File: ECAD/SolarConditioning.sch (KiCad schematic (older format))
At the start: 2 parts

Commit message: First version MPPT
Parts:
- added J?: S2A, symbol Connector:Conn_01x05_Female
- added J?: S2B, symbol Connector:Conn_01x05_Female
- added J?: S3A, symbol Connector:Conn_01x05_Female
- added J?: S3B, symbol Connector:Conn_01x05_Female
- added U?: ATtiny1604-SS, Package_SO:SOIC-14_3.9x8.7mm_P1.27mm, symbol MCU_Microchip_ATtiny:ATtiny1604-SS
Connections:
- wire segments 4 -> 12
Changed lines of the file:
@@
 $Descr A4 11693 8268
 encoding utf-8
-Sheet 5 6
+Sheet 5 8
 Title ""
 Date ""
@@
 $EndDescr
 $Sheet
-S 2700 1850 2000 950
+S 2600 1800 1050 550
 U 61BEC848
 F0 "MPPT1" 50
 F1 "MPPT.sch" 50
+F2 "VOUT" I R 3650 1850 50
+F3 "ARRAY_PWR" I L 2600 1850 50
+F4 "ARRAY_RTN" I L 2600 1950 50
+F5 "GATE" I L 2600 2050 50
+F6 "TELEM_VIN" I R 3650 1950 50
+F7 "TELEM_VOUT" I R 3650 2050 50
+F8 "TELEM_IIN" I R 3650 2150 50
+F9 "TELEM_IOUT" I R 3650 2250 50
 $EndSheet
 $Comp
@@
 Wire Wire Line
 	1700 1900 1700 2650
+$Comp
+L Connector:Conn_01x05_Female J?
+U 1 1 61BFAD9A
+P 1400 3700
+F 0 "J?" H 1292 4085 50  0000 C CNN
+F 1 "S2A" H 1292 3994 50  0000 C CNN
+F 2 "" H 1400 3700 50  0001 C CNN
+F 3 "~" H 1400 3700 50  0001 C CNN
+	1    1400 3700
+	-1   0    0    -1
+$EndComp
+$Comp
+L Connector:Conn_01x05_Female J?
+U 1 1 61BFADA0
+P 1400 4450
+F 0 "J?" H 1292 4835 50  0000 C CNN
+F 1 "S2B" H 1292 4744 50  0000 C CNN
+F 2 "" H 1400 4450 50  0001 C CNN
+F 3 "~" H 1400 4450 50  0001 C CNN
+	1    1400 4450
+	-1   0    0    -1
+$EndComp
+$Comp
+L power:GND #PWR?
+U 1 1 61BFADA6
+P 1700 4700
+F 0 "#PWR?" H 1700 4450 50  0001 C CNN
+F 1 "GND" H 1705 4527 50  0000 C CNN
+F 2 "" H 1700 4700 50  0001 C CNN
+F 3 "" H 1700 4700 50  0001 C CNN
+	1    1700 4700
+	1    0    0    -1
+$EndComp
+Wire Wire Line
+	1700 4700 1700 4550
+Wire Wire Line
+	1700 4550 1600 4550
+Connection ~ 1700 4550
+Wire Wire Line
+	1700 3800 1600 3800
+Wire Wire Line
+	1700 3800 1700 4550
+$Sheet
+S 2600 3750 1050 550
+U 61BFB023
+F0 "MPPT2" 50
+F1 "MPPT.sch" 50
+F2 "VOUT" I R 3650 3800 50
+F3 "ARRAY_PWR" I L 2600 3800 50
+F4 "ARRAY_RTN" I L 2600 3900 50
+F5 "GATE" I L 2600 4000 50
+F6 "TELEM_VIN" I R 3650 3900 50
+F7 "TELEM_VOUT" I R 3650 4000 50
+F8 "TELEM_IIN" I R 3650 4100 50
+F9 "TELEM_IOUT" I R 3650 4200 50
+$EndSheet
+$Comp
+L Connector:Conn_01x05_Female J?
+U 1 1 61BFC761
+P 1400 5500
+F 0 "J?" H 1292 5885 50  0000 C CNN
+F 1 "S3A" H 1292 5794 50  0000 C CNN
+F 2 "" H 1400 5500 50  0001 C CNN
+F 3 "~" H 1400 5500 50  0001 C CNN
+	1    1400 5500
+	-1   0    0    -1
+$EndComp
+$Comp
+L Connector:Conn_01x05_Female J?
+U 1 1 61BFC767
+P 1400 6250
+F 0 "J?" H 1292 6635 50  0000 C CNN
+F 1 "S3B" H 1292 6544 50  0000 C CNN
+F 2 "" H 1400 6250 50  0001 C CNN
+F 3 "~" H 1400 6250 50  0001 C CNN
+	1    1400 6250
+	-1   0    0    -1
+$EndComp
+$Comp
+L power:GND #PWR?
+U 1 1 61BFC76D
+P 1700 6500
+F 0 "#PWR?" H 1700 6250 50  0001 C CNN
+F 1 "GND" H 1705 6327 50  0000 C CNN
+F 2 "" H 1700 6500 50  0001 C CNN
+F 3 "" H 1700 6500 50  0001 C CNN
+	1    1700 6500
+	1    0    0    -1
+$EndComp
+Wire Wire Line
+	1700 6500 1700 6350
+Wire Wire Line
+	1700 6350 1600 6350
+Connection ~ 1700 6350
+Wire Wire Line
+	1700 5600 1600 5600
+Wire Wire Line
+	1700 5600 1700 6350
+$Sheet
+S 2600 5550 1050 550
+U 61BFCA72
+F0 "MPPT3" 50
+F1 "MPPT.sch" 50
+F2 "VOUT" I R 3650 5600 50
+F3 "ARRAY_PWR" I L 2600 5600 50
+F4 "ARRAY_RTN" I L 2600 5700 50
+F5 "GATE" I L 2600 5800 50
+F6 "TELEM_VIN" I R 3650 5700 50
+F7 "TELEM_VOUT" I R 3650 5800 50
+F8 "TELEM_IIN" I R 3650 5900 50
+F9 "TELEM_IOUT" I R 3650 6000 50
+$EndSheet
+$Comp
+L MCU_Microchip_ATtiny:ATtiny1604-SS U?
+U 1 1 61BFEAB5
+P 5100 3950
+F 0 "U?" H 5100 4831 50  0000 C CNN
+F 1 "ATtiny1604-SS" H 5100 4740 50  0000 C CNN
+F 2 "Package_SO:SOIC-14_3.9x8.7mm_P1.27mm" H 5100 3950 50  0001 C CIN
+F 3 "http://ww1.microchip.com/downloads/en/DeviceDoc/ATtiny804_1604-Data-Sheet-40002028A.pdf" H 5100 3950 50  0001 C CNN
+	1    5100 3950
+	1    0    0    -1
+$EndComp
 $EndSCHEMATC

Commit message: revamp solar conditioning, use lt3652 instead of homebrew buck converter
Parts:
- removed U?: ATtiny1604-SS, Package_SO:SOIC-14_3.9x8.7mm_P1.27mm, symbol MCU_Microchip_ATtiny:ATtiny1604-SS
- added C?: 0.47uF, symbol Device:C
- added C? (x3): 0.1uF, symbol Device:C
- added D? (x6): 1N4148, symbol Device:D
- added U? (x2): MCP4812, symbol Analog_DAC:MCP4812
- added U?: ATtiny85-20SU, Package_SO:SOIJ-8_5.3x5.3mm_P1.27mm, symbol MCU_Microchip_ATtiny:ATtiny85-20SU
- added U?: L78L33_SO8, Package_SO:SOIC-8_3.9x4.9mm_P1.27mm, symbol Regulator_Linear:L78L33_SO8
Connections:
- net labels added: +3.3VA, BCR_OUT, Vset1, Vset2, Vset3
- wire segments 12 -> 106
Other:
- note added: "MPPT Setpoint Controller"
- moved on the sheet: J?

Commit message: Spec out switching controllers for PCMs
Parts:
- added D?: 3v3 Zener, symbol Device:D_Zener
- added Q?: IRF7425, Package_SO:SOIC-8_3.9x4.9mm_P1.27mm, symbol Transistor_FET:IRF7404
- added R?: 220K, symbol Device:R
- added R?: 100K, symbol Device:R
- added R?: 10K, symbol Device:R
- added R?: 100R, symbol Device:R
- added SW?: INHIBIT 1, symbol Switch:SW_SPST
Connections:
- net BCR_OUT: now also Q?.1 (S), Q?.2 (S), Q?.3 (S)
- net GND: now also D?.2 (A), R?.2, SW?.1 (A)
- new net: Q?.4 (G), R?.1, R?.2
- new net: R?.2, SW?.2 (B)
- new net MPPT1/VOUT: Q?.5 (D), Q?.6 (D), Q?.7 (D), Q?.8 (D), R?.1, R?.1
- new net TELEM_VOUT: D?.1 (K), R?.1, R?.2
Changed lines of the file:
@@
 $Descr A4 11693 8268
 encoding utf-8
-Sheet 11 14
+Sheet 11 15
 Title ""
 Date ""
@@
 F0 "MPPT1" 50
 F1 "MPPT.sch" 50
-F2 "TELEM_VOUT" I R 2450 1300 50
-F3 "A_PWR" I L 1500 1200 50
-F4 "Vset" I L 1500 1400 50
-F5 "TELEM_I_A" I R 2450 1400 50
-F6 "TELEM_VIN" I R 2450 1200 50
-F7 "B_PWR" I L 1500 1300 50
-F8 "TELEM_I_B" I R 2450 1500 50
-F9 "VOUT" I R 2450 1600 50
+F2 "A_PWR" I L 1500 1200 50
+F3 "Vset" I L 1500 1400 50
+F4 "TELEM_I_A" I R 2450 1300 50
+F5 "TELEM_VIN" I R 2450 1200 50
+F6 "B_PWR" I L 1500 1300 50
+F7 "TELEM_I_B" I R 2450 1400 50
+F8 "VOUT" I R 2450 1500 50
 $EndSheet
 $Comp
@@
 F0 "MPPT2" 50
 F1 "MPPT.sch" 50
-F2 "TELEM_VOUT" I R 2450 2900 50
-F3 "A_PWR" I L 1500 2800 50
-F4 "Vset" I L 1500 3000 50
-F5 "TELEM_I_A" I R 2450 3000 50
-F6 "TELEM_VIN" I R 2450 2800 50
-F7 "B_PWR" I L 1500 2900 50
-F8 "TELEM_I_B" I R 2450 3100 50
-F9 "VOUT" I R 2450 3200 50
+F2 "A_PWR" I L 1500 2800 50
+F3 "Vset" I L 1500 3000 50
+F4 "TELEM_I_A" I R 2450 2900 50
+F5 "TELEM_VIN" I R 2450 2800 50
+F6 "B_PWR" I L 1500 2900 50
+F7 "TELEM_I_B" I R 2450 3000 50
+F8 "VOUT" I R 2450 3100 50
 $EndSheet
 $Sheet
@@
 F0 "MPPT3" 50
 F1 "MPPT.sch" 50
-F2 "TELEM_VOUT" I R 2450 4500 50
-F3 "A_PWR" I L 1500 4400 50
-F4 "Vset" I L 1500 4600 50
-F5 "TELEM_I_A" I R 2450 4600 50
-F6 "TELEM_VIN" I R 2450 4400 50
-F7 "B_PWR" I L 1500 4500 50
-F8 "TELEM_I_B" I R 2450 4700 50
-F9 "VOUT" I R 2450 4800 50
+F2 "A_PWR" I L 1500 4400 50
+F3 "Vset" I L 1500 4600 50
+F4 "TELEM_I_A" I R 2450 4500 50
+F5 "TELEM_VIN" I R 2450 4400 50
+F6 "B_PWR" I L 1500 4500 50
+F7 "TELEM_I_B" I R 2450 4600 50
+F8 "VOUT" I R 2450 4700 50
 $EndSheet
 Wire Wire Line
@@
 $EndComp
 Wire Wire Line
-	2450 1600 2650 1600
-Wire Wire Line
-	2650 1600 2650 3200
-Wire Wire Line
-	2650 3200 2450 3200
-Wire Wire Line
-	2650 3200 2650 4800
-Wire Wire Line
-	2650 4800 2450 4800
-Connection ~ 2650 3200
-Wire Wire Line
-	2650 3200 3000 3200
-Text GLabel 3000 3200 2    50   Input ~ 0
+	2450 1500 2650 1500
+Wire Wire Line
+	2650 1500 2650 3100
+Wire Wire Line
+	2650 3100 2450 3100
+Wire Wire Line
+	2650 3100 2650 4700
+Wire Wire Line
+	2650 4700 2450 4700
+Connection ~ 2650 3100
+Wire Wire Line
+	2650 3100 2900 3100
+Text GLabel 4450 3100 2    50   Input ~ 0
 BCR_OUT
+$Comp
+L Device:R R?
+U 1 1 61C37B40
+P 2900 3250
+AR Path="/61BEC565/61BEC848/61C37B40" Ref="R?"  Part="1"
+AR Path="/61BEC565/61BFB023/61C37B40" Ref="R?"  Part="1"
+AR Path="/61BEC565/61BFCA72/61C37B40" Ref="R?"  Part="1"
+AR Path="/61BEC565/61E10014/61C37B40" Ref="R?"  Part="1"
+AR Path="/61BEC565/61E1083C/61C37B40" Ref="R?"  Part="1"
+AR Path="/61BEC565/61C37B40" Ref="R?"  Part="1"
+F 0 "R?" H 2950 3250 50  0000 L CNN
+F 1 "220K" V 2900 3150 50  0000 L CNN
+F 2 "" V 2830 3250 50  0001 C CNN
+F 3 "~" H 2900 3250 50  0001 C CNN
+	1    2900 3250
+	1    0    0    -1
+$EndComp
+$Comp
+L Device:R R?
+U 1 1 61C37B46
+P 2900 3650
+AR Path="/61BEC565/61BEC848/61C37B46" Ref="R?"  Part="1"
+AR Path="/61BEC565/61BFB023/61C37B46" Ref="R?"  Part="1"
+AR Path="/61BEC565/61BFCA72/61C37B46" Ref="R?"  Part="1"
+AR Path="/61BEC565/61E10014/61C37B46" Ref="R?"  Part="1"
+AR Path="/61BEC565/61E1083C/61C37B46" Ref="R?"  Part="1"
+AR Path="/61BEC565/61C37B46" Ref="R?"  Part="1"
+F 0 "R?" H 2950 3650 50  0000 L CNN
+F 1 "100K" V 2900 3550 50  0000 L CNN
+F 2 "" V 2830 3650 50  0001 C CNN
+F 3 "~" H 2900 3650 50  0001 C CNN
+	1    2900 3650
+	1    0    0    -1
+$EndComp
+Wire Wire Line
+	2900 3500 2900 3450
+Wire Wire Line
+	3150 3500 3150 3450
+Wire Wire Line
+	3150 3450 2900 3450
+Connection ~ 2900 3450
+Wire Wire Line
+	2900 3450 2900 3400
+$Comp
+L Device:D_Zener D?
+U 1 1 61C37B51
+P 3150 3650
+AR Path="/61BEC565/61BEC848/61C37B51" Ref="D?"  Part="1"
+AR Path="/61BEC565/61BFB023/61C37B51" Ref="D?"  Part="1"
+AR Path="/61BEC565/61BFCA72/61C37B51" Ref="D?"  Part="1"
+AR Path="/61BEC565/61E10014/61C37B51" Ref="D?"  Part="1"
+AR Path="/61BEC565/61E1083C/61C37B51" Ref="D?"  Part="1"
+AR Path="/61BEC565/61C37B51" Ref="D?"  Part="1"
+F 0 "D?" V 3104 3730 50  0000 L CNN
+F 1 "3v3 Zener" V 3195 3730 50  0000 L CNN
+F 2 "" H 3150 3650 50  0001 C CNN
+F 3 "~" H 3150 3650 50  0001 C CNN
+	1    3150 3650
+	0    1    1    0
+$EndComp
+Text HLabel 3150 3450 2    50   Input ~ 0
+TELEM_VOUT
+Connection ~ 2900 3100
+Wire Wire Line
+	3150 3800 2900 3800
+$Comp
+L power:GND #PWR?
+U 1 1 61C41272
+P 2900 3800
+F 0 "#PWR?" H 2900 3550 50  0001 C CNN
+F 1 "GND" H 2905 3627 50  0000 C CNN
+F 2 "" H 2900 3800 50  0001 C CNN
+F 3 "" H 2900 3800 50  0001 C CNN
+	1    2900 3800
+	1    0    0    -1
+$EndComp
+Connection ~ 2900 3800
+$Comp
+L Transistor_FET:IRF7404 Q?
+U 1 1 61C4B7C5
+P 4100 3200
+F 0 "Q?" V 4442 3200 50  0000 C CNN
+F 1 "IRF7425" V 4351 3200 50  0000 C CNN
+F 2 "Package_SO:SOIC-8_3.9x4.9mm_P1.27mm" H 4300 3125 50  0001 L CIN
+F 3 "http://www.infineon.com/dgdl/irf7404.pdf?fileId=5546d462533600a4015355fa2b5b1b9e" V 4100 3200 50  0001 L CNN
+	1    4100 3200
+	0    -1   -1   0
+$EndComp
+$Comp
+L Device:R R?
+U 1 1 61C55D97
+P 3750 3250
+F 0 "R?" H 3800 3250 50  0000 L CNN
+F 1 "10K" V 3750 3250 50  0000 C CNN
+F 2 "" V 3680 3250 50  0001 C CNN
+F 3 "~" H 3750 3250 50  0001 C CNN
+	1    3750 3250
+	1    0    0    -1
+$EndComp
+Wire Wire Line
+	3900 3100 3750 3100
+Wire Wire Line
+	2900 3100 3750 3100
+Connection ~ 3750 3100
+Wire Wire Line
+	3750 3400 4100 3400
+Wire Wire Line
+	4300 3100 4450 3100
+$Comp
+L Switch:SW_SPST SW?
+U 1 1 61C66266
+P 3850 3800
+F 0 "SW?" H 3850 4035 50  0000 C CNN
+F 1 "INHIBIT 1" H 3850 3944 50  0000 C CNN
+F 2 "" H 3850 3800 50  0001 C CNN
+F 3 "~" H 3850 3800 50  0001 C CNN
+	1    3850 3800
+	1    0    0    -1
+$EndComp
+$Comp
+L Device:R R?
+U 1 1 61C70AB7
+P 4100 3550
+F 0 "R?" H 4150 3550 50  0000 L CNN
+F 1 "100R" V 4100 3450 50  0000 L CNN
+F 2 "" V 4030 3550 50  0001 C CNN
+F 3 "~" H 4100 3550 50  0001 C CNN
+	1    4100 3550
+	1    0    0    -1
+$EndComp
+Connection ~ 4100 3400
+Wire Wire Line
+	3650 3800 3150 3800
+Connection ~ 3150 3800
+Wire Wire Line
+	4050 3800 4100 3800
+Wire Wire Line
+	4100 3800 4100 3700
 $EndSCHEMATC

Commit message: Finish components for buck converters, add UVLO feature, correct all mosfet orientations
Parts:
- added D? (x6): CMSH3-40MA, symbol Device:D_Schottky
Connections:
- net BCR_OUT: now also Q?.5 (D), Q?.6 (D), Q?.7 (D), Q?.8 (D); no longer Q?.1 (S), Q?.2 (S), Q?.3 (S)
- net MPPT1/A_PWR: now also D?.1 (K); no longer J?.1 (Pin_1)
- net MPPT1/B_PWR: now also D?.1 (K); no longer J?.1 (Pin_1)
- net MPPT1/VOUT: now also Q?.1 (S), Q?.2 (S), Q?.3 (S); no longer Q?.5 (D), Q?.6 (D), Q?.7 (D), Q?.8 (D)
- net MPPT2/A_PWR: now also D?.1 (K); no longer J?.1 (Pin_1)
- net MPPT2/B_PWR: now also D?.1 (K); no longer J?.1 (Pin_1)
- net MPPT3/A_PWR: now also D?.1 (K); no longer J?.1 (Pin_1)
- net MPPT3/B_PWR: now also D?.1 (K); no longer J?.1 (Pin_1)
- net TELEM_VOUT renamed TELEM_VBCROUT
- new net: D?.2 (A), J?.1 (Pin_1) (x6)
Other:
- moved on the sheet: C?, D?, Q?, R?, SW?, U?

Commit message: Finish speccing out components for 12V boost
Parts:
- added U?: ATtiny84A-SSU, Package_SO:SOIC-14_3.9x8.7mm_P1.27mm, symbol MCU_Microchip_ATtiny:ATtiny84A-SSU
- added U?: MCP3208, symbol Analog_ADC:MCP3208
Connections:
- new net MISO: U?.8 (PA5)
- new net MOSI: U?.7 (PA6)
- new net SCK: U?.9 (PA4)

Commit message: Remove zeners, add PDMs, correct MPPT setpoint controller
Parts:
- removed D?: 3v3 Zener, symbol Device:D_Zener
- removed U?: ATtiny85-20SU, Package_SO:SOIJ-8_5.3x5.3mm_P1.27mm, symbol MCU_Microchip_ATtiny:ATtiny85-20SU
- added C? (x2): 0.1uF, symbol Device:C
Connections:
- net +3.3VA: now also U?.1 (VCC), U?.15 (Vref), U?.16 (Vdd), C?.1, C?.1
- net GND: now also U?.14 (AGND), U?.14 (GND), U?.9 (DGND), C?.2, C?.2
- net MISO: now also U?.12 (Dout)
- net MOSI: now also U?.11 (Din), U?.4 (SDI), U?.4 (SDI)
- net SCK: now also U?.13 (CLK), U?.3 (SCK), U?.3 (SCK)
- net DAC2CS: now reaches U?.2 (~CS)
- net DAC2CS: now also U?.5 (PB2)
- net DAC1CS: now reaches U?.2 (~CS)
- net DAC1CS: now also U?.3 (XTAL2/PB1)
- net V_SA3: now reaches U?.11 (PA2)
- net V_SA2: now reaches U?.12 (PA1)
- net V_SA1: now reaches U?.13 (AREF/PA0)
- net ADCCS: now reaches U?.2 (XTAL1/PB0)
- net ADCCS: now also U?.10 (~CS~/SHDN)
- net I_SA1A: now reaches U?.1 (CH0)
- net I_SA1B: now reaches U?.2 (CH1)
- net I_SA2A: now reaches U?.3 (CH2)
- net I_SA2B: now reaches U?.4 (CH3)
- net I_SA3A: now reaches U?.5 (CH4)
- net I_SA3B: now reaches U?.6 (CH5)
- net PANEL_OR: now reaches C?.1, D?.1 (K), D?.1 (K), D?.1 (K), D?.1 (K), D?.1 (K), D?.1 (K), U?.8 (IN)
Other:
- moved on the sheet: C?, U?
