File: ECAD/SolarConditioning.sch (KiCad schematic (older format))
At the start: 52 parts, among them J10 S3B, J11 S4A, J12 S4B, J13 TELEM_IN, J5 S1A, J6 S1B, J7 S2A, J8 S2B, J9 S3A, Q33 IRF7425, Q34 IRF7458, SW3 INHIBIT 1, U15 LTC4412xS6, U16 MCP3208, U17 LT6106, U18 ATtiny84A-SSU, U19 L78L33_SO8, U20 MCP4812, U21 MCP4812

Commit message: add some more footprints
Parts:
- D10, D11, D12, D13, D14, D15, D16, D17, D2, D3, D4, D5, D6, D7, D8, D9: footprint (none) -> Diode_SMD:D_SMA
Changed lines of the file:
@@
 F 0 "D7" H 1200 4100 50  0000 C CNN
 F 1 "CMSH3-40MA" H 1200 4200 50  0000 C CNN
-F 2 "" H 1200 4300 50  0001 C CNN
+F 2 "Diode_SMD:D_SMA" H 1200 4300 50  0001 C CNN
 F 3 "~" H 1200 4300 50  0001 C CNN
 	1    1200 4300
@@
 F 0 "D6" H 1200 3817 50  0000 C CNN
 F 1 "CMSH3-40MA" H 1200 3726 50  0000 C CNN
-F 2 "" H 1200 3600 50  0001 C CNN
+F 2 "Diode_SMD:D_SMA" H 1200 3600 50  0001 C CNN
 F 3 "~" H 1200 3600 50  0001 C CNN
 	1    1200 3600
@@
 F 0 "D15" V 1800 4200 50  0000 L CNN
 F 1 "1N4004" V 1700 4200 50  0000 L CNN
-F 2 "" H 1750 4150 50  0001 C CNN
+F 2 "Diode_SMD:D_SMA" H 1750 4150 50  0001 C CNN
 F 3 "~" H 1750 4150 50  0001 C CNN
 	1    1750 4150
@@
 F 0 "D14" V 1800 3700 50  0000 R CNN
 F 1 "1N4004" V 1700 3700 50  0000 R CNN
-F 2 "" H 1750 3750 50  0001 C CNN
+F 2 "Diode_SMD:D_SMA" H 1750 3750 50  0001 C CNN
 F 3 "~" H 1750 3750 50  0001 C CNN
 	1    1750 3750
@@
 F 0 "D5" H 1200 2650 50  0000 C CNN
 F 1 "CMSH3-40MA" H 1200 2750 50  0000 C CNN
-F 2 "" H 1200 2850 50  0001 C CNN
+F 2 "Diode_SMD:D_SMA" H 1200 2850 50  0001 C CNN
 F 3 "~" H 1200 2850 50  0001 C CNN
 	1    1200 2850
@@
 F 0 "D3" H 1200 1200 50  0000 C CNN
 F 1 "CMSH3-40MA" H 1200 1300 50  0000 C CNN
-F 2 "" H 1200 1400 50  0001 C CNN
+F 2 "Diode_SMD:D_SMA" H 1200 1400 50  0001 C CNN
 F 3 "~" H 1200 1400 50  0001 C CNN
 	1    1200 1400
@@
 F 0 "D2" H 1200 917 50  0000 C CNN
 F 1 "CMSH3-40MA" H 1200 826 50  0000 C CNN
-F 2 "" H 1200 700 50  0001 C CNN
+F 2 "Diode_SMD:D_SMA" H 1200 700 50  0001 C CNN
 F 3 "~" H 1200 700 50  0001 C CNN
 	1    1200 700
@@
 F 0 "D13" V 1800 2750 50  0000 L CNN
 F 1 "1N4004" V 1700 2750 50  0000 L CNN
-F 2 "" H 1750 2700 50  0001 C CNN
+F 2 "Diode_SMD:D_SMA" H 1750 2700 50  0001 C CNN
 F 3 "~" H 1750 2700 50  0001 C CNN
 	1    1750 2700
@@
 F 0 "D12" V 1800 2250 50  0000 R CNN
 F 1 "1N4004" V 1700 2250 50  0000 R CNN
-F 2 "" H 1750 2300 50  0001 C CNN
+F 2 "Diode_SMD:D_SMA" H 1750 2300 50  0001 C CNN
 F 3 "~" H 1750 2300 50  0001 C CNN
 	1    1750 2300
@@
 F 0 "D11" V 1800 1300 50  0000 L CNN
 F 1 "1N4004" V 1700 1300 50  0000 L CNN
-F 2 "" H 1750 1250 50  0001 C CNN
+F 2 "Diode_SMD:D_SMA" H 1750 1250 50  0001 C CNN
 F 3 "~" H 1750 1250 50  0001 C CNN
 	1    1750 1250
@@
 F 0 "D10" V 1800 800 50  0000 R CNN
 F 1 "1N4004" V 1700 800 50  0000 R CNN
-F 2 "" H 1750 850 50  0001 C CNN
+F 2 "Diode_SMD:D_SMA" H 1750 850 50  0001 C CNN
 F 3 "~" H 1750 850 50  0001 C CNN
 	1    1750 850
@@
 F 0 "D4" H 1200 2367 50  0000 C CNN
 F 1 "CMSH3-40MA" H 1200 2276 50  0000 C CNN
-F 2 "" H 1200 2150 50  0001 C CNN
+F 2 "Diode_SMD:D_SMA" H 1200 2150 50  0001 C CNN
 F 3 "~" H 1200 2150 50  0001 C CNN
 	1    1200 2150
@@
 F 0 "D9" H 1200 5550 50  0000 C CNN
 F 1 "CMSH3-40MA" H 1200 5650 50  0000 C CNN
-F 2 "" H 1200 5750 50  0001 C CNN
+F 2 "Diode_SMD:D_SMA" H 1200 5750 50  0001 C CNN
 F 3 "~" H 1200 5750 50  0001 C CNN
 	1    1200 5750
@@
 F 0 "D8" H 1200 5267 50  0000 C CNN
 F 1 "CMSH3-40MA" H 1200 5176 50  0000 C CNN
-F 2 "" H 1200 5050 50  0001 C CNN
+F 2 "Diode_SMD:D_SMA" H 1200 5050 50  0001 C CNN
 F 3 "~" H 1200 5050 50  0001 C CNN
 	1    1200 5050
@@
 F 0 "D17" V 1800 5650 50  0000 L CNN
 F 1 "1N4004" V 1700 5650 50  0000 L CNN
-F 2 "" H 1750 5600 50  0001 C CNN
+F 2 "Diode_SMD:D_SMA" H 1750 5600 50  0001 C CNN
 F 3 "~" H 1750 5600 50  0001 C CNN
 	1    1750 5600
@@
 F 0 "D16" V 1800 5150 50  0000 R CNN
 F 1 "1N4004" V 1700 5150 50  0000 R CNN
-F 2 "" H 1750 5200 50  0001 C CNN
+F 2 "Diode_SMD:D_SMA" H 1750 5200 50  0001 C CNN
 F 3 "~" H 1750 5200 50  0001 C CNN
 	1    1750 5200

Commit message: Add all IC footprints
Parts:
- U16: footprint (none) -> Package_SO:SO-16_3.9x9.9mm_P1.27mm
- U20, U21: footprint (none) -> Package_SO:MSOP-8_3x3mm_P0.65mm
Changed lines of the file:
@@
 F 0 "U21" H 9250 5000 50  0000 C CNN
 F 1 "MCP4812" H 9350 4900 50  0000 C CNN
-F 2 "" H 9950 4250 50  0001 C CNN
+F 2 "Package_SO:MSOP-8_3x3mm_P0.65mm" H 9950 4250 50  0001 C CNN
 F 3 "http://ww1.microchip.com/downloads/en/DeviceDoc/20002249B.pdf" H 9950 4250 50  0001 C CNN
 	1    9150 4550
@@
 F 0 "U20" H 9250 3800 50  0000 C CNN
 F 1 "MCP4812" H 9350 3700 50  0000 C CNN
-F 2 "" H 9950 3050 50  0001 C CNN
+F 2 "Package_SO:MSOP-8_3x3mm_P0.65mm" H 9950 3050 50  0001 C CNN
 F 3 "http://ww1.microchip.com/downloads/en/DeviceDoc/20002249B.pdf" H 9950 3050 50  0001 C CNN
 	1    9150 3350
@@
 F 0 "U16" H 4900 4931 50  0000 C CNN
 F 1 "MCP3208" H 4900 4840 50  0000 C CNN
-F 2 "" H 5000 4350 50  0001 C CNN
+F 2 "Package_SO:SO-16_3.9x9.9mm_P1.27mm" H 5000 4350 50  0001 C CNN
 F 3 "http://ww1.microchip.com/downloads/en/DeviceDoc/21298c.pdf" H 5000 4350 50  0001 C CNN
 	1    4900 4250

Commit message: add a bunch of cap and shunt resistor footprints
Parts:
- J13: footprint (none) -> Connector_PinHeader_1.27mm:PinHeader_1x07_P1.27mm_Vertical
- R78: footprint (none) -> Resistor_SMD:R_2010_5025Metric
Changed lines of the file:
@@
 F 0 "R78" V 6000 1450 50  0000 C CNN
 F 1 "10m" V 6100 1450 50  0000 C CNN
-F 2 "" V 6030 1450 50  0001 C CNN
+F 2 "Resistor_SMD:R_2010_5025Metric" V 6030 1450 50  0001 C CNN
 F 3 "~" H 6100 1450 50  0001 C CNN
 	1    6100 1450
@@
 F 0 "J13" H 8658 1931 50  0000 C CNN
 F 1 "TELEM_IN" H 8658 1840 50  0000 C CNN
-F 2 "" H 8550 1450 50  0001 C CNN
+F 2 "Connector_PinHeader_1.27mm:PinHeader_1x07_P1.27mm_Vertical" H 8550 1450 50  0001 C CNN
 F 3 "~" H 8550 1450 50  0001 C CNN
 	1    8550 1450
