File: ECAD/BatteryMaster.sch (KiCad schematic (older format))
At the start: 33 parts

Commit message: rearrange the stack headers to make some damn sense *looks at clydespace*
Parts:
- removed H?: Stack Header 2, symbol Connector_Generic:Conn_02x26_Odd_Even
- removed H?: Stack Header 1, symbol Connector_Generic:Conn_02x26_Odd_Even
- added H?: Stack Header 2, symbol Connector_Generic:Conn_02x26_Odd_Even
- added H?: Stack Header 1, symbol Connector_Generic:Conn_02x26_Odd_Even
Connections:
- net +12V: now also H?.23 (Pin_23), H?.24 (Pin_24)
- net +3V3: now also H?.29 (Pin_29), H?.30 (Pin_30)
- net +5V: now also H?.27 (Pin_27), H?.28 (Pin_28)
- net +BATT: now also H?.25 (Pin_25), H?.26 (Pin_26)
- net BCR_OUT: now also H?.41 (Pin_41), H?.42 (Pin_42), H?.43 (Pin_43), H?.44 (Pin_44)
- net GND: now also H?.21 (Pin_21), H?.22 (Pin_22), H?.31 (Pin_31), H?.32 (Pin_32), H?.45 (Pin_45), H?.46 (Pin_46), H?.5 (Pin_5), H?.6 (Pin_6)
- net PCM_IN: now also H?.35 (Pin_35), H?.36 (Pin_36)
- net SCL: now also H?.43 (Pin_43)
- net SDA: now also H?.41 (Pin_41)
- net SW1: now also H?.7 (Pin_7)
- net SW10: now also H?.15 (Pin_15)
- net SW2: now also H?.8 (Pin_8)
- net SW3: now also H?.9 (Pin_9)
- net SW4: now also H?.10 (Pin_10)
- net SW5: now also H?.12 (Pin_12)
- net SW6: now also H?.11 (Pin_11)
- net SW7: now also H?.14 (Pin_14)
- net SW8: now also H?.13 (Pin_13)
- net SW9: now also H?.16 (Pin_16)
- net VUSB: now also H?.32 (Pin_32)
- new net SW11: H?.18 (Pin_18)
- new net SW12: H?.17 (Pin_17)
- new net SW13: H?.20 (Pin_20)
- new net SW14: H?.19 (Pin_19)
- no-connect marks 18 -> 16

Commit message: spec out new cell protection IC and mosfets, figured out current limit calculation
Parts:
- removed R?: 15R, symbol Device:R
- added F?: 6A, symbol Device:Polyfuse
- added Q?: Si4186DY, Package_SO:SOIC-8_3.9x4.9mm_P1.27mm, symbol Transistor_FET:Si4162DY
- added R?: 100K, symbol Device:R
- added R?: 790K, symbol Device:R
- added R?: 50K, symbol Device:R
- added U?: LTC4365TS8-1, symbol Power_Management:LTC4365TS8-1
Connections:
- net +BATT: now also F?.1; no longer Q?.5 (D), Q?.6 (D), Q?.7 (D), Q?.8 (D)
- net -BATT: now also Q?.1 (S), Q?.2 (S), Q?.3 (S), Q?.5 (D), Q?.6 (D), Q?.7 (D), Q?.8 (D), R?.2, U?.4 (GND); no longer F?.1
- net at Q?.5 (D), Q?.6 (D), Q?.7 (D)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: now also F?.2, F?.1
- net at Q?.1 (S), Q?.2 (S), Q?.3 (S)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: now also R?.1, U?.3 (-); no longer U?.2 (-)
- new net: F?.2, Q?.1 (S), Q?.2 (S), Q?.3 (S), U?.7 (Vout)
- new net: Q?.5 (D), Q?.5 (D), Q?.6 (D), Q?.6 (D), Q?.7 (D), Q?.7 (D), Q?.8 (D), Q?.8 (D), R?.1, R?.1, U?.1 (Vin)
- new net: R?.2, U?.2 (UV), U?.5 (~SHDN)
- new net: R?.1, R?.2, U?.3 (OV)
- new net: Q?.4 (G), U?.8 (GATE)
Other:
- note added: "OUT is pulled high in OV condition, after 3 second delay\nOV is fixed at 4.3V per cell"
- note added: "Semidestructive protection in case \nOVP exists for more than 3 seconds"
- note removed: "Low resistance, high power\nShunt resistor, as OVP\nExternally connected"
- note removed: "OUT is pulled high in OV condition\nOV is fixed at 4.3V per cell"
- moved on the sheet: C?, F?, Q?, R?, SW?, U?, U?A, U?B, U?C

Commit message: Add OCP, resize some sheets
Parts:
- added D?: 1.2V zener, symbol Device:D_Zener
- added Q?: IRF7425, Package_SO:SOIC-8_3.9x4.9mm_P1.27mm, symbol Transistor_FET:IRF7404
- added R?: 100K, symbol Device:R
- F? (x2): value 6A -> 7A
Connections:
- net -BATT: now also D?.2 (A)
- net TELEM_IBAT: now also U?.5 (+)
- net TELEM_VBAT: now also R?.1, R?.2; no longer U?.6 (-), U?.7
- net at Q?.5 (D), Q?.6 (D), Q?.7 (D)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: now also Q?.5 (D), Q?.6 (D), Q?.7 (D), Q?.8 (D); no longer Q?.5 (D), Q?.6 (D), Q?.7 (D), Q?.8 (D)
- new net: Q?.1 (S), Q?.2 (S), Q?.3 (S), Q?.5 (D), Q?.6 (D), Q?.7 (D), Q?.8 (D), R?.1
- new net: D?.1 (K), R?.2, U?.6 (-)
- new net: Q?.4 (G), U?.7
Other:
- note added: "~~6A Bidirectional OCP"
- moved on the sheet: C?, F?, Q?, R?, SW?, U?, U?A, U?B, U?C

Commit message: fix the bidirectional ocp to actually be bidirectional
Parts:
- added Q?: IRF7425, Package_SO:SOIC-8_3.9x4.9mm_P1.27mm, symbol Transistor_FET:IRF7404
Connections:
- net at Q?.5 (D), Q?.6 (D), Q?.7 (D)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: now also Q?.1 (S), Q?.2 (S), Q?.3 (S); no longer Q?.5 (D), Q?.6 (D), Q?.7 (D), Q?.8 (D)
- net at Q?.4 (G), U?.7: now also Q?.4 (G)
- new net: Q?.5 (D), Q?.5 (D), Q?.6 (D), Q?.6 (D), Q?.7 (D), Q?.7 (D), Q?.8 (D), Q?.8 (D)
Other:
- moved on the sheet: Q?, U?B
Changed lines of the file:
@@
 L Amplifier_Operational:LM358 U?
 U 2 1 61DFA6F3
-P 5300 1300
-F 0 "U?" H 5300 1667 50  0000 C CNN
-F 1 "LM358" H 5300 1576 50  0000 C CNN
-F 2 "" H 5300 1300 50  0001 C CNN
-F 3 "http://www.ti.com/lit/ds/symlink/lm2904-n.pdf" H 5300 1300 50  0001 C CNN
-	2    5300 1300
+P 5200 1300
+F 0 "U?" H 5200 1667 50  0000 C CNN
+F 1 "LM358" H 5200 1576 50  0000 C CNN
+F 2 "" H 5200 1300 50  0001 C CNN
+F 3 "http://www.ti.com/lit/ds/symlink/lm2904-n.pdf" H 5200 1300 50  0001 C CNN
+	2    5200 1300
 	1    0    0    -1
 $EndComp
@@
 	4400 1100 4400 800
 Connection ~ 4400 1400
-Text Label 4600 1200 0    50   ~ 0
+Text Label 4500 1200 0    50   ~ 0
 TELEM_IBAT
 Wire Wire Line
-	4600 1200 5000 1200
-Wire Wire Line
-	4400 800  5400 800
+	4500 1200 4900 1200
+Wire Wire Line
+	4400 800  5300 800
 Wire Wire Line
 	6850 1100 6850 1200
@@
 L Transistor_FET:IRF7404 Q?
 U 1 1 622A211E
-P 5600 900
-F 0 "Q?" V 5942 900 50  0000 C CNN
-F 1 "IRF7425" V 5851 900 50  0000 C CNN
-F 2 "Package_SO:SOIC-8_3.9x4.9mm_P1.27mm" H 5800 825 50  0001 L CIN
-F 3 "http://www.infineon.com/dgdl/irf7404.pdf?fileId=5546d462533600a4015355fa2b5b1b9e" V 5600 900 50  0001 L CNN
-	1    5600 900
+P 5500 900
+F 0 "Q?" V 5842 900 50  0000 C CNN
+F 1 "IRF7425" V 5751 900 50  0000 C CNN
+F 2 "Package_SO:SOIC-8_3.9x4.9mm_P1.27mm" H 5700 825 50  0001 L CIN
+F 3 "http://www.infineon.com/dgdl/irf7404.pdf?fileId=5546d462533600a4015355fa2b5b1b9e" V 5500 900 50  0001 L CNN
+	1    5500 900
 	0    1    -1   0
 $EndComp
-Wire Wire Line
-	4400 1400 5000 1400
 Connection ~ 4400 800
 Wire Wire Line
-	5600 1300 5600 1100
-Wire Wire Line
-	5800 800  6150 800
-Connection ~ 6150 800
+	5500 1300 5500 1100
 Wire Wire Line
 	4400 2250 6150 2250
@@
 Wire Notes Line
 	500  500  3150 500
+$Comp
+L Transistor_FET:IRF7404 Q?
+U 1 1 61CCE42A
+P 5900 900
+F 0 "Q?" V 6242 900 50  0000 C CNN
+F 1 "IRF7425" V 6151 900 50  0000 C CNN
+F 2 "Package_SO:SOIC-8_3.9x4.9mm_P1.27mm" H 6100 825 50  0001 L CIN
+F 3 "http://www.infineon.com/dgdl/irf7404.pdf?fileId=5546d462533600a4015355fa2b5b1b9e" V 5900 900 50  0001 L CNN
+	1    5900 900
+	0    -1   -1   0
+$EndComp
+Wire Wire Line
+	4400 1400 4900 1400
+Wire Wire Line
+	5900 1100 5900 1300
+Wire Wire Line
+	5900 1300 5500 1300
+Connection ~ 5500 1300
+Wire Wire Line
+	6150 800  6100 800
+Connection ~ 6150 800
 $EndSCHEMATC

Commit message: start placing battery telemetry node
Parts:
- added C?: 0.1uF, symbol Device:C
- added R?: 22K, symbol Device:R
- added R?: 10K, symbol Device:R
- R?: value 87K -> 22K
- R?: value 100K -> 10K
Connections:
- net +3V3: now also U?.1 (VBAT), U?.24 (VDD), U?.36 (VDD), U?.48 (VDD), U?.9 (VDDA)
- net GND: now also U?.23 (VSS), U?.35 (VSS), U?.47 (VSS), U?.8 (VSSA), C?.2, R?.2
- net TELEM_IBAT: now also U?.15 (PA5)
- net TELEM_IBATDIR: now also R?.1
- net TELEM_VBAT: now also U?.14 (PA4), C?.1
- net SCK: now reaches H?.29 (Pin_29)
- net SCK: now also U?.39 (PB3)
- net MISO: now reaches H?.31 (Pin_31)
- net MISO: now also U?.40 (PB4)
- net MOSI: now reaches H?.33 (Pin_33)
- net MOSI: now also U?.41 (PB5)
- net SS: now reaches H?.35 (Pin_35)
- net SS: now also U?.38 (PA15)
- net TBAT1: now reaches U?.10 (PA0)
- net TBAT2: now reaches U?.11 (PA1)
- net TBAT3: now reaches U?.12 (PA2)
- net TBAT4: now reaches U?.13 (PA3)
- net at U?.16 (PA6): now also R?.1, R?.2
- net H2TOP: now reaches U?.21 (PB10)
- net H2BOT: now reaches U?.22 (PB11)
- net H3TOP: now reaches U?.25 (PB12)
- net H3BOT: now reaches U?.26 (PB13)
- net H4TOP: now reaches U?.27 (PB14)
- net H4BOT: now reaches U?.28 (PB15)
- net H1TOP: now reaches U?.45 (PB8)
- net H1BOT: now reaches U?.46 (PB9)
Other:
- moved on the sheet: C?, D?, F?, Q?, R?, SW?, U?, U?A, U?B, U?C

Commit message: bidirectional inhibits, remove unrealistic zener, replace all irf7425 with irf7458
Parts:
- removed R? (x2): 10K, symbol Device:R
- added C? (x2): 0.1uF, symbol Device:C
- added Q?: IRF7458, Package_SO:SOIC-8_3.9x4.9mm_P1.27mm, symbol Transistor_FET:IRF7404
- added Q?: Si4186DY, Package_SO:SOIC-8_3.9x4.9mm_P1.27mm, symbol Transistor_FET:Si4162DY
- added R? (x2): 100K, symbol Device:R
- added R?: 20K, symbol Device:R
- added R?: 10K, symbol Device:R
- D?: value 1.2V zener -> 3.6V Zener
- Q? (x3): value IRF7425 -> IRF7458
- R?: value 10K -> R
Connections:
- net +BATT: now also R?.1
- net -BATT: now also Q?.5 (D), Q?.6 (D), Q?.7 (D), Q?.8 (D), R?.2; no longer Q?.5 (D), Q?.6 (D), Q?.7 (D), Q?.8 (D)
- net Cell1/-: no longer R?.1
- net GND: now also Q?.5 (D), Q?.6 (D), Q?.7 (D), Q?.8 (D); no longer Q?.1 (S), Q?.2 (S), Q?.3 (S), R?.2
- net at Q?.4 (G), SW?.1 (A): now also C?.1, Q?.4 (G), R?.2
- net at Q?.1 (S), Q?.2 (S), Q?.3 (S)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: now also C?.1, Q?.1 (S), Q?.2 (S), Q?.3 (S), R?.1; no longer R?.1, R?.1, U?.3 (-), U?.4 (+)
- net at Q?.4 (G): now also SW?.2 (B), C?.2, Q?.4 (G), R?.1; no longer SW?.1 (A)
- net at Q?.5 (D), Q?.6 (D), Q?.7 (D)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: now also R?.1, U?.2 (-), U?.4 (+); no longer Q?.1 (S), Q?.2 (S), Q?.3 (S), R?.1
- net at Q?.5 (D), Q?.6 (D), Q?.7 (D)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: now also Q?.5 (D), Q?.6 (D), Q?.7 (D), Q?.8 (D); no longer Q?.1 (S), Q?.2 (S), Q?.3 (S)
- net at Q?.5 (D), Q?.6 (D), Q?.7 (D)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: now also R?.1, Q?.5 (D), Q?.6 (D), Q?.7 (D), Q?.8 (D); no longer Q?.5 (D), Q?.6 (D), Q?.7 (D), Q?.8 (D)
- net at R?.2: now also SW?.1 (A); no longer SW?.2 (B)
- net at D?.1 (K), R?.2: now also R?.1; no longer U?.6 (-)
- new net: C?.2, Q?.1 (S), Q?.1 (S), Q?.2 (S), Q?.2 (S), Q?.3 (S), Q?.3 (S), R?.2, R?.2
- new net: Q?.1 (S), Q?.1 (S), Q?.2 (S), Q?.2 (S), Q?.3 (S), Q?.3 (S)
- new net: R?.1, U?.3 (-)
- new net: R?.1, R?.2, U?.6 (-)
- no-connect marks 16 -> 17
Other:
- moved on the sheet: C?, D?, F?, Q?, R?, SW?, U?, U?B

Commit message: add programming to micro
Parts:
- added C? (x4): 0.1uF, symbol Device:C
- added C?: 10uF, symbol Device:C
- added C? (x2): 20pF, symbol Device:C
- added J?: SWD, symbol Connector:Conn_01x04_Male
- added R?: 10K, symbol Device:R
- added Y?: 8MHz, symbol Device:Crystal
Connections:
- net +3V3: now also C?.1, C?.1, C?.1, C?.1, C?.1, J?.1 (Pin_1), R?.1
- net GND: now also C?.2, C?.2, C?.2, C?.2, C?.2, C?.2, C?.2, J?.4 (Pin_4)
- net BOOT1: now reaches U?.20 (PB2)
- net SWDIO: now reaches U?.34 (PA13)
- net SWDIO: now also J?.2 (Pin_2)
- net SWDCLK: now reaches U?.37 (PA14)
- net SWDCLK: now also J?.3 (Pin_3)
- net BOOT0: now reaches U?.44 (BOOT0)
- net at U?.5 (PD0): now also C?.1, Y?.1
- net at U?.6 (PD1): now also C?.1, Y?.2
- net at U?.7 (NRST): now also R?.2

Commit message: Boot jumper
Parts:
- added J?: BOOT, symbol Connector:Conn_01x03_Male
- added R? (x2): 100K, symbol Device:R
Connections:
- net +3V3: now also J?.1 (Pin_1)
- net BOOT0: now also R?.1
- net BOOT1: now also R?.1
- net GND: now also J?.3 (Pin_3), R?.2
- new net: J?.2 (Pin_2), R?.2
Changed lines of the file:
@@
+	1    0    0    -1
+$EndComp
+Wire Wire Line
+	8900 3350 9200 3350
+Text Label 9200 3350 2    50   ~ 0
+BOOT0
+Wire Wire Line
+	8200 3250 7900 3250
+Text Label 7900 3250 0    50   ~ 0
+BOOT1
+$Comp
+L Device:R R?
+U 1 1 61D8C5EC
+P 8200 3400
+F 0 "R?" V 8100 3400 50  0000 C CNN
+F 1 "100K" V 8200 3400 50  0000 C CNN
+F 2 "" V 8130 3400 50  0001 C CNN
+F 3 "~" H 8200 3400 50  0001 C CNN
+	1    8200 3400
+	1    0    0    -1
+$EndComp
+$Comp
+L Device:R R?
+U 1 1 61D9FB1D
+P 8750 3350
+F 0 "R?" V 8650 3350 50  0000 C CNN
+F 1 "100K" V 8750 3350 50  0000 C CNN
+F 2 "" V 8680 3350 50  0001 C CNN
+F 3 "~" H 8750 3350 50  0001 C CNN
+	1    8750 3350
+	0    1    1    0
+$EndComp
+$Comp
+L Connector:Conn_01x03_Male J?
+U 1 1 61DD6434
+P 8400 3350
+F 0 "J?" H 8508 3631 50  0000 C CNN
+F 1 "BOOT" H 8508 3540 50  0000 C CNN
+F 2 "" H 8400 3350 50  0001 C CNN
+F 3 "~" H 8400 3350 50  0001 C CNN
+	1    8400 3350
+	1    0    0    -1
+$EndComp
+Wire Wire Line
+	8600 3250 8700 3250
+Wire Wire Line
+	8700 3250 8700 3150
+Wire Wire Line
+	8600 3450 8700 3450
+$Comp
+L power:+3V3 #PWR?
+U 1 1 61E560DB
+P 8700 3150
+AR Path="/61E560DB" Ref="#PWR?"  Part="1"
+AR Path="/61BD4B7D/61E560DB" Ref="#PWR?"  Part="1"
+F 0 "#PWR?" H 8700 3000 50  0001 C CNN
+F 1 "+3V3" V 8715 3278 50  0000 L CNN
+F 2 "" H 8700 3150 50  0001 C CNN
+F 3 "" H 8700 3150 50  0001 C CNN
+	1    8700 3150
+	1    0    0    -1
+$EndComp
+Wire Wire Line
+	8700 3450 8700 3550
+$Comp
+L power:GND #PWR?
+U 1 1 61E7AC27
+P 8700 3550
+AR Path="/61E7AC27" Ref="#PWR?"  Part="1"
+AR Path="/61BD4B7D/61E7AC27" Ref="#PWR?"  Part="1"
+F 0 "#PWR?" H 8700 3300 50  0001 C CNN
+F 1 "GND" H 8705 3377 50  0000 C CNN
+F 2 "" H 8700 3550 50  0001 C CNN
+F 3 "" H 8700 3550 50  0001 C CNN
+	1    8700 3550
+	1    0    0    -1
+$EndComp
+$Comp
+L power:GND #PWR?
+U 1 1 61EC69E9
+P 8200 3550
+AR Path="/61EC69E9" Ref="#PWR?"  Part="1"
+AR Path="/61BD4B7D/61EC69E9" Ref="#PWR?"  Part="1"
+F 0 "#PWR?" H 8200 3300 50  0001 C CNN
+F 1 "GND" H 8205 3377 50  0000 C CNN
+F 2 "" H 8200 3550 50  0001 C CNN
+F 3 "" H 8200 3550 50  0001 C CNN
+	1    8200 3550
 	1    0    0    -1
 $EndComp
