File: ECAD/PowerConditioning.sch (KiCad schematic (older format))
At the start: 17 parts

Commit message: Finish components for buck converters, add UVLO feature, correct all mosfet orientations
Parts:
- removed C? (x4): C, symbol Device:C
- added C? (x16): 220uF, symbol Device:CP
- added C? (x4): 0.1uF, symbol Device:C
- added C? (x2): 10uF, symbol Device:C
- added C? (x2): 1uF, symbol Device:C
- added L?: L, symbol Device:L
- added Q?: IRF7425, Package_SO:SOIC-8_3.9x4.9mm_P1.27mm, symbol Transistor_FET:IRF7404
- added Q?: 2N7002, Package_TO_SOT_SMD:SOT-23, symbol Transistor_FET:2N7002
- added Q?: Si7336ADP, Package_SO:PowerPAK_SO-8_Single, symbol Transistor_FET:Si7336ADP
- added R?: 40K, symbol Device:R
- added R?: 30K, symbol Device:R
- added R?: 7.5K, symbol Device:R
- added R?: 40m, symbol Device:R
- added U? (x3): LM358, symbol Amplifier_Operational:LM358
- added U?: ADR4530, Package_SO:SOIC-8_3.9x4.9mm_P1.27mm, symbol Reference_Voltage:ADR4530
- D? (x2): value D_Schottky -> RB051MM-2Y
- Q? (x2): value Si7141DP -> SIR167DP
Connections:
- net labels added: PCM_FILT, PCM_IN
- wire segments 47 -> 134
Other:
- note added: "Lower resistor provides hysteresis for UVLO\nFalling threshold, with the mosfet conducting, is 6.2V \n(6.199 taking into account 7.5 ohm Rds(on))\nRising threshold, with mosfet open, is 7V"
- note added: "UV Active High\nCompares with a 3V ref\n"
- note added: "Undervoltage Protection"
- moved on the sheet: C?, D?, L?, Q?, R?, U?

Commit message: Finish speccing out components for 12V boost
Parts:
- removed C?: 1uF, symbol Device:C
- added C? (x2): 220uF, symbol Device:CP
- added C?: 100uF, symbol Device:CP
- added C?: 330pF, symbol Device:C
- added C?: 100pF, symbol Device:C
- added D?: RB051MM-2Y, symbol Device:D_Schottky
- added R?: 91K, symbol Device:R
- added R?: 10K, symbol Device:R
- added R?: 3.3K, symbol Device:R
- L? (x2): value 47uH -> 68uH
- L?: value L -> 100uH
- R?: value 40m -> 25m
Connections:
- net GND: now also C?.1, Q?.1 (S), Q?.2 (S), Q?.3 (S), U?.4 (GND), U?.5 (SW), C?.2, C?.2, C?.2, C?.2, R?.2, R?.2
- net PCM_FILT: now also R?.1, U?.8 (Vin), C?.1
- net at R?.2, U?.1 (SENSE-): now also L?.1; no longer Q?.5 (D)
- net at U?.2 (Ith/RUN): now also C?.1
- net at U?.3 (Vfb): now also C?.1, R?.1, R?.2
- net at L?.2: now also Q?.5 (D), D?.2 (A)
- new net: C?.1, C?.1, D?.1 (K), R?.1
- new net: C?.2, R?.1
Other:
- note added: "Vout = 1.19V * (Rtop/Rbottom + 1)"
- moved on the sheet: C?, L?, Q?, R?, U?

Commit message: Remove zeners, add PDMs, correct MPPT setpoint controller
Parts:
- added C?: 220uF, symbol Device:CP
- C?: value 220uF -> 100uF
Connections:
- net GND: now also C?.2
- net at C?.1, C?.1, D?.1 (K)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: now also C?.1
Changed lines of the file:
@@
 $Descr A4 11693 8268
 encoding utf-8
-Sheet 15 15
+Sheet 15 30
 Title ""
 Date ""
@@
 P 8000 2700
 F 0 "C?" H 8118 2746 50  0000 L CNN
-F 1 "220uF" H 8118 2655 50  0000 L CNN
+F 1 "100uF" H 8118 2655 50  0000 L CNN
 F 2 "" H 8038 2550 50  0001 C CNN
 F 3 "~" H 8000 2700 50  0001 C CNN
@@
 	4900 1950 5200 1950
 Connection ~ 5200 1950
+$Comp
+L Device:CP C?
+U 1 1 61E67A6A
+P 8900 2700
+F 0 "C?" H 9018 2746 50  0000 L CNN
+F 1 "220uF" H 9018 2655 50  0000 L CNN
+F 2 "" H 8938 2550 50  0001 C CNN
+F 3 "~" H 8900 2700 50  0001 C CNN
+	1    8900 2700
+	1    0    0    -1
+$EndComp
+Wire Wire Line
+	8900 2550 8450 2550
+Connection ~ 8450 2550
+Wire Wire Line
+	8450 3250 8900 3250
+Wire Wire Line
+	8900 3250 8900 2850
+Connection ~ 8450 3250
 $EndSCHEMATC

Commit message: Cleanup, add yellow fill to symbols, add MAX4373
Parts:
- added R? (x2): 10K, symbol Device:R
- added U? (x3): MAX4373F, symbol symbols:MAX4373F
Connections:
- net GND: now also R?.2, R?.2; no longer U?.3 (SHDN), U?.3 (SHDN)
- new net: R?.1, U?.3 (SHDN) (x2)
Changed lines of the file:
@@
 	2100 5800 1650 5800
-Wire Wire Line
-	1650 5800 1650 6150
-Connection ~ 1650 6150
 Wire Wire Line
 	2000 4450 2000 3750
@@
 	3200 3750 3200 4100
 Connection ~ 3200 4100
-Wire Wire Line
-	1650 4100 1650 5150
 $Comp
 L Device:C C?
@@
 Wire Wire Line
 	1650 4100 2100 4100
-Wire Wire Line
-	1650 5150 1800 5150
 Connection ~ 1800 5150
 Wire Wire Line
@@
 Wire Wire Line
 	3200 6850 2500 6850
-Connection ~ 1650 5150
 Wire Wire Line
 	1350 5750 1350 6850
@@
 U 1 1 61CB8B7D
 P 3200 5950
-F 0 "R?" H 3270 5996 50  0000 L CNN
+F 0 "R?" H 3250 5950 50  0000 L CNN
 F 1 "15m" V 3200 5950 50  0000 C CNN
 F 2 "" V 3130 5950 50  0001 C CNN
@@
 U 1 1 61CA3226
 P 3200 4250
-F 0 "R?" H 3270 4296 50  0000 L CNN
+F 0 "R?" H 3250 4250 50  0000 L CNN
 F 1 "15m" V 3200 4250 50  0000 C CNN
 F 2 "" V 3130 4250 50  0001 C CNN
@@
 Wire Wire Line
 	1350 5150 1350 4050
-Wire Wire Line
-	1350 5150 1650 5150
 Connection ~ 1350 4050
 Wire Wire Line
@@
 	8900 3250 8900 2850
 Connection ~ 8450 3250
+Wire Wire Line
+	1350 5150 1650 5150
+$Comp
+L Device:R R?
+U 1 1 621D1188
+P 1650 4250
+F 0 "R?" H 1700 4250 50  0000 L CNN
+F 1 "10K" V 1650 4250 50  0000 C CNN
+F 2 "" V 1580 4250 50  0001 C CNN
+F 3 "~" H 1650 4250 50  0001 C CNN
+	1    1650 4250
+	1    0    0    -1
+$EndComp
+Wire Wire Line
+	1650 4400 1650 5150
+Connection ~ 1650 5150
+Wire Wire Line
+	1650 5150 1800 5150
+$Comp
+L Device:R R?
+U 1 1 621EBB75
+P 1650 5950
+F 0 "R?" H 1700 5950 50  0000 L CNN
+F 1 "10K" V 1650 5950 50  0000 C CNN
+F 2 "" V 1580 5950 50  0001 C CNN
+F 3 "~" H 1650 5950 50  0001 C CNN
+	1    1650 5950
+	1    0    0    -1
+$EndComp
+Wire Wire Line
+	1650 6100 1650 6150
+Connection ~ 1650 6150
+$Comp
+L symbols:MAX4373F U?
+U 1 1 62204B6C
+P 10350 2550
+F 0 "U?" H 10350 1411 50  0000 C CNN
+F 1 "MAX4373F" H 10350 1320 50  0000 C CNN
+F 2 "" H 10350 2650 50  0001 C CNN
+F 3 "" H 10350 2650 50  0001 C CNN
+	1    10350 2550
+	1    0    0    -1
+$EndComp
+$Comp
+L symbols:MAX4373F U?
+U 1 1 62206289
+P 6900 4250
+F 0 "U?" H 6900 3111 50  0000 C CNN
+F 1 "MAX4373F" H 6900 3020 50  0000 C CNN
+F 2 "" H 6900 4350 50  0001 C CNN
+F 3 "" H 6900 4350 50  0001 C CNN
+	1    6900 4250
+	1    0    0    -1
+$EndComp
+$Comp
+L symbols:MAX4373F U?
+U 1 1 6220D7B9
+P 6950 5950
+F 0 "U?" H 6950 4811 50  0000 C CNN
+F 1 "MAX4373F" H 6950 4720 50  0000 C CNN
+F 2 "" H 6950 6050 50  0001 C CNN
+F 3 "" H 6950 6050 50  0001 C CNN
+	1    6950 5950
+	1    0    0    -1
+$EndComp
 $EndSCHEMATC

Commit message: Add OCP, resize some sheets
Parts:
- removed U? (x2): MAX4373F, symbol symbols:MAX4373F
- added C? (x4): 0.1uF, symbol Device:C
- added C? (x2): 10uF, symbol Device:C
- added Q? (x4): 2N7002, Package_TO_SOT_SMD:SOT-23, symbol Transistor_FET:2N7002
- added Q? (x4): IRF7425, Package_SO:SOIC-8_3.9x4.9mm_P1.27mm, symbol Transistor_FET:IRF7404
- added R? (x12): 10K, symbol Device:R
- added R?: 25m, symbol Device:R
- added R? (x2): 9.5K, symbol Device:R
- added R? (x2): 3K, symbol Device:R
- added R? (x3): 10m, symbol Device:R
- added R? (x2): 11K, symbol Device:R
- added R? (x2): 4K, symbol Device:R
- added U? (x3): MAX4373F, symbol symbols:MAX4373F
- added U?: LM1117-3.3, symbol Regulator_Linear:LM1117-3.3
Connections:
- net GND: now also C?.2, C?.2, C?.2, C?.2, C?.2, C?.2, U?.4 (GND), C?.2, C?.2, C?.2, C?.2, C?.2, C?.2, Q?.2 (S), Q?.2 (S), Q?.2 (S), Q?.2 (S), R?.2, R?.2, R?.2, R?.2, U?.1 (GND), U?.4 (GND), U?.4 (GND), U?.4 (GND)
- net PCM_FILT: now also C?.1, Q?.1 (S), Q?.2 (S), Q?.3 (S), R?.1, U?.3 (VI)
- net at C?.1, C?.1, C?.1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: now also Q?.1 (S), Q?.2 (S), Q?.3 (S), R?.1 (x2)
- net at C?.1, C?.1, C?.1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: now also Q?.1 (S), Q?.2 (S), Q?.3 (S), R?.1
- net VCC: now reaches U?.1 (Vcc)
- net VCC: now also C?.1, C?.1, C?.1, C?.1, C?.1, R?.1, R?.1, R?.1, R?.1, R?.1, R?.1, R?.1, R?.1, U?.1 (Vcc), U?.1 (Vcc), U?.1 (Vcc), U?.2 (VO)
- net TELEM_I12V: now reaches U?.2 (OUT)
- net TELEM_I12V: now also R?.1
- net at U?.3 (CIN1): now also R?.1, R?.2
- net RST12VOCP: now reaches U?.5 (~RESET)
- net RST12VOCP: now also R?.2
- net at U?.6 (COUT1): now also Q?.1 (G), R?.2
- net +12V: now reaches U?.7 (RS-)
- net +12V: now also R?.1
- net at U?.8 (RS+): now also Q?.5 (D), Q?.6 (D), Q?.7 (D), Q?.8 (D), R?.2
- new net: Q?.3 (D), Q?.4 (G), R?.2 (x4)
- new net: R?.1, R?.2, U?.3 (CIN1) (x3)
- new net: Q?.1 (G), R?.2, U?.6 (COUT1) (x3)
- new net: Q?.5 (D), Q?.6 (D), Q?.7 (D), Q?.8 (D), R?.2, U?.8 (RS+) (x3)
- new net +3V3: R?.1, U?.7 (RS-)
- new net +5V: R?.1, U?.7 (RS-)
- new net +BATT: R?.1, U?.7 (RS-)
- new net RST3V3OCP: R?.2, U?.5 (~RESET)
- new net RST5VOCP: R?.2, U?.5 (~RESET)
- new net RSTBATVOCP: R?.2, U?.5 (~RESET)
- new net TELEM_I3V3: R?.1, U?.2 (OUT)
- new net TELEM_I5V: R?.1, U?.2 (OUT)
- new net TELEM_IBATV: R?.1, U?.2 (OUT)
Other:
- note added: "2A OCP\nIover = (0.6V / (Rsense * Av)) * (Rtop + Rbottom) / Rbottom"
- note added: "5V and 3V3 OCP set to 4.5A"
- note added: "Battery OCP set to 5A"
- moved on the sheet: C?, D?, L?, Q?, R?, U?

Commit message: bidirectional inhibits, remove unrealistic zener, replace all irf7425 with irf7458
Parts:
- Q? (x5): value IRF7425 -> IRF7458
Changed lines of the file:
@@
 P 3250 900
 F 0 "Q?" V 3592 900 50  0000 C CNN
-F 1 "IRF7425" V 3501 900 50  0000 C CNN
+F 1 "IRF7458" V 3501 900 50  0000 C CNN
 F 2 "Package_SO:SOIC-8_3.9x4.9mm_P1.27mm" H 3450 825 50  0001 L CIN
 F 3 "http://www.infineon.com/dgdl/irf7404.pdf?fileId=5546d462533600a4015355fa2b5b1b9e" V 3250 900 50  0001 L CNN
@@
 P 9100 1350
 F 0 "Q?" V 9442 1350 50  0000 C CNN
-F 1 "IRF7425" V 9351 1350 50  0000 C CNN
+F 1 "IRF7458" V 9351 1350 50  0000 C CNN
 F 2 "Package_SO:SOIC-8_3.9x4.9mm_P1.27mm" H 9300 1275 50  0001 L CIN
 F 3 "http://www.infineon.com/dgdl/irf7404.pdf?fileId=5546d462533600a4015355fa2b5b1b9e" V 9100 1350 50  0001 L CNN
@@
 P 7400 4450
 F 0 "Q?" V 7742 4450 50  0000 C CNN
-F 1 "IRF7425" V 7651 4450 50  0000 C CNN
+F 1 "IRF7458" V 7651 4450 50  0000 C CNN
 F 2 "Package_SO:SOIC-8_3.9x4.9mm_P1.27mm" H 7600 4375 50  0001 L CIN
 F 3 "http://www.infineon.com/dgdl/irf7404.pdf?fileId=5546d462533600a4015355fa2b5b1b9e" V 7400 4450 50  0001 L CNN
@@
 P 6500 2750
 F 0 "Q?" V 6842 2750 50  0000 C CNN
-F 1 "IRF7425" V 6751 2750 50  0000 C CNN
+F 1 "IRF7458" V 6751 2750 50  0000 C CNN
 F 2 "Package_SO:SOIC-8_3.9x4.9mm_P1.27mm" H 6700 2675 50  0001 L CIN
 F 3 "http://www.infineon.com/dgdl/irf7404.pdf?fileId=5546d462533600a4015355fa2b5b1b9e" V 6500 2750 50  0001 L CNN
@@
 P 7400 6150
 F 0 "Q?" V 7742 6150 50  0000 C CNN
-F 1 "IRF7425" V 7651 6150 50  0000 C CNN
+F 1 "IRF7458" V 7651 6150 50  0000 C CNN
 F 2 "Package_SO:SOIC-8_3.9x4.9mm_P1.27mm" H 7600 6075 50  0001 L CIN
 F 3 "http://www.infineon.com/dgdl/irf7404.pdf?fileId=5546d462533600a4015355fa2b5b1b9e" V 7400 6150 50  0001 L CNN
