File: ECAD/PowerConditioning.sch (KiCad schematic (older format))
At the start: 103 parts

Commit message: ceramics
Parts:
- removed C? (x4): 220uF, symbol Device:CP
- removed C?: 100uF, symbol Device:CP
- added C? (x5): 47uF, symbol Device:C
- L? (x2): value 68uH -> 100uH
- L?: value 100uH -> 220uH
Connections:
- net GND: now also C?.2, C?.2, C?.2, C?.2, C?.2
- net PCM_FILT: now also C?.1, C?.1, C?.1, C?.1, C?.1
Other:
- moved on the sheet: C?, D?, L?, Q?, R?, U?

Commit message: 555 retry timer?
Connections:
- net VCC: now also U?.6 (COUT1)
- net at Q?.1 (G), R?.2: no longer U?.6 (COUT1)
Other:
- moved on the sheet: R?, U?
Changed lines of the file:
@@
 $Descr USLegal 14000 8500
 encoding utf-8
-Sheet 16 31
+Sheet 16 32
 Title "TJ Custom EPS"
 Date ""
@@
 L symbols:MAX4373F U?
 U 1 1 62204B6C
-P 10250 1350
-F 0 "U?" H 10250 211 50  0000 C CNN
-F 1 "MAX4373F" H 10250 120 50  0000 C CNN
-F 2 "" H 10250 1450 50  0001 C CNN
-F 3 "" H 10250 1450 50  0001 C CNN
-	1    10250 1350
+P 10400 1350
+F 0 "U?" H 10400 211 50  0000 C CNN
+F 1 "MAX4373F" H 10400 120 50  0000 C CNN
+F 2 "" H 10400 1450 50  0001 C CNN
+F 3 "" H 10400 1450 50  0001 C CNN
+	1    10400 1350
 	1    0    0    -1
 $EndComp
@@
 L Device:R R?
 U 1 1 61D990E5
-P 10250 1250
-F 0 "R?" V 10150 1250 50  0000 C CNN
-F 1 "25m" V 10250 1250 50  0000 C CNN
-F 2 "" V 10180 1250 50  0001 C CNN
-F 3 "~" H 10250 1250 50  0001 C CNN
-	1    10250 1250
+P 10400 1250
+F 0 "R?" V 10300 1250 50  0000 C CNN
+F 1 "25m" V 10400 1250 50  0000 C CNN
+F 2 "" V 10330 1250 50  0001 C CNN
+F 3 "~" H 10400 1250 50  0001 C CNN
+	1    10400 1250
 	0    1    1    0
 $EndComp
 Wire Wire Line
-	10100 1350 10100 1250
-Wire Wire Line
-	10400 1350 10400 1250
-Connection ~ 10100 1250
+	10250 1350 10250 1250
+Wire Wire Line
+	10550 1350 10550 1250
+Connection ~ 10250 1250
 $Comp
 L Device:C C?
@@
 $EndComp
 Wire Wire Line
-	9500 1850 9850 1850
+	9650 1850 10000 1850
 Wire Wire Line
 	9200 1650 9200 1600
@@
 $EndComp
 Wire Wire Line
-	9200 2400 9650 2400
-Wire Wire Line
-	9650 2100 9650 1700
-Wire Wire Line
-	9400 1250 10100 1250
-Connection ~ 9650 2400
-Wire Wire Line
-	9650 2400 9900 2400
-Wire Wire Line
-	9650 1700 9700 1700
+	9650 2100 9650 1850
 $Comp
 L power:VCC #PWR?
@@
 $EndComp
 Wire Wire Line
-	9650 1700 9650 1550
-Wire Wire Line
 	9650 1550 9500 1550
-Connection ~ 9650 1700
 $Comp
 L Device:R R?
 U 1 1 61D75536
-P 9700 1950
-F 0 "R?" H 9750 1950 50  0000 L CNN
-F 1 "10K" V 9700 1950 50  0000 C CNN
-F 2 "" V 9630 1950 50  0001 C CNN
-F 3 "~" H 9700 1950 50  0001 C CNN
-	1    9700 1950
-	1    0    0    -1
-$EndComp
-Wire Wire Line
-	9700 1800 9700 1700
-Connection ~ 9700 1700
-Wire Wire Line
-	9700 1700 9850 1700
+P 9850 1950
+F 0 "R?" H 9900 1950 50  0000 L CNN
+F 1 "10K" V 9850 1950 50  0000 C CNN
+F 2 "" V 9780 1950 50  0001 C CNN
+F 3 "~" H 9850 1950 50  0001 C CNN
+	1    9850 1950
+	1    0    0    -1
+$EndComp
+Wire Wire Line
+	9850 1800 9850 1700
+Connection ~ 9850 1700
+Wire Wire Line
+	9850 1700 10000 1700
 Connection ~ 9500 1550
-Connection ~ 9500 1850
-Wire Wire Line
-	9850 2150 9700 2150
-Wire Wire Line
-	9700 2150 9700 2100
-Wire Wire Line
-	9700 2150 9500 2150
-Connection ~ 9700 2150
-Text GLabel 9500 2150 0    50   Input ~ 0
+Wire Wire Line
+	10000 2150 9850 2150
+Wire Wire Line
+	9850 2150 9850 2100
+Text GLabel 9150 2150 0    50   Input ~ 0
 RST12VOCP
 $Comp
 L Device:R R?
 U 1 1 61DA1480
-P 10700 1900
-F 0 "R?" H 10750 1900 50  0000 L CNN
-F 1 "9.5K" V 10700 1900 50  0000 C CNN
-F 2 "" V 10630 1900 50  0001 C CNN
-F 3 "~" H 10700 1900 50  0001 C CNN
-	1    10700 1900
+P 10850 1900
+F 0 "R?" H 10900 1900 50  0000 L CNN
+F 1 "9.5K" V 10850 1900 50  0000 C CNN
+F 2 "" V 10780 1900 50  0001 C CNN
+F 3 "~" H 10850 1900 50  0001 C CNN
+	1    10850 1900
 	1    0    0    -1
 $EndComp
@@
 L Device:R R?
 U 1 1 61DB22B4
-P 10700 2200
-F 0 "R?" H 10750 2200 50  0000 L CNN
-F 1 "3K" V 10700 2200 50  0000 C CNN
-F 2 "" V 10630 2200 50  0001 C CNN
-F 3 "~" H 10700 2200 50  0001 C CNN
-	1    10700 2200
-	1    0    0    -1
-$EndComp
-Wire Wire Line
-	10700 2050 10650 2050
-Connection ~ 10700 2050
-Wire Wire Line
-	10650 1750 10700 1750
-Wire Wire Line
-	10250 2400 10700 2400
-Wire Wire Line
-	10700 2400 10700 2350
-Connection ~ 10250 2400
+P 10850 2200
+F 0 "R?" H 10900 2200 50  0000 L CNN
+F 1 "3K" V 10850 2200 50  0000 C CNN
+F 2 "" V 10780 2200 50  0001 C CNN
+F 3 "~" H 10850 2200 50  0001 C CNN
+	1    10850 2200
+	1    0    0    -1
+$EndComp
+Wire Wire Line
+	10850 2050 10800 2050
+Connection ~ 10850 2050
+Wire Wire Line
+	10800 1750 10850 1750
 $Comp
 L power:GND #PWR?
@@
 $EndComp
 Connection ~ 9900 2400
-Wire Wire Line
-	9900 2400 10250 2400
-Text GLabel 10800 1750 2    50   Input ~ 0
+Text GLabel 10950 1750 2    50   Input ~ 0
 TELEM_I12V
 Wire Wire Line
-	10800 1750 10700 1750
-Connection ~ 10700 1750
+	10950 1750 10850 1750
+Connection ~ 10850 1750
 Text Notes 8550 2700 0    50   ~ 0
 2A OCP\nIover = (0.6V / (Rsense * Av)) * (Rtop + Rbottom) / Rbottom
@@
 Connection ~ 8400 1250
 Wire Wire Line
-	10400 1250 10900 1250
-Connection ~ 10400 1250
+	10550 1250 11050 1250
+Connection ~ 10550 1250
 $Comp
 L power:+12V #PWR?
 U 1 1 61E11F2A
-P 10900 1250
-F 0 "#PWR?" H 10900 1100 50  0001 C CNN
-F 1 "+12V" H 10915 1423 50  0000 C CNN
-F 2 "" H 10900 1250 50  0001 C CNN
-F 3 "" H 10900 1250 50  0001 C CNN
-	1    10900 1250
+P 11050 1250
+F 0 "#PWR?" H 11050 1100 50  0001 C CNN
+F 1 "+12V" H 11065 1423 50  0000 C CNN
+F 2 "" H 11050 1250 50  0001 C CNN
+F 3 "" H 11050 1250 50  0001 C CNN
+	1    11050 1250
 	1    0    0    -1
 $EndComp
@@
 	4300 650  4700 650
 Connection ~ 4700 650
+Connection ~ 9650 1850
+Connection ~ 10400 2400
+Wire Wire Line
+	9200 2400 9650 2400
+Wire Wire Line
+	9650 1550 9650 1700
+Wire Wire Line
+	9900 2400 10400 2400
+Connection ~ 9650 2400
+Wire Wire Line
+	9650 2400 9900 2400
+Wire Wire Line
+	10850 2400 10850 2350
+Wire Wire Line
+	10400 2400 10850 2400
+Wire Wire Line
+	9650 1700 9850 1700
+Connection ~ 9650 1700
+Wire Wire Line
+	9650 1700 9650 1850
+Wire Wire Line
+	9400 1250 10250 1250
+Wire Wire Line
+	9850 2150 9150 2150
+Connection ~ 9850 2150
+$Sheet
+S 12100 1550 1250 850
+U 61DD1DB6
+F0 "RetryTimer12V" 50
+F1 "RetryTimer.sch" 50
+$EndSheet
 $EndSCHEMATC

Commit message: implement a retry timer
Parts:
- L? (x2): value 100uH -> 330uH
- L?: value 220uH -> 330uH
Changed lines of the file:
@@
 $Descr USLegal 14000 8500
 encoding utf-8
-Sheet 16 32
+Sheet 16 35
 Title "TJ Custom EPS"
 Date ""
@@
 P 5200 4900
 F 0 "L?" V 5390 4900 50  0000 C CNN
-F 1 "100uH" V 5299 4900 50  0000 C CNN
+F 1 "330uH" V 5299 4900 50  0000 C CNN
 F 2 "" H 5200 4900 50  0001 C CNN
 F 3 "~" H 5200 4900 50  0001 C CNN
@@
 P 5200 6600
 F 0 "L?" V 5390 6600 50  0000 C CNN
-F 1 "100uH" V 5299 6600 50  0000 C CNN
+F 1 "330uH" V 5299 6600 50  0000 C CNN
 F 2 "" H 5200 6600 50  0001 C CNN
 F 3 "~" H 5200 6600 50  0001 C CNN
@@
 P 6450 1250
 F 0 "L?" V 6640 1250 50  0000 C CNN
-F 1 "220uH" V 6549 1250 50  0000 C CNN
+F 1 "330uH" V 6549 1250 50  0000 C CNN
 F 2 "" H 6450 1250 50  0001 C CNN
 F 3 "~" H 6450 1250 50  0001 C CNN
@@
 Connection ~ 9850 2150
 $Sheet
-S 12100 1550 1250 850
+S 12000 1650 800  250
 U 61DD1DB6
 F0 "RetryTimer12V" 50
 F1 "RetryTimer.sch" 50
+F2 "OUT" I R 12800 1750 50
+F3 "IN" I L 12000 1750 50
+$EndSheet
+$Sheet
+S 8950 3600 800  250
+U 61DAECDC
+F0 "RetryTimerBATV" 50
+F1 "RetryTimer.sch" 50
+F2 "OUT" I R 9750 3700 50
+F3 "IN" I L 8950 3700 50
+$EndSheet
+$Sheet
+S 9300 5150 800  250
+U 61DC440E
+F0 "RetryTimer5V" 50
+F1 "RetryTimer.sch" 50
+F2 "OUT" I R 10100 5250 50
+F3 "IN" I L 9300 5250 50
+$EndSheet
+$Sheet
+S 9800 6300 800  250
+U 61DD9B5B
+F0 "RetryTimer3V3" 50
+F1 "RetryTimer.sch" 50
+F2 "OUT" I R 10600 6400 50
+F3 "IN" I L 9800 6400 50
 $EndSheet
 $EndSCHEMATC

Commit message: fix a minor wire mixup
Connections:
- net VCC: no longer U?.6 (COUT1)
- net at Q?.1 (G), R?.2: now also U?.6 (COUT1)
Changed lines of the file:
@@
 $EndComp
-Wire Wire Line
-	9650 1850 10000 1850
 Wire Wire Line
 	9200 1650 9200 1600
@@
 	1    0    0    -1
 $EndComp
-Wire Wire Line
-	9650 2100 9650 1850
 $Comp
 L power:VCC #PWR?
@@
 	4300 650  4700 650
 Connection ~ 4700 650
-Connection ~ 9650 1850
 Connection ~ 10400 2400
 Wire Wire Line
@@
 	9650 1700 9850 1700
 Connection ~ 9650 1700
-Wire Wire Line
-	9650 1700 9650 1850
 Wire Wire Line
 	9400 1250 10250 1250
@@
 F3 "IN" I L 9800 6400 50
 $EndSheet
+Wire Wire Line
+	9650 1700 9650 2100
+Wire Wire Line
+	9500 1850 10000 1850
+Connection ~ 9500 1850
 $EndSCHEMATC

Commit message: connect retry timers, organize sheet
Parts:
- removed C? (x3): 0.1uF, symbol Device:C
- removed Q? (x3): 2N7002, Package_TO_SOT_SMD:SOT-23, symbol Transistor_FET:2N7002
- removed Q? (x3): IRF7458, Package_SO:SOIC-8_3.9x4.9mm_P1.27mm, symbol Transistor_FET:IRF7404
- removed R? (x3): 10m, symbol Device:R
- removed R? (x9): 10K, symbol Device:R
- removed R? (x2): 11K, symbol Device:R
- removed R? (x2): 4K, symbol Device:R
- removed R?: 9.5K, symbol Device:R
- removed R?: 3K, symbol Device:R
- removed U? (x3): MAX4373F, symbol symbols:MAX4373F
- added C? (x3): 0.1uF, symbol Device:C
- added Q? (x3): 2N7002, Package_TO_SOT_SMD:SOT-23, symbol Transistor_FET:2N7002
- added Q? (x3): IRF7458, Package_SO:SOIC-8_3.9x4.9mm_P1.27mm, symbol Transistor_FET:IRF7404
- added R? (x9): 10K, symbol Device:R
- added R?: 3K, symbol Device:R
- added R?: 9.5K, symbol Device:R
- added R? (x3): 10m, symbol Device:R
- added R? (x2): 4K, symbol Device:R
- added R? (x2): 11K, symbol Device:R
- added U? (x3): MAX4373F, symbol symbols:MAX4373F
Connections:
- net +3V3: now also R?.1, U?.7 (RS-)
- net +5V: now also R?.1, U?.7 (RS-)
- net +BATT: now also R?.1, U?.7 (RS-)
- net GND: now also C?.2, C?.2, C?.2, Q?.2 (S), Q?.2 (S), Q?.2 (S), R?.2, R?.2, R?.2, U?.4 (GND), U?.4 (GND), U?.4 (GND)
- net PCM_FILT: now also Q?.1 (S), Q?.2 (S), Q?.3 (S), R?.1
- net TELEM_I3V3: now also R?.1, U?.2 (OUT)
- net TELEM_I5V: now also R?.1, U?.2 (OUT)
- net TELEM_IBATV: now also R?.1, U?.2 (OUT)
- net VCC: now also C?.1, C?.1, C?.1, R?.1, R?.1, R?.1, R?.1, R?.1, R?.1, U?.1 (Vcc), U?.1 (Vcc), U?.1 (Vcc)
- net at C?.1, C?.1, C?.1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: now also Q?.1 (S), Q?.2 (S), Q?.3 (S), R?.1 (x2)
- net GATE12V: now reaches Q?.1 (G), R?.2, U?.6 (COUT1)
- net RST12VOCP renamed RST12V
- new net: Q?.3 (D), Q?.4 (G), R?.2 (x3)
- new net: Q?.5 (D), Q?.6 (D), Q?.7 (D), Q?.8 (D), R?.2, U?.8 (RS+) (x3)
- new net: R?.1, R?.2, U?.3 (CIN1) (x3)
- new net GATE3V3: Q?.1 (G), R?.2, U?.6 (COUT1)
- new net GATE5V: Q?.1 (G), R?.2, U?.6 (COUT1)
- new net GATEBATV: Q?.1 (G), R?.2, U?.6 (COUT1)
- new net RST3V3: R?.2, U?.5 (~RESET)
- new net RST5V: R?.2, U?.5 (~RESET)
- new net RSTBATV: R?.2, U?.5 (~RESET)
Other:
- note added: "12V Boost PCM"
- note added: "5V and 3V3 Buck PCMs"
- note added: "Always On Regulator"
- note added: "BATV PCM (OCP)"
- moved on the sheet: C?, D?, L?, Q?, R?, U?

Commit message: update values
Parts:
- C?: value 0.1uF -> 1nF
- L? (x3): value 330uH -> 270uH
Changed lines of the file:
@@
 P 3600 5500
 F 0 "L?" V 3790 5500 50  0000 C CNN
-F 1 "330uH" V 3699 5500 50  0000 C CNN
+F 1 "270uH" V 3699 5500 50  0000 C CNN
 F 2 "" H 3600 5500 50  0001 C CNN
 F 3 "~" H 3600 5500 50  0001 C CNN
@@
 P 3600 7200
 F 0 "L?" V 3790 7200 50  0000 C CNN
-F 1 "330uH" V 3699 7200 50  0000 C CNN
+F 1 "270uH" V 3699 7200 50  0000 C CNN
 F 2 "" H 3600 7200 50  0001 C CNN
 F 3 "~" H 3600 7200 50  0001 C CNN
@@
 $EndComp
 $Comp
-L Device:C C?
-U 1 1 62011AC8
-P 6200 1900
-F 0 "C?" H 6315 1946 50  0000 L CNN
-F 1 "0.1uF" H 6315 1855 50  0000 L CNN
-F 2 "" H 6238 1750 50  0001 C CNN
-F 3 "~" H 6200 1900 50  0001 C CNN
-	1    6200 1900
-	1    0    0    -1
-$EndComp
-$Comp
 L Device:L L?
 U 1 1 620059FF
 P 6500 1350
 F 0 "L?" V 6690 1350 50  0000 C CNN
-F 1 "330uH" V 6599 1350 50  0000 C CNN
+F 1 "270uH" V 6599 1350 50  0000 C CNN
 F 2 "" H 6500 1350 50  0001 C CNN
 F 3 "~" H 6500 1350 50  0001 C CNN
@@
 Text Notes 4350 600  0    50   ~ 0
 12V Boost PCM
+$Comp
+L Device:C C?
+U 1 1 62011AC8
+P 6200 1900
+F 0 "C?" H 6315 1946 50  0000 L CNN
+F 1 "1nF" H 6315 1855 50  0000 L CNN
+F 2 "" H 6238 1750 50  0001 C CNN
+F 3 "~" H 6200 1900 50  0001 C CNN
+	1    6200 1900
+	1    0    0    -1
+$EndComp
 $EndSCHEMATC

Commit message: Implement pulse resets
Parts:
- added Q? (x4): 2N7002, Package_TO_SOT_SMD:SOT-23, symbol Transistor_FET:2N7002
Connections:
- net GND: now also Q?.2 (S), Q?.2 (S), Q?.2 (S), Q?.2 (S); no longer Q?.2 (S), Q?.2 (S), Q?.2 (S), Q?.2 (S)
- net RST12V: no longer R?.2, U?.5 (~RESET)
- net RST3V3: no longer R?.2, U?.5 (~RESET)
- net RST5V: no longer R?.2, U?.5 (~RESET)
- net RSTBATV: no longer R?.2, U?.5 (~RESET)
- new net: Q?.2 (S), Q?.3 (D) (x4)
- new net RST12VOCP: R?.2, U?.5 (~RESET)
- new net RST12VPLS: Q?.1 (G)
- new net RST3V3OCP: R?.2, U?.5 (~RESET)
- new net RST3V3PLS: Q?.1 (G)
- new net RST5VOCP: R?.2, U?.5 (~RESET)
- new net RST5VPLS: Q?.1 (G)
- new net RSTBATVOCP: R?.2, U?.5 (~RESET)
- new net RSTBATVPLS: Q?.1 (G)
Other:
- moved on the sheet: C?, U?
