File: ECAD/USB+Boost-BuckMPPT.sch (KiCad schematic (older format))
At the start: 37 parts

Commit message: add comments and titles
Parts:
- added U?: LTC4412xS6, Package_TO_SOT_SMD:TSOT-23-6, symbol Power_Management:LTC4412xS6
Changed lines of the file:
@@
 encoding utf-8
 Sheet 15 31
-Title ""
+Title "TJ Custom EPS"
 Date ""
-Rev ""
-Comp ""
-Comment1 ""
-Comment2 ""
+Rev "0.1"
+Comp "TJHSST Nanosatellite Club"
+Comment1 "Buck-Boost MPPT Converter"
+Comment2 "Boosts voltage by a factor of two before feeding into an MPPT buck IC"
 Comment3 ""
-Comment4 ""
+Comment4 "Engineer: Alan Hsu"
 $EndDescr
 $Comp
@@
 	1    0    0    -1
 $EndComp
+$Comp
+L Power_Management:LTC4412xS6 U?
+U 1 1 61D94799
+P 4600 -850
+F 0 "U?" H 4600 -269 50  0000 C CNN
+F 1 "LTC4412xS6" H 4600 -360 50  0000 C CNN
+F 2 "Package_TO_SOT_SMD:TSOT-23-6" H 5250 -1200 50  0001 C CNN
+F 3 "https://www.analog.com/media/en/technical-documentation/data-sheets/4412fb.pdf" H 6700 -1050 50  0001 C CNN
+	1    4600 -850
+	1    0    0    -1
+$EndComp
