File: ECAD/PDM3V3.sch (KiCad schematic (older format))
At the start: 12 parts

Commit message: bidirectional inhibits, remove unrealistic zener, replace all irf7425 with irf7458
Parts:
- Q?: value IRF7425 -> IRF7458
Changed lines of the file:
@@
 AR Path="/61E87E93/61EF42FB/61E8B663" Ref="Q?"  Part="1"
 F 0 "Q?" H 4755 2196 50  0000 L CNN
-F 1 "IRF7425" H 4755 2105 50  0000 L CNN
+F 1 "IRF7458" H 4755 2105 50  0000 L CNN
 F 2 "Package_SO:SOIC-8_3.9x4.9mm_P1.27mm" H 4750 2075 50  0001 L CIN
 F 3 "http://www.infineon.com/dgdl/irf7404.pdf?fileId=5546d462533600a4015355fa2b5b1b9e" V 4550 2150 50  0001 L CNN
@@
 AR Path="/61E87E93/61EF422C/61E9FA3A" Ref="#PWR0192"  Part="1"
 AR Path="/61E87E93/61EF42FB/61E9FA3A" Ref="#PWR0194"  Part="1"
-F 0 "#PWR0194" H 4650 2900 50  0001 C CNN
+F 0 "#PWR0188" H 4650 2900 50  0001 C CNN
 F 1 "GND" H 4655 2977 50  0000 C CNN
 F 2 "" H 4650 3150 50  0001 C CNN
@@
 AR Path="/61E87E93/61EF422C/61EF2CDD" Ref="#PWR0193"  Part="1"
 AR Path="/61E87E93/61EF42FB/61EF2CDD" Ref="#PWR0195"  Part="1"
-F 0 "#PWR0195" H 4650 1550 50  0001 C CNN
+F 0 "#PWR0189" H 4650 1550 50  0001 C CNN
 F 1 "+3V3" H 4665 1873 50  0000 C CNN
 F 2 "" H 4650 1700 50  0001 C CNN

Commit message: Connect PDMs, add stm32 on eps board, add bcrout current telemetry, improve spacing
Parts:
- removed D?: 1N4148, symbol Device:D
- removed Q?: IRF7458, Package_SO:SOIC-8_3.9x4.9mm_P1.27mm, symbol Transistor_FET:IRF7404
- removed Q?: 2N7002, Package_TO_SOT_SMD:SOT-23, symbol Transistor_FET:2N7002
- removed R?: 100R, symbol Device:R
- removed R? (x2): 100K, symbol Device:R
- added D?: 1N4148, symbol Device:D
- added Q?: IRF7458, Package_SO:SOIC-8_3.9x4.9mm_P1.27mm, symbol Transistor_FET:IRF7404
- added Q?: 2N7002, Package_TO_SOT_SMD:SOT-23, symbol Transistor_FET:2N7002
- added R?: 100R, symbol Device:R
- added R? (x2): 100K, symbol Device:R
Connections:
- net +3V3: now also Q?.5 (D), Q?.6 (D), Q?.7 (D), Q?.8 (D)
- net GATE: now also R?.2
- net GND: now also D?.2 (A), Q?.2 (S), R?.2
- net TELEM_VOUT: now also R?.1, R?.2
- net at R?.2, R?.2, U?.5 (V+): now also D?.1 (K), Q?.1 (S), Q?.2 (S), Q?.3 (S), R?.1
- net at R?.2: now also Q?.3 (D), Q?.4 (G)
- net at R?.1: now also Q?.1 (G), R?.1

Commit message: implement a retry timer
Parts:
- D?: value 1N4148 -> 1N4004
Changed lines of the file:
@@
 $Descr A4 11693 8268
 encoding utf-8
-Sheet 28 32
+Sheet 28 35
 Title "TJ Custom EPS"
 Date ""
@@
 AR Path="/61E87E93/61EF42FB/61F7AEBB" Ref="D?"  Part="1"
 F 0 "D?" V 4604 2630 50  0000 L CNN
-F 1 "1N4148" V 4695 2630 50  0000 L CNN
+F 1 "1N4004" V 4695 2630 50  0000 L CNN
 F 2 "" H 4650 2550 50  0001 C CNN
 F 3 "~" H 4650 2550 50  0001 C CNN
