File: ECAD/PDM3V3.sch (KiCad schematic (older format))
At the start: 12 parts

Commit message: Annotate and begin adding footprints
Parts:
- R322, R323, R324, R325, R326, R328, R329: renamed from R?; footprint (none) -> Resistor_SMD:R_0805_2012Metric
- gave numbers to parts that had none: 5

Commit message: add some more footprints
Parts:
- D40: footprint (none) -> Diode_SMD:D_SMA
Changed lines of the file:
@@
 F 0 "D43" V 4604 2630 50  0000 L CNN
 F 1 "1N4004" V 4695 2630 50  0000 L CNN
-F 2 "" H 4650 2550 50  0001 C CNN
+F 2 "Diode_SMD:D_SMA" H 4650 2550 50  0001 C CNN
 F 3 "~" H 4650 2550 50  0001 C CNN
 	1    4650 2550

Commit message: add a bunch of cap and shunt resistor footprints
Parts:
- R327: footprint (none) -> Resistor_SMD:R_2010_5025Metric
Changed lines of the file:
@@
 $Descr A4 11693 8268
 encoding utf-8
-Sheet 44 44
+Sheet 42 44
 Title "TJ Custom EPS"
 Date ""
@@
 AR Path="/61E87E93/61EF422C/61F7AEB8" Ref="Q86"  Part="1"
 AR Path="/61E87E93/61EF42FB/61F7AEB8" Ref="Q88"  Part="1"
-F 0 "Q88" H 4755 2196 50  0000 L CNN
+F 0 "Q84" H 4755 2196 50  0000 L CNN
 F 1 "IRF7458" H 4755 2105 50  0000 L CNN
 F 2 "Package_SO:SOIC-8_3.9x4.9mm_P1.27mm" H 4750 2075 50  0001 L CIN
@@
 AR Path="/61E87E93/61EF422C/61F7AEB9" Ref="Q85"  Part="1"
 AR Path="/61E87E93/61EF42FB/61F7AEB9" Ref="Q87"  Part="1"
-F 0 "Q87" H 4304 2546 50  0000 L CNN
+F 0 "Q83" H 4304 2546 50  0000 L CNN
 F 1 "2N7002" H 4304 2455 50  0000 L CNN
 F 2 "Package_TO_SOT_SMD:SOT-23" H 4300 2425 50  0001 L CIN
@@
 AR Path="/61E87E93/61EF422C/61E98108" Ref="R340"  Part="1"
 AR Path="/61E87E93/61EF42FB/61E98108" Ref="R348"  Part="1"
-F 0 "R348" H 4250 1850 50  0000 L CNN
+F 0 "R332" H 4250 1850 50  0000 L CNN
 F 1 "10K" V 4200 1850 50  0000 C CNN
 F 2 "Resistor_SMD:R_0805_2012Metric" V 4130 1850 50  0001 C CNN
@@
 AR Path="/61E87E93/61EF422C/61F7AEBB" Ref="D42"  Part="1"
 AR Path="/61E87E93/61EF42FB/61F7AEBB" Ref="D43"  Part="1"
-F 0 "D43" V 4604 2630 50  0000 L CNN
+F 0 "D41" V 4604 2630 50  0000 L CNN
 F 1 "1N4004" V 4695 2630 50  0000 L CNN
 F 2 "Diode_SMD:D_SMA" H 4650 2550 50  0001 C CNN
@@
 AR Path="/61E87E93/61EF422C/61F7AEBC" Ref="R338"  Part="1"
 AR Path="/61E87E93/61EF42FB/61F7AEBC" Ref="R346"  Part="1"
-F 0 "R346" V 3450 2500 50  0000 C CNN
+F 0 "R330" V 3450 2500 50  0000 C CNN
 F 1 "100R" V 3550 2500 50  0000 C CNN
 F 2 "Resistor_SMD:R_0805_2012Metric" V 3480 2500 50  0001 C CNN
@@
 AR Path="/61E87E93/61EF422C/61E9E045" Ref="R339"  Part="1"
 AR Path="/61E87E93/61EF42FB/61E9E045" Ref="R347"  Part="1"
-F 0 "R347" H 3850 2650 50  0000 L CNN
+F 0 "R331" H 3850 2650 50  0000 L CNN
 F 1 "10K" V 3800 2650 50  0000 C CNN
 F 2 "Resistor_SMD:R_0805_2012Metric" V 3730 2650 50  0001 C CNN
@@
 AR Path="/61E87E93/61EF422C/61E9FA3A" Ref="#PWR0192"  Part="1"
 AR Path="/61E87E93/61EF42FB/61E9FA3A" Ref="#PWR0194"  Part="1"
-F 0 "#PWR0194" H 4650 2900 50  0001 C CNN
+F 0 "#PWR0190" H 4650 2900 50  0001 C CNN
 F 1 "GND" H 4655 2977 50  0000 C CNN
 F 2 "" H 4650 3150 50  0001 C CNN
@@
 AR Path="/61E87E93/61EF422C/61EB1F38" Ref="R343"  Part="1"
 AR Path="/61E87E93/61EF42FB/61EB1F38" Ref="R351"  Part="1"
-F 0 "R351" V 5650 2350 50  0000 C CNN
+F 0 "R335" V 5650 2350 50  0000 C CNN
 F 1 "10m" V 5750 2350 50  0000 C CNN
-F 2 "" V 5680 2350 50  0001 C CNN
+F 2 "Resistor_SMD:R_2010_5025Metric" V 5680 2350 50  0001 C CNN
 F 3 "~" H 5750 2350 50  0001 C CNN
 	1    5750 2350
@@
 AR Path="/61E87E93/61EF422C/61EB1F3E" Ref="U83"  Part="1"
 AR Path="/61E87E93/61EF42FB/61EB1F3E" Ref="U84"  Part="1"
-F 0 "U84" H 6594 2896 50  0000 L CNN
+F 0 "U82" H 6594 2896 50  0000 L CNN
 F 1 "LT6106" H 6594 2805 50  0000 L CNN
 F 2 "Package_TO_SOT_SMD:SOT-23-5" H 6250 2850 50  0001 C CNN
@@
 AR Path="/61E87E93/61EF422C/61EB1F4B" Ref="R345"  Part="1"
 AR Path="/61E87E93/61EF42FB/61EB1F4B" Ref="R353"  Part="1"
-F 0 "R353" H 6600 3000 50  0000 L CNN
+F 0 "R337" H 6600 3000 50  0000 L CNN
 F 1 "2K" V 6550 2950 50  0000 L CNN
 F 2 "Resistor_SMD:R_0805_2012Metric" V 6480 3000 50  0001 C CNN
@@
 AR Path="/61E87E93/61EF422C/61EB1F51" Ref="R344"  Part="1"
 AR Path="/61E87E93/61EF42FB/61EB1F51" Ref="R352"  Part="1"
-F 0 "R352" V 5700 2950 50  0000 C CNN
+F 0 "R336" V 5700 2950 50  0000 C CNN
 F 1 "100R" V 5800 2950 50  0000 C CNN
 F 2 "Resistor_SMD:R_0805_2012Metric" V 5730 2950 50  0001 C CNN
@@
 AR Path="/61E87E93/61EF422C/61F7AEC3" Ref="R341"  Part="1"
 AR Path="/61E87E93/61EF42FB/61F7AEC3" Ref="R349"  Part="1"
-F 0 "R349" H 5150 2550 50  0000 L CNN
+F 0 "R333" H 5150 2550 50  0000 L CNN
 F 1 "100K" V 5100 2550 50  0000 C CNN
 F 2 "Resistor_SMD:R_0805_2012Metric" V 5030 2550 50  0001 C CNN
@@
 AR Path="/61E87E93/61EF422C/61F7AEC4" Ref="R342"  Part="1"
 AR Path="/61E87E93/61EF42FB/61F7AEC4" Ref="R350"  Part="1"
-F 0 "R350" H 5150 2950 50  0000 L CNN
+F 0 "R334" H 5150 2950 50  0000 L CNN
 F 1 "100K" V 5100 2950 50  0000 C CNN
 F 2 "Resistor_SMD:R_0805_2012Metric" V 5030 2950 50  0001 C CNN
@@
 AR Path="/61E87E93/61EF422C/61EF2CDD" Ref="#PWR0193"  Part="1"
 AR Path="/61E87E93/61EF42FB/61EF2CDD" Ref="#PWR0195"  Part="1"
-F 0 "#PWR0195" H 4650 1550 50  0001 C CNN
+F 0 "#PWR0191" H 4650 1550 50  0001 C CNN
 F 1 "+3V3" H 4665 1873 50  0000 C CNN
 F 2 "" H 4650 1700 50  0001 C CNN

Commit message: Update stack header pinouts and re-annotate
Parts:
- renumbered D40 to D31, Q81 to Q53, Q82 to Q54, R322 to R238, R323 to R239, R324 to R240, R325 to R241, R326 to R242, R327 to R243, R328 to R244, R329 to R245, U81 to U67
