File: ECAD/Boost-BuckMPPT.sch (KiCad schematic (older format))
At the start: 38 parts

Commit message: Add USB charge to BCR3B
Parts:
- removed U?: LTC4412xS6, Package_TO_SOT_SMD:TSOT-23-6, symbol Power_Management:LTC4412xS6
Changed lines of the file:
@@
-	1    0    0    -1
-$EndComp
-$Comp
-L Power_Management:LTC4412xS6 U?
-U 1 1 61D94799
-P 4600 -850
-F 0 "U?" H 4600 -269 50  0000 C CNN
-F 1 "LTC4412xS6" H 4600 -360 50  0000 C CNN
-F 2 "Package_TO_SOT_SMD:TSOT-23-6" H 5250 -1200 50  0001 C CNN
-F 3 "https://www.analog.com/media/en/technical-documentation/data-sheets/4412fb.pdf" H 6700 -1050 50  0001 C CNN
-	1    4600 -850
 	1    0    0    -1
 $EndComp

Commit message: Annotate and begin adding footprints
Parts:
- C52, C53, C54, C55, C56: renamed from C?; footprint (none) -> Capacitor_SMD:C_0805_2012Metric
- R123, R124, R127, R128, R129, R130, R131, R132, R133, R134, R135, R136, R138: renamed from R?; footprint (none) -> Resistor_SMD:R_0805_2012Metric
- U34: renamed from U?; footprint (none) -> Package_SO:SO-8_3.9x4.9mm_P1.27mm
- gave numbers to parts that had none: 16

Commit message: add some more footprints
Parts:
- D24, D26: footprint (none) -> Diode_SMD:D_SMA
Changed lines of the file:
@@
 F 0 "D26" H 6950 1183 50  0000 C CNN
 F 1 "CMSH3-40MA" H 6950 1274 50  0000 C CNN
-F 2 "" H 6950 1400 50  0001 C CNN
+F 2 "Diode_SMD:D_SMA" H 6950 1400 50  0001 C CNN
 F 3 "~" H 6950 1400 50  0001 C CNN
 	1    6950 1400
@@
 F 0 "D24" H 4650 3917 50  0000 C CNN
 F 1 "CMSH3-40MA" H 4650 3826 50  0000 C CNN
-F 2 "" H 4650 3700 50  0001 C CNN
+F 2 "Diode_SMD:D_SMA" H 4650 3700 50  0001 C CNN
 F 3 "~" H 4650 3700 50  0001 C CNN
 	1    4650 3700

Commit message: Add all IC footprints
Parts:
- D25: value CMDSH2-4L -> RB051MM-2Y; footprint (none) -> Diode_SMD:D_SOD-123F
Changed lines of the file:
@@
 AR Path="/61BEC565/61D120A6/61D7BBA8" Ref="D25"  Part="1"
 F 0 "D25" H 4900 4417 50  0000 C CNN
-F 1 "CMDSH2-4L" H 4900 4326 50  0000 C CNN
-F 2 "" H 4900 4200 50  0001 C CNN
+F 1 "RB051MM-2Y" H 4900 4326 50  0000 C CNN
+F 2 "Diode_SMD:D_SOD-123F" H 4900 4200 50  0001 C CNN
 F 3 "~" H 4900 4200 50  0001 C CNN
 	1    4900 4200
