File: ECAD/Heater+Thermistor.sch (KiCad schematic (older format))
At the start: 12 parts

Commit message: Annotate and begin adding footprints
Parts:
- C36: renamed from C?; footprint (none) -> Capacitor_SMD:C_0805_2012Metric
- R67, R68, R69, R70, R71, R73: renamed from R?; footprint (none) -> Resistor_SMD:R_0805_2012Metric
- gave numbers to parts that had none: 5

Commit message: Add all IC footprints
Parts:
- R72, TH5: footprint (none) -> Connector_PinHeader_2.54mm:PinHeader_1x02_P2.54mm_Vertical
Changed lines of the file:
@@
 $Descr A4 11693 8268
 encoding utf-8
-Sheet 7 44
+Sheet 9 44
 Title "TJ Custom EPS"
 Date ""
@@
 AR Path="/61BD4B7D/62045EF1/620332F7" Ref="Q26"  Part="1"
 AR Path="/61BD4B7D/6204A8C5/620332F7" Ref="Q29"  Part="1"
-F 0 "Q23" H 3955 3346 50  0000 L CNN
+F 0 "Q29" H 3955 3346 50  0000 L CNN
 F 1 "Si4186DY" H 3955 3255 50  0000 L CNN
 F 2 "Package_SO:SOIC-8_3.9x4.9mm_P1.27mm" H 3950 3200 50  0001 L CNN
@@
 AR Path="/61BD4B7D/62045EF1/620332FD" Ref="R56"  Part="1"
 AR Path="/61BD4B7D/6204A8C5/620332FD" Ref="R63"  Part="1"
-F 0 "R49" V 3200 3300 50  0000 C CNN
+F 0 "R63" V 3200 3300 50  0000 C CNN
 F 1 "100R" V 3300 3300 50  0000 C CNN
 F 2 "Resistor_SMD:R_0805_2012Metric" V 3230 3300 50  0001 C CNN
@@
 AR Path="/61BD4B7D/62045EF1/62033303" Ref="R57"  Part="1"
 AR Path="/61BD4B7D/6204A8C5/62033303" Ref="R64"  Part="1"
-F 0 "R50" H 3400 3450 50  0000 C CNN
+F 0 "R64" H 3400 3450 50  0000 C CNN
 F 1 "10K" V 3500 3450 50  0000 C CNN
 F 2 "Resistor_SMD:R_0805_2012Metric" V 3430 3450 50  0001 C CNN
@@
 AR Path="/61BD4B7D/62045EF1/62033309" Ref="R58"  Part="1"
 AR Path="/61BD4B7D/6204A8C5/62033309" Ref="R65"  Part="1"
-F 0 "R51" H 3920 2996 50  0000 L CNN
+F 0 "R65" H 3920 2996 50  0000 L CNN
 F 1 "Heater (125R)" H 3920 2905 50  0000 L CNN
-F 2 "" V 3780 2950 50  0001 C CNN
+F 2 "Connector_PinHeader_2.54mm:PinHeader_1x02_P2.54mm_Vertical" V 3780 2950 50  0001 C CNN
 F 3 "~" H 3850 2950 50  0001 C CNN
 	1    3850 2950
@@
 AR Path="/61BD4B7D/62045EF1/6203330F" Ref="Q25"  Part="1"
 AR Path="/61BD4B7D/6204A8C5/6203330F" Ref="Q28"  Part="1"
-F 0 "Q22" H 3955 2646 50  0000 L CNN
+F 0 "Q28" H 3955 2646 50  0000 L CNN
 F 1 "IRF7458" H 3955 2555 50  0000 L CNN
 F 2 "Package_SO:SOIC-8_3.9x4.9mm_P1.27mm" H 3950 2525 50  0001 L CIN
@@
 AR Path="/61BD4B7D/62045EF1/62033315" Ref="#PWR0126"  Part="1"
 AR Path="/61BD4B7D/6204A8C5/62033315" Ref="#PWR0130"  Part="1"
-F 0 "#PWR0134" H 3850 2150 50  0001 C CNN
+F 0 "#PWR0130" H 3850 2150 50  0001 C CNN
 F 1 "+5V" H 3865 2473 50  0000 C CNN
 F 2 "" H 3850 2300 50  0001 C CNN
@@
 AR Path="/61BD4B7D/62045EF1/6203331C" Ref="Q24"  Part="1"
 AR Path="/61BD4B7D/6204A8C5/6203331C" Ref="Q27"  Part="1"
-F 0 "Q21" H 3104 2846 50  0000 L CNN
+F 0 "Q27" H 3104 2846 50  0000 L CNN
 F 1 "2N7002" H 3104 2755 50  0000 L CNN
 F 2 "Package_TO_SOT_SMD:SOT-23" H 3100 2725 50  0001 L CIN
@@
 AR Path="/61BD4B7D/62045EF1/62033324" Ref="R55"  Part="1"
 AR Path="/61BD4B7D/6204A8C5/62033324" Ref="R62"  Part="1"
-F 0 "R48" H 2900 2450 50  0000 C CNN
+F 0 "R62" H 2900 2450 50  0000 C CNN
 F 1 "10K" V 3000 2450 50  0000 C CNN
 F 2 "Resistor_SMD:R_0805_2012Metric" V 2930 2450 50  0001 C CNN
@@
 AR Path="/61BD4B7D/62045EF1/6203332E" Ref="R53"  Part="1"
 AR Path="/61BD4B7D/6204A8C5/6203332E" Ref="R60"  Part="1"
-F 0 "R46" V 2350 2800 50  0000 C CNN
+F 0 "R60" V 2350 2800 50  0000 C CNN
 F 1 "100R" V 2450 2800 50  0000 C CNN
 F 2 "Resistor_SMD:R_0805_2012Metric" V 2380 2800 50  0001 C CNN
@@
 AR Path="/61BD4B7D/62045EF1/62033334" Ref="R54"  Part="1"
 AR Path="/61BD4B7D/6204A8C5/62033334" Ref="R61"  Part="1"
-F 0 "R47" H 2550 2950 50  0000 C CNN
+F 0 "R61" H 2550 2950 50  0000 C CNN
 F 1 "10K" V 2650 2950 50  0000 C CNN
 F 2 "Resistor_SMD:R_0805_2012Metric" V 2580 2950 50  0001 C CNN
@@
 AR Path="/61BD4B7D/62045EF1/62034CCA" Ref="#PWR0127"  Part="1"
 AR Path="/61BD4B7D/6204A8C5/62034CCA" Ref="#PWR0131"  Part="1"
-F 0 "#PWR0135" H 3850 3350 50  0001 C CNN
+F 0 "#PWR0131" H 3850 3350 50  0001 C CNN
 F 1 "GND" H 3855 3427 50  0000 C CNN
 F 2 "" H 3850 3600 50  0001 C CNN
@@
 AR Path="/61BD4B7D/62045EF1/62036CA9" Ref="C34"  Part="1"
 AR Path="/61BD4B7D/6204A8C5/62036CA9" Ref="C35"  Part="1"
-F 0 "C33" H 6065 3496 50  0000 L CNN
+F 0 "C35" H 6065 3496 50  0000 L CNN
 F 1 "0.1uF" H 6065 3405 50  0000 L CNN
 F 2 "Capacitor_SMD:C_0805_2012Metric" H 5988 3300 50  0001 C CNN
@@
 AR Path="/61BD4B7D/62045EF1/620379E8" Ref="R59"  Part="1"
 AR Path="/61BD4B7D/6204A8C5/620379E8" Ref="R66"  Part="1"
-F 0 "R52" H 5400 3150 50  0000 L CNN
+F 0 "R66" H 5400 3150 50  0000 L CNN
 F 1 "270K" V 5350 3050 50  0000 L CNN
 F 2 "Resistor_SMD:R_0805_2012Metric" V 5280 3150 50  0001 C CNN
@@
 AR Path="/61BD4B7D/62045EF1/62035C98" Ref="TH3"  Part="1"
 AR Path="/61BD4B7D/6204A8C5/62035C98" Ref="TH4"  Part="1"
-F 0 "TH2" H 5448 3496 50  0000 L CNN
+F 0 "TH4" H 5448 3496 50  0000 L CNN
 F 1 "100K NTC" H 5448 3405 50  0000 L CNN
-F 2 "" H 5350 3500 50  0001 C CNN
+F 2 "Connector_PinHeader_2.54mm:PinHeader_1x02_P2.54mm_Vertical" H 5350 3500 50  0001 C CNN
 F 3 "~" H 5350 3500 50  0001 C CNN
 	1    5350 3450
@@
 AR Path="/61BD4B7D/62045EF1/6203964D" Ref="#PWR0128"  Part="1"
 AR Path="/61BD4B7D/6204A8C5/6203964D" Ref="#PWR0132"  Part="1"
-F 0 "#PWR0136" H 5350 2850 50  0001 C CNN
+F 0 "#PWR0132" H 5350 2850 50  0001 C CNN
 F 1 "+3V3" H 5365 3173 50  0000 C CNN
 F 2 "" H 5350 3000 50  0001 C CNN
@@
 AR Path="/61BD4B7D/62045EF1/6203B674" Ref="#PWR0129"  Part="1"
 AR Path="/61BD4B7D/6204A8C5/6203B674" Ref="#PWR0133"  Part="1"
-F 0 "#PWR0137" H 5350 3350 50  0001 C CNN
+F 0 "#PWR0133" H 5350 3350 50  0001 C CNN
 F 1 "GND" H 5355 3427 50  0000 C CNN
 F 2 "" H 5350 3600 50  0001 C CNN
