File: ECAD/PDM12V.sch (KiCad schematic (older format))
At the start: 12 parts

Commit message: Annotate and begin adding footprints
Parts:
- R242, R243, R244, R245, R246, R248, R249: renamed from R?; footprint (none) -> Resistor_SMD:R_0805_2012Metric
- gave numbers to parts that had none: 5

Commit message: add some more footprints
Parts:
- D30: footprint (none) -> Diode_SMD:D_SMA
Changed lines of the file:
@@
 F 0 "D32" V 4604 2630 50  0000 L CNN
 F 1 "1N4004" V 4695 2630 50  0000 L CNN
-F 2 "" H 4650 2550 50  0001 C CNN
+F 2 "Diode_SMD:D_SMA" H 4650 2550 50  0001 C CNN
 F 3 "~" H 4650 2550 50  0001 C CNN
 	1    4650 2550

Commit message: Add all IC footprints
Changed lines of the file:
@@
 $Descr A4 11693 8268
 encoding utf-8
-Sheet 33 44
+Sheet 31 44
 Title "TJ Custom EPS"
 Date ""
@@
 AR Path="/61E87E93/61EE5674/61E8B663" Ref="Q66"  Part="1"
 AR Path="/61E87E93/61EE57E7/61E8B663" Ref="Q?"  Part="1"
-F 0 "Q66" H 4755 2196 50  0000 L CNN
+F 0 "Q62" H 4755 2196 50  0000 L CNN
 F 1 "IRF7458" H 4755 2105 50  0000 L CNN
 F 2 "Package_SO:SOIC-8_3.9x4.9mm_P1.27mm" H 4750 2075 50  0001 L CIN
@@
 AR Path="/61E87E93/61EE5674/61E8DB1F" Ref="Q65"  Part="1"
 AR Path="/61E87E93/61EE57E7/61E8DB1F" Ref="Q?"  Part="1"
-F 0 "Q65" H 4304 2546 50  0000 L CNN
+F 0 "Q61" H 4304 2546 50  0000 L CNN
 F 1 "2N7002" H 4304 2455 50  0000 L CNN
 F 2 "Package_TO_SOT_SMD:SOT-23" H 4300 2425 50  0001 L CIN
@@
 AR Path="/61E87E93/61EE5674/61F7AEBA" Ref="R260"  Part="1"
 AR Path="/61E87E93/61EE57E7/61F7AEBA" Ref="R?"  Part="1"
-F 0 "R260" H 4250 1850 50  0000 L CNN
+F 0 "R244" H 4250 1850 50  0000 L CNN
 F 1 "10K" V 4200 1850 50  0000 C CNN
 F 2 "Resistor_SMD:R_0805_2012Metric" V 4130 1850 50  0001 C CNN
@@
 AR Path="/61E87E93/61EE5674/61EEB9E1" Ref="D32"  Part="1"
 AR Path="/61E87E93/61EE57E7/61EEB9E1" Ref="D?"  Part="1"
-F 0 "D32" V 4604 2630 50  0000 L CNN
+F 0 "D30" V 4604 2630 50  0000 L CNN
 F 1 "1N4004" V 4695 2630 50  0000 L CNN
 F 2 "Diode_SMD:D_SMA" H 4650 2550 50  0001 C CNN
@@
 AR Path="/61E87E93/61EE5674/61E9D23B" Ref="R258"  Part="1"
 AR Path="/61E87E93/61EE57E7/61E9D23B" Ref="R?"  Part="1"
-F 0 "R258" V 3450 2500 50  0000 C CNN
+F 0 "R242" V 3450 2500 50  0000 C CNN
 F 1 "100R" V 3550 2500 50  0000 C CNN
 F 2 "Resistor_SMD:R_0805_2012Metric" V 3480 2500 50  0001 C CNN
@@
 AR Path="/61E87E93/61EE5674/61F7AEBD" Ref="R259"  Part="1"
 AR Path="/61E87E93/61EE57E7/61F7AEBD" Ref="R?"  Part="1"
-F 0 "R259" H 3850 2650 50  0000 L CNN
+F 0 "R243" H 3850 2650 50  0000 L CNN
 F 1 "10K" V 3800 2650 50  0000 C CNN
 F 2 "Resistor_SMD:R_0805_2012Metric" V 3730 2650 50  0001 C CNN
@@
 AR Path="/61E87E93/61EE5674/61EF1EBB" Ref="R263"  Part="1"
 AR Path="/61E87E93/61EE57E7/61EF1EBB" Ref="R?"  Part="1"
-F 0 "R263" V 5650 2350 50  0000 C CNN
+F 0 "R247" V 5650 2350 50  0000 C CNN
 F 1 "10m" V 5750 2350 50  0000 C CNN
 F 2 "" V 5680 2350 50  0001 C CNN
@@
 AR Path="/61E87E93/61EE5674/61EEB9E6" Ref="U73"  Part="1"
 AR Path="/61E87E93/61EE57E7/61EEB9E6" Ref="U?"  Part="1"
-F 0 "U73" H 6594 2896 50  0000 L CNN
+F 0 "U71" H 6594 2896 50  0000 L CNN
 F 1 "LT6106" H 6594 2805 50  0000 L CNN
 F 2 "Package_TO_SOT_SMD:SOT-23-5" H 6250 2850 50  0001 C CNN
@@
 AR Path="/61E87E93/61EE5674/61EEB9E7" Ref="R265"  Part="1"
 AR Path="/61E87E93/61EE57E7/61EEB9E7" Ref="R?"  Part="1"
-F 0 "R265" H 6600 3000 50  0000 L CNN
+F 0 "R249" H 6600 3000 50  0000 L CNN
 F 1 "2K" V 6550 2950 50  0000 L CNN
 F 2 "Resistor_SMD:R_0805_2012Metric" V 6480 3000 50  0001 C CNN
@@
 AR Path="/61E87E93/61EE5674/61EEB9E8" Ref="R264"  Part="1"
 AR Path="/61E87E93/61EE57E7/61EEB9E8" Ref="R?"  Part="1"
-F 0 "R264" V 5700 2950 50  0000 C CNN
+F 0 "R248" V 5700 2950 50  0000 C CNN
 F 1 "100R" V 5800 2950 50  0000 C CNN
 F 2 "Resistor_SMD:R_0805_2012Metric" V 5730 2950 50  0001 C CNN
@@
 AR Path="/61E87E93/61EE5674/61EEB9E9" Ref="R261"  Part="1"
 AR Path="/61E87E93/61EE57E7/61EEB9E9" Ref="R?"  Part="1"
-F 0 "R261" H 5150 2550 50  0000 L CNN
+F 0 "R245" H 5150 2550 50  0000 L CNN
 F 1 "400K" V 5100 2550 50  0000 C CNN
 F 2 "Resistor_SMD:R_0805_2012Metric" V 5030 2550 50  0001 C CNN
@@
 AR Path="/61E87E93/61EE5674/61EC73C7" Ref="R262"  Part="1"
 AR Path="/61E87E93/61EE57E7/61EC73C7" Ref="R?"  Part="1"
-F 0 "R262" H 5150 2950 50  0000 L CNN
+F 0 "R246" H 5150 2950 50  0000 L CNN
 F 1 "100K" V 5100 2950 50  0000 C CNN
 F 2 "Resistor_SMD:R_0805_2012Metric" V 5030 2950 50  0001 C CNN

Commit message: add a bunch of cap and shunt resistor footprints
Parts:
- R247: footprint (none) -> Resistor_SMD:R_2010_5025Metric
Changed lines of the file:
@@
 $Descr A4 11693 8268
 encoding utf-8
-Sheet 31 44
+Sheet 33 44
 Title "TJ Custom EPS"
 Date ""
@@
 AR Path="/61E87E93/61EE5674/61E8B663" Ref="Q66"  Part="1"
 AR Path="/61E87E93/61EE57E7/61E8B663" Ref="Q?"  Part="1"
-F 0 "Q62" H 4755 2196 50  0000 L CNN
+F 0 "Q66" H 4755 2196 50  0000 L CNN
 F 1 "IRF7458" H 4755 2105 50  0000 L CNN
 F 2 "Package_SO:SOIC-8_3.9x4.9mm_P1.27mm" H 4750 2075 50  0001 L CIN
@@
 AR Path="/61E87E93/61EE5674/61E8DB1F" Ref="Q65"  Part="1"
 AR Path="/61E87E93/61EE57E7/61E8DB1F" Ref="Q?"  Part="1"
-F 0 "Q61" H 4304 2546 50  0000 L CNN
+F 0 "Q65" H 4304 2546 50  0000 L CNN
 F 1 "2N7002" H 4304 2455 50  0000 L CNN
 F 2 "Package_TO_SOT_SMD:SOT-23" H 4300 2425 50  0001 L CIN
@@
 AR Path="/61E87E93/61EE5674/61F7AEBA" Ref="R260"  Part="1"
 AR Path="/61E87E93/61EE57E7/61F7AEBA" Ref="R?"  Part="1"
-F 0 "R244" H 4250 1850 50  0000 L CNN
+F 0 "R260" H 4250 1850 50  0000 L CNN
 F 1 "10K" V 4200 1850 50  0000 C CNN
 F 2 "Resistor_SMD:R_0805_2012Metric" V 4130 1850 50  0001 C CNN
@@
 AR Path="/61E87E93/61EE5674/61EEB9E1" Ref="D32"  Part="1"
 AR Path="/61E87E93/61EE57E7/61EEB9E1" Ref="D?"  Part="1"
-F 0 "D30" V 4604 2630 50  0000 L CNN
+F 0 "D32" V 4604 2630 50  0000 L CNN
 F 1 "1N4004" V 4695 2630 50  0000 L CNN
 F 2 "Diode_SMD:D_SMA" H 4650 2550 50  0001 C CNN
@@
 AR Path="/61E87E93/61EE5674/61E9D23B" Ref="R258"  Part="1"
 AR Path="/61E87E93/61EE57E7/61E9D23B" Ref="R?"  Part="1"
-F 0 "R242" V 3450 2500 50  0000 C CNN
+F 0 "R258" V 3450 2500 50  0000 C CNN
 F 1 "100R" V 3550 2500 50  0000 C CNN
 F 2 "Resistor_SMD:R_0805_2012Metric" V 3480 2500 50  0001 C CNN
@@
 AR Path="/61E87E93/61EE5674/61F7AEBD" Ref="R259"  Part="1"
 AR Path="/61E87E93/61EE57E7/61F7AEBD" Ref="R?"  Part="1"
-F 0 "R243" H 3850 2650 50  0000 L CNN
+F 0 "R259" H 3850 2650 50  0000 L CNN
 F 1 "10K" V 3800 2650 50  0000 C CNN
 F 2 "Resistor_SMD:R_0805_2012Metric" V 3730 2650 50  0001 C CNN
@@
 AR Path="/61E87E93/61EE5674/61EF1EBB" Ref="R263"  Part="1"
 AR Path="/61E87E93/61EE57E7/61EF1EBB" Ref="R?"  Part="1"
-F 0 "R247" V 5650 2350 50  0000 C CNN
+F 0 "R263" V 5650 2350 50  0000 C CNN
 F 1 "10m" V 5750 2350 50  0000 C CNN
-F 2 "" V 5680 2350 50  0001 C CNN
+F 2 "Resistor_SMD:R_2010_5025Metric" V 5680 2350 50  0001 C CNN
 F 3 "~" H 5750 2350 50  0001 C CNN
 	1    5750 2350
@@
 AR Path="/61E87E93/61EE5674/61EEB9E6" Ref="U73"  Part="1"
 AR Path="/61E87E93/61EE57E7/61EEB9E6" Ref="U?"  Part="1"
-F 0 "U71" H 6594 2896 50  0000 L CNN
+F 0 "U73" H 6594 2896 50  0000 L CNN
 F 1 "LT6106" H 6594 2805 50  0000 L CNN
 F 2 "Package_TO_SOT_SMD:SOT-23-5" H 6250 2850 50  0001 C CNN
@@
 AR Path="/61E87E93/61EE5674/61EEB9E7" Ref="R265"  Part="1"
 AR Path="/61E87E93/61EE57E7/61EEB9E7" Ref="R?"  Part="1"
-F 0 "R249" H 6600 3000 50  0000 L CNN
+F 0 "R265" H 6600 3000 50  0000 L CNN
 F 1 "2K" V 6550 2950 50  0000 L CNN
 F 2 "Resistor_SMD:R_0805_2012Metric" V 6480 3000 50  0001 C CNN
@@
 AR Path="/61E87E93/61EE5674/61EEB9E8" Ref="R264"  Part="1"
 AR Path="/61E87E93/61EE57E7/61EEB9E8" Ref="R?"  Part="1"
-F 0 "R248" V 5700 2950 50  0000 C CNN
+F 0 "R264" V 5700 2950 50  0000 C CNN
 F 1 "100R" V 5800 2950 50  0000 C CNN
 F 2 "Resistor_SMD:R_0805_2012Metric" V 5730 2950 50  0001 C CNN
@@
 AR Path="/61E87E93/61EE5674/61EEB9E9" Ref="R261"  Part="1"
 AR Path="/61E87E93/61EE57E7/61EEB9E9" Ref="R?"  Part="1"
-F 0 "R245" H 5150 2550 50  0000 L CNN
+F 0 "R261" H 5150 2550 50  0000 L CNN
 F 1 "400K" V 5100 2550 50  0000 C CNN
 F 2 "Resistor_SMD:R_0805_2012Metric" V 5030 2550 50  0001 C CNN
@@
 AR Path="/61E87E93/61EE5674/61EC73C7" Ref="R262"  Part="1"
 AR Path="/61E87E93/61EE57E7/61EC73C7" Ref="R?"  Part="1"
-F 0 "R246" H 5150 2950 50  0000 L CNN
+F 0 "R262" H 5150 2950 50  0000 L CNN
 F 1 "100K" V 5100 2950 50  0000 C CNN
 F 2 "Resistor_SMD:R_0805_2012Metric" V 5030 2950 50  0001 C CNN
