File: ECAD/PDM5V.sch (KiCad schematic (older format))
At the start: 12 parts

Commit message: Annotate and begin adding footprints
Parts:
- R290, R291, R292, R293, R294, R296, R297: renamed from R?; footprint (none) -> Resistor_SMD:R_0805_2012Metric
- gave numbers to parts that had none: 5

Commit message: add some more footprints
Parts:
- D36: footprint (none) -> Diode_SMD:D_SMA
Changed lines of the file:
@@
 F 0 "D39" V 4604 2630 50  0000 L CNN
 F 1 "1N4004" V 4695 2630 50  0000 L CNN
-F 2 "" H 4650 2550 50  0001 C CNN
+F 2 "Diode_SMD:D_SMA" H 4650 2550 50  0001 C CNN
 F 3 "~" H 4650 2550 50  0001 C CNN
 	1    4650 2550

Commit message: add a bunch of cap and shunt resistor footprints
Parts:
- R295: footprint (none) -> Resistor_SMD:R_2010_5025Metric
Changed lines of the file:
@@
 F 0 "R319" V 5650 2350 50  0000 C CNN
 F 1 "10m" V 5750 2350 50  0000 C CNN
-F 2 "" V 5680 2350 50  0001 C CNN
+F 2 "Resistor_SMD:R_2010_5025Metric" V 5680 2350 50  0001 C CNN
 F 3 "~" H 5750 2350 50  0001 C CNN
 	1    5750 2350

Commit message: Update stack header pinouts and re-annotate
Parts:
- renumbered D36 to D35, Q73 to Q61, Q74 to Q62, R290 to R270, R291 to R271, R292 to R272, R293 to R273, R294 to R274, R295 to R275, R296 to R276, R297 to R277, U77 to U71
