File: ECAD/PDMBATV.sch (KiCad schematic (older format))
At the start: 12 parts

Commit message: Annotate and begin adding footprints
Parts:
- R266, R267, R268, R269, R270, R272, R273: renamed from R?; footprint (none) -> Resistor_SMD:R_0805_2012Metric
- gave numbers to parts that had none: 5
Changed lines of the file:
@@
 $Descr A4 11693 8268
 encoding utf-8
-Sheet 34 44
+Sheet 36 44
 Title "TJ Custom EPS"
 Date ""
@@
 AR Path="/61E87E93/61EE54AF/61EEB9DE" Ref="Q?"  Part="1"
 AR Path="/61E87E93/61EE5674/61EEB9DE" Ref="Q?"  Part="1"
-AR Path="/61E87E93/61EE57E7/61EEB9DE" Ref="Q?"  Part="1"
-AR Path="/61E87E93/61EE7EE1/61EEB9DE" Ref="Q?"  Part="1"
-AR Path="/61E87E93/61EE7FDA/61EEB9DE" Ref="Q?"  Part="1"
+AR Path="/61E87E93/61EE57E7/61EEB9DE" Ref="Q68"  Part="1"
+AR Path="/61E87E93/61EE7EE1/61EEB9DE" Ref="Q70"  Part="1"
+AR Path="/61E87E93/61EE7FDA/61EEB9DE" Ref="Q72"  Part="1"
 AR Path="/61E87E93/61EEB97A/61EEB9DE" Ref="Q?"  Part="1"
-F 0 "Q?" H 4755 2196 50  0000 L CNN
+F 0 "Q72" H 4755 2196 50  0000 L CNN
 F 1 "IRF7458" H 4755 2105 50  0000 L CNN
 F 2 "Package_SO:SOIC-8_3.9x4.9mm_P1.27mm" H 4750 2075 50  0001 L CIN
@@
 AR Path="/61E87E93/61EE54AF/61EEB9DF" Ref="Q?"  Part="1"
 AR Path="/61E87E93/61EE5674/61EEB9DF" Ref="Q?"  Part="1"
-AR Path="/61E87E93/61EE57E7/61EEB9DF" Ref="Q?"  Part="1"
-AR Path="/61E87E93/61EE7EE1/61EEB9DF" Ref="Q?"  Part="1"
-AR Path="/61E87E93/61EE7FDA/61EEB9DF" Ref="Q?"  Part="1"
+AR Path="/61E87E93/61EE57E7/61EEB9DF" Ref="Q67"  Part="1"
+AR Path="/61E87E93/61EE7EE1/61EEB9DF" Ref="Q69"  Part="1"
+AR Path="/61E87E93/61EE7FDA/61EEB9DF" Ref="Q71"  Part="1"
 AR Path="/61E87E93/61EEB97A/61EEB9DF" Ref="Q?"  Part="1"
-F 0 "Q?" H 4304 2546 50  0000 L CNN
+F 0 "Q71" H 4304 2546 50  0000 L CNN
 F 1 "2N7002" H 4304 2455 50  0000 L CNN
 F 2 "Package_TO_SOT_SMD:SOT-23" H 4300 2425 50  0001 L CIN
@@
 AR Path="/61E87E93/61EE54AF/61EEB9E0" Ref="R?"  Part="1"
 AR Path="/61E87E93/61EE5674/61EEB9E0" Ref="R?"  Part="1"
-AR Path="/61E87E93/61EE57E7/61EEB9E0" Ref="R?"  Part="1"
-AR Path="/61E87E93/61EE7EE1/61EEB9E0" Ref="R?"  Part="1"
-AR Path="/61E87E93/61EE7FDA/61EEB9E0" Ref="R?"  Part="1"
+AR Path="/61E87E93/61EE57E7/61EEB9E0" Ref="R268"  Part="1"
+AR Path="/61E87E93/61EE7EE1/61EEB9E0" Ref="R276"  Part="1"
+AR Path="/61E87E93/61EE7FDA/61EEB9E0" Ref="R284"  Part="1"
 AR Path="/61E87E93/61EEB97A/61EEB9E0" Ref="R?"  Part="1"
-F 0 "R?" H 4250 1850 50  0000 L CNN
+F 0 "R284" H 4250 1850 50  0000 L CNN
 F 1 "10K" V 4200 1850 50  0000 C CNN
-F 2 "" V 4130 1850 50  0001 C CNN
+F 2 "Resistor_SMD:R_0805_2012Metric" V 4130 1850 50  0001 C CNN
 F 3 "~" H 4200 1850 50  0001 C CNN
 	1    4200 1850
@@
 AR Path="/61E87E93/61EE54AF/61E99672" Ref="D?"  Part="1"
 AR Path="/61E87E93/61EE5674/61E99672" Ref="D?"  Part="1"
-AR Path="/61E87E93/61EE57E7/61E99672" Ref="D?"  Part="1"
-AR Path="/61E87E93/61EE7EE1/61E99672" Ref="D?"  Part="1"
-AR Path="/61E87E93/61EE7FDA/61E99672" Ref="D?"  Part="1"
+AR Path="/61E87E93/61EE57E7/61E99672" Ref="D33"  Part="1"
+AR Path="/61E87E93/61EE7EE1/61E99672" Ref="D34"  Part="1"
+AR Path="/61E87E93/61EE7FDA/61E99672" Ref="D35"  Part="1"
 AR Path="/61E87E93/61EEB97A/61E99672" Ref="D?"  Part="1"
-F 0 "D?" V 4604 2630 50  0000 L CNN
+F 0 "D35" V 4604 2630 50  0000 L CNN
 F 1 "1N4004" V 4695 2630 50  0000 L CNN
 F 2 "" H 4650 2550 50  0001 C CNN
@@
 AR Path="/61E87E93/61EE54AF/61EEB9E2" Ref="R?"  Part="1"
 AR Path="/61E87E93/61EE5674/61EEB9E2" Ref="R?"  Part="1"
-AR Path="/61E87E93/61EE57E7/61EEB9E2" Ref="R?"  Part="1"
-AR Path="/61E87E93/61EE7EE1/61EEB9E2" Ref="R?"  Part="1"
-AR Path="/61E87E93/61EE7FDA/61EEB9E2" Ref="R?"  Part="1"
+AR Path="/61E87E93/61EE57E7/61EEB9E2" Ref="R266"  Part="1"
+AR Path="/61E87E93/61EE7EE1/61EEB9E2" Ref="R274"  Part="1"
+AR Path="/61E87E93/61EE7FDA/61EEB9E2" Ref="R282"  Part="1"
 AR Path="/61E87E93/61EEB97A/61EEB9E2" Ref="R?"  Part="1"
-F 0 "R?" V 3450 2500 50  0000 C CNN
+F 0 "R282" V 3450 2500 50  0000 C CNN
 F 1 "100R" V 3550 2500 50  0000 C CNN
-F 2 "" V 3480 2500 50  0001 C CNN
+F 2 "Resistor_SMD:R_0805_2012Metric" V 3480 2500 50  0001 C CNN
 F 3 "~" H 3550 2500 50  0001 C CNN
 	1    3550 2500
@@
 AR Path="/61E87E93/61EE54AF/61EEB9E3" Ref="R?"  Part="1"
 AR Path="/61E87E93/61EE5674/61EEB9E3" Ref="R?"  Part="1"
-AR Path="/61E87E93/61EE57E7/61EEB9E3" Ref="R?"  Part="1"
-AR Path="/61E87E93/61EE7EE1/61EEB9E3" Ref="R?"  Part="1"
-AR Path="/61E87E93/61EE7FDA/61EEB9E3" Ref="R?"  Part="1"
+AR Path="/61E87E93/61EE57E7/61EEB9E3" Ref="R267"  Part="1"
+AR Path="/61E87E93/61EE7EE1/61EEB9E3" Ref="R275"  Part="1"
+AR Path="/61E87E93/61EE7FDA/61EEB9E3" Ref="R283"  Part="1"
 AR Path="/61E87E93/61EEB97A/61EEB9E3" Ref="R?"  Part="1"
-F 0 "R?" H 3850 2650 50  0000 L CNN
+F 0 "R283" H 3850 2650 50  0000 L CNN
 F 1 "10K" V 3800 2650 50  0000 C CNN
-F 2 "" V 3730 2650 50  0001 C CNN
+F 2 "Resistor_SMD:R_0805_2012Metric" V 3730 2650 50  0001 C CNN
 F 3 "~" H 3800 2650 50  0001 C CNN
 	1    3800 2650
@@
 AR Path="/61E87E93/61EE7FDA/61EEB9E4" Ref="#PWR0178"  Part="1"
 AR Path="/61E87E93/61EEB97A/61EEB9E4" Ref="#PWR?"  Part="1"
-F 0 "#PWR0174" H 4650 2900 50  0001 C CNN
+F 0 "#PWR0178" H 4650 2900 50  0001 C CNN
 F 1 "GND" H 4655 2977 50  0000 C CNN
 F 2 "" H 4650 3150 50  0001 C CNN
@@
 AR Path="/61E87E93/61EE54AF/61EEB9E5" Ref="R?"  Part="1"
 AR Path="/61E87E93/61EE5674/61EEB9E5" Ref="R?"  Part="1"
-AR Path="/61E87E93/61EE57E7/61EEB9E5" Ref="R?"  Part="1"
-AR Path="/61E87E93/61EE7EE1/61EEB9E5" Ref="R?"  Part="1"
-AR Path="/61E87E93/61EE7FDA/61EEB9E5" Ref="R?"  Part="1"
+AR Path="/61E87E93/61EE57E7/61EEB9E5" Ref="R271"  Part="1"
+AR Path="/61E87E93/61EE7EE1/61EEB9E5" Ref="R279"  Part="1"
+AR Path="/61E87E93/61EE7FDA/61EEB9E5" Ref="R287"  Part="1"
 AR Path="/61E87E93/61EEB97A/61EEB9E5" Ref="R?"  Part="1"
-F 0 "R?" V 5650 2350 50  0000 C CNN
+F 0 "R287" V 5650 2350 50  0000 C CNN
 F 1 "10m" V 5750 2350 50  0000 C CNN
 F 2 "" V 5680 2350 50  0001 C CNN
@@
 AR Path="/61E87E93/61EE54AF/61EF1EBC" Ref="U?"  Part="1"
 AR Path="/61E87E93/61EE5674/61EF1EBC" Ref="U?"  Part="1"
-AR Path="/61E87E93/61EE57E7/61EF1EBC" Ref="U?"  Part="1"
-AR Path="/61E87E93/61EE7EE1/61EF1EBC" Ref="U?"  Part="1"
-AR Path="/61E87E93/61EE7FDA/61EF1EBC" Ref="U?"  Part="1"
+AR Path="/61E87E93/61EE57E7/61EF1EBC" Ref="U74"  Part="1"
+AR Path="/61E87E93/61EE7EE1/61EF1EBC" Ref="U75"  Part="1"
+AR Path="/61E87E93/61EE7FDA/61EF1EBC" Ref="U76"  Part="1"
 AR Path="/61E87E93/61EEB97A/61EF1EBC" Ref="U?"  Part="1"
-F 0 "U?" H 6594 2896 50  0000 L CNN
+F 0 "U76" H 6594 2896 50  0000 L CNN
 F 1 "LT6106" H 6594 2805 50  0000 L CNN
 F 2 "Package_TO_SOT_SMD:SOT-23-5" H 6250 2850 50  0001 C CNN
@@
 AR Path="/61E87E93/61EE54AF/61EF1EBD" Ref="R?"  Part="1"
 AR Path="/61E87E93/61EE5674/61EF1EBD" Ref="R?"  Part="1"
-AR Path="/61E87E93/61EE57E7/61EF1EBD" Ref="R?"  Part="1"
-AR Path="/61E87E93/61EE7EE1/61EF1EBD" Ref="R?"  Part="1"
-AR Path="/61E87E93/61EE7FDA/61EF1EBD" Ref="R?"  Part="1"
+AR Path="/61E87E93/61EE57E7/61EF1EBD" Ref="R273"  Part="1"
+AR Path="/61E87E93/61EE7EE1/61EF1EBD" Ref="R281"  Part="1"
+AR Path="/61E87E93/61EE7FDA/61EF1EBD" Ref="R289"  Part="1"
 AR Path="/61E87E93/61EEB97A/61EF1EBD" Ref="R?"  Part="1"
-F 0 "R?" H 6600 3000 50  0000 L CNN
+F 0 "R289" H 6600 3000 50  0000 L CNN
 F 1 "2K" V 6550 2950 50  0000 L CNN
-F 2 "" V 6480 3000 50  0001 C CNN
+F 2 "Resistor_SMD:R_0805_2012Metric" V 6480 3000 50  0001 C CNN
 F 3 "~" H 6550 3000 50  0001 C CNN
 	1    6550 3000
@@
 AR Path="/61E87E93/61EE54AF/61F7AEC2" Ref="R?"  Part="1"
 AR Path="/61E87E93/61EE5674/61F7AEC2" Ref="R?"  Part="1"
-AR Path="/61E87E93/61EE57E7/61F7AEC2" Ref="R?"  Part="1"
-AR Path="/61E87E93/61EE7EE1/61F7AEC2" Ref="R?"  Part="1"
-AR Path="/61E87E93/61EE7FDA/61F7AEC2" Ref="R?"  Part="1"
+AR Path="/61E87E93/61EE57E7/61F7AEC2" Ref="R272"  Part="1"
+AR Path="/61E87E93/61EE7EE1/61F7AEC2" Ref="R280"  Part="1"
+AR Path="/61E87E93/61EE7FDA/61F7AEC2" Ref="R288"  Part="1"
 AR Path="/61E87E93/61EEB97A/61F7AEC2" Ref="R?"  Part="1"
-F 0 "R?" V 5700 2950 50  0000 C CNN
+F 0 "R288" V 5700 2950 50  0000 C CNN
 F 1 "100R" V 5800 2950 50  0000 C CNN
-F 2 "" V 5730 2950 50  0001 C CNN
+F 2 "Resistor_SMD:R_0805_2012Metric" V 5730 2950 50  0001 C CNN
 F 3 "~" H 5800 2950 50  0001 C CNN
 	1    5800 2950
@@
 AR Path="/61E87E93/61EE54AF/61EC6843" Ref="R?"  Part="1"
 AR Path="/61E87E93/61EE5674/61EC6843" Ref="R?"  Part="1"
-AR Path="/61E87E93/61EE57E7/61EC6843" Ref="R?"  Part="1"
-AR Path="/61E87E93/61EE7EE1/61EC6843" Ref="R?"  Part="1"
-AR Path="/61E87E93/61EE7FDA/61EC6843" Ref="R?"  Part="1"
+AR Path="/61E87E93/61EE57E7/61EC6843" Ref="R269"  Part="1"
+AR Path="/61E87E93/61EE7EE1/61EC6843" Ref="R277"  Part="1"
+AR Path="/61E87E93/61EE7FDA/61EC6843" Ref="R285"  Part="1"
 AR Path="/61E87E93/61EEB97A/61EC6843" Ref="R?"  Part="1"
-F 0 "R?" H 5150 2550 50  0000 L CNN
+F 0 "R285" H 5150 2550 50  0000 L CNN
 F 1 "200K" V 5100 2550 50  0000 C CNN
-F 2 "" V 5030 2550 50  0001 C CNN
+F 2 "Resistor_SMD:R_0805_2012Metric" V 5030 2550 50  0001 C CNN
 F 3 "~" H 5100 2550 50  0001 C CNN
 	1    5100 2550
@@
 AR Path="/61E87E93/61EE54AF/61EEB9EA" Ref="R?"  Part="1"
 AR Path="/61E87E93/61EE5674/61EEB9EA" Ref="R?"  Part="1"
-AR Path="/61E87E93/61EE57E7/61EEB9EA" Ref="R?"  Part="1"
-AR Path="/61E87E93/61EE7EE1/61EEB9EA" Ref="R?"  Part="1"
-AR Path="/61E87E93/61EE7FDA/61EEB9EA" Ref="R?"  Part="1"
+AR Path="/61E87E93/61EE57E7/61EEB9EA" Ref="R270"  Part="1"
+AR Path="/61E87E93/61EE7EE1/61EEB9EA" Ref="R278"  Part="1"
+AR Path="/61E87E93/61EE7FDA/61EEB9EA" Ref="R286"  Part="1"
 AR Path="/61E87E93/61EEB97A/61EEB9EA" Ref="R?"  Part="1"
-F 0 "R?" H 5150 2950 50  0000 L CNN
+F 0 "R286" H 5150 2950 50  0000 L CNN
 F 1 "100K" V 5100 2950 50  0000 C CNN
-F 2 "" V 5030 2950 50  0001 C CNN
+F 2 "Resistor_SMD:R_0805_2012Metric" V 5030 2950 50  0001 C CNN
 F 3 "~" H 5100 2950 50  0001 C CNN
 	1    5100 2950
@@
 AR Path="/61E87E93/61EE7FDA/61EEA4DE" Ref="#PWR0179"  Part="1"
 AR Path="/61E87E93/61EEB97A/61EEA4DE" Ref="#PWR?"  Part="1"
-F 0 "#PWR0175" H 4650 1550 50  0001 C CNN
+F 0 "#PWR0179" H 4650 1550 50  0001 C CNN
 F 1 "+BATT" H 4665 1873 50  0000 C CNN
 F 2 "" H 4650 1700 50  0001 C CNN

Commit message: add some more footprints
Parts:
- D33: footprint (none) -> Diode_SMD:D_SMA
Changed lines of the file:
@@
 F 0 "D35" V 4604 2630 50  0000 L CNN
 F 1 "1N4004" V 4695 2630 50  0000 L CNN
-F 2 "" H 4650 2550 50  0001 C CNN
+F 2 "Diode_SMD:D_SMA" H 4650 2550 50  0001 C CNN
 F 3 "~" H 4650 2550 50  0001 C CNN
 	1    4650 2550

Commit message: add a bunch of cap and shunt resistor footprints
Parts:
- R271: footprint (none) -> Resistor_SMD:R_2010_5025Metric
Changed lines of the file:
@@
 F 0 "R287" V 5650 2350 50  0000 C CNN
 F 1 "10m" V 5750 2350 50  0000 C CNN
-F 2 "" V 5680 2350 50  0001 C CNN
+F 2 "Resistor_SMD:R_2010_5025Metric" V 5680 2350 50  0001 C CNN
 F 3 "~" H 5750 2350 50  0001 C CNN
 	1    5750 2350

Commit message: Major descope, remove 12V boost and all related circuitry
Changed lines of the file:
@@
 $Descr A4 11693 8268
 encoding utf-8
-Sheet 36 44
+Sheet 36 37
 Title "TJ Custom EPS"
 Date ""
@@
 AR Path="/61E87E93/61EE7FDA/61EEB9DE" Ref="Q72"  Part="1"
 AR Path="/61E87E93/61EEB97A/61EEB9DE" Ref="Q?"  Part="1"
-F 0 "Q72" H 4755 2196 50  0000 L CNN
+AR Path="/61E87E93/61EB04DF/61EEB9DE" Ref="Q?"  Part="1"
+F 0 "Q?" H 4755 2196 50  0000 L CNN
 F 1 "IRF7458" H 4755 2105 50  0000 L CNN
 F 2 "Package_SO:SOIC-8_3.9x4.9mm_P1.27mm" H 4750 2075 50  0001 L CIN
@@
 AR Path="/61E87E93/61EE7FDA/61EEB9DF" Ref="Q71"  Part="1"
 AR Path="/61E87E93/61EEB97A/61EEB9DF" Ref="Q?"  Part="1"
-F 0 "Q71" H 4304 2546 50  0000 L CNN
+AR Path="/61E87E93/61EB04DF/61EEB9DF" Ref="Q?"  Part="1"
+F 0 "Q?" H 4304 2546 50  0000 L CNN
 F 1 "2N7002" H 4304 2455 50  0000 L CNN
 F 2 "Package_TO_SOT_SMD:SOT-23" H 4300 2425 50  0001 L CIN
@@
 AR Path="/61E87E93/61EE7FDA/61EEB9E0" Ref="R284"  Part="1"
 AR Path="/61E87E93/61EEB97A/61EEB9E0" Ref="R?"  Part="1"
-F 0 "R284" H 4250 1850 50  0000 L CNN
+AR Path="/61E87E93/61EB04DF/61EEB9E0" Ref="R?"  Part="1"
+F 0 "R?" H 4250 1850 50  0000 L CNN
 F 1 "10K" V 4200 1850 50  0000 C CNN
 F 2 "Resistor_SMD:R_0805_2012Metric" V 4130 1850 50  0001 C CNN
@@
 AR Path="/61E87E93/61EE7FDA/61E99672" Ref="D35"  Part="1"
 AR Path="/61E87E93/61EEB97A/61E99672" Ref="D?"  Part="1"
-F 0 "D35" V 4604 2630 50  0000 L CNN
+AR Path="/61E87E93/61EB04DF/61E99672" Ref="D?"  Part="1"
+F 0 "D?" V 4604 2630 50  0000 L CNN
 F 1 "1N4004" V 4695 2630 50  0000 L CNN
 F 2 "Diode_SMD:D_SMA" H 4650 2550 50  0001 C CNN
@@
 AR Path="/61E87E93/61EE7FDA/61EEB9E2" Ref="R282"  Part="1"
 AR Path="/61E87E93/61EEB97A/61EEB9E2" Ref="R?"  Part="1"
-F 0 "R282" V 3450 2500 50  0000 C CNN
+AR Path="/61E87E93/61EB04DF/61EEB9E2" Ref="R?"  Part="1"
+F 0 "R?" V 3450 2500 50  0000 C CNN
 F 1 "100R" V 3550 2500 50  0000 C CNN
 F 2 "Resistor_SMD:R_0805_2012Metric" V 3480 2500 50  0001 C CNN
@@
 AR Path="/61E87E93/61EE7FDA/61EEB9E3" Ref="R283"  Part="1"
 AR Path="/61E87E93/61EEB97A/61EEB9E3" Ref="R?"  Part="1"
-F 0 "R283" H 3850 2650 50  0000 L CNN
+AR Path="/61E87E93/61EB04DF/61EEB9E3" Ref="R?"  Part="1"
+F 0 "R?" H 3850 2650 50  0000 L CNN
 F 1 "10K" V 3800 2650 50  0000 C CNN
 F 2 "Resistor_SMD:R_0805_2012Metric" V 3730 2650 50  0001 C CNN
@@
 AR Path="/61E87E93/61EE7FDA/61EEB9E4" Ref="#PWR0178"  Part="1"
 AR Path="/61E87E93/61EEB97A/61EEB9E4" Ref="#PWR?"  Part="1"
-F 0 "#PWR0178" H 4650 2900 50  0001 C CNN
+AR Path="/61E87E93/61EB04DF/61EEB9E4" Ref="#PWR?"  Part="1"
+F 0 "#PWR?" H 4650 2900 50  0001 C CNN
 F 1 "GND" H 4655 2977 50  0000 C CNN
 F 2 "" H 4650 3150 50  0001 C CNN
@@
 AR Path="/61E87E93/61EE7FDA/61EEB9E5" Ref="R287"  Part="1"
 AR Path="/61E87E93/61EEB97A/61EEB9E5" Ref="R?"  Part="1"
-F 0 "R287" V 5650 2350 50  0000 C CNN
+AR Path="/61E87E93/61EB04DF/61EEB9E5" Ref="R?"  Part="1"
+F 0 "R?" V 5650 2350 50  0000 C CNN
 F 1 "10m" V 5750 2350 50  0000 C CNN
 F 2 "Resistor_SMD:R_2010_5025Metric" V 5680 2350 50  0001 C CNN
@@
 AR Path="/61E87E93/61EE7FDA/61EF1EBC" Ref="U76"  Part="1"
 AR Path="/61E87E93/61EEB97A/61EF1EBC" Ref="U?"  Part="1"
-F 0 "U76" H 6594 2896 50  0000 L CNN
+AR Path="/61E87E93/61EB04DF/61EF1EBC" Ref="U?"  Part="1"
+F 0 "U?" H 6594 2896 50  0000 L CNN
 F 1 "LT6106" H 6594 2805 50  0000 L CNN
 F 2 "Package_TO_SOT_SMD:SOT-23-5" H 6250 2850 50  0001 C CNN
@@
 AR Path="/61E87E93/61EE7FDA/61EF1EBD" Ref="R289"  Part="1"
 AR Path="/61E87E93/61EEB97A/61EF1EBD" Ref="R?"  Part="1"
-F 0 "R289" H 6600 3000 50  0000 L CNN
+AR Path="/61E87E93/61EB04DF/61EF1EBD" Ref="R?"  Part="1"
+F 0 "R?" H 6600 3000 50  0000 L CNN
 F 1 "2K" V 6550 2950 50  0000 L CNN
 F 2 "Resistor_SMD:R_0805_2012Metric" V 6480 3000 50  0001 C CNN
@@
 AR Path="/61E87E93/61EE7FDA/61F7AEC2" Ref="R288"  Part="1"
 AR Path="/61E87E93/61EEB97A/61F7AEC2" Ref="R?"  Part="1"
-F 0 "R288" V 5700 2950 50  0000 C CNN
+AR Path="/61E87E93/61EB04DF/61F7AEC2" Ref="R?"  Part="1"
+F 0 "R?" V 5700 2950 50  0000 C CNN
 F 1 "100R" V 5800 2950 50  0000 C CNN
 F 2 "Resistor_SMD:R_0805_2012Metric" V 5730 2950 50  0001 C CNN
@@
 AR Path="/61E87E93/61EE7FDA/61EC6843" Ref="R285"  Part="1"
 AR Path="/61E87E93/61EEB97A/61EC6843" Ref="R?"  Part="1"
-F 0 "R285" H 5150 2550 50  0000 L CNN
+AR Path="/61E87E93/61EB04DF/61EC6843" Ref="R?"  Part="1"
+F 0 "R?" H 5150 2550 50  0000 L CNN
 F 1 "200K" V 5100 2550 50  0000 C CNN
 F 2 "Resistor_SMD:R_0805_2012Metric" V 5030 2550 50  0001 C CNN
@@
 AR Path="/61E87E93/61EE7FDA/61EEB9EA" Ref="R286"  Part="1"
 AR Path="/61E87E93/61EEB97A/61EEB9EA" Ref="R?"  Part="1"
-F 0 "R286" H 5150 2950 50  0000 L CNN
+AR Path="/61E87E93/61EB04DF/61EEB9EA" Ref="R?"  Part="1"
+F 0 "R?" H 5150 2950 50  0000 L CNN
 F 1 "100K" V 5100 2950 50  0000 C CNN
 F 2 "Resistor_SMD:R_0805_2012Metric" V 5030 2950 50  0001 C CNN
@@
 AR Path="/61E87E93/61EE7FDA/61EEA4DE" Ref="#PWR0179"  Part="1"
 AR Path="/61E87E93/61EEB97A/61EEA4DE" Ref="#PWR?"  Part="1"
-F 0 "#PWR0179" H 4650 1550 50  0001 C CNN
+AR Path="/61E87E93/61EB04DF/61EEA4DE" Ref="#PWR?"  Part="1"
+F 0 "#PWR?" H 4650 1550 50  0001 C CNN
 F 1 "+BATT" H 4665 1873 50  0000 C CNN
 F 2 "" H 4650 1700 50  0001 C CNN

Commit message: Update stack header pinouts and re-annotate
Parts:
- renumbered D33 to D38, R266 to R294, R267 to R295, R268 to R296, R269 to R297, R270 to R298, R271 to R299, R272 to R300, R273 to R301
