File: ECAD/Pulse+RetryTimer.sch (KiCad schematic (older format))
At the start: 13 parts

Commit message: Annotate and begin adding footprints
Parts:
- C100, C105: renamed from C?; footprint (none) -> Capacitor_SMD:C_0805_2012Metric
- R214, R215, R216, R231, R232, R233, R234: renamed from R?; footprint (none) -> Resistor_SMD:R_0805_2012Metric
- gave numbers to parts that had none: 4

Commit message: Add all IC footprints
Changed lines of the file:
@@
 $Descr A4 11693 8268
 encoding utf-8
-Sheet 29 44
+Sheet 26 44
 Title "TJ Custom EPS"
 Date ""
@@
 AR Path="/61C9425D/6278B84C/61DD6209" Ref="#PWR0235"  Part="1"
 AR Path="/61C9425D/6286FCFD/61DD6209" Ref="#PWR0239"  Part="1"
-F 0 "#PWR0239" H 2950 1000 50  0001 C CNN
+F 0 "#PWR0227" H 2950 1000 50  0001 C CNN
 F 1 "VCC" H 2965 1323 50  0000 C CNN
 F 2 "" H 2950 1150 50  0001 C CNN
@@
 AR Path="/61C9425D/6278B84C/61DE485D" Ref="R228"  Part="1"
 AR Path="/61C9425D/6286FCFD/61DE485D" Ref="R235"  Part="1"
-F 0 "R235" H 2150 1300 50  0000 L CNN
+F 0 "R214" H 2150 1300 50  0000 L CNN
 F 1 "2.5M" V 2100 1300 50  0000 C CNN
 F 2 "Resistor_SMD:R_0805_2012Metric" V 2030 1300 50  0001 C CNN
@@
 AR Path="/61C9425D/6278B84C/61DEA269" Ref="C104"  Part="1"
 AR Path="/61C9425D/6286FCFD/61DEA269" Ref="C106"  Part="1"
-F 0 "C106" H 2215 1746 50  0000 L CNN
+F 0 "C100" H 2215 1746 50  0000 L CNN
 F 1 "22uF" H 2215 1655 50  0000 L CNN
 F 2 "Capacitor_SMD:C_0805_2012Metric" H 2138 1550 50  0001 C CNN
@@
 AR Path="/61C9425D/6278B84C/61E036B5" Ref="#PWR0236"  Part="1"
 AR Path="/61C9425D/6286FCFD/61E036B5" Ref="#PWR0240"  Part="1"
-F 0 "#PWR0240" H 2950 1800 50  0001 C CNN
+F 0 "#PWR0228" H 2950 1800 50  0001 C CNN
 F 1 "GND" H 2955 1877 50  0000 C CNN
 F 2 "" H 2950 2050 50  0001 C CNN
@@
 AR Path="/61C9425D/6278B84C/61D5F929" Ref="Q57"  Part="1"
 AR Path="/61C9425D/6286FCFD/61D5F929" Ref="Q59"  Part="1"
-F 0 "Q59" H 1704 1746 50  0000 L CNN
+F 0 "Q53" H 1704 1746 50  0000 L CNN
 F 1 "2N7002" H 1704 1655 50  0000 L CNN
 F 2 "Package_TO_SOT_SMD:SOT-23" H 1700 1625 50  0001 L CIN
@@
 AR Path="/61C9425D/6278B84C/61D6733E" Ref="U63"  Part="1"
 AR Path="/61C9425D/6286FCFD/61D6733E" Ref="U65"  Part="1"
-F 0 "U65" H 3394 1646 50  0000 L CNN
+F 0 "U59" H 3394 1646 50  0000 L CNN
 F 1 "AD8603" H 3394 1555 50  0000 L CNN
 F 2 "Package_TO_SOT_SMD:TSOT-23-5" H 3050 1600 50  0001 C CNN
@@
 AR Path="/61C9425D/6278B84C/61D73526" Ref="Q58"  Part="1"
 AR Path="/61C9425D/6286FCFD/61D73526" Ref="Q60"  Part="1"
-F 0 "Q60" H 4104 1646 50  0000 L CNN
+F 0 "Q54" H 4104 1646 50  0000 L CNN
 F 1 "2N7002" H 4104 1555 50  0000 L CNN
 F 2 "Package_TO_SOT_SMD:SOT-23" H 4100 1525 50  0001 L CIN
@@
 AR Path="/61C9425D/6278B84C/61D792CF" Ref="R229"  Part="1"
 AR Path="/61C9425D/6286FCFD/61D792CF" Ref="R236"  Part="1"
-F 0 "R236" H 2500 1300 50  0000 L CNN
+F 0 "R215" H 2500 1300 50  0000 L CNN
 F 1 "10K" V 2450 1300 50  0000 C CNN
 F 2 "Resistor_SMD:R_0805_2012Metric" V 2380 1300 50  0001 C CNN
@@
 AR Path="/61C9425D/6278B84C/61D79DBB" Ref="R230"  Part="1"
 AR Path="/61C9425D/6286FCFD/61D79DBB" Ref="R237"  Part="1"
-F 0 "R237" H 2500 1900 50  0000 L CNN
+F 0 "R216" H 2500 1900 50  0000 L CNN
 F 1 "20K" V 2450 1900 50  0000 C CNN
 F 2 "Resistor_SMD:R_0805_2012Metric" V 2380 1900 50  0001 C CNN
@@
 AR Path="/61C9425D/62734C35/628E3A19" Ref="U62"  Part="1"
 AR Path="/61C9425D/6286FCFD/628E3A19" Ref="U66"  Part="1"
-F 0 "U66" H 6600 1800 50  0000 L CNN
+F 0 "U60" H 6600 1800 50  0000 L CNN
 F 1 "LTC6993xS6-4" H 6600 1600 50  0000 L CNN
 F 2 "Package_TO_SOT_SMD:TSOT-23-6" H 6350 1300 50  0001 C CNN
@@
 AR Path="/61C9425D/62734C35/628E3A1F" Ref="#PWR0233"  Part="1"
 AR Path="/61C9425D/6286FCFD/628E3A1F" Ref="#PWR0241"  Part="1"
-F 0 "#PWR0241" H 6350 1150 50  0001 C CNN
+F 0 "#PWR0229" H 6350 1150 50  0001 C CNN
 F 1 "VCC" H 6365 1473 50  0000 C CNN
 F 2 "" H 6350 1300 50  0001 C CNN
@@
 AR Path="/61C9425D/62734C35/628E3A25" Ref="R225"  Part="1"
 AR Path="/61C9425D/6286FCFD/628E3A25" Ref="R239"  Part="1"
-F 0 "R239" H 5700 1900 50  0000 L CNN
+F 0 "R218" H 5700 1900 50  0000 L CNN
 F 1 "1K" V 5650 1900 50  0000 C CNN
 F 2 "Resistor_SMD:R_0805_2012Metric" V 5580 1900 50  0001 C CNN
@@
 AR Path="/61C9425D/62734C35/628E3A2B" Ref="R224"  Part="1"
 AR Path="/61C9425D/6286FCFD/628E3A2B" Ref="R238"  Part="1"
-F 0 "R238" H 5700 1450 50  0000 L CNN
+F 0 "R217" H 5700 1450 50  0000 L CNN
 F 1 "523R" V 5650 1450 50  0000 C CNN
 F 2 "Resistor_SMD:R_0805_2012Metric" V 5580 1450 50  0001 C CNN
@@
 AR Path="/61C9425D/62734C35/628E3A39" Ref="R227"  Part="1"
 AR Path="/61C9425D/6286FCFD/628E3A39" Ref="R241"  Part="1"
-F 0 "R241" H 6000 1950 50  0000 L CNN
+F 0 "R220" H 6000 1950 50  0000 L CNN
 F 1 "760K" V 5950 1950 50  0000 C CNN
 F 2 "Resistor_SMD:R_0805_2012Metric" V 5880 1950 50  0001 C CNN
@@
 AR Path="/61C9425D/62734C35/628E3A41" Ref="C103"  Part="1"
 AR Path="/61C9425D/6286FCFD/628E3A41" Ref="C107"  Part="1"
-F 0 "C107" H 5315 1496 50  0000 L CNN
+F 0 "C101" H 5315 1496 50  0000 L CNN
 F 1 "0.1uF" H 5315 1405 50  0000 L CNN
 F 2 "Capacitor_SMD:C_0805_2012Metric" H 5238 1300 50  0001 C CNN
@@
 AR Path="/61C9425D/62734C35/628E3A4F" Ref="R226"  Part="1"
 AR Path="/61C9425D/6286FCFD/628E3A4F" Ref="R240"  Part="1"
-F 0 "R240" H 5900 1500 50  0000 L CNN
+F 0 "R219" H 5900 1500 50  0000 L CNN
 F 1 "10K" V 5850 1500 50  0000 C CNN
 F 2 "Resistor_SMD:R_0805_2012Metric" V 5780 1500 50  0001 C CNN
@@
 AR Path="/61C9425D/6278B84C/628E8E71" Ref="#PWR0238"  Part="1"
 AR Path="/61C9425D/6286FCFD/628E8E71" Ref="#PWR0242"  Part="1"
-F 0 "#PWR0242" H 6350 1850 50  0001 C CNN
+F 0 "#PWR0230" H 6350 1850 50  0001 C CNN
 F 1 "GND" H 6355 1927 50  0000 C CNN
 F 2 "" H 6350 2100 50  0001 C CNN

Commit message: Update stack header pinouts and re-annotate
Parts:
- renumbered C100 to C87, C105 to C90, Q53 to Q41, Q54 to Q42, R214 to R193, R215 to R194, R216 to R195, R231 to R203, R232 to R204, R233 to R205, R234 to R206, U59 to U54, U64 to U57
