File: ECAD/PowerDistribution.sch (KiCad schematic (older format))
At the start: 0 parts

Commit message: add amux
Parts:
- added U? (x2): CD74HC4067SM, Package_SO:SSOP-24_5.3x8.2mm_P0.65mm, symbol 74xx:CD74HC4067SM
Connections:
- net TELEM_ISW1: now also U?.9 (I0)
- net TELEM_ISW10: now also U?.22 (I9)
- net TELEM_ISW11: now also U?.21 (I10)
- net TELEM_ISW12: now also U?.20 (I11)
- net TELEM_ISW13: now also U?.19 (I12)
- net TELEM_ISW14: now also U?.18 (I13)
- net TELEM_ISW2: now also U?.8 (I1)
- net TELEM_ISW3: now also U?.7 (I2)
- net TELEM_ISW4: now also U?.6 (I3)
- net TELEM_ISW5: now also U?.5 (I4)
- net TELEM_ISW6: now also U?.4 (I5)
- net TELEM_ISW7: now also U?.3 (I6)
- net TELEM_ISW8: now also U?.2 (I7)
- net TELEM_ISW9: now also U?.23 (I8)
- net TELEM_VSW1: now also U?.9 (I0)
- net TELEM_VSW10: now also U?.22 (I9)
- net TELEM_VSW11: now also U?.21 (I10)
- net TELEM_VSW12: now also U?.20 (I11)
- net TELEM_VSW13: now also U?.19 (I12)
- net TELEM_VSW14: now also U?.18 (I13)
- net TELEM_VSW2: now also U?.8 (I1)
- net TELEM_VSW3: now also U?.7 (I2)
- net TELEM_VSW4: now also U?.6 (I3)
- net TELEM_VSW5: now also U?.5 (I4)
- net TELEM_VSW6: now also U?.4 (I5)
- net TELEM_VSW7: now also U?.3 (I6)
- net TELEM_VSW8: now also U?.2 (I7)
- net TELEM_VSW9: now also U?.23 (I8)
- new net MUX2OUT: U?.1 (COM)
- new net MUX3OUT: U?.1 (COM)
Changed lines of the file:
@@
 $Descr A4 11693 8268
 encoding utf-8
-Sheet 21 44
+Sheet 30 44
 Title "TJ Custom EPS"
 Date ""
@@
 Text Notes 1500 4400 0    50   ~ 0
 3.3V PDMs
+$Comp
+L 74xx:CD74HC4067SM U?
+U 1 1 61D9F1B4
+P 3400 6150
+AR Path="/61D9F1B4" Ref="U?"  Part="1"
+AR Path="/61E87E93/61D9F1B4" Ref="U?"  Part="1"
+F 0 "U?" H 3400 7331 50  0000 C CNN
+F 1 "CD74HC4067SM" H 3400 7240 50  0000 C CNN
+F 2 "Package_SO:SSOP-24_5.3x8.2mm_P0.65mm" H 4450 5150 50  0001 C CIN
+F 3 "http://www.ti.com/lit/ds/symlink/cd74hc4067.pdf" H 3050 7000 50  0001 C CNN
+	1    3400 6150
+	-1   0    0    -1
+$EndComp
+Text GLabel 2900 5450 0    50   Input ~ 0
+TELEM_VSW1
+Text GLabel 2900 5550 0    50   Input ~ 0
+TELEM_VSW2
+Text GLabel 2900 5650 0    50   Input ~ 0
+TELEM_VSW3
+Text GLabel 2900 5750 0    50   Input ~ 0
+TELEM_VSW4
+Text GLabel 2900 5850 0    50   Input ~ 0
+TELEM_VSW5
+Text GLabel 2900 5950 0    50   Input ~ 0
+TELEM_VSW6
+Text GLabel 2900 6050 0    50   Input ~ 0
+TELEM_VSW7
+Text GLabel 2900 6150 0    50   Input ~ 0
+TELEM_VSW8
+Text GLabel 2900 6250 0    50   Input ~ 0
+TELEM_VSW9
+Text GLabel 2900 6350 0    50   Input ~ 0
+TELEM_VSW10
+Text GLabel 2900 6450 0    50   Input ~ 0
+TELEM_VSW11
+Text GLabel 2900 6550 0    50   Input ~ 0
+TELEM_VSW12
+Text GLabel 2900 6650 0    50   Input ~ 0
+TELEM_VSW13
+Text GLabel 2900 6750 0    50   Input ~ 0
+TELEM_VSW14
+$Comp
+L 74xx:CD74HC4067SM U?
+U 1 1 61DC574F
+P 5850 6150
+AR Path="/61DC574F" Ref="U?"  Part="1"
+AR Path="/61E87E93/61DC574F" Ref="U?"  Part="1"
+F 0 "U?" H 5850 7331 50  0000 C CNN
+F 1 "CD74HC4067SM" H 5850 7240 50  0000 C CNN
+F 2 "Package_SO:SSOP-24_5.3x8.2mm_P0.65mm" H 6900 5150 50  0001 C CIN
+F 3 "http://www.ti.com/lit/ds/symlink/cd74hc4067.pdf" H 5500 7000 50  0001 C CNN
+	1    5850 6150
+	-1   0    0    -1
+$EndComp
+Text GLabel 5350 5450 0    50   Input ~ 0
+TELEM_ISW1
+Text GLabel 5350 5550 0    50   Input ~ 0
+TELEM_ISW2
+Text GLabel 5350 5650 0    50   Input ~ 0
+TELEM_ISW3
+Text GLabel 5350 5750 0    50   Input ~ 0
+TELEM_ISW4
+Text GLabel 5350 5850 0    50   Input ~ 0
+TELEM_ISW5
+Text GLabel 5350 5950 0    50   Input ~ 0
+TELEM_ISW6
+Text GLabel 5350 6050 0    50   Input ~ 0
+TELEM_ISW7
+Text GLabel 5350 6150 0    50   Input ~ 0
+TELEM_ISW8
+Text GLabel 5350 6250 0    50   Input ~ 0
+TELEM_ISW9
+Text GLabel 5350 6350 0    50   Input ~ 0
+TELEM_ISW10
+Text GLabel 5350 6450 0    50   Input ~ 0
+TELEM_ISW11
+Text GLabel 5350 6550 0    50   Input ~ 0
+TELEM_ISW12
+Text GLabel 5350 6650 0    50   Input ~ 0
+TELEM_ISW13
+Text GLabel 5350 6750 0    50   Input ~ 0
+TELEM_ISW14
+Text GLabel 3900 5650 2    50   Input ~ 0
+MUX2OUT
+Text GLabel 6350 5650 2    50   Input ~ 0
+MUX3OUT
 $EndSCHEMATC

Commit message: connect amux
Parts:
- added C? (x2): 0.1uF, symbol Device:C
- added C? (x2): 0.01uF, symbol Device:C
- added U? (x2): 74HC595, symbol 74xx:74HC595
Connections:
- net MUX2OUT: now also C?.1
- net MUX3OUT: now also C?.1
- net S0: now reaches U?.10 (S0)
- net S0: now also U?.10 (S0)
- net S1: now reaches U?.11 (S1)
- net S1: now also U?.11 (S1)
- net GND: now reaches U?.12 (GND)
- net GND: now also U?.12 (GND), U?.15 (~E), U?.15 (~E), C?.2, C?.2, C?.2, C?.2
- net S3: now reaches U?.13 (S3)
- net S3: now also U?.13 (S3)
- net S2: now reaches U?.14 (S2)
- net S2: now also U?.14 (S2)
- net +3V3: now reaches U?.24 (VCC)
- net +3V3: now also U?.24 (VCC), C?.1, C?.1
Other:
- moved on the sheet: U?

Commit message: Add PDM control using shift registers
Parts:
- added C? (x2): 0.1uF, symbol Device:C
Connections:
- net +3V3: now also U?.10 (~SRCLR), U?.10 (~SRCLR), U?.16 (VCC), U?.16 (VCC), C?.1, C?.1
- net GND: now also U?.13 (~OE), U?.13 (~OE), U?.8 (GND), U?.8 (GND), C?.2, C?.2
- net SW1: now also U?.15 (QA)
- net SW10: now also U?.1 (QB)
- net SW11: now also U?.2 (QC)
- net SW12: now also U?.3 (QD)
- net SW13: now also U?.4 (QE)
- net SW14: now also U?.5 (QF)
- net SW2: now also U?.1 (QB)
- net SW3: now also U?.2 (QC)
- net SW4: now also U?.3 (QD)
- net SW5: now also U?.4 (QE)
- net SW6: now also U?.5 (QF)
- net SW7: now also U?.6 (QG)
- net SW8: now also U?.7 (QH)
- net SW9: now also U?.15 (QA)
- net SRCLK: now reaches U?.11 (SRCLK)
- net SRCLK: now also U?.11 (SRCLK)
- net SRLCH: now reaches U?.12 (RCLK)
- net SRLCH: now also U?.12 (RCLK)
- net SRSERIN: now reaches U?.14 (SER)
- net at U?.9 (QH'): now also U?.14 (SER)
- no-connect marks 0 -> 1
Other:
- note added: "74hc595 are rising edge clock"
- moved on the sheet: U?
Changed lines of the file:
@@
 L 74xx:74HC595 U?
 U 1 1 622C9B64
-P 8400 1900
-F 0 "U?" H 8400 2681 50  0000 C CNN
-F 1 "74HC595" H 8400 2590 50  0000 C CNN
-F 2 "" H 8400 1900 50  0001 C CNN
-F 3 "http://www.ti.com/lit/ds/symlink/sn74hc595.pdf" H 8400 1900 50  0001 C CNN
-	1    8400 1900
+P 8750 1750
+F 0 "U?" H 8750 2531 50  0000 C CNN
+F 1 "74HC595" H 8750 2440 50  0000 C CNN
+F 2 "" H 8750 1750 50  0001 C CNN
+F 3 "http://www.ti.com/lit/ds/symlink/sn74hc595.pdf" H 8750 1750 50  0001 C CNN
+	1    8750 1750
 	1    0    0    -1
 $EndComp
@@
 L 74xx:74HC595 U?
 U 1 1 622C9F3C
-P 9550 1900
-F 0 "U?" H 9550 2681 50  0000 C CNN
-F 1 "74HC595" H 9550 2590 50  0000 C CNN
-F 2 "" H 9550 1900 50  0001 C CNN
-F 3 "http://www.ti.com/lit/ds/symlink/sn74hc595.pdf" H 9550 1900 50  0001 C CNN
-	1    9550 1900
+P 10500 1750
+F 0 "U?" H 10500 2531 50  0000 C CNN
+F 1 "74HC595" H 10500 2440 50  0000 C CNN
+F 2 "" H 10500 1750 50  0001 C CNN
+F 3 "http://www.ti.com/lit/ds/symlink/sn74hc595.pdf" H 10500 1750 50  0001 C CNN
+	1    10500 1750
 	1    0    0    -1
 $EndComp
@@
 	5400 7300 5200 7300
 Connection ~ 5200 7300
+$Comp
+L power:+3V3 #PWR?
+U 1 1 61DA7D11
+P 9550 1150
+AR Path="/61DA7D11" Ref="#PWR?"  Part="1"
+AR Path="/61BD4B7D/61DA7D11" Ref="#PWR?"  Part="1"
+AR Path="/61E87E93/61DA7D11" Ref="#PWR?"  Part="1"
+F 0 "#PWR?" H 9550 1000 50  0001 C CNN
+F 1 "+3V3" V 9565 1278 50  0000 L CNN
+F 2 "" H 9550 1150 50  0001 C CNN
+F 3 "" H 9550 1150 50  0001 C CNN
+	1    9550 1150
+	1    0    0    -1
+$EndComp
+$Comp
+L power:GND #PWR?
+U 1 1 61DA8643
+P 9550 2450
+AR Path="/61DA8643" Ref="#PWR?"  Part="1"
+AR Path="/61BD4B7D/61DA8643" Ref="#PWR?"  Part="1"
+AR Path="/61E87E93/61DA8643" Ref="#PWR?"  Part="1"
+F 0 "#PWR?" H 9550 2200 50  0001 C CNN
+F 1 "GND" H 9555 2277 50  0000 C CNN
+F 2 "" H 9550 2450 50  0001 C CNN
+F 3 "" H 9550 2450 50  0001 C CNN
+	1    9550 2450
+	1    0    0    -1
+$EndComp
+$Comp
+L Device:C C?
+U 1 1 61DA8C08
+P 9550 1300
+F 0 "C?" H 9665 1346 50  0000 L CNN
+F 1 "0.1uF" H 9665 1255 50  0000 L CNN
+F 2 "" H 9588 1150 50  0001 C CNN
+F 3 "~" H 9550 1300 50  0001 C CNN
+	1    9550 1300
+	1    0    0    -1
+$EndComp
+$Comp
+L Device:C C?
+U 1 1 61DA9C99
+P 7750 1300
+F 0 "C?" H 7865 1346 50  0000 L CNN
+F 1 "0.1uF" H 7865 1255 50  0000 L CNN
+F 2 "" H 7788 1150 50  0001 C CNN
+F 3 "~" H 7750 1300 50  0001 C CNN
+	1    7750 1300
+	1    0    0    -1
+$EndComp
+Wire Wire Line
+	10500 1150 10000 1150
+Connection ~ 8750 1150
+Wire Wire Line
+	8750 1150 8250 1150
+Wire Wire Line
+	7750 1450 7750 2450
+Wire Wire Line
+	8750 2450 9550 2450
+Connection ~ 8750 2450
+Wire Wire Line
+	8350 1650 8250 1650
+Wire Wire Line
+	8250 1650 8250 1150
+Connection ~ 8250 1150
+Wire Wire Line
+	10100 1650 10000 1650
+Wire Wire Line
+	10000 1650 10000 1150
+Connection ~ 10000 1150
+Wire Wire Line
+	8350 1950 8250 1950
+Text Notes 8600 700  0    50   ~ 0
+74hc595 are rising edge clock
+Wire Wire Line
+	10050 1350 10050 2250
+Wire Wire Line
+	10100 1950 10000 1950
+Wire Wire Line
+	10000 1950 10000 2450
+Connection ~ 10000 2450
+Wire Wire Line
+	10000 2450 10500 2450
+Wire Wire Line
+	8250 1950 8250 2450
+Connection ~ 8250 2450
+Wire Wire Line
+	8250 2450 8750 2450
+Wire Wire Line
+	10050 1350 10100 1350
+Wire Wire Line
+	9150 2250 10050 2250
+Wire Wire Line
+	8350 1350 8350 1050
+Wire Wire Line
+	8350 1050 8050 1050
+Wire Wire Line
+	8350 1850 8200 1850
+Wire Wire Line
+	8350 1550 8200 1550
+Wire Wire Line
+	10100 1550 9950 1550
+Wire Wire Line
+	10100 1850 9950 1850
+Text GLabel 8200 1550 0    50   Input ~ 0
+SRCLK
+Text GLabel 9950 1550 0    50   Input ~ 0
+SRCLK
+Text GLabel 8200 1850 0    50   Input ~ 0
+SRLCH
+Text GLabel 9950 1850 0    50   Input ~ 0
+SRLCH
+Text GLabel 8050 1050 0    50   Input ~ 0
+SRSERIN
+Text GLabel 9150 1350 2    50   Input ~ 0
+SW1
+Text GLabel 9150 1450 2    50   Input ~ 0
+SW2
+Text GLabel 9150 1550 2    50   Input ~ 0
+SW3
+Text GLabel 9150 1650 2    50   Input ~ 0
+SW4
+Text GLabel 9150 1750 2    50   Input ~ 0
+SW5
+Text GLabel 9150 1850 2    50   Input ~ 0
+SW6
+Text GLabel 9150 1950 2    50   Input ~ 0
+SW7
+Text GLabel 9150 2050 2    50   Input ~ 0
+SW8
+Text GLabel 10900 1350 2    50   Input ~ 0
+SW9
+Text GLabel 10900 1450 2    50   Input ~ 0
+SW10
+Text GLabel 10900 1550 2    50   Input ~ 0
+SW11
+Text GLabel 10900 1650 2    50   Input ~ 0
+SW12
+Text GLabel 10900 1750 2    50   Input ~ 0
+SW13
+Text GLabel 10900 1850 2    50   Input ~ 0
+SW14
+Connection ~ 9550 1150
+Wire Wire Line
+	9550 1150 8750 1150
+Connection ~ 9550 2450
+Wire Wire Line
+	9550 2450 10000 2450
+Wire Wire Line
+	9550 1450 9550 2450
+Wire Wire Line
+	9550 1150 10000 1150
+NoConn ~ 10900 2250
+Wire Wire Line
+	7750 1150 8250 1150
+Wire Wire Line
+	7750 2450 8250 2450
 $EndSCHEMATC

Commit message: Annotate and begin adding footprints
Parts:
- C108, C109, C110, C111, C112, C113: renamed from C?; footprint (none) -> Capacitor_SMD:C_0805_2012Metric
- U69, U70: renamed from U?; footprint (none) -> Package_SO:SOIC-16_3.9x9.9mm_P1.27mm
- gave numbers to parts that had none: 2
Changed lines of the file:
@@
 P 2500 6200
 AR Path="/61D9F1B4" Ref="U?"  Part="1"
-AR Path="/61E87E93/61D9F1B4" Ref="U?"  Part="1"
-F 0 "U?" H 2500 7381 50  0000 C CNN
+AR Path="/61E87E93/61D9F1B4" Ref="U67"  Part="1"
+F 0 "U67" H 2500 7381 50  0000 C CNN
 F 1 "CD74HC4067SM" H 2500 7290 50  0000 C CNN
 F 2 "Package_SO:SSOP-24_5.3x8.2mm_P0.65mm" H 3550 5200 50  0001 C CIN
@@
 P 4700 6200
 AR Path="/61DC574F" Ref="U?"  Part="1"
-AR Path="/61E87E93/61DC574F" Ref="U?"  Part="1"
-F 0 "U?" H 4700 7381 50  0000 C CNN
+AR Path="/61E87E93/61DC574F" Ref="U68"  Part="1"
+F 0 "U68" H 4700 7381 50  0000 C CNN
 F 1 "CD74HC4067SM" H 4700 7290 50  0000 C CNN
 F 2 "Package_SO:SSOP-24_5.3x8.2mm_P0.65mm" H 5750 5200 50  0001 C CIN
@@
 MUX3OUT
 $Comp
-L 74xx:74HC595 U?
+L 74xx:74HC595 U69
 U 1 1 622C9B64
 P 8750 1750
-F 0 "U?" H 8750 2531 50  0000 C CNN
+F 0 "U69" H 8750 2531 50  0000 C CNN
 F 1 "74HC595" H 8750 2440 50  0000 C CNN
-F 2 "" H 8750 1750 50  0001 C CNN
+F 2 "Package_SO:SOIC-16_3.9x9.9mm_P1.27mm" H 8750 1750 50  0001 C CNN
 F 3 "http://www.ti.com/lit/ds/symlink/sn74hc595.pdf" H 8750 1750 50  0001 C CNN
 	1    8750 1750
@@
 $EndComp
 $Comp
-L 74xx:74HC595 U?
+L 74xx:74HC595 U70
 U 1 1 622C9F3C
 P 10500 1750
-F 0 "U?" H 10500 2531 50  0000 C CNN
+F 0 "U70" H 10500 2531 50  0000 C CNN
 F 1 "74HC595" H 10500 2440 50  0000 C CNN
-F 2 "" H 10500 1750 50  0001 C CNN
+F 2 "Package_SO:SOIC-16_3.9x9.9mm_P1.27mm" H 10500 1750 50  0001 C CNN
 F 3 "http://www.ti.com/lit/ds/symlink/sn74hc595.pdf" H 10500 1750 50  0001 C CNN
 	1    10500 1750
@@
 AR Path="/62361C29" Ref="#PWR?"  Part="1"
 AR Path="/61BD4B7D/62361C29" Ref="#PWR?"  Part="1"
-AR Path="/61E87E93/62361C29" Ref="#PWR?"  Part="1"
-F 0 "#PWR?" H 3600 5050 50  0001 C CNN
+AR Path="/61E87E93/62361C29" Ref="#PWR0243"  Part="1"
+F 0 "#PWR0243" H 3600 5050 50  0001 C CNN
 F 1 "+3V3" V 3615 5328 50  0000 L CNN
 F 2 "" H 3600 5200 50  0001 C CNN
@@
 AR Path="/62361C33" Ref="#PWR?"  Part="1"
 AR Path="/61BD4B7D/62361C33" Ref="#PWR?"  Part="1"
-AR Path="/61E87E93/62361C33" Ref="#PWR?"  Part="1"
-F 0 "#PWR?" H 3600 7050 50  0001 C CNN
+AR Path="/61E87E93/62361C33" Ref="#PWR0244"  Part="1"
+F 0 "#PWR0244" H 3600 7050 50  0001 C CNN
 F 1 "GND" H 3605 7127 50  0000 C CNN
 F 2 "" H 3600 7300 50  0001 C CNN
@@
 AR Path="/61BD4B7D/62361C3B" Ref="C?"  Part="1"
 AR Path="/62361C3B" Ref="C?"  Part="1"
-AR Path="/61E87E93/62361C3B" Ref="C?"  Part="1"
-F 0 "C?" H 3715 5396 50  0000 L CNN
+AR Path="/61E87E93/62361C3B" Ref="C110"  Part="1"
+F 0 "C110" H 3715 5396 50  0000 L CNN
 F 1 "0.1uF" H 3715 5305 50  0000 L CNN
-F 2 "" H 3638 5200 50  0001 C CNN
+F 2 "Capacitor_SMD:C_0805_2012Metric" H 3638 5200 50  0001 C CNN
 F 3 "~" H 3600 5350 50  0001 C CNN
 	1    3600 5350
@@
 AR Path="/61BD4B7D/6236CC02" Ref="C?"  Part="1"
 AR Path="/6236CC02" Ref="C?"  Part="1"
-AR Path="/61E87E93/6236CC02" Ref="C?"  Part="1"
-F 0 "C?" H 1515 5396 50  0000 L CNN
+AR Path="/61E87E93/6236CC02" Ref="C108"  Part="1"
+F 0 "C108" H 1515 5396 50  0000 L CNN
 F 1 "0.1uF" H 1515 5305 50  0000 L CNN
-F 2 "" H 1438 5200 50  0001 C CNN
+F 2 "Capacitor_SMD:C_0805_2012Metric" H 1438 5200 50  0001 C CNN
 F 3 "~" H 1400 5350 50  0001 C CNN
 	1    1400 5350
@@
 AR Path="/61BD4B7D/623E18AC" Ref="C?"  Part="1"
 AR Path="/623E18AC" Ref="C?"  Part="1"
-AR Path="/61E87E93/623E18AC" Ref="C?"  Part="1"
-F 0 "C?" H 3315 5896 50  0000 L CNN
+AR Path="/61E87E93/623E18AC" Ref="C109"  Part="1"
+F 0 "C109" H 3315 5896 50  0000 L CNN
 F 1 "0.01uF" H 3315 5805 50  0000 L CNN
-F 2 "" H 3238 5700 50  0001 C CNN
+F 2 "Capacitor_SMD:C_0805_2012Metric" H 3238 5700 50  0001 C CNN
 F 3 "~" H 3200 5850 50  0001 C CNN
 	1    3200 5850
@@
 AR Path="/61BD4B7D/623E402C" Ref="C?"  Part="1"
 AR Path="/623E402C" Ref="C?"  Part="1"
-AR Path="/61E87E93/623E402C" Ref="C?"  Part="1"
-F 0 "C?" H 5515 5896 50  0000 L CNN
+AR Path="/61E87E93/623E402C" Ref="C111"  Part="1"
+F 0 "C111" H 5515 5896 50  0000 L CNN
 F 1 "0.01uF" H 5515 5805 50  0000 L CNN
-F 2 "" H 5438 5700 50  0001 C CNN
+F 2 "Capacitor_SMD:C_0805_2012Metric" H 5438 5700 50  0001 C CNN
 F 3 "~" H 5400 5850 50  0001 C CNN
 	1    5400 5850
@@
 AR Path="/61DA7D11" Ref="#PWR?"  Part="1"
 AR Path="/61BD4B7D/61DA7D11" Ref="#PWR?"  Part="1"
-AR Path="/61E87E93/61DA7D11" Ref="#PWR?"  Part="1"
-F 0 "#PWR?" H 9550 1000 50  0001 C CNN
+AR Path="/61E87E93/61DA7D11" Ref="#PWR0245"  Part="1"
+F 0 "#PWR0245" H 9550 1000 50  0001 C CNN
 F 1 "+3V3" V 9565 1278 50  0000 L CNN
 F 2 "" H 9550 1150 50  0001 C CNN
@@
 AR Path="/61DA8643" Ref="#PWR?"  Part="1"
 AR Path="/61BD4B7D/61DA8643" Ref="#PWR?"  Part="1"
-AR Path="/61E87E93/61DA8643" Ref="#PWR?"  Part="1"
-F 0 "#PWR?" H 9550 2200 50  0001 C CNN
+AR Path="/61E87E93/61DA8643" Ref="#PWR0246"  Part="1"
+F 0 "#PWR0246" H 9550 2200 50  0001 C CNN
 F 1 "GND" H 9555 2277 50  0000 C CNN
 F 2 "" H 9550 2450 50  0001 C CNN
@@
 $EndComp
 $Comp
-L Device:C C?
+L Device:C C113
 U 1 1 61DA8C08
 P 9550 1300
-F 0 "C?" H 9665 1346 50  0000 L CNN
+F 0 "C113" H 9665 1346 50  0000 L CNN
 F 1 "0.1uF" H 9665 1255 50  0000 L CNN
-F 2 "" H 9588 1150 50  0001 C CNN
+F 2 "Capacitor_SMD:C_0805_2012Metric" H 9588 1150 50  0001 C CNN
 F 3 "~" H 9550 1300 50  0001 C CNN
 	1    9550 1300
@@
 $EndComp
 $Comp
-L Device:C C?
+L Device:C C112
 U 1 1 61DA9C99
 P 7750 1300
-F 0 "C?" H 7865 1346 50  0000 L CNN
+F 0 "C112" H 7865 1346 50  0000 L CNN
 F 1 "0.1uF" H 7865 1255 50  0000 L CNN
-F 2 "" H 7788 1150 50  0001 C CNN
+F 2 "Capacitor_SMD:C_0805_2012Metric" H 7788 1150 50  0001 C CNN
 F 3 "~" H 7750 1300 50  0001 C CNN
 	1    7750 1300

Commit message: Major descope, remove 12V boost and all related circuitry
Connections:
- net SW13: no longer names the net of U70.4 (QE)
- net SW14: no longer names the net of U70.5 (QF)
- net TELEM_ISW13: no longer names the net of U68.19 (I12)
- net TELEM_ISW14: no longer names the net of U68.18 (I13)
- net TELEM_VSW13: no longer names the net of U67.19 (I12)
- net TELEM_VSW14: no longer names the net of U67.18 (I13)
Other:
- note removed: "12V PDMs"
- moved on the sheet: C112, C113, U69, U70

Commit message: Update stack header pinouts and re-annotate
Parts:
- renumbered C108 to C93, C109 to C94, C110 to C95, C111 to C96, C112 to C97, C113 to C98, U67 to U60, U68 to U61, U69 to U62, U70 to U63
Changed lines of the file:
@@
 P 2500 6200
 AR Path="/61D9F1B4" Ref="U?"  Part="1"
-AR Path="/61E87E93/61D9F1B4" Ref="U67"  Part="1"
-F 0 "U67" H 2500 7381 50  0000 C CNN
+AR Path="/61E87E93/61D9F1B4" Ref="U60"  Part="1"
+F 0 "U60" H 2500 7381 50  0000 C CNN
 F 1 "CD74HC4067SM" H 2500 7290 50  0000 C CNN
 F 2 "Package_SO:SSOP-24_5.3x8.2mm_P0.65mm" H 3550 5200 50  0001 C CIN
@@
 P 4700 6200
 AR Path="/61DC574F" Ref="U?"  Part="1"
-AR Path="/61E87E93/61DC574F" Ref="U68"  Part="1"
-F 0 "U68" H 4700 7381 50  0000 C CNN
+AR Path="/61E87E93/61DC574F" Ref="U61"  Part="1"
+F 0 "U61" H 4700 7381 50  0000 C CNN
 F 1 "CD74HC4067SM" H 4700 7290 50  0000 C CNN
 F 2 "Package_SO:SSOP-24_5.3x8.2mm_P0.65mm" H 5750 5200 50  0001 C CIN
@@
 MUX3OUT
 $Comp
-L 74xx:74HC595 U69
+L 74xx:74HC595 U62
 U 1 1 622C9B64
 P 7750 5500
-F 0 "U69" H 7750 6281 50  0000 C CNN
+F 0 "U62" H 7750 6281 50  0000 C CNN
 F 1 "74HC595" H 7750 6190 50  0000 C CNN
 F 2 "Package_SO:SOIC-16_3.9x9.9mm_P1.27mm" H 7750 5500 50  0001 C CNN
@@
 $EndComp
 $Comp
-L 74xx:74HC595 U70
+L 74xx:74HC595 U63
 U 1 1 622C9F3C
 P 9500 5500
-F 0 "U70" H 9500 6281 50  0000 C CNN
+F 0 "U63" H 9500 6281 50  0000 C CNN
 F 1 "74HC595" H 9500 6190 50  0000 C CNN
 F 2 "Package_SO:SOIC-16_3.9x9.9mm_P1.27mm" H 9500 5500 50  0001 C CNN
@@
 AR Path="/62361C29" Ref="#PWR?"  Part="1"
 AR Path="/61BD4B7D/62361C29" Ref="#PWR?"  Part="1"
-AR Path="/61E87E93/62361C29" Ref="#PWR0243"  Part="1"
-F 0 "#PWR0243" H 3600 5050 50  0001 C CNN
+AR Path="/61E87E93/62361C29" Ref="#PWR0200"  Part="1"
+F 0 "#PWR0200" H 3600 5050 50  0001 C CNN
 F 1 "+3V3" V 3615 5328 50  0000 L CNN
 F 2 "" H 3600 5200 50  0001 C CNN
@@
 AR Path="/62361C33" Ref="#PWR?"  Part="1"
 AR Path="/61BD4B7D/62361C33" Ref="#PWR?"  Part="1"
-AR Path="/61E87E93/62361C33" Ref="#PWR0244"  Part="1"
-F 0 "#PWR0244" H 3600 7050 50  0001 C CNN
+AR Path="/61E87E93/62361C33" Ref="#PWR0201"  Part="1"
+F 0 "#PWR0201" H 3600 7050 50  0001 C CNN
 F 1 "GND" H 3605 7127 50  0000 C CNN
 F 2 "" H 3600 7300 50  0001 C CNN
@@
 AR Path="/61BD4B7D/62361C3B" Ref="C?"  Part="1"
 AR Path="/62361C3B" Ref="C?"  Part="1"
-AR Path="/61E87E93/62361C3B" Ref="C110"  Part="1"
-F 0 "C110" H 3715 5396 50  0000 L CNN
+AR Path="/61E87E93/62361C3B" Ref="C95"  Part="1"
+F 0 "C95" H 3715 5396 50  0000 L CNN
 F 1 "0.1uF" H 3715 5305 50  0000 L CNN
 F 2 "Capacitor_SMD:C_0805_2012Metric" H 3638 5200 50  0001 C CNN
@@
 AR Path="/61BD4B7D/6236CC02" Ref="C?"  Part="1"
 AR Path="/6236CC02" Ref="C?"  Part="1"
-AR Path="/61E87E93/6236CC02" Ref="C108"  Part="1"
-F 0 "C108" H 1515 5396 50  0000 L CNN
+AR Path="/61E87E93/6236CC02" Ref="C93"  Part="1"
+F 0 "C93" H 1515 5396 50  0000 L CNN
 F 1 "0.1uF" H 1515 5305 50  0000 L CNN
 F 2 "Capacitor_SMD:C_0805_2012Metric" H 1438 5200 50  0001 C CNN
@@
 AR Path="/61BD4B7D/623E18AC" Ref="C?"  Part="1"
 AR Path="/623E18AC" Ref="C?"  Part="1"
-AR Path="/61E87E93/623E18AC" Ref="C109"  Part="1"
-F 0 "C109" H 3315 5896 50  0000 L CNN
+AR Path="/61E87E93/623E18AC" Ref="C94"  Part="1"
+F 0 "C94" H 3315 5896 50  0000 L CNN
 F 1 "0.01uF" H 3315 5805 50  0000 L CNN
 F 2 "Capacitor_SMD:C_0805_2012Metric" H 3238 5700 50  0001 C CNN
@@
 AR Path="/61BD4B7D/623E402C" Ref="C?"  Part="1"
 AR Path="/623E402C" Ref="C?"  Part="1"
-AR Path="/61E87E93/623E402C" Ref="C111"  Part="1"
-F 0 "C111" H 5515 5896 50  0000 L CNN
+AR Path="/61E87E93/623E402C" Ref="C96"  Part="1"
+F 0 "C96" H 5515 5896 50  0000 L CNN
 F 1 "0.01uF" H 5515 5805 50  0000 L CNN
 F 2 "Capacitor_SMD:C_0805_2012Metric" H 5438 5700 50  0001 C CNN
@@
 AR Path="/61DA7D11" Ref="#PWR?"  Part="1"
 AR Path="/61BD4B7D/61DA7D11" Ref="#PWR?"  Part="1"
-AR Path="/61E87E93/61DA7D11" Ref="#PWR0245"  Part="1"
-F 0 "#PWR0245" H 8550 4750 50  0001 C CNN
+AR Path="/61E87E93/61DA7D11" Ref="#PWR0202"  Part="1"
+F 0 "#PWR0202" H 8550 4750 50  0001 C CNN
 F 1 "+3V3" V 8565 5028 50  0000 L CNN
 F 2 "" H 8550 4900 50  0001 C CNN
@@
 AR Path="/61DA8643" Ref="#PWR?"  Part="1"
 AR Path="/61BD4B7D/61DA8643" Ref="#PWR?"  Part="1"
-AR Path="/61E87E93/61DA8643" Ref="#PWR0246"  Part="1"
-F 0 "#PWR0246" H 8550 5950 50  0001 C CNN
+AR Path="/61E87E93/61DA8643" Ref="#PWR0203"  Part="1"
+F 0 "#PWR0203" H 8550 5950 50  0001 C CNN
 F 1 "GND" H 8555 6027 50  0000 C CNN
 F 2 "" H 8550 6200 50  0001 C CNN
@@
 $EndComp
 $Comp
-L Device:C C113
+L Device:C C98
 U 1 1 61DA8C08
 P 8550 5050
-F 0 "C113" H 8665 5096 50  0000 L CNN
+F 0 "C98" H 8665 5096 50  0000 L CNN
 F 1 "0.1uF" H 8665 5005 50  0000 L CNN
 F 2 "Capacitor_SMD:C_0805_2012Metric" H 8588 4900 50  0001 C CNN
@@
 $EndComp
 $Comp
-L Device:C C112
+L Device:C C97
 U 1 1 61DA9C99
 P 6750 5050
-F 0 "C112" H 6865 5096 50  0000 L CNN
+F 0 "C97" H 6865 5096 50  0000 L CNN
 F 1 "0.1uF" H 6865 5005 50  0000 L CNN
 F 2 "Capacitor_SMD:C_0805_2012Metric" H 6788 4900 50  0001 C CNN

Commit message: Condense muxes and add srrst
Parts:
- removed C93, C95: 0.1uF, Capacitor_SMD:C_0805_2012Metric, symbol Device:C
- removed C94, C96: 0.01uF, Capacitor_SMD:C_0805_2012Metric, symbol Device:C
- removed U60, U61: CD74HC4067SM, Package_SO:SSOP-24_5.3x8.2mm_P0.65mm, symbol 74xx:CD74HC4067SM
- added R310: 10K, symbol Device:R
Connections:
- net +3V3: now also R310.1; no longer U62.10 (~SRCLR)
- new net PDMRST: R310.2, U62.10 (~SRCLR)
Other:
- moved on the sheet: C97, C98, U62, U63
