File: ECAD/TJ-EPS.sch (KiCad schematic (older format))
At the start: 29 parts

Commit message: add amux
Parts:
- added C?: 0.1uF, symbol Device:C
- added R?: 270K, symbol Device:R
- added TH?: 100K NTC, symbol Device:Thermistor_NTC
- added U? (x2): CD74HC4067SM, Package_SO:SSOP-24_5.3x8.2mm_P0.65mm, symbol 74xx:CD74HC4067SM
- added U?: 74HC595, symbol 74xx:74HC595
Connections:
- net +3V3: now also R?.1
- net GND: now also C?.2, TH?.2
- net SOLAR_CS1: now reaches U?.22 (PB11)
- net SOLAR_CS0: now reaches U?.25 (PB12)
- net SOLAR_SCK: now reaches U?.26 (PB13)
- net SOLAR_MISO: now reaches U?.27 (PB14)
- net SOLAR_MOSI: now reaches U?.28 (PB15)
- new net I_SA1A: U?.8 (I1)
- new net I_SA1B: U?.7 (I2)
- new net I_SA2A: U?.5 (I4)
- new net I_SA2B: U?.4 (I5)
- new net I_SA3A: U?.2 (I7)
- new net I_SA3B: U?.23 (I8)
- new net I_SA4A: U?.21 (I10)
- new net I_SA4B: U?.20 (I11)
- new net MUX0OUT: U?.1 (COM)
- new net MUX1OUT: U?.1 (COM)
- new net TELEM_I12V: U?.9 (I0)
- new net TELEM_I3V3: U?.6 (I3)
- new net TELEM_I5V: U?.7 (I2)
- new net TELEM_IBATV: U?.8 (I1)
- new net TELEM_IBCROUT: U?.18 (I13)
- new net TELEM_TBRD: C?.1, R?.2, TH?.1, U?.23 (I8)
- new net TELEM_V12V: U?.5 (I4)
- new net TELEM_V3V3: U?.2 (I7)
- new net TELEM_V5V: U?.3 (I6)
- new net TELEM_VBATV: U?.4 (I5)
- new net TELEM_VBCROUT: U?.19 (I12)
- new net V_SA1: U?.9 (I0)
- new net V_SA2: U?.6 (I3)
- new net V_SA3: U?.3 (I6)
- new net V_SA4: U?.22 (I9)
Other:
- note added: "Top resistor selected for 5C center operating temperature"
Changed lines of the file:
@@
 Wire Wire Line
 	550  3050 750  3050
+$Comp
+L 74xx:CD74HC4067SM U?
+U 1 1 61D924A0
+P 4350 5850
+F 0 "U?" H 4350 7031 50  0000 C CNN
+F 1 "CD74HC4067SM" H 4350 6940 50  0000 C CNN
+F 2 "Package_SO:SSOP-24_5.3x8.2mm_P0.65mm" H 5400 4850 50  0001 C CIN
+F 3 "http://www.ti.com/lit/ds/symlink/cd74hc4067.pdf" H 4000 6700 50  0001 C CNN
+	1    4350 5850
+	-1   0    0    -1
+$EndComp
+Text GLabel 3850 5250 0    50   Input ~ 0
+I_SA1A
+Text GLabel 3850 5550 0    50   Input ~ 0
+I_SA2A
+Text GLabel 3850 5650 0    50   Input ~ 0
+I_SA2B
+Text GLabel 3850 5850 0    50   Input ~ 0
+I_SA3A
+Text GLabel 3850 5950 0    50   Input ~ 0
+I_SA3B
+Text GLabel 3850 6150 0    50   Input ~ 0
+I_SA4A
+Text GLabel 3850 6250 0    50   Input ~ 0
+I_SA4B
+Text GLabel 3850 5350 0    50   Input ~ 0
+I_SA1B
+Text GLabel 3850 5150 0    50   Input ~ 0
+V_SA1
+Text GLabel 3850 5450 0    50   Input ~ 0
+V_SA2
+Text GLabel 3850 5750 0    50   Input ~ 0
+V_SA3
+Text GLabel 3850 6050 0    50   Input ~ 0
+V_SA4
+Text GLabel 3850 6350 0    50   Input ~ 0
+TELEM_VBCROUT
+Text GLabel 3850 6450 0    50   Input ~ 0
+TELEM_IBCROUT
+Text GLabel 6000 5150 0    50   Input ~ 0
+TELEM_I12V
+Text GLabel 6000 5250 0    50   Input ~ 0
+TELEM_IBATV
+Text GLabel 6000 5350 0    50   Input ~ 0
+TELEM_I5V
+Text GLabel 6000 5450 0    50   Input ~ 0
+TELEM_I3V3
+Text GLabel 6000 5550 0    50   Input ~ 0
+TELEM_V12V
+Text GLabel 6000 5650 0    50   Input ~ 0
+TELEM_VBATV
+Text GLabel 6000 5750 0    50   Input ~ 0
+TELEM_V5V
+Text GLabel 6000 5850 0    50   Input ~ 0
+TELEM_V3V3
+$Comp
+L Device:R R?
+U 1 1 6225F84D
+P 4150 3050
+AR Path="/61BD4B7D/62026259/6225F84D" Ref="R?"  Part="1"
+AR Path="/61BD4B7D/62041525/6225F84D" Ref="R?"  Part="1"
+AR Path="/61BD4B7D/62045EF1/6225F84D" Ref="R?"  Part="1"
+AR Path="/61BD4B7D/6204A8C5/6225F84D" Ref="R?"  Part="1"
+AR Path="/6225F84D" Ref="R?"  Part="1"
+F 0 "R?" H 4200 3050 50  0000 L CNN
+F 1 "270K" V 4150 2950 50  0000 L CNN
+F 2 "" V 4080 3050 50  0001 C CNN
+F 3 "~" H 4150 3050 50  0001 C CNN
+	1    4150 3050
+	1    0    0    -1
+$EndComp
+$Comp
+L Device:Thermistor_NTC TH?
+U 1 1 6225F853
+P 4150 3350
+AR Path="/61BD4B7D/62026259/6225F853" Ref="TH?"  Part="1"
+AR Path="/61BD4B7D/62041525/6225F853" Ref="TH?"  Part="1"
+AR Path="/61BD4B7D/62045EF1/6225F853" Ref="TH?"  Part="1"
+AR Path="/61BD4B7D/6204A8C5/6225F853" Ref="TH?"  Part="1"
+AR Path="/6225F853" Ref="TH?"  Part="1"
+F 0 "TH?" H 4248 3396 50  0000 L CNN
+F 1 "100K NTC" H 4248 3305 50  0000 L CNN
+F 2 "" H 4150 3400 50  0001 C CNN
+F 3 "~" H 4150 3400 50  0001 C CNN
+	1    4150 3350
+	1    0    0    -1
+$EndComp
+Text Notes 3350 2600 0    50   ~ 0
+Top resistor selected for 5C center operating temperature
+$Comp
+L power:+3V3 #PWR?
+U 1 1 6225F85A
+P 4150 2900
+AR Path="/61BD4B7D/62026259/6225F85A" Ref="#PWR?"  Part="1"
+AR Path="/61BD4B7D/62041525/6225F85A" Ref="#PWR?"  Part="1"
+AR Path="/61BD4B7D/62045EF1/6225F85A" Ref="#PWR?"  Part="1"
+AR Path="/61BD4B7D/6204A8C5/6225F85A" Ref="#PWR?"  Part="1"
+AR Path="/6225F85A" Ref="#PWR?"  Part="1"
+F 0 "#PWR?" H 4150 2750 50  0001 C CNN
+F 1 "+3V3" H 4165 3073 50  0000 C CNN
+F 2 "" H 4150 2900 50  0001 C CNN
+F 3 "" H 4150 2900 50  0001 C CNN
+	1    4150 2900
+	1    0    0    -1
+$EndComp
+Wire Wire Line
+	4150 3200 4750 3200
+Connection ~ 4150 3200
+$Comp
+L power:GND #PWR?
+U 1 1 6225F863
+P 4150 3500
+AR Path="/61BD4B7D/62026259/6225F863" Ref="#PWR?"  Part="1"
+AR Path="/61BD4B7D/62041525/6225F863" Ref="#PWR?"  Part="1"
+AR Path="/61BD4B7D/62045EF1/6225F863" Ref="#PWR?"  Part="1"
+AR Path="/61BD4B7D/6204A8C5/6225F863" Ref="#PWR?"  Part="1"
+AR Path="/6225F863" Ref="#PWR?"  Part="1"
+F 0 "#PWR?" H 4150 3250 50  0001 C CNN
+F 1 "GND" H 4155 3327 50  0000 C CNN
+F 2 "" H 4150 3500 50  0001 C CNN
+F 3 "" H 4150 3500 50  0001 C CNN
+	1    4150 3500
+	1    0    0    -1
+$EndComp
+Text GLabel 4750 3200 2    50   Input ~ 0
+TELEM_TBRD
+Connection ~ 4150 3500
+Wire Wire Line
+	4150 3500 4750 3500
+$Comp
+L Device:C C?
+U 1 1 6225F847
+P 4750 3350
+AR Path="/61BD4B7D/62026259/6225F847" Ref="C?"  Part="1"
+AR Path="/61BD4B7D/62041525/6225F847" Ref="C?"  Part="1"
+AR Path="/61BD4B7D/62045EF1/6225F847" Ref="C?"  Part="1"
+AR Path="/61BD4B7D/6204A8C5/6225F847" Ref="C?"  Part="1"
+AR Path="/6225F847" Ref="C?"  Part="1"
+F 0 "C?" H 4865 3396 50  0000 L CNN
+F 1 "0.1uF" H 4865 3305 50  0000 L CNN
+F 2 "" H 4788 3200 50  0001 C CNN
+F 3 "~" H 4750 3350 50  0001 C CNN
+	1    4750 3350
+	1    0    0    -1
+$EndComp
+$Comp
+L 74xx:CD74HC4067SM U?
+U 1 1 622718CA
+P 6500 5850
+F 0 "U?" H 6500 7031 50  0000 C CNN
+F 1 "CD74HC4067SM" H 6500 6940 50  0000 C CNN
+F 2 "Package_SO:SSOP-24_5.3x8.2mm_P0.65mm" H 7550 4850 50  0001 C CIN
+F 3 "http://www.ti.com/lit/ds/symlink/cd74hc4067.pdf" H 6150 6700 50  0001 C CNN
+	1    6500 5850
+	-1   0    0    -1
+$EndComp
+Text GLabel 6000 5950 0    50   Input ~ 0
+TELEM_TBRD
+Text GLabel 7800 3450 0    50   Input ~ 0
+SOLAR_SCK
+Text GLabel 7800 3550 0    50   Input ~ 0
+SOLAR_MISO
+Text GLabel 7800 3650 0    50   Input ~ 0
+SOLAR_MOSI
+Text GLabel 7800 3350 0    50   Input ~ 0
+SOLAR_CS0
+Text GLabel 7800 3250 0    50   Input ~ 0
+SOLAR_CS1
+Text GLabel 4850 5350 2    50   Input ~ 0
+MUX0OUT
+Text GLabel 7000 5350 2    50   Input ~ 0
+MUX1OUT
+$Comp
+L 74xx:74HC595 U?
+U 1 1 622B9EC0
+P 2700 7150
+F 0 "U?" H 2700 7931 50  0000 C CNN
+F 1 "74HC595" H 2700 7840 50  0000 C CNN
+F 2 "" H 2700 7150 50  0001 C CNN
+F 3 "http://www.ti.com/lit/ds/symlink/sn74hc595.pdf" H 2700 7150 50  0001 C CNN
+	1    2700 7150
+	1    0    0    -1
+$EndComp
 $EndSCHEMATC

Commit message: connect amux
Parts:
- removed U?: 74HC595, symbol 74xx:74HC595
- added C? (x2): 0.1uF, symbol Device:C
- added C? (x2): 0.01uF, symbol Device:C
Connections:
- net +3V3: now also U?.24 (VCC), U?.24 (VCC), C?.1, C?.1
- net GND: now also U?.12 (GND), U?.12 (GND), U?.15 (~E), U?.15 (~E), C?.2, C?.2, C?.2, C?.2
- net HANDSHAKE: now also U?.25 (PB12); no longer U?.18 (PB0)
- net MUX0OUT: now also U?.10 (PA0), C?.1
- net MUX1OUT: now also U?.11 (PA1), C?.1
- net SOLAR_CS0: now also U?.18 (PB0); no longer U?.25 (PB12)
- net SOLAR_CS1: now also U?.19 (PB1); no longer U?.22 (PB11)
- net S0: now reaches U?.10 (S0)
- net S0: now also U?.10 (S0), U?.45 (PB8)
- net S1: now reaches U?.11 (S1)
- net S1: now also U?.11 (S1), U?.46 (PB9)
- net S3: now reaches U?.13 (S3)
- net S3: now also U?.13 (S3), U?.22 (PB11)
- net S2: now reaches U?.14 (S2)
- net S2: now also U?.14 (S2), U?.21 (PB10)
- net MUX2OUT: now reaches U?.12 (PA2)
- net MUX3OUT: now reaches U?.13 (PA3)
- net RST3V3: now reaches U?.17 (PA7)
- net RST5V: now reaches U?.29 (PA8)
- net RSTBATV: now reaches U?.30 (PA9)
- net RST12V: now reaches U?.31 (PA10)
Other:
- moved on the sheet: U?

Commit message: Add PDM control using shift registers
Connections:
- net SRCLK: now reaches U?.14 (PA4)
- net SRLCH: now reaches U?.15 (PA5)
- net SRSERIN: now reaches U?.16 (PA6)
Changed lines of the file:
@@
 Text GLabel 9100 2850 2    50   Input ~ 0
 RST3V3
+Text GLabel 9100 2550 2    50   Input ~ 0
+SRCLK
+Text GLabel 9100 2650 2    50   Input ~ 0
+SRLCH
+Text GLabel 9100 2750 2    50   Input ~ 0
+SRSERIN
 $EndSCHEMATC

Commit message: Annotate and begin adding footprints
Parts:
- C1, C10, C11, C12, C13, C2, C3, C4, C5, C6, C7, C8, C9: renamed from C?; footprint (none) -> Capacitor_SMD:C_0805_2012Metric
- H1, H2: footprint (none) -> Connector_PinSocket_2.54mm:PinSocket_2x26_P2.54mm_Vertical
- J1: renamed from J?; footprint (none) -> Connector_PinHeader_2.54mm:PinHeader_1x04_P2.54mm_Horizontal
- J2: renamed from J?; footprint (none) -> Connector_PinHeader_2.54mm:PinHeader_1x03_P2.54mm_Vertical
- MH1, MH2, MH3, MH4: renamed from MH?; footprint (none) -> MountingHole:MountingHole_3.2mm_M3_DIN965_Pad_TopBottom
- R1, R2, R3, R4, R5, R6, R7, R8, R9: renamed from R?; footprint (none) -> Resistor_SMD:R_0805_2012Metric
- Y1: renamed from Y?; footprint (none) -> Crystal:Crystal_HC49-4H_Vertical
- gave numbers to parts that had none: 7

Commit message: Add all IC footprints
Parts:
- TH1: footprint (none) -> Resistor_SMD:R_1206_3216Metric
Changed lines of the file:
@@
 F 0 "TH1" H 4248 3396 50  0000 L CNN
 F 1 "100K NTC" H 4248 3305 50  0000 L CNN
-F 2 "" H 4150 3400 50  0001 C CNN
+F 2 "Resistor_SMD:R_1206_3216Metric" H 4150 3400 50  0001 C CNN
 F 3 "~" H 4150 3400 50  0001 C CNN
 	1    4150 3350

Commit message: Major descope, remove 12V boost and all related circuitry
Connections:
- net +12V is gone; now on net +BATT: H1.23 (Pin_23), H1.24 (Pin_24)
- net SW13 is gone; now on net GND: H1.20 (Pin_20)
- net SW14 is gone; now on net GND: H1.19 (Pin_19)
- net TELEM_I12V is gone; now on net TELEM_IBATV: U3.9 (I0)
- net TELEM_V12V is gone; now on net TELEM_V5V: U3.5 (I4)
- net +3V3: now also H1.27 (Pin_27), H1.28 (Pin_28); no longer H1.29 (Pin_29), H1.30 (Pin_30)
- net +5V: now also H1.25 (Pin_25), H1.26 (Pin_26); no longer H1.27 (Pin_27), H1.28 (Pin_28)
- net +BATT: no longer H1.25 (Pin_25), H1.26 (Pin_26)
- net GND: now also H1.29 (Pin_29), H1.30 (Pin_30)
- net TELEM_I3V3: now also U3.7 (I2); no longer U3.6 (I3)
- net TELEM_I5V: now also U3.8 (I1); no longer U3.7 (I2)
- net TELEM_IBATV: no longer U3.8 (I1)
- net TELEM_TBRD: now also U3.3 (I6); no longer U3.23 (I8)
- net TELEM_V3V3: now also U3.4 (I5); no longer U3.2 (I7)
- net TELEM_V5V: no longer U3.3 (I6)
- net TELEM_VBATV: now also U3.6 (I3); no longer U3.4 (I5)
- net RST12V: no longer names the net of U4.31 (PA10)
Changed lines of the file:
@@
 $Descr A4 11693 8268
 encoding utf-8
-Sheet 1 44
+Sheet 1 37
 Title "TJ Custom EPS"
 Date ""
@@
 SW10
 $Comp
-L power:+12V #PWR0101
-U 1 1 61BC2B50
-P 2400 2050
-F 0 "#PWR0101" H 2400 1900 50  0001 C CNN
-F 1 "+12V" V 2415 2178 50  0000 L CNN
-F 2 "" H 2400 2050 50  0001 C CNN
-F 3 "" H 2400 2050 50  0001 C CNN
-	1    2400 2050
-	0    1    1    0
-$EndComp
-$Comp
-L power:+12V #PWR0102
-U 1 1 61BC30BA
-P 1900 2050
-F 0 "#PWR0102" H 1900 1900 50  0001 C CNN
-F 1 "+12V" V 1915 2178 50  0000 L CNN
-F 2 "" H 1900 2050 50  0001 C CNN
-F 3 "" H 1900 2050 50  0001 C CNN
-	1    1900 2050
-	0    -1   -1   0
-$EndComp
-$Comp
 L power:+5V #PWR0103
 U 1 1 61BC34F8
+P 1900 2150
+F 0 "#PWR0103" H 1900 2000 50  0001 C CNN
+F 1 "+5V" V 1915 2278 50  0000 L CNN
+F 2 "" H 1900 2150 50  0001 C CNN
+F 3 "" H 1900 2150 50  0001 C CNN
+	1    1900 2150
+	0    -1   -1   0
+$EndComp
+$Comp
+L power:+5V #PWR0104
+U 1 1 61BC3941
+P 2400 2150
+F 0 "#PWR0104" H 2400 2000 50  0001 C CNN
+F 1 "+5V" V 2415 2278 50  0000 L CNN
+F 2 "" H 2400 2150 50  0001 C CNN
+F 3 "" H 2400 2150 50  0001 C CNN
+	1    2400 2150
+	0    1    1    0
+$EndComp
+$Comp
+L power:+3V3 #PWR0105
+U 1 1 61BC3DF9
 P 1900 2250
-F 0 "#PWR0103" H 1900 2100 50  0001 C CNN
-F 1 "+5V" V 1915 2378 50  0000 L CNN
+F 0 "#PWR0105" H 1900 2100 50  0001 C CNN
+F 1 "+3V3" V 1915 2378 50  0000 L CNN
 F 2 "" H 1900 2250 50  0001 C CNN
 F 3 "" H 1900 2250 50  0001 C CNN
@@
 $EndComp
 $Comp
-L power:+5V #PWR0104
-U 1 1 61BC3941
+L power:+3V3 #PWR0106
+U 1 1 61BC42A2
 P 2400 2250
-F 0 "#PWR0104" H 2400 2100 50  0001 C CNN
-F 1 "+5V" V 2415 2378 50  0000 L CNN
+F 0 "#PWR0106" H 2400 2100 50  0001 C CNN
+F 1 "+3V3" V 2415 2378 50  0000 L CNN
 F 2 "" H 2400 2250 50  0001 C CNN
 F 3 "" H 2400 2250 50  0001 C CNN
 	1    2400 2250
-	0    1    1    0
-$EndComp
-$Comp
-L power:+3V3 #PWR0105
-U 1 1 61BC3DF9
-P 1900 2350
-F 0 "#PWR0105" H 1900 2200 50  0001 C CNN
-F 1 "+3V3" V 1915 2478 50  0000 L CNN
-F 2 "" H 1900 2350 50  0001 C CNN
-F 3 "" H 1900 2350 50  0001 C CNN
-	1    1900 2350
-	0    -1   -1   0
-$EndComp
-$Comp
-L power:+3V3 #PWR0106
-U 1 1 61BC42A2
-P 2400 2350
-F 0 "#PWR0106" H 2400 2200 50  0001 C CNN
-F 1 "+3V3" V 2415 2478 50  0000 L CNN
-F 2 "" H 2400 2350 50  0001 C CNN
-F 3 "" H 2400 2350 50  0001 C CNN
-	1    2400 2350
 	0    1    1    0
 $EndComp
@@
 L power:+BATT #PWR0107
 U 1 1 61BC5790
-P 2400 2150
-F 0 "#PWR0107" H 2400 2000 50  0001 C CNN
-F 1 "+BATT" V 2415 2278 50  0000 L CNN
-F 2 "" H 2400 2150 50  0001 C CNN
-F 3 "" H 2400 2150 50  0001 C CNN
-	1    2400 2150
+P 2400 2050
+F 0 "#PWR0107" H 2400 1900 50  0001 C CNN
+F 1 "+BATT" V 2415 2178 50  0000 L CNN
+F 2 "" H 2400 2050 50  0001 C CNN
+F 3 "" H 2400 2050 50  0001 C CNN
+	1    2400 2050
 	0    1    1    0
 $EndComp
@@
 L power:+BATT #PWR0108
 U 1 1 61BC64DC
-P 1900 2150
-F 0 "#PWR0108" H 1900 2000 50  0001 C CNN
-F 1 "+BATT" V 1915 2278 50  0000 L CNN
-F 2 "" H 1900 2150 50  0001 C CNN
-F 3 "" H 1900 2150 50  0001 C CNN
-	1    1900 2150
+P 1900 2050
+F 0 "#PWR0108" H 1900 1900 50  0001 C CNN
+F 1 "+BATT" V 1915 2178 50  0000 L CNN
+F 2 "" H 1900 2050 50  0001 C CNN
+F 3 "" H 1900 2050 50  0001 C CNN
+	1    1900 2050
 	0    -1   -1   0
 $EndComp
@@
 Text GLabel 2400 1750 2    50   Input ~ 0
 SW11
-Text GLabel 2400 1850 2    50   Input ~ 0
-SW13
 Text GLabel 1900 1750 0    50   Input ~ 0
 SW12
-Text GLabel 1900 1850 0    50   Input ~ 0
-SW14
 $Comp
 L Connector_Generic:Conn_02x26_Odd_Even H1
@@
 	2800 1150 2400 1150
 Wire Wire Line
-	2800 1150 2800 1950
+	2800 1150 2800 1850
 Wire Wire Line
 	1900 1150 1500 1150
 Wire Wire Line
-	1500 1150 1500 1950
+	1500 1150 1500 1850
 Connection ~ 1500 2450
 Wire Wire Line
 	1500 2450 1500 3150
-Wire Wire Line
-	1500 1950 1500 2450
 Connection ~ 2800 2450
 Wire Wire Line
 	2800 2450 2800 3150
-Wire Wire Line
-	2800 1950 2800 2450
 Connection ~ 2800 3150
 Wire Wire Line
@@
 TELEM_IBCROUT
 Text GLabel 5350 5150 0    50   Input ~ 0
-TELEM_I12V
+TELEM_IBATV
 Text GLabel 5350 5250 0    50   Input ~ 0
-TELEM_IBATV
+TELEM_I5V
 Text GLabel 5350 5350 0    50   Input ~ 0
-TELEM_I5V
+TELEM_I3V3
 Text GLabel 5350 5450 0    50   Input ~ 0
-TELEM_I3V3
+TELEM_VBATV
 Text GLabel 5350 5550 0    50   Input ~ 0
-TELEM_V12V
+TELEM_V5V
 Text GLabel 5350 5650 0    50   Input ~ 0
-TELEM_VBATV
-Text GLabel 5350 5750 0    50   Input ~ 0
-TELEM_V5V
-Text GLabel 5350 5850 0    50   Input ~ 0
 TELEM_V3V3
 $Comp
@@
 	-1   0    0    -1
 $EndComp
-Text GLabel 5350 5950 0    50   Input ~ 0
+Text GLabel 5350 5750 0    50   Input ~ 0
 TELEM_TBRD
 Text GLabel 7800 3450 0    50   Input ~ 0
@@
 Text GLabel 9100 2450 2    50   Input ~ 0
 MUX3OUT
-Text GLabel 9100 3150 2    50   Input ~ 0
-RST12V
 Text GLabel 9100 3050 2    50   Input ~ 0
 RSTBATV
@@
 Text GLabel 9100 2750 2    50   Input ~ 0
 SRSERIN
+Wire Wire Line
+	2400 2350 2800 2350
+Wire Wire Line
+	1900 2350 1500 2350
+Wire Wire Line
+	2400 1850 2800 1850
+Connection ~ 2800 1850
+Wire Wire Line
+	2800 1850 2800 1950
+Wire Wire Line
+	1900 1850 1500 1850
+Connection ~ 1500 1850
+Wire Wire Line
+	1500 1850 1500 1950
+Wire Wire Line
+	2800 1950 2800 2350
+Wire Wire Line
+	1500 1950 1500 2350
+Connection ~ 2800 2350
+Wire Wire Line
+	2800 2350 2800 2450
+Connection ~ 1500 2350
+Wire Wire Line
+	1500 2350 1500 2450
 $EndSCHEMATC

Commit message: Update stack header pinouts and re-annotate
Parts:
- renumbered H2 to H1, H1 to H2
Connections:
- net +3V3: now also H2.29 (Pin_29), H2.30 (Pin_30); no longer H2.27 (Pin_27), H2.28 (Pin_28)
- net +5V: now also H2.27 (Pin_27), H2.28 (Pin_28); no longer H2.25 (Pin_25), H2.26 (Pin_26)
- net +BATT: now also H2.25 (Pin_25), H2.26 (Pin_26); no longer H2.23 (Pin_23), H2.24 (Pin_24)
- net BCR_OUT: now also H2.39 (Pin_39), H2.40 (Pin_40); no longer H2.43 (Pin_43), H2.44 (Pin_44)
- net GND: now also H2.10 (Pin_10), H2.23 (Pin_23), H2.24 (Pin_24), H2.43 (Pin_43), H2.44 (Pin_44), H2.9 (Pin_9); no longer H2.19 (Pin_19), H2.20 (Pin_20), H2.21 (Pin_21), H2.22 (Pin_22), H2.29 (Pin_29), H2.30 (Pin_30), H2.45 (Pin_45), H2.46 (Pin_46), H2.5 (Pin_5), H2.6 (Pin_6)
- net SW1: now also H2.11 (Pin_11); no longer H2.7 (Pin_7)
- net SW10: now also H2.19 (Pin_19); no longer H2.15 (Pin_15)
- net SW11: now also H2.22 (Pin_22); no longer H2.18 (Pin_18)
- net SW12: now also H2.21 (Pin_21); no longer H2.17 (Pin_17)
- net SW2: now also H2.12 (Pin_12); no longer H2.8 (Pin_8)
- net SW3: now also H2.13 (Pin_13); no longer H2.9 (Pin_9)
- net SW4: now also H2.14 (Pin_14); no longer H2.10 (Pin_10)
- net SW5: now also H2.16 (Pin_16); no longer H2.12 (Pin_12)
- net SW6: now also H2.15 (Pin_15); no longer H2.11 (Pin_11)
- net SW7: now also H2.18 (Pin_18); no longer H2.14 (Pin_14)
- net SW8: now also H2.17 (Pin_17); no longer H2.13 (Pin_13)
- net SW9: now also H2.20 (Pin_20); no longer H2.16 (Pin_16)
- net VUSB: now also H2.45 (Pin_45), H2.46 (Pin_46); no longer H1.32 (Pin_32)
- no-connect marks 16 -> 18

Commit message: Condense muxes and add srrst
Parts:
- added C93: 0.1uF, Capacitor_SMD:C_0805_2012Metric, symbol Device:C
- added C94: 0.01uF, Capacitor_SMD:C_0805_2012Metric, symbol Device:C
- added U60: CD74HC4067SM, Package_SO:SSOP-24_5.3x8.2mm_P0.65mm, symbol 74xx:CD74HC4067SM
Connections:
- net +3V3: now also C93.1, U60.24 (VCC)
- net GND: now also C93.2, C94.2, U60.12 (GND), U60.15 (~E)
- net MUX2OUT: now also C94.1, U60.1 (COM)
- net RST3V3: now also U4.29 (PA8); no longer U4.17 (PA7)
- net RST5V: now also U4.30 (PA9); no longer U4.29 (PA8)
- net RSTBATV: now also U4.31 (PA10); no longer U4.30 (PA9)
- net S0: now also U60.10 (S0)
- net S1: now also U60.11 (S1)
- net S2: now also U60.14 (S2)
- net S3: now also U60.13 (S3)
- net TELEM_I3V3: now also U60.17 (I14); no longer U3.7 (I2)
- net TELEM_I5V: now also U60.18 (I13); no longer U3.8 (I1)
- net TELEM_IBATV: now also U60.19 (I12); no longer U3.9 (I0)
- net TELEM_TBRD: now also U1.16 (I15); no longer U3.3 (I6)
- net TELEM_V3V3: now also U3.17 (I14); no longer U3.4 (I5)
- net TELEM_V5V: now also U3.18 (I13); no longer U3.5 (I4)
- net TELEM_VBATV: now also U3.19 (I12); no longer U3.6 (I3)
- net TELEM_VSW8: now reaches U3.2 (I7)
- net TELEM_VSW12: now reaches U3.20 (I11)
- net TELEM_VSW11: now reaches U3.21 (I10)
- net TELEM_VSW10: now reaches U3.22 (I9)
- net TELEM_VSW9: now reaches U3.23 (I8)
- new net PDMRST: U4.17 (PA7)
- new net TELEM_ISW1: U60.9 (I0)
- new net TELEM_ISW10: U60.22 (I9)
- new net TELEM_ISW11: U60.21 (I10)
- new net TELEM_ISW12: U60.20 (I11)
- new net TELEM_ISW2: U60.8 (I1)
- new net TELEM_ISW3: U60.7 (I2)
- new net TELEM_ISW4: U60.6 (I3)
- new net TELEM_ISW5: U60.5 (I4)
- new net TELEM_ISW6: U60.4 (I5)
- new net TELEM_ISW7: U60.3 (I6)
- new net TELEM_ISW8: U60.2 (I7)
- new net TELEM_ISW9: U60.23 (I8)
- new net TELEM_VSW1: U3.9 (I0)
- new net TELEM_VSW2: U3.8 (I1)
- new net TELEM_VSW3: U3.7 (I2)
- new net TELEM_VSW4: U3.6 (I3)
- new net TELEM_VSW5: U3.5 (I4)
- new net TELEM_VSW6: U3.4 (I5)
- new net TELEM_VSW7: U3.3 (I6)
Other:
- moved on the sheet: C1, C3, U1
