File: ECAD/MPPT.sch (KiCad schematic (older format))
At the start: 24 parts, among them U30 LT6106, U31 LT6106, U32 LM358, U33 LT3652EMSE

Commit message: add some more footprints
Parts:
- D22: footprint (none) -> Diode_SMD:D_SMA
Changed lines of the file:
@@
 $Descr A4 11693 8268
 encoding utf-8
-Sheet 12 44
+Sheet 14 44
 Title "TJ Custom EPS"
 Date ""
@@
 AR Path="/61BEC565/61E10014/61BF0603" Ref="R97"  Part="1"
 AR Path="/61BEC565/61E1083C/61BF0603" Ref="R83"  Part="1"
-F 0 "R83" V 950 750 50  0000 C CNN
+F 0 "R111" V 950 750 50  0000 C CNN
 F 1 "20m" V 1050 750 50  0000 C CNN
 F 2 "" V 980 750 50  0001 C CNN
@@
 AR Path="/61BEC565/61E10014/61C169BE" Ref="R95"  Part="1"
 AR Path="/61BEC565/61E1083C/61C169BE" Ref="R81"  Part="1"
-F 0 "R81" H 900 1150 50  0000 L CNN
+F 0 "R109" H 900 1150 50  0000 L CNN
 F 1 "50R" V 850 1150 50  0000 C CNN
 F 2 "Resistor_SMD:R_0805_2012Metric" V 780 1150 50  0001 C CNN
@@
 AR Path="/61BEC565/61E10014/61C24A1A" Ref="U29"  Part="1"
 AR Path="/61BEC565/61E1083C/61C24A1A" Ref="U25"  Part="1"
-F 0 "U25" H 6900 2531 50  0000 C CNN
+F 0 "U33" H 6900 2531 50  0000 C CNN
 F 1 "LT3652EMSE" H 6900 2440 50  0000 C CNN
 F 2 "Package_SO:MSOP-12-1EP_3x4mm_P0.65mm_EP1.65x2.85mm" H 6900 1250 50  0001 C CNN
@@
 AR Path="/61BEC565/61E10014/61C384AF" Ref="U28"  Part="1"
 AR Path="/61BEC565/61E1083C/61C384AF" Ref="U24"  Part="1"
-F 0 "U24" H 4750 2217 50  0000 C CNN
+F 0 "U32" H 4750 2217 50  0000 C CNN
 F 1 "LM358" H 4750 2126 50  0000 C CNN
 F 2 "Package_SO:SO-8_3.9x4.9mm_P1.27mm" H 4750 1850 50  0001 C CNN
@@
 AR Path="/61BEC565/61E10014/61C39A83" Ref="U28"  Part="2"
 AR Path="/61BEC565/61E1083C/61C39A83" Ref="U24"  Part="2"
-F 0 "U24" H 5500 2117 50  0000 C CNN
+F 0 "U32" H 5500 2117 50  0000 C CNN
 F 1 "LM358" H 5500 2026 50  0000 C CNN
 F 2 "Package_SO:SO-8_3.9x4.9mm_P1.27mm" H 5500 1750 50  0001 C CNN
@@
 AR Path="/61BEC565/61E10014/61C3AED7" Ref="U28"  Part="3"
 AR Path="/61BEC565/61E1083C/61C3AED7" Ref="U24"  Part="3"
-F 0 "U24" H 3800 1700 50  0000 L CNN
+F 0 "U32" H 3800 1700 50  0000 L CNN
 F 1 "LM358" H 3700 1600 50  0000 L CNN
 F 2 "Package_SO:SO-8_3.9x4.9mm_P1.27mm" H 4100 1650 50  0001 C CNN
@@
 AR Path="/61BEC565/61E10014/61C732C6" Ref="R104"  Part="1"
 AR Path="/61BEC565/61E1083C/61C732C6" Ref="R90"  Part="1"
-F 0 "R90" V 4850 2150 50  0000 C CNN
+F 0 "R118" V 4850 2150 50  0000 C CNN
 F 1 "7.5K" V 4750 2150 50  0000 C CNN
 F 2 "Resistor_SMD:R_0805_2012Metric" V 4680 2150 50  0001 C CNN
@@
 AR Path="/61BEC565/61E10014/61C738CF" Ref="R103"  Part="1"
 AR Path="/61BEC565/61E1083C/61C738CF" Ref="R89"  Part="1"
-F 0 "R89" H 4500 2300 50  0000 L CNN
+F 0 "R117" H 4500 2300 50  0000 L CNN
 F 1 "1K" V 4450 2300 50  0000 C CNN
 F 2 "Resistor_SMD:R_0805_2012Metric" V 4380 2300 50  0001 C CNN
@@
 AR Path="/61BEC565/61E10014/61C7C0FE" Ref="#PWR0152"  Part="1"
 AR Path="/61BEC565/61E1083C/61C7C0FE" Ref="#PWR0148"  Part="1"
-F 0 "#PWR0148" H 5050 2300 50  0001 C CNN
+F 0 "#PWR0156" H 5050 2300 50  0001 C CNN
 F 1 "GND" H 5055 2377 50  0000 C CNN
 F 2 "" H 5050 2550 50  0001 C CNN
@@
 AR Path="/61BEC565/61E10014/61C7D2EA" Ref="C46"  Part="1"
 AR Path="/61BEC565/61E1083C/61C7D2EA" Ref="C43"  Part="1"
-F 0 "C43" H 6115 1546 50  0000 L CNN
+F 0 "C49" H 6115 1546 50  0000 L CNN
 F 1 "10uF" H 6115 1455 50  0000 L CNN
 F 2 "Capacitor_SMD:C_0805_2012Metric" H 6038 1350 50  0001 C CNN
@@
 AR Path="/61BEC565/61E10014/61C10EDC" Ref="R99"  Part="1"
 AR Path="/61BEC565/61E1083C/61C10EDC" Ref="R85"  Part="1"
-F 0 "R85" H 1950 1350 50  0000 L CNN
+F 0 "R113" H 1950 1350 50  0000 L CNN
 F 1 "5K" V 1900 1350 50  0000 C CNN
 F 2 "Resistor_SMD:R_0805_2012Metric" V 1830 1350 50  0001 C CNN
@@
 AR Path="/61BEC565/61E10014/61C105A2" Ref="#PWR0153"  Part="1"
 AR Path="/61BEC565/61E1083C/61C105A2" Ref="#PWR0149"  Part="1"
-F 0 "#PWR0149" H 1500 1250 50  0001 C CNN
+F 0 "#PWR0157" H 1500 1250 50  0001 C CNN
 F 1 "GND" H 1505 1327 50  0000 C CNN
 F 2 "" H 1500 1500 50  0001 C CNN
@@
 AR Path="/61BEC565/61E10014/61C0AC32" Ref="U26"  Part="1"
 AR Path="/61BEC565/61E1083C/61C0AC32" Ref="U22"  Part="1"
-F 0 "U22" H 1944 1246 50  0000 L CNN
+F 0 "U30" H 1944 1246 50  0000 L CNN
 F 1 "LT6106" H 1944 1155 50  0000 L CNN
 F 2 "Package_TO_SOT_SMD:SOT-23-5" H 1600 1200 50  0001 C CNN
@@
 AR Path="/61BEC565/61E10014/61BF13FC" Ref="R102"  Part="1"
 AR Path="/61BEC565/61E1083C/61BF13FC" Ref="R88"  Part="1"
-F 0 "R88" H 3200 2200 50  0000 L CNN
+F 0 "R116" H 3200 2200 50  0000 L CNN
 F 1 "100K" V 3150 2100 50  0000 L CNN
 F 2 "Resistor_SMD:R_0805_2012Metric" V 3080 2200 50  0001 C CNN
@@
 AR Path="/61BEC565/61E10014/61BF0C42" Ref="R101"  Part="1"
 AR Path="/61BEC565/61E1083C/61BF0C42" Ref="R87"  Part="1"
-F 0 "R87" H 3200 1600 50  0000 L CNN
+F 0 "R115" H 3200 1600 50  0000 L CNN
 F 1 "750K" V 3150 1500 50  0000 L CNN
 F 2 "Resistor_SMD:R_0805_2012Metric" V 3080 1600 50  0001 C CNN
@@
 AR Path="/61BEC565/61E10014/61D167BB" Ref="R98"  Part="1"
 AR Path="/61BEC565/61E1083C/61D167BB" Ref="R84"  Part="1"
-F 0 "R84" V 1000 1900 50  0000 C CNN
+F 0 "R112" V 1000 1900 50  0000 C CNN
 F 1 "20m" V 1100 1900 50  0000 C CNN
 F 2 "" V 1030 1900 50  0001 C CNN
@@
 AR Path="/61BEC565/61E10014/61D167C5" Ref="R96"  Part="1"
 AR Path="/61BEC565/61E1083C/61D167C5" Ref="R82"  Part="1"
-F 0 "R82" H 950 2300 50  0000 L CNN
+F 0 "R110" H 950 2300 50  0000 L CNN
 F 1 "50R" V 900 2300 50  0000 C CNN
 F 2 "Resistor_SMD:R_0805_2012Metric" V 830 2300 50  0001 C CNN
@@
 AR Path="/61BEC565/61E10014/61D167D4" Ref="R100"  Part="1"
 AR Path="/61BEC565/61E1083C/61D167D4" Ref="R86"  Part="1"
-F 0 "R86" H 2000 2500 50  0000 L CNN
+F 0 "R114" H 2000 2500 50  0000 L CNN
 F 1 "5K" V 1950 2500 50  0000 C CNN
 F 2 "Resistor_SMD:R_0805_2012Metric" V 1880 2500 50  0001 C CNN
@@
 AR Path="/61BEC565/61E10014/61D167DA" Ref="#PWR0154"  Part="1"
 AR Path="/61BEC565/61E1083C/61D167DA" Ref="#PWR0150"  Part="1"
-F 0 "#PWR0150" H 1550 2400 50  0001 C CNN
+F 0 "#PWR0158" H 1550 2400 50  0001 C CNN
 F 1 "GND" H 1555 2477 50  0000 C CNN
 F 2 "" H 1550 2650 50  0001 C CNN
@@
 AR Path="/61BEC565/61E10014/61D167E0" Ref="U27"  Part="1"
 AR Path="/61BEC565/61E1083C/61D167E0" Ref="U23"  Part="1"
-F 0 "U23" H 1994 2396 50  0000 L CNN
+F 0 "U31" H 1994 2396 50  0000 L CNN
 F 1 "LT6106" H 1994 2305 50  0000 L CNN
 F 2 "Package_TO_SOT_SMD:SOT-23-5" H 1650 2350 50  0001 C CNN
@@
 AR Path="/61BEC565/61E10014/61D5E781" Ref="R105"  Part="1"
 AR Path="/61BEC565/61E1083C/61D5E781" Ref="R91"  Part="1"
-F 0 "R91" V 7500 2250 50  0000 C CNN
+F 0 "R119" V 7500 2250 50  0000 C CNN
 F 1 "52.8K" V 7600 2250 50  0000 C CNN
 F 2 "Resistor_SMD:R_0805_2012Metric" V 7530 2250 50  0001 C CNN
@@
 AR Path="/61BEC565/61E10014/61D6D602" Ref="R107"  Part="1"
 AR Path="/61BEC565/61E1083C/61D6D602" Ref="R93"  Part="1"
-F 0 "R93" H 7750 2400 50  0000 R CNN
+F 0 "R121" H 7750 2400 50  0000 R CNN
 F 1 "330K" V 7800 2400 50  0000 C CNN
 F 2 "Resistor_SMD:R_0805_2012Metric" V 7730 2400 50  0001 C CNN
@@
 AR Path="/61BEC565/61E10014/61D73998" Ref="R106"  Part="1"
 AR Path="/61BEC565/61E1083C/61D73998" Ref="R92"  Part="1"
-F 0 "R92" H 7750 2100 50  0000 R CNN
+F 0 "R120" H 7750 2100 50  0000 R CNN
 F 1 "490K" V 7800 2100 50  0000 C CNN
 F 2 "Resistor_SMD:R_0805_2012Metric" V 7730 2100 50  0001 C CNN
@@
 AR Path="/61BEC565/61E10014/61D9F858" Ref="D21"  Part="1"
 AR Path="/61BEC565/61E1083C/61D9F858" Ref="D19"  Part="1"
-F 0 "D19" H 7950 1967 50  0000 C CNN
+F 0 "D23" H 7950 1967 50  0000 C CNN
 F 1 "CMDSH2-4L" H 7950 1876 50  0000 C CNN
 F 2 "" H 7950 1750 50  0001 C CNN
@@
 AR Path="/61BEC565/61E10014/61DA5795" Ref="C47"  Part="1"
 AR Path="/61BEC565/61E1083C/61DA5795" Ref="C44"  Part="1"
-F 0 "C44" H 7550 1700 50  0000 L CNN
+F 0 "C50" H 7550 1700 50  0000 L CNN
 F 1 "1uF" H 7550 1500 50  0000 L CNN
 F 2 "Capacitor_SMD:C_0805_2012Metric" H 7588 1450 50  0001 C CNN
@@
 AR Path="/61BEC565/61E10014/61DAD2DF" Ref="D20"  Part="1"
 AR Path="/61BEC565/61E1083C/61DAD2DF" Ref="D18"  Part="1"
-F 0 "D18" H 7700 1467 50  0000 C CNN
+F 0 "D22" H 7700 1467 50  0000 C CNN
 F 1 "CMSH3-40MA" H 7700 1376 50  0000 C CNN
-F 2 "" H 7700 1250 50  0001 C CNN
+F 2 "Diode_SMD:D_SMA" H 7700 1250 50  0001 C CNN
 F 3 "~" H 7700 1250 50  0001 C CNN
 	1    7700 1250
@@
 AR Path="/61BEC565/61E10014/61DB925A" Ref="#PWR0155"  Part="1"
 AR Path="/61BEC565/61E1083C/61DB925A" Ref="#PWR0151"  Part="1"
-F 0 "#PWR0151" H 7850 1000 50  0001 C CNN
+F 0 "#PWR0159" H 7850 1000 50  0001 C CNN
 F 1 "GND" H 7855 1077 50  0000 C CNN
 F 2 "" H 7850 1250 50  0001 C CNN
@@
 AR Path="/61BEC565/61E10014/61DBC37B" Ref="L2"  Part="1"
 AR Path="/61BEC565/61E1083C/61DBC37B" Ref="L1"  Part="1"
-F 0 "L1" H 8303 1696 50  0000 L CNN
+F 0 "L3" H 8303 1696 50  0000 L CNN
 F 1 "22uH" H 8300 1600 50  0000 L CNN
 F 2 "" H 8250 1650 50  0001 C CNN
@@
 AR Path="/61BEC565/61E10014/61DC7062" Ref="R108"  Part="1"
 AR Path="/61BEC565/61E1083C/61DC7062" Ref="R94"  Part="1"
-F 0 "R94" V 8350 2000 50  0000 C CNN
+F 0 "R122" V 8350 2000 50  0000 C CNN
 F 1 "50m" V 8450 1850 50  0000 C CNN
 F 2 "" V 8380 1850 50  0001 C CNN
@@
 AR Path="/61BEC565/61E10014/61DD561E" Ref="C48"  Part="1"
 AR Path="/61BEC565/61E1083C/61DD561E" Ref="C45"  Part="1"
-F 0 "C45" H 8365 2146 50  0000 L CNN
+F 0 "C51" H 8365 2146 50  0000 L CNN
 F 1 "10uF" H 8365 2055 50  0000 L CNN
 F 2 "Capacitor_SMD:C_0805_2012Metric" H 8288 1950 50  0001 C CNN

Commit message: Add all IC footprints
Parts:
- D23: value CMDSH2-4L -> RB051MM-2Y; footprint (none) -> Diode_SMD:D_SOD-123F
Changed lines of the file:
@@
 $Descr A4 11693 8268
 encoding utf-8
-Sheet 14 44
+Sheet 12 44
 Title "TJ Custom EPS"
 Date ""
@@
 AR Path="/61BEC565/61E10014/61BF0603" Ref="R97"  Part="1"
 AR Path="/61BEC565/61E1083C/61BF0603" Ref="R83"  Part="1"
-F 0 "R111" V 950 750 50  0000 C CNN
+F 0 "R83" V 950 750 50  0000 C CNN
 F 1 "20m" V 1050 750 50  0000 C CNN
 F 2 "" V 980 750 50  0001 C CNN
@@
 AR Path="/61BEC565/61E10014/61C169BE" Ref="R95"  Part="1"
 AR Path="/61BEC565/61E1083C/61C169BE" Ref="R81"  Part="1"
-F 0 "R109" H 900 1150 50  0000 L CNN
+F 0 "R81" H 900 1150 50  0000 L CNN
 F 1 "50R" V 850 1150 50  0000 C CNN
 F 2 "Resistor_SMD:R_0805_2012Metric" V 780 1150 50  0001 C CNN
@@
 AR Path="/61BEC565/61E10014/61C24A1A" Ref="U29"  Part="1"
 AR Path="/61BEC565/61E1083C/61C24A1A" Ref="U25"  Part="1"
-F 0 "U33" H 6900 2531 50  0000 C CNN
+F 0 "U25" H 6900 2531 50  0000 C CNN
 F 1 "LT3652EMSE" H 6900 2440 50  0000 C CNN
 F 2 "Package_SO:MSOP-12-1EP_3x4mm_P0.65mm_EP1.65x2.85mm" H 6900 1250 50  0001 C CNN
@@
 AR Path="/61BEC565/61E10014/61C384AF" Ref="U28"  Part="1"
 AR Path="/61BEC565/61E1083C/61C384AF" Ref="U24"  Part="1"
-F 0 "U32" H 4750 2217 50  0000 C CNN
+F 0 "U24" H 4750 2217 50  0000 C CNN
 F 1 "LM358" H 4750 2126 50  0000 C CNN
 F 2 "Package_SO:SO-8_3.9x4.9mm_P1.27mm" H 4750 1850 50  0001 C CNN
@@
 AR Path="/61BEC565/61E10014/61C39A83" Ref="U28"  Part="2"
 AR Path="/61BEC565/61E1083C/61C39A83" Ref="U24"  Part="2"
-F 0 "U32" H 5500 2117 50  0000 C CNN
+F 0 "U24" H 5500 2117 50  0000 C CNN
 F 1 "LM358" H 5500 2026 50  0000 C CNN
 F 2 "Package_SO:SO-8_3.9x4.9mm_P1.27mm" H 5500 1750 50  0001 C CNN
@@
 AR Path="/61BEC565/61E10014/61C3AED7" Ref="U28"  Part="3"
 AR Path="/61BEC565/61E1083C/61C3AED7" Ref="U24"  Part="3"
-F 0 "U32" H 3800 1700 50  0000 L CNN
+F 0 "U24" H 3800 1700 50  0000 L CNN
 F 1 "LM358" H 3700 1600 50  0000 L CNN
 F 2 "Package_SO:SO-8_3.9x4.9mm_P1.27mm" H 4100 1650 50  0001 C CNN
@@
 AR Path="/61BEC565/61E10014/61C732C6" Ref="R104"  Part="1"
 AR Path="/61BEC565/61E1083C/61C732C6" Ref="R90"  Part="1"
-F 0 "R118" V 4850 2150 50  0000 C CNN
+F 0 "R90" V 4850 2150 50  0000 C CNN
 F 1 "7.5K" V 4750 2150 50  0000 C CNN
 F 2 "Resistor_SMD:R_0805_2012Metric" V 4680 2150 50  0001 C CNN
@@
 AR Path="/61BEC565/61E10014/61C738CF" Ref="R103"  Part="1"
 AR Path="/61BEC565/61E1083C/61C738CF" Ref="R89"  Part="1"
-F 0 "R117" H 4500 2300 50  0000 L CNN
+F 0 "R89" H 4500 2300 50  0000 L CNN
 F 1 "1K" V 4450 2300 50  0000 C CNN
 F 2 "Resistor_SMD:R_0805_2012Metric" V 4380 2300 50  0001 C CNN
@@
 AR Path="/61BEC565/61E10014/61C7C0FE" Ref="#PWR0152"  Part="1"
 AR Path="/61BEC565/61E1083C/61C7C0FE" Ref="#PWR0148"  Part="1"
-F 0 "#PWR0156" H 5050 2300 50  0001 C CNN
+F 0 "#PWR0148" H 5050 2300 50  0001 C CNN
 F 1 "GND" H 5055 2377 50  0000 C CNN
 F 2 "" H 5050 2550 50  0001 C CNN
@@
 AR Path="/61BEC565/61E10014/61C7D2EA" Ref="C46"  Part="1"
 AR Path="/61BEC565/61E1083C/61C7D2EA" Ref="C43"  Part="1"
-F 0 "C49" H 6115 1546 50  0000 L CNN
+F 0 "C43" H 6115 1546 50  0000 L CNN
 F 1 "10uF" H 6115 1455 50  0000 L CNN
 F 2 "Capacitor_SMD:C_0805_2012Metric" H 6038 1350 50  0001 C CNN
@@
 AR Path="/61BEC565/61E10014/61C10EDC" Ref="R99"  Part="1"
 AR Path="/61BEC565/61E1083C/61C10EDC" Ref="R85"  Part="1"
-F 0 "R113" H 1950 1350 50  0000 L CNN
+F 0 "R85" H 1950 1350 50  0000 L CNN
 F 1 "5K" V 1900 1350 50  0000 C CNN
 F 2 "Resistor_SMD:R_0805_2012Metric" V 1830 1350 50  0001 C CNN
@@
 AR Path="/61BEC565/61E10014/61C105A2" Ref="#PWR0153"  Part="1"
 AR Path="/61BEC565/61E1083C/61C105A2" Ref="#PWR0149"  Part="1"
-F 0 "#PWR0157" H 1500 1250 50  0001 C CNN
+F 0 "#PWR0149" H 1500 1250 50  0001 C CNN
 F 1 "GND" H 1505 1327 50  0000 C CNN
 F 2 "" H 1500 1500 50  0001 C CNN
@@
 AR Path="/61BEC565/61E10014/61C0AC32" Ref="U26"  Part="1"
 AR Path="/61BEC565/61E1083C/61C0AC32" Ref="U22"  Part="1"
-F 0 "U30" H 1944 1246 50  0000 L CNN
+F 0 "U22" H 1944 1246 50  0000 L CNN
 F 1 "LT6106" H 1944 1155 50  0000 L CNN
 F 2 "Package_TO_SOT_SMD:SOT-23-5" H 1600 1200 50  0001 C CNN
@@
 AR Path="/61BEC565/61E10014/61BF13FC" Ref="R102"  Part="1"
 AR Path="/61BEC565/61E1083C/61BF13FC" Ref="R88"  Part="1"
-F 0 "R116" H 3200 2200 50  0000 L CNN
+F 0 "R88" H 3200 2200 50  0000 L CNN
 F 1 "100K" V 3150 2100 50  0000 L CNN
 F 2 "Resistor_SMD:R_0805_2012Metric" V 3080 2200 50  0001 C CNN
@@
 AR Path="/61BEC565/61E10014/61BF0C42" Ref="R101"  Part="1"
 AR Path="/61BEC565/61E1083C/61BF0C42" Ref="R87"  Part="1"
-F 0 "R115" H 3200 1600 50  0000 L CNN
+F 0 "R87" H 3200 1600 50  0000 L CNN
 F 1 "750K" V 3150 1500 50  0000 L CNN
 F 2 "Resistor_SMD:R_0805_2012Metric" V 3080 1600 50  0001 C CNN
@@
 AR Path="/61BEC565/61E10014/61D167BB" Ref="R98"  Part="1"
 AR Path="/61BEC565/61E1083C/61D167BB" Ref="R84"  Part="1"
-F 0 "R112" V 1000 1900 50  0000 C CNN
+F 0 "R84" V 1000 1900 50  0000 C CNN
 F 1 "20m" V 1100 1900 50  0000 C CNN
 F 2 "" V 1030 1900 50  0001 C CNN
@@
 AR Path="/61BEC565/61E10014/61D167C5" Ref="R96"  Part="1"
 AR Path="/61BEC565/61E1083C/61D167C5" Ref="R82"  Part="1"
-F 0 "R110" H 950 2300 50  0000 L CNN
+F 0 "R82" H 950 2300 50  0000 L CNN
 F 1 "50R" V 900 2300 50  0000 C CNN
 F 2 "Resistor_SMD:R_0805_2012Metric" V 830 2300 50  0001 C CNN
@@
 AR Path="/61BEC565/61E10014/61D167D4" Ref="R100"  Part="1"
 AR Path="/61BEC565/61E1083C/61D167D4" Ref="R86"  Part="1"
-F 0 "R114" H 2000 2500 50  0000 L CNN
+F 0 "R86" H 2000 2500 50  0000 L CNN
 F 1 "5K" V 1950 2500 50  0000 C CNN
 F 2 "Resistor_SMD:R_0805_2012Metric" V 1880 2500 50  0001 C CNN
@@
 AR Path="/61BEC565/61E10014/61D167DA" Ref="#PWR0154"  Part="1"
 AR Path="/61BEC565/61E1083C/61D167DA" Ref="#PWR0150"  Part="1"
-F 0 "#PWR0158" H 1550 2400 50  0001 C CNN
+F 0 "#PWR0150" H 1550 2400 50  0001 C CNN
 F 1 "GND" H 1555 2477 50  0000 C CNN
 F 2 "" H 1550 2650 50  0001 C CNN
@@
 AR Path="/61BEC565/61E10014/61D167E0" Ref="U27"  Part="1"
 AR Path="/61BEC565/61E1083C/61D167E0" Ref="U23"  Part="1"
-F 0 "U31" H 1994 2396 50  0000 L CNN
+F 0 "U23" H 1994 2396 50  0000 L CNN
 F 1 "LT6106" H 1994 2305 50  0000 L CNN
 F 2 "Package_TO_SOT_SMD:SOT-23-5" H 1650 2350 50  0001 C CNN
@@
 AR Path="/61BEC565/61E10014/61D5E781" Ref="R105"  Part="1"
 AR Path="/61BEC565/61E1083C/61D5E781" Ref="R91"  Part="1"
-F 0 "R119" V 7500 2250 50  0000 C CNN
+F 0 "R91" V 7500 2250 50  0000 C CNN
 F 1 "52.8K" V 7600 2250 50  0000 C CNN
 F 2 "Resistor_SMD:R_0805_2012Metric" V 7530 2250 50  0001 C CNN
@@
 AR Path="/61BEC565/61E10014/61D6D602" Ref="R107"  Part="1"
 AR Path="/61BEC565/61E1083C/61D6D602" Ref="R93"  Part="1"
-F 0 "R121" H 7750 2400 50  0000 R CNN
+F 0 "R93" H 7750 2400 50  0000 R CNN
 F 1 "330K" V 7800 2400 50  0000 C CNN
 F 2 "Resistor_SMD:R_0805_2012Metric" V 7730 2400 50  0001 C CNN
@@
 AR Path="/61BEC565/61E10014/61D73998" Ref="R106"  Part="1"
 AR Path="/61BEC565/61E1083C/61D73998" Ref="R92"  Part="1"
-F 0 "R120" H 7750 2100 50  0000 R CNN
+F 0 "R92" H 7750 2100 50  0000 R CNN
 F 1 "490K" V 7800 2100 50  0000 C CNN
 F 2 "Resistor_SMD:R_0805_2012Metric" V 7730 2100 50  0001 C CNN
@@
 AR Path="/61BEC565/61E10014/61D9F858" Ref="D21"  Part="1"
 AR Path="/61BEC565/61E1083C/61D9F858" Ref="D19"  Part="1"
-F 0 "D23" H 7950 1967 50  0000 C CNN
-F 1 "CMDSH2-4L" H 7950 1876 50  0000 C CNN
-F 2 "" H 7950 1750 50  0001 C CNN
+F 0 "D19" H 7950 1967 50  0000 C CNN
+F 1 "RB051MM-2Y" H 7950 1876 50  0000 C CNN
+F 2 "Diode_SMD:D_SOD-123F" H 7950 1750 50  0001 C CNN
 F 3 "~" H 7950 1750 50  0001 C CNN
 	1    7950 1750
@@
 AR Path="/61BEC565/61E10014/61DA5795" Ref="C47"  Part="1"
 AR Path="/61BEC565/61E1083C/61DA5795" Ref="C44"  Part="1"
-F 0 "C50" H 7550 1700 50  0000 L CNN
+F 0 "C44" H 7550 1700 50  0000 L CNN
 F 1 "1uF" H 7550 1500 50  0000 L CNN
 F 2 "Capacitor_SMD:C_0805_2012Metric" H 7588 1450 50  0001 C CNN
@@
 AR Path="/61BEC565/61E10014/61DAD2DF" Ref="D20"  Part="1"
 AR Path="/61BEC565/61E1083C/61DAD2DF" Ref="D18"  Part="1"
-F 0 "D22" H 7700 1467 50  0000 C CNN
+F 0 "D18" H 7700 1467 50  0000 C CNN
 F 1 "CMSH3-40MA" H 7700 1376 50  0000 C CNN
 F 2 "Diode_SMD:D_SMA" H 7700 1250 50  0001 C CNN
@@
 AR Path="/61BEC565/61E10014/61DB925A" Ref="#PWR0155"  Part="1"
 AR Path="/61BEC565/61E1083C/61DB925A" Ref="#PWR0151"  Part="1"
-F 0 "#PWR0159" H 7850 1000 50  0001 C CNN
+F 0 "#PWR0151" H 7850 1000 50  0001 C CNN
 F 1 "GND" H 7855 1077 50  0000 C CNN
 F 2 "" H 7850 1250 50  0001 C CNN
@@
 AR Path="/61BEC565/61E10014/61DBC37B" Ref="L2"  Part="1"
 AR Path="/61BEC565/61E1083C/61DBC37B" Ref="L1"  Part="1"
-F 0 "L3" H 8303 1696 50  0000 L CNN
+F 0 "L1" H 8303 1696 50  0000 L CNN
 F 1 "22uH" H 8300 1600 50  0000 L CNN
 F 2 "" H 8250 1650 50  0001 C CNN
@@
 AR Path="/61BEC565/61E10014/61DC7062" Ref="R108"  Part="1"
 AR Path="/61BEC565/61E1083C/61DC7062" Ref="R94"  Part="1"
-F 0 "R122" V 8350 2000 50  0000 C CNN
+F 0 "R94" V 8350 2000 50  0000 C CNN
 F 1 "50m" V 8450 1850 50  0000 C CNN
 F 2 "" V 8380 1850 50  0001 C CNN
@@
 AR Path="/61BEC565/61E10014/61DD561E" Ref="C48"  Part="1"
 AR Path="/61BEC565/61E1083C/61DD561E" Ref="C45"  Part="1"
-F 0 "C51" H 8365 2146 50  0000 L CNN
+F 0 "C45" H 8365 2146 50  0000 L CNN
 F 1 "10uF" H 8365 2055 50  0000 L CNN
 F 2 "Capacitor_SMD:C_0805_2012Metric" H 8288 1950 50  0001 C CNN

Commit message: add a bunch of cap and shunt resistor footprints
Parts:
- R111, R112, R122: footprint (none) -> Resistor_SMD:R_2512_6332Metric
Changed lines of the file:
@@
 F 0 "R83" V 950 750 50  0000 C CNN
 F 1 "20m" V 1050 750 50  0000 C CNN
-F 2 "" V 980 750 50  0001 C CNN
+F 2 "Resistor_SMD:R_2512_6332Metric" V 980 750 50  0001 C CNN
 F 3 "~" H 1050 750 50  0001 C CNN
 	1    1050 750
@@
 F 0 "R84" V 1000 1900 50  0000 C CNN
 F 1 "20m" V 1100 1900 50  0000 C CNN
-F 2 "" V 1030 1900 50  0001 C CNN
+F 2 "Resistor_SMD:R_2512_6332Metric" V 1030 1900 50  0001 C CNN
 F 3 "~" H 1100 1900 50  0001 C CNN
 	1    1100 1900
@@
 F 0 "R94" V 8350 2000 50  0000 C CNN
 F 1 "50m" V 8450 1850 50  0000 C CNN
-F 2 "" V 8380 1850 50  0001 C CNN
+F 2 "Resistor_SMD:R_2512_6332Metric" V 8380 1850 50  0001 C CNN
 F 3 "~" H 8450 1850 50  0001 C CNN
 	1    8450 1850

Commit message: Update stack header pinouts and re-annotate
Parts:
- renumbered C49 to C47, C50 to C48, C51 to C49, D22 to D21, D23 to D22, R109 to R100, R110 to R101, R111 to R102, R112 to R103, R113 to R104, R114 to R105, R115 to R106, R116 to R107, R117 to R108, R118 to R109, R119 to R110, R120 to R111, R121 to R112, R122 to R113, U30 to U27, U31 to U28, U32 to U29, U33 to U30

Commit message: Despec inductor for buck converters, finish adding footprints, general schematic cleanup
Parts:
- L3: footprint (none) -> Inductor_SMD:L_Bourns_SRP7028A_7.3x6.6mm
Changed lines of the file:
@@
 $Descr A4 11693 8268
 encoding utf-8
-Sheet 12 37
+Sheet 10 37
 Title "TJ Custom EPS"
 Date ""
@@
 F 0 "L3" H 8303 1696 50  0000 L CNN
 F 1 "22uH" H 8300 1600 50  0000 L CNN
-F 2 "" H 8250 1650 50  0001 C CNN
+F 2 "Inductor_SMD:L_Bourns_SRP7028A_7.3x6.6mm" H 8250 1650 50  0001 C CNN
 F 3 "~" H 8250 1650 50  0001 C CNN
 	1    8250 1650
