File: ECAD/SolarTelem.sch (KiCad schematic (older format))
At the start: 8 parts

Commit message: Implement solar telemetry, add a sheet layout
Parts:
- added C? (x2): 0.1uF, symbol Device:C
- added H? (x4): M2.5, symbol Mechanical:MountingHole_Pad
- added J?: OUT, symbol Connector:Conn_01x07_Female
- added U? (x2): MCP3208, symbol Analog_ADC:MCP3208
Connections:
- net S1ATelem/TEMPIN: now reaches J?.2 (Pin_2)
- net S1ATelem/PHOTOIN: now reaches J?.3 (Pin_3)
- net S1BTelem/TEMPIN: now reaches J?.2 (Pin_2)
- net S1BTelem/PHOTOIN: now reaches J?.3 (Pin_3)
- net S2ATelem/TEMPIN: now reaches J?.2 (Pin_2)
- net S2ATelem/PHOTOIN: now reaches J?.3 (Pin_3)
- net S2BTelem/TEMPIN: now reaches J?.2 (Pin_2)
- net S2BTelem/PHOTOIN: now reaches J?.3 (Pin_3)
- net S3ATelem/TEMPIN: now reaches J?.2 (Pin_2)
- net S3ATelem/PHOTOIN: now reaches J?.3 (Pin_3)
- net S3BTelem/TEMPIN: now reaches J?.2 (Pin_2)
- net S3BTelem/PHOTOIN: now reaches J?.3 (Pin_3)
- net S4ATelem/TEMPIN: now reaches J?.2 (Pin_2)
- net S4ATelem/PHOTOIN: now reaches J?.3 (Pin_3)
- net S4BTelem/TEMPIN: now reaches J?.2 (Pin_2)
- net S4BTelem/PHOTOIN: now reaches J?.3 (Pin_3)
- new net +3.3VA: C?.1, C?.1, J?.1 (Pin_1), U?.15 (Vref), U?.15 (Vref), U?.16 (Vdd), U?.16 (Vdd)
- new net CS0: J?.5 (Pin_5), U?.10 (~CS~/SHDN)
- new net CS1: J?.6 (Pin_6), U?.10 (~CS~/SHDN)
- new net GND: C?.2, C?.2, H?.1, H?.1, H?.1, H?.1, J?.7 (Pin_7), U?.14 (AGND), U?.14 (AGND), U?.9 (DGND), U?.9 (DGND)
- new net MISO: J?.3 (Pin_3), U?.12 (Dout), U?.12 (Dout)
- new net MOSI: J?.4 (Pin_4), U?.11 (Din), U?.11 (Din)
- new net S1ATelem/PHOTOOUT: U?.2 (CH1)
- new net S1ATelem/TEMPOUT: U?.1 (CH0)
- new net S1BTelem/PHOTOOUT: U?.4 (CH3)
- new net S1BTelem/TEMPOUT: U?.3 (CH2)
- new net S2ATelem/PHOTOOUT: U?.6 (CH5)
- new net S2ATelem/TEMPOUT: U?.5 (CH4)
- new net S2BTelem/PHOTOOUT: U?.8 (CH7)
- new net S2BTelem/TEMPOUT: U?.7 (CH6)
- new net S3ATelem/PHOTOOUT: U?.2 (CH1)
- new net S3ATelem/TEMPOUT: U?.1 (CH0)
- new net S3BTelem/PHOTOOUT: U?.4 (CH3)
- new net S3BTelem/TEMPOUT: U?.3 (CH2)
- new net S4ATelem/PHOTOOUT: U?.6 (CH5)
- new net S4ATelem/TEMPOUT: U?.5 (CH4)
- new net S4BTelem/PHOTOOUT: U?.8 (CH7)
- new net S4BTelem/TEMPOUT: U?.7 (CH6)
- new net SCK: J?.2 (Pin_2), U?.13 (CLK), U?.13 (CLK)

Commit message: Annotate and begin adding footprints
Parts:
- C60, C61: renamed from C?; footprint (none) -> Capacitor_SMD:C_0805_2012Metric
- H17, H18, H19, H20: renamed from H?; footprint (none) -> MountingHole:MountingHole_2.7mm_M2.5_DIN965_Pad
- J14, J15, J16, J17, J18, J19, J20, J21: renamed from J?; footprint (none) -> Connector_Hirose:Hirose_DF13-04P-1.25DSA_1x04_P1.25mm_Vertical
- gave numbers to parts that had none: 3

Commit message: Add all IC footprints
Parts:
- U39, U40: footprint (none) -> Package_SO:SO-16_3.9x9.9mm_P1.27mm
Changed lines of the file:
@@
 F 0 "U39" H 4200 3281 50  0000 C CNN
 F 1 "MCP3208" H 4200 3190 50  0000 C CNN
-F 2 "" H 4300 2700 50  0001 C CNN
+F 2 "Package_SO:SO-16_3.9x9.9mm_P1.27mm" H 4300 2700 50  0001 C CNN
 F 3 "http://ww1.microchip.com/downloads/en/DeviceDoc/21298c.pdf" H 4300 2700 50  0001 C CNN
 	1    4200 2600
@@
 F 0 "U40" H 4200 5031 50  0000 C CNN
 F 1 "MCP3208" H 4200 4940 50  0000 C CNN
-F 2 "" H 4300 4450 50  0001 C CNN
+F 2 "Package_SO:SO-16_3.9x9.9mm_P1.27mm" H 4300 4450 50  0001 C CNN
 F 3 "http://ww1.microchip.com/downloads/en/DeviceDoc/21298c.pdf" H 4300 4450 50  0001 C CNN
 	1    4200 4350

Commit message: add a bunch of cap and shunt resistor footprints
Parts:
- J22: footprint (none) -> Connector_PinSocket_1.27mm:PinSocket_1x07_P1.27mm_Vertical
Changed lines of the file:
@@
 F 0 "J22" H 6078 3426 50  0000 L CNN
 F 1 "OUT" H 6078 3335 50  0000 L CNN
-F 2 "" H 6050 3400 50  0001 C CNN
+F 2 "Connector_PinSocket_1.27mm:PinSocket_1x07_P1.27mm_Vertical" H 6050 3400 50  0001 C CNN
 F 3 "~" H 6050 3400 50  0001 C CNN
 	1    6050 3400

Commit message: Update stack header pinouts and re-annotate
Parts:
- renumbered C60 to C58, C61 to C59, H18 to H10, H19 to H11, H20 to H12, H17 to H9, U39 to U36, U40 to U37
Changed lines of the file:
@@
 	1200 6600 1650 6600
 $Comp
-L Mechanical:MountingHole_Pad H17
+L Mechanical:MountingHole_Pad H9
 U 1 1 61DDA086
 P 6650 2100
-F 0 "H17" H 6750 2149 50  0000 L CNN
+F 0 "H9" H 6750 2149 50  0000 L CNN
 F 1 "M2.5" H 6750 2058 50  0000 L CNN
 F 2 "MountingHole:MountingHole_2.7mm_M2.5_DIN965_Pad" H 6650 2100 50  0001 C CNN
@@
 AR Path="/61BEC565/636144E9/61DD520E/61DDAE75" Ref="#PWR?"  Part="1"
 AR Path="/61BEC565/636144E9/61DD5214/61DDAE75" Ref="#PWR?"  Part="1"
-AR Path="/61BEC565/636144E9/61DDAE75" Ref="#PWR066"  Part="1"
-F 0 "#PWR066" H 6650 1950 50  0001 C CNN
+AR Path="/61BEC565/636144E9/61DDAE75" Ref="#PWR0119"  Part="1"
+F 0 "#PWR0119" H 6650 1950 50  0001 C CNN
 F 1 "GND" H 6655 2027 50  0000 C CNN
 F 2 "" H 6650 2200 50  0001 C CNN
@@
 $EndComp
 $Comp
-L Mechanical:MountingHole_Pad H19
+L Mechanical:MountingHole_Pad H11
 U 1 1 61DDD34E
 P 7050 2100
-F 0 "H19" H 7150 2149 50  0000 L CNN
+F 0 "H11" H 7150 2149 50  0000 L CNN
 F 1 "M2.5" H 7150 2058 50  0000 L CNN
 F 2 "MountingHole:MountingHole_2.7mm_M2.5_DIN965_Pad" H 7050 2100 50  0001 C CNN
@@
 AR Path="/61BEC565/636144E9/61DD520E/61DDD354" Ref="#PWR?"  Part="1"
 AR Path="/61BEC565/636144E9/61DD5214/61DDD354" Ref="#PWR?"  Part="1"
-AR Path="/61BEC565/636144E9/61DDD354" Ref="#PWR068"  Part="1"
-F 0 "#PWR068" H 7050 1950 50  0001 C CNN
+AR Path="/61BEC565/636144E9/61DDD354" Ref="#PWR0121"  Part="1"
+F 0 "#PWR0121" H 7050 1950 50  0001 C CNN
 F 1 "GND" H 7055 2027 50  0000 C CNN
 F 2 "" H 7050 2200 50  0001 C CNN
@@
 $EndComp
 $Comp
-L Mechanical:MountingHole_Pad H18
+L Mechanical:MountingHole_Pad H10
 U 1 1 61DDE165
 P 6650 2650
-F 0 "H18" H 6750 2699 50  0000 L CNN
+F 0 "H10" H 6750 2699 50  0000 L CNN
 F 1 "M2.5" H 6750 2608 50  0000 L CNN
 F 2 "MountingHole:MountingHole_2.7mm_M2.5_DIN965_Pad" H 6650 2650 50  0001 C CNN
@@
 AR Path="/61BEC565/636144E9/61DD520E/61DDE16B" Ref="#PWR?"  Part="1"
 AR Path="/61BEC565/636144E9/61DD5214/61DDE16B" Ref="#PWR?"  Part="1"
-AR Path="/61BEC565/636144E9/61DDE16B" Ref="#PWR067"  Part="1"
-F 0 "#PWR067" H 6650 2500 50  0001 C CNN
+AR Path="/61BEC565/636144E9/61DDE16B" Ref="#PWR0120"  Part="1"
+F 0 "#PWR0120" H 6650 2500 50  0001 C CNN
 F 1 "GND" H 6655 2577 50  0000 C CNN
 F 2 "" H 6650 2750 50  0001 C CNN
@@
 $EndComp
 $Comp
-L Mechanical:MountingHole_Pad H20
+L Mechanical:MountingHole_Pad H12
 U 1 1 61DDEDFA
 P 7050 2650
-F 0 "H20" H 7150 2699 50  0000 L CNN
+F 0 "H12" H 7150 2699 50  0000 L CNN
 F 1 "M2.5" H 7150 2608 50  0000 L CNN
 F 2 "MountingHole:MountingHole_2.7mm_M2.5_DIN965_Pad" H 7050 2650 50  0001 C CNN
@@
 AR Path="/61BEC565/636144E9/61DD520E/61DDEE00" Ref="#PWR?"  Part="1"
 AR Path="/61BEC565/636144E9/61DD5214/61DDEE00" Ref="#PWR?"  Part="1"
-AR Path="/61BEC565/636144E9/61DDEE00" Ref="#PWR069"  Part="1"
-F 0 "#PWR069" H 7050 2500 50  0001 C CNN
+AR Path="/61BEC565/636144E9/61DDEE00" Ref="#PWR0122"  Part="1"
+F 0 "#PWR0122" H 7050 2500 50  0001 C CNN
 F 1 "GND" H 7055 2577 50  0000 C CNN
 F 2 "" H 7050 2750 50  0001 C CNN
@@
 $EndComp
 $Comp
-L Analog_ADC:MCP3208 U39
+L Analog_ADC:MCP3208 U36
 U 1 1 61DF1A1E
 P 4200 2600
-F 0 "U39" H 4200 3281 50  0000 C CNN
+F 0 "U36" H 4200 3281 50  0000 C CNN
 F 1 "MCP3208" H 4200 3190 50  0000 C CNN
 F 2 "Package_SO:SO-16_3.9x9.9mm_P1.27mm" H 4300 2700 50  0001 C CNN
@@
 $EndComp
 $Comp
-L Analog_ADC:MCP3208 U40
+L Analog_ADC:MCP3208 U37
 U 1 1 61DF4003
 P 4200 4350
-F 0 "U40" H 4200 5031 50  0000 C CNN
+F 0 "U37" H 4200 5031 50  0000 C CNN
 F 1 "MCP3208" H 4200 4940 50  0000 C CNN
 F 2 "Package_SO:SO-16_3.9x9.9mm_P1.27mm" H 4300 4450 50  0001 C CNN
@@
 $EndComp
 $Comp
-L power:+3.3VA #PWR061
+L power:+3.3VA #PWR0114
 U 1 1 61DF4DA9
 P 4950 2100
-F 0 "#PWR061" H 4950 1950 50  0001 C CNN
+F 0 "#PWR0114" H 4950 1950 50  0001 C CNN
 F 1 "+3.3VA" H 4965 2273 50  0000 C CNN
 F 2 "" H 4950 2100 50  0001 C CNN
@@
 	4400 3850 4100 3850
 $Comp
-L Device:C C60
+L Device:C C58
 U 1 1 61DF73F3
 P 5250 2250
-F 0 "C60" H 5365 2296 50  0000 L CNN
+F 0 "C58" H 5365 2296 50  0000 L CNN
 F 1 "0.1uF" H 5365 2205 50  0000 L CNN
 F 2 "Capacitor_SMD:C_0805_2012Metric" H 5288 2100 50  0001 C CNN
@@
 $EndComp
 $Comp
-L Device:C C61
+L Device:C C59
 U 1 1 61DF7CC1
 P 5250 4000
-F 0 "C61" H 5365 4046 50  0000 L CNN
+F 0 "C59" H 5365 4046 50  0000 L CNN
 F 1 "0.1uF" H 5365 3955 50  0000 L CNN
 F 2 "Capacitor_SMD:C_0805_2012Metric" H 5288 3850 50  0001 C CNN
@@
 AR Path="/61BEC565/636144E9/61DD520E/61DFA512" Ref="#PWR?"  Part="1"
 AR Path="/61BEC565/636144E9/61DD5214/61DFA512" Ref="#PWR?"  Part="1"
-AR Path="/61BEC565/636144E9/61DFA512" Ref="#PWR063"  Part="1"
-F 0 "#PWR063" H 5250 3900 50  0001 C CNN
+AR Path="/61BEC565/636144E9/61DFA512" Ref="#PWR0116"  Part="1"
+F 0 "#PWR0116" H 5250 3900 50  0001 C CNN
 F 1 "GND" H 5255 3977 50  0000 C CNN
 F 2 "" H 5250 4150 50  0001 C CNN
@@
 AR Path="/61BEC565/636144E9/61DD520E/61DFA518" Ref="#PWR?"  Part="1"
 AR Path="/61BEC565/636144E9/61DD5214/61DFA518" Ref="#PWR?"  Part="1"
-AR Path="/61BEC565/636144E9/61DFA518" Ref="#PWR062"  Part="1"
-F 0 "#PWR062" H 5250 2150 50  0001 C CNN
+AR Path="/61BEC565/636144E9/61DFA518" Ref="#PWR0115"  Part="1"
+F 0 "#PWR0115" H 5250 2150 50  0001 C CNN
 F 1 "GND" H 5255 2227 50  0000 C CNN
 F 2 "" H 5250 2400 50  0001 C CNN
@@
 AR Path="/61BEC565/636144E9/61DD520E/61DFCEA1" Ref="#PWR?"  Part="1"
 AR Path="/61BEC565/636144E9/61DD5214/61DFCEA1" Ref="#PWR?"  Part="1"
-AR Path="/61BEC565/636144E9/61DFCEA1" Ref="#PWR060"  Part="1"
-F 0 "#PWR060" H 4100 4700 50  0001 C CNN
+AR Path="/61BEC565/636144E9/61DFCEA1" Ref="#PWR0113"  Part="1"
+F 0 "#PWR0113" H 4100 4700 50  0001 C CNN
 F 1 "GND" H 4105 4777 50  0000 C CNN
 F 2 "" H 4100 4950 50  0001 C CNN
@@
 AR Path="/61BEC565/636144E9/61DD520E/61DFCEA7" Ref="#PWR?"  Part="1"
 AR Path="/61BEC565/636144E9/61DD5214/61DFCEA7" Ref="#PWR?"  Part="1"
-AR Path="/61BEC565/636144E9/61DFCEA7" Ref="#PWR059"  Part="1"
-F 0 "#PWR059" H 4100 2950 50  0001 C CNN
+AR Path="/61BEC565/636144E9/61DFCEA7" Ref="#PWR0112"  Part="1"
+F 0 "#PWR0112" H 4100 2950 50  0001 C CNN
 F 1 "GND" H 4105 3027 50  0000 C CNN
 F 2 "" H 4100 3200 50  0001 C CNN
@@
 CS1
 $Comp
-L power:+3.3VA #PWR064
+L power:+3.3VA #PWR0117
 U 1 1 61E820B7
 P 5750 3100
-F 0 "#PWR064" H 5750 2950 50  0001 C CNN
+F 0 "#PWR0117" H 5750 2950 50  0001 C CNN
 F 1 "+3.3VA" H 5765 3273 50  0000 C CNN
 F 2 "" H 5750 3100 50  0001 C CNN
@@
 AR Path="/61BEC565/636144E9/61DD520E/61E8CD3E" Ref="#PWR?"  Part="1"
 AR Path="/61BEC565/636144E9/61DD5214/61E8CD3E" Ref="#PWR?"  Part="1"
-AR Path="/61BEC565/636144E9/61E8CD3E" Ref="#PWR065"  Part="1"
-F 0 "#PWR065" H 5750 3450 50  0001 C CNN
+AR Path="/61BEC565/636144E9/61E8CD3E" Ref="#PWR0118"  Part="1"
+F 0 "#PWR0118" H 5750 3450 50  0001 C CNN
 F 1 "GND" H 5755 3527 50  0000 C CNN
 F 2 "" H 5750 3700 50  0001 C CNN
