File: ECAD/Temp+Light.sch (KiCad schematic (older format))
At the start: 7 parts

Commit message: Annotate and begin adding footprints
Parts:
- R139, R140, R141, R142: renamed from R?; footprint (none) -> Resistor_SMD:R_0805_2012Metric
- U41: renamed from U?; footprint (none) -> Package_SO:SO-8_3.9x4.9mm_P1.27mm

Commit message: Add all IC footprints
Changed lines of the file:
@@
 $Descr A4 11693 8268
 encoding utf-8
-Sheet 24 44
+Sheet 17 44
 Title "TJ Custom EPS"
 Date ""
@@
 AR Path="/61BEC565/636144E9/61DD520E/61D7F18C" Ref="R163"  Part="1"
 AR Path="/61BEC565/636144E9/61DD5214/61D7F18C" Ref="R167"  Part="1"
-F 0 "R167" H 3400 2150 50  0000 L CNN
+F 0 "R139" H 3400 2150 50  0000 L CNN
 F 1 "100K" V 3350 2150 50  0000 C CNN
 F 2 "Resistor_SMD:R_0805_2012Metric" V 3280 2150 50  0001 C CNN
@@
 AR Path="/61BEC565/636144E9/61DD520E/61D7F747" Ref="R165"  Part="1"
 AR Path="/61BEC565/636144E9/61DD5214/61D7F747" Ref="R169"  Part="1"
-F 0 "R169" V 3750 3750 50  0000 C CNN
+F 0 "R141" V 3750 3750 50  0000 C CNN
 F 1 "3K" V 3650 3750 50  0000 C CNN
 F 2 "Resistor_SMD:R_0805_2012Metric" V 3580 3750 50  0001 C CNN
@@
 AR Path="/61BEC565/636144E9/61DD520E/61D89596" Ref="U47"  Part="1"
 AR Path="/61BEC565/636144E9/61DD5214/61D89596" Ref="U48"  Part="1"
-F 0 "U48" H 3900 2767 50  0000 C CNN
+F 0 "U41" H 3900 2767 50  0000 C CNN
 F 1 "LM358" H 3900 2676 50  0000 C CNN
 F 2 "Package_SO:SO-8_3.9x4.9mm_P1.27mm" H 3900 2400 50  0001 C CNN
@@
 AR Path="/61BEC565/636144E9/61DD520E/61D8A9E1" Ref="U47"  Part="2"
 AR Path="/61BEC565/636144E9/61DD5214/61D8A9E1" Ref="U48"  Part="2"
-F 0 "U48" H 3650 4667 50  0000 C CNN
+F 0 "U41" H 3650 4667 50  0000 C CNN
 F 1 "LM358" H 3650 4576 50  0000 C CNN
 F 2 "Package_SO:SO-8_3.9x4.9mm_P1.27mm" H 3650 4300 50  0001 C CNN
@@
 AR Path="/61BEC565/636144E9/61DD520E/61D8B59A" Ref="U47"  Part="3"
 AR Path="/61BEC565/636144E9/61DD5214/61D8B59A" Ref="U48"  Part="3"
-F 0 "U48" H 2408 3096 50  0000 L CNN
+F 0 "U41" H 2408 3096 50  0000 L CNN
 F 1 "LM358" H 2408 3005 50  0000 L CNN
 F 2 "Package_SO:SO-8_3.9x4.9mm_P1.27mm" H 2450 3050 50  0001 C CNN
@@
 AR Path="/61BEC565/636144E9/61DD520E/61D92CEE" Ref="#PWR0100"  Part="1"
 AR Path="/61BEC565/636144E9/61DD5214/61D92CEE" Ref="#PWR0198"  Part="1"
-F 0 "#PWR0198" H 2350 2600 50  0001 C CNN
+F 0 "#PWR070" H 2350 2600 50  0001 C CNN
 F 1 "+3.3VA" H 2365 2923 50  0000 C CNN
 F 2 "" H 2350 2750 50  0001 C CNN
@@
 AR Path="/61BEC565/636144E9/61DD520E/61D93C4C" Ref="#PWR0142"  Part="1"
 AR Path="/61BEC565/636144E9/61DD5214/61D93C4C" Ref="#PWR0199"  Part="1"
-F 0 "#PWR0199" H 2350 3100 50  0001 C CNN
+F 0 "#PWR071" H 2350 3100 50  0001 C CNN
 F 1 "GND" H 2355 3177 50  0000 C CNN
 F 2 "" H 2350 3350 50  0001 C CNN
@@
 AR Path="/61BEC565/636144E9/61DD520E/61D9B58C" Ref="#PWR0145"  Part="1"
 AR Path="/61BEC565/636144E9/61DD5214/61D9B58C" Ref="#PWR0200"  Part="1"
-F 0 "#PWR0200" H 3350 1850 50  0001 C CNN
+F 0 "#PWR072" H 3350 1850 50  0001 C CNN
 F 1 "+3.3VA" H 3365 2173 50  0000 C CNN
 F 2 "" H 3350 2000 50  0001 C CNN
@@
 AR Path="/61BEC565/636144E9/61DD520E/61D9C312" Ref="R164"  Part="1"
 AR Path="/61BEC565/636144E9/61DD5214/61D9C312" Ref="R168"  Part="1"
-F 0 "R168" H 3650 3000 50  0000 L CNN
+F 0 "R140" H 3650 3000 50  0000 L CNN
 F 1 "1K" V 3600 3000 50  0000 C CNN
 F 2 "Resistor_SMD:R_0805_2012Metric" V 3530 3000 50  0001 C CNN
@@
 AR Path="/61BEC565/636144E9/61DD520E/61D9C6FD" Ref="R166"  Part="1"
 AR Path="/61BEC565/636144E9/61DD5214/61D9C6FD" Ref="R170"  Part="1"
-F 0 "R170" V 4000 2700 50  0000 L CNN
+F 0 "R142" V 4000 2700 50  0000 L CNN
 F 1 "120K" V 3900 2750 50  0000 C CNN
 F 2 "Resistor_SMD:R_0805_2012Metric" V 3830 2750 50  0001 C CNN
@@
 AR Path="/61BEC565/636144E9/61DD520E/61D9E166" Ref="#PWR0197"  Part="1"
 AR Path="/61BEC565/636144E9/61DD5214/61D9E166" Ref="#PWR0202"  Part="1"
-F 0 "#PWR0202" H 3600 2900 50  0001 C CNN
+F 0 "#PWR074" H 3600 2900 50  0001 C CNN
 F 1 "GND" H 3605 2977 50  0000 C CNN
 F 2 "" H 3600 3150 50  0001 C CNN
@@
 AR Path="/61BEC565/636144E9/61DD520E/61DA7F11" Ref="#PWR0196"  Part="1"
 AR Path="/61BEC565/636144E9/61DD5214/61DA7F11" Ref="#PWR0201"  Part="1"
-F 0 "#PWR0201" H 3350 4400 50  0001 C CNN
+F 0 "#PWR073" H 3350 4400 50  0001 C CNN
 F 1 "GND" H 3355 4477 50  0000 C CNN
 F 2 "" H 3350 4650 50  0001 C CNN

Commit message: Update stack header pinouts and re-annotate
Parts:
- renumbered R139 to R130, R140 to R131, R141 to R132, R142 to R133, U41 to U38

Commit message: Schematic Cleanup
Changed lines of the file:
@@
 EELAYER 30 0
 EELAYER END
-$Descr A4 11693 8268
+$Descr USLetter 11000 8500
 encoding utf-8
-Sheet 17 37
+Sheet 13 37
 Title "TJ Custom EPS"
 Date ""
@@
 AR Path="/61BEC565/636144E9/61DD520E/61D7F18C" Ref="R154"  Part="1"
 AR Path="/61BEC565/636144E9/61DD5214/61D7F18C" Ref="R158"  Part="1"
-F 0 "R158" H 3400 2150 50  0000 L CNN
+F 0 "R130" H 3400 2150 50  0000 L CNN
 F 1 "100K" V 3350 2150 50  0000 C CNN
 F 2 "Resistor_SMD:R_0805_2012Metric" V 3280 2150 50  0001 C CNN
@@
 AR Path="/61BEC565/636144E9/61DD520E/61D7F747" Ref="R156"  Part="1"
 AR Path="/61BEC565/636144E9/61DD5214/61D7F747" Ref="R160"  Part="1"
-F 0 "R160" V 3750 3750 50  0000 C CNN
+F 0 "R132" V 3750 3750 50  0000 C CNN
 F 1 "3K" V 3650 3750 50  0000 C CNN
 F 2 "Resistor_SMD:R_0805_2012Metric" V 3580 3750 50  0001 C CNN
@@
 AR Path="/61BEC565/636144E9/61DD520E/61D89596" Ref="U44"  Part="1"
 AR Path="/61BEC565/636144E9/61DD5214/61D89596" Ref="U45"  Part="1"
-F 0 "U45" H 3900 2767 50  0000 C CNN
+F 0 "U38" H 3900 2767 50  0000 C CNN
 F 1 "LM358" H 3900 2676 50  0000 C CNN
 F 2 "Package_SO:SO-8_3.9x4.9mm_P1.27mm" H 3900 2400 50  0001 C CNN
@@
 AR Path="/61BEC565/636144E9/61DD520E/61D8A9E1" Ref="U44"  Part="2"
 AR Path="/61BEC565/636144E9/61DD5214/61D8A9E1" Ref="U45"  Part="2"
-F 0 "U45" H 3650 4667 50  0000 C CNN
+F 0 "U38" H 3650 4667 50  0000 C CNN
 F 1 "LM358" H 3650 4576 50  0000 C CNN
 F 2 "Package_SO:SO-8_3.9x4.9mm_P1.27mm" H 3650 4300 50  0001 C CNN
@@
 AR Path="/61BEC565/636144E9/61DD520E/61D8B59A" Ref="U44"  Part="3"
 AR Path="/61BEC565/636144E9/61DD5214/61D8B59A" Ref="U45"  Part="3"
-F 0 "U45" H 2408 3096 50  0000 L CNN
+F 0 "U38" H 2408 3096 50  0000 L CNN
 F 1 "LM358" H 2408 3005 50  0000 L CNN
 F 2 "Package_SO:SO-8_3.9x4.9mm_P1.27mm" H 2450 3050 50  0001 C CNN
@@
 AR Path="/61BEC565/636144E9/61DD520E/61D92CEE" Ref="#PWR0153"  Part="1"
 AR Path="/61BEC565/636144E9/61DD5214/61D92CEE" Ref="#PWR0158"  Part="1"
-F 0 "#PWR0158" H 2350 2600 50  0001 C CNN
+F 0 "#PWR0123" H 2350 2600 50  0001 C CNN
 F 1 "+3.3VA" H 2365 2923 50  0000 C CNN
 F 2 "" H 2350 2750 50  0001 C CNN
@@
 AR Path="/61BEC565/636144E9/61DD520E/61D93C4C" Ref="#PWR0154"  Part="1"
 AR Path="/61BEC565/636144E9/61DD5214/61D93C4C" Ref="#PWR0159"  Part="1"
-F 0 "#PWR0159" H 2350 3100 50  0001 C CNN
+F 0 "#PWR0124" H 2350 3100 50  0001 C CNN
 F 1 "GND" H 2355 3177 50  0000 C CNN
 F 2 "" H 2350 3350 50  0001 C CNN
@@
 AR Path="/61BEC565/636144E9/61DD520E/61D9B58C" Ref="#PWR0155"  Part="1"
 AR Path="/61BEC565/636144E9/61DD5214/61D9B58C" Ref="#PWR0160"  Part="1"
-F 0 "#PWR0160" H 3350 1850 50  0001 C CNN
+F 0 "#PWR0125" H 3350 1850 50  0001 C CNN
 F 1 "+3.3VA" H 3365 2173 50  0000 C CNN
 F 2 "" H 3350 2000 50  0001 C CNN
@@
 AR Path="/61BEC565/636144E9/61DD520E/61D9C312" Ref="R155"  Part="1"
 AR Path="/61BEC565/636144E9/61DD5214/61D9C312" Ref="R159"  Part="1"
-F 0 "R159" H 3650 3000 50  0000 L CNN
+F 0 "R131" H 3650 3000 50  0000 L CNN
 F 1 "1K" V 3600 3000 50  0000 C CNN
 F 2 "Resistor_SMD:R_0805_2012Metric" V 3530 3000 50  0001 C CNN
@@
 AR Path="/61BEC565/636144E9/61DD520E/61D9C6FD" Ref="R157"  Part="1"
 AR Path="/61BEC565/636144E9/61DD5214/61D9C6FD" Ref="R161"  Part="1"
-F 0 "R161" V 4000 2700 50  0000 L CNN
+F 0 "R133" V 4000 2700 50  0000 L CNN
 F 1 "120K" V 3900 2750 50  0000 C CNN
 F 2 "Resistor_SMD:R_0805_2012Metric" V 3830 2750 50  0001 C CNN
@@
 AR Path="/61BEC565/636144E9/61DD520E/61D9E166" Ref="#PWR0157"  Part="1"
 AR Path="/61BEC565/636144E9/61DD5214/61D9E166" Ref="#PWR0162"  Part="1"
-F 0 "#PWR0162" H 3600 2900 50  0001 C CNN
+F 0 "#PWR0127" H 3600 2900 50  0001 C CNN
 F 1 "GND" H 3605 2977 50  0000 C CNN
 F 2 "" H 3600 3150 50  0001 C CNN
@@
 AR Path="/61BEC565/636144E9/61DD520E/61DA7F11" Ref="#PWR0156"  Part="1"
 AR Path="/61BEC565/636144E9/61DD5214/61DA7F11" Ref="#PWR0161"  Part="1"
-F 0 "#PWR0161" H 3350 4400 50  0001 C CNN
+F 0 "#PWR0126" H 3350 4400 50  0001 C CNN
 F 1 "GND" H 3355 4477 50  0000 C CNN
 F 2 "" H 3350 4650 50  0001 C CNN
