File: ECAD/TJ-EPS.kicad_pcb (KiCad board)
At the start: 2 copper layers, 654 parts, among them J1 SWD, J10 S3B, J11 S4A, J12 S4B, J13 TELEM_IN, J14 S1A, J15 S1B, J16 S2A, J17 S2B, J18 S3A, J19 S3B, J2 BOOT, J20 S4A, J21 S4B, J22 OUT, J3 SWD, J4 BOOT, J5 S1A, J6 S1B, J7 S2A, J8 S2B, J9 S3A, Q1 2N7002, Q10 Si4186DY, Q11 IRF7425, Q12 Si4186DY, Q13 2N7002, Q14 IRF7458, Q15 Si4186DY, Q16 2N7002, Q17 IRF7458, Q18 Si4186DY, Q19 2N7002, Q2 IRF7425, Q20 IRF7458, Q21 Si4186DY, Q22 2N7002, Q23 IRF7458, Q24 Si4186DY, Q25 IRF7425, Q26 IRF7458, Q27 Si4186DY, Q28 SIR167DP, Q29 SIR167DP, Q3 IRF7458, Q30 2N7002, Q31 IRF7458, Q32 2N7002, Q33 IRF7458, Q34 2N7002, Q35 2N7002, Q36 2N7002, Q37 IRF7458, Q38 IRF7458, Q39 2N7002, Q4 Si4186DY, Q40 2N7002, Q41 2N7002, Q42 2N7002, Q43 2N7002, Q44 2N7002, Q45 2N7002, Q46 2N7002, Q47 2N7002, Q48 IRF7458, Q49 2N7002, Q5 IRF7458, Q50 IRF7458, Q51 2N7002, Q52 IRF7458, Q53 2N7002, Q54 IRF7458, Q55 2N7002, Q56 IRF7458, Q57 2N7002, Q58 IRF7458, Q59 2N7002, Q6 Si4186DY, Q60 IRF7458, Q61 2N7002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

Commit message: move bat board stuff aside
Parts:
- moved Q22 324.7 mm to (-67.0, -8.69)
- moved R58 324.7 mm to (-62.6, -6.48)
- moved R59 324.7 mm to (-58.1, -9.49)
- moved R61 324.7 mm to (-53.3, -16.7)
- moved R63 324.7 mm to (-62.2, -15.8)
- moved C34 324.7 mm to (-62.5, -9.46)
- moved Q23 324.7 mm to (-73.4, -14.9)
- moved Q24 324.7 mm to (-73.4, -8.49)
- moved R60 324.7 mm to (-57.7, -13.7)
- moved R62 324.7 mm to (-67.0, -4.94)
- moved R64 324.7 mm to (-57.7, -16.7)
- moved TH5 324.7 mm to (-66.9, -15.8)
- moved C31 276.3 mm to (-46.9, 10.8)
- moved Q13 276.3 mm to (-51.3, 11.6)
- moved Q14 276.3 mm to (-57.8, 11.8)
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