File: Concepts/555 boost converter/555 boost converter.sch (KiCad schematic (older format))
At the start: 1 part

Commit message: spec out new cell protection IC and mosfets, figured out current limit calculation
Parts:
- removed U?: NE555D, Package_SO:SOIC-8_3.9x4.9mm_P1.27mm, symbol Timer:NE555D
- added U?: LMC555xM, Package_SO:SOIC-8_3.9x4.9mm_P1.27mm, symbol Timer:LMC555xM
Changed lines of the file:
@@
 $EndDescr
 $Comp
-L Timer:NE555D U?
-U 1 1 61C55B22
-P 6000 2550
-F 0 "U?" H 6000 3131 50  0000 C CNN
-F 1 "NE555D" H 6000 3040 50  0000 C CNN
-F 2 "Package_SO:SOIC-8_3.9x4.9mm_P1.27mm" H 6850 2150 50  0001 C CNN
-F 3 "http://www.ti.com/lit/ds/symlink/ne555.pdf" H 6850 2150 50  0001 C CNN
-	1    6000 2550
+L Timer:LMC555xM U?
+U 1 1 61C68AC5
+P 5450 3200
+F 0 "U?" H 5450 3781 50  0000 C CNN
+F 1 "LMC555xM" H 5450 3690 50  0000 C CNN
+F 2 "Package_SO:SOIC-8_3.9x4.9mm_P1.27mm" H 6300 2800 50  0001 C CNN
+F 3 "http://www.ti.com/lit/ds/symlink/lmc555.pdf" H 6300 2800 50  0001 C CNN
+	1    5450 3200
 	1    0    0    -1
 $EndComp
