File: ECAD/SolarTelem/SolarTelem.kicad_pcb (KiCad board)
At the start: 2 copper layers, 57 parts, among them J1 S1A, J2 S1B, J3 S2A, J4 S2B, J5 S3A, J6 S3B, J7 S4A, J8 S4B, J9 OUT, U1 MCP3208, U10 LM358, U2 MCP3208, U3 LM358, U4 LM358, U5 LM358, U6 LM358, U7 LM358, U8 LM358, U9 LM358

Commit message: 18500 footprint
Parts:
- moved U1 16.9 mm to (112.8, 67.6)
- moved U2 16.3 mm to (112.8, 80.3)

Commit message: Further descope: remove SA4
Parts:
- removed J7: S4A, Connector_Hirose:Hirose_DF13-04P-1.25DSA_1x04_P1.25mm_Vertical
- removed J8: S4B, Connector_Hirose:Hirose_DF13-04P-1.25DSA_1x04_P1.25mm_Vertical
- removed R25, R29: 100K, Resistor_SMD:R_0805_2012Metric
- removed R26, R30: 1K, Resistor_SMD:R_0805_2012Metric
- removed R27, R31: 3K, Resistor_SMD:R_0805_2012Metric
- removed R28, R32: 120K, Resistor_SMD:R_0805_2012Metric
- removed U10, U9: LM358, Package_SO:SO-8_3.9x4.9mm_P1.27mm
Connections:
- U2 pad 5: /S4ATelem/TEMPOUT -> (no net)
- U2 pad 6: /S4ATelem/PHOTOOUT -> (no net)
- U2 pad 7: /S4BTelem/TEMPOUT -> (no net)
- U2 pad 8: /S4BTelem/PHOTOOUT -> (no net)

Commit message: Push KiCAD v6
Other:
- net class Default removed
