File: ECAD/Battery/BatteryMaster.kicad_pcb (KiCad board)
At the start: 2 copper layers, 126 parts, among them J1 BOOT, J2 SWD, Q1 IRF7458, Q10 Si4186DY, Q11 2N7002, Q12 IRF7458, Q13 Si4186DY, Q14 2N7002, Q15 IRF7458, Q16 Si4186DY, Q17 2N7002, Q18 IRF7458, Q19 Si4186DY, Q2 Si4186DY, Q20 2N7002, Q21 IRF7458, Q22 Si4186DY, Q3 IRF7458, Q4 Si4186DY, Q5 IRF7458, Q6 2N7002, Q7 IRF7458, Q8 IRF7425, Q9 Si4186DY, SW1 INHIBIT3, SW2 INHIBIT4, U1 LM358, U2 LT6106, U3 ADR4530, U4 MAX6369, U5 LTC4365TS8-1, U6 STM32F103C8Tx, U7 BQ29209, Y1 8MHz

Commit message: Add standard dimensions to batt
TODO: replace footprint of 18650
Parts:
- BT1, BT4: footprint Battery:BatteryHolder_Keystone_1042_1x18650 -> Battery:BatteryHolder_MPD_BH-18650-PC2
- BT2: renamed from BT3; footprint Battery:BatteryHolder_Keystone_1042_1x18650 -> Battery:BatteryHolder_MPD_BH-18650-PC2
- BT3: renamed from BT2; footprint Battery:BatteryHolder_Keystone_1042_1x18650 -> Battery:BatteryHolder_MPD_BH-18650-PC2
- moved BT4 199.6 mm to (283.7, 68.2), turned to 270 degrees
- moved BT3 172.2 mm to (262.9, 68.2), turned to 270 degrees
- moved BT1 157.8 mm to (221.2, 140.2), turned to 90 degrees
- moved BT2 157.3 mm to (242.1, 140.2), turned to 90 degrees
- moved Q10 153.9 mm to (-13.7, 95.5)
- moved C6 146.0 mm to (24.7, 99.7)
- moved J2 146.0 mm to (7.47, 64.8)
- moved R20 146.0 mm to (20.2, 102.7)
- moved U2 146.0 mm to (24.5, 95.9)
- moved C14 146.0 mm to (7.37, 76.2)
- moved C15 146.0 mm to (11.8, 76.2)
- moved C16 146.0 mm to (16.3, 76.2)
- moved C17 146.0 mm to (25.4, 77.0)
- moved C18 146.0 mm to (90.1, 89.5)
- moved C19 146.0 mm to (90.1, 108.0)
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- renumbered H2 to H1, H1 to H2
Connections:
- H2 pad 29: /SCK -> (no net)
- H2 pad 30: (no net) -> /SCK
- H2 pad 31: /MISO -> (no net)
- H2 pad 32: (no net) -> /MISO
- H2 pad 33: /MOSI -> (no net)
- H2 pad 34: (no net) -> /MOSI
- H2 pad 35: /SS -> (no net)
- H2 pad 36: (no net) -> /SS
- R1 pad 1: (no net) -> BCR_OUT
Routing:
- net Net-(BT1-Pad2): track 0.00 -> 62.5 mm
- net Net-(BT3-Pad2): track 0.00 -> 20.8 mm
- net Net-(BT1-Pad1): track 0.00 -> 20.8 mm
Other:
- board outline added: 90.3 x 95.9 mm

Commit message: 254 footprint
Parts:
- BT1, BT2, BT3, BT4: footprint Battery:BatteryHolder_MPD_BH-18650-PC2 -> footprints:Keystone-254
- C1, C10, C11, C12, C13, C14, C15, C16, C17, C18, C19, C2, C20, C21, C3, C4, C5, C6, C7, C8, C9, F1, F2, J1, J2, Q1, Q10, Q11, Q12, Q13, Q14, Q15, Q16, Q17, Q18, Q19, Q2, Q20, Q21, Q22, Q3, Q4, Q5, Q6, Q7, Q8, Q9, R1, R10, R11, R12, R13, R14, R15, R16, R17, R18, R19, R2, R20, R21, R22, R23, R24, R25, R26, R27, R28, R29, R3, R30, R31, R32, R33, R34, R35, R36, R37, R38, R39, R4, R40, R41, R42, R43, R44, R45, R46, R47, R48, R49, R5, R50, R51, R52, R53, R54, R55, R6, R7, R8, R9, SW1, SW2, TH1, TH2, TH3, TH4, U1, U2, U3, U4, U5, U6, U7, Y1: moved to B.Cu
- moved Q10 126.6 mm to (112.8, 90.9), turned to 180 degrees
- moved R31 99.7 mm to (-0.26, 77.7), turned to 180 degrees
- moved R38 99.7 mm to (-0.26, 96.2), turned to 180 degrees
- moved R44 99.7 mm to (-0.26, 114.6), turned to 180 degrees
- moved R52 99.7 mm to (-0.26, 59.3), turned to 180 degrees
- moved R29 90.9 mm to (4.15, 77.7), turned to 180 degrees
- moved R32 90.9 mm to (4.15, 80.7), turned to 180 degrees
- moved R36 90.9 mm to (4.15, 96.2), turned to 180 degrees
- moved R37 90.9 mm to (4.15, 99.1), turned to 180 degrees
- moved R43 90.9 mm to (4.15, 117.5), turned to 180 degrees
- moved R46 90.9 mm to (4.15, 114.6), turned to 180 degrees
- moved R50 90.9 mm to (4.15, 59.3), turned to 180 degrees
- moved R53 90.9 mm to (4.15, 62.3), turned to 180 degrees
- moved R34 90.1 mm to (4.55, 84.9), turned to 180 degrees
- moved R35 90.1 mm to (4.55, 103.4), turned to 180 degrees
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Routing:
- net Net-(BT1-Pad2): track 62.5 -> 0.00 mm
- net Net-(BT1-Pad1): track 20.8 -> 0.00 mm
- net Net-(BT3-Pad2): track 20.8 -> 1.99 mm

Commit message: 18500 footprint
Parts:
- BT1, BT2, BT3, BT4: value 18650 -> 18500
- moved BT3 135.1 mm to (165.9, 103.3)
- moved BT4 135.1 mm to (186.7, 103.3)
- moved BT1 106.2 mm to (121.7, 103.1)
- moved BT2 106.2 mm to (142.5, 103.1)

Commit message: welded 18650
Parts:
- BT1, BT2, BT3, BT4: footprint footprints:Keystone-254 -> footprints:18650-weld
- moved R44 185.6 mm to (174.0, 178.6), turned to 270 degrees
- moved R42 184.1 mm to (181.2, 173.8), turned to 270 degrees
- moved R43 181.8 mm to (177.0, 174.2), turned to 270 degrees
- moved R45 180.8 mm to (184.2, 169.3), turned to 270 degrees
- moved R46 180.0 mm to (174.0, 174.2), turned to 270 degrees
- moved C20 178.7 mm to (181.2, 169.3), turned to 270 degrees
- moved R48 176.6 mm to (185.8, 164.9), turned to 270 degrees
- moved R38 176.3 mm to (155.6, 178.6), turned to 270 degrees
- moved TH3 174.8 mm to (174.9, 169.6), turned to 270 degrees
- moved Q17 173.8 mm to (182.0, 164.9), turned to 270 degrees
- moved R35 173.2 mm to (162.8, 173.8), turned to 270 degrees
- moved R37 171.7 mm to (158.5, 174.2), turned to 270 degrees
- moved R31 170.5 mm to (137.2, 178.6), turned to 270 degrees
- moved R36 170.3 mm to (155.6, 174.2), turned to 270 degrees
- moved R41 169.0 mm to (165.8, 169.3), turned to 270 degrees
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Routing:
- net Net-(BT1-Pad2): track 0.00 -> 60.2 mm
- net Net-(BT3-Pad2): track 1.99 -> 22.5 mm
- net Net-(BT1-Pad1): track 0.00 -> 20.1 mm
- net Net-(F1-Pad1): track 0.00 -> 10.3 mm
- net Net-(C9-Pad1): track 0.00 -> 6.40 mm
- net Net-(C16-Pad1): track 0.00 -> 3.28 mm

Commit message: wip: refine shunt resistor selection, add inhibits
Parts:
- J2: footprint Connector_PinHeader_2.54mm:PinHeader_1x04_P2.54mm_Horizontal -> Connector_PinHeader_2.54mm:PinHeader_1x04_P2.54mm_Vertical; moved to F.Cu
- moved J2 106.4 mm to (194.3, 87.9), turned to 0 degrees
- moved J1 87.9 mm to (163.3, 88.6)
- moved C15 22.8 mm to (137.9, 105.9)
- moved C16 22.8 mm to (138.9, 134.4)
- moved C9 22.8 mm to (128.5, 133.6)
- moved R25 22.8 mm to (127.8, 109.5)
- moved C14 22.8 mm to (132.1, 105.9)
- moved F1 22.8 mm to (123.4, 112.8)
- moved F2 22.8 mm to (123.4, 126.0)
- moved Q10 22.8 mm to (126.0, 119.4)
- moved R21 22.8 mm to (128.5, 129.5)
- moved R26 22.8 mm to (135.1, 101.1)
- moved R22 22.8 mm to (132.1, 127.5)
- moved R27 22.8 mm to (140.7, 101.1)
- moved U7 22.8 mm to (134.4, 131.8)
Connections:
- net Net-(BT3-Pad2) renamed -BATT
Routing:
- net -BATT: track 22.5 -> 25.1 mm

Commit message: footprint and layout update
Parts:
- removed the C5 at (80.5, 120.2)
- removed the C6 at (74.3, 95.1)
- removed the R13 at (87.3, 107.0)
- removed the R14 at (91.7, 107.0)
- removed the R23 at (74.1, 98.1)
- removed the U3 at (81.2, 77.4)
- added C1: 10uF, Capacitor_SMD:C_0805_2012Metric, B.Cu at (87.9, 144.8)
- added C12: 0.1uF, Capacitor_SMD:C_0805_2012Metric, B.Cu at (87.9, 147.8)
- added C2: 0.1uF, Capacitor_SMD:C_0805_2012Metric, B.Cu at (77.5, 138.7)
- added C8: 0.1uF, Capacitor_SMD:C_0805_2012Metric, B.Cu at (83.7, 141.3)
- added JP1: LTDIS, Connector_PinHeader_1.27mm:PinHeader_1x02_P1.27mm_Vertical, B.Cu at (83.6, 145.8)
- added JP2: LTDIS, Connector_PinHeader_1.27mm:PinHeader_1x02_P1.27mm_Vertical, B.Cu at (92.1, 152.3)
- added Q7: IRF7458, Package_SO:SOIC-8_3.9x4.9mm_P1.27mm, B.Cu at (71.1, 142.5)
- added Q8: IRF7458, Package_SO:SOIC-8_3.9x4.9mm_P1.27mm, B.Cu at (80.9, 150.7)
- added R11: 285K, Resistor_SMD:R_0805_2012Metric, B.Cu at (92.3, 144.9)
- added R12: 45K, Resistor_SMD:R_0805_2012Metric, B.Cu at (86.4, 138.4)
- added R25: 100R, Resistor_SMD:R_0805_2012Metric, B.Cu at (90.8, 138.8)
- added R6: 45K, Resistor_SMD:R_0805_2012Metric, B.Cu at (92.3, 147.8)
- added R7: 285K, Resistor_SMD:R_0805_2012Metric, B.Cu at (88.2, 141.8)
- added SW1: INHIBIT4, Connector_Hirose:Hirose_DF13-02P-1.25DSA_1x02_P1.25mm_Vertical, B.Cu at (77.8, 142.5)
- added U1: LM1117-3.3, Package_TO_SOT_SMD:SOT-223-3_TabPin2, B.Cu at (71.8, 149.8)
- R1: renamed from R3; value 10m -> 4m; footprint Resistor_SMD:R_2010_5025Metric -> Resistor_SMD:R_1206_3216Metric
- R24: value 22K -> 100K
- R4: value 100R -> 100K
- R5: value 2K -> 100K
- SW2: renamed from SW1; value INHIBIT3 -> INHIBIT5
- SW3: renamed from SW2; value INHIBIT4 -> INHIBIT6
- U2: value LT6106 -> INA181A2; footprint Package_TO_SOT_SMD:SOT-23-5 -> Package_TO_SOT_SMD:SOT-23-6
- moved R4 88.6 mm to (82.0, 138.4), turned to 0 degrees
- moved U2 61.7 mm to (87.6, 151.6), turned to 0 degrees
- moved R24 43.2 mm to (92.6, 141.9), turned to 0 degrees
- moved R5 39.7 mm to (95.2, 139.0), turned to 0 degrees
- renumbered BT3 to BT2, BT2 to BT3, C7 to C10, C8 to C11, C10 to C13, C11 to C14, C12 to C15, C13 to C16, C2 to C17, C17 to C18, C3 to C19, C18 to C20, C19 to C21, C20 to C22, C21 to C23, C9 to C3, C14 to C4, C15 to C5, C16 to C6, C4 to C7, C1 to C9, Q10 to Q1, Q2 to Q10, Q3 to Q11, Q4 to Q12, Q11 to Q13, Q12 to Q14, Q13 to Q15, Q14 to Q16, Q15 to Q17, Q16 to Q18, Q17 to Q19, Q5 to Q2, Q18 to Q20, Q19 to Q21, Q20 to Q22, Q21 to Q23, Q22 to Q24, Q7 to Q3, Q9 to Q4, Q6 to Q5, Q8 to Q6, Q1 to Q9, R27 to R10, R10 to R13, R11 to R14, R12 to R15, R17 to R16, R18 to R17, R19 to R18, R15 to R19, R21 to R2, R16 to R20, R1 to R21, R2 to R22, R20 to R23, R6 to R26, R7 to R27, R8 to R28, R9 to R29, R22 to R3, R28 to R30, R29 to R31, R30 to R32, R31 to R33, R32 to R34, R33 to R35, R34 to R36, R35 to R37, R36 to R38, R37 to R39, R38 to R40, R39 to R41, R40 to R42, R41 to R43, R42 to R44, R43 to R45, R44 to R46, R45 to R47, R46 to R48, R47 to R49, R48 to R50, R49 to R51, R50 to R52, R51 to R53, R52 to R54, R53 to R55, R54 to R56, R55 to R57, R25 to R8, R26 to R9, U7 to U3, U1 to U4, U4 to U5, U5 to U6, U6 to U7
Connections:
- C17 pad 2: Net-(C2-Pad2) -> Net-(C17-Pad2)
- C19 pad 1: Net-(C3-Pad1) (its old number) -> Net-(C19-Pad1)
- F1 pad 2: Net-(F1-Pad2) -> /BAT_RAW
- H1 pad 35: PCM_IN -> BCR_OUT
- H1 pad 36: PCM_IN -> BCR_OUT
- Q10 pad 4: Net-(C3-Pad1) (its old number) -> Net-(C19-Pad1)
- Q11 pad 4: Net-(C2-Pad2) -> Net-(C17-Pad2)
- Q11 pad 5: Net-(C5-Pad1) -> /BAT_RAW
- Q11 pad 6: Net-(C5-Pad1) -> /BAT_RAW
- Q11 pad 7: Net-(C5-Pad1) -> /BAT_RAW
- Q11 pad 8: Net-(C5-Pad1) -> /BAT_RAW
- Q12 pad 4: Net-(C3-Pad1) (its old number) -> Net-(C19-Pad1)
- Q2 pad 1: Net-(Q5-Pad1) (its old number) -> Net-(C8-Pad1)
- Q2 pad 2: Net-(Q5-Pad1) (its old number) -> Net-(C8-Pad1)
- Q2 pad 3: Net-(Q5-Pad1) (its old number) -> Net-(C8-Pad1)
- Q2 pad 4: Net-(Q5-Pad4) -> Net-(Q2-Pad4)
- Q2 pad 5: Net-(C5-Pad1) -> Net-(Q2-Pad5)
- Q2 pad 6: Net-(C5-Pad1) -> Net-(Q2-Pad5)
- Q2 pad 7: Net-(C5-Pad1) -> Net-(Q2-Pad5)
- Q2 pad 8: Net-(C5-Pad1) -> Net-(Q2-Pad5)
- Q3 pad 1: Net-(Q5-Pad1) (its old number) -> Net-(C8-Pad1)
- Q3 pad 2: Net-(Q5-Pad1) (its old number) -> Net-(C8-Pad1)
- Q3 pad 3: Net-(Q5-Pad1) (its old number) -> Net-(C8-Pad1)
- Q3 pad 4: Net-(Q5-Pad4) -> Net-(Q3-Pad4)
- Q4 pad 1: Net-(F1-Pad2) -> Net-(Q4-Pad1)
- Q4 pad 2: Net-(F1-Pad2) -> Net-(Q4-Pad1)
- Q4 pad 3: Net-(F1-Pad2) -> Net-(Q4-Pad1)
- Q9 pad 4: Net-(C2-Pad2) -> Net-(C17-Pad2)
- Q9 pad 5: Net-(Q1-Pad5) -> Net-(Q8-Pad5)
- Q9 pad 6: Net-(Q1-Pad5) -> Net-(Q8-Pad5)
- Q9 pad 7: Net-(Q1-Pad5) -> Net-(Q8-Pad5)
- Q9 pad 8: Net-(Q1-Pad5) -> Net-(Q8-Pad5)
- R1 pad 1: Net-(Q1-Pad5) -> Net-(Q2-Pad5)
- R17 pad 2: -BATT -> GND
- R21 pad 1: BCR_OUT -> Net-(Q4-Pad1)
- R24 pad 1: /TELEM_IBATDIR -> Net-(C12-Pad2)
- R24 pad 2: Net-(R23-Pad1) -> GND
- R26 pad 1: Net-(C2-Pad2) -> Net-(JP1-Pad2)
- R29 pad 2: Net-(C3-Pad1) (its old number) -> Net-(JP2-Pad1)
- R4 pad 2: BCR_OUT -> GND
- R5 pad 1: /TELEM_IBAT -> Net-(R4-Pad1)
- R5 pad 2: GND -> +3.3VA
- SW2 pad 2: Net-(C2-Pad2) -> Net-(C17-Pad2)
- SW3 pad 1: Net-(C3-Pad1) (its old number) -> Net-(C19-Pad1)
- U2 pad 3: Net-(R4-Pad1) -> BCR_OUT
- U2 pad 4: Net-(Q1-Pad5) -> Net-(Q2-Pad5)
- U2 pad 5: BCR_OUT -> Net-(R4-Pad1)
- U4 pad 1: /TELEM_IBATDIR -> Net-(Q3-Pad4)
- U4 pad 2: Net-(Q1-Pad5) -> Net-(R6-Pad2)
- U4 pad 3: BCR_OUT -> /TELEM_IBAT
- U4 pad 5: /TELEM_IBAT -> Net-(R11-Pad2)
- U4 pad 6: Net-(R13-Pad2) -> /TELEM_IBAT
- U4 pad 7: Net-(Q5-Pad4) -> Net-(Q2-Pad4)
- U4 pad 8: BCR_OUT -> Net-(C8-Pad1)
- U6 pad 4: -BATT -> GND
- U6 pad 7: Net-(F1-Pad2) -> Net-(Q4-Pad1)
- U7 pad 16: Net-(R23-Pad1) -> (no net)

Commit message: Restandardize stack headers a bit
Connections:
- H1 pad 10: GND -> (no net)
- H1 pad 21: (no net) -> GND
- H1 pad 22: (no net) -> GND
- H1 pad 23: GND -> (no net)
- H1 pad 24: GND -> (no net)
- H1 pad 25: +BATT -> +5V
- H1 pad 26: +BATT -> +5V
- H1 pad 27: +5V -> +3V3
- H1 pad 28: +5V -> +3V3
- H1 pad 29: +3V3 -> GND
- H1 pad 30: +3V3 -> GND
- H1 pad 39: BCR_OUT -> (no net)
- H1 pad 40: BCR_OUT -> (no net)
- H1 pad 43: GND -> BCR_OUT
- H1 pad 44: GND -> BCR_OUT
- H1 pad 45: VUSB -> +BATT
- H1 pad 46: VUSB -> +BATT
- H1 pad 9: GND -> (no net)
- H2 pad 30: /SCK -> (no net)
- H2 pad 32: /MISO -> (no net)
- H2 pad 33: (no net) -> /SCK
- H2 pad 34: /MOSI -> (no net)
- H2 pad 35: (no net) -> /MISO
- H2 pad 36: /SS -> (no net)
- H2 pad 37: (no net) -> /MOSI
- H2 pad 39: (no net) -> /SS

Commit message: moving some connectors
Parts:
- H1, H2: moved to B.Cu
- R42, R49, R56, SW1, SW2, SW3, TH1: moved to F.Cu
- moved U5 100.9 mm to (168.9, 81.3)
- moved Q5 100.2 mm to (186.7, 80.0)
- moved Q6 89.5 mm to (179.1, 78.7)
- moved R49 34.8 mm to (194.9, 136.5), turned to 180 degrees
- moved SW1 32.9 mm to (109.2, 132.7), turned to 90 degrees
- moved R42 29.6 mm to (171.4, 144.1), turned to 90 degrees
- moved TH1 24.6 mm to (151.1, 144.1), turned to 90 degrees
- moved R56 23.6 mm to (130.8, 144.1), turned to 90 degrees
- moved H1 2.54 mm to (120.8, 60.5), turned to 270 degrees
- moved H2 2.54 mm to (120.8, 65.6), turned to 270 degrees
