File: ECAD/Battery/BatteryMaster.sch (KiCad schematic (older format))
At the start: 84 parts, among them J1 BOOT, J2 SWD, Q1 IRF7458, Q10 Si4186DY, Q2 Si4186DY, Q3 IRF7458, Q4 Si4186DY, Q5 IRF7458, Q6 2N7002, Q7 IRF7458, Q8 IRF7425, Q9 Si4186DY, SW1 INHIBIT5, SW2 INHIBIT6, U1 LM358, U2 INA181A2, U3 ADR4530, U4 MAX6369, U5 LTC4365TS8-1, U6 STM32F103C8Tx, U7 BQ29209, Y1 8MHz

Commit message: Finish revamp of protection layout
Parts:
- removed C6: 0.1uF, Capacitor_SMD:C_0805_2012Metric, symbol Device:C
- removed R13: 24K, Resistor_SMD:R_0805_2012Metric, symbol Device:R
- removed R14: 16K, Resistor_SMD:R_0805_2012Metric, symbol Device:R
- removed U3: ADR4530, Package_SO:SOIC-8_3.9x4.9mm_P1.27mm, symbol Reference_Voltage:ADR4530
- added C?: 10uF, Capacitor_SMD:C_0805_2012Metric, symbol Device:C
- added C? (x2): 0.1uF, Capacitor_SMD:C_0805_2012Metric, symbol Device:C
- added R? (x2): 100K, Resistor_SMD:R_0805_2012Metric, symbol Device:R
- added R? (x2): 45K, Resistor_SMD:R_0805_2012Metric, symbol Device:R
- added R? (x2): 285K, Resistor_SMD:R_0805_2012Metric, symbol Device:R
- added unit 1 of U1
- added unit 3 of U1
Connections:
- net labels added: +3.3VA, BAT_RAW
- wire segments 275 -> 299
Other:
- note added: "50V/V gain\n200mV/A, 0A = 1.65V out\nDischarge Vout < 1.65\nCharge Vout > 1.65"
- note added: "6A Bidirectional OCP"
- note added: "Charge"
- note added: "Discharge"
- note added: "V and I Telemetry, OCP, OVP"
- note removed: "V and I Telemetry"
- note removed: "~~6A Bidirectional OCP"
- moved on the sheet: BT1, BT2, BT3, BT4, C1, C14, C15, C16, C2, C3, C4, C9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

Commit message: footprint and layout update
Parts:
- removed R23: 10K, Resistor_SMD:R_0805_2012Metric, symbol Device:R
- removed R24: 22K, Resistor_SMD:R_0805_2012Metric, symbol Device:R
- JP1, JP2: renamed from JP?; footprint (none) -> Connector_PinHeader_1.27mm:PinHeader_1x02_P1.27mm_Vertical
- U1: renamed from U?; footprint (none) -> Package_TO_SOT_SMD:SOT-223-3_TabPin2
- U4: renamed from U1; footprint (none) -> Package_SO:SO-8_3.9x4.9mm_P1.27mm
- gave numbers to parts that had none: 15
- renumbered BT3 to BT2, BT2 to BT3, C7 to C10, C8 to C11, C10 to C13, C11 to C14, C12 to C15, C13 to C16, C2 to C17, C17 to C18, C3 to C19, C9 to C3, C14 to C4, C15 to C5, C16 to C6, C4 to C7, C1 to C9, Q10 to Q1, Q2 to Q10, Q3 to Q11, Q4 to Q12, Q5 to Q2, Q7 to Q3, Q9 to Q4, Q6 to Q5, Q8 to Q6, Q1 to Q9, R3 to R1, R27 to R10, R10 to R13, R11 to R14, R12 to R15, R17 to R16, R18 to R17, R19 to R18, R15 to R19, R21 to R2, R16 to R20, R1 to R21, R2 to R22, R20 to R23, R6 to R26, R7 to R27, R8 to R28, R9 to R29, R22 to R3, R25 to R8, R26 to R9, SW1 to SW2, SW2 to SW3, U7 to U3, U1 to U4, U4 to U5, U5 to U6, U6 to U7

Commit message: Restandardize stack headers a bit
Connections:
- net +3V3: now also H1.27 (Pin_27), H1.28 (Pin_28); no longer H1.29 (Pin_29), H1.30 (Pin_30)
- net +5V: now also H1.25 (Pin_25), H1.26 (Pin_26); no longer H1.27 (Pin_27), H1.28 (Pin_28)
- net +BATT: now also H1.45 (Pin_45), H1.46 (Pin_46); no longer H1.25 (Pin_25), H1.26 (Pin_26)
- net BCR_OUT: now also H1.43 (Pin_43), H1.44 (Pin_44); no longer H1.39 (Pin_39), H1.40 (Pin_40)
- net GND: now also H1.21 (Pin_21), H1.22 (Pin_22), H1.29 (Pin_29), H1.30 (Pin_30); no longer H1.10 (Pin_10), H1.23 (Pin_23), H1.24 (Pin_24), H1.43 (Pin_43), H1.44 (Pin_44), H1.9 (Pin_9)
- net MISO: now also H2.35 (Pin_35); no longer H2.32 (Pin_32)
- net MOSI: now also H2.37 (Pin_37); no longer H2.34 (Pin_34)
- net SCK: now also H2.33 (Pin_33); no longer H2.30 (Pin_30)
- net SCL: now also H2.43 (Pin_43); no longer H2.44 (Pin_44)
- net SDA: now also H2.41 (Pin_41); no longer H2.42 (Pin_42)
- net SS: now also H2.39 (Pin_39); no longer H2.36 (Pin_36)
- net SW1: now also H1.9 (Pin_9); no longer H1.11 (Pin_11)
- net SW10: now also H1.18 (Pin_18); no longer H1.19 (Pin_19)
- net SW11: now also H1.19 (Pin_19); no longer H1.22 (Pin_22)
- net SW12: now also H1.20 (Pin_20); no longer H1.21 (Pin_21)
- net SW2: now also H1.10 (Pin_10); no longer H1.12 (Pin_12)
- net SW3: now also H1.11 (Pin_11); no longer H1.13 (Pin_13)
- net SW4: now also H1.12 (Pin_12); no longer H1.14 (Pin_14)
- net SW5: now also H1.13 (Pin_13); no longer H1.16 (Pin_16)
- net SW6: now also H1.14 (Pin_14); no longer H1.15 (Pin_15)
- net SW7: now also H1.15 (Pin_15); no longer H1.18 (Pin_18)
- net SW8: now also H1.16 (Pin_16); no longer H1.17 (Pin_17)
- net SW9: now also H1.17 (Pin_17); no longer H1.20 (Pin_20)
- net VUSB: now also H2.32 (Pin_32); no longer H1.45 (Pin_45), H1.46 (Pin_46)
- no-connect marks 19 -> 23
Other:
- moved on the sheet: H1, H2

Commit message: downspec heater mosfets
Parts:
- renumbered H2 to H1, H1 to H2
Changed lines of the file:
@@
 BCR_OUT
 $Comp
-L power:+BATT #PWR06
+L power:+BATT #PWR09
 U 1 1 6209177A
 P 2450 7400
-AR Path="/6209177A" Ref="#PWR06"  Part="1"
+AR Path="/6209177A" Ref="#PWR09"  Part="1"
 AR Path="/61BD4B7D/6209177A" Ref="#PWR?"  Part="1"
-F 0 "#PWR06" H 2450 7250 50  0001 C CNN
+F 0 "#PWR09" H 2450 7250 50  0001 C CNN
 F 1 "+BATT" V 2450 7500 50  0000 L CNN
 F 2 "" H 2450 7400 50  0001 C CNN
@@
 $EndComp
 $Comp
-L power:+BATT #PWR01
+L power:+BATT #PWR04
 U 1 1 62091780
 P 1950 7400
-AR Path="/62091780" Ref="#PWR01"  Part="1"
+AR Path="/62091780" Ref="#PWR04"  Part="1"
 AR Path="/61BD4B7D/62091780" Ref="#PWR?"  Part="1"
-F 0 "#PWR01" H 1950 7250 50  0001 C CNN
+F 0 "#PWR04" H 1950 7250 50  0001 C CNN
 F 1 "+BATT" V 1950 7500 50  0000 L CNN
 F 2 "" H 1950 7400 50  0001 C CNN
@@
 	1250 1650 1600 1650
 $Comp
-L power:GND #PWR04
+L power:GND #PWR01
 U 1 1 61FCA066
 P 1250 1650
-F 0 "#PWR04" H 1250 1400 50  0001 C CNN
+F 0 "#PWR01" H 1250 1400 50  0001 C CNN
 F 1 "GND" H 1255 1477 50  0000 C CNN
 F 2 "" H 1250 1650 50  0001 C CNN
@@
 Connection ~ 1600 1200
 $Comp
-L power:+3.3VA #PWR09
+L power:+3.3VA #PWR06
 U 1 1 6204AE89
 P 2350 1200
-F 0 "#PWR09" H 2350 1050 50  0001 C CNN
+F 0 "#PWR06" H 2350 1050 50  0001 C CNN
 F 1 "+3.3VA" H 2365 1373 50  0000 C CNN
 F 2 "" H 2350 1200 50  0001 C CNN
@@
 	2850 6600 2850 6700
 $Comp
-L Connector_Generic:Conn_02x26_Odd_Even H2
+L Connector_Generic:Conn_02x26_Odd_Even H1
 U 1 1 6209174D
 P 950 6400
-AR Path="/6209174D" Ref="H2"  Part="1"
+AR Path="/6209174D" Ref="H1"  Part="1"
 AR Path="/61BD4B7D/6209174D" Ref="H?"  Part="1"
-F 0 "H2" H 1000 7817 50  0000 C CNN
+F 0 "H1" H 1000 7817 50  0000 C CNN
 F 1 "Stack Header 2" H 1000 7726 50  0000 C CNN
 F 2 "Connector_PinSocket_2.54mm:PinSocket_2x26_P2.54mm_Vertical" H 950 6400 50  0001 C CNN
@@
 $EndComp
 $Comp
-L Connector_Generic:Conn_02x26_Odd_Even H1
+L Connector_Generic:Conn_02x26_Odd_Even H2
 U 1 1 620917C1
 P 2150 6400
-AR Path="/620917C1" Ref="H1"  Part="1"
+AR Path="/620917C1" Ref="H2"  Part="1"
 AR Path="/61BD4B7D/620917C1" Ref="H?"  Part="1"
-F 0 "H1" H 2200 7817 50  0000 C CNN
+F 0 "H2" H 2200 7817 50  0000 C CNN
 F 1 "Stack Header 1" H 2200 7726 50  0000 C CNN
 F 2 "Connector_PinSocket_2.54mm:PinSocket_2x26_P2.54mm_Vertical" H 2150 6400 50  0001 C CNN

Commit message: Finish routing vbat power path
Parts:
- added C24: 10uF, Capacitor_SMD:C_0805_2012Metric, symbol Device:C
- added Q25: Si4186DY, Package_SO:SOIC-8_3.9x4.9mm_P1.27mm, symbol Transistor_FET:Si4162DY
- added U8: LTC4359-MS8, Package_SO:MSOP-8_3x3mm_P0.65mm, symbol Power_Management:LTC4359-MS8
- H1, H2: footprint Connector_PinSocket_2.54mm:PinSocket_2x26_P2.54mm_Vertical -> footprints:PinSocket_2x26_P2.54mm_Vertical
Connections:
- net BCR_OUT: now also Q25.1 (S), Q25.2 (S), Q25.3 (S), U8.2 (SRC), U8.4 (IN), U8.5 (~SHDN); no longer H2.35 (Pin_35), H2.36 (Pin_36)
- net GND: now also C24.2, U8.6 (Vss), U8.7 (NC)
- net at C12.2, Q7.4 (G), Q8.4 (G)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: now also SW1.1 (A); no longer SW1.2 (B)
- net at R25.2: now also SW1.2 (B); no longer SW1.1 (A)
- new net: Q25.4 (G), U8.1 (GATE)
- new net PCM_IN: C24.1, H2.35 (Pin_35), H2.36 (Pin_36), Q25.5 (D), Q25.6 (D), Q25.7 (D), Q25.8 (D), U8.8 (OUT)
Other:
- note added: "Ideal Diode"
- moved on the sheet: C10, C11, C13, C14, C15, C16, C18, C7, H1, H2, J1, J2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

Commit message: swd with debug, and replace boot jumper with solder jumper
Parts:
- removed J1: BOOT, Connector_PinHeader_2.54mm:PinHeader_1x03_P2.54mm_Vertical, symbol Connector:Conn_01x03_Male
- removed J2: SWD, Connector_PinHeader_2.54mm:PinHeader_1x04_P2.54mm_Vertical, symbol Connector:Conn_01x04_Male
- added J1: SWD/DEBUG, Connector_PinHeader_2.54mm:PinHeader_1x06_P2.54mm_Vertical, symbol Connector:Conn_01x06_Male
- added JP1: BOOT, Jumper:SolderJumper-3_P1.3mm_Open_Pad1.0x1.5mm, symbol Jumper:SolderJumper_3_Open
- renumbered C9 to C10, C10 to C11, C11 to C12, C12 to C13, C13 to C14, C14 to C15, C17 to C16, C15 to C17, C16 to C18, C18 to C20, C8 to C7, C7 to C8, C24 to C9, JP1 to JP2, JP2 to JP3, Q9 to Q10, Q10 to Q11, Q11 to Q12, Q12 to Q13, Q25 to Q4, Q4 to Q5, Q5 to Q6, Q6 to Q7, Q7 to Q8, Q8 to Q9, R16 to R15, R17 to R16, R15 to R17, R24 to R23, R23 to R24, U8 to U5, U5 to U6, U6 to U7, U7 to U8
Connections:
- net GND: now also J1.4 (Pin_4), JP1.1 (A)
- net SWDCLK: now also J1.3 (Pin_3)
- net SWDIO: now also J1.2 (Pin_2)
- net VDD: now also J1.1 (Pin_1), JP1.3 (B)
- net at R17.2: now also JP1.2 (C)
- net D-: now reaches U8.32 (PA11)
- net D-: now also J1.5 (Pin_5)
- net D+: now reaches U8.33 (PA12)
- net D+: now also J1.6 (Pin_6)
Other:
- moved on the sheet: R17

Commit message: place heater and thermistor stuff
Parts:
- added Q26: Si4186DY, Package_SO:SOIC-8_3.9x4.9mm_P1.27mm, symbol Transistor_FET:Si4162DY
Connections:
- net -BATT: now also Q26.1 (S), Q26.2 (S), Q26.3 (S); no longer Q1.1 (S), Q1.2 (S), Q1.3 (S)
- net at Q1.4 (G), R3.1: now also Q26.4 (G)
- new net: Q1.1 (S), Q1.2 (S), Q1.3 (S), Q26.5 (D), Q26.6 (D), Q26.7 (D), Q26.8 (D)
Other:
- note added: "Redundant mosfets"
Changed lines of the file:
@@
 	1800 3550 2200 3550
 Connection ~ 2050 2950
-Wire Wire Line
-	1500 3750 1500 4400
 $Comp
 L Transistor_FET:Si4162DY Q1
@@
 Wire Wire Line
 	7500 5350 7650 5350
+$Comp
+L Transistor_FET:Si4162DY Q26
+U 1 1 61F5EB95
+P 1600 3950
+F 0 "Q26" H 1805 3996 50  0000 L CNN
+F 1 "Si4186DY" H 1805 3905 50  0000 L CNN
+F 2 "Package_SO:SOIC-8_3.9x4.9mm_P1.27mm" H 1800 3850 50  0001 L CNN
+F 3 "http://www.vishay.com/docs/68967/si4162dy.pdf" H 1600 3950 50  0001 L CNN
+	1    1600 3950
+	-1   0    0    -1
+$EndComp
+Wire Wire Line
+	1500 4400 1500 4150
+Wire Wire Line
+	1800 3950 1800 3550
+Connection ~ 1800 3550
+Text Notes 1150 4500 0    50   ~ 0
+Redundant mosfets
 $EndSCHEMATC

Commit message: Round off some corners and set up eps board for routing
Parts:
- renumbered H2 to H1, H1 to H2
Changed lines of the file:
@@
 	3250 6600 3250 6700
 $Comp
-L Connector_Generic:Conn_02x26_Odd_Even H1
+L Connector_Generic:Conn_02x26_Odd_Even H2
 U 1 1 6209174D
 P 1350 6400
-AR Path="/6209174D" Ref="H1"  Part="1"
+AR Path="/6209174D" Ref="H2"  Part="1"
 AR Path="/61BD4B7D/6209174D" Ref="H?"  Part="1"
-F 0 "H1" H 1400 7817 50  0000 C CNN
+F 0 "H2" H 1400 7817 50  0000 C CNN
 F 1 "Stack Header 2" H 1400 7726 50  0000 C CNN
 F 2 "footprints:PinSocket_2x26_P2.54mm_Vertical" H 1350 6400 50  0001 C CNN
@@
 $EndComp
 $Comp
-L Connector_Generic:Conn_02x26_Odd_Even H2
+L Connector_Generic:Conn_02x26_Odd_Even H1
 U 1 1 620917C1
 P 2550 6400
-AR Path="/620917C1" Ref="H2"  Part="1"
+AR Path="/620917C1" Ref="H1"  Part="1"
 AR Path="/61BD4B7D/620917C1" Ref="H?"  Part="1"
-F 0 "H2" H 2600 7817 50  0000 C CNN
+F 0 "H1" H 2600 7817 50  0000 C CNN
 F 1 "Stack Header 1" H 2600 7726 50  0000 C CNN
 F 2 "footprints:PinSocket_2x26_P2.54mm_Vertical" H 2550 6400 50  0001 C CNN
