File: ECAD/Battery/Heater+Thermistor.sch (KiCad schematic (older format))
At the start: 12 parts, among them Q11 2N7002, Q12 IRF7458, Q13 Si4186DY

Commit message: footprint and layout update
Parts:
- renumbered C18 to C20, Q11 to Q13, Q12 to Q14, Q13 to Q15, R28 to R30, R29 to R31, R30 to R32, R31 to R33, R32 to R34, R33 to R35, R34 to R36

Commit message: downspec heater mosfets
Parts:
- removed Q14: IRF7458, Package_SO:SOIC-8_3.9x4.9mm_P1.27mm, symbol Transistor_FET:IRF7404
- removed Q15: Si4186DY, Package_SO:SOIC-8_3.9x4.9mm_P1.27mm, symbol Transistor_FET:Si4162DY
- added Q23: BSS83P, Package_TO_SOT_SMD:SOT-23, symbol Transistor_FET:BSS83P
- added Q24: BSN20, Package_TO_SOT_SMD:SOT-23, symbol Transistor_FET:BSN20
Connections:
- net +5V: now also Q23.2 (S)
- net GND: now also Q24.2 (S)
- net at R33.1, R34.1: now also Q24.1 (G)
- net at R35.2: now also Q24.3 (D)
- net at R35.1: now also Q23.3 (D)
- net at Q13.3 (D), R32.2: now also Q23.1 (G)
Changed lines of the file:
@@
 $Descr USLetter 11000 8500
 encoding utf-8
-Sheet 6 5
+Sheet 2 5
 Title "TJ Custom EPS"
 Date ""
@@
 Comment4 "Engineer: Alan Hsu"
 $EndDescr
-$Comp
-L Transistor_FET:Si4162DY Q?
-U 1 1 620332F7
-P 3750 3300
-AR Path="/61BD4B7D/620332F7" Ref="Q?"  Part="1"
-AR Path="/61BD4B7D/62026259/620332F7" Ref="Q?"  Part="1"
-AR Path="/61BD4B7D/62041525/620332F7" Ref="Q?"  Part="1"
-AR Path="/61BD4B7D/62045EF1/620332F7" Ref="Q?"  Part="1"
-AR Path="/61BD4B7D/6204A8C5/620332F7" Ref="Q?"  Part="1"
-AR Path="/62041525/620332F7" Ref="Q15"  Part="1"
-AR Path="/62045EF1/620332F7" Ref="Q18"  Part="1"
-AR Path="/6204A8C5/620332F7" Ref="Q21"  Part="1"
-AR Path="/62026259/620332F7" Ref="Q24"  Part="1"
-F 0 "Q24" H 3955 3346 50  0000 L CNN
-F 1 "Si4186DY" H 3955 3255 50  0000 L CNN
-F 2 "Package_SO:SOIC-8_3.9x4.9mm_P1.27mm" H 3950 3200 50  0001 L CNN
-F 3 "http://www.vishay.com/docs/68967/si4162dy.pdf" H 3750 3300 50  0001 L CNN
-	1    3750 3300
-	1    0    0    -1
-$EndComp
 $Comp
 L Device:R R?
@@
 $EndComp
 $Comp
-L Transistor_FET:IRF7404 Q?
-U 1 1 6203330F
-P 3750 2600
-AR Path="/61BD4B7D/6203330F" Ref="Q?"  Part="1"
-AR Path="/61BD4B7D/62026259/6203330F" Ref="Q?"  Part="1"
-AR Path="/61BD4B7D/62041525/6203330F" Ref="Q?"  Part="1"
-AR Path="/61BD4B7D/62045EF1/6203330F" Ref="Q?"  Part="1"
-AR Path="/61BD4B7D/6204A8C5/6203330F" Ref="Q?"  Part="1"
-AR Path="/62041525/6203330F" Ref="Q14"  Part="1"
-AR Path="/62045EF1/6203330F" Ref="Q17"  Part="1"
-AR Path="/6204A8C5/6203330F" Ref="Q20"  Part="1"
-AR Path="/62026259/6203330F" Ref="Q23"  Part="1"
-F 0 "Q23" H 3955 2646 50  0000 L CNN
-F 1 "IRF7458" H 3955 2555 50  0000 L CNN
-F 2 "Package_SO:SOIC-8_3.9x4.9mm_P1.27mm" H 3950 2525 50  0001 L CIN
-F 3 "http://www.infineon.com/dgdl/irf7404.pdf?fileId=5546d462533600a4015355fa2b5b1b9e" V 3750 2600 50  0001 L CNN
-	1    3750 2600
-	1    0    0    1
-$EndComp
-$Comp
 L power:+5V #PWR?
 U 1 1 62033315
@@
 Text HLabel 5950 3300 2    50   Input ~ 0
 TELEM_TBAT
+$Comp
+L Transistor_FET:BSN20 Q24
+U 1 1 61F204F1
+P 3750 3300
+AR Path="/62026259/61F204F1" Ref="Q24"  Part="1"
+AR Path="/62041525/61F204F1" Ref="Q15"  Part="1"
+AR Path="/62045EF1/61F204F1" Ref="Q18"  Part="1"
+AR Path="/6204A8C5/61F204F1" Ref="Q21"  Part="1"
+F 0 "Q24" H 3955 3346 50  0000 L CNN
+F 1 "BSN20" H 3955 3255 50  0000 L CNN
+F 2 "Package_TO_SOT_SMD:SOT-23" H 3950 3225 50  0001 L CIN
+F 3 "http://www.diodes.com/assets/Datasheets/ds31898.pdf" H 3750 3300 50  0001 L CNN
+	1    3750 3300
+	1    0    0    -1
+$EndComp
+$Comp
+L Transistor_FET:BSS83P Q23
+U 1 1 61F25B8B
+P 3750 2600
+AR Path="/62026259/61F25B8B" Ref="Q23"  Part="1"
+AR Path="/62041525/61F25B8B" Ref="Q14"  Part="1"
+AR Path="/62045EF1/61F25B8B" Ref="Q17"  Part="1"
+AR Path="/6204A8C5/61F25B8B" Ref="Q20"  Part="1"
+F 0 "Q23" H 3954 2554 50  0000 L CNN
+F 1 "BSS83P" H 3954 2645 50  0000 L CNN
+F 2 "Package_TO_SOT_SMD:SOT-23" H 3950 2525 50  0001 L CIN
+F 3 "http://www.farnell.com/datasheets/1835997.pdf" H 3750 2600 50  0001 L CNN
+	1    3750 2600
+	1    0    0    1
+$EndComp
 $EndSCHEMATC

Commit message: swd with debug, and replace boot jumper with solder jumper
Parts:
- renumbered C20 to C21, Q13 to Q14, Q23 to Q24, Q24 to Q25
Changed lines of the file:
@@
 AR Path="/61BD4B7D/62045EF1/62033315" Ref="#PWR?"  Part="1"
 AR Path="/61BD4B7D/6204A8C5/62033315" Ref="#PWR?"  Part="1"
-AR Path="/62041525/62033315" Ref="#PWR035"  Part="1"
-AR Path="/62045EF1/62033315" Ref="#PWR039"  Part="1"
-AR Path="/6204A8C5/62033315" Ref="#PWR043"  Part="1"
-AR Path="/62026259/62033315" Ref="#PWR047"  Part="1"
-F 0 "#PWR047" H 3850 2150 50  0001 C CNN
+AR Path="/62041525/62033315" Ref="#PWR036"  Part="1"
+AR Path="/62045EF1/62033315" Ref="#PWR040"  Part="1"
+AR Path="/6204A8C5/62033315" Ref="#PWR044"  Part="1"
+AR Path="/62026259/62033315" Ref="#PWR048"  Part="1"
+F 0 "#PWR048" H 3850 2150 50  0001 C CNN
 F 1 "+5V" H 3865 2473 50  0000 C CNN
 F 2 "" H 3850 2300 50  0001 C CNN
@@
 AR Path="/61BD4B7D/62045EF1/6203331C" Ref="Q?"  Part="1"
 AR Path="/61BD4B7D/6204A8C5/6203331C" Ref="Q?"  Part="1"
-AR Path="/62041525/6203331C" Ref="Q13"  Part="1"
-AR Path="/62045EF1/6203331C" Ref="Q16"  Part="1"
-AR Path="/6204A8C5/6203331C" Ref="Q19"  Part="1"
-AR Path="/62026259/6203331C" Ref="Q22"  Part="1"
-F 0 "Q22" H 3104 2846 50  0000 L CNN
+AR Path="/62041525/6203331C" Ref="Q14"  Part="1"
+AR Path="/62045EF1/6203331C" Ref="Q17"  Part="1"
+AR Path="/6204A8C5/6203331C" Ref="Q20"  Part="1"
+AR Path="/62026259/6203331C" Ref="Q23"  Part="1"
+F 0 "Q23" H 3104 2846 50  0000 L CNN
 F 1 "2N7002" H 3104 2755 50  0000 L CNN
 F 2 "Package_TO_SOT_SMD:SOT-23" H 3100 2725 50  0001 L CIN
@@
 AR Path="/61BD4B7D/62045EF1/62034CCA" Ref="#PWR?"  Part="1"
 AR Path="/61BD4B7D/6204A8C5/62034CCA" Ref="#PWR?"  Part="1"
-AR Path="/62041525/62034CCA" Ref="#PWR036"  Part="1"
-AR Path="/62045EF1/62034CCA" Ref="#PWR040"  Part="1"
-AR Path="/6204A8C5/62034CCA" Ref="#PWR044"  Part="1"
-AR Path="/62026259/62034CCA" Ref="#PWR048"  Part="1"
-F 0 "#PWR048" H 3850 3350 50  0001 C CNN
+AR Path="/62041525/62034CCA" Ref="#PWR037"  Part="1"
+AR Path="/62045EF1/62034CCA" Ref="#PWR041"  Part="1"
+AR Path="/6204A8C5/62034CCA" Ref="#PWR045"  Part="1"
+AR Path="/62026259/62034CCA" Ref="#PWR049"  Part="1"
+F 0 "#PWR049" H 3850 3350 50  0001 C CNN
 F 1 "GND" H 3855 3427 50  0000 C CNN
 F 2 "" H 3850 3600 50  0001 C CNN
@@
 AR Path="/61BD4B7D/62045EF1/62036CA9" Ref="C?"  Part="1"
 AR Path="/61BD4B7D/6204A8C5/62036CA9" Ref="C?"  Part="1"
-AR Path="/62041525/62036CA9" Ref="C20"  Part="1"
-AR Path="/62045EF1/62036CA9" Ref="C21"  Part="1"
-AR Path="/6204A8C5/62036CA9" Ref="C22"  Part="1"
-AR Path="/62026259/62036CA9" Ref="C23"  Part="1"
-F 0 "C23" H 6065 3496 50  0000 L CNN
+AR Path="/62041525/62036CA9" Ref="C21"  Part="1"
+AR Path="/62045EF1/62036CA9" Ref="C22"  Part="1"
+AR Path="/6204A8C5/62036CA9" Ref="C23"  Part="1"
+AR Path="/62026259/62036CA9" Ref="C24"  Part="1"
+F 0 "C24" H 6065 3496 50  0000 L CNN
 F 1 "0.1uF" H 6065 3405 50  0000 L CNN
 F 2 "Capacitor_SMD:C_0805_2012Metric" H 5988 3300 50  0001 C CNN
@@
 AR Path="/61BD4B7D/62045EF1/6203964D" Ref="#PWR?"  Part="1"
 AR Path="/61BD4B7D/6204A8C5/6203964D" Ref="#PWR?"  Part="1"
-AR Path="/62041525/6203964D" Ref="#PWR037"  Part="1"
-AR Path="/62045EF1/6203964D" Ref="#PWR041"  Part="1"
-AR Path="/6204A8C5/6203964D" Ref="#PWR045"  Part="1"
-AR Path="/62026259/6203964D" Ref="#PWR049"  Part="1"
-F 0 "#PWR049" H 5350 2850 50  0001 C CNN
+AR Path="/62041525/6203964D" Ref="#PWR038"  Part="1"
+AR Path="/62045EF1/6203964D" Ref="#PWR042"  Part="1"
+AR Path="/6204A8C5/6203964D" Ref="#PWR046"  Part="1"
+AR Path="/62026259/6203964D" Ref="#PWR050"  Part="1"
+F 0 "#PWR050" H 5350 2850 50  0001 C CNN
 F 1 "+3V3" H 5365 3173 50  0000 C CNN
 F 2 "" H 5350 3000 50  0001 C CNN
@@
 AR Path="/61BD4B7D/62045EF1/6203B674" Ref="#PWR?"  Part="1"
 AR Path="/61BD4B7D/6204A8C5/6203B674" Ref="#PWR?"  Part="1"
-AR Path="/62041525/6203B674" Ref="#PWR038"  Part="1"
-AR Path="/62045EF1/6203B674" Ref="#PWR042"  Part="1"
-AR Path="/6204A8C5/6203B674" Ref="#PWR046"  Part="1"
-AR Path="/62026259/6203B674" Ref="#PWR050"  Part="1"
-F 0 "#PWR050" H 5350 3350 50  0001 C CNN
+AR Path="/62041525/6203B674" Ref="#PWR039"  Part="1"
+AR Path="/62045EF1/6203B674" Ref="#PWR043"  Part="1"
+AR Path="/6204A8C5/6203B674" Ref="#PWR047"  Part="1"
+AR Path="/62026259/6203B674" Ref="#PWR051"  Part="1"
+F 0 "#PWR051" H 5350 3350 50  0001 C CNN
 F 1 "GND" H 5355 3427 50  0000 C CNN
 F 2 "" H 5350 3600 50  0001 C CNN
@@
 TELEM_TBAT
 $Comp
-L Transistor_FET:BSN20 Q24
+L Transistor_FET:BSN20 Q25
 U 1 1 61F204F1
 P 3750 3300
-AR Path="/62026259/61F204F1" Ref="Q24"  Part="1"
-AR Path="/62041525/61F204F1" Ref="Q15"  Part="1"
-AR Path="/62045EF1/61F204F1" Ref="Q18"  Part="1"
-AR Path="/6204A8C5/61F204F1" Ref="Q21"  Part="1"
-F 0 "Q24" H 3955 3346 50  0000 L CNN
+AR Path="/62026259/61F204F1" Ref="Q25"  Part="1"
+AR Path="/62041525/61F204F1" Ref="Q16"  Part="1"
+AR Path="/62045EF1/61F204F1" Ref="Q19"  Part="1"
+AR Path="/6204A8C5/61F204F1" Ref="Q22"  Part="1"
+F 0 "Q25" H 3955 3346 50  0000 L CNN
 F 1 "BSN20" H 3955 3255 50  0000 L CNN
 F 2 "Package_TO_SOT_SMD:SOT-23" H 3950 3225 50  0001 L CIN
@@
 $EndComp
 $Comp
-L Transistor_FET:BSS83P Q23
+L Transistor_FET:BSS83P Q24
 U 1 1 61F25B8B
 P 3750 2600
-AR Path="/62026259/61F25B8B" Ref="Q23"  Part="1"
-AR Path="/62041525/61F25B8B" Ref="Q14"  Part="1"
-AR Path="/62045EF1/61F25B8B" Ref="Q17"  Part="1"
-AR Path="/6204A8C5/61F25B8B" Ref="Q20"  Part="1"
-F 0 "Q23" H 3954 2554 50  0000 L CNN
+AR Path="/62026259/61F25B8B" Ref="Q24"  Part="1"
+AR Path="/62041525/61F25B8B" Ref="Q15"  Part="1"
+AR Path="/62045EF1/61F25B8B" Ref="Q18"  Part="1"
+AR Path="/6204A8C5/61F25B8B" Ref="Q21"  Part="1"
+F 0 "Q24" H 3954 2554 50  0000 L CNN
 F 1 "BSS83P" H 3954 2645 50  0000 L CNN
 F 2 "Package_TO_SOT_SMD:SOT-23" H 3950 2525 50  0001 L CIN

Commit message: place heater and thermistor stuff
Parts:
- TH1: footprint Connector_PinHeader_2.54mm:PinHeader_1x02_P2.54mm_Vertical -> Connector_Hirose:Hirose_DF13-02P-1.25DSA_1x02_P1.25mm_Vertical
Changed lines of the file:
@@
 F 0 "TH4" H 5448 3496 50  0000 L CNN
 F 1 "100K NTC" H 5448 3405 50  0000 L CNN
-F 2 "Connector_PinHeader_2.54mm:PinHeader_1x02_P2.54mm_Vertical" H 5350 3500 50  0001 C CNN
+F 2 "Connector_Hirose:Hirose_DF13-02P-1.25DSA_1x02_P1.25mm_Vertical" H 5350 3500 50  0001 C CNN
 F 3 "~" H 5350 3500 50  0001 C CNN
 	1    5350 3450

Commit message: change some power flags for latchup prevention
Connections:
- net +3V3 renamed VDD
Changed lines of the file:
@@
 Text Notes 4550 2700 0    50   ~ 0
 Top resistor selected for 5C center operating temperature
-$Comp
-L power:+3V3 #PWR?
-U 1 1 6203964D
-P 5350 3000
-AR Path="/61BD4B7D/62026259/6203964D" Ref="#PWR?"  Part="1"
-AR Path="/61BD4B7D/62041525/6203964D" Ref="#PWR?"  Part="1"
-AR Path="/61BD4B7D/62045EF1/6203964D" Ref="#PWR?"  Part="1"
-AR Path="/61BD4B7D/6204A8C5/6203964D" Ref="#PWR?"  Part="1"
-AR Path="/62041525/6203964D" Ref="#PWR038"  Part="1"
-AR Path="/62045EF1/6203964D" Ref="#PWR042"  Part="1"
-AR Path="/6204A8C5/6203964D" Ref="#PWR046"  Part="1"
-AR Path="/62026259/6203964D" Ref="#PWR050"  Part="1"
-F 0 "#PWR050" H 5350 2850 50  0001 C CNN
-F 1 "+3V3" H 5365 3173 50  0000 C CNN
-F 2 "" H 5350 3000 50  0001 C CNN
-F 3 "" H 5350 3000 50  0001 C CNN
-	1    5350 3000
-	1    0    0    -1
-$EndComp
 Wire Wire Line
 	5350 3300 5950 3300
-Connection ~ 5350 3300
 Wire Wire Line
 	5350 3600 5950 3600
@@
 	1    0    0    1
 $EndComp
+$Comp
+L power:VDD #PWR?
+U 1 1 61FDBD41
+P 5350 3000
+F 0 "#PWR?" H 5350 2850 50  0001 C CNN
+F 1 "VDD" H 5365 3173 50  0000 C CNN
+F 2 "" H 5350 3000 50  0001 C CNN
+F 3 "" H 5350 3000 50  0001 C CNN
+	1    5350 3000
+	1    0    0    -1
+$EndComp
+Connection ~ 5350 3300
 $EndSCHEMATC
