File: ECAD/Battery/BatteryMaster.kicad_sch (KiCad schematic)
At the start: 91 parts, among them J1 SWD/DEBUG, Q1 Si4186DY, Q10 IRF7458, Q11 Si4186DY, Q12 IRF7458, Q13 Si4186DY, Q2 IRF7458, Q26 Si4186DY, Q3 IRF7458, Q4 Si4186DY, Q5 Si4186DY, Q6 2N7002, Q7 IRF7425, Q8 IRF7458, Q9 IRF7458, SW1 INHIBIT4, SW2 INHIBIT5, SW3 INHIBIT6, U1 LM1117-3.3, U2 INA181A2, U3 BQ29209, U4 LM358, U5 LTC4359-MS8, U6 MAX6369, U7 LTC4365TS8-1, U8 STM32F103C8Tx, Y1 8MHz

Commit message: remove separate spi interface
Connections:
- net SCL: now also U8.42 (PB6)
- net SDA: now also U8.43 (PB7)
- net MISO: no longer names the net of H2.35 (Pin_35)
- net MISO: no longer U8.40 (PB4)
- net MOSI: no longer names the net of H2.37 (Pin_37)
- net MOSI: no longer U8.41 (PB5)
- net SCK: no longer names the net of H2.33 (Pin_33)
- net SCK: no longer U8.39 (PB3)
- net SS: no longer names the net of H2.39 (Pin_39)
- net SS: no longer U8.38 (PA15)
Changed lines of the file:
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@@
     (stroke (width 0) (type default) (color 0 0 0 0))
   )
-  (wire (pts (xy 241.3 121.92) (xy 246.38 121.92))
-    (stroke (width 0) (type default) (color 0 0 0 0))
-  )
   (wire (pts (xy 209.55 91.44) (xy 209.55 93.98))
     (stroke (width 0) (type default) (color 0 0 0 0))
@@
     (stroke (width 0) (type default) (color 0 0 0 0))
   )
-  (wire (pts (xy 24.13 172.72) (xy 29.21 172.72))
-    (stroke (width 0) (type default) (color 0 0 0 0))
-  )
-  (wire (pts (xy 241.3 119.38) (xy 246.38 119.38))
-    (stroke (width 0) (type default) (color 0 0 0 0))
-  )
   (wire (pts (xy 86.36 104.14) (xy 83.82 104.14))
     (stroke (width 0) (type default) (color 0 0 0 0))
@@
     (stroke (width 0) (type default) (color 0 0 0 0))
   )
-  (wire (pts (xy 24.13 175.26) (xy 29.21 175.26))
-    (stroke (width 0) (type default) (color 0 0 0 0))
-  )
   (wire (pts (xy 96.52 181.61) (xy 88.9 181.61))
     (stroke (width 0) (type default) (color 0 0 0 0))
@@
     (stroke (width 0) (type default) (color 0 0 0 0))
   )
-  (wire (pts (xy 24.13 177.8) (xy 29.21 177.8))
-    (stroke (width 0) (type default) (color 0 0 0 0))
-  )
   (wire (pts (xy 246.38 139.7) (xy 238.76 139.7))
     (stroke (width 0) (type default) (color 0 0 0 0))
@@
     (stroke (width 0) (type default) (color 0 0 0 0))
   )
-  (wire (pts (xy 241.3 116.84) (xy 246.38 116.84))
-    (stroke (width 0) (type default) (color 0 0 0 0))
-  )
   (wire (pts (xy 238.76 21.59) (xy 243.84 21.59))
     (stroke (width 0) (type default) (color 0 0 0 0))
@@
     (stroke (width 0) (type default) (color 0 0 0 0))
   )
-  (wire (pts (xy 24.13 180.34) (xy 29.21 180.34))
-    (stroke (width 0) (type default) (color 0 0 0 0))
-  )
   (wire (pts (xy 148.59 21.59) (xy 152.4 21.59))
     (stroke (width 0) (type default) (color 0 0 0 0))
@@
     (stroke (width 0) (type default) (color 0 0 0 0))
   )
-  (wire (pts (xy 283.21 147.32) (xy 279.4 147.32))
-    (stroke (width 0) (type default) (color 0 0 0 0))
-  )
   (wire (pts (xy 294.64 73.66) (xy 283.21 73.66))
     (stroke (width 0) (type default) (color 0 0 0 0))
@@
     (stroke (width 0) (type default) (color 0 0 0 0))
   )
+  (wire (pts (xy 241.3 127) (xy 246.38 127))
+    (stroke (width 0) (type default) (color 0 0 0 0))
+  )
   (wire (pts (xy 38.1 74.93) (xy 38.1 85.09))
     (stroke (width 0) (type default) (color 0 0 0 0))
@@
     (stroke (width 0) (type default) (color 0 0 0 0))
   )
+  (wire (pts (xy 241.3 124.46) (xy 246.38 124.46))
+    (stroke (width 0) (type default) (color 0 0 0 0))
+  )
   (wire (pts (xy 240.03 29.21) (xy 243.84 29.21))
     (stroke (width 0) (type default) (color 0 0 0 0))
@@
     (effects (font (size 1.27 1.27)) (justify right bottom))
   )
-  (label "MOSI" (at 24.13 177.8 0)
-    (effects (font (size 1.27 1.27)) (justify left bottom))
-  )
   (label "H3BOT" (at 238.76 142.24 0)
     (effects (font (size 1.27 1.27)) (justify left bottom))
@@
     (effects (font (size 1.27 1.27)) (justify left bottom))
   )
-  (label "SCK" (at 24.13 172.72 0)
-    (effects (font (size 1.27 1.27)) (justify left bottom))
-  )
   (label "BAT_RAW" (at 13.97 74.93 0)
     (effects (font (size 1.27 1.27)) (justify left bottom))
@@
     (effects (font (size 1.27 1.27)) (justify right bottom))
   )
-  (label "MISO" (at 241.3 119.38 0)
-    (effects (font (size 1.27 1.27)) (justify left bottom))
-  )
   (label "H2BOT" (at 88.9 158.75 0)
     (effects (font (size 1.27 1.27)) (justify left bottom))
@@
     (effects (font (size 1.27 1.27)) (justify right bottom))
   )
-  (label "MISO" (at 24.13 175.26 0)
-    (effects (font (size 1.27 1.27)) (justify left bottom))
-  )
   (label "TBAT4" (at 132.08 181.61 180)
     (effects (font (size 1.27 1.27)) (justify right bottom))
@@
     (effects (font (size 1.27 1.27)) (justify right bottom))
   )
-  (label "SS" (at 24.13 180.34 0)
-    (effects (font (size 1.27 1.27)) (justify left bottom))
-  )
-  (label "MOSI" (at 241.3 121.92 0)
-    (effects (font (size 1.27 1.27)) (justify left bottom))
-  )
   (label "H2TOP" (at 238.76 134.62 0)
     (effects (font (size 1.27 1.27)) (justify left bottom))
@@
     (effects (font (size 1.27 1.27)) (justify left bottom))
   )
-  (label "SS" (at 283.21 147.32 180)
-    (effects (font (size 1.27 1.27)) (justify right bottom))
-  )
   (label "TELEM_IBAT" (at 104.14 38.1 0)
     (effects (font (size 1.27 1.27)) (justify left bottom))
   )
-  (label "SCK" (at 241.3 116.84 0)
-    (effects (font (size 1.27 1.27)) (justify left bottom))
-  )
   (label "SWDCLK" (at 287.02 144.78 180)
     (effects (font (size 1.27 1.27)) (justify right bottom))
@@
     (effects (font (size 1.27 1.27)) (justify left bottom))
   )
+  (label "SCL" (at 241.3 124.46 0)
+    (effects (font (size 1.27 1.27)) (justify left bottom))
+  )
   (label "TELEM_VBAT" (at 219.71 39.37 180)
     (effects (font (size 1.27 1.27)) (justify right bottom))
@@
     (effects (font (size 1.27 1.27)) (justify right bottom))
   )
+  (label "SDA" (at 241.3 127 0)
+    (effects (font (size 1.27 1.27)) (justify left bottom))
+  )
   (label "TBAT1" (at 132.08 143.51 180)
     (effects (font (size 1.27 1.27)) (justify right bottom))
@@
       (reference "#PWR051") (unit 1) (value "GND") (footprint "")
     )
-    (path "/00000000-0000-0000-0000-000062045ef1/00000000-0000-0000-0000-000061fdbd41"
+    (path "/00000000-0000-0000-0000-000062026259/00000000-0000-0000-0000-000061fdbd41"
       (reference "#PWR?") (unit 1) (value "VDD") (footprint "")
     )
-    (path "/00000000-0000-0000-0000-00006204a8c5/00000000-0000-0000-0000-000061fdbd41"
+    (path "/00000000-0000-0000-0000-000062045ef1/00000000-0000-0000-0000-000061fdbd41"
       (reference "#PWR?") (unit 1) (value "VDD") (footprint "")
     )
@@
       (reference "#PWR?") (unit 1) (value "VDD") (footprint "")
     )
-    (path "/00000000-0000-0000-0000-000062026259/00000000-0000-0000-0000-000061fdbd41"
+    (path "/00000000-0000-0000-0000-00006204a8c5/00000000-0000-0000-0000-000061fdbd41"
       (reference "#PWR?") (unit 1) (value "VDD") (footprint "")
     )

Commit message: who needs ovp anyways
Parts:
- removed C13: 0.1uF, Capacitor_SMD:C_0805_2012Metric, symbol Device:C
- removed F2: 7A, Resistor_SMD:R_1206_3216Metric, symbol Device:Polyfuse
- removed Q1, Q26: Si4186DY, Package_SO:SOIC-8_3.9x4.9mm_P1.27mm, symbol Transistor_FET:Si4162DY
- removed Q8, Q9: IRF7458, Package_SO:SOIC-8_3.9x4.9mm_P1.27mm, symbol Transistor_FET:IRF7404
- removed R23: 100K, Resistor_SMD:R_0805_2012Metric, symbol Device:R
- removed R25: 100R, Resistor_SMD:R_0805_2012Metric, symbol Device:R
- removed R3: 1K, Resistor_SMD:R_0805_2012Metric, symbol Device:R
- removed SW1: INHIBIT4, Connector_Hirose:Hirose_DF13-02P-1.25DSA_1x02_P1.25mm_Vertical, symbol Switch:SW_SPST
- C6: value 0.33uF -> (none)
- F1: value 7A -> (none)
- H1: renamed from H2; value Stack Header 2 -> (none); footprint footprints:PinSocket_2x26_P2.54mm_Vertical -> (none)
- H2: renamed from H1; value Stack Header 1 -> (none)
Connections:
- net at BT1.1 (+), BT3.1 (+), R2.1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: now also F1.1
- net at Q10.5 (D), Q10.6 (D), Q10.7 (D)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: now also Q5.1 (S), Q5.2 (S), Q5.3 (S), R21.1, U7.7 (Vout)
- no-connect marks 23 -> 24
Other:
- note removed: "Inhibit (B)"
- note removed: "OUT is pulled high in OV condition, after 3 second delay OV is fixed at 4.3V per cell"
- note removed: "Redundant mosfets"
- note removed: "Semidestructive protection in case OVP exists for more than 3 seconds"
- moved on the sheet: C16, C19, F1, JP2, JP3, Q10, Q11, Q12, Q13, R26, R27, R28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

Commit message: move inhibits to battery, resize sheet
Parts:
- added Q? (x3): IRF7458, Package_SO:SOIC-8_3.9x4.9mm_P1.27mm, symbol Transistor_FET:IRF7404
- added R? (x3): 100K, Resistor_SMD:R_0805_2012Metric, symbol Device:R
- added R? (x3): 100R, Resistor_SMD:R_0805_2012Metric, symbol Device:R
- added SW? (x2): (no value), Connector_Hirose:Hirose_DF13-02P-1.25DSA_1x02_P1.25mm_Vertical, symbol Switch:SW_SPST
- added SW?: INHIBIT, Connector_Hirose:Hirose_DF13-02P-1.25DSA_1x02_P1.25mm_Vertical, symbol Switch:SW_SPST
- SW2: value INHIBIT5 -> (none)
- SW3: value INHIBIT6 -> (none)
Connections:
- net BCR_OUT: now also Q?.1 (S), Q?.2 (S), Q?.3 (S), R?.1; no longer C1.1, Q4.1 (S), Q4.2 (S), Q4.3 (S), R1.2, U1.3 (VI), U2.3 (+), U5.2 (SRC), U5.4 (IN), U5.5 (~{SHDN})
- net GND: now also R?.2, R?.2, R?.2
- net PCM_IN: now also Q?.5 (D), Q?.6 (D), Q?.7 (D), Q?.8 (D); no longer C9.1, Q4.5 (D), Q4.6 (D), Q4.7 (D), Q4.8 (D), U5.8 (OUT)
- net BAT_RAW: no longer names the net of F1.2, Q12.5 (D), Q12.6 (D), Q12.7 (D), Q12.8 (D)
- new net: C1.1, Q4.1 (S), Q4.2 (S), Q4.3 (S), Q?.5 (D), Q?.6 (D), Q?.7 (D), Q?.8 (D), R1.2, U1.3 (VI), U2.3 (+), U5.2 (SRC), U5.4 (IN), U5.5 (~{SHDN})
- new net: C9.1, Q4.5 (D), Q4.6 (D), Q4.7 (D), Q4.8 (D), Q?.1 (S), Q?.2 (S), Q?.3 (S), R?.1, U5.8 (OUT)
- new net: Q?.4 (G), R?.1, SW?.2 (B) (x3)
- new net: Q?.1 (S), Q?.2 (S), Q?.3 (S), Q?.5 (D), Q?.6 (D), Q?.7 (D), Q?.8 (D), R?.1
- new net: R?.2, SW?.1 (A) (x3)
Other:
- note added: "Inhibit (B)"
- note added: "Inhibit (C)"
- note removed: "V TELEM"
- moved on the sheet: BT1, BT2, BT3, BT4, C1, C10, C11, C12, C14, C15, C16, C17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

Commit message: move heater circuitry
Parts:
- added J?: (no value), symbol Connector:Conn_01x12_Female
- C6: value (none) -> 0.1uF
- F1: value (none) -> 6A
- H1: value (none) -> Stack Header; footprint (none) -> footprints:PinSocket_2x26_P2.54mm_Vertical
- H2: value (none) -> Stack Header
- SW1, SW4: renamed from SW?; value (none) -> INHIBIT
- SW2, SW3: value (none) -> INHIBIT
- gave numbers to parts that had none: 10
Connections:
- net +5V: now also J?.1 (Pin_1)
- net GND: now also J?.11 (Pin_11), J?.12 (Pin_12)
- net TBAT1: now also J?.7 (Pin_7)
- net TBAT2: now also J?.8 (Pin_8)
- net TBAT3: now also J?.9 (Pin_9)
- net TBAT4: now also J?.10 (Pin_10)
- net VDD: now also J?.2 (Pin_2)
- new net H1CTRL: J?.3 (Pin_3)
- new net H2CTRL: J?.4 (Pin_4)
- new net H3CTRL: J?.5 (Pin_5)
- new net H4CTRL: J?.6 (Pin_6)
Other:
- removed sheet HBAT1
- removed sheet HBAT2
- removed sheet HBAT3
- removed sheet HBAT4
- note removed: "Cell Heaters/Thermistors"
- moved on the sheet: H1, H2

Commit message: minor fixes
Parts:
- J?: value (none) -> Conn_01x12_Female
Connections:
- net H1BOT is gone; now on net H2CTRL: U8.46 (PB9)
- net H1TOP is gone; now on net H1CTRL: U8.45 (PB8)
- net H2BOT is gone; now on net H4CTRL: U8.22 (PB11)
- net H2TOP is gone; now on net H3CTRL: U8.21 (PB10)
- net H3BOT: no longer names the net of U8.26 (PB13)
- net H3TOP: no longer names the net of U8.25 (PB12)
- net H4BOT: no longer names the net of U8.28 (PB15)
- net H4TOP: no longer names the net of U8.27 (PB14)
Changed lines of the file:
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@@
     (stroke (width 0) (type default) (color 0 0 0 0))
   )
-  (wire (pts (xy 242.57 199.39) (xy 234.95 199.39))
-    (stroke (width 0) (type default) (color 0 0 0 0))
-  )
   (wire (pts (xy 377.19 95.25) (xy 392.43 95.25))
     (stroke (width 0) (type default) (color 0 0 0 0))
@@
     (stroke (width 0) (type default) (color 0 0 0 0))
   )
-  (wire (pts (xy 242.57 184.15) (xy 234.95 184.15))
-    (stroke (width 0) (type default) (color 0 0 0 0))
-  )
   (wire (pts (xy 330.2 101.6) (xy 330.2 110.49))
     (stroke (width 0) (type default) (color 0 0 0 0))
@@
     (stroke (width 0) (type default) (color 0 0 0 0))
   )
-  (wire (pts (xy 242.57 191.77) (xy 234.95 191.77))
-    (stroke (width 0) (type default) (color 0 0 0 0))
-  )
   (wire (pts (xy 233.68 73.66) (xy 241.3 73.66))
     (stroke (width 0) (type default) (color 0 0 0 0))
@@
     (stroke (width 0) (type default) (color 0 0 0 0))
   )
+  (wire (pts (xy 234.95 181.61) (xy 242.57 181.61))
+    (stroke (width 0) (type default) (color 0 0 0 0))
+  )
   (wire (pts (xy 99.06 212.09) (xy 115.57 212.09))
     (stroke (width 0) (type default) (color 0 0 0 0))
@@
     (stroke (width 0) (type default) (color 0 0 0 0))
   )
-  (wire (pts (xy 242.57 186.69) (xy 234.95 186.69))
-    (stroke (width 0) (type default) (color 0 0 0 0))
-  )
   (wire (pts (xy 64.77 41.91) (xy 64.77 24.13))
     (stroke (width 0) (type default) (color 0 0 0 0))
@@
     (stroke (width 0) (type default) (color 0 0 0 0))
   )
-  (wire (pts (xy 242.57 194.31) (xy 234.95 194.31))
-    (stroke (width 0) (type default) (color 0 0 0 0))
-  )
   (polyline (pts (xy 99.06 15.24) (xy 99.06 60.96))
     (stroke (width 0) (type default) (color 0 0 0 0))
@@
     (stroke (width 0) (type default) (color 0 0 0 0))
   )
+  (wire (pts (xy 234.95 186.69) (xy 242.57 186.69))
+    (stroke (width 0) (type default) (color 0 0 0 0))
+  )
+  (wire (pts (xy 234.95 184.15) (xy 242.57 184.15))
+    (stroke (width 0) (type default) (color 0 0 0 0))
+  )
   (wire (pts (xy 73.66 198.12) (xy 78.74 198.12))
     (stroke (width 0) (type default) (color 0 0 0 0))
@@
     (stroke (width 0) (type default) (color 0 0 0 0))
   )
-  (wire (pts (xy 242.57 189.23) (xy 234.95 189.23))
-    (stroke (width 0) (type default) (color 0 0 0 0))
-  )
   (wire (pts (xy 97.79 97.79) (xy 97.79 110.49))
     (stroke (width 0) (type default) (color 0 0 0 0))
@@
     (stroke (width 0) (type default) (color 0 0 0 0))
   )
-  (wire (pts (xy 242.57 196.85) (xy 234.95 196.85))
-    (stroke (width 0) (type default) (color 0 0 0 0))
-  )
   (wire (pts (xy 275.59 171.45) (xy 287.02 171.45))
     (stroke (width 0) (type default) (color 0 0 0 0))
@@
     (stroke (width 0) (type default) (color 0 0 0 0))
   )
-  (wire (pts (xy 242.57 181.61) (xy 234.95 181.61))
-    (stroke (width 0) (type default) (color 0 0 0 0))
-  )
   (wire (pts (xy 48.26 35.56) (xy 48.26 31.75))
     (stroke (width 0) (type default) (color 0 0 0 0))
@@
     (stroke (width 0) (type default) (color 0 0 0 0))
   )
+  (wire (pts (xy 234.95 189.23) (xy 242.57 189.23))
+    (stroke (width 0) (type default) (color 0 0 0 0))
+  )
   (wire (pts (xy 242.57 166.37) (xy 234.95 166.37))
     (stroke (width 0) (type default) (color 0 0 0 0))
@@
     (effects (font (size 1.27 1.27)) (justify right bottom))
   )
-  (label "H2BOT" (at 234.95 189.23 0)
-    (effects (font (size 1.27 1.27)) (justify left bottom))
-  )
-  (label "H4TOP" (at 234.95 196.85 0)
-    (effects (font (size 1.27 1.27)) (justify left bottom))
-  )
   (label "TBAT3" (at 330.2 184.15 0)
     (effects (font (size 1.27 1.27)) (justify left bottom))
   )
-  (label "H3BOT" (at 234.95 194.31 0)
-    (effects (font (size 1.27 1.27)) (justify left bottom))
-  )
   (label "TELEM_VBAT" (at 287.02 171.45 180)
     (effects (font (size 1.27 1.27)) (justify right bottom))
@@
     (effects (font (size 1.27 1.27)) (justify right bottom))
   )
-  (label "H1CTRL" (at 330.2 168.91 0)
+  (label "H3CTRL" (at 234.95 186.69 0)
     (effects (font (size 1.27 1.27)) (justify left bottom))
   )
-  (label "SWDIO" (at 194.31 194.31 180)
-    (effects (font (size 1.27 1.27)) (justify right bottom))
-  )
-  (label "H3TOP" (at 234.95 191.77 0)
+  (label "H2CTRL" (at 234.95 184.15 0)
     (effects (font (size 1.27 1.27)) (justify left bottom))
   )
-  (label "H1BOT" (at 234.95 184.15 0)
+  (label "H1CTRL" (at 330.2 168.91 0)
     (effects (font (size 1.27 1.27)) (justify left bottom))
   )
+  (label "SWDIO" (at 194.31 194.31 180)
+    (effects (font (size 1.27 1.27)) (justify right bottom))
+  )
   (label "D+" (at 279.4 191.77 180)
     (effects (font (size 1.27 1.27)) (justify right bottom))
@@
     (effects (font (size 1.27 1.27)) (justify left bottom))
   )
+  (label "H4CTRL" (at 234.95 189.23 0)
+    (effects (font (size 1.27 1.27)) (justify left bottom))
+  )
   (label "D+" (at 190.5 204.47 180)
     (effects (font (size 1.27 1.27)) (justify right bottom))
@@
     (effects (font (size 1.27 1.27)) (justify right bottom))
   )
-  (label "H4BOT" (at 234.95 199.39 0)
+  (label "H1CTRL" (at 234.95 181.61 0)
     (effects (font (size 1.27 1.27)) (justify left bottom))
   )
@@
     (effects (font (size 1.27 1.27)) (justify right bottom))
   )
-  (label "H2TOP" (at 234.95 186.69 0)
-    (effects (font (size 1.27 1.27)) (justify left bottom))
-  )
-  (label "H1TOP" (at 234.95 181.61 0)
-    (effects (font (size 1.27 1.27)) (justify left bottom))
-  )
   (label "TELEM_IBAT" (at 142.24 90.17 0)
     (effects (font (size 1.27 1.27)) (justify left bottom))
@@
       (effects (font (size 1.27 1.27)) hide)
     )
-    (property "Value" "" (id 1) (at 334.01 161.29 0))
+    (property "Value" "VDD" (id 1) (at 334.01 161.29 0))
     (property "Footprint" "" (id 2) (at 334.01 166.37 0)
       (effects (font (size 1.27 1.27)) hide)
@@
       (effects (font (size 1.27 1.27)) hide)
     )
-    (property "Value" "" (id 1) (at 337.82 196.85 0))
+    (property "Value" "GND" (id 1) (at 337.82 196.85 0))
     (property "Footprint" "" (id 2) (at 337.82 191.77 0)
       (effects (font (size 1.27 1.27)) hide)
@@
       (effects (font (size 1.27 1.27)) hide)
     )
-    (property "Value" "" (id 1) (at 337.82 158.75 0))
+    (property "Value" "+5V" (id 1) (at 337.82 158.75 0))
     (property "Footprint" "" (id 2) (at 337.82 163.83 0)
       (effects (font (size 1.27 1.27)) hide)
@@
       (effects (font (size 1.27 1.27)) (justify left))
     )
-    (property "Value" "" (id 1) (at 344.17 179.0699 0)
+    (property "Value" "Conn_01x12_Female" (id 1) (at 344.17 179.0699 0)
       (effects (font (size 1.27 1.27)) (justify left))
     )

Commit message: move UVP to battery
Parts:
- added C13, C21: (no value), symbol Device:C
- added Q14: (no value), symbol Transistor_FET:2N7002
- added Q15: (no value), symbol Transistor_FET:IRF7404
- added R30, R31, R32: (no value), symbol Device:R
- added U10: (no value), symbol Reference_Voltage:ADR4530
- added U9: (no value), symbol Amplifier_Operational:LM358
- gave numbers to parts that had none: 1
Connections:
- net GND: now also C13.2, C21.2, Q14.2 (S), R32.2, U10.4 (GND), U9.4 (V-), U9.5 (+)
- net at C9.1, Q4.5 (D), Q4.6 (D)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: now also C13.1, C21.1, Q15.1 (S), Q15.2 (S), Q15.3 (S), R30.1, U10.2 (IN), U9.8 (V+); no longer Q8.1 (S), Q8.2 (S), Q8.3 (S), R25.1
- new net: R30.2, R31.1, U9.2 (-)
- new net: Q14.3 (D), R31.2, R32.1
- new net: Q15.5 (D), Q15.6 (D), Q15.7 (D), Q15.8 (D), Q8.1 (S), Q8.2 (S), Q8.3 (S), R25.1
- new net: Q14.1 (G), Q15.4 (G), U9.1
- new net: U10.6 (OUT), U9.3 (+)
- new net: U9.6 (-), U9.7
Other:
- note added: "Lower resistor provides hysteresis for UVLO Falling threshold, with the mosfet conducting, is 6.2V (6.199 taking into account 7.5 ohm Rds(on)) Rising threshold, with mosfet open, is 7V"
- note added: "UV Active High Compares with a 3V ref"
- note added: "UVP and Inhibit"
- moved on the sheet: BT1, BT2, BT3, BT4, C1, C10, C11, C12, C14, C15, C16, C17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

Commit message: enlarge comment
Parts:
- C13: value (none) -> 1uF; footprint (none) -> Capacitor_SMD:C_0805_2012Metric
- C21: value (none) -> 0.1uF; footprint (none) -> Capacitor_SMD:C_0805_2012Metric
- Q14: value (none) -> 2N7002; footprint (none) -> Package_TO_SOT_SMD:SOT-23
- Q15: value (none) -> IRF7458; footprint (none) -> Package_SO:SOIC-8_3.9x4.9mm_P1.27mm
- R30: value (none) -> 40K; footprint (none) -> Resistor_SMD:R_0805_2012Metric
- R31: value (none) -> 30K; footprint (none) -> Resistor_SMD:R_0805_2012Metric
- R32: value (none) -> 7.5K; footprint (none) -> Resistor_SMD:R_0805_2012Metric
- U10: value (none) -> ADR4530; footprint (none) -> Package_SO:SOIC-8_3.9x4.9mm_P1.27mm
- U9: value (none) -> LM358; footprint (none) -> Package_SO:SO-8_3.9x4.9mm_P1.27mm
Other:
- moved on the sheet: Q8, Q9, R25, R58, R59, R60, SW4, SW5

Commit message: remove flex pcb, move to battery board
Parts:
- removed J2: Conn_01x12_Female, symbol Connector:Conn_01x12_Female
- renumbered C14 to C11, C15 to C12, C16 to C13, C17 to C14, C18 to C15, C19 to C16, C20 to C17, C3 to C18, C4 to C19, C5 to C20, C6 to C21, C9 to C3, C13 to C4, C21 to C5, C8 to C6, C11 to C8, C12 to C9, Q8 to Q10, Q9 to Q11, Q10 to Q12, Q11 to Q13, Q12 to Q14, Q13 to Q15, Q4 to Q2, Q14 to Q3, Q15 to Q4, Q2 to Q5, Q3 to Q7, Q7 to Q8, Q5 to Q9, R3 to R1, R13 to R10, R30 to R11, R31 to R12, R32 to R13, R17 to R15, R19 to R16, R20 to R17, R15 to R18, R16 to R19, R23 to R2, R18 to R20, R25 to R21, R58 to R22, R21 to R23, R22 to R24, R59 to R25, R24 to R26, R60 to R27, R26 to R28, R27 to R29, R1 to R3, R28 to R30, R29 to R31, R2 to R32, R8 to R33, R9 to R34, R10 to R35, R11 to R8, R12 to R9, SW4 to SW2, SW5 to SW3, SW2 to SW4, SW3 to SW5, U3 to U10, U5 to U2, U2 to U3, U9 to U4, U10 to U5, U4 to U6, U6 to U7, U7 to U8, U8 to U9
Other:
- added sheet Cell 1 Heater (Heater.kicad_sch)
- added sheet Cell 2 Heater (Heater.kicad_sch)
- added sheet Cell 3 Heater (Heater.kicad_sch)
- added sheet Cell 4 Heater (Heater.kicad_sch)
