File: ECAD/Battery/Heater.kicad_sch (KiCad schematic)
At the start: 11 parts, among them Q16 2N7002, Q17 BSS83P, Q18 BSN20

Commit message: push rev 2 (no more silly numbering conventions)
Changed lines of the file:
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@@
 (kicad_sch (version 20211123) (generator eeschema)
   (paper "A4")
+  (title_block
+    (rev "2")
+  )
   (junction (at 175.26 97.79) (diameter 0) (color 0 0 0 0)
   )
@@
       (effects (font (size 1.27 1.27)) hide)
     )
-    (property "Value" "" (id 1) (at 137.16 67.31 0))
+    (property "Value" "+3V3" (id 1) (at 137.16 67.31 0))
     (property "Footprint" "" (id 2) (at 137.16 72.39 0)
       (effects (font (size 1.27 1.27)) hide)

Commit message: comment update
Parts:
- added C?: (no value), symbol Device:C
Other:
- note added: "10 Ohm PCB Traces"
- note removed: "20 Ohm PCB Traces"
Changed lines of the file:
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@@
     (stroke (width 0) (type default) (color 0 0 0 0))
   )
-  (text "20 Ohm PCB Traces" (at 148.59 97.79 0)
+  (text "10 Ohm PCB Traces" (at 148.59 97.79 0)
     (effects (font (size 1.27 1.27)) (justify left bottom))
   )
@@
     (pin "1")
   )
+  (symbol (lib_id "Device:C") (at 156.21 106.68 0) (unit 1)
+    (in_bom yes) (on_board yes) (fields_autoplaced)
+    (property "Reference" "C?" (id 0) (at 160.02 105.4099 0)
+      (effects (font (size 1.27 1.27)) (justify left))
+    )
+    (property "Value" "" (id 1) (at 160.02 107.9499 0)
+      (effects (font (size 1.27 1.27)) (justify left))
+    )
+    (property "Footprint" "" (id 2) (at 157.1752 110.49 0)
+      (effects (font (size 1.27 1.27)) hide)
+    )
+    (property "Datasheet" "~" (id 3) (at 156.21 106.68 0)
+      (effects (font (size 1.27 1.27)) hide)
+    )
+    (pin "1")
+    (pin "2")
+  )
 )

Commit message: regulator
Parts:
- C?: value (none) -> C
Connections:
- net +3V3 renamed +1V0
Changed lines of the file:
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@@
   (junction (at 106.68 85.09) (diameter 0) (color 0 0 0 0)
   )
+  (junction (at 137.16 72.39) (diameter 0) (color 0 0 0 0)
+  )
   (junction (at 137.16 129.54) (diameter 0) (color 0 0 0 0)
-  )
-  (junction (at 137.16 72.39) (diameter 0) (color 0 0 0 0)
   )
   (junction (at 128.27 129.54) (diameter 0) (color 0 0 0 0)
@@
     (pin "3")
   )
-  (symbol (lib_id "power:+3V3") (at 137.16 72.39 0) (unit 1)
+  (symbol (lib_id "power:+1V0") (at 137.16 72.39 0) (unit 1)
     (in_bom yes) (on_board yes) (fields_autoplaced)
     (property "Reference" "#PWR?" (id 0) (at 137.16 76.2 0)
       (effects (font (size 1.27 1.27)) hide)
     )
-    (property "Value" "+3V3" (id 1) (at 137.16 67.31 0))
+    (property "Value" "" (id 1) (at 137.16 67.31 0))
     (property "Footprint" "" (id 2) (at 137.16 72.39 0)
       (effects (font (size 1.27 1.27)) hide)
@@
       (effects (font (size 1.27 1.27)) (justify left))
     )
-    (property "Value" "" (id 1) (at 160.02 107.9499 0)
-      (effects (font (size 1.27 1.27)) (justify left))
-    )
+    (property "Value" "C" (id 1) (at 160.02 107.9499 0)
+      (effects (font (size 1.27 1.27)) (justify left))
+    )

Commit message: Respect mosfets for heaters, organize, inductor footprint
Parts:
- removed C?: C, symbol Device:C
- removed Q16: 2N7002, Package_TO_SOT_SMD:SOT-23, symbol Transistor_FET:2N7002
- removed Q17: BSS83P, Package_TO_SOT_SMD:SOT-23, symbol Transistor_FET:BSS83P
- removed R38: 10K, Resistor_SMD:R_0805_2012Metric, symbol Device:R
- added Q16: (no value), symbol Transistor_FET:BSN20
- Q18: value BSN20 -> (none)
Connections:
- net +1V0: now also Q16.3 (D)
- net GND: no longer R37.2
- net at R36.1, R37.1: now also Q16.1 (G)
- net at Q18.3 (D): now also R37.2, Q16.2 (S)
Other:
- moved on the sheet: Q18, R36, R37, R39, R40

Commit message: layout and footprints
Parts:
- Q16: value (none) -> DMG6968U-7; footprint (none) -> Package_TO_SOT_SMD:SOT-23
- Q18: value (none) -> DMG6968U-7
Changed lines of the file:
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@@
       (effects (font (size 1.27 1.27)) (justify left))
     )
-    (property "Value" "" (id 1) (at 122.047 76.073 0)
+    (property "Value" "DMG6968U-7" (id 1) (at 122.047 76.073 0)
       (effects (font (size 1.27 1.27)) (justify left))
     )
-    (property "Footprint" "" (id 2) (at 121.92 76.835 0)
+    (property "Footprint" "Package_TO_SOT_SMD:SOT-23" (id 2) (at 121.92 76.835 0)
       (effects (font (size 1.27 1.27) italic) (justify left) hide)
     )
@@
       (effects (font (size 1.27 1.27)) (justify left))
     )
-    (property "Value" "" (id 1) (at 122.047 117.983 0)
+    (property "Value" "DMG6968U-7" (id 1) (at 122.047 117.983 0)
       (effects (font (size 1.27 1.27)) (justify left))
     )

Commit message: routing and stuff
Parts:
- renumbered C22 to C25, Q18 to Q17, R36 to R38, R37 to R40, R40 to R41, R41 to R42
Changed lines of the file:
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@@
   (symbol (lib_id "Device:R") (at 105.41 74.93 270) (unit 1)
     (in_bom yes) (on_board yes)
-    (property "Reference" "R36" (id 0) (at 105.41 72.39 90))
+    (property "Reference" "R38" (id 0) (at 105.41 72.39 90))
     (property "Value" "100R" (id 1) (at 105.41 74.93 90))
     (property "Footprint" "Resistor_SMD:R_0805_2012Metric" (id 2) (at 105.41 73.152 90)
@@
   (symbol (lib_id "power:+1V0") (at 119.38 67.31 0) (unit 1)
     (in_bom yes) (on_board yes) (fields_autoplaced)
-    (property "Reference" "#PWR051" (id 0) (at 119.38 71.12 0)
+    (property "Reference" "#PWR042" (id 0) (at 119.38 71.12 0)
       (effects (font (size 1.27 1.27)) hide)
     )
@@
   (symbol (lib_id "Device:C") (at 190.5 101.6 0) (unit 1)
     (in_bom yes) (on_board yes)
-    (property "Reference" "C22" (id 0) (at 193.421 100.4316 0)
+    (property "Reference" "C25" (id 0) (at 193.421 100.4316 0)
       (effects (font (size 1.27 1.27)) (justify left))
     )
@@
   (symbol (lib_id "power:VDD") (at 175.26 90.17 0) (unit 1)
     (in_bom yes) (on_board yes)
-    (property "Reference" "#PWR041" (id 0) (at 175.26 93.98 0)
+    (property "Reference" "#PWR044" (id 0) (at 175.26 93.98 0)
       (effects (font (size 1.27 1.27)) hide)
     )
@@
   (symbol (lib_id "Device:R") (at 175.26 93.98 0) (unit 1)
     (in_bom yes) (on_board yes)
-    (property "Reference" "R41" (id 0) (at 176.53 93.98 0)
+    (property "Reference" "R42" (id 0) (at 176.53 93.98 0)
       (effects (font (size 1.27 1.27)) (justify left))
     )
@@
   (symbol (lib_id "power:GND") (at 175.26 105.41 0) (unit 1)
     (in_bom yes) (on_board yes)
-    (property "Reference" "#PWR042" (id 0) (at 175.26 111.76 0)
+    (property "Reference" "#PWR045" (id 0) (at 175.26 111.76 0)
       (effects (font (size 1.27 1.27)) hide)
     )
@@
   (symbol (lib_id "Device:R") (at 110.49 120.65 0) (unit 1)
     (in_bom yes) (on_board yes)
-    (property "Reference" "R40" (id 0) (at 109.22 120.65 0)
+    (property "Reference" "R41" (id 0) (at 109.22 120.65 0)
       (effects (font (size 1.27 1.27)) (justify right))
     )
@@
   (symbol (lib_id "Device:R") (at 110.49 78.74 0) (unit 1)
     (in_bom yes) (on_board yes)
-    (property "Reference" "R37" (id 0) (at 109.22 78.74 0)
+    (property "Reference" "R40" (id 0) (at 109.22 78.74 0)
       (effects (font (size 1.27 1.27)) (justify right))
     )
@@
   (symbol (lib_id "Transistor_FET:BSN20") (at 116.84 116.84 0) (unit 1)
     (in_bom yes) (on_board yes)
-    (property "Reference" "Q18" (id 0) (at 122.047 115.6716 0)
+    (property "Reference" "Q17" (id 0) (at 122.047 115.6716 0)
       (effects (font (size 1.27 1.27)) (justify left))
     )
@@
   (symbol (lib_id "power:GND") (at 119.38 124.46 0) (unit 1)
     (in_bom yes) (on_board yes)
-    (property "Reference" "#PWR040" (id 0) (at 119.38 130.81 0)
+    (property "Reference" "#PWR043" (id 0) (at 119.38 130.81 0)
       (effects (font (size 1.27 1.27)) hide)
     )

Commit message: route
Parts:
- renumbered C25 to C24
Changed lines of the file:
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@@
   (symbol (lib_id "Device:C") (at 190.5 101.6 0) (unit 1)
     (in_bom yes) (on_board yes)
-    (property "Reference" "C25" (id 0) (at 193.421 100.4316 0)
+    (property "Reference" "C24" (id 0) (at 193.421 100.4316 0)
       (effects (font (size 1.27 1.27)) (justify left))
     )

Commit message: remove jank heater trace
Parts:
- added R58: (no value), symbol Device:Heater
Connections:
- net at Q16.2 (S), R40.2: now also R58.1; no longer Q17.3 (D)
- new net: Q17.3 (D), R58.2
Other:
- note added: "10 Ohm Nichrome Wire (24 Gauge?)"
- note removed: "10 Ohm PCB Traces"
Changed lines of the file:
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@@
   (junction (at 175.26 105.41) (diameter 0) (color 0 0 0 0)
   )
+  (junction (at 119.38 82.55) (diameter 0) (color 0 0 0 0)
+  )
   (junction (at 110.49 74.93) (diameter 0) (color 0 0 0 0)
-  )
-  (junction (at 119.38 82.55) (diameter 0) (color 0 0 0 0)
   )
   (junction (at 119.38 124.46) (diameter 0) (color 0 0 0 0)
@@
     (stroke (width 0) (type default) (color 0 0 0 0))
   )
-  (wire (pts (xy 129.54 107.95) (xy 129.54 109.22))
-    (stroke (width 0) (type default) (color 0 0 0 0))
-  )
-  (wire (pts (xy 109.22 97.79) (xy 129.54 97.79))
-    (stroke (width 0) (type default) (color 0 0 0 0))
-  )
-  (wire (pts (xy 109.22 107.95) (xy 129.54 107.95))
-    (stroke (width 0) (type default) (color 0 0 0 0))
-  )
-  (wire (pts (xy 109.22 101.6) (xy 129.54 101.6))
-    (stroke (width 0) (type default) (color 0 0 0 0))
-  )
-  (wire (pts (xy 129.54 97.79) (xy 129.54 99.06))
-    (stroke (width 0) (type default) (color 0 0 0 0))
-  )
-  (wire (pts (xy 109.22 93.98) (xy 129.54 93.98))
-    (stroke (width 0) (type default) (color 0 0 0 0))
-  )
-  (wire (pts (xy 109.22 93.98) (xy 109.22 95.25))
-    (stroke (width 0) (type default) (color 0 0 0 0))
-  )
-  (wire (pts (xy 109.22 87.63) (xy 129.54 87.63))
-    (stroke (width 0) (type default) (color 0 0 0 0))
-  )
-  (wire (pts (xy 109.22 99.06) (xy 129.54 99.06))
-    (stroke (width 0) (type default) (color 0 0 0 0))
-  )
-  (wire (pts (xy 109.22 92.71) (xy 129.54 92.71))
-    (stroke (width 0) (type default) (color 0 0 0 0))
-  )
   (wire (pts (xy 119.38 124.46) (xy 119.38 121.92))
     (stroke (width 0) (type default) (color 0 0 0 0))
   )
-  (wire (pts (xy 109.22 106.68) (xy 109.22 107.95))
-    (stroke (width 0) (type default) (color 0 0 0 0))
-  )
   (wire (pts (xy 109.22 74.93) (xy 110.49 74.93))
-    (stroke (width 0) (type default) (color 0 0 0 0))
-  )
-  (wire (pts (xy 129.54 110.49) (xy 129.54 111.76))
-    (stroke (width 0) (type default) (color 0 0 0 0))
-  )
-  (wire (pts (xy 129.54 105.41) (xy 129.54 106.68))
-    (stroke (width 0) (type default) (color 0 0 0 0))
-  )
-  (wire (pts (xy 129.54 82.55) (xy 129.54 83.82))
     (stroke (width 0) (type default) (color 0 0 0 0))
   )
@@
     (stroke (width 0) (type default) (color 0 0 0 0))
   )
-  (wire (pts (xy 109.22 99.06) (xy 109.22 100.33))
-    (stroke (width 0) (type default) (color 0 0 0 0))
-  )
-  (wire (pts (xy 109.22 95.25) (xy 129.54 95.25))
-    (stroke (width 0) (type default) (color 0 0 0 0))
-  )
-  (wire (pts (xy 109.22 88.9) (xy 129.54 88.9))
-    (stroke (width 0) (type default) (color 0 0 0 0))
-  )
-  (wire (pts (xy 109.22 91.44) (xy 109.22 92.71))
-    (stroke (width 0) (type default) (color 0 0 0 0))
-  )
-  (wire (pts (xy 109.22 96.52) (xy 129.54 96.52))
-    (stroke (width 0) (type default) (color 0 0 0 0))
-  )
   (wire (pts (xy 110.49 82.55) (xy 119.38 82.55))
-    (stroke (width 0) (type default) (color 0 0 0 0))
-  )
-  (wire (pts (xy 109.22 102.87) (xy 129.54 102.87))
     (stroke (width 0) (type default) (color 0 0 0 0))
   )
@@
     (stroke (width 0) (type default) (color 0 0 0 0))
   )
-  (wire (pts (xy 109.22 83.82) (xy 109.22 85.09))
-    (stroke (width 0) (type default) (color 0 0 0 0))
-  )
-  (wire (pts (xy 109.22 90.17) (xy 129.54 90.17))
-    (stroke (width 0) (type default) (color 0 0 0 0))
-  )
-  (wire (pts (xy 109.22 88.9) (xy 109.22 90.17))
-    (stroke (width 0) (type default) (color 0 0 0 0))
-  )
-  (wire (pts (xy 129.54 87.63) (xy 129.54 88.9))
-    (stroke (width 0) (type default) (color 0 0 0 0))
-  )
-  (wire (pts (xy 109.22 91.44) (xy 129.54 91.44))
+  (wire (pts (xy 119.38 97.79) (xy 119.38 111.76))
     (stroke (width 0) (type default) (color 0 0 0 0))
   )
@@
     (stroke (width 0) (type default) (color 0 0 0 0))
   )
-  (wire (pts (xy 119.38 82.55) (xy 129.54 82.55))
-    (stroke (width 0) (type default) (color 0 0 0 0))
-  )
-  (wire (pts (xy 129.54 100.33) (xy 129.54 101.6))
-    (stroke (width 0) (type default) (color 0 0 0 0))
-  )
-  (wire (pts (xy 129.54 92.71) (xy 129.54 93.98))
-    (stroke (width 0) (type default) (color 0 0 0 0))
-  )
-  (wire (pts (xy 109.22 109.22) (xy 109.22 110.49))
-    (stroke (width 0) (type default) (color 0 0 0 0))
-  )
-  (wire (pts (xy 109.22 100.33) (xy 129.54 100.33))
-    (stroke (width 0) (type default) (color 0 0 0 0))
-  )
-  (wire (pts (xy 109.22 96.52) (xy 109.22 97.79))
-    (stroke (width 0) (type default) (color 0 0 0 0))
-  )
-  (wire (pts (xy 129.54 102.87) (xy 129.54 104.14))
+  (wire (pts (xy 119.38 82.55) (xy 119.38 90.17))
     (stroke (width 0) (type default) (color 0 0 0 0))
   )
@@
     (stroke (width 0) (type default) (color 0 0 0 0))
   )
-  (wire (pts (xy 109.22 83.82) (xy 129.54 83.82))
-    (stroke (width 0) (type default) (color 0 0 0 0))
-  )
-  (wire (pts (xy 129.54 85.09) (xy 129.54 86.36))
-    (stroke (width 0) (type default) (color 0 0 0 0))
-  )
-  (wire (pts (xy 109.22 110.49) (xy 129.54 110.49))
-    (stroke (width 0) (type default) (color 0 0 0 0))
-  )
-  (wire (pts (xy 109.22 105.41) (xy 129.54 105.41))
-    (stroke (width 0) (type default) (color 0 0 0 0))
-  )
-  (wire (pts (xy 129.54 106.68) (xy 109.22 106.68))
-    (stroke (width 0) (type default) (color 0 0 0 0))
-  )
-  (wire (pts (xy 129.54 90.17) (xy 129.54 91.44))
-    (stroke (width 0) (type default) (color 0 0 0 0))
-  )
-  (wire (pts (xy 109.22 101.6) (xy 109.22 102.87))
-    (stroke (width 0) (type default) (color 0 0 0 0))
-  )
   (wire (pts (xy 109.22 116.84) (xy 110.49 116.84))
     (stroke (width 0) (type default) (color 0 0 0 0))
   )
-  (wire (pts (xy 109.22 104.14) (xy 129.54 104.14))
-    (stroke (width 0) (type default) (color 0 0 0 0))
-  )
-  (wire (pts (xy 109.22 104.14) (xy 109.22 105.41))
-    (stroke (width 0) (type default) (color 0 0 0 0))
-  )
-  (wire (pts (xy 129.54 95.25) (xy 129.54 96.52))
-    (stroke (width 0) (type default) (color 0 0 0 0))
-  )
-  (wire (pts (xy 129.54 109.22) (xy 109.22 109.22))
-    (stroke (width 0) (type default) (color 0 0 0 0))
-  )
-  (wire (pts (xy 109.22 85.09) (xy 129.54 85.09))
-    (stroke (width 0) (type default) (color 0 0 0 0))
-  )
-  (wire (pts (xy 129.54 111.76) (xy 119.38 111.76))
-    (stroke (width 0) (type default) (color 0 0 0 0))
-  )
-  (wire (pts (xy 109.22 86.36) (xy 129.54 86.36))
-    (stroke (width 0) (type default) (color 0 0 0 0))
-  )
-  (wire (pts (xy 109.22 86.36) (xy 109.22 87.63))
-    (stroke (width 0) (type default) (color 0 0 0 0))
-  )
-  (text "10 Ohm PCB Traces" (at 130.81 92.71 0)
+  (text "10 Ohm Nichrome Wire (24 Gauge?)" (at 130.81 92.71 0)
     (effects (font (size 1.27 1.27)) (justify left bottom))
   )
@@
     (pin "1")
   )
+  (symbol (lib_id "Device:Heater") (at 119.38 93.98 0) (unit 1)
+    (in_bom yes) (on_board yes) (fields_autoplaced)
+    (property "Reference" "R58" (id 0) (at 121.92 92.7099 0)
+      (effects (font (size 1.27 1.27)) (justify left))
+    )
+    (property "Value" "" (id 1) (at 121.92 95.2499 0)
+      (effects (font (size 1.27 1.27)) (justify left))
+    )
+    (property "Footprint" "" (id 2) (at 117.602 93.98 90)
+      (effects (font (size 1.27 1.27)) hide)
+    )
+    (property "Datasheet" "~" (id 3) (at 119.38 93.98 0)
+      (effects (font (size 1.27 1.27)) hide)
+    )
+    (pin "1")
+    (pin "2")
+  )
   (symbol (lib_id "Device:R") (at 175.26 93.98 0) (unit 1)
