File: ECAD/EPS/TJ-EPS.kicad_pcb (KiCad board)
At the start: 2 copper layers, 471 parts, among them J1 SWD, J10 S3B, J11 S4A, J12 S4B, J13 TELEM_IN, J2 BOOT, J5 S1A, J6 S1B, J7 S2A, J8 S2B, J9 S3A, Q1 2N7002, Q2 IRF7425, Q25 IRF7425, Q26 IRF7458, Q27 Si4186DY, Q28 SIR167DP, Q29 SIR167DP, Q30 2N7002, Q31 IRF7458, Q32 2N7002, Q33 IRF7458, Q34 2N7002, Q35 2N7002, Q36 2N7002, Q37 IRF7458, Q38 IRF7458, Q39 2N7002, Q40 2N7002, Q41 2N7002, Q42 2N7002, Q43 2N7002, Q44 2N7002, Q45 2N7002, Q46 2N7002, Q47 2N7002, Q48 IRF7458, Q49 2N7002, Q50 IRF7458, Q51 2N7002, Q52 IRF7458, Q53 2N7002, Q54 IRF7458, Q55 2N7002, Q56 IRF7458, Q57 2N7002, Q58 IRF7458, Q59 2N7002, Q60 IRF7458, Q61 2N7002, Q62 IRF7458, Q63 2N7002, Q64 IRF7458, Q65 2N7002, Q66 IRF7458, Q67 2N7002, Q68 IRF7458, Q69 2N7002, Q70 IRF7458, SW3 INHIBIT 1, U1 CD74HC4067SM, U12 LTC4412xS6, U13 MCP3208, U14 LT6106, U15 ATtiny84A-SSU, U16 L78L33_SO8, U17 MCP4812, U18 MCP4812, U19 LT6106, U2 MAX6369, U20 LT6106, U21 LM358, U22 LT3652EMSE, U23 LT6106, U24 LT6106, U25 LM358, U26 LT3652EMSE, U27 LT6106, U28 LT6106, U29 LM358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

Commit message: Add standard dimensions to batt
TODO: replace footprint of 18650
Parts:
- renumbered H2 to H1, H1 to H2
Connections:
- H2 pad 29: /SCK -> (no net)
- H2 pad 30: (no net) -> /SCK
- H2 pad 31: /MISO -> (no net)
- H2 pad 32: (no net) -> /MISO
- H2 pad 33: /MOSI -> (no net)
- H2 pad 34: (no net) -> /MOSI
- H2 pad 35: /SS -> (no net)
- H2 pad 36: (no net) -> /SS
- H2 pad 41: /SDA -> (no net)
- H2 pad 42: (no net) -> /SDA
- H2 pad 43: /SCL -> (no net)
- H2 pad 44: (no net) -> /SCL

Commit message: 18500 footprint
Parts:
- moved C1 121.8 mm to (90.7, 45.4)
- moved C12 121.8 mm to (82.2, 48.4)
- moved C13 121.8 mm to (86.7, 48.4)
- moved C3 121.8 mm to (86.3, 44.2)
- moved C4 121.8 mm to (81.8, 44.2)
- moved C6 121.8 mm to (86.3, 41.2)
- moved C7 121.8 mm to (81.8, 41.2)
- moved H1 121.8 mm to (65.7, 22.2)
- moved H2 121.8 mm to (72.9, 22.2)
- moved J1 121.8 mm to (77.5, 22.2)
- moved MH3 121.8 mm to (96.8, 43.7)
- moved MH4 121.8 mm to (103.9, 43.7)
- moved Q2 121.8 mm to (97.4, 29.7)
- moved R1 121.8 mm to (99.9, 51.7)
- moved R6 121.8 mm to (86.2, 54.4)
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
Commit message: Further descope: remove SA4
Parts:
- removed C41, C43: 10uF, Capacitor_SMD:C_0805_2012Metric
- removed C42: 1uF, Capacitor_SMD:C_0805_2012Metric
- removed the D13 at (140.4, 131.0)
- removed the D14 at (157.1, 114.6)
- removed D17: CMSH3-40MA, Diode_SMD:D_SMA
- removed D18: RB051MM-2Y, Diode_SMD:D_SOD-123F
- removed the D5 at (165.2, 114.6)
- removed the D6 at (149.1, 114.6)
- removed J10: S3B, Connector_Hirose:Hirose_DF13-04P-1.25DSA_1x04_P1.25mm_Vertical
- removed J9: S3A, Connector_Hirose:Hirose_DF13-04P-1.25DSA_1x04_P1.25mm_Vertical
- removed L1: 22uH, Inductor_SMD:L_Bourns_SRP7028A_7.3x6.6mm
- removed R72, R73: 50R, Resistor_SMD:R_0805_2012Metric
- removed R74, R75: 20m, Resistor_SMD:R_2512_6332Metric
- removed R76, R77: 5K, Resistor_SMD:R_0805_2012Metric
- removed R78: 750K, Resistor_SMD:R_0805_2012Metric
- removed R79: 100K, Resistor_SMD:R_0805_2012Metric
- removed R80: 1K, Resistor_SMD:R_0805_2012Metric
- removed R81: 7.5K, Resistor_SMD:R_0805_2012Metric
- removed R82: 52.8K, Resistor_SMD:R_0805_2012Metric
- removed R83: 490K, Resistor_SMD:R_0805_2012Metric
- removed R84: 330K, Resistor_SMD:R_0805_2012Metric
- removed R85: 50m, Resistor_SMD:R_2512_6332Metric
- removed U19, U20: LT6106, Package_TO_SOT_SMD:SOT-23-5
- removed U21: LM358, Package_SO:SO-8_3.9x4.9mm_P1.27mm
- removed U22: LT3652EMSE, Package_SO:MSOP-12-1EP_3x4mm_P0.65mm_EP1.65x2.85mm
- J11: value S4A -> S3A
- J12: value S4B -> S3B
- renumbered D15 to D13, D16 to D14, D7 to D5, D8 to D6
Connections:
- R120 pad 1: I_SA4A -> I_SA3A
- R121 pad 1: I_SA4B -> I_SA3B
- R122 pad 2: V_SA4 -> V_SA3
- R123 pad 1: V_SA4 -> V_SA3
- U1 pad 18: TELEM_IBCROUT -> (no net)
- U1 pad 19: TELEM_VBCROUT -> (no net)
- U1 pad 20: I_SA4B -> (no net)
- U1 pad 21: I_SA4A -> TELEM_IBCROUT
- U1 pad 22: V_SA4 -> TELEM_VBCROUT
- U13 pad 7: I_SA4A -> (no net)
- U13 pad 8: I_SA4B -> (no net)
- U15 pad 10: V_SA4 -> (no net)
- U18 pad 6: /SolarConditioning/Vset4 -> (no net)
- U31 pad 3: /SolarConditioning/Vset4 -> /SolarConditioning/Vset3
- U32 pad 1: I_SA4A -> I_SA3A
- U33 pad 1: I_SA4B -> I_SA3B

Commit message: wip: refine shunt resistor selection, add inhibits
Parts:
- added Q5: IRF7458, Package_SO:SOIC-8_3.9x4.9mm_P1.27mm, F.Cu at (286.0, 143.0)
- added Q7: IRF7458, Package_SO:SOIC-8_3.9x4.9mm_P1.27mm, F.Cu at (306.3, 143.0)
- added R12: 10K, Resistor_SMD:R_0805_2012Metric, F.Cu at (284.0, 147.7)
- added R13: 100R, Resistor_SMD:R_0805_2012Metric, F.Cu at (292.4, 146.7)
- added R63: 10K, Resistor_SMD:R_0805_2012Metric, F.Cu at (304.2, 147.7)
- added R64: 100R, Resistor_SMD:R_0805_2012Metric, F.Cu at (312.7, 146.7)
- added SW2: INHIBIT 2, Connector_Hirose:Hirose_DF13-02P-1.25DSA_1x02_P1.25mm_Vertical, F.Cu at (292.7, 143.0)
- added SW3: INHIBIT 3, Connector_Hirose:Hirose_DF13-02P-1.25DSA_1x02_P1.25mm_Vertical, F.Cu at (313.0, 143.0)
- R123: renamed from R219; footprint Resistor_SMD:R_2010_5025Metric -> Resistor_SMD:R_1206_3216Metric
- R131: renamed from R227; footprint Resistor_SMD:R_2010_5025Metric -> Resistor_SMD:R_1206_3216Metric
- R139: renamed from R235; footprint Resistor_SMD:R_2010_5025Metric -> Resistor_SMD:R_1206_3216Metric
- R147: renamed from R243; footprint Resistor_SMD:R_2010_5025Metric -> Resistor_SMD:R_1206_3216Metric
- R155: renamed from R251; footprint Resistor_SMD:R_2010_5025Metric -> Resistor_SMD:R_1206_3216Metric
- R16: renamed from R69; footprint Resistor_SMD:R_2010_5025Metric -> Resistor_SMD:R_1206_3216Metric
- R163: renamed from R259; footprint Resistor_SMD:R_2010_5025Metric -> Resistor_SMD:R_1206_3216Metric
- R171: renamed from R267; footprint Resistor_SMD:R_2010_5025Metric -> Resistor_SMD:R_1206_3216Metric
- R179: renamed from R275; footprint Resistor_SMD:R_2010_5025Metric -> Resistor_SMD:R_1206_3216Metric
- R187: renamed from R283; footprint Resistor_SMD:R_2010_5025Metric -> Resistor_SMD:R_1206_3216Metric
- R195: renamed from R291; footprint Resistor_SMD:R_2010_5025Metric -> Resistor_SMD:R_1206_3216Metric
- R203: renamed from R299; footprint Resistor_SMD:R_2010_5025Metric -> Resistor_SMD:R_1206_3216Metric
- R21: renamed from R88; value 20m -> 10m; footprint Resistor_SMD:R_2512_6332Metric -> Resistor_SMD:R_1206_3216Metric
- R211: renamed from R307; footprint Resistor_SMD:R_2010_5025Metric -> Resistor_SMD:R_1206_3216Metric
- R22: renamed from R89; value 20m -> 10m; footprint Resistor_SMD:R_2512_6332Metric -> Resistor_SMD:R_1206_3216Metric
- R35: renamed from R102; value 20m -> 10m; footprint Resistor_SMD:R_2512_6332Metric -> Resistor_SMD:R_1206_3216Metric
- R36: renamed from R103; value 20m -> 10m; footprint Resistor_SMD:R_2512_6332Metric -> Resistor_SMD:R_1206_3216Metric
- R49: renamed from R116; value 20m -> 10m; footprint Resistor_SMD:R_2512_6332Metric -> Resistor_SMD:R_1206_3216Metric
- R50: renamed from R117; value 20m -> 10m; footprint Resistor_SMD:R_2512_6332Metric -> Resistor_SMD:R_1206_3216Metric
- R81: renamed from R178; footprint Resistor_SMD:R_2010_5025Metric -> Resistor_SMD:R_1206_3216Metric
- R82: renamed from R181; footprint Resistor_SMD:R_2010_5025Metric -> Resistor_SMD:R_1206_3216Metric
- R83: renamed from R182; footprint Resistor_SMD:R_2010_5025Metric -> Resistor_SMD:R_1206_3216Metric
- renumbered C94 to C10, C9 to C11, C10 to C12, C11 to C13, C12 to C14, C13 to C15, C35 to C16, C36 to C17, C37 to C18, C38 to C19, C4 to C2, C39 to C20, C40 to C21, C44 to C22, C45 to C23, C46 to C24, C47 to C25, C48 to C26, C49 to C27, C50 to C28, C51 to C29, C52 to C30, C53 to C31, C54 to C32, C55 to C33, C56 to C34, C57 to C35, C60 to C36, C61 to C37, C63 to C38, C64 to C39, C5 to C4, C65 to C40, C66 to C41, C68 to C42, C69 to C43, C62 to C44, C70 to C45, C71 to C46, C72 to C47, C73 to C48, C74 to C49, C2 to C5, C75 to C50, C67 to C51, C76 to C52, C77 to C53, C78 to C54, C79 to C55, C80 to C56, C81 to C57, C82 to C58, C83 to C59, C84 to C60, C85 to C61, C86 to C62, C87 to C63, C88 to C64, C89 to C65, C90 to C66, C91 to C67, C92 to C68, C97 to C69, C93 to C7, C98 to C70, C7 to C8, C8 to C9, D12 to D10, D13 to D11, D14 to D12, D19 to D13, D20 to D14, D21 to D15, D22 to D16, D23 to D17, D24 to D18, D25 to D19, D26 to D20, D27 to D21, D28 to D22, D29 to D23, D30 to D24, D31 to D25, D32 to D26, D33 to D27, D34 to D28, D35 to D29, D36 to D30, D37 to D31, D38 to D32, D39 to D33, D9 to D7, D10 to D8, D11 to D9, H5 to H3, H6 to H4, H7 to H5, H8 to H6, J5 to J3, J6 to J4, J7 to J5, J8 to J6, J11 to J7, J12 to J8, J13 to J9, L2 to L1, L3 to L2, L4 to L3, L5 to L4, L6 to L5, L7 to L6, Q28 to Q10, Q29 to Q11, Q32 to Q12, Q33 to Q13, Q35 to Q14, Q36 to Q15, Q34 to Q16, Q37 to Q17, Q38 to Q18, Q39 to Q19, Q40 to Q20, Q41 to Q21, Q42 to Q22, Q43 to Q23, Q44 to Q24, Q45 to Q25, Q46 to Q26, Q47 to Q27, Q48 to Q28, Q49 to Q29, Q25 to Q3, Q50 to Q30, Q51 to Q31, Q52 to Q32, Q53 to Q33, Q54 to Q34, Q55 to Q35, Q56 to Q36, Q57 to Q37, Q58 to Q38, Q59 to Q39, Q26 to Q4, Q60 to Q40, Q61 to Q41, Q62 to Q42, Q63 to Q43, Q64 to Q44, Q65 to Q45, Q66 to Q46, Q67 to Q47, Q68 to Q48, Q69 to Q49, Q70 to Q50, Q27 to Q6, Q30 to Q8, Q31 to Q9, R2 to R1, R65 to R10, R197 to R100, R198 to R101, R199 to R102, R200 to R103, R201 to R104, R202 to R105, R203 to R106, R204 to R107, R205 to R108, R206 to R109, R66 to R11, R207 to R110, R208 to R111, R209 to R112, R210 to R113, R211 to R114, R212 to R115, R213 to R116, R310 to R117, R214 to R118, R215 to R119, R216 to R120, R217 to R121, R218 to R122, R220 to R124, R221 to R125, R222 to R126, R223 to R127, R224 to R128, R225 to R129, R226 to R130, R228 to R132, R229 to R133, R230 to R134, R231 to R135, R232 to R136, R233 to R137, R234 to R138, R67 to R14, R236 to R140, R237 to R141, R238 to R142, R239 to R143, R240 to R144, R241 to R145, R242 to R146, R244 to R148, R245 to R149, R68 to R15, R246 to R150, R247 to R151, R248 to R152, R249 to R153, R250 to R154, R252 to R156, R253 to R157, R254 to R158, R255 to R159, R256 to R160, R257 to R161, R258 to R162, R260 to R164, R261 to R165, R262 to R166, R263 to R167, R264 to R168, R265 to R169, R70 to R17, R266 to R170, R268 to R172, R269 to R173, R270 to R174, R271 to R175, R272 to R176, R273 to R177, R274 to R178, R71 to R18, R276 to R180, R277 to R181, R278 to R182, R279 to R183, R280 to R184, R281 to R185, R282 to R186, R284 to R188, R285 to R189, R86 to R19, R286 to R190, R287 to R191, R288 to R192, R289 to R193, R290 to R194, R292 to R196, R293 to R197, R294 to R198, R295 to R199, R1 to R2, R87 to R20, R296 to R200, R297 to R201, R298 to R202, R300 to R204, R301 to R205, R302 to R206, R303 to R207, R304 to R208, R305 to R209, R306 to R210, R308 to R212, R309 to R213, R90 to R23, R91 to R24, R92 to R25, R93 to R26, R94 to R27, R95 to R28, R96 to R29, R97 to R30, R98 to R31, R99 to R32, R100 to R33, R101 to R34, R104 to R37, R105 to R38, R106 to R39, R5 to R4, R107 to R40, R108 to R41, R109 to R42, R110 to R43, R111 to R44, R112 to R45, R113 to R46, R114 to R47, R115 to R48, R4 to R5, R118 to R51, R119 to R52, R120 to R53, R121 to R54, R122 to R55, R123 to R56, R124 to R57, R125 to R58, R126 to R59, R127 to R60, R128 to R61, R129 to R62, R164 to R65, R165 to R66, R166 to R67, R162 to R68, R163 to R69, R167 to R70, R168 to R71, R169 to R72, R170 to R73, R171 to R74, R172 to R75, R174 to R76, R175 to R77, R173 to R78, R176 to R79, R177 to R80, R179 to R84, R180 to R85, R183 to R86, R184 to R87, R185 to R88, R186 to R89, R187 to R90, R188 to R91, R189 to R92, R190 to R93, R191 to R94, R192 to R95, R193 to R96, R194 to R97, R195 to R98, R196 to R99, SW3 to SW1, U16 to U10, U17 to U11, U18 to U12, U23 to U13, U24 to U14, U25 to U15, U26 to U16, U27 to U17, U28 to U18, U29 to U19, U3 to U2, U30 to U20, U31 to U21, U32 to U22, U33 to U23, U34 to U24, U35 to U25, U46 to U26, U48 to U27, U49 to U28, U50 to U29, U2 to U3, U47 to U30, U51 to U31, U52 to U32, U53 to U33, U54 to U34, U55 to U35, U56 to U36, U57 to U37, U58 to U38, U59 to U39, U60 to U4, U62 to U40, U63 to U41, U64 to U42, U65 to U43, U66 to U44, U67 to U45, U68 to U46, U69 to U47, U70 to U48, U71 to U49, U4 to U5, U72 to U50, U73 to U51, U74 to U52, U75 to U53, U12 to U6, U13 to U7, U15 to U8, U14 to U9
Connections:
- C36 pad 1: PCM_IN -> Net-(C36-Pad1)
- C37 pad 1: PCM_IN -> Net-(C36-Pad1)
- Q4 pad 5: Net-(Q26-Pad5) -> Net-(Q4-Pad5)
- Q4 pad 6: Net-(Q26-Pad5) -> Net-(Q4-Pad5)
- Q4 pad 7: Net-(Q26-Pad5) -> Net-(Q4-Pad5)
- Q4 pad 8: Net-(Q26-Pad5) -> Net-(Q4-Pad5)
- Q9 pad 1: PCM_IN -> Net-(C36-Pad1)
- Q9 pad 2: PCM_IN -> Net-(C36-Pad1)
- Q9 pad 3: PCM_IN -> Net-(C36-Pad1)
- R14 pad 1: Net-(Q26-Pad5) -> Net-(Q5-Pad5)
- R16 pad 2: Net-(Q26-Pad5) -> Net-(Q5-Pad5)
- R17 pad 2: Net-(Q26-Pad5) -> Net-(Q5-Pad5)
- R65 pad 1: PCM_IN -> Net-(C36-Pad1)
- U26 pad 8: PCM_IN -> Net-(C36-Pad1)
- U27 pad 2: PCM_IN -> Net-(C36-Pad1)

Commit message: inhibit resistor values, among other things
Parts:
- Q2, Q3: value IRF7425 -> IRF7458

Commit message: Restandardize stack headers a bit
Parts:
- R10, R12, R63: value 10K -> 100K
Connections:
- H1 pad 10: GND -> SW2
- H1 pad 11: SW1 -> SW3
- H1 pad 12: SW2 -> SW4
- H1 pad 13: SW3 -> SW5
- H1 pad 14: SW4 -> SW6
- H1 pad 15: SW6 -> SW7
- H1 pad 16: SW5 -> SW8
- H1 pad 17: SW8 -> SW9
- H1 pad 18: SW7 -> SW10
- H1 pad 19: SW10 -> SW11
- H1 pad 20: SW9 -> SW12
- H1 pad 21: SW12 -> GND
- H1 pad 22: SW11 -> GND
- H1 pad 23: GND -> (no net)
- H1 pad 24: GND -> (no net)
- H1 pad 25: +BATT -> +5V
- H1 pad 26: +BATT -> +5V
- H1 pad 27: +5V -> +3V3
- H1 pad 28: +5V -> +3V3
- H1 pad 29: +3V3 -> GND
- H1 pad 30: +3V3 -> GND
- H1 pad 39: BCR_OUT -> (no net)
- H1 pad 40: BCR_OUT -> (no net)
- H1 pad 43: GND -> BCR_OUT
- H1 pad 44: GND -> BCR_OUT
- H1 pad 45: VUSB -> +BATT
- H1 pad 46: VUSB -> +BATT
- H1 pad 9: GND -> SW1
- H2 pad 30: /SCK -> (no net)
- H2 pad 32: /MISO -> VUSB
- H2 pad 33: (no net) -> /SCK
- H2 pad 34: /MOSI -> (no net)
- H2 pad 35: (no net) -> /MISO
- H2 pad 36: /SS -> (no net)
- H2 pad 37: (no net) -> /MOSI
- H2 pad 39: (no net) -> /SS
- H2 pad 41: (no net) -> /SDA
- H2 pad 42: /SDA -> (no net)
- H2 pad 43: (no net) -> /SCL
- H2 pad 44: /SCL -> (no net)
- R10 pad 1: /SolarConditioning/MPPT1/VOUT -> Net-(Q4-Pad4)
- R10 pad 2: Net-(Q4-Pad4) -> GND
- R11 pad 1: Net-(Q4-Pad4) -> /SolarConditioning/MPPT1/VOUT
- R12 pad 1: Net-(Q4-Pad5) -> Net-(Q5-Pad4)
- R12 pad 2: Net-(Q5-Pad4) -> GND
- R13 pad 1: Net-(Q5-Pad4) -> Net-(Q4-Pad5)
- R63 pad 1: PCM_IN -> Net-(Q7-Pad4)
- R63 pad 2: Net-(Q7-Pad4) -> GND
- R64 pad 1: Net-(Q7-Pad4) -> PCM_IN
- SW1 pad 2: GND -> Net-(Q4-Pad4)
- SW2 pad 2: GND -> Net-(Q5-Pad4)
- SW3 pad 2: GND -> Net-(Q7-Pad4)

Commit message: replace stack header footprint
Parts:
- H1, H2: footprint Connector_PinSocket_2.54mm:PinSocket_2x26_P2.54mm_Vertical -> footprints:PinSocket_2x26_P2.54mm_Vertical

Commit message: Round off some corners and set up eps board for routing
Parts:
- removed J2: BOOT, Connector_PinHeader_2.54mm:PinHeader_1x03_P2.54mm_Vertical
- added JP1: BOOT, Jumper:SolderJumper-3_P1.3mm_Open_Pad1.0x1.5mm, F.Cu at (79.6, 170.9)
- H1, H2: moved to B.Cu
- J1: value SWD -> SWD/DEBUG; footprint Connector_PinHeader_2.54mm:PinHeader_1x04_P2.54mm_Horizontal -> Connector_PinHeader_2.54mm:PinHeader_1x06_P2.54mm_Vertical
- moved C25 158.5 mm to (127.7, 325.4)
- moved D16 158.5 mm to (112.2, 328.9)
- moved D33 158.5 mm to (214.8, 305.1)
- moved H4 158.5 mm to (163.0, 283.0)
- moved J4 158.5 mm to (137.6, 274.0)
- moved J7 158.5 mm to (128.9, 274.0)
- moved Q35 158.5 mm to (235.8, 261.0)
- moved Q45 158.5 mm to (264.6, 260.1)
- moved Q50 158.5 mm to (215.0, 299.6)
- moved R105 158.5 mm to (246.8, 283.7)
- moved R11 158.5 mm to (168.3, 286.0)
- moved R150 158.5 mm to (237.2, 264.8)
- moved R153 158.5 mm to (232.8, 264.8)
- moved R19 158.5 mm to (201.3, 260.0)
- moved R191 158.5 mm to (261.6, 263.9)
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Connections:
- U5 pad 32: (no net) -> /D-
- U5 pad 33: (no net) -> /D+
Other:
- board outline added: 90.2 x 95.9 mm
