File: ECAD/EPS/TJ-EPS.sch (KiCad schematic (older format))
At the start: 41 parts, among them J1 SWD, J2 BOOT, Q1 2N7002, Q2 IRF7425, U1 CD74HC4067SM, U2 MAX6369, U3 CD74HC4067SM, U4 STM32F103C8Tx, U60 CD74HC4067SM, Y1 8MHz

Commit message: Split up into 3 projects for separate boards
Connections:
- net MUX3OUT: no longer names the net of U4.13 (PA3)
Changed lines of the file:
@@
 $Descr USLegal 14000 8500
 encoding utf-8
-Sheet 1 37
+Sheet 1 32
 Title "TJ Custom EPS"
 Date ""
@@
 $Sheet
 S 10400 2550 1100 250
-U 61BD4B7D
-F0 "Battery" 50
-F1 "BatteryMaster.sch" 50
-$EndSheet
-$Sheet
-S 10400 2100 1100 250
 U 61BEC565
 F0 "SolarConditioning" 50
@@
 Text GLabel 8650 2450 2    50   Input ~ 0
 MUX2OUT
-Text GLabel 8650 2550 2    50   Input ~ 0
-MUX3OUT
 Text GLabel 8650 3250 2    50   Input ~ 0
 RSTBATV

Commit message: Add standard dimensions to batt
TODO: replace footprint of 18650
Parts:
- renumbered H2 to H1, H1 to H2
Connections:
- net MISO: now also H2.32 (Pin_32); no longer H2.31 (Pin_31)
- net MOSI: now also H2.34 (Pin_34); no longer H2.33 (Pin_33)
- net SCK: now also H2.30 (Pin_30); no longer H2.29 (Pin_29)
- net SCL: now also H2.44 (Pin_44); no longer H2.43 (Pin_43)
- net SDA: now also H2.42 (Pin_42); no longer H2.41 (Pin_41)
- net SS: now also H2.36 (Pin_36); no longer H2.35 (Pin_35)
Other:
- moved on the sheet: H1, H2

Commit message: Further descope: remove SA4
Connections:
- net I_SA4A is gone; now on net TELEM_IBCROUT: U1.21 (I10)
- net V_SA4 is gone; now on net TELEM_VBCROUT: U1.22 (I9)
- net TELEM_IBCROUT: no longer U1.18 (I13)
- net TELEM_VBCROUT: no longer U1.19 (I12)
- net I_SA4B: no longer names the net of U1.20 (I11)
Changed lines of the file:
@@
 $Descr USLegal 14000 8500
 encoding utf-8
-Sheet 1 23
+Sheet 1 22
 Title "TJ Custom EPS"
 Date ""
@@
 Text GLabel 1450 6650 0    50   Input ~ 0
 I_SA3B
-Text GLabel 1450 6850 0    50   Input ~ 0
-I_SA4A
-Text GLabel 1450 6950 0    50   Input ~ 0
-I_SA4B
 Text GLabel 1450 6050 0    50   Input ~ 0
 I_SA1B
@@
 V_SA3
 Text GLabel 1450 6750 0    50   Input ~ 0
-V_SA4
-Text GLabel 1450 7050 0    50   Input ~ 0
 TELEM_VBCROUT
-Text GLabel 1450 7150 0    50   Input ~ 0
+Text GLabel 1450 6850 0    50   Input ~ 0
 TELEM_IBCROUT
 $Comp

Commit message: wip: refine shunt resistor selection, add inhibits
Parts:
- renumbered C94 to C10, C9 to C11, C10 to C12, C11 to C13, C12 to C14, C13 to C15, C4 to C2, C5 to C4, C2 to C5, C93 to C7, C7 to C8, C8 to C9, R2 to R1, R1 to R2, R5 to R4, R4 to R5, U3 to U2, U2 to U3, U60 to U4, U4 to U5

Commit message: inhibit resistor values, among other things
Parts:
- Q2: value IRF7425 -> IRF7458
Changed lines of the file:
@@
 P 5800 1250
 F 0 "Q2" H 6005 1204 50  0000 L CNN
-F 1 "IRF7425" H 6005 1295 50  0000 L CNN
+F 1 "IRF7458" H 6005 1295 50  0000 L CNN
 F 2 "Package_SO:SOIC-8_3.9x4.9mm_P1.27mm" H 6000 1175 50  0001 L CIN
 F 3 "http://www.infineon.com/dgdl/irf7404.pdf?fileId=5546d462533600a4015355fa2b5b1b9e" V 5800 1250 50  0001 L CNN

Commit message: Restandardize stack headers a bit
Connections:
- net +3V3: now also H1.27 (Pin_27), H1.28 (Pin_28); no longer H1.29 (Pin_29), H1.30 (Pin_30)
- net +5V: now also H1.25 (Pin_25), H1.26 (Pin_26); no longer H1.27 (Pin_27), H1.28 (Pin_28)
- net +BATT: now also H1.45 (Pin_45), H1.46 (Pin_46); no longer H1.25 (Pin_25), H1.26 (Pin_26)
- net BCR_OUT: now also H1.43 (Pin_43), H1.44 (Pin_44); no longer H1.39 (Pin_39), H1.40 (Pin_40)
- net GND: now also H1.21 (Pin_21), H1.22 (Pin_22), H1.29 (Pin_29), H1.30 (Pin_30); no longer H1.10 (Pin_10), H1.23 (Pin_23), H1.24 (Pin_24), H1.43 (Pin_43), H1.44 (Pin_44), H1.9 (Pin_9)
- net MISO: now also H2.35 (Pin_35); no longer H2.32 (Pin_32)
- net MOSI: now also H2.37 (Pin_37); no longer H2.34 (Pin_34)
- net SCK: now also H2.33 (Pin_33); no longer H2.30 (Pin_30)
- net SCL: now also H2.43 (Pin_43); no longer H2.44 (Pin_44)
- net SDA: now also H2.41 (Pin_41); no longer H2.42 (Pin_42)
- net SS: now also H2.39 (Pin_39); no longer H2.36 (Pin_36)
- net SW1: now also H1.9 (Pin_9); no longer H1.11 (Pin_11)
- net SW10: now also H1.18 (Pin_18); no longer H1.19 (Pin_19)
- net SW11: now also H1.19 (Pin_19); no longer H1.22 (Pin_22)
- net SW12: now also H1.20 (Pin_20); no longer H1.21 (Pin_21)
- net SW2: now also H1.10 (Pin_10); no longer H1.12 (Pin_12)
- net SW3: now also H1.11 (Pin_11); no longer H1.13 (Pin_13)
- net SW4: now also H1.12 (Pin_12); no longer H1.14 (Pin_14)
- net SW5: now also H1.13 (Pin_13); no longer H1.16 (Pin_16)
- net SW6: now also H1.14 (Pin_14); no longer H1.15 (Pin_15)
- net SW7: now also H1.15 (Pin_15); no longer H1.18 (Pin_18)
- net SW8: now also H1.16 (Pin_16); no longer H1.17 (Pin_17)
- net SW9: now also H1.17 (Pin_17); no longer H1.20 (Pin_20)
- net VUSB: now also H2.32 (Pin_32); no longer H1.45 (Pin_45), H1.46 (Pin_46)
- no-connect marks 18 -> 22
Other:
- moved on the sheet: H1, H2

Commit message: replace stack header footprint
Parts:
- H1, H2: footprint Connector_PinSocket_2.54mm:PinSocket_2x26_P2.54mm_Vertical -> footprints:PinSocket_2x26_P2.54mm_Vertical
Changed lines of the file:
@@
 F 0 "H2" H 1150 3667 50  0000 C CNN
 F 1 "Stack Header 2" H 1150 3576 50  0000 C CNN
-F 2 "Connector_PinSocket_2.54mm:PinSocket_2x26_P2.54mm_Vertical" H 1100 2250 50  0001 C CNN
+F 2 "footprints:PinSocket_2x26_P2.54mm_Vertical" H 1100 2250 50  0001 C CNN
 F 3 "~" H 1100 2250 50  0001 C CNN
 	1    1100 2250
@@
 F 0 "H1" H 2350 3667 50  0000 C CNN
 F 1 "Stack Header 1" H 2350 3576 50  0000 C CNN
-F 2 "Connector_PinSocket_2.54mm:PinSocket_2x26_P2.54mm_Vertical" H 2300 2250 50  0001 C CNN
+F 2 "footprints:PinSocket_2x26_P2.54mm_Vertical" H 2300 2250 50  0001 C CNN
 F 3 "~" H 2300 2250 50  0001 C CNN
 	1    2300 2250

Commit message: Round off some corners and set up eps board for routing
Parts:
- removed J1: SWD, Connector_PinHeader_2.54mm:PinHeader_1x04_P2.54mm_Horizontal, symbol Connector:Conn_01x04_Male
- removed J2: BOOT, Connector_PinHeader_2.54mm:PinHeader_1x03_P2.54mm_Vertical, symbol Connector:Conn_01x03_Male
- added J1: SWD/DEBUG, Connector_PinHeader_2.54mm:PinHeader_1x06_P2.54mm_Vertical, symbol Connector:Conn_01x06_Male
- added JP1: BOOT, Jumper:SolderJumper-3_P1.3mm_Open_Pad1.0x1.5mm, symbol Jumper:SolderJumper_3_Open
Connections:
- net GND: now also J1.4 (Pin_4), JP1.1 (A)
- net SWDCLK: now also J1.3 (Pin_3)
- net SWDIO: now also J1.2 (Pin_2)
- net VDD: now also J1.1 (Pin_1), JP1.3 (B)
- net at R6.2: now also JP1.2 (C)
- net D-: now reaches U5.32 (PA11)
- net D-: now also J1.5 (Pin_5)
- net D+: now reaches U5.33 (PA12)
- net D+: now also J1.6 (Pin_6)
Other:
- moved on the sheet: R4, R6
Changed lines of the file:
@@
 Wire Notes Line
 	6400 600  6400 4450
-Wire Notes Line
-	6350 2250 6350 4000
-Wire Notes Line
-	4700 2250 4700 4000
 Text Notes 4750 2350 0    50   ~ 0
 Programming Headers & the like
@@
 	6350 2250 4700 2250
 Wire Notes Line
-	4700 4000 6350 4000
+	4700 4450 6350 4450
+Wire Wire Line
+	5350 3850 5650 3850
+Wire Wire Line
+	5350 3550 5650 3550
 Wire Wire Line
 	5350 3750 5650 3750
 Wire Wire Line
-	5350 3450 5650 3450
-Wire Wire Line
 	5350 3650 5650 3650
-Wire Wire Line
-	5350 3550 5650 3550
 $Comp
 L power:VDD #PWR017
 U 1 1 629CA474
-P 5650 3450
-F 0 "#PWR017" H 5650 3300 50  0001 C CNN
-F 1 "VDD" H 5665 3623 50  0000 C CNN
-F 2 "" H 5650 3450 50  0001 C CNN
-F 3 "" H 5650 3450 50  0001 C CNN
-	1    5650 3450
+P 5650 3550
+F 0 "#PWR017" H 5650 3400 50  0001 C CNN
+F 1 "VDD" H 5665 3723 50  0000 C CNN
+F 2 "" H 5650 3550 50  0001 C CNN
+F 3 "" H 5650 3550 50  0001 C CNN
+	1    5650 3550
 	1    0    0    -1
 $EndComp
@@
 L power:VDD #PWR015
 U 1 1 629C1F75
-P 5650 2600
-F 0 "#PWR015" H 5650 2450 50  0001 C CNN
-F 1 "VDD" H 5665 2773 50  0000 C CNN
-F 2 "" H 5650 2600 50  0001 C CNN
-F 3 "" H 5650 2600 50  0001 C CNN
-	1    5650 2600
+P 5400 2550
+F 0 "#PWR015" H 5400 2400 50  0001 C CNN
+F 1 "VDD" H 5415 2723 50  0000 C CNN
+F 2 "" H 5400 2550 50  0001 C CNN
+F 3 "" H 5400 2550 50  0001 C CNN
+	1    5400 2550
 	1    0    0    -1
 $EndComp
@@
 L power:GND #PWR?
 U 1 1 61DD0707
-P 5650 3750
+P 5650 3850
 AR Path="/61BD4B7D/61DD0707" Ref="#PWR?"  Part="1"
 AR Path="/61DD0707" Ref="#PWR018"  Part="1"
-F 0 "#PWR018" H 5650 3500 50  0001 C CNN
-F 1 "GND" H 5655 3577 50  0000 C CNN
-F 2 "" H 5650 3750 50  0001 C CNN
-F 3 "" H 5650 3750 50  0001 C CNN
-	1    5650 3750
-	1    0    0    -1
-$EndComp
+F 0 "#PWR018" H 5650 3600 50  0001 C CNN
+F 1 "GND" H 5655 3677 50  0000 C CNN
+F 2 "" H 5650 3850 50  0001 C CNN
+F 3 "" H 5650 3850 50  0001 C CNN
+	1    5650 3850
+	1    0    0    -1
+$EndComp
+Text Label 5650 3750 2    50   ~ 0
+SWDCLK
 Text Label 5650 3650 2    50   ~ 0
-SWDCLK
-Text Label 5650 3550 2    50   ~ 0
 SWDIO
-$Comp
-L Connector:Conn_01x04_Male J?
-U 1 1 61DD06F5
-P 5150 3550
-AR Path="/61BD4B7D/61DD06F5" Ref="J?"  Part="1"
-AR Path="/61DD06F5" Ref="J1"  Part="1"
-F 0 "J1" H 5258 3831 50  0000 C CNN
-F 1 "SWD" H 5258 3740 50  0000 C CNN
-F 2 "Connector_PinHeader_2.54mm:PinHeader_1x04_P2.54mm_Horizontal" H 5150 3550 50  0001 C CNN
-F 3 "~" H 5150 3550 50  0001 C CNN
-	1    5150 3550
-	1    0    0    -1
-$EndComp
 $Comp
 L power:GND #PWR012
 U 1 1 61DB8500
-P 5150 3000
+P 5050 3000
 AR Path="/61DB8500" Ref="#PWR012"  Part="1"
 AR Path="/61BD4B7D/61DB8500" Ref="#PWR?"  Part="1"
-F 0 "#PWR012" H 5150 2750 50  0001 C CNN
-F 1 "GND" H 5155 2827 50  0000 C CNN
-F 2 "" H 5150 3000 50  0001 C CNN
-F 3 "" H 5150 3000 50  0001 C CNN
-	1    5150 3000
+F 0 "#PWR012" H 5050 2750 50  0001 C CNN
+F 1 "GND" H 5055 2827 50  0000 C CNN
+F 2 "" H 5050 3000 50  0001 C CNN
+F 3 "" H 5050 3000 50  0001 C CNN
+	1    5050 3000
 	1    0    0    -1
 $EndComp
@@
 L power:GND #PWR016
 U 1 1 61DB84FA
-P 5650 3000
+P 5400 3150
 AR Path="/61DB84FA" Ref="#PWR016"  Part="1"
 AR Path="/61BD4B7D/61DB84FA" Ref="#PWR?"  Part="1"
-F 0 "#PWR016" H 5650 2750 50  0001 C CNN
-F 1 "GND" H 5655 2827 50  0000 C CNN
-F 2 "" H 5650 3000 50  0001 C CNN
-F 3 "" H 5650 3000 50  0001 C CNN
-	1    5650 3000
-	1    0    0    -1
-$EndComp
-Wire Wire Line
-	5650 2900 5650 3000
-Wire Wire Line
-	5550 2900 5650 2900
-Wire Wire Line
-	5650 2700 5650 2600
-Wire Wire Line
-	5550 2700 5650 2700
-$Comp
-L Connector:Conn_01x03_Male J?
-U 1 1 61DB84EA
-P 5350 2800
-AR Path="/61BD4B7D/61DB84EA" Ref="J?"  Part="1"
-AR Path="/61DB84EA" Ref="J2"  Part="1"
-F 0 "J2" H 5458 3081 50  0000 C CNN
-F 1 "BOOT" H 5458 2990 50  0000 C CNN
-F 2 "Connector_PinHeader_2.54mm:PinHeader_1x03_P2.54mm_Vertical" H 5350 2800 50  0001 C CNN
-F 3 "~" H 5350 2800 50  0001 C CNN
-	1    5350 2800
-	1    0    0    -1
-$EndComp
+F 0 "#PWR016" H 5400 2900 50  0001 C CNN
+F 1 "GND" H 5405 2977 50  0000 C CNN
+F 2 "" H 5400 3150 50  0001 C CNN
+F 3 "" H 5400 3150 50  0001 C CNN
+	1    5400 3150
+	1    0    0    -1
+$EndComp
+Wire Wire Line
+	5400 3050 5400 3150
+Wire Wire Line
+	5400 2650 5400 2550
 $Comp
 L Device:R R?
 U 1 1 61DB84E4
-P 5700 2800
+P 5700 2850
 AR Path="/61BD4B7D/61DB84E4" Ref="R?"  Part="1"
 AR Path="/61DB84E4" Ref="R6"  Part="1"
-F 0 "R6" V 5600 2800 50  0000 C CNN
-F 1 "100K" V 5700 2800 50  0000 C CNN
-F 2 "Resistor_SMD:R_0805_2012Metric" V 5630 2800 50  0001 C CNN
-F 3 "~" H 5700 2800 50  0001 C CNN
-	1    5700 2800
+F 0 "R6" V 5600 2850 50  0000 C CNN
+F 1 "100K" V 5700 2850 50  0000 C CNN
+F 2 "Resistor_SMD:R_0805_2012Metric" V 5630 2850 50  0001 C CNN
+F 3 "~" H 5700 2850 50  0001 C CNN
+	1    5700 2850
 	0    1    1    0
 $EndComp
@@
 L Device:R R?
 U 1 1 61DB84DE
-P 5150 2850
+P 5050 2850
 AR Path="/61BD4B7D/61DB84DE" Ref="R?"  Part="1"
 AR Path="/61DB84DE" Ref="R4"  Part="1"
-F 0 "R4" V 5050 2850 50  0000 C CNN
-F 1 "100K" V 5150 2850 50  0000 C CNN
-F 2 "Resistor_SMD:R_0805_2012Metric" V 5080 2850 50  0001 C CNN
-F 3 "~" H 5150 2850 50  0001 C CNN
-	1    5150 2850
-	1    0    0    -1
-$EndComp
-Text Label 4850 2700 0    50   ~ 0
+F 0 "R4" V 4950 2850 50  0000 C CNN
+F 1 "100K" V 5050 2850 50  0000 C CNN
+F 2 "Resistor_SMD:R_0805_2012Metric" V 4980 2850 50  0001 C CNN
+F 3 "~" H 5050 2850 50  0001 C CNN
+	1    5050 2850
+	1    0    0    -1
+$EndComp
+Text Label 4750 2700 0    50   ~ 0
 BOOT1
 Wire Wire Line
-	5150 2700 4850 2700
-Text Label 6150 2800 2    50   ~ 0
+	5050 2700 4750 2700
+Text Label 6150 2850 2    50   ~ 0
 BOOT0
 Wire Wire Line
-	5850 2800 6150 2800
+	5850 2850 6150 2850
 Text Notes 3150 700  0    50   ~ 0
 Latchup WDT
@@
 NoConn ~ 2100 2150
 NoConn ~ 2600 2150
+$Comp
+L Jumper:SolderJumper_3_Open JP1
+U 1 1 61F77E37
+P 5400 2850
+F 0 "JP1" V 5446 2917 50  0000 L CNN
+F 1 "BOOT" V 5355 2917 50  0000 L CNN
+F 2 "Jumper:SolderJumper-3_P1.3mm_Open_Pad1.0x1.5mm" H 5400 2850 50  0001 C CNN
+F 3 "~" H 5400 2850 50  0001 C CNN
+	1    5400 2850
+	0    -1   -1   0
+$EndComp
+Wire Notes Line
+	6350 2250 6350 4450
+Wire Notes Line
+	4700 2250 4700 4450
+$Comp
+L Connector:Conn_01x06_Male J1
+U 1 1 61FB2226
+P 5150 3750
+F 0 "J1" H 5258 4131 50  0000 C CNN
+F 1 "SWD/DEBUG" H 5258 4040 50  0000 C CNN
+F 2 "Connector_PinHeader_2.54mm:PinHeader_1x06_P2.54mm_Vertical" H 5150 3750 50  0001 C CNN
+F 3 "~" H 5150 3750 50  0001 C CNN
+	1    5150 3750
+	1    0    0    -1
+$EndComp
+Wire Wire Line
+	5350 3950 5550 3950
+Wire Wire Line
+	5350 4050 5550 4050
+Text Label 5550 3950 2    50   ~ 0
+D-
+Text Label 5550 4050 2    50   ~ 0
+D+
+Wire Wire Line
+	8650 3350 8850 3350
+Wire Wire Line
+	8650 3450 8850 3450
+Text Label 8850 3350 2    50   ~ 0
+D-
+Text Label 8850 3450 2    50   ~ 0
+D+
 $EndSCHEMATC
