File: ECAD/EPS/TJ-EPS.sch (KiCad schematic (older format))
At the start: 41 parts, among them J1 SWD/DEBUG, Q1 2N7002, Q2 IRF7458, U1 CD74HC4067SM, U2 CD74HC4067SM, U3 MAX6369, U4 CD74HC4067SM, U5 STM32F103C8Tx, Y1 8MHz

Commit message: Replace EVERY LT6106 with INA180A3
Friendship ended with LT6106
now ina180 is my best friend
Parts:
- renumbered H2 to H1, H1 to H2, R4 to R3, R3 to R4
Changed lines of the file:
@@
 $EndDescr
 $Comp
-L Connector_Generic:Conn_02x26_Odd_Even H2
+L Connector_Generic:Conn_02x26_Odd_Even H1
 U 1 1 61BB9DA8
 P 1100 2250
-F 0 "H2" H 1150 3667 50  0000 C CNN
+F 0 "H1" H 1150 3667 50  0000 C CNN
 F 1 "Stack Header 2" H 1150 3576 50  0000 C CNN
 F 2 "footprints:PinSocket_2x26_P2.54mm_Vertical" H 1100 2250 50  0001 C CNN
@@
 SW10
 $Comp
-L power:+5V #PWR04
+L power:+5V #PWR03
 U 1 1 61BC34F8
 P 2100 2250
-F 0 "#PWR04" H 2100 2100 50  0001 C CNN
+F 0 "#PWR03" H 2100 2100 50  0001 C CNN
 F 1 "+5V" V 2115 2378 50  0000 L CNN
 F 2 "" H 2100 2250 50  0001 C CNN
@@
 $EndComp
 $Comp
-L power:+5V #PWR08
+L power:+5V #PWR07
 U 1 1 61BC3941
 P 2600 2250
-F 0 "#PWR08" H 2600 2100 50  0001 C CNN
+F 0 "#PWR07" H 2600 2100 50  0001 C CNN
 F 1 "+5V" V 2615 2378 50  0000 L CNN
 F 2 "" H 2600 2250 50  0001 C CNN
@@
 $EndComp
 $Comp
-L power:+3V3 #PWR05
+L power:+3V3 #PWR04
 U 1 1 61BC3DF9
 P 2100 2350
-F 0 "#PWR05" H 2100 2200 50  0001 C CNN
+F 0 "#PWR04" H 2100 2200 50  0001 C CNN
 F 1 "+3V3" V 2115 2478 50  0000 L CNN
 F 2 "" H 2100 2350 50  0001 C CNN
@@
 $EndComp
 $Comp
-L power:+3V3 #PWR09
+L power:+3V3 #PWR08
 U 1 1 61BC42A2
 P 2600 2350
-F 0 "#PWR09" H 2600 2200 50  0001 C CNN
+F 0 "#PWR08" H 2600 2200 50  0001 C CNN
 F 1 "+3V3" V 2615 2478 50  0000 L CNN
 F 2 "" H 2600 2350 50  0001 C CNN
@@
 BCR_OUT
 $Comp
-L power:+BATT #PWR07
+L power:+BATT #PWR09
 U 1 1 61BC5790
 P 2600 3250
-F 0 "#PWR07" H 2600 3100 50  0001 C CNN
+F 0 "#PWR09" H 2600 3100 50  0001 C CNN
 F 1 "+BATT" V 2600 3350 50  0000 L CNN
 F 2 "" H 2600 3250 50  0001 C CNN
@@
 $EndComp
 $Comp
-L power:+BATT #PWR03
+L power:+BATT #PWR05
 U 1 1 61BC64DC
 P 2100 3250
-F 0 "#PWR03" H 2100 3100 50  0001 C CNN
+F 0 "#PWR05" H 2100 3100 50  0001 C CNN
 F 1 "+BATT" V 2100 3350 50  0000 L CNN
 F 2 "" H 2100 3250 50  0001 C CNN
@@
 P 5150 1100
 AR Path="/61BD4B7D/6296E260" Ref="R?"  Part="1"
-AR Path="/6296E260" Ref="R3"  Part="1"
-F 0 "R3" H 5200 1100 50  0000 L CNN
+AR Path="/6296E260" Ref="R4"  Part="1"
+F 0 "R4" H 5200 1100 50  0000 L CNN
 F 1 "10K" V 5150 1100 50  0000 C CNN
 F 2 "Resistor_SMD:R_0805_2012Metric" V 5080 1100 50  0001 C CNN
@@
 NoConn ~ 2100 1350
 $Comp
-L Connector_Generic:Conn_02x26_Odd_Even H1
+L Connector_Generic:Conn_02x26_Odd_Even H2
 U 1 1 61BBDB62
 P 2300 2250
-F 0 "H1" H 2350 3667 50  0000 C CNN
+F 0 "H2" H 2350 3667 50  0000 C CNN
 F 1 "Stack Header 1" H 2350 3576 50  0000 C CNN
 F 2 "footprints:PinSocket_2x26_P2.54mm_Vertical" H 2300 2250 50  0001 C CNN
@@
 P 5050 2850
 AR Path="/61BD4B7D/61DB84DE" Ref="R?"  Part="1"
-AR Path="/61DB84DE" Ref="R4"  Part="1"
-F 0 "R4" V 4950 2850 50  0000 C CNN
+AR Path="/61DB84DE" Ref="R3"  Part="1"
+F 0 "R3" V 4950 2850 50  0000 C CNN
 F 1 "100K" V 5050 2850 50  0000 C CNN
 F 2 "Resistor_SMD:R_0805_2012Metric" V 4980 2850 50  0001 C CNN

Commit message: change some power flags for latchup prevention
Connections:
- net +3V3: no longer C1.1, C4.1, C7.1, R7.1, R8.1, U1.24 (VCC), U2.24 (VCC), U4.24 (VCC)
- net VDD: now also C1.1, C4.1, C7.1, R7.1, R8.1, U1.24 (VCC), U2.24 (VCC), U4.24 (VCC)
Changed lines of the file:
@@
 	8650 850  8650 1400
 Connection ~ 8800 1400
-Connection ~ 6650 2550
-$Comp
-L power:+3V3 #PWR022
-U 1 1 61D61EDB
-P 6650 2550
-AR Path="/61D61EDB" Ref="#PWR022"  Part="1"
-AR Path="/61BD4B7D/61D61EDB" Ref="#PWR?"  Part="1"
-F 0 "#PWR022" H 6650 2400 50  0001 C CNN
-F 1 "+3V3" V 6665 2678 50  0000 L CNN
-F 2 "" H 6650 2550 50  0001 C CNN
-F 3 "" H 6650 2550 50  0001 C CNN
-	1    6650 2550
-	1    0    0    -1
-$EndComp
 Wire Wire Line
 	700  3050 900  3050
@@
 Text GLabel 7150 6050 2    50   Input ~ 0
 MUX2OUT
-$Comp
-L power:+3V3 #PWR013
-U 1 1 61EACF2A
-P 5350 5550
-AR Path="/61EACF2A" Ref="#PWR013"  Part="1"
-AR Path="/61BD4B7D/61EACF2A" Ref="#PWR?"  Part="1"
-AR Path="/61E87E93/61EACF2A" Ref="#PWR?"  Part="1"
-F 0 "#PWR013" H 5350 5400 50  0001 C CNN
-F 1 "+3V3" V 5365 5678 50  0000 L CNN
-F 2 "" H 5350 5550 50  0001 C CNN
-F 3 "" H 5350 5550 50  0001 C CNN
-	1    5350 5550
-	1    0    0    -1
-$EndComp
 Wire Wire Line
 	6450 5550 5350 5550
@@
 	4950 7650 5350 7650
 Connection ~ 4950 7650
-Wire Wire Line
-	4250 5550 5350 5550
 Connection ~ 4250 5550
 $Comp
@@
 Text Label 8850 3450 2    50   ~ 0
 D+
+$Comp
+L power:VDD #PWR?
+U 1 1 61FB25F1
+P 6650 2550
+F 0 "#PWR?" H 6650 2400 50  0001 C CNN
+F 1 "VDD" H 6665 2723 50  0000 C CNN
+F 2 "" H 6650 2550 50  0001 C CNN
+F 3 "" H 6650 2550 50  0001 C CNN
+	1    6650 2550
+	1    0    0    -1
+$EndComp
+Connection ~ 6650 2550
+$Comp
+L power:VDD #PWR?
+U 1 1 61FCB802
+P 5350 5550
+F 0 "#PWR?" H 5350 5400 50  0001 C CNN
+F 1 "VDD" H 5365 5723 50  0000 C CNN
+F 2 "" H 5350 5550 50  0001 C CNN
+F 3 "" H 5350 5550 50  0001 C CNN
+	1    5350 5550
+	1    0    0    -1
+$EndComp
+Wire Wire Line
+	4250 5550 5350 5550
 $EndSCHEMATC
