File: ECAD/EPS/PDMBATV.sch (KiCad schematic (older format))
At the start: 12 parts, among them Q67 2N7002, Q68 IRF7458, U74 LT6106

Commit message: wip: refine shunt resistor selection, add inhibits
Parts:
- R203: renamed from R299; footprint Resistor_SMD:R_2010_5025Metric -> Resistor_SMD:R_1206_3216Metric
- renumbered D38 to D32, Q67 to Q47, Q68 to Q48, R294 to R198, R295 to R199, R296 to R200, R297 to R201, R298 to R202, R300 to R204, R301 to R205, U74 to U52

Commit message: work
Parts:
- D32: value 1N4004 -> RR264MM; footprint Diode_SMD:D_SMA -> Diode_SMD:D_SOD-123F
Connections:
- net VOUT: now also D32.1 (K)
- net at Q48.1 (S), Q48.2 (S), Q48.3 (S)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: no longer D32.1 (K)
Other:
- moved on the sheet: D32
Changed lines of the file:
@@
 $Descr A4 11693 8268
 encoding utf-8
-Sheet 20 22
+Sheet 21 22
 Title "TJ Custom EPS"
 Date ""
@@
 Text HLabel 3300 2500 0    50   Input ~ 0
 GATE
-Text HLabel 6000 2350 2    50   Input ~ 0
+Text HLabel 7450 2350 2    50   Input ~ 0
 VOUT
 Text HLabel 6900 2850 2    50   Input ~ 0
@@
 AR Path="/61E87E93/61EEB97A/61EEB9DE" Ref="Q?"  Part="1"
 AR Path="/61E87E93/61EB04DF/61EEB9DE" Ref="Q50"  Part="1"
-F 0 "Q50" H 4755 2196 50  0000 L CNN
+F 0 "Q48" H 4755 2196 50  0000 L CNN
 F 1 "IRF7458" H 4755 2105 50  0000 L CNN
 F 2 "Package_SO:SOIC-8_3.9x4.9mm_P1.27mm" H 4750 2075 50  0001 L CIN
@@
 AR Path="/61E87E93/61EEB97A/61EEB9DF" Ref="Q?"  Part="1"
 AR Path="/61E87E93/61EB04DF/61EEB9DF" Ref="Q49"  Part="1"
-F 0 "Q49" H 4304 2546 50  0000 L CNN
+F 0 "Q47" H 4304 2546 50  0000 L CNN
 F 1 "2N7002" H 4304 2455 50  0000 L CNN
 F 2 "Package_TO_SOT_SMD:SOT-23" H 4300 2425 50  0001 L CIN
@@
 AR Path="/61E87E93/61EEB97A/61EEB9E0" Ref="R?"  Part="1"
 AR Path="/61E87E93/61EB04DF/61EEB9E0" Ref="R208"  Part="1"
-F 0 "R208" H 4250 1850 50  0000 L CNN
+F 0 "R200" H 4250 1850 50  0000 L CNN
 F 1 "10K" V 4200 1850 50  0000 C CNN
 F 2 "Resistor_SMD:R_0805_2012Metric" V 4130 1850 50  0001 C CNN
@@
 L Device:D D?
 U 1 1 61E99672
-P 4650 2550
+P 7450 2500
 AR Path="/61E87E93/61E898DE/61E99672" Ref="D?"  Part="1"
 AR Path="/61E87E93/61ED0AEF/61E99672" Ref="D?"  Part="1"
@@
 AR Path="/61E87E93/61EEB97A/61E99672" Ref="D?"  Part="1"
 AR Path="/61E87E93/61EB04DF/61E99672" Ref="D33"  Part="1"
-F 0 "D33" V 4604 2630 50  0000 L CNN
-F 1 "1N4004" V 4695 2630 50  0000 L CNN
-F 2 "Diode_SMD:D_SMA" H 4650 2550 50  0001 C CNN
-F 3 "~" H 4650 2550 50  0001 C CNN
-	1    4650 2550
+F 0 "D32" V 7404 2580 50  0000 L CNN
+F 1 "RR264MM" V 7495 2580 50  0000 L CNN
+F 2 "Diode_SMD:D_SOD-123F" H 7450 2500 50  0001 C CNN
+F 3 "~" H 7450 2500 50  0001 C CNN
+	1    7450 2500
 	0    1    1    0
 $EndComp
-Wire Wire Line
-	4650 2350 4650 2400
 $Comp
 L Device:R R?
@@
 AR Path="/61E87E93/61EEB97A/61EEB9E2" Ref="R?"  Part="1"
 AR Path="/61E87E93/61EB04DF/61EEB9E2" Ref="R206"  Part="1"
-F 0 "R206" V 3450 2500 50  0000 C CNN
+F 0 "R198" V 3450 2500 50  0000 C CNN
 F 1 "100R" V 3550 2500 50  0000 C CNN
 F 2 "Resistor_SMD:R_0805_2012Metric" V 3480 2500 50  0001 C CNN
@@
 AR Path="/61E87E93/61EEB97A/61EEB9E3" Ref="R?"  Part="1"
 AR Path="/61E87E93/61EB04DF/61EEB9E3" Ref="R207"  Part="1"
-F 0 "R207" H 3850 2650 50  0000 L CNN
+F 0 "R199" H 3850 2650 50  0000 L CNN
 F 1 "10K" V 3800 2650 50  0000 C CNN
 F 2 "Resistor_SMD:R_0805_2012Metric" V 3730 2650 50  0001 C CNN
@@
 AR Path="/61E87E93/61EEB97A/61EEB9E4" Ref="#PWR?"  Part="1"
 AR Path="/61E87E93/61EB04DF/61EEB9E4" Ref="#PWR0123"  Part="1"
-F 0 "#PWR0123" H 4650 2900 50  0001 C CNN
+F 0 "#PWR0121" H 4650 2900 50  0001 C CNN
 F 1 "GND" H 4655 2977 50  0000 C CNN
 F 2 "" H 4650 3150 50  0001 C CNN
@@
 AR Path="/61E87E93/61EEB97A/61EEB9E5" Ref="R?"  Part="1"
 AR Path="/61E87E93/61EB04DF/61EEB9E5" Ref="R211"  Part="1"
-F 0 "R211" V 5650 2350 50  0000 C CNN
+F 0 "R203" V 5650 2350 50  0000 C CNN
 F 1 "10m" V 5750 2350 50  0000 C CNN
 F 2 "Resistor_SMD:R_1206_3216Metric" V 5680 2350 50  0001 C CNN
@@
 AR Path="/61E87E93/61EEB97A/61EF1EBC" Ref="U?"  Part="1"
 AR Path="/61E87E93/61EB04DF/61EF1EBC" Ref="U53"  Part="1"
-F 0 "U53" H 6594 2896 50  0000 L CNN
+F 0 "U52" H 6594 2896 50  0000 L CNN
 F 1 "LT6106" H 6594 2805 50  0000 L CNN
 F 2 "Package_TO_SOT_SMD:SOT-23-5" H 6250 2850 50  0001 C CNN
@@
 AR Path="/61E87E93/61EEB97A/61EF1EBD" Ref="R?"  Part="1"
 AR Path="/61E87E93/61EB04DF/61EF1EBD" Ref="R213"  Part="1"
-F 0 "R213" H 6600 3000 50  0000 L CNN
+F 0 "R205" H 6600 3000 50  0000 L CNN
 F 1 "2K" V 6550 2950 50  0000 L CNN
 F 2 "Resistor_SMD:R_0805_2012Metric" V 6480 3000 50  0001 C CNN
@@
 AR Path="/61E87E93/61EEB97A/61F7AEC2" Ref="R?"  Part="1"
 AR Path="/61E87E93/61EB04DF/61F7AEC2" Ref="R212"  Part="1"
-F 0 "R212" V 5700 2950 50  0000 C CNN
+F 0 "R204" V 5700 2950 50  0000 C CNN
 F 1 "100R" V 5800 2950 50  0000 C CNN
 F 2 "Resistor_SMD:R_0805_2012Metric" V 5730 2950 50  0001 C CNN
@@
 Connection ~ 6550 2850
 Connection ~ 5600 2350
-Wire Wire Line
-	6000 2350 5900 2350
-Connection ~ 5900 2350
 Text Notes 7000 2750 0    50   ~ 0
 200mV/A
@@
 AR Path="/61E87E93/61EEB97A/61EC6843" Ref="R?"  Part="1"
 AR Path="/61E87E93/61EB04DF/61EC6843" Ref="R209"  Part="1"
-F 0 "R209" H 5150 2550 50  0000 L CNN
+F 0 "R201" H 5150 2550 50  0000 L CNN
 F 1 "200K" V 5100 2550 50  0000 C CNN
 F 2 "Resistor_SMD:R_0805_2012Metric" V 5030 2550 50  0001 C CNN
@@
 AR Path="/61E87E93/61EEB97A/61EEB9EA" Ref="R?"  Part="1"
 AR Path="/61E87E93/61EB04DF/61EEB9EA" Ref="R210"  Part="1"
-F 0 "R210" H 5150 2950 50  0000 L CNN
+F 0 "R202" H 5150 2950 50  0000 L CNN
 F 1 "100K" V 5100 2950 50  0000 C CNN
 F 2 "Resistor_SMD:R_0805_2012Metric" V 5030 2950 50  0001 C CNN
@@
 Connection ~ 4650 3150
 Wire Wire Line
-	4650 2700 4650 3150
-Wire Wire Line
 	4200 2700 4200 3150
 Connection ~ 4200 3150
@@
 Wire Wire Line
 	4650 2350 5100 2350
-Connection ~ 4650 2350
 Wire Wire Line
 	5100 2400 5100 2350
@@
 AR Path="/61E87E93/61EEB97A/61EEA4DE" Ref="#PWR?"  Part="1"
 AR Path="/61E87E93/61EB04DF/61EEA4DE" Ref="#PWR0122"  Part="1"
-F 0 "#PWR0122" H 4650 1550 50  0001 C CNN
+F 0 "#PWR0120" H 4650 1550 50  0001 C CNN
 F 1 "+BATT" H 4665 1873 50  0000 C CNN
 F 2 "" H 4650 1700 50  0001 C CNN
@@
 $EndComp
 Connection ~ 4650 1700
+Wire Wire Line
+	6550 3150 7450 3150
+Connection ~ 6550 3150
+Connection ~ 5900 2350
+Wire Wire Line
+	5900 2350 7450 2350
+Wire Wire Line
+	7450 2650 7450 3150
 $EndSCHEMATC

Commit message: Replace EVERY LT6106 with INA180A3
Friendship ended with LT6106
now ina180 is my best friend
Parts:
- removed R204: 100R, Resistor_SMD:R_0805_2012Metric, symbol Device:R
- removed R205: 2K, Resistor_SMD:R_0805_2012Metric, symbol Device:R
- removed U52: LT6106, Package_TO_SOT_SMD:SOT-23-5, symbol Amplifier_Current:LT6106
- added C88: 0.1uF, Capacitor_SMD:C_0603_1608Metric, symbol Device:C
- added U52: INA180A3, Package_TO_SOT_SMD:SOT-23-5, symbol Amplifier_Current:INA138
- R169: renamed from R203; value 10m -> 4m
- renumbered R198 to R164, R199 to R165, R200 to R166, R201 to R167, R202 to R168
Connections:
- net GND: now also C88.2, U52.2 (GND)
- net TELEM_IOUT: now also U52.1
- net VOUT: now also U52.4 (-)
- net at Q48.1 (S), Q48.2 (S), Q48.3 (S)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: now also U52.3 (+)
- new net VCC: C88.1, U52.5 (V+)
Other:
- note added: "400mV/A"
- note removed: "200mV/A"
- moved on the sheet: R173, R174, R175
