File: ECAD/EPS/PowerConditioning.sch (KiCad schematic (older format))
At the start: 83 parts, among them Q28 SIR167DP, Q29 SIR167DP, Q30 2N7002, Q31 IRF7458, Q32 2N7002, Q33 IRF7458, Q34 2N7002, Q35 2N7002, Q36 2N7002, Q37 IRF7458, Q38 IRF7458, Q39 2N7002, Q40 2N7002, U46 LM358, U47 LM1117-3.3, U48 ADR4530, U49 MAX1626, U50 MAX1626, U51 MAX4373F, U52 MAX4373F, U53 MAX4373F

Commit message: wip: refine shunt resistor selection, add inhibits
Parts:
- added Q7: IRF7458, Package_SO:SOIC-8_3.9x4.9mm_P1.27mm, symbol Transistor_FET:IRF7404
- added R63: 10K, Resistor_SMD:R_0805_2012Metric, symbol Device:R
- added R64: 100R, Resistor_SMD:R_0805_2012Metric, symbol Device:R
- added SW3: INHIBIT 3, Connector_Hirose:Hirose_DF13-02P-1.25DSA_1x02_P1.25mm_Vertical, symbol Switch:SW_SPST
- R81: renamed from R178; footprint Resistor_SMD:R_2010_5025Metric -> Resistor_SMD:R_1206_3216Metric
- R82: renamed from R181; footprint Resistor_SMD:R_2010_5025Metric -> Resistor_SMD:R_1206_3216Metric
- R83: renamed from R182; footprint Resistor_SMD:R_2010_5025Metric -> Resistor_SMD:R_1206_3216Metric
- renumbered C60 to C36, C61 to C37, C63 to C38, C64 to C39, C65 to C40, C66 to C41, C68 to C42, C69 to C43, C62 to C44, C70 to C45, C71 to C46, C72 to C47, C73 to C48, C74 to C49, C75 to C50, C67 to C51, C76 to C52, C77 to C53, C78 to C54, C79 to C55, C80 to C56, C81 to C57, C82 to C58, C83 to C59, C84 to C60, C85 to C61, C86 to C62, D26 to D20, D27 to D21, L6 to L5, L7 to L6, Q28 to Q10, Q29 to Q11, Q32 to Q12, Q33 to Q13, Q35 to Q14, Q36 to Q15, Q34 to Q16, Q37 to Q17, Q38 to Q18, Q39 to Q19, Q40 to Q20, Q30 to Q8, Q31 to Q9, R164 to R65, R165 to R66, R166 to R67, R162 to R68, R163 to R69, R167 to R70, R168 to R71, R169 to R72, R170 to R73, R171 to R74, R172 to R75, R174 to R76, R175 to R77, R173 to R78, R176 to R79, R177 to R80, R179 to R84, R180 to R85, R183 to R86, R184 to R87, R185 to R88, R186 to R89, R187 to R90, R188 to R91, R189 to R92, R190 to R93, R191 to R94, R192 to R95, U46 to U26, U48 to U27, U49 to U28, U50 to U29, U47 to U30, U51 to U31, U52 to U32, U53 to U33
Connections:
- net GND: now also SW3.2 (B)
- net PCM_IN: now also Q7.1 (S), Q7.2 (S), Q7.3 (S), R63.1; no longer C36.1, C37.1, Q9.1 (S), Q9.2 (S), Q9.3 (S), R65.1, U26.8 (V+), U27.2 (IN)
- new net: C36.1, C37.1, Q7.5 (D), Q7.6 (D), Q7.7 (D), Q7.8 (D), Q9.1 (S), Q9.2 (S), Q9.3 (S), R65.1, U26.8 (V+), U27.2 (IN)
- new net: Q7.4 (G), R63.2, R64.1
- new net: R64.2, SW3.1 (A)
Other:
- note added: "UVP and Inhibit"
- note removed: "Undervoltage Protection"
- moved on the sheet: C36, C37, C38, C39, C40, C41, C42, C43, C44, C45, C46, C47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

Commit message: inhibit resistor values, among other things
Parts:
- R63: value 10K -> 100K
Connections:
- net GND: now also R63.2; no longer SW3.2 (B)
- net PCM_IN: now also R64.1; no longer R63.1
- new net: Q7.4 (G), R63.1, SW3.2 (B)
Other:
- moved on the sheet: R63, R64, SW3
Changed lines of the file:
@@
 	0    1    1    0
 $EndComp
-Connection ~ 1450 1100
 $Comp
 L Device:R R?
 U 1 1 61ECA4CA
-P 1450 1250
+P 1050 950
 AR Path="/61BEC565/61ECA4CA" Ref="R?"  Part="1"
 AR Path="/61C9425D/61ECA4CA" Ref="R64"  Part="1"
-F 0 "R64" H 1500 1250 50  0000 L CNN
-F 1 "100R" V 1450 1150 50  0000 L CNN
-F 2 "Resistor_SMD:R_0805_2012Metric" V 1380 1250 50  0001 C CNN
-F 3 "~" H 1450 1250 50  0001 C CNN
-	1    1450 1250
+F 0 "R64" H 1100 950 50  0000 L CNN
+F 1 "100R" V 1050 950 50  0000 C CNN
+F 2 "Resistor_SMD:R_0805_2012Metric" V 980 950 50  0001 C CNN
+F 3 "~" H 1050 950 50  0001 C CNN
+	1    1050 950
 	1    0    0    -1
 $EndComp
 $Comp
-L Switch:SW_SPST SW?
-U 1 1 61ECA4D0
-P 1450 1850
-AR Path="/61BEC565/61ECA4D0" Ref="SW?"  Part="1"
-AR Path="/61C9425D/61ECA4D0" Ref="SW3"  Part="1"
-F 0 "SW3" V 1500 1950 50  0000 L CNN
-F 1 "INHIBIT 3" V 1400 1950 50  0000 L CNN
-F 2 "Connector_Hirose:Hirose_DF13-02P-1.25DSA_1x02_P1.25mm_Vertical" H 1450 1850 50  0001 C CNN
-F 3 "~" H 1450 1850 50  0001 C CNN
-	1    1450 1850
-	0    1    1    0
-$EndComp
-Wire Wire Line
-	1100 1100 1450 1100
-Wire Wire Line
-	1250 800  1100 800
-$Comp
 L Device:R R?
 U 1 1 61ECA4D8
-P 1100 950
+P 1450 1700
 AR Path="/61BEC565/61ECA4D8" Ref="R?"  Part="1"
 AR Path="/61C9425D/61ECA4D8" Ref="R63"  Part="1"
-F 0 "R63" H 1150 950 50  0000 L CNN
-F 1 "10K" V 1100 950 50  0000 C CNN
-F 2 "Resistor_SMD:R_0805_2012Metric" V 1030 950 50  0001 C CNN
-F 3 "~" H 1100 950 50  0001 C CNN
-	1    1100 950
+F 0 "R63" H 1500 1700 50  0000 L CNN
+F 1 "100K" V 1450 1700 50  0000 C CNN
+F 2 "Resistor_SMD:R_0805_2012Metric" V 1380 1700 50  0001 C CNN
+F 3 "~" H 1450 1700 50  0001 C CNN
+	1    1450 1700
 	1    0    0    -1
 $EndComp
@@
 $EndComp
 Wire Wire Line
-	900  800  1100 800
-Connection ~ 1100 800
-Wire Wire Line
-	1450 1400 1450 1650
-Wire Wire Line
 	1650 800  2800 800
 Connection ~ 2800 800
-Wire Wire Line
-	1450 2050 1450 2400
 Wire Wire Line
 	1450 2400 1900 2400
@@
 Wire Notes Line
 	500  500  5500 500
+$Comp
+L Switch:SW_SPST SW?
+U 1 1 61ECA4D0
+P 1250 1250
+AR Path="/61BEC565/61ECA4D0" Ref="SW?"  Part="1"
+AR Path="/61C9425D/61ECA4D0" Ref="SW3"  Part="1"
+F 0 "SW3" H 1250 1150 50  0000 C CNN
+F 1 "INHIBIT 3" H 1250 1050 50  0000 C CNN
+F 2 "Connector_Hirose:Hirose_DF13-02P-1.25DSA_1x02_P1.25mm_Vertical" H 1250 1250 50  0001 C CNN
+F 3 "~" H 1250 1250 50  0001 C CNN
+	1    1250 1250
+	1    0    0    -1
+$EndComp
+Wire Wire Line
+	900  800  1050 800
+Connection ~ 1050 800
+Wire Wire Line
+	1050 800  1250 800
+Wire Wire Line
+	1450 1550 1450 1250
+Connection ~ 1450 1250
+Wire Wire Line
+	1450 1250 1450 1100
+Wire Wire Line
+	1050 1100 1050 1250
+Wire Wire Line
+	1450 1850 1450 2400
 $EndSCHEMATC

Commit message: Replace EVERY LT6106 with INA180A3
Friendship ended with LT6106
now ina180 is my best friend
Parts:
- renumbered C36 to C43, C37 to C44, C38 to C45, C39 to C46, C40 to C47, C41 to C48, C42 to C49, C43 to C50, C44 to C51, C45 to C52, C46 to C53, C47 to C54, C48 to C55, C49 to C56, C50 to C57, C51 to C58, C52 to C59, C53 to C60, C54 to C61, C55 to C62, C56 to C63, C57 to C64, C58 to C65, C59 to C66, C60 to C67, C61 to C68, C62 to C69, R64 to R49, R63 to R50, R65 to R51, R66 to R52, R67 to R53, R68 to R54, R69 to R55, R70 to R56, R71 to R57, R72 to R58, R73 to R59, R74 to R60, R75 to R61, R76 to R62, R77 to R63, R78 to R64, R79 to R65, R80 to R66, R81 to R67, R82 to R68, R83 to R69, R84 to R70, R85 to R71, R86 to R72, R87 to R73, R88 to R74, R89 to R75, R90 to R76, R91 to R77, R92 to R78, R93 to R79, R94 to R80, R95 to R81
