File: ECAD/EPS/Pulse+RetryTimer.sch (KiCad schematic (older format))
At the start: 13 parts, among them Q41 2N7002, Q42 2N7002, U54 AD8603, U57 LTC6993xS6-4

Commit message: wip: refine shunt resistor selection, add inhibits
Parts:
- renumbered C87 to C63, C90 to C66, Q41 to Q21, Q42 to Q22, R203 to R106, R204 to R107, R205 to R108, R206 to R109, R193 to R96, R194 to R97, R195 to R98, U54 to U34, U57 to U37

Commit message: Replace EVERY LT6106 with INA180A3
Friendship ended with LT6106
now ina180 is my best friend
Parts:
- renumbered C63 to C70, C66 to C73, R96 to R82, R97 to R83, R98 to R84, R106 to R92, R107 to R93, R108 to R94, R109 to R95
Changed lines of the file:
@@
 AR Path="/61C9425D/61DD9B5B/61DD6209" Ref="#PWR?"  Part="1"
 AR Path="/61C9425D/62429382/61DD6209" Ref="#PWR?"  Part="1"
-AR Path="/61C9425D/62734C35/61DD6209" Ref="#PWR086"  Part="1"
-AR Path="/61C9425D/6278B84C/61DD6209" Ref="#PWR090"  Part="1"
-AR Path="/61C9425D/6286FCFD/61DD6209" Ref="#PWR094"  Part="1"
-F 0 "#PWR094" H 2950 1000 50  0001 C CNN
+AR Path="/61C9425D/62734C35/61DD6209" Ref="#PWR0100"  Part="1"
+AR Path="/61C9425D/6278B84C/61DD6209" Ref="#PWR0104"  Part="1"
+AR Path="/61C9425D/6286FCFD/61DD6209" Ref="#PWR0108"  Part="1"
+F 0 "#PWR0108" H 2950 1000 50  0001 C CNN
 F 1 "VCC" H 2965 1323 50  0000 C CNN
 F 2 "" H 2950 1150 50  0001 C CNN
@@
 AR Path="/61C9425D/61DD9B5B/61DE485D" Ref="R?"  Part="1"
 AR Path="/61C9425D/62429382/61DE485D" Ref="R?"  Part="1"
-AR Path="/61C9425D/62734C35/61DE485D" Ref="R96"  Part="1"
-AR Path="/61C9425D/6278B84C/61DE485D" Ref="R103"  Part="1"
-AR Path="/61C9425D/6286FCFD/61DE485D" Ref="R110"  Part="1"
-F 0 "R110" H 2150 1300 50  0000 L CNN
+AR Path="/61C9425D/62734C35/61DE485D" Ref="R82"  Part="1"
+AR Path="/61C9425D/6278B84C/61DE485D" Ref="R89"  Part="1"
+AR Path="/61C9425D/6286FCFD/61DE485D" Ref="R96"  Part="1"
+F 0 "R96" H 2150 1300 50  0000 L CNN
 F 1 "2.5M" V 2100 1300 50  0000 C CNN
 F 2 "Resistor_SMD:R_0805_2012Metric" V 2030 1300 50  0001 C CNN
@@
 AR Path="/61C9425D/61DD9B5B/61DEA269" Ref="C?"  Part="1"
 AR Path="/61C9425D/62429382/61DEA269" Ref="C?"  Part="1"
-AR Path="/61C9425D/62734C35/61DEA269" Ref="C63"  Part="1"
-AR Path="/61C9425D/6278B84C/61DEA269" Ref="C65"  Part="1"
-AR Path="/61C9425D/6286FCFD/61DEA269" Ref="C67"  Part="1"
-F 0 "C67" H 2215 1746 50  0000 L CNN
+AR Path="/61C9425D/62734C35/61DEA269" Ref="C70"  Part="1"
+AR Path="/61C9425D/6278B84C/61DEA269" Ref="C72"  Part="1"
+AR Path="/61C9425D/6286FCFD/61DEA269" Ref="C74"  Part="1"
+F 0 "C74" H 2215 1746 50  0000 L CNN
 F 1 "22uF" H 2215 1655 50  0000 L CNN
 F 2 "Capacitor_SMD:C_0805_2012Metric" H 2138 1550 50  0001 C CNN
@@
 AR Path="/61C9425D/61DD9B5B/61E036B5" Ref="#PWR?"  Part="1"
 AR Path="/61C9425D/62429382/61E036B5" Ref="#PWR?"  Part="1"
-AR Path="/61C9425D/62734C35/61E036B5" Ref="#PWR087"  Part="1"
-AR Path="/61C9425D/6278B84C/61E036B5" Ref="#PWR091"  Part="1"
-AR Path="/61C9425D/6286FCFD/61E036B5" Ref="#PWR095"  Part="1"
-F 0 "#PWR095" H 2950 1800 50  0001 C CNN
+AR Path="/61C9425D/62734C35/61E036B5" Ref="#PWR0101"  Part="1"
+AR Path="/61C9425D/6278B84C/61E036B5" Ref="#PWR0105"  Part="1"
+AR Path="/61C9425D/6286FCFD/61E036B5" Ref="#PWR0109"  Part="1"
+F 0 "#PWR0109" H 2950 1800 50  0001 C CNN
 F 1 "GND" H 2955 1877 50  0000 C CNN
 F 2 "" H 2950 2050 50  0001 C CNN
@@
 AR Path="/61C9425D/61DD9B5B/61D792CF" Ref="R?"  Part="1"
 AR Path="/61C9425D/62429382/61D792CF" Ref="R?"  Part="1"
-AR Path="/61C9425D/62734C35/61D792CF" Ref="R97"  Part="1"
-AR Path="/61C9425D/6278B84C/61D792CF" Ref="R104"  Part="1"
-AR Path="/61C9425D/6286FCFD/61D792CF" Ref="R111"  Part="1"
-F 0 "R111" H 2500 1300 50  0000 L CNN
+AR Path="/61C9425D/62734C35/61D792CF" Ref="R83"  Part="1"
+AR Path="/61C9425D/6278B84C/61D792CF" Ref="R90"  Part="1"
+AR Path="/61C9425D/6286FCFD/61D792CF" Ref="R97"  Part="1"
+F 0 "R97" H 2500 1300 50  0000 L CNN
 F 1 "10K" V 2450 1300 50  0000 C CNN
 F 2 "Resistor_SMD:R_0805_2012Metric" V 2380 1300 50  0001 C CNN
@@
 AR Path="/61C9425D/61DD9B5B/61D79DBB" Ref="R?"  Part="1"
 AR Path="/61C9425D/62429382/61D79DBB" Ref="R?"  Part="1"
-AR Path="/61C9425D/62734C35/61D79DBB" Ref="R98"  Part="1"
-AR Path="/61C9425D/6278B84C/61D79DBB" Ref="R105"  Part="1"
-AR Path="/61C9425D/6286FCFD/61D79DBB" Ref="R112"  Part="1"
-F 0 "R112" H 2500 1900 50  0000 L CNN
+AR Path="/61C9425D/62734C35/61D79DBB" Ref="R84"  Part="1"
+AR Path="/61C9425D/6278B84C/61D79DBB" Ref="R91"  Part="1"
+AR Path="/61C9425D/6286FCFD/61D79DBB" Ref="R98"  Part="1"
+F 0 "R98" H 2500 1900 50  0000 L CNN
 F 1 "20K" V 2450 1900 50  0000 C CNN
 F 2 "Resistor_SMD:R_0805_2012Metric" V 2380 1900 50  0001 C CNN
@@
 P 6350 1300
 AR Path="/61C9425D/628E3A1F" Ref="#PWR?"  Part="1"
-AR Path="/61C9425D/6278B84C/628E3A1F" Ref="#PWR092"  Part="1"
+AR Path="/61C9425D/6278B84C/628E3A1F" Ref="#PWR0106"  Part="1"
 AR Path="/61C9425D/61DD1DB6/628E3A1F" Ref="#PWR?"  Part="1"
-AR Path="/61C9425D/62734C35/628E3A1F" Ref="#PWR088"  Part="1"
-AR Path="/61C9425D/6286FCFD/628E3A1F" Ref="#PWR096"  Part="1"
-F 0 "#PWR096" H 6350 1150 50  0001 C CNN
+AR Path="/61C9425D/62734C35/628E3A1F" Ref="#PWR0102"  Part="1"
+AR Path="/61C9425D/6286FCFD/628E3A1F" Ref="#PWR0110"  Part="1"
+F 0 "#PWR0110" H 6350 1150 50  0001 C CNN
 F 1 "VCC" H 6365 1473 50  0000 C CNN
 F 2 "" H 6350 1300 50  0001 C CNN
@@
 P 5650 1900
 AR Path="/61C9425D/628E3A25" Ref="R?"  Part="1"
-AR Path="/61C9425D/6278B84C/628E3A25" Ref="R107"  Part="1"
+AR Path="/61C9425D/6278B84C/628E3A25" Ref="R93"  Part="1"
 AR Path="/61C9425D/61DD1DB6/628E3A25" Ref="R?"  Part="1"
-AR Path="/61C9425D/62734C35/628E3A25" Ref="R100"  Part="1"
-AR Path="/61C9425D/6286FCFD/628E3A25" Ref="R114"  Part="1"
-F 0 "R114" H 5700 1900 50  0000 L CNN
+AR Path="/61C9425D/62734C35/628E3A25" Ref="R86"  Part="1"
+AR Path="/61C9425D/6286FCFD/628E3A25" Ref="R100"  Part="1"
+F 0 "R100" H 5700 1900 50  0000 L CNN
 F 1 "1K" V 5650 1900 50  0000 C CNN
 F 2 "Resistor_SMD:R_0805_2012Metric" V 5580 1900 50  0001 C CNN
@@
 P 5650 1450
 AR Path="/61C9425D/628E3A2B" Ref="R?"  Part="1"
-AR Path="/61C9425D/6278B84C/628E3A2B" Ref="R106"  Part="1"
+AR Path="/61C9425D/6278B84C/628E3A2B" Ref="R92"  Part="1"
 AR Path="/61C9425D/61DD1DB6/628E3A2B" Ref="R?"  Part="1"
-AR Path="/61C9425D/62734C35/628E3A2B" Ref="R99"  Part="1"
-AR Path="/61C9425D/6286FCFD/628E3A2B" Ref="R113"  Part="1"
-F 0 "R113" H 5700 1450 50  0000 L CNN
+AR Path="/61C9425D/62734C35/628E3A2B" Ref="R85"  Part="1"
+AR Path="/61C9425D/6286FCFD/628E3A2B" Ref="R99"  Part="1"
+F 0 "R99" H 5700 1450 50  0000 L CNN
 F 1 "523R" V 5650 1450 50  0000 C CNN
 F 2 "Resistor_SMD:R_0805_2012Metric" V 5580 1450 50  0001 C CNN
@@
 P 5950 1950
 AR Path="/61C9425D/628E3A39" Ref="R?"  Part="1"
-AR Path="/61C9425D/6278B84C/628E3A39" Ref="R109"  Part="1"
+AR Path="/61C9425D/6278B84C/628E3A39" Ref="R95"  Part="1"
 AR Path="/61C9425D/61DD1DB6/628E3A39" Ref="R?"  Part="1"
-AR Path="/61C9425D/62734C35/628E3A39" Ref="R102"  Part="1"
-AR Path="/61C9425D/6286FCFD/628E3A39" Ref="R116"  Part="1"
-F 0 "R116" H 6000 1950 50  0000 L CNN
+AR Path="/61C9425D/62734C35/628E3A39" Ref="R88"  Part="1"
+AR Path="/61C9425D/6286FCFD/628E3A39" Ref="R102"  Part="1"
+F 0 "R102" H 6000 1950 50  0000 L CNN
 F 1 "760K" V 5950 1950 50  0000 C CNN
 F 2 "Resistor_SMD:R_0805_2012Metric" V 5880 1950 50  0001 C CNN
@@
 P 5200 1450
 AR Path="/61C9425D/628E3A41" Ref="C?"  Part="1"
-AR Path="/61C9425D/6278B84C/628E3A41" Ref="C66"  Part="1"
+AR Path="/61C9425D/6278B84C/628E3A41" Ref="C73"  Part="1"
 AR Path="/61C9425D/61DD1DB6/628E3A41" Ref="C?"  Part="1"
-AR Path="/61C9425D/62734C35/628E3A41" Ref="C64"  Part="1"
-AR Path="/61C9425D/6286FCFD/628E3A41" Ref="C68"  Part="1"
-F 0 "C68" H 5315 1496 50  0000 L CNN
+AR Path="/61C9425D/62734C35/628E3A41" Ref="C71"  Part="1"
+AR Path="/61C9425D/6286FCFD/628E3A41" Ref="C75"  Part="1"
+F 0 "C75" H 5315 1496 50  0000 L CNN
 F 1 "0.1uF" H 5315 1405 50  0000 L CNN
 F 2 "Capacitor_SMD:C_0805_2012Metric" H 5238 1300 50  0001 C CNN
@@
 P 5850 1500
 AR Path="/61C9425D/628E3A4F" Ref="R?"  Part="1"
-AR Path="/61C9425D/6278B84C/628E3A4F" Ref="R108"  Part="1"
+AR Path="/61C9425D/6278B84C/628E3A4F" Ref="R94"  Part="1"
 AR Path="/61C9425D/61DD1DB6/628E3A4F" Ref="R?"  Part="1"
-AR Path="/61C9425D/62734C35/628E3A4F" Ref="R101"  Part="1"
-AR Path="/61C9425D/6286FCFD/628E3A4F" Ref="R115"  Part="1"
-F 0 "R115" H 5900 1500 50  0000 L CNN
+AR Path="/61C9425D/62734C35/628E3A4F" Ref="R87"  Part="1"
+AR Path="/61C9425D/6286FCFD/628E3A4F" Ref="R101"  Part="1"
+F 0 "R101" H 5900 1500 50  0000 L CNN
 F 1 "10K" V 5850 1500 50  0000 C CNN
 F 2 "Resistor_SMD:R_0805_2012Metric" V 5780 1500 50  0001 C CNN
@@
 AR Path="/61C9425D/61DD9B5B/628E8E71" Ref="#PWR?"  Part="1"
 AR Path="/61C9425D/62429382/628E8E71" Ref="#PWR?"  Part="1"
-AR Path="/61C9425D/62734C35/628E8E71" Ref="#PWR089"  Part="1"
-AR Path="/61C9425D/6278B84C/628E8E71" Ref="#PWR093"  Part="1"
-AR Path="/61C9425D/6286FCFD/628E8E71" Ref="#PWR097"  Part="1"
-F 0 "#PWR097" H 6350 1850 50  0001 C CNN
+AR Path="/61C9425D/62734C35/628E8E71" Ref="#PWR0103"  Part="1"
+AR Path="/61C9425D/6278B84C/628E8E71" Ref="#PWR0107"  Part="1"
+AR Path="/61C9425D/6286FCFD/628E8E71" Ref="#PWR0111"  Part="1"
+F 0 "#PWR0111" H 6350 1850 50  0001 C CNN
 F 1 "GND" H 6355 1927 50  0000 C CNN
 F 2 "" H 6350 2100 50  0001 C CNN
