File: ECAD/EPS/SolarConditioning.sch (KiCad schematic (older format))
At the start: 52 parts, among them J10 S3B, J11 S4A, J12 S4B, J13 TELEM_IN, J5 S1A, J6 S1B, J7 S2A, J8 S2B, J9 S3A, Q25 IRF7425, Q26 IRF7458, SW3 INHIBIT 1, U12 LTC4412xS6, U13 MCP3208, U14 LT6106, U15 ATtiny84A-SSU, U16 L78L33_SO8, U17 MCP4812, U18 MCP4812

Commit message: Split up into 3 projects for separate boards
Changed lines of the file:
@@
 $Descr USLetter 11000 8500
 encoding utf-8
-Sheet 7 37
+Sheet 2 32
 Title "TJ Custom EPS"
 Date ""
@@
 Wire Wire Line
 	2150 5750 2150 6400
-$Sheet
-S 9400 1200 1000 500
-U 636144E9
-F0 "SolarTelem" 50
-F1 "SolarTelem.sch" 50
-$EndSheet
 $Comp
 L Mechanical:MountingHole_Pad H?

Commit message: Further descope: remove SA4
Parts:
- removed D13, D14: 1N4004, Diode_SMD:D_SMA, symbol Device:D
- removed D5, D6: CMSH3-40MA, Diode_SMD:D_SMA, symbol Device:D_Schottky
- removed J10: S3B, Connector_Hirose:Hirose_DF13-04P-1.25DSA_1x04_P1.25mm_Vertical, symbol Connector:Conn_01x04_Female
- removed J9: S3A, Connector_Hirose:Hirose_DF13-04P-1.25DSA_1x04_P1.25mm_Vertical, symbol Connector:Conn_01x04_Female
- J11: value S4A -> S3A
- J12: value S4B -> S3B
- renumbered D15 to D13, D16 to D14, D7 to D5, D8 to D6
Connections:
- net I_SA4A: no longer names the net of U13.7 (CH6)
- net I_SA4B: no longer names the net of U13.8 (CH7)
- net V_SA4: no longer names the net of U15.10 (PA3)
- net Vset4: no longer names the net of U18.6 (VB)
Other:
- moved on the sheet: D13, D14, D5, D6, J11, J12, Q25, U12

Commit message: wip: refine shunt resistor selection, add inhibits
Parts:
- added Q5: IRF7458, Package_SO:SOIC-8_3.9x4.9mm_P1.27mm, symbol Transistor_FET:IRF7404
- added R12: 10K, Resistor_SMD:R_0805_2012Metric, symbol Device:R
- added R13: 100R, Resistor_SMD:R_0805_2012Metric, symbol Device:R
- added SW2: INHIBIT 2, Connector_Hirose:Hirose_DF13-02P-1.25DSA_1x02_P1.25mm_Vertical, symbol Switch:SW_SPST
- R16: renamed from R69; footprint Resistor_SMD:R_2010_5025Metric -> Resistor_SMD:R_1206_3216Metric
- renumbered C35 to C16, C36 to C17, C37 to C18, C38 to C19, C39 to C20, C40 to C21, D12 to D10, D13 to D11, D14 to D12, D9 to D7, D10 to D8, D11 to D9, H5 to H3, H6 to H4, H7 to H5, H8 to H6, J5 to J3, J6 to J4, J7 to J5, J8 to J6, J11 to J7, J12 to J8, J13 to J9, Q25 to Q3, Q26 to Q4, R65 to R10, R66 to R11, R67 to R14, R68 to R15, R70 to R17, R71 to R18, SW3 to SW1, U16 to U10, U17 to U11, U18 to U12, U12 to U6, U13 to U7, U15 to U8, U14 to U9
Connections:
- net GND: now also SW2.2 (B)
- net at Q4.5 (D), Q4.6 (D), Q4.7 (D)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: now also Q5.1 (S), Q5.2 (S), Q5.3 (S), R12.1; no longer R14.1, R16.2, R17.2
- new net: Q5.5 (D), Q5.6 (D), Q5.7 (D), Q5.8 (D), R14.1, R16.2, R17.2
- new net: Q5.4 (G), R12.2, R13.1
- new net: R13.2, SW2.1 (A)
Other:
- moved on the sheet: J9, R14, R15, R16, R17, R18, SW1, U9

Commit message: inhibit resistor values, among other things
Parts:
- Q3: value IRF7425 -> IRF7458
- R10, R12: value 10K -> 100K
Connections:
- net GND: now also R10.2, R12.2; no longer SW1.2 (B), SW2.2 (B)
- net MPPT1/VOUT: now also R11.1; no longer R10.1
- net at Q4.5 (D), Q4.6 (D), Q4.7 (D)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: now also R13.1; no longer R12.1
- new net: Q4.4 (G), R10.1, SW1.2 (B)
- new net: Q5.4 (G), R12.1, SW2.2 (B)
Other:
- moved on the sheet: R10, R11, R12, R13, SW1, SW2
Changed lines of the file:
@@
 	-1   0    0    1
 $EndComp
-Connection ~ 4300 1750
 $Comp
 L Device:R R11
 U 1 1 61C70AB7
-P 4300 1900
-F 0 "R11" H 4350 1900 50  0000 L CNN
-F 1 "100R" V 4300 1800 50  0000 L CNN
-F 2 "Resistor_SMD:R_0805_2012Metric" V 4230 1900 50  0001 C CNN
-F 3 "~" H 4300 1900 50  0001 C CNN
-	1    4300 1900
-	1    0    0    -1
-$EndComp
-Wire Wire Line
-	3950 1750 4300 1750
-Wire Wire Line
-	4100 1450 3950 1450
+P 3900 1600
+F 0 "R11" H 3950 1600 50  0000 L CNN
+F 1 "100R" V 3900 1600 50  0000 C CNN
+F 2 "Resistor_SMD:R_0805_2012Metric" V 3830 1600 50  0001 C CNN
+F 3 "~" H 3900 1600 50  0001 C CNN
+	1    3900 1600
+	1    0    0    -1
+$EndComp
 $Comp
 L Device:R R10
 U 1 1 61C55D97
-P 3950 1600
-F 0 "R10" H 4000 1600 50  0000 L CNN
-F 1 "10K" V 3950 1600 50  0000 C CNN
-F 2 "Resistor_SMD:R_0805_2012Metric" V 3880 1600 50  0001 C CNN
-F 3 "~" H 3950 1600 50  0001 C CNN
-	1    3950 1600
-	1    0    0    -1
-$EndComp
-$Comp
-L Transistor_FET:IRF7404 Q4
-U 1 1 61C4B7C5
-P 4300 1550
-F 0 "Q4" V 4642 1550 50  0000 C CNN
-F 1 "IRF7458" V 4551 1550 50  0000 C CNN
-F 2 "Package_SO:SOIC-8_3.9x4.9mm_P1.27mm" H 4500 1475 50  0001 L CIN
-F 3 "http://www.infineon.com/dgdl/irf7404.pdf?fileId=5546d462533600a4015355fa2b5b1b9e" V 4300 1550 50  0001 L CNN
-	1    4300 1550
-	0    1    -1   0
+P 4300 2300
+F 0 "R10" H 4350 2300 50  0000 L CNN
+F 1 "100K" V 4300 2300 50  0000 C CNN
+F 2 "Resistor_SMD:R_0805_2012Metric" V 4230 2300 50  0001 C CNN
+F 3 "~" H 4300 2300 50  0001 C CNN
+	1    4300 2300
+	1    0    0    -1
 $EndComp
 $Comp
@@
 Wire Wire Line
 	3400 4350 3750 4350
-Wire Wire Line
-	3750 1450 3950 1450
 Connection ~ 3750 1450
-Connection ~ 3950 1450
 Wire Wire Line
 	1750 1000 1750 1050
@@
 P 1650 5050
 F 0 "Q3" V 2000 5050 50  0000 C CNN
-F 1 "IRF7425" V 1900 5050 50  0000 C CNN
+F 1 "IRF7458" V 1900 5050 50  0000 C CNN
 F 2 "Package_SO:SOIC-8_3.9x4.9mm_P1.27mm" H 1850 4975 50  0001 L CIN
 F 3 "http://www.infineon.com/dgdl/irf7404.pdf?fileId=5546d462533600a4015355fa2b5b1b9e" V 1650 5050 50  0001 L CNN
@@
 L Switch:SW_SPST SW1
 U 1 1 61C66266
-P 4300 2250
-F 0 "SW1" V 4350 2350 50  0000 L CNN
-F 1 "INHIBIT 1" V 4250 2350 50  0000 L CNN
-F 2 "Connector_Hirose:Hirose_DF13-02P-1.25DSA_1x02_P1.25mm_Vertical" H 4300 2250 50  0001 C CNN
-F 3 "~" H 4300 2250 50  0001 C CNN
-	1    4300 2250
-	0    1    1    0
-$EndComp
-Connection ~ 5050 1750
+P 4100 1900
+F 0 "SW1" H 4100 1800 50  0000 C CNN
+F 1 "INHIBIT 1" H 4100 1700 50  0000 C CNN
+F 2 "Connector_Hirose:Hirose_DF13-02P-1.25DSA_1x02_P1.25mm_Vertical" H 4100 1900 50  0001 C CNN
+F 3 "~" H 4100 1900 50  0001 C CNN
+	1    4100 1900
+	1    0    0    -1
+$EndComp
 $Comp
 L Device:R R13
 U 1 1 621825FF
-P 5050 1900
-F 0 "R13" H 5100 1900 50  0000 L CNN
-F 1 "100R" V 5050 1800 50  0000 L CNN
-F 2 "Resistor_SMD:R_0805_2012Metric" V 4980 1900 50  0001 C CNN
-F 3 "~" H 5050 1900 50  0001 C CNN
-	1    5050 1900
-	1    0    0    -1
-$EndComp
-Wire Wire Line
-	4700 1750 5050 1750
-Wire Wire Line
-	4850 1450 4700 1450
+P 4650 1600
+F 0 "R13" H 4700 1600 50  0000 L CNN
+F 1 "100R" V 4650 1600 50  0000 C CNN
+F 2 "Resistor_SMD:R_0805_2012Metric" V 4580 1600 50  0001 C CNN
+F 3 "~" H 4650 1600 50  0001 C CNN
+	1    4650 1600
+	1    0    0    -1
+$EndComp
 $Comp
 L Device:R R12
 U 1 1 62182607
-P 4700 1600
-F 0 "R12" H 4750 1600 50  0000 L CNN
-F 1 "10K" V 4700 1600 50  0000 C CNN
-F 2 "Resistor_SMD:R_0805_2012Metric" V 4630 1600 50  0001 C CNN
-F 3 "~" H 4700 1600 50  0001 C CNN
-	1    4700 1600
+P 5050 2300
+F 0 "R12" H 5100 2300 50  0000 L CNN
+F 1 "100K" V 5050 2300 50  0000 C CNN
+F 2 "Resistor_SMD:R_0805_2012Metric" V 4980 2300 50  0001 C CNN
+F 3 "~" H 5050 2300 50  0001 C CNN
+	1    5050 2300
 	1    0    0    -1
 $EndComp
@@
 	0    1    -1   0
 $EndComp
-Wire Wire Line
-	4500 1450 4700 1450
-Connection ~ 4700 1450
 $Comp
 L Switch:SW_SPST SW2
 U 1 1 621E79D7
-P 5050 2250
-F 0 "SW2" V 5100 2350 50  0000 L CNN
-F 1 "INHIBIT 2" V 5000 2350 50  0000 L CNN
-F 2 "Connector_Hirose:Hirose_DF13-02P-1.25DSA_1x02_P1.25mm_Vertical" H 5050 2250 50  0001 C CNN
-F 3 "~" H 5050 2250 50  0001 C CNN
-	1    5050 2250
-	0    1    1    0
+P 4850 1900
+F 0 "SW2" H 4850 1800 50  0000 C CNN
+F 1 "INHIBIT 2" H 4850 1700 50  0000 C CNN
+F 2 "Connector_Hirose:Hirose_DF13-02P-1.25DSA_1x02_P1.25mm_Vertical" H 4850 1900 50  0001 C CNN
+F 3 "~" H 4850 1900 50  0001 C CNN
+	1    4850 1900
+	1    0    0    -1
 $EndComp
 Wire Wire Line
 	4300 2450 4700 2450
 Connection ~ 4700 2450
-Wire Wire Line
-	4700 2450 5050 2450
 Connection ~ 7250 2250
 $Comp
@@
 TELEM_VBCROUT
 Wire Wire Line
+	5850 2450 5850 2150
+Wire Wire Line
+	3750 1450 3900 1450
+Wire Wire Line
+	4700 2450 5050 2450
+Connection ~ 5050 2450
+Wire Wire Line
 	5050 2450 5850 2450
 Wire Wire Line
-	5850 2450 5850 2150
-Connection ~ 5050 2450
+	4500 1450 4650 1450
+$Comp
+L Transistor_FET:IRF7404 Q4
+U 1 1 61C4B7C5
+P 4300 1550
+F 0 "Q4" V 4642 1550 50  0000 C CNN
+F 1 "IRF7458" V 4551 1550 50  0000 C CNN
+F 2 "Package_SO:SOIC-8_3.9x4.9mm_P1.27mm" H 4500 1475 50  0001 L CIN
+F 3 "http://www.infineon.com/dgdl/irf7404.pdf?fileId=5546d462533600a4015355fa2b5b1b9e" V 4300 1550 50  0001 L CNN
+	1    4300 1550
+	0    1    -1   0
+$EndComp
+Connection ~ 4650 1450
+Wire Wire Line
+	4650 1450 4850 1450
+Wire Wire Line
+	5050 1750 5050 1900
+Connection ~ 5050 1900
+Wire Wire Line
+	5050 1900 5050 2150
+Wire Wire Line
+	4650 1750 4650 1900
+Connection ~ 3900 1450
+Wire Wire Line
+	3900 1450 4100 1450
+Wire Wire Line
+	4300 2150 4300 1900
+Connection ~ 4300 1900
+Wire Wire Line
+	4300 1900 4300 1750
+Wire Wire Line
+	3900 1750 3900 1900
 $EndSCHEMATC

Commit message: work
Parts:
- D10, D11, D12, D7, D8, D9: value 1N4004 -> RR264MM; footprint Diode_SMD:D_SMA -> Diode_SMD:D_SOD-123F
Changed lines of the file:
@@
 P 1750 2700
 F 0 "D10" V 1800 2750 50  0000 L CNN
-F 1 "1N4004" V 1700 2750 50  0000 L CNN
-F 2 "Diode_SMD:D_SMA" H 1750 2700 50  0001 C CNN
+F 1 "RR264MM" V 1700 2750 50  0000 L CNN
+F 2 "Diode_SMD:D_SOD-123F" H 1750 2700 50  0001 C CNN
 F 3 "~" H 1750 2700 50  0001 C CNN
 	1    1750 2700
@@
 P 1750 2300
 F 0 "D9" V 1800 2250 50  0000 R CNN
-F 1 "1N4004" V 1700 2250 50  0000 R CNN
-F 2 "Diode_SMD:D_SMA" H 1750 2300 50  0001 C CNN
+F 1 "RR264MM" V 1700 2250 50  0000 R CNN
+F 2 "Diode_SMD:D_SOD-123F" H 1750 2300 50  0001 C CNN
 F 3 "~" H 1750 2300 50  0001 C CNN
 	1    1750 2300
@@
 P 1750 1250
 F 0 "D8" V 1800 1300 50  0000 L CNN
-F 1 "1N4004" V 1700 1300 50  0000 L CNN
-F 2 "Diode_SMD:D_SMA" H 1750 1250 50  0001 C CNN
+F 1 "RR264MM" V 1700 1300 50  0000 L CNN
+F 2 "Diode_SMD:D_SOD-123F" H 1750 1250 50  0001 C CNN
 F 3 "~" H 1750 1250 50  0001 C CNN
 	1    1750 1250
@@
 P 1750 850
 F 0 "D7" V 1800 800 50  0000 R CNN
-F 1 "1N4004" V 1700 800 50  0000 R CNN
-F 2 "Diode_SMD:D_SMA" H 1750 850 50  0001 C CNN
+F 1 "RR264MM" V 1700 800 50  0000 R CNN
+F 2 "Diode_SMD:D_SOD-123F" H 1750 850 50  0001 C CNN
 F 3 "~" H 1750 850 50  0001 C CNN
 	1    1750 850
@@
 P 1750 4150
 F 0 "D12" V 1800 4200 50  0000 L CNN
-F 1 "1N4004" V 1700 4200 50  0000 L CNN
-F 2 "Diode_SMD:D_SMA" H 1750 4150 50  0001 C CNN
+F 1 "RR264MM" V 1700 4200 50  0000 L CNN
+F 2 "Diode_SMD:D_SOD-123F" H 1750 4150 50  0001 C CNN
 F 3 "~" H 1750 4150 50  0001 C CNN
 	1    1750 4150
@@
 P 1750 3750
 F 0 "D11" V 1800 3700 50  0000 R CNN
-F 1 "1N4004" V 1700 3700 50  0000 R CNN
-F 2 "Diode_SMD:D_SMA" H 1750 3750 50  0001 C CNN
+F 1 "RR264MM" V 1700 3700 50  0000 R CNN
+F 2 "Diode_SMD:D_SOD-123F" H 1750 3750 50  0001 C CNN
 F 3 "~" H 1750 3750 50  0001 C CNN
 	1    1750 3750

Commit message: Replace EVERY LT6106 with INA180A3
Friendship ended with LT6106
now ina180 is my best friend
Parts:
- removed R17: 100R, Resistor_SMD:R_0805_2012Metric, symbol Device:R
- removed R18: 2K, Resistor_SMD:R_0805_2012Metric, symbol Device:R
- removed U9: LT6106, Package_TO_SOT_SMD:SOT-23-5, symbol Amplifier_Current:LT6106
- added C19: 0.1uF, Capacitor_SMD:C_0603_1608Metric, symbol Device:C
- added U9: INA180A3, Package_TO_SOT_SMD:SOT-23-5, symbol Amplifier_Current:INA138
- R16: value 10m -> 4m
- renumbered C19 to C20, C20 to C21, C21 to C22, J3 to J2, J4 to J3, J5 to J4, J6 to J5, J7 to J6, J8 to J7, J9 to J8, R11 to R10, R10 to R11, R13 to R12, R12 to R13
Connections:
- net +3.3VA: now also C19.1, U9.5 (V+)
- net BCR_OUT: now also U9.4 (-)
- net GND: now also C19.2, U9.2 (GND)
- net TELEM_IBCROUT: now also U9.1
- net at Q5.5 (D), Q5.6 (D), Q5.7 (D)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: now also U9.3 (+)
Other:
- note added: "400mV/A"
- note removed: "200mV/A"
