File: ECAD/EPS/PowerDistribution.sch (KiCad schematic (older format))
At the start: 5 parts, among them U62 74HC595, U63 74HC595

Commit message: wip: refine shunt resistor selection, add inhibits
Parts:
- renumbered C97 to C69, C98 to C70, R310 to R117, U62 to U40, U63 to U41
Changed lines of the file:
@@
 3.3V PDMs
 $Comp
-L 74xx:74HC595 U62
+L 74xx:74HC595 U40
 U 1 1 622C9B64
 P 4650 4700
-F 0 "U62" H 4650 5481 50  0000 C CNN
+F 0 "U40" H 4650 5481 50  0000 C CNN
 F 1 "74HC595" H 4650 5390 50  0000 C CNN
 F 2 "Package_SO:SOIC-16_3.9x9.9mm_P1.27mm" H 4650 4700 50  0001 C CNN
@@
 $EndComp
 $Comp
-L 74xx:74HC595 U63
+L 74xx:74HC595 U41
 U 1 1 622C9F3C
 P 6400 4700
-F 0 "U63" H 6400 5481 50  0000 C CNN
+F 0 "U41" H 6400 5481 50  0000 C CNN
 F 1 "74HC595" H 6400 5390 50  0000 C CNN
 F 2 "Package_SO:SOIC-16_3.9x9.9mm_P1.27mm" H 6400 4700 50  0001 C CNN
@@
 AR Path="/61DA7D11" Ref="#PWR?"  Part="1"
 AR Path="/61BD4B7D/61DA7D11" Ref="#PWR?"  Part="1"
-AR Path="/61E87E93/61DA7D11" Ref="#PWR0202"  Part="1"
-F 0 "#PWR0202" H 5450 3950 50  0001 C CNN
+AR Path="/61E87E93/61DA7D11" Ref="#PWR098"  Part="1"
+F 0 "#PWR098" H 5450 3950 50  0001 C CNN
 F 1 "+3V3" V 5465 4228 50  0000 L CNN
 F 2 "" H 5450 4100 50  0001 C CNN
@@
 AR Path="/61DA8643" Ref="#PWR?"  Part="1"
 AR Path="/61BD4B7D/61DA8643" Ref="#PWR?"  Part="1"
-AR Path="/61E87E93/61DA8643" Ref="#PWR0203"  Part="1"
-F 0 "#PWR0203" H 5450 5150 50  0001 C CNN
+AR Path="/61E87E93/61DA8643" Ref="#PWR099"  Part="1"
+F 0 "#PWR099" H 5450 5150 50  0001 C CNN
 F 1 "GND" H 5455 5227 50  0000 C CNN
 F 2 "" H 5450 5400 50  0001 C CNN
@@
 $EndComp
 $Comp
-L Device:C C98
+L Device:C C70
 U 1 1 61DA8C08
 P 5450 4250
-F 0 "C98" H 5565 4296 50  0000 L CNN
+F 0 "C70" H 5565 4296 50  0000 L CNN
 F 1 "0.1uF" H 5565 4205 50  0000 L CNN
 F 2 "Capacitor_SMD:C_0805_2012Metric" H 5488 4100 50  0001 C CNN
@@
 $EndComp
 $Comp
-L Device:C C97
+L Device:C C69
 U 1 1 61DA9C99
 P 3650 4250
-F 0 "C97" H 3750 4300 50  0000 L CNN
+F 0 "C69" H 3750 4300 50  0000 L CNN
 F 1 "0.1uF" H 3750 4200 50  0000 L CNN
 F 2 "Capacitor_SMD:C_0805_2012Metric" H 3688 4100 50  0001 C CNN
@@
 	3650 4100 4150 4100
 $Comp
-L Device:R R310
+L Device:R R117
 U 1 1 61EFFA0D
 P 4150 4250
-F 0 "R310" H 4100 4250 50  0000 R CNN
+F 0 "R117" H 4100 4250 50  0000 R CNN
 F 1 "10K" V 4150 4250 50  0000 C CNN
 F 2 "Resistor_SMD:R_0805_2012Metric" V 4080 4250 50  0001 C CNN

Commit message: Replace EVERY LT6106 with INA180A3
Friendship ended with LT6106
now ina180 is my best friend
Parts:
- renumbered C69 to C76, C70 to C77, R117 to R103
Changed lines of the file:
@@
 AR Path="/61DA7D11" Ref="#PWR?"  Part="1"
 AR Path="/61BD4B7D/61DA7D11" Ref="#PWR?"  Part="1"
-AR Path="/61E87E93/61DA7D11" Ref="#PWR098"  Part="1"
-F 0 "#PWR098" H 5450 3950 50  0001 C CNN
+AR Path="/61E87E93/61DA7D11" Ref="#PWR0112"  Part="1"
+F 0 "#PWR0112" H 5450 3950 50  0001 C CNN
 F 1 "+3V3" V 5465 4228 50  0000 L CNN
 F 2 "" H 5450 4100 50  0001 C CNN
@@
 AR Path="/61DA8643" Ref="#PWR?"  Part="1"
 AR Path="/61BD4B7D/61DA8643" Ref="#PWR?"  Part="1"
-AR Path="/61E87E93/61DA8643" Ref="#PWR099"  Part="1"
-F 0 "#PWR099" H 5450 5150 50  0001 C CNN
+AR Path="/61E87E93/61DA8643" Ref="#PWR0113"  Part="1"
+F 0 "#PWR0113" H 5450 5150 50  0001 C CNN
 F 1 "GND" H 5455 5227 50  0000 C CNN
 F 2 "" H 5450 5400 50  0001 C CNN
@@
 $EndComp
 $Comp
-L Device:C C70
+L Device:C C77
 U 1 1 61DA8C08
 P 5450 4250
-F 0 "C70" H 5565 4296 50  0000 L CNN
+F 0 "C77" H 5565 4296 50  0000 L CNN
 F 1 "0.1uF" H 5565 4205 50  0000 L CNN
 F 2 "Capacitor_SMD:C_0805_2012Metric" H 5488 4100 50  0001 C CNN
@@
 $EndComp
 $Comp
-L Device:C C69
+L Device:C C76
 U 1 1 61DA9C99
 P 3650 4250
-F 0 "C69" H 3750 4300 50  0000 L CNN
+F 0 "C76" H 3750 4300 50  0000 L CNN
 F 1 "0.1uF" H 3750 4200 50  0000 L CNN
 F 2 "Capacitor_SMD:C_0805_2012Metric" H 3688 4100 50  0001 C CNN
@@
 	3650 4100 4150 4100
 $Comp
-L Device:R R117
+L Device:R R103
 U 1 1 61EFFA0D
 P 4150 4250
-F 0 "R117" H 4100 4250 50  0000 R CNN
+F 0 "R103" H 4100 4250 50  0000 R CNN
 F 1 "10K" V 4150 4250 50  0000 C CNN
 F 2 "Resistor_SMD:R_0805_2012Metric" V 4080 4250 50  0001 C CNN

Commit message: change some power flags for latchup prevention
Connections:
- net +3V3 renamed VDD
Changed lines of the file:
@@
-$EndComp
-$Comp
-L power:+3V3 #PWR?
-U 1 1 61DA7D11
-P 5450 4100
-AR Path="/61DA7D11" Ref="#PWR?"  Part="1"
-AR Path="/61BD4B7D/61DA7D11" Ref="#PWR?"  Part="1"
-AR Path="/61E87E93/61DA7D11" Ref="#PWR0112"  Part="1"
-F 0 "#PWR0112" H 5450 3950 50  0001 C CNN
-F 1 "+3V3" V 5465 4228 50  0000 L CNN
-F 2 "" H 5450 4100 50  0001 C CNN
-F 3 "" H 5450 4100 50  0001 C CNN
-	1    5450 4100
-	1    0    0    -1
 $EndComp
 $Comp
@@
 Wire Notes Line
 	7250 3700 3500 3700
+$Comp
+L power:VDD #PWR?
+U 1 1 61FC1BD8
+P 5450 4100
+F 0 "#PWR?" H 5450 3950 50  0001 C CNN
+F 1 "VDD" H 5465 4273 50  0000 C CNN
+F 2 "" H 5450 4100 50  0001 C CNN
+F 3 "" H 5450 4100 50  0001 C CNN
+	1    5450 4100
+	1    0    0    -1
+$EndComp
 $EndSCHEMATC
