File: ECAD/EPS/PDM3V3.sch (KiCad schematic (older format))
At the start: 12 parts, among them Q53 2N7002, Q54 IRF7458, U67 LT6106

Commit message: wip: refine shunt resistor selection, add inhibits
Parts:
- R147: renamed from R243; footprint Resistor_SMD:R_2010_5025Metric -> Resistor_SMD:R_1206_3216Metric
- renumbered D31 to D25, Q53 to Q33, Q54 to Q34, R238 to R142, R239 to R143, R240 to R144, R241 to R145, R242 to R146, R244 to R148, R245 to R149, U67 to U45

Commit message: work
Parts:
- D25: value 1N4004 -> RR264MM; footprint Diode_SMD:D_SMA -> Diode_SMD:D_SOD-123F
Connections:
- net VOUT: now also D25.1 (K)
- net at Q34.1 (S), Q34.2 (S), Q34.3 (S)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: no longer D25.1 (K)
Other:
- moved on the sheet: D25
Changed lines of the file:
@@
 $Descr A4 11693 8268
 encoding utf-8
-Sheet 11 22
+Sheet 14 22
 Title "TJ Custom EPS"
 Date ""
@@
 Text HLabel 3300 2500 0    50   Input ~ 0
 GATE
-Text HLabel 6000 2350 2    50   Input ~ 0
+Text HLabel 7450 2350 2    50   Input ~ 0
 VOUT
 Text HLabel 6900 2850 2    50   Input ~ 0
@@
 L Device:D D?
 U 1 1 61F7AEBB
-P 4650 2550
+P 7450 2500
 AR Path="/61E87E93/61E898DE/61F7AEBB" Ref="D?"  Part="1"
 AR Path="/61E87E93/61ED0AEF/61F7AEBB" Ref="D?"  Part="1"
@@
 AR Path="/61E87E93/61EF422C/61F7AEBB" Ref="D22"  Part="1"
 AR Path="/61E87E93/61EF42FB/61F7AEBB" Ref="D23"  Part="1"
-F 0 "D25" V 4604 2630 50  0000 L CNN
-F 1 "1N4004" V 4695 2630 50  0000 L CNN
-F 2 "Diode_SMD:D_SMA" H 4650 2550 50  0001 C CNN
-F 3 "~" H 4650 2550 50  0001 C CNN
-	1    4650 2550
+F 0 "D25" V 7404 2580 50  0000 L CNN
+F 1 "RR264MM" V 7495 2580 50  0000 L CNN
+F 2 "Diode_SMD:D_SOD-123F" H 7450 2500 50  0001 C CNN
+F 3 "~" H 7450 2500 50  0001 C CNN
+	1    7450 2500
 	0    1    1    0
 $EndComp
-Wire Wire Line
-	4650 2350 4650 2400
 $Comp
 L Device:R R?
@@
 Connection ~ 6550 2850
 Connection ~ 5600 2350
-Wire Wire Line
-	6000 2350 5900 2350
 Connection ~ 5900 2350
 Text Notes 7000 2750 0    50   ~ 0
@@
 Connection ~ 4650 3150
 Wire Wire Line
-	4650 2700 4650 3150
-Wire Wire Line
 	4200 2700 4200 3150
 Connection ~ 4200 3150
@@
 Wire Wire Line
 	4650 2350 5100 2350
-Connection ~ 4650 2350
 Wire Wire Line
 	5100 2400 5100 2350
@@
 $EndComp
 Connection ~ 4650 1700
+Wire Wire Line
+	7450 3150 6550 3150
+Connection ~ 6550 3150
+Wire Wire Line
+	7450 2650 7450 3150
+Wire Wire Line
+	5900 2350 7450 2350
 $EndSCHEMATC

Commit message: Replace EVERY LT6106 with INA180A3
Friendship ended with LT6106
now ina180 is my best friend
Parts:
- removed R147: 10m, Resistor_SMD:R_1206_3216Metric, symbol Device:R
- removed R148: 100R, Resistor_SMD:R_0805_2012Metric, symbol Device:R
- removed R149: 2K, Resistor_SMD:R_0805_2012Metric, symbol Device:R
- removed U45: LT6106, Package_TO_SOT_SMD:SOT-23-5, symbol Amplifier_Current:LT6106
- added C78: 0.1uF, Capacitor_SMD:C_0603_1608Metric, symbol Device:C
- added R109: 4m, Resistor_SMD:R_1206_3216Metric, symbol Device:R
- added U42: INA180A3, Package_TO_SOT_SMD:SOT-23-5, symbol Amplifier_Current:INA138
- renumbered R142 to R122, R143 to R123, R144 to R124, R145 to R125, R146 to R126
Connections:
- net GND: now also C78.2, U42.2 (GND)
- net TELEM_IOUT: now also U42.1
- net VOUT: now also C78.1, R109.1, U42.4 (-), U42.5 (V+)
- net at Q34.1 (S), Q34.2 (S), Q34.3 (S)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: now also R109.2, U42.3 (+)
Other:
- note added: "400mV/A"
- note removed: "200mV/A"
- moved on the sheet: R125, R126

Commit message: 4 layer + fix pdm gate SRs
Changed lines of the file:
@@
 $Descr A4 11693 8268
 encoding utf-8
-Sheet 14 22
+Sheet 13 22
 Title "TJ Custom EPS"
 Date ""
@@
 AR Path="/61E87E93/61EF422C/61F7AEB8" Ref="Q28"  Part="1"
 AR Path="/61E87E93/61EF42FB/61F7AEB8" Ref="Q30"  Part="1"
-F 0 "Q34" H 4755 2196 50  0000 L CNN
+F 0 "Q32" H 4755 2196 50  0000 L CNN
 F 1 "IRF7458" H 4755 2105 50  0000 L CNN
 F 2 "Package_SO:SOIC-8_3.9x4.9mm_P1.27mm" H 4750 2075 50  0001 L CIN
@@
 AR Path="/61E87E93/61EF422C/61F7AEB9" Ref="Q27"  Part="1"
 AR Path="/61E87E93/61EF42FB/61F7AEB9" Ref="Q29"  Part="1"
-F 0 "Q33" H 4304 2546 50  0000 L CNN
+F 0 "Q31" H 4304 2546 50  0000 L CNN
 F 1 "2N7002" H 4304 2455 50  0000 L CNN
 F 2 "Package_TO_SOT_SMD:SOT-23" H 4300 2425 50  0001 L CIN
@@
 AR Path="/61E87E93/61EF422C/61E98108" Ref="R106"  Part="1"
 AR Path="/61E87E93/61EF42FB/61E98108" Ref="R112"  Part="1"
-F 0 "R124" H 4250 1850 50  0000 L CNN
+F 0 "R118" H 4250 1850 50  0000 L CNN
 F 1 "10K" V 4200 1850 50  0000 C CNN
 F 2 "Resistor_SMD:R_0805_2012Metric" V 4130 1850 50  0001 C CNN
@@
 AR Path="/61E87E93/61EF422C/61F7AEBB" Ref="D22"  Part="1"
 AR Path="/61E87E93/61EF42FB/61F7AEBB" Ref="D23"  Part="1"
-F 0 "D25" V 7404 2580 50  0000 L CNN
+F 0 "D24" V 7404 2580 50  0000 L CNN
 F 1 "RR264MM" V 7495 2580 50  0000 L CNN
 F 2 "Diode_SMD:D_SOD-123F" H 7450 2500 50  0001 C CNN
@@
 AR Path="/61E87E93/61EF422C/61F7AEBC" Ref="R104"  Part="1"
 AR Path="/61E87E93/61EF42FB/61F7AEBC" Ref="R110"  Part="1"
-F 0 "R122" V 3450 2500 50  0000 C CNN
+F 0 "R116" V 3450 2500 50  0000 C CNN
 F 1 "100R" V 3550 2500 50  0000 C CNN
 F 2 "Resistor_SMD:R_0805_2012Metric" V 3480 2500 50  0001 C CNN
@@
 AR Path="/61E87E93/61EF422C/61E9E045" Ref="R105"  Part="1"
 AR Path="/61E87E93/61EF42FB/61E9E045" Ref="R111"  Part="1"
-F 0 "R123" H 3850 2650 50  0000 L CNN
+F 0 "R117" H 3850 2650 50  0000 L CNN
 F 1 "10K" V 3800 2650 50  0000 C CNN
 F 2 "Resistor_SMD:R_0805_2012Metric" V 3730 2650 50  0001 C CNN
@@
 AR Path="/61E87E93/61EF422C/61E9FA3A" Ref="#PWR0115"  Part="1"
 AR Path="/61E87E93/61EF42FB/61E9FA3A" Ref="#PWR0118"  Part="1"
-F 0 "#PWR0124" H 4650 2900 50  0001 C CNN
+F 0 "#PWR0121" H 4650 2900 50  0001 C CNN
 F 1 "GND" H 4655 2977 50  0000 C CNN
 F 2 "" H 4650 3150 50  0001 C CNN
@@
 AR Path="/61E87E93/61EF422C/61F7AEC3" Ref="R107"  Part="1"
 AR Path="/61E87E93/61EF42FB/61F7AEC3" Ref="R113"  Part="1"
-F 0 "R125" H 4700 2550 50  0000 L CNN
+F 0 "R119" H 4700 2550 50  0000 L CNN
 F 1 "100K" V 4650 2550 50  0000 C CNN
 F 2 "Resistor_SMD:R_0805_2012Metric" V 4580 2550 50  0001 C CNN
@@
 AR Path="/61E87E93/61EF422C/61F7AEC4" Ref="R108"  Part="1"
 AR Path="/61E87E93/61EF42FB/61F7AEC4" Ref="R114"  Part="1"
-F 0 "R126" H 4700 2950 50  0000 L CNN
+F 0 "R120" H 4700 2950 50  0000 L CNN
 F 1 "100K" V 4650 2950 50  0000 C CNN
 F 2 "Resistor_SMD:R_0805_2012Metric" V 4580 2950 50  0001 C CNN
@@
 AR Path="/61E87E93/61EF422C/61EF2CDD" Ref="#PWR0114"  Part="1"
 AR Path="/61E87E93/61EF42FB/61EF2CDD" Ref="#PWR0117"  Part="1"
-F 0 "#PWR0123" H 4650 1550 50  0001 C CNN
+F 0 "#PWR0120" H 4650 1550 50  0001 C CNN
 F 1 "+3V3" H 4665 1873 50  0000 C CNN
 F 2 "" H 4650 1700 50  0001 C CNN
@@
 AR Path="/61E87E93/61EF4153/61FDAC13" Ref="R121"  Part="1"
 AR Path="/61E87E93/61EF1E50/61FDAC13" Ref="R127"  Part="1"
-F 0 "R127" V 5600 2350 50  0000 C CNN
+F 0 "R121" V 5600 2350 50  0000 C CNN
 F 1 "4m" V 5700 2350 50  0000 C CNN
 F 2 "Resistor_SMD:R_1206_3216Metric" V 5630 2350 50  0001 C CNN
@@
 AR Path="/61E87E93/61EF4153/61FDAC1C" Ref="U44"  Part="1"
 AR Path="/61E87E93/61EF1E50/61FDAC1C" Ref="U45"  Part="1"
-F 0 "U45" H 6594 2896 50  0000 L CNN
+F 0 "U44" H 6594 2896 50  0000 L CNN
 F 1 "INA180A3" H 6594 2805 50  0000 L CNN
 F 2 "Package_TO_SOT_SMD:SOT-23-5" H 6250 2850 50  0001 C CNN
@@
 AR Path="/61E87E93/61EF4153/61FDAC29" Ref="C80"  Part="1"
 AR Path="/61E87E93/61EF1E50/61FDAC29" Ref="C81"  Part="1"
-F 0 "C81" V 6450 2500 50  0000 R CNN
+F 0 "C80" V 6450 2500 50  0000 R CNN
 F 1 "0.1uF" V 6350 2500 50  0000 R CNN
 F 2 "Capacitor_SMD:C_0603_1608Metric" H 6338 2400 50  0001 C CNN
@@
 AR Path="/61E87E93/61EF4153/61FDAC30" Ref="#PWR0122"  Part="1"
 AR Path="/61E87E93/61EF1E50/61FDAC30" Ref="#PWR0125"  Part="1"
-F 0 "#PWR0125" H 6450 2300 50  0001 C CNN
+F 0 "#PWR0122" H 6450 2300 50  0001 C CNN
 F 1 "GND" H 6455 2377 50  0000 C CNN
 F 2 "" H 6450 2550 50  0001 C CNN

Commit message: 0603 and route
Parts:
- R122, R123, R124, R125, R126: footprint Resistor_SMD:R_0805_2012Metric -> Resistor_SMD:R_0603_1608Metric
Changed lines of the file:
@@
 $Descr A4 11693 8268
 encoding utf-8
-Sheet 13 22
+Sheet 14 22
 Title "TJ Custom EPS"
 Date ""
@@
 AR Path="/61E87E93/61EF422C/61F7AEB8" Ref="Q28"  Part="1"
 AR Path="/61E87E93/61EF42FB/61F7AEB8" Ref="Q30"  Part="1"
-F 0 "Q32" H 4755 2196 50  0000 L CNN
+F 0 "Q34" H 4755 2196 50  0000 L CNN
 F 1 "IRF7458" H 4755 2105 50  0000 L CNN
 F 2 "Package_SO:SOIC-8_3.9x4.9mm_P1.27mm" H 4750 2075 50  0001 L CIN
@@
 AR Path="/61E87E93/61EF422C/61F7AEB9" Ref="Q27"  Part="1"
 AR Path="/61E87E93/61EF42FB/61F7AEB9" Ref="Q29"  Part="1"
-F 0 "Q31" H 4304 2546 50  0000 L CNN
+F 0 "Q33" H 4304 2546 50  0000 L CNN
 F 1 "2N7002" H 4304 2455 50  0000 L CNN
 F 2 "Package_TO_SOT_SMD:SOT-23" H 4300 2425 50  0001 L CIN
@@
 AR Path="/61E87E93/61EF422C/61E98108" Ref="R106"  Part="1"
 AR Path="/61E87E93/61EF42FB/61E98108" Ref="R112"  Part="1"
-F 0 "R118" H 4250 1850 50  0000 L CNN
+F 0 "R124" H 4250 1850 50  0000 L CNN
 F 1 "10K" V 4200 1850 50  0000 C CNN
-F 2 "Resistor_SMD:R_0805_2012Metric" V 4130 1850 50  0001 C CNN
+F 2 "Resistor_SMD:R_0603_1608Metric" V 4130 1850 50  0001 C CNN
 F 3 "~" H 4200 1850 50  0001 C CNN
 	1    4200 1850
@@
 AR Path="/61E87E93/61EF422C/61F7AEBB" Ref="D22"  Part="1"
 AR Path="/61E87E93/61EF42FB/61F7AEBB" Ref="D23"  Part="1"
-F 0 "D24" V 7404 2580 50  0000 L CNN
+F 0 "D25" V 7404 2580 50  0000 L CNN
 F 1 "RR264MM" V 7495 2580 50  0000 L CNN
 F 2 "Diode_SMD:D_SOD-123F" H 7450 2500 50  0001 C CNN
@@
 AR Path="/61E87E93/61EF422C/61F7AEBC" Ref="R104"  Part="1"
 AR Path="/61E87E93/61EF42FB/61F7AEBC" Ref="R110"  Part="1"
-F 0 "R116" V 3450 2500 50  0000 C CNN
+F 0 "R122" V 3450 2500 50  0000 C CNN
 F 1 "100R" V 3550 2500 50  0000 C CNN
-F 2 "Resistor_SMD:R_0805_2012Metric" V 3480 2500 50  0001 C CNN
+F 2 "Resistor_SMD:R_0603_1608Metric" V 3480 2500 50  0001 C CNN
 F 3 "~" H 3550 2500 50  0001 C CNN
 	1    3550 2500
@@
 AR Path="/61E87E93/61EF422C/61E9E045" Ref="R105"  Part="1"
 AR Path="/61E87E93/61EF42FB/61E9E045" Ref="R111"  Part="1"
-F 0 "R117" H 3850 2650 50  0000 L CNN
+F 0 "R123" H 3850 2650 50  0000 L CNN
 F 1 "10K" V 3800 2650 50  0000 C CNN
-F 2 "Resistor_SMD:R_0805_2012Metric" V 3730 2650 50  0001 C CNN
+F 2 "Resistor_SMD:R_0603_1608Metric" V 3730 2650 50  0001 C CNN
 F 3 "~" H 3800 2650 50  0001 C CNN
 	1    3800 2650
@@
 AR Path="/61E87E93/61EF422C/61E9FA3A" Ref="#PWR0115"  Part="1"
 AR Path="/61E87E93/61EF42FB/61E9FA3A" Ref="#PWR0118"  Part="1"
-F 0 "#PWR0121" H 4650 2900 50  0001 C CNN
+F 0 "#PWR0124" H 4650 2900 50  0001 C CNN
 F 1 "GND" H 4655 2977 50  0000 C CNN
 F 2 "" H 4650 3150 50  0001 C CNN
@@
 AR Path="/61E87E93/61EF422C/61F7AEC3" Ref="R107"  Part="1"
 AR Path="/61E87E93/61EF42FB/61F7AEC3" Ref="R113"  Part="1"
-F 0 "R119" H 4700 2550 50  0000 L CNN
+F 0 "R125" H 4700 2550 50  0000 L CNN
 F 1 "100K" V 4650 2550 50  0000 C CNN
-F 2 "Resistor_SMD:R_0805_2012Metric" V 4580 2550 50  0001 C CNN
+F 2 "Resistor_SMD:R_0603_1608Metric" V 4580 2550 50  0001 C CNN
 F 3 "~" H 4650 2550 50  0001 C CNN
 	1    4650 2550
@@
 AR Path="/61E87E93/61EF422C/61F7AEC4" Ref="R108"  Part="1"
 AR Path="/61E87E93/61EF42FB/61F7AEC4" Ref="R114"  Part="1"
-F 0 "R120" H 4700 2950 50  0000 L CNN
+F 0 "R126" H 4700 2950 50  0000 L CNN
 F 1 "100K" V 4650 2950 50  0000 C CNN
-F 2 "Resistor_SMD:R_0805_2012Metric" V 4580 2950 50  0001 C CNN
+F 2 "Resistor_SMD:R_0603_1608Metric" V 4580 2950 50  0001 C CNN
 F 3 "~" H 4650 2950 50  0001 C CNN
 	1    4650 2950
@@
 AR Path="/61E87E93/61EF422C/61EF2CDD" Ref="#PWR0114"  Part="1"
 AR Path="/61E87E93/61EF42FB/61EF2CDD" Ref="#PWR0117"  Part="1"
-F 0 "#PWR0120" H 4650 1550 50  0001 C CNN
+F 0 "#PWR0123" H 4650 1550 50  0001 C CNN
 F 1 "+3V3" H 4665 1873 50  0000 C CNN
 F 2 "" H 4650 1700 50  0001 C CNN
@@
 AR Path="/61E87E93/61EF4153/61FDAC13" Ref="R121"  Part="1"
 AR Path="/61E87E93/61EF1E50/61FDAC13" Ref="R127"  Part="1"
-F 0 "R121" V 5600 2350 50  0000 C CNN
+F 0 "R127" V 5600 2350 50  0000 C CNN
 F 1 "4m" V 5700 2350 50  0000 C CNN
 F 2 "Resistor_SMD:R_1206_3216Metric" V 5630 2350 50  0001 C CNN
@@
 AR Path="/61E87E93/61EF4153/61FDAC1C" Ref="U44"  Part="1"
 AR Path="/61E87E93/61EF1E50/61FDAC1C" Ref="U45"  Part="1"
-F 0 "U44" H 6594 2896 50  0000 L CNN
+F 0 "U45" H 6594 2896 50  0000 L CNN
 F 1 "INA180A3" H 6594 2805 50  0000 L CNN
 F 2 "Package_TO_SOT_SMD:SOT-23-5" H 6250 2850 50  0001 C CNN
@@
 AR Path="/61E87E93/61EF4153/61FDAC29" Ref="C80"  Part="1"
 AR Path="/61E87E93/61EF1E50/61FDAC29" Ref="C81"  Part="1"
-F 0 "C80" V 6450 2500 50  0000 R CNN
+F 0 "C81" V 6450 2500 50  0000 R CNN
 F 1 "0.1uF" V 6350 2500 50  0000 R CNN
 F 2 "Capacitor_SMD:C_0603_1608Metric" H 6338 2400 50  0001 C CNN
@@
 AR Path="/61E87E93/61EF4153/61FDAC30" Ref="#PWR0122"  Part="1"
 AR Path="/61E87E93/61EF1E50/61FDAC30" Ref="#PWR0125"  Part="1"
-F 0 "#PWR0122" H 6450 2300 50  0001 C CNN
+F 0 "#PWR0125" H 6450 2300 50  0001 C CNN
 F 1 "GND" H 6455 2377 50  0000 C CNN
 F 2 "" H 6450 2550 50  0001 C CNN
