File: ECAD/EPS/PDM5V.sch (KiCad schematic (older format))
At the start: 12 parts, among them Q61 2N7002, Q62 IRF7458, U71 LT6106

Commit message: wip: refine shunt resistor selection, add inhibits
Parts:
- R179: renamed from R275; footprint Resistor_SMD:R_2010_5025Metric -> Resistor_SMD:R_1206_3216Metric
- renumbered D35 to D29, Q61 to Q41, Q62 to Q42, R270 to R174, R271 to R175, R272 to R176, R273 to R177, R274 to R178, R276 to R180, R277 to R181, U71 to U49

Commit message: work
Parts:
- D29: value 1N4004 -> RR264MM; footprint Diode_SMD:D_SMA -> Diode_SMD:D_SOD-123F
Connections:
- net VOUT: now also D29.1 (K)
- net at Q42.1 (S), Q42.2 (S), Q42.3 (S)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: no longer D29.1 (K)
Other:
- moved on the sheet: D29
Changed lines of the file:
@@
 $Descr A4 11693 8268
 encoding utf-8
-Sheet 15 22
+Sheet 18 22
 Title "TJ Custom EPS"
 Date ""
@@
 Text HLabel 3300 2500 0    50   Input ~ 0
 GATE
-Text HLabel 6000 2350 2    50   Input ~ 0
+Text HLabel 7500 2350 2    50   Input ~ 0
 VOUT
 Text HLabel 6900 2850 2    50   Input ~ 0
@@
 L Device:D D?
 U 1 1 61EF1EB7
-P 4650 2550
+P 7500 2500
 AR Path="/61E87E93/61E898DE/61EF1EB7" Ref="D?"  Part="1"
 AR Path="/61E87E93/61ED0AEF/61EF1EB7" Ref="D?"  Part="1"
@@
 AR Path="/61E87E93/61EF1CFC/61EF1EB7" Ref="D26"  Part="1"
 AR Path="/61E87E93/61EF1E50/61EF1EB7" Ref="D?"  Part="1"
-F 0 "D29" V 4604 2630 50  0000 L CNN
-F 1 "1N4004" V 4695 2630 50  0000 L CNN
-F 2 "Diode_SMD:D_SMA" H 4650 2550 50  0001 C CNN
-F 3 "~" H 4650 2550 50  0001 C CNN
-	1    4650 2550
+F 0 "D29" V 7454 2580 50  0000 L CNN
+F 1 "RR264MM" V 7545 2580 50  0000 L CNN
+F 2 "Diode_SMD:D_SOD-123F" H 7500 2500 50  0001 C CNN
+F 3 "~" H 7500 2500 50  0001 C CNN
+	1    7500 2500
 	0    1    1    0
 $EndComp
-Wire Wire Line
-	4650 2350 4650 2400
 $Comp
 L Device:R R?
@@
 Connection ~ 6550 2850
 Connection ~ 5600 2350
-Wire Wire Line
-	6000 2350 5900 2350
 Connection ~ 5900 2350
 Text Notes 7000 2750 0    50   ~ 0
@@
 Connection ~ 4650 3150
 Wire Wire Line
-	4650 2700 4650 3150
-Wire Wire Line
 	4200 2700 4200 3150
 Connection ~ 4200 3150
@@
 Wire Wire Line
 	4650 2350 5100 2350
-Connection ~ 4650 2350
 Wire Wire Line
 	5100 2400 5100 2350
@@
 $EndComp
 Connection ~ 4650 1700
+Wire Wire Line
+	7500 3150 6550 3150
+Connection ~ 6550 3150
+Wire Wire Line
+	5900 2350 7500 2350
+Wire Wire Line
+	7500 2650 7500 3150
 $EndSCHEMATC

Commit message: Replace EVERY LT6106 with INA180A3
Friendship ended with LT6106
now ina180 is my best friend
Parts:
- removed R179: 10m, Resistor_SMD:R_1206_3216Metric, symbol Device:R
- removed R180: 100R, Resistor_SMD:R_0805_2012Metric, symbol Device:R
- removed R181: 2K, Resistor_SMD:R_0805_2012Metric, symbol Device:R
- removed U49: LT6106, Package_TO_SOT_SMD:SOT-23-5, symbol Amplifier_Current:LT6106
- added C82: 0.1uF, Capacitor_SMD:C_0603_1608Metric, symbol Device:C
- added R151: 4m, Resistor_SMD:R_1206_3216Metric, symbol Device:R
- added U46: INA180A3, Package_TO_SOT_SMD:SOT-23-5, symbol Amplifier_Current:INA138
- renumbered R174 to R146, R175 to R147, R176 to R148, R177 to R149, R178 to R150
Connections:
- net GND: now also C82.2, U46.2 (GND)
- net TELEM_IOUT: now also U46.1
- net VOUT: now also C82.1, R151.1, U46.4 (-), U46.5 (V+)
- net at Q42.1 (S), Q42.2 (S), Q42.3 (S)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: now also R151.2, U46.3 (+)
Other:
- note added: "400mV/A"
- note removed: "200mV/A"
- moved on the sheet: D29, R149, R150

Commit message: 0603 and route
Parts:
- R146, R147, R148, R149, R150: footprint Resistor_SMD:R_0805_2012Metric -> Resistor_SMD:R_0603_1608Metric
Changed lines of the file:
@@
 F 0 "R148" H 4250 1850 50  0000 L CNN
 F 1 "10K" V 4200 1850 50  0000 C CNN
-F 2 "Resistor_SMD:R_0805_2012Metric" V 4130 1850 50  0001 C CNN
+F 2 "Resistor_SMD:R_0603_1608Metric" V 4130 1850 50  0001 C CNN
 F 3 "~" H 4200 1850 50  0001 C CNN
 	1    4200 1850
@@
 F 0 "R146" V 3450 2500 50  0000 C CNN
 F 1 "100R" V 3550 2500 50  0000 C CNN
-F 2 "Resistor_SMD:R_0805_2012Metric" V 3480 2500 50  0001 C CNN
+F 2 "Resistor_SMD:R_0603_1608Metric" V 3480 2500 50  0001 C CNN
 F 3 "~" H 3550 2500 50  0001 C CNN
 	1    3550 2500
@@
 F 0 "R147" H 3850 2650 50  0000 L CNN
 F 1 "10K" V 3800 2650 50  0000 C CNN
-F 2 "Resistor_SMD:R_0805_2012Metric" V 3730 2650 50  0001 C CNN
+F 2 "Resistor_SMD:R_0603_1608Metric" V 3730 2650 50  0001 C CNN
 F 3 "~" H 3800 2650 50  0001 C CNN
 	1    3800 2650
@@
 F 0 "R149" H 4700 2550 50  0000 L CNN
 F 1 "100K" V 4650 2550 50  0000 C CNN
-F 2 "Resistor_SMD:R_0805_2012Metric" V 4580 2550 50  0001 C CNN
+F 2 "Resistor_SMD:R_0603_1608Metric" V 4580 2550 50  0001 C CNN
 F 3 "~" H 4650 2550 50  0001 C CNN
 	1    4650 2550
@@
 F 0 "R150" H 4700 2950 50  0000 L CNN
 F 1 "100K" V 4650 2950 50  0000 C CNN
-F 2 "Resistor_SMD:R_0805_2012Metric" V 4580 2950 50  0001 C CNN
+F 2 "Resistor_SMD:R_0603_1608Metric" V 4580 2950 50  0001 C CNN
 F 3 "~" H 4650 2950 50  0001 C CNN
 	1    4650 2950
