File: ECAD/EPS/Boost-BuckMPPT.sch (KiCad schematic (older format))
At the start: 35 parts, among them Q27 Si4186DY, U31 LM358, U32 LT6106, U33 LT6106, U34 LT3652EMSE, U35 LMC555xM

Commit message: wip: refine shunt resistor selection, add inhibits
Parts:
- R49: renamed from R116; value 20m -> 10m; footprint Resistor_SMD:R_2512_6332Metric -> Resistor_SMD:R_1206_3216Metric
- R50: renamed from R117; value 20m -> 10m; footprint Resistor_SMD:R_2512_6332Metric -> Resistor_SMD:R_1206_3216Metric
- renumbered C50 to C28, C51 to C29, C52 to C30, C53 to C31, C54 to C32, C55 to C33, C56 to C34, C57 to C35, D23 to D17, D24 to D18, D25 to D19, L4 to L3, L5 to L4, Q27 to Q6, R114 to R47, R115 to R48, R118 to R51, R119 to R52, R120 to R53, R121 to R54, R122 to R55, R123 to R56, R124 to R57, R125 to R58, R126 to R59, R127 to R60, R128 to R61, R129 to R62, U31 to U21, U32 to U22, U33 to U23, U34 to U24, U35 to U25
Other:
- note added: "Gain = Rout/Rin = 100\n1V/A"
- note removed: "Gain = Rout/Rin = 100\n2V/A"

Commit message: Replace EVERY LT6106 with INA180A3
Friendship ended with LT6106
now ina180 is my best friend
Parts:
- removed R47, R48: 50R, Resistor_SMD:R_0805_2012Metric, symbol Device:R
- removed R49, R50: 10m, Resistor_SMD:R_1206_3216Metric, symbol Device:R
- removed R53, R54: 5K, Resistor_SMD:R_0805_2012Metric, symbol Device:R
- removed U22, U23: LT6106, Package_TO_SOT_SMD:SOT-23-5, symbol Amplifier_Current:LT6106
- added C33, C34: 0.1uF, Capacitor_SMD:C_0603_1608Metric, symbol Device:C
- added R37, R38: 4m, Resistor_SMD:R_1206_3216Metric, symbol Device:R
- added U22, U23: INA180A3, Package_TO_SOT_SMD:SOT-23-5, symbol Amplifier_Current:INA138
- renumbered C28 to C35, C29 to C36, C30 to C37, C31 to C38, C32 to C39, C33 to C40, C34 to C41, C35 to C42, R51 to R39, R52 to R40, R55 to R41, R56 to R42, R57 to R43, R58 to R44, R59 to R45, R60 to R46, R61 to R47, R62 to R48
Connections:
- net A_PWR: now also R37.2, U22.3 (+)
- net B_PWR: now also R38.2, U23.3 (+)
- net GND: now also C33.2, C34.2, U22.2 (GND), U23.2 (GND)
- net TELEM_I_A: now also U22.1
- net TELEM_I_B: now also U23.1
- net at C40.1, L4.1, R41.1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: now also R37.1, R38.1, U22.4 (-), U23.4 (-)
- new net +3.3VA: C33.1, C34.1, U22.5 (V+), U23.5 (V+)
Other:
- note added: "100V/V Gain\n400mV/A"
- note removed: "Gain = Rout/Rin = 100\n1V/A"

Commit message: correct setpoint circuitry
Parts:
- R39: value 1K -> 10K
- R40: value 7.5K -> 75K
Connections:
- net +3.3VA: now also U21.8 (V+)
- net TELEM_VIN: now also U21.1, U21.2 (-); no longer R41.2, R42.1
- net VBOOST: now also R40.1; no longer U21.5 (+), U21.8 (V+)
- net Vset: now also U21.6 (-); no longer U21.3 (+)
- net at R39.1, R40.2: now also U21.5 (+); no longer U21.2 (-)
- new net: R41.2, R42.1, U21.3 (+)
Other:
- moved on the sheet: R39, R40, U21A, U21B, U21C
Changed lines of the file:
@@
 	1    0    0    -1
 $EndComp
-Wire Wire Line
-	1400 5000 950  5000
-Connection ~ 1400 5000
-Wire Wire Line
-	1400 4900 1400 5000
-Wire Wire Line
-	950  4400 950  5000
-Wire Wire Line
-	2950 5000 2000 5000
 Connection ~ 2950 5000
 Wire Wire Line
@@
 Wire Wire Line
 	3850 4800 3850 5000
-Wire Wire Line
-	2000 5000 1400 5000
 Connection ~ 2000 5000
 Wire Wire Line
@@
 	0    1    1    0
 $EndComp
-Wire Wire Line
-	2750 4200 3350 4200
-Connection ~ 2150 3800
-Wire Wire Line
-	2150 3800 2950 3800
 Text Notes 600  3050 0    50   ~ 0
 Vmp Setpoint
@@
 	1    0    0    -1
 $EndComp
-Connection ~ 1400 4600
-Wire Wire Line
-	1400 4600 1400 4400
-Wire Wire Line
-	1550 4600 1400 4600
-Connection ~ 2000 4300
-Wire Wire Line
-	1850 4600 2000 4600
-Wire Wire Line
-	2000 4600 2000 4300
 $Comp
 L Device:R R?
 U 1 1 61D7BAE9
-P 1400 4750
+P 2000 4800
 AR Path="/61BEC565/61BEC848/61D7BAE9" Ref="R?"  Part="1"
 AR Path="/61BEC565/61BFB023/61D7BAE9" Ref="R?"  Part="1"
@@
 AR Path="/61BEC565/61E1083C/61D7BAE9" Ref="R?"  Part="1"
 AR Path="/61BEC565/61D120A6/61D7BAE9" Ref="R39"  Part="1"
-F 0 "R39" H 1450 4750 50  0000 L CNN
-F 1 "1K" V 1400 4750 50  0000 C CNN
-F 2 "Resistor_SMD:R_0805_2012Metric" V 1330 4750 50  0001 C CNN
-F 3 "~" H 1400 4750 50  0001 C CNN
-	1    1400 4750
+F 0 "R39" H 2050 4800 50  0000 L CNN
+F 1 "10K" V 2000 4800 50  0000 C CNN
+F 2 "Resistor_SMD:R_0805_2012Metric" V 1930 4800 50  0001 C CNN
+F 3 "~" H 2000 4800 50  0001 C CNN
+	1    2000 4800
 	1    0    0    -1
 $EndComp
@@
 L Device:R R?
 U 1 1 61D7BAE3
-P 1700 4600
+P 2000 4000
 AR Path="/61BEC565/61BEC848/61D7BAE3" Ref="R?"  Part="1"
 AR Path="/61BEC565/61BFB023/61D7BAE3" Ref="R?"  Part="1"
@@
 AR Path="/61BEC565/61E1083C/61D7BAE3" Ref="R?"  Part="1"
 AR Path="/61BEC565/61D120A6/61D7BAE3" Ref="R40"  Part="1"
-F 0 "R40" V 1800 4600 50  0000 C CNN
-F 1 "7.5K" V 1700 4600 50  0000 C CNN
-F 2 "Resistor_SMD:R_0805_2012Metric" V 1630 4600 50  0001 C CNN
-F 3 "~" H 1700 4600 50  0001 C CNN
-	1    1700 4600
-	0    1    1    0
-$EndComp
-Text HLabel 1300 4200 0    50   Input ~ 0
+F 0 "R40" H 2050 4000 50  0000 L CNN
+F 1 "75K" V 2000 4000 50  0000 C CNN
+F 2 "Resistor_SMD:R_0805_2012Metric" V 1930 4000 50  0001 C CNN
+F 3 "~" H 2000 4000 50  0001 C CNN
+	1    2000 4000
+	1    0    0    -1
+$EndComp
+Text HLabel 1950 4400 0    50   Input ~ 0
 Vset
-Wire Wire Line
-	1400 4200 1300 4200
-Wire Wire Line
-	950  3800 2150 3800
-Wire Wire Line
-	2150 4100 2150 3800
-Wire Wire Line
-	2000 4300 2150 4300
 $Comp
 L Amplifier_Operational:LM358 U?
 U 3 1 61D7BAD6
-P 1050 4100
+P 1400 4700
 AR Path="/61BEC565/61BEC848/61D7BAD6" Ref="U?"  Part="3"
 AR Path="/61BEC565/61BFB023/61D7BAD6" Ref="U?"  Part="3"
@@
 AR Path="/61BEC565/61E1083C/61D7BAD6" Ref="U?"  Part="3"
 AR Path="/61BEC565/61D120A6/61D7BAD6" Ref="U21"  Part="3"
-F 0 "U21" H 750 4150 50  0000 L CNN
-F 1 "LM358" H 650 4050 50  0000 L CNN
-F 2 "Package_SO:SO-8_3.9x4.9mm_P1.27mm" H 1050 4100 50  0001 C CNN
-F 3 "http://www.ti.com/lit/ds/symlink/lm2904-n.pdf" H 1050 4100 50  0001 C CNN
-	3    1050 4100
+F 0 "U21" H 1100 4750 50  0000 L CNN
+F 1 "LM358" H 1000 4650 50  0000 L CNN
+F 2 "Package_SO:SO-8_3.9x4.9mm_P1.27mm" H 1400 4700 50  0001 C CNN
+F 3 "http://www.ti.com/lit/ds/symlink/lm2904-n.pdf" H 1400 4700 50  0001 C CNN
+	3    1400 4700
 	1    0    0    -1
 $EndComp
@@
 L Amplifier_Operational:LM358 U?
 U 2 1 61D7BAD0
-P 2450 4200
+P 2400 4300
 AR Path="/61BEC565/61BEC848/61D7BAD0" Ref="U?"  Part="2"
 AR Path="/61BEC565/61BFB023/61D7BAD0" Ref="U?"  Part="2"
@@
 AR Path="/61BEC565/61E1083C/61D7BAD0" Ref="U?"  Part="2"
 AR Path="/61BEC565/61D120A6/61D7BAD0" Ref="U21"  Part="2"
-F 0 "U21" H 2450 4567 50  0000 C CNN
-F 1 "LM358" H 2450 4476 50  0000 C CNN
-F 2 "Package_SO:SO-8_3.9x4.9mm_P1.27mm" H 2450 4200 50  0001 C CNN
-F 3 "http://www.ti.com/lit/ds/symlink/lm2904-n.pdf" H 2450 4200 50  0001 C CNN
-	2    2450 4200
+F 0 "U21" H 2400 4667 50  0000 C CNN
+F 1 "LM358" H 2400 4576 50  0000 C CNN
+F 2 "Package_SO:SO-8_3.9x4.9mm_P1.27mm" H 2400 4300 50  0001 C CNN
+F 3 "http://www.ti.com/lit/ds/symlink/lm2904-n.pdf" H 2400 4300 50  0001 C CNN
+	2    2400 4300
 	1    0    0    -1
 $EndComp
@@
 L Amplifier_Operational:LM358 U?
 U 1 1 61D7BACA
-P 1700 4300
+P 3700 2200
 AR Path="/61BEC565/61BEC848/61D7BACA" Ref="U?"  Part="1"
 AR Path="/61BEC565/61BFB023/61D7BACA" Ref="U?"  Part="1"
@@
 AR Path="/61BEC565/61E1083C/61D7BACA" Ref="U?"  Part="1"
 AR Path="/61BEC565/61D120A6/61D7BACA" Ref="U21"  Part="1"
-F 0 "U21" H 1700 4667 50  0000 C CNN
-F 1 "LM358" H 1700 4576 50  0000 C CNN
-F 2 "Package_SO:SO-8_3.9x4.9mm_P1.27mm" H 1700 4300 50  0001 C CNN
-F 3 "http://www.ti.com/lit/ds/symlink/lm2904-n.pdf" H 1700 4300 50  0001 C CNN
-	1    1700 4300
+F 0 "U21" H 3700 2567 50  0000 C CNN
+F 1 "LM358" H 3700 2476 50  0000 C CNN
+F 2 "Package_SO:SO-8_3.9x4.9mm_P1.27mm" H 3700 2200 50  0001 C CNN
+F 3 "http://www.ti.com/lit/ds/symlink/lm2904-n.pdf" H 3700 2200 50  0001 C CNN
+	1    3700 2200
 	1    0    0    -1
 $EndComp
@@
 Wire Wire Line
 	3200 1500 3200 1400
-Wire Wire Line
-	3200 1950 3200 2100
-Connection ~ 3200 1950
-Wire Wire Line
-	3200 1950 3450 1950
-Wire Wire Line
-	3200 1800 3200 1950
 $Comp
 L Device:R R?
@@
 	1    0    0    -1
 $EndComp
-Text HLabel 3450 1950 2    50   Input ~ 0
+Text HLabel 4000 2200 2    50   Input ~ 0
 TELEM_VIN
 Wire Wire Line
@@
 Text Label 600  3800 0    50   ~ 0
 VBOOST
-Wire Wire Line
-	600  3800 950  3800
-Connection ~ 950  3800
 Wire Notes Line
 	2750 5300 550  5300
@@
 Wire Wire Line
 	1300 1850 3000 1850
+Wire Wire Line
+	2000 5000 2950 5000
+Wire Wire Line
+	2000 4150 2000 4200
+Wire Wire Line
+	2000 4200 2100 4200
+Connection ~ 2000 4200
+Wire Wire Line
+	2000 3850 2000 3800
+Connection ~ 2000 3800
+Wire Wire Line
+	2000 3800 2950 3800
+Wire Wire Line
+	2000 4200 2000 4650
+Wire Wire Line
+	2100 4400 1950 4400
+Wire Wire Line
+	2700 4300 3050 4300
+Wire Wire Line
+	3050 4300 3050 4200
+Wire Wire Line
+	3050 4200 3350 4200
+Wire Wire Line
+	3200 1800 3200 2100
+Wire Wire Line
+	3400 2100 3200 2100
+Connection ~ 3200 2100
+Wire Wire Line
+	3400 2300 3400 2500
+Wire Wire Line
+	3400 2500 4000 2500
+Wire Wire Line
+	4000 2500 4000 2200
+Wire Wire Line
+	600  3800 2000 3800
+Wire Wire Line
+	1300 5000 2000 5000
+$Comp
+L power:+3.3VA #PWR?
+U 1 1 6219DE8C
+P 1300 4400
+F 0 "#PWR?" H 1300 4250 50  0001 C CNN
+F 1 "+3.3VA" H 1315 4573 50  0000 C CNN
+F 2 "" H 1300 4400 50  0001 C CNN
+F 3 "" H 1300 4400 50  0001 C CNN
+	1    1300 4400
+	1    0    0    -1
+$EndComp
+Wire Wire Line
+	2000 4950 2000 5000
 $EndSCHEMATC
