File: ECAD/EPS/MPPT.sch (KiCad schematic (older format))
At the start: 24 parts, among them U27 LT6106, U28 LT6106, U29 LM358, U30 LT3652EMSE

Commit message: wip: refine shunt resistor selection, add inhibits
Parts:
- R35: renamed from R102; value 20m -> 10m; footprint Resistor_SMD:R_2512_6332Metric -> Resistor_SMD:R_1206_3216Metric
- R36: renamed from R103; value 20m -> 10m; footprint Resistor_SMD:R_2512_6332Metric -> Resistor_SMD:R_1206_3216Metric
- renumbered C47 to C25, C48 to C26, C49 to C27, D21 to D15, D22 to D16, L3 to L2, R100 to R33, R101 to R34, R104 to R37, R105 to R38, R106 to R39, R107 to R40, R108 to R41, R109 to R42, R110 to R43, R111 to R44, R112 to R45, R113 to R46, U27 to U17, U28 to U18, U29 to U19, U30 to U20
Other:
- note added: "Gain = Rout/Rin = 100\n1V/A"
- note removed: "Gain = Rout/Rin = 100\n2V/A"

Commit message: Round off some corners and set up eps board for routing
Changed lines of the file:
@@
 $Descr USLetter 11000 8500
 encoding utf-8
-Sheet 4 22
+Sheet 3 22
 Title "TJ Custom EPS"
 Date ""
@@
 AR Path="/61BEC565/61E10014/61BF0603" Ref="R21"  Part="1"
 AR Path="/61BEC565/61E1083C/61BF0603" Ref="R?"  Part="1"
-F 0 "R35" V 950 750 50  0000 C CNN
+F 0 "R21" V 950 750 50  0000 C CNN
 F 1 "10m" V 1050 750 50  0000 C CNN
 F 2 "Resistor_SMD:R_1206_3216Metric" V 980 750 50  0001 C CNN
@@
 AR Path="/61BEC565/61E10014/61C169BE" Ref="R19"  Part="1"
 AR Path="/61BEC565/61E1083C/61C169BE" Ref="R?"  Part="1"
-F 0 "R33" H 900 1150 50  0000 L CNN
+F 0 "R19" H 900 1150 50  0000 L CNN
 F 1 "50R" V 850 1150 50  0000 C CNN
 F 2 "Resistor_SMD:R_0805_2012Metric" V 780 1150 50  0001 C CNN
@@
 AR Path="/61BEC565/61E10014/61C24A1A" Ref="U16"  Part="1"
 AR Path="/61BEC565/61E1083C/61C24A1A" Ref="U?"  Part="1"
-F 0 "U20" H 6900 2531 50  0000 C CNN
+F 0 "U16" H 6900 2531 50  0000 C CNN
 F 1 "LT3652EMSE" H 6900 2440 50  0000 C CNN
 F 2 "Package_SO:MSOP-12-1EP_3x4mm_P0.65mm_EP1.65x2.85mm" H 6900 1250 50  0001 C CNN
@@
 AR Path="/61BEC565/61E10014/61C384AF" Ref="U15"  Part="1"
 AR Path="/61BEC565/61E1083C/61C384AF" Ref="U?"  Part="1"
-F 0 "U19" H 4750 2217 50  0000 C CNN
+F 0 "U15" H 4750 2217 50  0000 C CNN
 F 1 "LM358" H 4750 2126 50  0000 C CNN
 F 2 "Package_SO:SO-8_3.9x4.9mm_P1.27mm" H 4750 1850 50  0001 C CNN
@@
 AR Path="/61BEC565/61E10014/61C39A83" Ref="U15"  Part="2"
 AR Path="/61BEC565/61E1083C/61C39A83" Ref="U?"  Part="2"
-F 0 "U19" H 5500 2117 50  0000 C CNN
+F 0 "U15" H 5500 2117 50  0000 C CNN
 F 1 "LM358" H 5500 2026 50  0000 C CNN
 F 2 "Package_SO:SO-8_3.9x4.9mm_P1.27mm" H 5500 1750 50  0001 C CNN
@@
 AR Path="/61BEC565/61E10014/61C3AED7" Ref="U15"  Part="3"
 AR Path="/61BEC565/61E1083C/61C3AED7" Ref="U?"  Part="3"
-F 0 "U19" H 3800 1700 50  0000 L CNN
+F 0 "U15" H 3800 1700 50  0000 L CNN
 F 1 "LM358" H 3700 1600 50  0000 L CNN
 F 2 "Package_SO:SO-8_3.9x4.9mm_P1.27mm" H 4100 1650 50  0001 C CNN
@@
 AR Path="/61BEC565/61E10014/61C732C6" Ref="R28"  Part="1"
 AR Path="/61BEC565/61E1083C/61C732C6" Ref="R?"  Part="1"
-F 0 "R42" V 4850 2150 50  0000 C CNN
+F 0 "R28" V 4850 2150 50  0000 C CNN
 F 1 "7.5K" V 4750 2150 50  0000 C CNN
 F 2 "Resistor_SMD:R_0805_2012Metric" V 4680 2150 50  0001 C CNN
@@
 AR Path="/61BEC565/61E10014/61C738CF" Ref="R27"  Part="1"
 AR Path="/61BEC565/61E1083C/61C738CF" Ref="R?"  Part="1"
-F 0 "R41" H 4500 2300 50  0000 L CNN
+F 0 "R27" H 4500 2300 50  0000 L CNN
 F 1 "1K" V 4450 2300 50  0000 C CNN
 F 2 "Resistor_SMD:R_0805_2012Metric" V 4380 2300 50  0001 C CNN
@@
 AR Path="/61BEC565/61E10014/61C7C0FE" Ref="#PWR051"  Part="1"
 AR Path="/61BEC565/61E1083C/61C7C0FE" Ref="#PWR?"  Part="1"
-F 0 "#PWR055" H 5050 2300 50  0001 C CNN
+F 0 "#PWR051" H 5050 2300 50  0001 C CNN
 F 1 "GND" H 5055 2377 50  0000 C CNN
 F 2 "" H 5050 2550 50  0001 C CNN
@@
 AR Path="/61BEC565/61E10014/61C7D2EA" Ref="C22"  Part="1"
 AR Path="/61BEC565/61E1083C/61C7D2EA" Ref="C?"  Part="1"
-F 0 "C25" H 6115 1546 50  0000 L CNN
+F 0 "C22" H 6115 1546 50  0000 L CNN
 F 1 "10uF" H 6115 1455 50  0000 L CNN
 F 2 "Capacitor_SMD:C_0805_2012Metric" H 6038 1350 50  0001 C CNN
@@
 AR Path="/61BEC565/61E10014/61C10EDC" Ref="R23"  Part="1"
 AR Path="/61BEC565/61E1083C/61C10EDC" Ref="R?"  Part="1"
-F 0 "R37" H 1950 1350 50  0000 L CNN
+F 0 "R23" H 1950 1350 50  0000 L CNN
 F 1 "5K" V 1900 1350 50  0000 C CNN
 F 2 "Resistor_SMD:R_0805_2012Metric" V 1830 1350 50  0001 C CNN
@@
 AR Path="/61BEC565/61E10014/61C105A2" Ref="#PWR049"  Part="1"
 AR Path="/61BEC565/61E1083C/61C105A2" Ref="#PWR?"  Part="1"
-F 0 "#PWR053" H 1500 1250 50  0001 C CNN
+F 0 "#PWR049" H 1500 1250 50  0001 C CNN
 F 1 "GND" H 1505 1327 50  0000 C CNN
 F 2 "" H 1500 1500 50  0001 C CNN
@@
 AR Path="/61BEC565/61E10014/61C0AC32" Ref="U13"  Part="1"
 AR Path="/61BEC565/61E1083C/61C0AC32" Ref="U?"  Part="1"
-F 0 "U17" H 1944 1246 50  0000 L CNN
+F 0 "U13" H 1944 1246 50  0000 L CNN
 F 1 "LT6106" H 1944 1155 50  0000 L CNN
 F 2 "Package_TO_SOT_SMD:SOT-23-5" H 1600 1200 50  0001 C CNN
@@
 AR Path="/61BEC565/61E10014/61BF13FC" Ref="R26"  Part="1"
 AR Path="/61BEC565/61E1083C/61BF13FC" Ref="R?"  Part="1"
-F 0 "R40" H 3200 2200 50  0000 L CNN
+F 0 "R26" H 3200 2200 50  0000 L CNN
 F 1 "100K" V 3150 2100 50  0000 L CNN
 F 2 "Resistor_SMD:R_0805_2012Metric" V 3080 2200 50  0001 C CNN
@@
 AR Path="/61BEC565/61E10014/61BF0C42" Ref="R25"  Part="1"
 AR Path="/61BEC565/61E1083C/61BF0C42" Ref="R?"  Part="1"
-F 0 "R39" H 3200 1600 50  0000 L CNN
+F 0 "R25" H 3200 1600 50  0000 L CNN
 F 1 "750K" V 3150 1500 50  0000 L CNN
 F 2 "Resistor_SMD:R_0805_2012Metric" V 3080 1600 50  0001 C CNN
@@
 AR Path="/61BEC565/61E10014/61D167BB" Ref="R22"  Part="1"
 AR Path="/61BEC565/61E1083C/61D167BB" Ref="R?"  Part="1"
-F 0 "R36" V 1000 1900 50  0000 C CNN
+F 0 "R22" V 1000 1900 50  0000 C CNN
 F 1 "10m" V 1100 1900 50  0000 C CNN
 F 2 "Resistor_SMD:R_1206_3216Metric" V 1030 1900 50  0001 C CNN
@@
 AR Path="/61BEC565/61E10014/61D167C5" Ref="R20"  Part="1"
 AR Path="/61BEC565/61E1083C/61D167C5" Ref="R?"  Part="1"
-F 0 "R34" H 950 2300 50  0000 L CNN
+F 0 "R20" H 950 2300 50  0000 L CNN
 F 1 "50R" V 900 2300 50  0000 C CNN
 F 2 "Resistor_SMD:R_0805_2012Metric" V 830 2300 50  0001 C CNN
@@
 AR Path="/61BEC565/61E10014/61D167D4" Ref="R24"  Part="1"
 AR Path="/61BEC565/61E1083C/61D167D4" Ref="R?"  Part="1"
-F 0 "R38" H 2000 2500 50  0000 L CNN
+F 0 "R24" H 2000 2500 50  0000 L CNN
 F 1 "5K" V 1950 2500 50  0000 C CNN
 F 2 "Resistor_SMD:R_0805_2012Metric" V 1880 2500 50  0001 C CNN
@@
 AR Path="/61BEC565/61E10014/61D167DA" Ref="#PWR050"  Part="1"
 AR Path="/61BEC565/61E1083C/61D167DA" Ref="#PWR?"  Part="1"
-F 0 "#PWR054" H 1550 2400 50  0001 C CNN
+F 0 "#PWR050" H 1550 2400 50  0001 C CNN
 F 1 "GND" H 1555 2477 50  0000 C CNN
 F 2 "" H 1550 2650 50  0001 C CNN
@@
 AR Path="/61BEC565/61E10014/61D167E0" Ref="U14"  Part="1"
 AR Path="/61BEC565/61E1083C/61D167E0" Ref="U?"  Part="1"
-F 0 "U18" H 1994 2396 50  0000 L CNN
+F 0 "U14" H 1994 2396 50  0000 L CNN
 F 1 "LT6106" H 1994 2305 50  0000 L CNN
 F 2 "Package_TO_SOT_SMD:SOT-23-5" H 1650 2350 50  0001 C CNN
@@
 AR Path="/61BEC565/61E10014/61D5E781" Ref="R29"  Part="1"
 AR Path="/61BEC565/61E1083C/61D5E781" Ref="R?"  Part="1"
-F 0 "R43" V 7500 2250 50  0000 C CNN
+F 0 "R29" V 7500 2250 50  0000 C CNN
 F 1 "52.8K" V 7600 2250 50  0000 C CNN
 F 2 "Resistor_SMD:R_0805_2012Metric" V 7530 2250 50  0001 C CNN
@@
 AR Path="/61BEC565/61E10014/61D6D602" Ref="R31"  Part="1"
 AR Path="/61BEC565/61E1083C/61D6D602" Ref="R?"  Part="1"
-F 0 "R45" H 7750 2400 50  0000 R CNN
+F 0 "R31" H 7750 2400 50  0000 R CNN
 F 1 "330K" V 7800 2400 50  0000 C CNN
 F 2 "Resistor_SMD:R_0805_2012Metric" V 7730 2400 50  0001 C CNN
@@
 AR Path="/61BEC565/61E10014/61D73998" Ref="R30"  Part="1"
 AR Path="/61BEC565/61E1083C/61D73998" Ref="R?"  Part="1"
-F 0 "R44" H 7750 2100 50  0000 R CNN
+F 0 "R30" H 7750 2100 50  0000 R CNN
 F 1 "490K" V 7800 2100 50  0000 C CNN
 F 2 "Resistor_SMD:R_0805_2012Metric" V 7730 2100 50  0001 C CNN
@@
 AR Path="/61BEC565/61E10014/61D9F858" Ref="D14"  Part="1"
 AR Path="/61BEC565/61E1083C/61D9F858" Ref="D?"  Part="1"
-F 0 "D16" H 7950 1967 50  0000 C CNN
+F 0 "D14" H 7950 1967 50  0000 C CNN
 F 1 "RB051MM-2Y" H 7950 1876 50  0000 C CNN
 F 2 "Diode_SMD:D_SOD-123F" H 7950 1750 50  0001 C CNN
@@
 AR Path="/61BEC565/61E10014/61DA5795" Ref="C23"  Part="1"
 AR Path="/61BEC565/61E1083C/61DA5795" Ref="C?"  Part="1"
-F 0 "C26" H 7550 1700 50  0000 L CNN
+F 0 "C23" H 7550 1700 50  0000 L CNN
 F 1 "1uF" H 7550 1500 50  0000 L CNN
 F 2 "Capacitor_SMD:C_0805_2012Metric" H 7588 1450 50  0001 C CNN
@@
 AR Path="/61BEC565/61E10014/61DAD2DF" Ref="D13"  Part="1"
 AR Path="/61BEC565/61E1083C/61DAD2DF" Ref="D?"  Part="1"
-F 0 "D15" H 7700 1467 50  0000 C CNN
+F 0 "D13" H 7700 1467 50  0000 C CNN
 F 1 "CMSH3-40MA" H 7700 1376 50  0000 C CNN
 F 2 "Diode_SMD:D_SMA" H 7700 1250 50  0001 C CNN
@@
 AR Path="/61BEC565/61E10014/61DB925A" Ref="#PWR052"  Part="1"
 AR Path="/61BEC565/61E1083C/61DB925A" Ref="#PWR?"  Part="1"
-F 0 "#PWR056" H 7850 1000 50  0001 C CNN
+F 0 "#PWR052" H 7850 1000 50  0001 C CNN
 F 1 "GND" H 7855 1077 50  0000 C CNN
 F 2 "" H 7850 1250 50  0001 C CNN
@@
 AR Path="/61BEC565/61E10014/61DBC37B" Ref="L1"  Part="1"
 AR Path="/61BEC565/61E1083C/61DBC37B" Ref="L?"  Part="1"
-F 0 "L2" H 8303 1696 50  0000 L CNN
+F 0 "L1" H 8303 1696 50  0000 L CNN
 F 1 "22uH" H 8300 1600 50  0000 L CNN
 F 2 "Inductor_SMD:L_Bourns_SRP7028A_7.3x6.6mm" H 8250 1650 50  0001 C CNN
@@
 AR Path="/61BEC565/61E10014/61DC7062" Ref="R32"  Part="1"
 AR Path="/61BEC565/61E1083C/61DC7062" Ref="R?"  Part="1"
-F 0 "R46" V 8350 2000 50  0000 C CNN
+F 0 "R32" V 8350 2000 50  0000 C CNN
 F 1 "50m" V 8450 1850 50  0000 C CNN
 F 2 "Resistor_SMD:R_2512_6332Metric" V 8380 1850 50  0001 C CNN
@@
 AR Path="/61BEC565/61E10014/61DD561E" Ref="C24"  Part="1"
 AR Path="/61BEC565/61E1083C/61DD561E" Ref="C?"  Part="1"
-F 0 "C27" H 8365 2146 50  0000 L CNN
+F 0 "C24" H 8365 2146 50  0000 L CNN
 F 1 "10uF" H 8365 2055 50  0000 L CNN
 F 2 "Capacitor_SMD:C_0805_2012Metric" H 8288 1950 50  0001 C CNN

Commit message: Replace EVERY LT6106 with INA180A3
Friendship ended with LT6106
now ina180 is my best friend
Parts:
- removed R33, R34: 50R, Resistor_SMD:R_0805_2012Metric, symbol Device:R
- removed R35, R36: 10m, Resistor_SMD:R_1206_3216Metric, symbol Device:R
- removed R37, R38: 5K, Resistor_SMD:R_0805_2012Metric, symbol Device:R
- removed U17, U18: LT6106, Package_TO_SOT_SMD:SOT-23-5, symbol Amplifier_Current:LT6106
- added C23, C24: 0.1uF, Capacitor_SMD:C_0603_1608Metric, symbol Device:C
- added R17, R28: 4m, Resistor_SMD:R_1206_3216Metric, symbol Device:R
- added U13, U14: INA180A3, Package_TO_SOT_SMD:SOT-23-5, symbol Amplifier_Current:INA138
- renumbered C25 to C30, C26 to C31, C27 to C32, R39 to R29, R40 to R30, R41 to R31, R42 to R32, R43 to R33, R44 to R34, R45 to R35, R46 to R36
Connections:
- net A_PWR: now also R17.2, U13.3 (+)
- net B_PWR: now also R28.2, U14.3 (+)
- net GND: now also C23.2, C24.2, U13.2 (GND), U14.2 (GND)
- net TELEM_I_A: now also U13.1
- net TELEM_I_B: now also U14.1
- net at C30.1, R29.1, U19.5 (+)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: now also R17.1, R28.1, U13.4 (-), U14.4 (-)
- new net +3.3VA: C23.1, C24.1, U13.5 (V+), U14.5 (V+)
Other:
- note added: "100V/V Gain\n400mV/A"
- note removed: "Gain = Rout/Rin = 100\n1V/A"

Commit message: correct setpoint circuitry
Parts:
- R31: value 1K -> 10K
- R32: value 7.5K -> 75K
Connections:
- net +3.3VA: now also U19.8 (V+)
- net TELEM_VIN: now also U19.1, U19.2 (-); no longer R29.2, R30.1
- net Vset: now also U19.6 (-); no longer U19.3 (+)
- net at C30.1, R17.1, R28.1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: now also R32.1; no longer U19.5 (+), U19.8 (V+)
- net at R31.1, R32.2: now also U19.5 (+); no longer U19.2 (-)
- new net: R29.2, R30.1, U19.3 (+)
Other:
- moved on the sheet: R31, R32, U19A, U19B, U19C
Changed lines of the file:
@@
 L Amplifier_Operational:LM358 U19
 U 1 1 61C384AF
-P 4750 1850
+P 3750 2000
 AR Path="/61BEC565/61BEC848/61C384AF" Ref="U19"  Part="1"
 AR Path="/61BEC565/61BFB023/61C384AF" Ref="U?"  Part="1"
@@
 AR Path="/61BEC565/61E10014/61C384AF" Ref="U15"  Part="1"
 AR Path="/61BEC565/61E1083C/61C384AF" Ref="U?"  Part="1"
-F 0 "U19" H 4750 2217 50  0000 C CNN
-F 1 "LM358" H 4750 2126 50  0000 C CNN
-F 2 "Package_SO:SO-8_3.9x4.9mm_P1.27mm" H 4750 1850 50  0001 C CNN
-F 3 "http://www.ti.com/lit/ds/symlink/lm2904-n.pdf" H 4750 1850 50  0001 C CNN
-	1    4750 1850
+F 0 "U19" H 3750 2367 50  0000 C CNN
+F 1 "LM358" H 3750 2276 50  0000 C CNN
+F 2 "Package_SO:SO-8_3.9x4.9mm_P1.27mm" H 3750 2000 50  0001 C CNN
+F 3 "http://www.ti.com/lit/ds/symlink/lm2904-n.pdf" H 3750 2000 50  0001 C CNN
+	1    3750 2000
 	1    0    0    -1
 $EndComp
@@
 L Amplifier_Operational:LM358 U19
 U 2 1 61C39A83
-P 5500 1750
+P 5450 1850
 AR Path="/61BEC565/61BEC848/61C39A83" Ref="U19"  Part="2"
 AR Path="/61BEC565/61BFB023/61C39A83" Ref="U?"  Part="2"
@@
 AR Path="/61BEC565/61E10014/61C39A83" Ref="U15"  Part="2"
 AR Path="/61BEC565/61E1083C/61C39A83" Ref="U?"  Part="2"
-F 0 "U19" H 5500 2117 50  0000 C CNN
-F 1 "LM358" H 5500 2026 50  0000 C CNN
-F 2 "Package_SO:SO-8_3.9x4.9mm_P1.27mm" H 5500 1750 50  0001 C CNN
-F 3 "http://www.ti.com/lit/ds/symlink/lm2904-n.pdf" H 5500 1750 50  0001 C CNN
-	2    5500 1750
+F 0 "U19" H 5450 2217 50  0000 C CNN
+F 1 "LM358" H 5450 2126 50  0000 C CNN
+F 2 "Package_SO:SO-8_3.9x4.9mm_P1.27mm" H 5450 1850 50  0001 C CNN
+F 3 "http://www.ti.com/lit/ds/symlink/lm2904-n.pdf" H 5450 1850 50  0001 C CNN
+	2    5450 1850
 	1    0    0    -1
 $EndComp
@@
 L Amplifier_Operational:LM358 U19
 U 3 1 61C3AED7
-P 4100 1650
+P 4750 2250
 AR Path="/61BEC565/61BEC848/61C3AED7" Ref="U19"  Part="3"
 AR Path="/61BEC565/61BFB023/61C3AED7" Ref="U?"  Part="3"
@@
 AR Path="/61BEC565/61E10014/61C3AED7" Ref="U15"  Part="3"
 AR Path="/61BEC565/61E1083C/61C3AED7" Ref="U?"  Part="3"
-F 0 "U19" H 3800 1700 50  0000 L CNN
-F 1 "LM358" H 3700 1600 50  0000 L CNN
-F 2 "Package_SO:SO-8_3.9x4.9mm_P1.27mm" H 4100 1650 50  0001 C CNN
-F 3 "http://www.ti.com/lit/ds/symlink/lm2904-n.pdf" H 4100 1650 50  0001 C CNN
-	3    4100 1650
+F 0 "U19" H 4450 2300 50  0000 L CNN
+F 1 "LM358" H 4350 2200 50  0000 L CNN
+F 2 "Package_SO:SO-8_3.9x4.9mm_P1.27mm" H 4750 2250 50  0001 C CNN
+F 3 "http://www.ti.com/lit/ds/symlink/lm2904-n.pdf" H 4750 2250 50  0001 C CNN
+	3    4750 2250
 	1    0    0    -1
 $EndComp
 Text HLabel 900  750  0    50   Input ~ 0
 A_PWR
-Wire Wire Line
-	5050 1850 5200 1850
-Wire Wire Line
-	5200 1650 5200 1350
-Wire Wire Line
-	4000 1350 5200 1350
-Wire Wire Line
-	4450 1750 4350 1750
-Text HLabel 4350 1750 0    50   Input ~ 0
+Text HLabel 5000 1950 0    50   Input ~ 0
 Vset
 $Comp
 L Device:R R32
 U 1 1 61C732C6
-P 4750 2150
+P 5050 1550
 AR Path="/61BEC565/61BEC848/61C732C6" Ref="R32"  Part="1"
 AR Path="/61BEC565/61BFB023/61C732C6" Ref="R?"  Part="1"
@@
 AR Path="/61BEC565/61E10014/61C732C6" Ref="R22"  Part="1"
 AR Path="/61BEC565/61E1083C/61C732C6" Ref="R?"  Part="1"
-F 0 "R32" V 4850 2150 50  0000 C CNN
-F 1 "7.5K" V 4750 2150 50  0000 C CNN
-F 2 "Resistor_SMD:R_0805_2012Metric" V 4680 2150 50  0001 C CNN
-F 3 "~" H 4750 2150 50  0001 C CNN
-	1    4750 2150
-	0    1    1    0
+F 0 "R32" H 5100 1550 50  0000 L CNN
+F 1 "75K" V 5050 1550 50  0000 C CNN
+F 2 "Resistor_SMD:R_0805_2012Metric" V 4980 1550 50  0001 C CNN
+F 3 "~" H 5050 1550 50  0001 C CNN
+	1    5050 1550
+	1    0    0    -1
 $EndComp
 $Comp
 L Device:R R31
 U 1 1 61C738CF
-P 4450 2300
+P 5050 2350
 AR Path="/61BEC565/61BEC848/61C738CF" Ref="R31"  Part="1"
 AR Path="/61BEC565/61BFB023/61C738CF" Ref="R?"  Part="1"
@@
 AR Path="/61BEC565/61E10014/61C738CF" Ref="R21"  Part="1"
 AR Path="/61BEC565/61E1083C/61C738CF" Ref="R?"  Part="1"
-F 0 "R31" H 4500 2300 50  0000 L CNN
-F 1 "1K" V 4450 2300 50  0000 C CNN
-F 2 "Resistor_SMD:R_0805_2012Metric" V 4380 2300 50  0001 C CNN
-F 3 "~" H 4450 2300 50  0001 C CNN
-	1    4450 2300
-	1    0    0    -1
-$EndComp
-Wire Wire Line
-	5050 2150 5050 1850
-Wire Wire Line
-	4900 2150 5050 2150
-Connection ~ 5050 1850
-Wire Wire Line
-	4600 2150 4450 2150
-Wire Wire Line
-	4450 2150 4450 1950
-Connection ~ 4450 2150
+F 0 "R31" H 5100 2350 50  0000 L CNN
+F 1 "10K" V 5050 2350 50  0000 C CNN
+F 2 "Resistor_SMD:R_0805_2012Metric" V 4980 2350 50  0001 C CNN
+F 3 "~" H 5050 2350 50  0001 C CNN
+	1    5050 2350
+	1    0    0    -1
+$EndComp
 $Comp
 L power:GND #PWR065
@@
 Text HLabel 2300 1250 2    50   Input ~ 0
 TELEM_I_A
-Text HLabel 3400 1900 2    50   Input ~ 0
+Text HLabel 4050 2000 2    50   Input ~ 0
 TELEM_VIN
 $Comp
@@
 Wire Wire Line
 	3150 1750 3150 1900
-Wire Wire Line
-	3150 1900 3400 1900
 Connection ~ 3150 1900
 Wire Wire Line
@@
 Wire Wire Line
 	3150 1450 3150 1350
-Wire Wire Line
-	3150 1350 4000 1350
-Connection ~ 4000 1350
 Text HLabel 900  1800 0    50   Input ~ 0
 B_PWR
@@
 Text Notes 3100 600  0    50   ~ 0
 Input Voltage Telemetry and Vmp Setpoint
-Wire Wire Line
-	5200 1350 6000 1350
-Connection ~ 5200 1350
-Wire Wire Line
-	5800 1750 6400 1750
 $Comp
 L Device:R R33
@@
 Connection ~ 5050 2550
 Wire Wire Line
-	5050 2550 4450 2550
-Wire Wire Line
 	6900 2350 6900 2550
 Connection ~ 6900 2550
@@
 Wire Wire Line
 	6000 2550 5050 2550
-Wire Wire Line
-	4000 1950 4000 2550
-Connection ~ 4000 2550
-Wire Wire Line
-	4450 2450 4450 2550
-Connection ~ 4450 2550
-Wire Wire Line
-	4450 2550 4000 2550
 $Comp
 L Device:D_Schottky D16
@@
 Text Notes 8400 1500 0    50   ~ 0
 Imax = 0.1V/Rsense\nMaximum allowed is 2A\nTermination at C/10 = 0.2A
-Wire Wire Line
-	3150 2550 4000 2550
 $Comp
 L power:GND #PWR?
@@
 Wire Wire Line
 	1250 1800 2950 1800
+Wire Wire Line
+	5050 1400 5050 1350
+Connection ~ 5050 1350
+Wire Wire Line
+	5050 1350 6000 1350
+Wire Wire Line
+	5050 2500 5050 2550
+Wire Wire Line
+	5050 1700 5050 1750
+Wire Wire Line
+	5150 1750 5050 1750
+Connection ~ 5050 1750
+Wire Wire Line
+	5050 1750 5050 2200
+Wire Wire Line
+	5000 1950 5150 1950
+Wire Wire Line
+	5750 1850 6100 1850
+Wire Wire Line
+	6100 1850 6100 1750
+Wire Wire Line
+	6100 1750 6400 1750
+Wire Wire Line
+	3150 1350 5050 1350
+Wire Wire Line
+	3150 2550 4650 2550
+Wire Wire Line
+	3150 1900 3450 1900
+Wire Wire Line
+	3450 2100 3450 2300
+Wire Wire Line
+	3450 2300 4050 2300
+Wire Wire Line
+	4050 2300 4050 2000
+Connection ~ 4650 2550
+Wire Wire Line
+	4650 2550 5050 2550
+$Comp
+L power:+3.3VA #PWR?
+U 1 1 6211F03B
+P 4650 1950
+AR Path="/61BEC565/61BEC848/6211F03B" Ref="#PWR?"  Part="1"
+AR Path="/61BEC565/61E10014/6211F03B" Ref="#PWR?"  Part="1"
+F 0 "#PWR?" H 4650 1800 50  0001 C CNN
+F 1 "+3.3VA" H 4665 2123 50  0000 C CNN
+F 2 "" H 4650 1950 50  0001 C CNN
+F 3 "" H 4650 1950 50  0001 C CNN
+	1    4650 1950
+	1    0    0    -1
+$EndComp
 $EndSCHEMATC
