File: ECAD/EPS/PDM3V3.kicad_sch (KiCad schematic)
At the start: 11 parts, among them Q33 2N7002, Q34 IRF7458, U45 INA180A3

Commit message: respec and consolidate
Parts:
- renumbered C81 to C69, D25 to D26, Q33 to Q29, Q34 to Q30, R122 to R116, R123 to R117, R124 to R118, R125 to R119, R126 to R120, R127 to R121, U45 to U43
Changed lines of the file:
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@@
   (symbol (lib_id "Device:R") (at 106.68 46.99 0) (unit 1)
     (in_bom yes) (on_board yes)
-    (property "Reference" "R124" (id 0) (at 107.95 46.99 0)
+    (property "Reference" "R118" (id 0) (at 107.95 46.99 0)
       (effects (font (size 1.27 1.27)) (justify left))
     )
@@
   (symbol (lib_id "Device:R") (at 96.52 67.31 0) (unit 1)
     (in_bom yes) (on_board yes)
-    (property "Reference" "R123" (id 0) (at 97.79 67.31 0)
+    (property "Reference" "R117" (id 0) (at 97.79 67.31 0)
       (effects (font (size 1.27 1.27)) (justify left))
     )
@@
   (symbol (lib_id "power:GND") (at 118.11 80.01 0) (unit 1)
     (in_bom yes) (on_board yes)
-    (property "Reference" "#PWR0124" (id 0) (at 118.11 86.36 0)
+    (property "Reference" "#PWR0122" (id 0) (at 118.11 86.36 0)
       (effects (font (size 1.27 1.27)) hide)
     )
@@
   (symbol (lib_id "power:+3V3") (at 118.11 43.18 0) (unit 1)
     (in_bom yes) (on_board yes)
-    (property "Reference" "#PWR0123" (id 0) (at 118.11 46.99 0)
+    (property "Reference" "#PWR0121" (id 0) (at 118.11 46.99 0)
       (effects (font (size 1.27 1.27)) hide)
     )
@@
   (symbol (lib_id "Transistor_FET:IRF7404") (at 115.57 54.61 0) (unit 1)
     (in_bom yes) (on_board yes)
-    (property "Reference" "Q34" (id 0) (at 120.777 53.4416 0)
+    (property "Reference" "Q30" (id 0) (at 120.777 53.4416 0)
       (effects (font (size 1.27 1.27)) (justify left))
     )
@@
   (symbol (lib_id "Transistor_FET:2N7002") (at 104.14 63.5 0) (unit 1)
     (in_bom yes) (on_board yes)
-    (property "Reference" "Q33" (id 0) (at 109.3216 62.3316 0)
+    (property "Reference" "Q29" (id 0) (at 109.3216 62.3316 0)
       (effects (font (size 1.27 1.27)) (justify left))
     )
@@
   (symbol (lib_id "Device:D") (at 189.23 63.5 270) (unit 1)
     (in_bom yes) (on_board yes)
-    (property "Reference" "D25" (id 0) (at 191.262 62.3316 90)
+    (property "Reference" "D26" (id 0) (at 191.262 62.3316 90)
       (effects (font (size 1.27 1.27)) (justify left))
     )
@@
   (symbol (lib_id "Device:R") (at 90.17 63.5 270) (unit 1)
     (in_bom yes) (on_board yes)
-    (property "Reference" "R122" (id 0) (at 90.17 60.96 90))
+    (property "Reference" "R116" (id 0) (at 90.17 60.96 90))
     (property "Value" "100R" (id 1) (at 90.17 63.5 90))
     (property "Footprint" "Resistor_SMD:R_0603_1608Metric" (id 2) (at 90.17 61.722 90)
@@
   (symbol (lib_id "Device:R") (at 118.11 64.77 0) (unit 1)
     (in_bom yes) (on_board yes)
-    (property "Reference" "R125" (id 0) (at 119.38 64.77 0)
+    (property "Reference" "R119" (id 0) (at 119.38 64.77 0)
       (effects (font (size 1.27 1.27)) (justify left))
     )
@@
   (symbol (lib_id "Device:R") (at 118.11 74.93 0) (unit 1)
     (in_bom yes) (on_board yes)
-    (property "Reference" "R126" (id 0) (at 119.38 74.93 0)
+    (property "Reference" "R120" (id 0) (at 119.38 74.93 0)
       (effects (font (size 1.27 1.27)) (justify left))
     )
@@
   (symbol (lib_id "Device:R") (at 144.78 59.69 270) (unit 1)
     (in_bom yes) (on_board yes)
-    (property "Reference" "R127" (id 0) (at 144.78 57.15 90))
+    (property "Reference" "R121" (id 0) (at 144.78 57.15 90))
     (property "Value" "4m" (id 1) (at 144.78 59.69 90))
     (property "Footprint" "Resistor_SMD:R_1206_3216Metric" (id 2) (at 144.78 57.912 90)
@@
   (symbol (lib_id "Amplifier_Current:INA138") (at 158.75 72.39 0) (unit 1)
     (in_bom yes) (on_board yes)
-    (property "Reference" "U45" (id 0) (at 167.4876 71.2216 0)
+    (property "Reference" "U43" (id 0) (at 167.4876 71.2216 0)
       (effects (font (size 1.27 1.27)) (justify left))
     )
@@
   (symbol (lib_id "Device:C") (at 160.02 64.77 90) (unit 1)
     (in_bom yes) (on_board yes)
-    (property "Reference" "C81" (id 0) (at 161.29 60.96 90)
+    (property "Reference" "C69" (id 0) (at 161.29 60.96 90)
       (effects (font (size 1.27 1.27)) (justify right))
     )
@@
   (symbol (lib_id "power:GND") (at 163.83 64.77 0) (unit 1)
     (in_bom yes) (on_board yes)
-    (property "Reference" "#PWR0125" (id 0) (at 163.83 71.12 0)
-      (effects (font (size 1.27 1.27)) hide)
-    )
+    (property "Reference" "#PWR0123" (id 0) (at 163.83 71.12 0)
+      (effects (font (size 1.27 1.27)) hide)
+    )
