File: ECAD/EPS/PDM5V.kicad_sch (KiCad schematic)
At the start: 11 parts, among them Q41 2N7002, Q42 IRF7458, U49 INA180A3

Commit message: respec and consolidate
Parts:
- renumbered C85 to C68, D29 to D25, Q41 to Q27, Q42 to Q28, R146 to R110, R147 to R111, R148 to R112, R149 to R113, R150 to R114, R151 to R115, U49 to U42
Changed lines of the file:
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@@
   (symbol (lib_id "power:+5V") (at 118.11 43.18 0) (unit 1)
     (in_bom yes) (on_board yes)
-    (property "Reference" "#PWR0135" (id 0) (at 118.11 46.99 0)
+    (property "Reference" "#PWR0118" (id 0) (at 118.11 46.99 0)
       (effects (font (size 1.27 1.27)) hide)
     )
@@
   (symbol (lib_id "Transistor_FET:IRF7404") (at 115.57 54.61 0) (unit 1)
     (in_bom yes) (on_board yes)
-    (property "Reference" "Q42" (id 0) (at 120.777 53.4416 0)
+    (property "Reference" "Q28" (id 0) (at 120.777 53.4416 0)
       (effects (font (size 1.27 1.27)) (justify left))
     )
@@
   (symbol (lib_id "Transistor_FET:2N7002") (at 104.14 63.5 0) (unit 1)
     (in_bom yes) (on_board yes)
-    (property "Reference" "Q41" (id 0) (at 109.3216 62.3316 0)
+    (property "Reference" "Q27" (id 0) (at 109.3216 62.3316 0)
       (effects (font (size 1.27 1.27)) (justify left))
     )
@@
   (symbol (lib_id "Device:R") (at 106.68 46.99 0) (unit 1)
     (in_bom yes) (on_board yes)
-    (property "Reference" "R148" (id 0) (at 107.95 46.99 0)
+    (property "Reference" "R112" (id 0) (at 107.95 46.99 0)
       (effects (font (size 1.27 1.27)) (justify left))
     )
@@
   (symbol (lib_id "Device:D") (at 189.23 63.5 270) (unit 1)
     (in_bom yes) (on_board yes)
-    (property "Reference" "D29" (id 0) (at 191.262 62.3316 90)
+    (property "Reference" "D25" (id 0) (at 191.262 62.3316 90)
       (effects (font (size 1.27 1.27)) (justify left))
     )
@@
   (symbol (lib_id "Device:R") (at 90.17 63.5 270) (unit 1)
     (in_bom yes) (on_board yes)
-    (property "Reference" "R146" (id 0) (at 90.17 60.96 90))
+    (property "Reference" "R110" (id 0) (at 90.17 60.96 90))
     (property "Value" "100R" (id 1) (at 90.17 63.5 90))
     (property "Footprint" "Resistor_SMD:R_0603_1608Metric" (id 2) (at 90.17 61.722 90)
@@
   (symbol (lib_id "Device:R") (at 96.52 67.31 0) (unit 1)
     (in_bom yes) (on_board yes)
-    (property "Reference" "R147" (id 0) (at 97.79 67.31 0)
+    (property "Reference" "R111" (id 0) (at 97.79 67.31 0)
       (effects (font (size 1.27 1.27)) (justify left))
     )
@@
   (symbol (lib_id "Device:R") (at 118.11 64.77 0) (unit 1)
     (in_bom yes) (on_board yes)
-    (property "Reference" "R149" (id 0) (at 119.38 64.77 0)
+    (property "Reference" "R113" (id 0) (at 119.38 64.77 0)
       (effects (font (size 1.27 1.27)) (justify left))
     )
@@
   (symbol (lib_id "Device:R") (at 118.11 74.93 0) (unit 1)
     (in_bom yes) (on_board yes)
-    (property "Reference" "R150" (id 0) (at 119.38 74.93 0)
+    (property "Reference" "R114" (id 0) (at 119.38 74.93 0)
       (effects (font (size 1.27 1.27)) (justify left))
     )
@@
   (symbol (lib_id "power:GND") (at 118.11 80.01 0) (unit 1)
     (in_bom yes) (on_board yes)
-    (property "Reference" "#PWR0136" (id 0) (at 118.11 86.36 0)
+    (property "Reference" "#PWR0119" (id 0) (at 118.11 86.36 0)
       (effects (font (size 1.27 1.27)) hide)
     )
@@
   (symbol (lib_id "Device:R") (at 144.78 59.69 270) (unit 1)
     (in_bom yes) (on_board yes)
-    (property "Reference" "R151" (id 0) (at 144.78 57.15 90))
+    (property "Reference" "R115" (id 0) (at 144.78 57.15 90))
     (property "Value" "4m" (id 1) (at 144.78 59.69 90))
     (property "Footprint" "Resistor_SMD:R_1206_3216Metric" (id 2) (at 144.78 57.912 90)
@@
   (symbol (lib_id "Amplifier_Current:INA138") (at 158.75 72.39 0) (unit 1)
     (in_bom yes) (on_board yes)
-    (property "Reference" "U49" (id 0) (at 167.4876 71.2216 0)
+    (property "Reference" "U42" (id 0) (at 167.4876 71.2216 0)
       (effects (font (size 1.27 1.27)) (justify left))
     )
@@
   (symbol (lib_id "Device:C") (at 160.02 64.77 90) (unit 1)
     (in_bom yes) (on_board yes)
-    (property "Reference" "C85" (id 0) (at 161.29 60.96 90)
+    (property "Reference" "C68" (id 0) (at 161.29 60.96 90)
       (effects (font (size 1.27 1.27)) (justify right))
     )
@@
   (symbol (lib_id "power:GND") (at 163.83 64.77 0) (unit 1)
     (in_bom yes) (on_board yes)
-    (property "Reference" "#PWR0137" (id 0) (at 163.83 71.12 0)
-      (effects (font (size 1.27 1.27)) hide)
-    )
+    (property "Reference" "#PWR0120" (id 0) (at 163.83 71.12 0)
+      (effects (font (size 1.27 1.27)) hide)
+    )
