File: ECAD/EPS/PDMBATV.kicad_sch (KiCad schematic)
At the start: 11 parts, among them Q47 2N7002, Q48 IRF7458, U52 INA180A3

Commit message: respec and consolidate
Parts:
- renumbered C88 to C67, D32 to D24, Q47 to Q25, Q48 to Q26, R164 to R104, R165 to R105, R166 to R106, R167 to R107, R168 to R108, R169 to R109, U52 to U41
Changed lines of the file:
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@@
   (symbol (lib_id "Device:D") (at 189.23 63.5 270) (unit 1)
     (in_bom yes) (on_board yes)
-    (property "Reference" "D32" (id 0) (at 191.262 62.3316 90)
+    (property "Reference" "D24" (id 0) (at 191.262 62.3316 90)
       (effects (font (size 1.27 1.27)) (justify left))
     )
@@
   (symbol (lib_id "Device:R") (at 118.11 64.77 0) (unit 1)
     (in_bom yes) (on_board yes)
-    (property "Reference" "R167" (id 0) (at 119.38 64.77 0)
+    (property "Reference" "R107" (id 0) (at 119.38 64.77 0)
       (effects (font (size 1.27 1.27)) (justify left))
     )
@@
   (symbol (lib_id "power:+BATT") (at 118.11 43.18 0) (unit 1)
     (in_bom yes) (on_board yes)
-    (property "Reference" "#PWR0146" (id 0) (at 118.11 46.99 0)
+    (property "Reference" "#PWR0114" (id 0) (at 118.11 46.99 0)
       (effects (font (size 1.27 1.27)) hide)
     )
@@
   (symbol (lib_id "Transistor_FET:IRF7404") (at 115.57 54.61 0) (unit 1)
     (in_bom yes) (on_board yes)
-    (property "Reference" "Q48" (id 0) (at 120.777 53.4416 0)
+    (property "Reference" "Q26" (id 0) (at 120.777 53.4416 0)
       (effects (font (size 1.27 1.27)) (justify left))
     )
@@
   (symbol (lib_id "Transistor_FET:2N7002") (at 104.14 63.5 0) (unit 1)
     (in_bom yes) (on_board yes)
-    (property "Reference" "Q47" (id 0) (at 109.3216 62.3316 0)
+    (property "Reference" "Q25" (id 0) (at 109.3216 62.3316 0)
       (effects (font (size 1.27 1.27)) (justify left))
     )
@@
   (symbol (lib_id "Device:R") (at 106.68 46.99 0) (unit 1)
     (in_bom yes) (on_board yes)
-    (property "Reference" "R166" (id 0) (at 107.95 46.99 0)
+    (property "Reference" "R106" (id 0) (at 107.95 46.99 0)
       (effects (font (size 1.27 1.27)) (justify left))
     )
@@
   (symbol (lib_id "Device:R") (at 90.17 63.5 270) (unit 1)
     (in_bom yes) (on_board yes)
-    (property "Reference" "R164" (id 0) (at 90.17 60.96 90))
+    (property "Reference" "R104" (id 0) (at 90.17 60.96 90))
     (property "Value" "100R" (id 1) (at 90.17 63.5 90))
     (property "Footprint" "Resistor_SMD:R_0603_1608Metric" (id 2) (at 90.17 61.722 90)
@@
   (symbol (lib_id "Device:R") (at 96.52 67.31 0) (unit 1)
     (in_bom yes) (on_board yes)
-    (property "Reference" "R165" (id 0) (at 97.79 67.31 0)
+    (property "Reference" "R105" (id 0) (at 97.79 67.31 0)
       (effects (font (size 1.27 1.27)) (justify left))
     )
@@
   (symbol (lib_id "power:GND") (at 118.11 80.01 0) (unit 1)
     (in_bom yes) (on_board yes)
-    (property "Reference" "#PWR0147" (id 0) (at 118.11 86.36 0)
+    (property "Reference" "#PWR0115" (id 0) (at 118.11 86.36 0)
       (effects (font (size 1.27 1.27)) hide)
     )
@@
   (symbol (lib_id "Device:R") (at 144.78 59.69 270) (unit 1)
     (in_bom yes) (on_board yes)
-    (property "Reference" "R169" (id 0) (at 144.78 57.15 90))
+    (property "Reference" "R109" (id 0) (at 144.78 57.15 90))
     (property "Value" "4m" (id 1) (at 144.78 59.69 90))
     (property "Footprint" "Resistor_SMD:R_1206_3216Metric" (id 2) (at 144.78 57.912 90)
@@
   (symbol (lib_id "Device:R") (at 118.11 74.93 0) (unit 1)
     (in_bom yes) (on_board yes)
-    (property "Reference" "R168" (id 0) (at 119.38 74.93 0)
+    (property "Reference" "R108" (id 0) (at 119.38 74.93 0)
       (effects (font (size 1.27 1.27)) (justify left))
     )
@@
   (symbol (lib_id "Amplifier_Current:INA138") (at 158.75 72.39 0) (unit 1)
     (in_bom yes) (on_board yes)
-    (property "Reference" "U52" (id 0) (at 167.4876 71.2216 0)
+    (property "Reference" "U41" (id 0) (at 167.4876 71.2216 0)
       (effects (font (size 1.27 1.27)) (justify left))
     )
@@
   (symbol (lib_id "power:VCC") (at 156.21 64.77 0) (unit 1)
     (in_bom yes) (on_board yes)
-    (property "Reference" "#PWR0148" (id 0) (at 156.21 68.58 0)
+    (property "Reference" "#PWR0116" (id 0) (at 156.21 68.58 0)
       (effects (font (size 1.27 1.27)) hide)
     )
@@
   (symbol (lib_id "Device:C") (at 160.02 64.77 90) (unit 1)
     (in_bom yes) (on_board yes)
-    (property "Reference" "C88" (id 0) (at 161.29 60.96 90)
+    (property "Reference" "C67" (id 0) (at 161.29 60.96 90)
       (effects (font (size 1.27 1.27)) (justify right))
     )
@@
   (symbol (lib_id "power:GND") (at 163.83 64.77 0) (unit 1)
     (in_bom yes) (on_board yes)
-    (property "Reference" "#PWR0149" (id 0) (at 163.83 71.12 0)
-      (effects (font (size 1.27 1.27)) hide)
-    )
+    (property "Reference" "#PWR0117" (id 0) (at 163.83 71.12 0)
+      (effects (font (size 1.27 1.27)) hide)
+    )
