File: ECAD/EPS/PowerDistribution.kicad_sch (KiCad schematic)
At the start: 5 parts, among them U40 74HC595, U41 74HC595

Commit message: respec and consolidate
Parts:
- renumbered C76 to C65, C77 to C66, U40 to U39, U41 to U40
Changed lines of the file:
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@@
   (symbol (lib_id "Device:C") (at 142.24 107.95 0) (unit 1)
     (in_bom yes) (on_board yes)
-    (property "Reference" "C77" (id 0) (at 145.161 106.7816 0)
+    (property "Reference" "C66" (id 0) (at 145.161 106.7816 0)
       (effects (font (size 1.27 1.27)) (justify left))
     )
@@
   (symbol (lib_id "Device:C") (at 92.71 107.95 0) (unit 1)
     (in_bom yes) (on_board yes)
-    (property "Reference" "C76" (id 0) (at 95.25 106.68 0)
+    (property "Reference" "C65" (id 0) (at 95.25 106.68 0)
       (effects (font (size 1.27 1.27)) (justify left))
     )
@@
   (symbol (lib_id "power:VDD") (at 142.24 104.14 0) (unit 1)
     (in_bom yes) (on_board yes)
-    (property "Reference" "#PWR0155" (id 0) (at 142.24 107.95 0)
+    (property "Reference" "#PWR0112" (id 0) (at 142.24 107.95 0)
       (effects (font (size 1.27 1.27)) hide)
     )
@@
   (symbol (lib_id "74xx:74HC595") (at 118.11 119.38 0) (unit 1)
     (in_bom yes) (on_board yes)
-    (property "Reference" "U40" (id 0) (at 118.11 99.5426 0))
+    (property "Reference" "U39" (id 0) (at 118.11 99.5426 0))
     (property "Value" "74HC595" (id 1) (at 118.11 101.854 0))
     (property "Footprint" "Package_SO:SOIC-16_3.9x9.9mm_P1.27mm" (id 2) (at 118.11 119.38 0)
@@
   (symbol (lib_id "74xx:74HC595") (at 166.37 119.38 0) (unit 1)
     (in_bom yes) (on_board yes)
-    (property "Reference" "U41" (id 0) (at 166.37 99.5426 0))
+    (property "Reference" "U40" (id 0) (at 166.37 99.5426 0))
     (property "Value" "74HC595" (id 1) (at 166.37 101.854 0))
     (property "Footprint" "Package_SO:SOIC-16_3.9x9.9mm_P1.27mm" (id 2) (at 166.37 119.38 0)
