File: ECAD/EPS/Boost-BuckMPPT.kicad_sch (KiCad schematic)
At the start: 34 parts, among them Q6 Si4186DY, U21 LM358, U22 INA180A3, U23 INA180A3, U24 LT3652EMSE, U25 LMC555xM, U57 MCP14A0902-E/SN

Commit message: layout and footprints
Parts:
- renumbered C33 to C37, C34 to C38, C35 to C39, C36 to C40, C37 to C41, C38 to C42, C39 to C43, C40 to C44, C41 to C45, C42 to C46, Q6 to Q4, R37 to R33, R38 to R34, R39 to R35, R40 to R36, R41 to R37, R42 to R38, R43 to R39, R44 to R40, R45 to R41, R46 to R42, R47 to R43, R48 to R44, U57 to U26
Changed lines of the file:
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@@
   (symbol (lib_id "Device:R") (at 148.59 39.37 90) (unit 1)
     (in_bom yes) (on_board yes)
-    (property "Reference" "R48" (id 0) (at 149.86 36.83 90)
+    (property "Reference" "R44" (id 0) (at 149.86 36.83 90)
       (effects (font (size 1.27 1.27)) (justify left))
     )
@@
   (symbol (lib_id "Device:C") (at 102.87 50.8 0) (unit 1)
     (in_bom yes) (on_board yes)
-    (property "Reference" "C36" (id 0) (at 105.791 49.6316 0)
+    (property "Reference" "C40" (id 0) (at 105.791 49.6316 0)
       (effects (font (size 1.27 1.27)) (justify left))
     )
@@
   (symbol (lib_id "Device:C") (at 115.57 57.15 0) (unit 1)
     (in_bom yes) (on_board yes)
-    (property "Reference" "C38" (id 0) (at 118.491 55.9816 0)
+    (property "Reference" "C42" (id 0) (at 118.491 55.9816 0)
       (effects (font (size 1.27 1.27)) (justify left))
     )
@@
   (symbol (lib_id "Device:R") (at 102.87 43.18 0) (unit 1)
     (in_bom yes) (on_board yes)
-    (property "Reference" "R43" (id 0) (at 104.14 43.18 0)
+    (property "Reference" "R39" (id 0) (at 104.14 43.18 0)
       (effects (font (size 1.27 1.27)) (justify left))
     )
@@
   (symbol (lib_id "Transistor_FET:Si4162DY") (at 181.61 46.99 0) (unit 1)
     (in_bom yes) (on_board yes)
-    (property "Reference" "Q6" (id 0) (at 186.69 45.72 0)
+    (property "Reference" "Q4" (id 0) (at 186.69 45.72 0)
       (effects (font (size 1.27 1.27)) (justify left))
     )
@@
   (symbol (lib_id "power:GND") (at 139.7 66.04 0) (unit 1)
     (in_bom yes) (on_board yes)
-    (property "Reference" "#PWR077" (id 0) (at 139.7 72.39 0)
+    (property "Reference" "#PWR073" (id 0) (at 139.7 72.39 0)
       (effects (font (size 1.27 1.27)) hide)
     )
@@
   (symbol (lib_id "Device:R") (at 50.8 101.6 0) (unit 1)
     (in_bom yes) (on_board yes)
-    (property "Reference" "R39" (id 0) (at 52.07 101.6 0)
+    (property "Reference" "R35" (id 0) (at 52.07 101.6 0)
       (effects (font (size 1.27 1.27)) (justify left))
     )
@@
   (symbol (lib_id "Device:R") (at 50.8 121.92 0) (unit 1)
     (in_bom yes) (on_board yes)
-    (property "Reference" "R40" (id 0) (at 52.07 121.92 0)
+    (property "Reference" "R36" (id 0) (at 52.07 121.92 0)
       (effects (font (size 1.27 1.27)) (justify left))
     )
@@
   (symbol (lib_id "power:GND") (at 50.8 127 0) (unit 1)
     (in_bom yes) (on_board yes)
-    (property "Reference" "#PWR075" (id 0) (at 50.8 133.35 0)
+    (property "Reference" "#PWR071" (id 0) (at 50.8 133.35 0)
       (effects (font (size 1.27 1.27)) hide)
     )
@@
   (symbol (lib_id "Device:C") (at 74.93 100.33 0) (unit 1)
     (in_bom yes) (on_board yes)
-    (property "Reference" "C35" (id 0) (at 77.851 99.1616 0)
+    (property "Reference" "C39" (id 0) (at 77.851 99.1616 0)
       (effects (font (size 1.27 1.27)) (justify left))
     )
@@
   (symbol (lib_id "Device:R") (at 115.57 119.38 270) (unit 1)
     (in_bom yes) (on_board yes)
-    (property "Reference" "R44" (id 0) (at 115.57 116.84 90))
+    (property "Reference" "R40" (id 0) (at 115.57 116.84 90))
     (property "Value" "52.8K" (id 1) (at 115.57 119.38 90))
     (property "Footprint" "Resistor_SMD:R_0805_2012Metric" (id 2) (at 115.57 117.602 90)
@@
   (symbol (lib_id "Device:R") (at 120.65 123.19 180) (unit 1)
     (in_bom yes) (on_board yes)
-    (property "Reference" "R46" (id 0) (at 121.92 123.19 0)
+    (property "Reference" "R42" (id 0) (at 121.92 123.19 0)
       (effects (font (size 1.27 1.27)) (justify right))
     )
@@
   (symbol (lib_id "Device:R") (at 120.65 115.57 180) (unit 1)
     (in_bom yes) (on_board yes)
-    (property "Reference" "R45" (id 0) (at 121.92 115.57 0)
+    (property "Reference" "R41" (id 0) (at 121.92 115.57 0)
       (effects (font (size 1.27 1.27)) (justify right))
     )
@@
   (symbol (lib_id "Device:C") (at 114.3 102.87 0) (unit 1)
     (in_bom yes) (on_board yes)
-    (property "Reference" "C37" (id 0) (at 114.3 100.33 0)
+    (property "Reference" "C41" (id 0) (at 114.3 100.33 0)
       (effects (font (size 1.27 1.27)) (justify left))
     )
@@
   (symbol (lib_id "power:GND") (at 121.92 93.98 0) (unit 1)
     (in_bom yes) (on_board yes)
-    (property "Reference" "#PWR076" (id 0) (at 121.92 100.33 0)
+    (property "Reference" "#PWR072" (id 0) (at 121.92 100.33 0)
       (effects (font (size 1.27 1.27)) hide)
     )
@@
   (symbol (lib_id "Device:R") (at 137.16 109.22 270) (unit 1)
     (in_bom yes) (on_board yes)
-    (property "Reference" "R47" (id 0) (at 140.97 106.68 90))
+    (property "Reference" "R43" (id 0) (at 140.97 106.68 90))
     (property "Value" "50m" (id 1) (at 137.16 109.22 90))
     (property "Footprint" "Resistor_SMD:R_2512_6332Metric" (id 2) (at 137.16 107.442 90)
@@
   (symbol (lib_id "Device:C") (at 132.08 115.57 0) (unit 1)
     (in_bom yes) (on_board yes)
-    (property "Reference" "C39" (id 0) (at 135.001 114.4016 0)
+    (property "Reference" "C43" (id 0) (at 135.001 114.4016 0)
       (effects (font (size 1.27 1.27)) (justify left))
     )
@@
   (symbol (lib_id "Device:C") (at 157.48 54.61 0) (unit 1)
     (in_bom yes) (on_board yes)
-    (property "Reference" "C40" (id 0) (at 160.401 53.4416 0)
+    (property "Reference" "C44" (id 0) (at 160.401 53.4416 0)
       (effects (font (size 1.27 1.27)) (justify left))
     )
@@
   (symbol (lib_id "Device:C") (at 200.66 46.99 0) (unit 1)
     (in_bom yes) (on_board yes)
-    (property "Reference" "C41" (id 0) (at 203.581 45.8216 0)
+    (property "Reference" "C45" (id 0) (at 203.581 45.8216 0)
       (effects (font (size 1.27 1.27)) (justify left))
     )
@@
   (symbol (lib_id "Device:C") (at 210.82 46.99 0) (unit 1)
     (in_bom yes) (on_board yes)
-    (property "Reference" "C42" (id 0) (at 213.741 45.8216 0)
+    (property "Reference" "C46" (id 0) (at 213.741 45.8216 0)
       (effects (font (size 1.27 1.27)) (justify left))
     )
@@
   (symbol (lib_id "Device:R") (at 81.28 41.91 0) (unit 1)
     (in_bom yes) (on_board yes)
-    (property "Reference" "R41" (id 0) (at 82.55 41.91 0)
+    (property "Reference" "R37" (id 0) (at 82.55 41.91 0)
       (effects (font (size 1.27 1.27)) (justify left))
     )
@@
   (symbol (lib_id "Device:R") (at 81.28 57.15 0) (unit 1)
     (in_bom yes) (on_board yes)
-    (property "Reference" "R42" (id 0) (at 82.55 57.15 0)
+    (property "Reference" "R38" (id 0) (at 82.55 57.15 0)
       (effects (font (size 1.27 1.27)) (justify left))
     )
@@
   (symbol (lib_id "power:GND") (at 40.64 40.64 0) (unit 1)
     (in_bom yes) (on_board yes)
-    (property "Reference" "#PWR070" (id 0) (at 40.64 46.99 0)
+    (property "Reference" "#PWR066" (id 0) (at 40.64 46.99 0)
       (effects (font (size 1.27 1.27)) hide)
     )
@@
   (symbol (lib_id "Device:R") (at 29.21 20.32 270) (unit 1)
     (in_bom yes) (on_board yes)
-    (property "Reference" "R37" (id 0) (at 29.21 17.78 90))
+    (property "Reference" "R33" (id 0) (at 29.21 17.78 90))
     (property "Value" "4m" (id 1) (at 29.21 20.32 90))
     (property "Footprint" "Resistor_SMD:R_1206_3216Metric" (id 2) (at 29.21 18.542 90)
@@
   (symbol (lib_id "Device:C") (at 44.45 25.4 90) (unit 1)
     (in_bom yes) (on_board yes)
-    (property "Reference" "C33" (id 0) (at 45.72 21.59 90)
+    (property "Reference" "C37" (id 0) (at 45.72 21.59 90)
       (effects (font (size 1.27 1.27)) (justify right))
     )
@@
   (symbol (lib_id "power:GND") (at 48.26 25.4 0) (unit 1)
     (in_bom yes) (on_board yes)
-    (property "Reference" "#PWR073" (id 0) (at 48.26 31.75 0)
+    (property "Reference" "#PWR069" (id 0) (at 48.26 31.75 0)
       (effects (font (size 1.27 1.27)) hide)
     )
@@
   (symbol (lib_id "power:+3.3VA") (at 40.64 25.4 0) (unit 1)
     (in_bom yes) (on_board yes)
-    (property "Reference" "#PWR069" (id 0) (at 40.64 29.21 0)
+    (property "Reference" "#PWR065" (id 0) (at 40.64 29.21 0)
       (effects (font (size 1.27 1.27)) hide)
     )
@@
   (symbol (lib_id "power:GND") (at 40.64 67.31 0) (unit 1)
     (in_bom yes) (on_board yes)
-    (property "Reference" "#PWR072" (id 0) (at 40.64 73.66 0)
+    (property "Reference" "#PWR068" (id 0) (at 40.64 73.66 0)
       (effects (font (size 1.27 1.27)) hide)
     )
@@
   (symbol (lib_id "Device:R") (at 29.21 46.99 270) (unit 1)
     (in_bom yes) (on_board yes)
-    (property "Reference" "R38" (id 0) (at 29.21 44.45 90))
+    (property "Reference" "R34" (id 0) (at 29.21 44.45 90))
     (property "Value" "4m" (id 1) (at 29.21 46.99 90))
     (property "Footprint" "Resistor_SMD:R_1206_3216Metric" (id 2) (at 29.21 45.212 90)
@@
   (symbol (lib_id "Device:C") (at 44.45 52.07 90) (unit 1)
     (in_bom yes) (on_board yes)
-    (property "Reference" "C34" (id 0) (at 45.72 48.26 90)
+    (property "Reference" "C38" (id 0) (at 45.72 48.26 90)
       (effects (font (size 1.27 1.27)) (justify right))
     )
@@
   (symbol (lib_id "power:GND") (at 48.26 52.07 0) (unit 1)
     (in_bom yes) (on_board yes)
-    (property "Reference" "#PWR074" (id 0) (at 48.26 58.42 0)
+    (property "Reference" "#PWR070" (id 0) (at 48.26 58.42 0)
       (effects (font (size 1.27 1.27)) hide)
     )
@@
   (symbol (lib_id "power:+3.3VA") (at 40.64 52.07 0) (unit 1)
     (in_bom yes) (on_board yes)
-    (property "Reference" "#PWR071" (id 0) (at 40.64 55.88 0)
+    (property "Reference" "#PWR067" (id 0) (at 40.64 55.88 0)
       (effects (font (size 1.27 1.27)) hide)
     )
@@
   (symbol (lib_id "power:+3.3VA") (at 33.02 111.76 0) (unit 1)
     (in_bom yes) (on_board yes)
-    (property "Reference" "#PWR068" (id 0) (at 33.02 115.57 0)
+    (property "Reference" "#PWR064" (id 0) (at 33.02 115.57 0)
       (effects (font (size 1.27 1.27)) hide)
     )
@@
   (symbol (lib_id "Driver_FET:MCP14A0902xMNY") (at 168.91 46.99 0) (unit 1)
     (in_bom yes) (on_board yes)
-    (property "Reference" "U57" (id 0) (at 173.99 50.8 0)
-      (effects (font (size 1.27 1.27)) (justify left))
-    )
+    (property "Reference" "U26" (id 0) (at 173.99 50.8 0)
+      (effects (font (size 1.27 1.27)) (justify left))
+    )

Commit message: routing and stuff
Parts:
- removed U21: LM358, Package_SO:SO-8_3.9x4.9mm_P1.27mm, symbol Amplifier_Operational:LM358
- added U?: (no value), symbol Amplifier_Operational:LM321
Connections:
- net +3.3VA: now also U?.5 (V+)
- net GND: now also U?.2 (V-)
- net TELEM_VIN: now also R37.2, R38.1
- net Vset: now also U?.3 (-)
- net at U24.2 (VIN_REG): now also U?.4
- net at R35.2, R36.1: now also U?.1 (+)
Changed lines of the file:
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@@
   (junction (at 152.4 46.99) (diameter 0) (color 0 0 0 0)
   )
-  (junction (at 81.28 53.34) (diameter 0) (color 0 0 0 0)
-  )
   (junction (at 102.87 35.56) (diameter 0) (color 0 0 0 0)
   )
@@
   )
   (junction (at 200.66 66.04) (diameter 0) (color 0 0 0 0)
+  )
+  (junction (at 58.42 127) (diameter 0) (color 0 0 0 0)
   )
   (junction (at 120.65 111.76) (diameter 0) (color 0 0 0 0)
@@
     (stroke (width 0) (type default) (color 0 0 0 0))
   )
-  (wire (pts (xy 33.02 127) (xy 50.8 127))
-    (stroke (width 0) (type default) (color 0 0 0 0))
-  )
   (wire (pts (xy 102.87 66.04) (xy 115.57 66.04))
     (stroke (width 0) (type default) (color 0 0 0 0))
@@
     (stroke (width 0) (type default) (color 0 0 0 0))
   )
-  (wire (pts (xy 101.6 63.5) (xy 101.6 55.88))
-    (stroke (width 0) (type default) (color 0 0 0 0))
-  )
   (wire (pts (xy 34.29 62.23) (xy 35.56 62.23))
     (stroke (width 0) (type default) (color 0 0 0 0))
@@
     (stroke (width 0) (type default) (color 0 0 0 0))
   )
+  (wire (pts (xy 58.42 127) (xy 74.93 127))
+    (stroke (width 0) (type default) (color 0 0 0 0))
+  )
   (wire (pts (xy 50.8 59.69) (xy 59.69 59.69))
     (stroke (width 0) (type default) (color 0 0 0 0))
@@
     (stroke (width 0) (type default) (color 0 0 0 0))
   )
-  (wire (pts (xy 86.36 63.5) (xy 101.6 63.5))
-    (stroke (width 0) (type default) (color 0 0 0 0))
-  )
   (wire (pts (xy 111.76 119.38) (xy 110.49 119.38))
     (stroke (width 0) (type default) (color 0 0 0 0))
@@
     (stroke (width 0) (type default) (color 0 0 0 0))
   )
-  (wire (pts (xy 50.8 127) (xy 74.93 127))
+  (wire (pts (xy 50.8 127) (xy 58.42 127))
     (stroke (width 0) (type default) (color 0 0 0 0))
   )
@@
     (stroke (width 0) (type default) (color 0 0 0 0))
   )
+  (wire (pts (xy 58.42 116.84) (xy 58.42 127))
+    (stroke (width 0) (type default) (color 0 0 0 0))
+  )
   (wire (pts (xy 74.93 104.14) (xy 74.93 127))
     (stroke (width 0) (type default) (color 0 0 0 0))
@@
     (stroke (width 0) (type default) (color 0 0 0 0))
   )
-  (wire (pts (xy 86.36 53.34) (xy 81.28 53.34))
-    (stroke (width 0) (type default) (color 0 0 0 0))
-  )
   (wire (pts (xy 120.65 111.76) (xy 128.27 111.76))
     (stroke (width 0) (type default) (color 0 0 0 0))
@@
   )
   (wire (pts (xy 111.76 63.5) (xy 152.4 63.5))
-    (stroke (width 0) (type default) (color 0 0 0 0))
-  )
-  (wire (pts (xy 86.36 58.42) (xy 86.36 63.5))
     (stroke (width 0) (type default) (color 0 0 0 0))
   )
@@
     (effects (font (size 1.27 1.27)) (justify left))
   )
-  (hierarchical_label "TELEM_VIN" (shape input) (at 101.6 55.88 0)
+  (hierarchical_label "TELEM_VIN" (shape input) (at 81.28 49.53 0)
     (effects (font (size 1.27 1.27)) (justify left))
   )
@@
     (pin "9")
   )
-  (symbol (lib_id "Amplifier_Operational:LM358") (at 93.98 55.88 0) (unit 1)
-    (in_bom yes) (on_board yes)
-    (property "Reference" "U21" (id 0) (at 93.98 46.5582 0))
-    (property "Value" "LM358" (id 1) (at 93.98 48.8696 0))
-    (property "Footprint" "Package_SO:SO-8_3.9x4.9mm_P1.27mm" (id 2) (at 93.98 55.88 0)
-      (effects (font (size 1.27 1.27)) hide)
-    )
-    (property "Datasheet" "http://www.ti.com/lit/ds/symlink/lm2904-n.pdf" (id 3) (at 93.98 55.88 0)
-      (effects (font (size 1.27 1.27)) hide)
-    )
-    (pin "1")
-    (pin "2")
-    (pin "3")
-    (pin "5")
-    (pin "6")
-    (pin "7")
-    (pin "4")
-    (pin "8")
-  )
-  (symbol (lib_id "Amplifier_Operational:LM358") (at 60.96 109.22 0) (unit 2)
-    (in_bom yes) (on_board yes)
-    (property "Reference" "U21" (id 0) (at 60.96 99.8982 0))
-    (property "Value" "LM358" (id 1) (at 60.96 102.2096 0))
-    (property "Footprint" "Package_SO:SO-8_3.9x4.9mm_P1.27mm" (id 2) (at 60.96 109.22 0)
-      (effects (font (size 1.27 1.27)) hide)
-    )
-    (property "Datasheet" "http://www.ti.com/lit/ds/symlink/lm2904-n.pdf" (id 3) (at 60.96 109.22 0)
-      (effects (font (size 1.27 1.27)) hide)
-    )
-    (pin "1")
-    (pin "2")
-    (pin "3")
-    (pin "5")
-    (pin "6")
-    (pin "7")
-    (pin "4")
-    (pin "8")
-  )
-  (symbol (lib_id "Amplifier_Operational:LM358") (at 35.56 119.38 0) (unit 3)
-    (in_bom yes) (on_board yes)
-    (property "Reference" "U21" (id 0) (at 27.94 118.11 0)
-      (effects (font (size 1.27 1.27)) (justify left))
-    )
-    (property "Value" "LM358" (id 1) (at 25.4 120.65 0)
-      (effects (font (size 1.27 1.27)) (justify left))
-    )
-    (property "Footprint" "Package_SO:SO-8_3.9x4.9mm_P1.27mm" (id 2) (at 35.56 119.38 0)
-      (effects (font (size 1.27 1.27)) hide)
-    )
-    (property "Datasheet" "http://www.ti.com/lit/ds/symlink/lm2904-n.pdf" (id 3) (at 35.56 119.38 0)
-      (effects (font (size 1.27 1.27)) hide)
-    )
-    (pin "1")
-    (pin "2")
-    (pin "3")
-    (pin "5")
-    (pin "6")
-    (pin "7")
-    (pin "4")
-    (pin "8")
-  )
   (symbol (lib_id "Device:R") (at 50.8 101.6 0) (unit 1)
     (in_bom yes) (on_board yes)
@@
     (pin "1")
   )
-  (symbol (lib_id "power:+3.3VA") (at 33.02 111.76 0) (unit 1)
-    (in_bom yes) (on_board yes)
-    (property "Reference" "#PWR064" (id 0) (at 33.02 115.57 0)
-      (effects (font (size 1.27 1.27)) hide)
-    )
-    (property "Value" "+3.3VA" (id 1) (at 33.401 107.3658 0))
-    (property "Footprint" "" (id 2) (at 33.02 111.76 0)
-      (effects (font (size 1.27 1.27)) hide)
-    )
-    (property "Datasheet" "" (id 3) (at 33.02 111.76 0)
-      (effects (font (size 1.27 1.27)) hide)
-    )
-    (pin "1")
+  (symbol (lib_id "Amplifier_Operational:LM321") (at 60.96 109.22 0) (unit 1)
+    (in_bom yes) (on_board yes) (fields_autoplaced)
+    (property "Reference" "U?" (id 0) (at 71.12 104.521 0))
+    (property "Value" "" (id 1) (at 71.12 107.061 0))
+    (property "Footprint" "" (id 2) (at 60.96 109.22 0)
+      (effects (font (size 1.27 1.27)) hide)
+    )
+    (property "Datasheet" "http://www.ti.com/lit/ds/symlink/lm321.pdf" (id 3) (at 60.96 109.22 0)
+      (effects (font (size 1.27 1.27)) hide)
+    )
+    (pin "1")
+    (pin "2")
+    (pin "3")
+    (pin "4")
+    (pin "5")
   )
   (symbol (lib_id "Driver_FET:MCP14A0902xMNY") (at 168.91 46.99 0) (unit 1)
@@
     (pin "9")
   )
+  (symbol (lib_id "power:+3.3VA") (at 58.42 101.6 0) (unit 1)
+    (in_bom yes) (on_board yes)
+    (property "Reference" "#PWR?" (id 0) (at 58.42 105.41 0)
+      (effects (font (size 1.27 1.27)) hide)
+    )
+    (property "Value" "" (id 1) (at 58.42 97.79 0))
+    (property "Footprint" "" (id 2) (at 58.42 101.6 0)
+      (effects (font (size 1.27 1.27)) hide)
+    )
+    (property "Datasheet" "" (id 3) (at 58.42 101.6 0)
+      (effects (font (size 1.27 1.27)) hide)
+    )
+    (pin "1")
+  )
 )
