File: ECAD/EPS/TJ-EPS.kicad_sch (KiCad schematic)
At the start: 41 parts, among them J1 SWD/DEBUG, Q1 2N7002, Q2 IRF7458, U1 CD74HC4067SM, U2 CD74HC4067SM, U3 MAX6369, U4 CD74HC4067SM, U5 STM32F103C8Tx, Y1 8MHz

Commit message: selectable voltages on PDMs
Parts:
- JP1: symbol TJ-EPS-rescue:SolderJumper_3_Open-Jumper -> Jumper:SolderJumper_3_Open
Other:
- removed sheet PowerDistribution

Commit message: descope to 10 pdms, replace mcp3208 with mcp3008 bc of stock
Connections:
- net TELEM_ISW11 is gone; now on net TELEM_IBATV: U4.21 (I10)
- net TELEM_ISW12 is gone; now on net TELEM_I5V: U4.20 (I11)
- net TELEM_VSW11 is gone; now on net TELEM_VBATV: U2.21 (I10)
- net TELEM_VSW12 is gone; now on net TELEM_V5V: U2.20 (I11)
- net TELEM_I3V3: now also U4.19 (I12); no longer U4.17 (I14)
- net TELEM_I5V: no longer U4.18 (I13)
- net TELEM_IBATV: no longer U4.19 (I12)
- net TELEM_V3V3: now also U2.19 (I12); no longer U2.17 (I14)
- net TELEM_V5V: no longer U2.18 (I13)
- net TELEM_VBATV: no longer U2.19 (I12)
- net SW11: no longer names the net of H2.19 (Pin_19)
- net SW12: no longer names the net of H2.20 (Pin_20)
- no-connect marks 22 -> 24

Commit message: layout and footprints
Parts:
- added C1, C2, C3, C4: 0.1uF, symbol Device:C
- renumbered C6 to C10, C7 to C11, C8 to C12, C9 to C13, C10 to C14, C11 to C15, C12 to C16, C13 to C17, C14 to C18, C15 to C19, C1 to C5, C2 to C6, C3 to C7, C4 to C8, C5 to C9
Connections:
- net GND: now also C1.2, C2.2, C3.2, C4.2; no longer MH1.1, MH2.1, MH3.1, MH4.1
- new net: C1.1, MH1.1
- new net: C2.1, MH2.1
- new net: C3.1, MH3.1
- new net: C4.1, MH4.1
Other:
- moved on the sheet: MH1, MH2, MH3, MH4

Commit message: routing and stuff
Parts:
- C1, C2, C3, C4: footprint (none) -> Capacitor_SMD:C_0805_2012Metric
Changed lines of the file:
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@@
       (effects (font (size 1.27 1.27)) (justify left))
     )
-    (property "Footprint" "" (id 2) (at 281.6352 49.53 0)
+    (property "Footprint" "Capacitor_SMD:C_0805_2012Metric" (id 2) (at 281.6352 49.53 0)
       (effects (font (size 1.27 1.27)) hide)
     )
@@
       (effects (font (size 1.27 1.27)) (justify left))
     )
-    (property "Footprint" "" (id 2) (at 270.2052 49.53 0)
+    (property "Footprint" "Capacitor_SMD:C_0805_2012Metric" (id 2) (at 270.2052 49.53 0)
       (effects (font (size 1.27 1.27)) hide)
     )
@@
       (effects (font (size 1.27 1.27)) (justify left))
     )
-    (property "Footprint" "" (id 2) (at 270.2052 29.21 0)
+    (property "Footprint" "Capacitor_SMD:C_0805_2012Metric" (id 2) (at 270.2052 29.21 0)
       (effects (font (size 1.27 1.27)) hide)
     )
@@
       (effects (font (size 1.27 1.27)) (justify left))
     )
-    (property "Footprint" "" (id 2) (at 281.6352 29.21 0)
+    (property "Footprint" "Capacitor_SMD:C_0805_2012Metric" (id 2) (at 281.6352 29.21 0)
       (effects (font (size 1.27 1.27)) hide)
     )
@@
       (reference "#PWR063") (unit 1) (value "GND") (footprint "")
     )
-    (path "/00000000-0000-0000-0000-000061bec565/00000000-0000-0000-0000-000061d120a6/00000000-0000-0000-0000-00006219de8c"
-      (reference "#PWR064") (unit 1) (value "+3.3VA") (footprint "")
-    )
     (path "/00000000-0000-0000-0000-000061bec565/00000000-0000-0000-0000-000061d120a6/00000000-0000-0000-0000-0000620d2dfc"
       (reference "#PWR065") (unit 1) (value "+3.3VA") (footprint "")
@@
       (reference "#PWR0177") (unit 1) (value "GND") (footprint "")
     )
+    (path "/00000000-0000-0000-0000-000061bec565/00000000-0000-0000-0000-000061d120a6/e3ead1dd-4db8-44b4-8d50-b8ecbf58917f"
+      (reference "#PWR?") (unit 1) (value "+3.3VA") (footprint "")
+    )
     (path "/7e3f1371-1389-4ebf-8bab-3a86b2caca4c"
       (reference "C1") (unit 1) (value "0.1uF") (footprint "Capacitor_SMD:C_0805_2012Metric")
@@
       (reference "U14") (unit 1) (value "INA180A3") (footprint "Package_TO_SOT_SMD:SOT-23-5")
     )
-    (path "/00000000-0000-0000-0000-000061bec565/00000000-0000-0000-0000-000061bec848/00000000-0000-0000-0000-000061c384af"
-      (reference "U15") (unit 1) (value "LM358") (footprint "Package_SO:SO-8_3.9x4.9mm_P1.27mm")
-    )
-    (path "/00000000-0000-0000-0000-000061bec565/00000000-0000-0000-0000-000061bec848/00000000-0000-0000-0000-000061c39a83"
-      (reference "U15") (unit 2) (value "LM358") (footprint "Package_SO:SO-8_3.9x4.9mm_P1.27mm")
-    )
-    (path "/00000000-0000-0000-0000-000061bec565/00000000-0000-0000-0000-000061bec848/00000000-0000-0000-0000-000061c3aed7"
-      (reference "U15") (unit 3) (value "LM358") (footprint "Package_SO:SO-8_3.9x4.9mm_P1.27mm")
-    )
     (path "/00000000-0000-0000-0000-000061bec565/00000000-0000-0000-0000-000061bec848/00000000-0000-0000-0000-000061c24a1a"
       (reference "U16") (unit 1) (value "LT3652EMSE") (footprint "Package_SO:MSOP-12-1EP_3x4mm_P0.65mm_EP1.65x2.85mm")
@@
       (reference "U18") (unit 1) (value "INA180A3") (footprint "Package_TO_SOT_SMD:SOT-23-5")
     )
-    (path "/00000000-0000-0000-0000-000061bec565/00000000-0000-0000-0000-000061e10014/00000000-0000-0000-0000-000061c384af"
-      (reference "U19") (unit 1) (value "LM358") (footprint "Package_SO:SO-8_3.9x4.9mm_P1.27mm")
-    )
-    (path "/00000000-0000-0000-0000-000061bec565/00000000-0000-0000-0000-000061e10014/00000000-0000-0000-0000-000061c39a83"
-      (reference "U19") (unit 2) (value "LM358") (footprint "Package_SO:SO-8_3.9x4.9mm_P1.27mm")
-    )
-    (path "/00000000-0000-0000-0000-000061bec565/00000000-0000-0000-0000-000061e10014/00000000-0000-0000-0000-000061c3aed7"
-      (reference "U19") (unit 3) (value "LM358") (footprint "Package_SO:SO-8_3.9x4.9mm_P1.27mm")
-    )
     (path "/00000000-0000-0000-0000-000061bec565/00000000-0000-0000-0000-000061e10014/00000000-0000-0000-0000-000061c24a1a"
       (reference "U20") (unit 1) (value "LT3652EMSE") (footprint "Package_SO:MSOP-12-1EP_3x4mm_P0.65mm_EP1.65x2.85mm")
     )
-    (path "/00000000-0000-0000-0000-000061bec565/00000000-0000-0000-0000-000061d120a6/00000000-0000-0000-0000-000061d7baca"
-      (reference "U21") (unit 1) (value "LM358") (footprint "Package_SO:SO-8_3.9x4.9mm_P1.27mm")
-    )
-    (path "/00000000-0000-0000-0000-000061bec565/00000000-0000-0000-0000-000061d120a6/00000000-0000-0000-0000-000061d7bad0"
-      (reference "U21") (unit 2) (value "LM358") (footprint "Package_SO:SO-8_3.9x4.9mm_P1.27mm")
-    )
-    (path "/00000000-0000-0000-0000-000061bec565/00000000-0000-0000-0000-000061d120a6/00000000-0000-0000-0000-000061d7bad6"
-      (reference "U21") (unit 3) (value "LM358") (footprint "Package_SO:SO-8_3.9x4.9mm_P1.27mm")
-    )
     (path "/00000000-0000-0000-0000-000061bec565/00000000-0000-0000-0000-000061d120a6/00000000-0000-0000-0000-0000620d2de5"
       (reference "U22") (unit 1) (value "INA180A3") (footprint "Package_TO_SOT_SMD:SOT-23-5")
@@
       (reference "U33") (unit 1) (value "MAX4373F") (footprint "Package_SO:SO-8_3.9x4.9mm_P1.27mm")
     )
-    (path "/00000000-0000-0000-0000-000061c9425d/00000000-0000-0000-0000-000062734c35/00000000-0000-0000-0000-000061d6733e"
-      (reference "U34") (unit 1) (value "AD8603") (footprint "Package_TO_SOT_SMD:TSOT-23-5")
+    (path "/00000000-0000-0000-0000-000061c9425d/00000000-0000-0000-0000-000062734c35/f8baf378-fa33-49d0-8b04-5731a7323f11"
+      (reference "U34") (unit 1) (value "LM321") (footprint "Package_TO_SOT_SMD:SOT-23-5")
     )
     (path "/00000000-0000-0000-0000-000061c9425d/00000000-0000-0000-0000-000062734c35/00000000-0000-0000-0000-0000628e3a19"
       (reference "U35") (unit 1) (value "LTC6993xS6-4") (footprint "Package_TO_SOT_SMD:TSOT-23-6")
     )
-    (path "/00000000-0000-0000-0000-000061c9425d/00000000-0000-0000-0000-00006278b84c/00000000-0000-0000-0000-000061d6733e"
-      (reference "U36") (unit 1) (value "AD8603") (footprint "Package_TO_SOT_SMD:TSOT-23-5")
+    (path "/00000000-0000-0000-0000-000061c9425d/00000000-0000-0000-0000-00006278b84c/f8baf378-fa33-49d0-8b04-5731a7323f11"
+      (reference "U36") (unit 1) (value "LM321") (footprint "Package_TO_SOT_SMD:SOT-23-5")
     )
     (path "/00000000-0000-0000-0000-000061c9425d/00000000-0000-0000-0000-00006278b84c/00000000-0000-0000-0000-0000628e3a19"
       (reference "U37") (unit 1) (value "LTC6993xS6-4") (footprint "Package_TO_SOT_SMD:TSOT-23-6")
     )
-    (path "/00000000-0000-0000-0000-000061c9425d/00000000-0000-0000-0000-00006286fcfd/00000000-0000-0000-0000-000061d6733e"
-      (reference "U38") (unit 1) (value "AD8603") (footprint "Package_TO_SOT_SMD:TSOT-23-5")
+    (path "/00000000-0000-0000-0000-000061c9425d/00000000-0000-0000-0000-00006286fcfd/f8baf378-fa33-49d0-8b04-5731a7323f11"
+      (reference "U38") (unit 1) (value "LM321") (footprint "Package_TO_SOT_SMD:SOT-23-5")
     )
     (path "/00000000-0000-0000-0000-000061c9425d/00000000-0000-0000-0000-00006286fcfd/00000000-0000-0000-0000-0000628e3a19"
@@
       (reference "U51") (unit 1) (value "INA180A3") (footprint "Package_TO_SOT_SMD:SOT-23-5")
     )
-    (path "/00000000-0000-0000-0000-000061bec565/3f3e5af9-b6d1-4725-9068-724c489d3608/00000000-0000-0000-0000-000061c384af"
-      (reference "U52") (unit 1) (value "LM358") (footprint "Package_SO:SO-8_3.9x4.9mm_P1.27mm")
-    )
-    (path "/00000000-0000-0000-0000-000061bec565/3f3e5af9-b6d1-4725-9068-724c489d3608/00000000-0000-0000-0000-000061c39a83"
-      (reference "U52") (unit 2) (value "LM358") (footprint "Package_SO:SO-8_3.9x4.9mm_P1.27mm")
-    )
-    (path "/00000000-0000-0000-0000-000061bec565/3f3e5af9-b6d1-4725-9068-724c489d3608/00000000-0000-0000-0000-000061c3aed7"
-      (reference "U52") (unit 3) (value "LM358") (footprint "Package_SO:SO-8_3.9x4.9mm_P1.27mm")
-    )
     (path "/00000000-0000-0000-0000-000061bec565/3f3e5af9-b6d1-4725-9068-724c489d3608/00000000-0000-0000-0000-000061c24a1a"
       (reference "U53") (unit 1) (value "LT3652EMSE") (footprint "Package_SO:MSOP-12-1EP_3x4mm_P0.65mm_EP1.65x2.85mm")
     )
+    (path "/00000000-0000-0000-0000-000061bec565/00000000-0000-0000-0000-000061d120a6/3c5b7bb6-ec62-4822-aa17-516f6ba3ea36"
+      (reference "U?") (unit 1) (value "LM321") (footprint "Package_TO_SOT_SMD:SOT-23-5")
+    )
+    (path "/00000000-0000-0000-0000-000061bec565/00000000-0000-0000-0000-000061bec848/71842248-20be-4a73-8117-eec39847c925"
+      (reference "U?") (unit 1) (value "LM321") (footprint "Package_TO_SOT_SMD:SOT-23-5")
+    )
+    (path "/00000000-0000-0000-0000-000061bec565/3f3e5af9-b6d1-4725-9068-724c489d3608/71842248-20be-4a73-8117-eec39847c925"
+      (reference "U?") (unit 1) (value "LM321") (footprint "Package_TO_SOT_SMD:SOT-23-5")
+    )
+    (path "/00000000-0000-0000-0000-000061bec565/00000000-0000-0000-0000-000061e10014/71842248-20be-4a73-8117-eec39847c925"
+      (reference "U?") (unit 1) (value "LM321") (footprint "Package_TO_SOT_SMD:SOT-23-5")
+    )
     (path "/00000000-0000-0000-0000-000061dbcdff"

Commit message: move solar to daughterboard... again. Also replace all 0603 resistor with 0805
Parts:
- removed C5: 0.1uF, Capacitor_SMD:C_0805_2012Metric, symbol Device:C
- removed C7: 0.01uF, Capacitor_SMD:C_0805_2012Metric, symbol Device:C
- removed U1: CD74HC4067SM, Package_SO:SSOP-24_5.3x8.2mm_P0.65mm, symbol 74xx:CD74HC4067SM
- added J2: (no value), symbol Connector_Generic:Conn_02x05_Counter_Clockwise
- added MH1, MH2, MH3, MH4: (no value), symbol Mechanical:MountingHole
- renumbered C8 to C1, C16 to C10, C17 to C11, C18 to C12, C19 to C13, C1 to C14, C2 to C15, C3 to C16, C4 to C17, C6 to C2, C10 to C3, C11 to C4, C9 to C5, C14 to C6, C12 to C7, C13 to C8, C15 to C9, MH1 to MH5, MH2 to MH6, MH3 to MH7, MH4 to MH8, U2 to U1, U4 to U2, U5 to U4
Connections:
- net MUX0OUT is gone; now on net MUX1OUT: U4.10 (PA0)
- net BCR_OUT: now also J2.3 (Pin_3), J2.4 (Pin_4)
- net GND: now also J2.5 (Pin_5), J2.6 (Pin_6)
- net MUX1OUT: now also J2.1 (Pin_1); no longer U4.11 (PA1)
- net MUX2OUT: now also U4.11 (PA1), J2.2 (Pin_2); no longer U4.12 (PA2)
- net S0: now also J2.10 (Pin_10)
- net S1: now also J2.9 (Pin_9)
- net S2: now also J2.8 (Pin_8)
- net S3: now also J2.7 (Pin_7)
- net TELEM_TBRD: now also U1.18 (I13)
- net MUX4OUT: now reaches U4.13 (PA3)
- new net MUX3OUT: U4.12 (PA2)
Other:
- removed sheet SolarConditioning
- moved on the sheet: C1, C3, C4, C6, U1, U2
