File: ECAD/EPS/PDM.kicad_sch (KiCad schematic)
At the start: 11 parts, among them Q29 2N7002, Q30 IRF7458, U43 INA180A3

Commit message: selectable voltages on PDMs
Parts:
- removed C69: 0.1uF, Capacitor_SMD:C_0603_1608Metric, symbol Device:C
- removed D26: RR264MM, Diode_SMD:D_SOD-123F, symbol Device:D
- removed Q29: 2N7002, Package_TO_SOT_SMD:SOT-23, symbol Transistor_FET:2N7002
- removed Q30: IRF7458, Package_SO:SOIC-8_3.9x4.9mm_P1.27mm, symbol Transistor_FET:IRF7404
- removed R116: 100R, Resistor_SMD:R_0603_1608Metric, symbol Device:R
- removed R117, R118: 10K, Resistor_SMD:R_0603_1608Metric, symbol Device:R
- removed R119, R120: 100K, Resistor_SMD:R_0603_1608Metric, symbol Device:R
- removed R121: 4m, Resistor_SMD:R_1206_3216Metric, symbol Device:R
- removed U43: INA180A3, Package_TO_SOT_SMD:SOT-23-5, symbol Amplifier_Current:INA138
- added C?: 0.1uF, Capacitor_SMD:C_0603_1608Metric, symbol Device:C
- added D?: RR264MM, Diode_SMD:D_SOD-123F, symbol Device:D
- added JP?: JP, symbol symbols:SolderJumper_4_Open
- added Q?: IRF7458, Package_SO:SOIC-8_3.9x4.9mm_P1.27mm, symbol Transistor_FET:IRF7404
- added Q?: 2N7002, Package_TO_SOT_SMD:SOT-23, symbol Transistor_FET:2N7002
- added R?: 200K, Resistor_SMD:R_0603_1608Metric, symbol Device:R
- added R? (x2): 10K, Resistor_SMD:R_0603_1608Metric, symbol Device:R
- added R?: 100R, Resistor_SMD:R_0603_1608Metric, symbol Device:R
- added R?: 4m, Resistor_SMD:R_1206_3216Metric, symbol Device:R
- added R?: 100K, Resistor_SMD:R_0603_1608Metric, symbol Device:R
- added U?: INA180A3, Package_TO_SOT_SMD:SOT-23-5, symbol Amplifier_Current:INA138
Connections:
- net +3V3: now also JP?.1 (A)
- net GATE: now also R?.2
- net GND: now also C?.2, D?.2 (A), Q?.2 (S), R?.2, R?.2, U?.2 (GND)
- net TELEM_IOUT: now also U?.1
- net TELEM_VOUT: now also R?.1, R?.2
- net VOUT: now also D?.1 (K), R?.1, U?.4 (-)
- new net: Q?.1 (S), Q?.2 (S), Q?.3 (S), R?.1, R?.2, U?.3 (+)
- new net: Q?.3 (D), Q?.4 (G), R?.2
- new net: JP?.2 (C), Q?.5 (D), Q?.6 (D), Q?.7 (D), Q?.8 (D), R?.1
- new net: Q?.1 (G), R?.1, R?.1
- new net +5V: JP?.3 (B)
- new net +BATT: JP?.4 (D)
- new net VCC: C?.1, U?.5 (V+)
Other:
- note added: "Select Voltage By Jumper"

Commit message: layout and footprints
Parts:
- JP8: renamed from JP?; footprint (none) -> footprints:SolderJumper-4_P1.3mm_Open_RoundedPad1.0x1.5mm
- gave numbers to parts that had none: 11
Changed lines of the file:
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@@
   (symbol (lib_id "Device:D") (at 189.23 63.5 270) (unit 1)
     (in_bom yes) (on_board yes)
-    (property "Reference" "D?" (id 0) (at 191.262 62.3316 90)
+    (property "Reference" "D30" (id 0) (at 191.262 62.3316 90)
       (effects (font (size 1.27 1.27)) (justify left))
     )
@@
   (symbol (lib_id "Device:R") (at 118.11 64.77 0) (unit 1)
     (in_bom yes) (on_board yes)
-    (property "Reference" "R?" (id 0) (at 119.38 64.77 0)
+    (property "Reference" "R134" (id 0) (at 119.38 64.77 0)
       (effects (font (size 1.27 1.27)) (justify left))
     )
@@
   (symbol (lib_id "power:+BATT") (at 118.11 34.29 0) (unit 1)
     (in_bom yes) (on_board yes)
-    (property "Reference" "#PWR?" (id 0) (at 118.11 38.1 0)
+    (property "Reference" "#PWR0146" (id 0) (at 118.11 38.1 0)
       (effects (font (size 1.27 1.27)) hide)
     )
@@
   (symbol (lib_id "Transistor_FET:IRF7404") (at 115.57 54.61 0) (unit 1)
     (in_bom yes) (on_board yes)
-    (property "Reference" "Q?" (id 0) (at 120.777 53.4416 0)
+    (property "Reference" "Q33" (id 0) (at 120.777 53.4416 0)
       (effects (font (size 1.27 1.27)) (justify left))
     )
@@
   (symbol (lib_id "Transistor_FET:2N7002") (at 104.14 63.5 0) (unit 1)
     (in_bom yes) (on_board yes)
-    (property "Reference" "Q?" (id 0) (at 109.3216 62.3316 0)
+    (property "Reference" "Q32" (id 0) (at 109.3216 62.3316 0)
       (effects (font (size 1.27 1.27)) (justify left))
     )
@@
   (symbol (lib_id "Device:R") (at 106.68 46.99 0) (unit 1)
     (in_bom yes) (on_board yes)
-    (property "Reference" "R?" (id 0) (at 107.95 46.99 0)
+    (property "Reference" "R133" (id 0) (at 107.95 46.99 0)
       (effects (font (size 1.27 1.27)) (justify left))
     )
@@
   (symbol (lib_id "Device:R") (at 90.17 63.5 270) (unit 1)
     (in_bom yes) (on_board yes)
-    (property "Reference" "R?" (id 0) (at 90.17 60.96 90))
+    (property "Reference" "R131" (id 0) (at 90.17 60.96 90))
     (property "Value" "100R" (id 1) (at 90.17 63.5 90))
     (property "Footprint" "Resistor_SMD:R_0603_1608Metric" (id 2) (at 90.17 61.722 90)
@@
   (symbol (lib_id "Device:R") (at 96.52 67.31 0) (unit 1)
     (in_bom yes) (on_board yes)
-    (property "Reference" "R?" (id 0) (at 97.79 67.31 0)
+    (property "Reference" "R132" (id 0) (at 97.79 67.31 0)
       (effects (font (size 1.27 1.27)) (justify left))
     )
@@
   (symbol (lib_id "power:GND") (at 118.11 80.01 0) (unit 1)
     (in_bom yes) (on_board yes)
-    (property "Reference" "#PWR?" (id 0) (at 118.11 86.36 0)
+    (property "Reference" "#PWR0147" (id 0) (at 118.11 86.36 0)
       (effects (font (size 1.27 1.27)) hide)
     )
@@
   (symbol (lib_id "Device:R") (at 144.78 59.69 270) (unit 1)
     (in_bom yes) (on_board yes)
-    (property "Reference" "R?" (id 0) (at 144.78 57.15 90))
+    (property "Reference" "R136" (id 0) (at 144.78 57.15 90))
     (property "Value" "4m" (id 1) (at 144.78 59.69 90))
     (property "Footprint" "Resistor_SMD:R_1206_3216Metric" (id 2) (at 144.78 57.912 90)
@@
   (symbol (lib_id "Device:R") (at 118.11 74.93 0) (unit 1)
     (in_bom yes) (on_board yes)
-    (property "Reference" "R?" (id 0) (at 119.38 74.93 0)
+    (property "Reference" "R135" (id 0) (at 119.38 74.93 0)
       (effects (font (size 1.27 1.27)) (justify left))
     )
@@
   (symbol (lib_id "Amplifier_Current:INA138") (at 158.75 72.39 0) (unit 1)
     (in_bom yes) (on_board yes)
-    (property "Reference" "U?" (id 0) (at 167.4876 71.2216 0)
+    (property "Reference" "U46" (id 0) (at 167.4876 71.2216 0)
       (effects (font (size 1.27 1.27)) (justify left))
     )
@@
   (symbol (lib_id "power:VCC") (at 156.21 64.77 0) (unit 1)
     (in_bom yes) (on_board yes)
-    (property "Reference" "#PWR?" (id 0) (at 156.21 68.58 0)
+    (property "Reference" "#PWR0149" (id 0) (at 156.21 68.58 0)
       (effects (font (size 1.27 1.27)) hide)
     )
@@
   (symbol (lib_id "Device:C") (at 160.02 64.77 90) (unit 1)
     (in_bom yes) (on_board yes)
-    (property "Reference" "C?" (id 0) (at 161.29 60.96 90)
+    (property "Reference" "C75" (id 0) (at 161.29 60.96 90)
       (effects (font (size 1.27 1.27)) (justify right))
     )
@@
   (symbol (lib_id "power:GND") (at 163.83 64.77 0) (unit 1)
     (in_bom yes) (on_board yes)
-    (property "Reference" "#PWR?" (id 0) (at 163.83 71.12 0)
+    (property "Reference" "#PWR0150" (id 0) (at 163.83 71.12 0)
       (effects (font (size 1.27 1.27)) hide)
     )
@@
   (symbol (lib_id "symbols:SolderJumper_4_Open") (at 118.11 39.37 0) (unit 1)
     (in_bom yes) (on_board yes)
-    (property "Reference" "JP?" (id 0) (at 120.65 35.56 0)
+    (property "Reference" "JP8" (id 0) (at 120.65 35.56 0)
       (effects (font (size 1.27 1.27)) (justify left))
     )
@@
       (effects (font (size 1.27 1.27)) (justify left))
     )
-    (property "Footprint" "" (id 2) (at 118.11 39.37 0)
+    (property "Footprint" "footprints:SolderJumper-4_P1.3mm_Open_RoundedPad1.0x1.5mm" (id 2) (at 118.11 39.37 0)
       (effects (font (size 1.27 1.27)) hide)
     )
@@
   (symbol (lib_id "power:+5V") (at 127 39.37 0) (unit 1)
     (in_bom yes) (on_board yes) (fields_autoplaced)
-    (property "Reference" "#PWR?" (id 0) (at 127 43.18 0)
+    (property "Reference" "#PWR0148" (id 0) (at 127 43.18 0)
       (effects (font (size 1.27 1.27)) hide)
     )
@@
   (symbol (lib_id "power:+3V3") (at 109.22 39.37 0) (unit 1)
     (in_bom yes) (on_board yes) (fields_autoplaced)
-    (property "Reference" "#PWR?" (id 0) (at 109.22 43.18 0)
-      (effects (font (size 1.27 1.27)) hide)
-    )
+    (property "Reference" "#PWR0145" (id 0) (at 109.22 43.18 0)
+      (effects (font (size 1.27 1.27)) hide)
+    )

Commit message: move solar to daughterboard... again. Also replace all 0603 resistor with 0805
Parts:
- R100: renamed from R135; footprint Resistor_SMD:R_0603_1608Metric -> (none)
- R96: renamed from R131; footprint Resistor_SMD:R_0603_1608Metric -> (none)
- R97: renamed from R132; footprint Resistor_SMD:R_0603_1608Metric -> (none)
- R98: renamed from R133; footprint Resistor_SMD:R_0603_1608Metric -> (none)
- R99: renamed from R134; footprint Resistor_SMD:R_0603_1608Metric -> (none)
- renumbered C75 to C46, D30 to D7, Q32 to Q30, Q33 to Q31, R136 to R101, U46 to U24
Connections:
- net at R101.2, R99.1, U24.3 (+): now also Q31.5 (D), Q31.6 (D), Q31.7 (D), Q31.8 (D); no longer Q31.1 (S), Q31.2 (S), Q31.3 (S)
- new net: JP8.2 (C), Q31.1 (S), Q31.2 (S), Q31.3 (S), R98.1
Changed lines of the file:
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@@
   (symbol (lib_id "Device:D") (at 189.23 63.5 270) (unit 1)
     (in_bom yes) (on_board yes)
-    (property "Reference" "D30" (id 0) (at 191.262 62.3316 90)
+    (property "Reference" "D7" (id 0) (at 191.262 62.3316 90)
       (effects (font (size 1.27 1.27)) (justify left))
     )
@@
   (symbol (lib_id "Device:R") (at 118.11 64.77 0) (unit 1)
     (in_bom yes) (on_board yes)
-    (property "Reference" "R134" (id 0) (at 119.38 64.77 0)
+    (property "Reference" "R99" (id 0) (at 119.38 64.77 0)
       (effects (font (size 1.27 1.27)) (justify left))
     )
     (property "Value" "200K" (id 1) (at 118.11 64.77 90))
-    (property "Footprint" "Resistor_SMD:R_0603_1608Metric" (id 2) (at 116.332 64.77 90)
+    (property "Footprint" "" (id 2) (at 116.332 64.77 90)
       (effects (font (size 1.27 1.27)) hide)
     )
@@
   (symbol (lib_id "power:+BATT") (at 118.11 34.29 0) (unit 1)
     (in_bom yes) (on_board yes)
-    (property "Reference" "#PWR0146" (id 0) (at 118.11 38.1 0)
+    (property "Reference" "#PWR0105" (id 0) (at 118.11 38.1 0)
       (effects (font (size 1.27 1.27)) hide)
     )
@@
     (pin "1")
   )
-  (symbol (lib_id "Transistor_FET:IRF7404") (at 115.57 54.61 0) (unit 1)
-    (in_bom yes) (on_board yes)
-    (property "Reference" "Q33" (id 0) (at 120.777 53.4416 0)
-      (effects (font (size 1.27 1.27)) (justify left))
-    )
-    (property "Value" "IRF7458" (id 1) (at 120.777 55.753 0)
-      (effects (font (size 1.27 1.27)) (justify left))
-    )
-    (property "Footprint" "Package_SO:SOIC-8_3.9x4.9mm_P1.27mm" (id 2) (at 120.65 56.515 0)
+  (symbol (lib_id "Transistor_FET:IRF7404") (at 115.57 54.61 0) (mirror x) (unit 1)
+    (in_bom yes) (on_board yes)
+    (property "Reference" "Q31" (id 0) (at 120.777 55.7784 0)
+      (effects (font (size 1.27 1.27)) (justify left))
+    )
+    (property "Value" "IRF7458" (id 1) (at 120.777 53.467 0)
+      (effects (font (size 1.27 1.27)) (justify left))
+    )
+    (property "Footprint" "Package_SO:SOIC-8_3.9x4.9mm_P1.27mm" (id 2) (at 120.65 52.705 0)
       (effects (font (size 1.27 1.27) italic) (justify left) hide)
     )
@@
   (symbol (lib_id "Transistor_FET:2N7002") (at 104.14 63.5 0) (unit 1)
     (in_bom yes) (on_board yes)
-    (property "Reference" "Q32" (id 0) (at 109.3216 62.3316 0)
+    (property "Reference" "Q30" (id 0) (at 109.3216 62.3316 0)
       (effects (font (size 1.27 1.27)) (justify left))
     )
@@
   (symbol (lib_id "Device:R") (at 106.68 46.99 0) (unit 1)
     (in_bom yes) (on_board yes)
-    (property "Reference" "R133" (id 0) (at 107.95 46.99 0)
+    (property "Reference" "R98" (id 0) (at 107.95 46.99 0)
       (effects (font (size 1.27 1.27)) (justify left))
     )
     (property "Value" "10K" (id 1) (at 106.68 46.99 90))
-    (property "Footprint" "Resistor_SMD:R_0603_1608Metric" (id 2) (at 104.902 46.99 90)
+    (property "Footprint" "" (id 2) (at 104.902 46.99 90)
       (effects (font (size 1.27 1.27)) hide)
     )
@@
   (symbol (lib_id "Device:R") (at 90.17 63.5 270) (unit 1)
     (in_bom yes) (on_board yes)
-    (property "Reference" "R131" (id 0) (at 90.17 60.96 90))
+    (property "Reference" "R96" (id 0) (at 90.17 60.96 90))
     (property "Value" "100R" (id 1) (at 90.17 63.5 90))
-    (property "Footprint" "Resistor_SMD:R_0603_1608Metric" (id 2) (at 90.17 61.722 90)
+    (property "Footprint" "" (id 2) (at 90.17 61.722 90)
       (effects (font (size 1.27 1.27)) hide)
     )
@@
   (symbol (lib_id "Device:R") (at 96.52 67.31 0) (unit 1)
     (in_bom yes) (on_board yes)
-    (property "Reference" "R132" (id 0) (at 97.79 67.31 0)
+    (property "Reference" "R97" (id 0) (at 97.79 67.31 0)
       (effects (font (size 1.27 1.27)) (justify left))
     )
     (property "Value" "10K" (id 1) (at 96.52 67.31 90))
-    (property "Footprint" "Resistor_SMD:R_0603_1608Metric" (id 2) (at 94.742 67.31 90)
+    (property "Footprint" "" (id 2) (at 94.742 67.31 90)
       (effects (font (size 1.27 1.27)) hide)
     )
@@
   (symbol (lib_id "power:GND") (at 118.11 80.01 0) (unit 1)
     (in_bom yes) (on_board yes)
-    (property "Reference" "#PWR0147" (id 0) (at 118.11 86.36 0)
+    (property "Reference" "#PWR0106" (id 0) (at 118.11 86.36 0)
       (effects (font (size 1.27 1.27)) hide)
     )
@@
   (symbol (lib_id "Device:R") (at 144.78 59.69 270) (unit 1)
     (in_bom yes) (on_board yes)
-    (property "Reference" "R136" (id 0) (at 144.78 57.15 90))
+    (property "Reference" "R101" (id 0) (at 144.78 57.15 90))
     (property "Value" "4m" (id 1) (at 144.78 59.69 90))
     (property "Footprint" "Resistor_SMD:R_1206_3216Metric" (id 2) (at 144.78 57.912 90)
@@
   (symbol (lib_id "Device:R") (at 118.11 74.93 0) (unit 1)
     (in_bom yes) (on_board yes)
-    (property "Reference" "R135" (id 0) (at 119.38 74.93 0)
+    (property "Reference" "R100" (id 0) (at 119.38 74.93 0)
       (effects (font (size 1.27 1.27)) (justify left))
     )
     (property "Value" "100K" (id 1) (at 118.11 74.93 90))
-    (property "Footprint" "Resistor_SMD:R_0603_1608Metric" (id 2) (at 116.332 74.93 90)
+    (property "Footprint" "" (id 2) (at 116.332 74.93 90)
       (effects (font (size 1.27 1.27)) hide)
     )
@@
   (symbol (lib_id "Amplifier_Current:INA138") (at 158.75 72.39 0) (unit 1)
     (in_bom yes) (on_board yes)
-    (property "Reference" "U46" (id 0) (at 167.4876 71.2216 0)
+    (property "Reference" "U24" (id 0) (at 167.4876 71.2216 0)
       (effects (font (size 1.27 1.27)) (justify left))
     )
@@
   (symbol (lib_id "power:VCC") (at 156.21 64.77 0) (unit 1)
     (in_bom yes) (on_board yes)
-    (property "Reference" "#PWR0149" (id 0) (at 156.21 68.58 0)
+    (property "Reference" "#PWR0108" (id 0) (at 156.21 68.58 0)
       (effects (font (size 1.27 1.27)) hide)
     )
@@
   (symbol (lib_id "Device:C") (at 160.02 64.77 90) (unit 1)
     (in_bom yes) (on_board yes)
-    (property "Reference" "C75" (id 0) (at 161.29 60.96 90)
+    (property "Reference" "C46" (id 0) (at 161.29 60.96 90)
       (effects (font (size 1.27 1.27)) (justify right))
     )
@@
   (symbol (lib_id "power:GND") (at 163.83 64.77 0) (unit 1)
     (in_bom yes) (on_board yes)
-    (property "Reference" "#PWR0150" (id 0) (at 163.83 71.12 0)
+    (property "Reference" "#PWR0109" (id 0) (at 163.83 71.12 0)
       (effects (font (size 1.27 1.27)) hide)
     )
@@
   (symbol (lib_id "power:+5V") (at 127 39.37 0) (unit 1)
     (in_bom yes) (on_board yes) (fields_autoplaced)
-    (property "Reference" "#PWR0148" (id 0) (at 127 43.18 0)
+    (property "Reference" "#PWR0107" (id 0) (at 127 43.18 0)
       (effects (font (size 1.27 1.27)) hide)
     )
@@
   (symbol (lib_id "power:+3V3") (at 109.22 39.37 0) (unit 1)
     (in_bom yes) (on_board yes) (fields_autoplaced)
-    (property "Reference" "#PWR0145" (id 0) (at 109.22 43.18 0)
-      (effects (font (size 1.27 1.27)) hide)
-    )
+    (property "Reference" "#PWR0104" (id 0) (at 109.22 43.18 0)
+      (effects (font (size 1.27 1.27)) hide)
+    )

Commit message: Micro + PCM blocks
Micro + PCM blocks
Parts:
- renumbered C46 to C45, D7 to D6, JP8 to JP7, Q30 to Q28, Q31 to Q29, R96 to R90, R97 to R91, R98 to R92, R99 to R93, R100 to R94, R101 to R95, U24 to U23
Changed lines of the file:
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@@
     (effects (font (size 1.27 1.27)) (justify left))
   )
-  (symbol (lib_id "Device:D") (at 189.23 63.5 270) (unit 1)
-    (in_bom yes) (on_board yes)
-    (property "Reference" "D7" (id 0) (at 191.262 62.3316 90)
+  (symbol (lib_id "Device:D") (at 189.23 63.5 270)
+    (in_bom yes) (on_board yes)
+    (property "Reference" "D6" (id 0) (at 191.262 62.3316 90)
       (effects (font (size 1.27 1.27)) (justify left))
     )
@@
     (pin "2")
   )
-  (symbol (lib_id "Device:R") (at 118.11 64.77 0) (unit 1)
-    (in_bom yes) (on_board yes)
-    (property "Reference" "R99" (id 0) (at 119.38 64.77 0)
+  (symbol (lib_id "Device:R") (at 118.11 64.77 0)
+    (in_bom yes) (on_board yes)
+    (property "Reference" "R93" (id 0) (at 119.38 64.77 0)
       (effects (font (size 1.27 1.27)) (justify left))
     )
@@
     (pin "2")
   )
-  (symbol (lib_id "power:+BATT") (at 118.11 34.29 0) (unit 1)
-    (in_bom yes) (on_board yes)
-    (property "Reference" "#PWR0105" (id 0) (at 118.11 38.1 0)
+  (symbol (lib_id "power:+BATT") (at 118.11 34.29 0)
+    (in_bom yes) (on_board yes)
+    (property "Reference" "#PWR099" (id 0) (at 118.11 38.1 0)
       (effects (font (size 1.27 1.27)) hide)
     )
@@
     (pin "1")
   )
-  (symbol (lib_id "Transistor_FET:IRF7404") (at 115.57 54.61 0) (mirror x) (unit 1)
-    (in_bom yes) (on_board yes)
-    (property "Reference" "Q31" (id 0) (at 120.777 55.7784 0)
+  (symbol (lib_id "Transistor_FET:IRF7404") (at 115.57 54.61 0) (mirror x)
+    (in_bom yes) (on_board yes)
+    (property "Reference" "Q29" (id 0) (at 120.777 55.7784 0)
       (effects (font (size 1.27 1.27)) (justify left))
     )
@@
     (pin "8")
   )
-  (symbol (lib_id "Transistor_FET:2N7002") (at 104.14 63.5 0) (unit 1)
-    (in_bom yes) (on_board yes)
-    (property "Reference" "Q30" (id 0) (at 109.3216 62.3316 0)
+  (symbol (lib_id "Transistor_FET:2N7002") (at 104.14 63.5 0)
+    (in_bom yes) (on_board yes)
+    (property "Reference" "Q28" (id 0) (at 109.3216 62.3316 0)
       (effects (font (size 1.27 1.27)) (justify left))
     )
@@
     (pin "3")
   )
-  (symbol (lib_id "Device:R") (at 106.68 46.99 0) (unit 1)
-    (in_bom yes) (on_board yes)
-    (property "Reference" "R98" (id 0) (at 107.95 46.99 0)
+  (symbol (lib_id "Device:R") (at 106.68 46.99 0)
+    (in_bom yes) (on_board yes)
+    (property "Reference" "R92" (id 0) (at 107.95 46.99 0)
       (effects (font (size 1.27 1.27)) (justify left))
     )
@@
     (pin "2")
   )
-  (symbol (lib_id "Device:R") (at 90.17 63.5 270) (unit 1)
-    (in_bom yes) (on_board yes)
-    (property "Reference" "R96" (id 0) (at 90.17 60.96 90))
+  (symbol (lib_id "Device:R") (at 90.17 63.5 270)
+    (in_bom yes) (on_board yes)
+    (property "Reference" "R90" (id 0) (at 90.17 60.96 90))
     (property "Value" "100R" (id 1) (at 90.17 63.5 90))
     (property "Footprint" "" (id 2) (at 90.17 61.722 90)
@@
     (pin "2")
   )
-  (symbol (lib_id "Device:R") (at 96.52 67.31 0) (unit 1)
-    (in_bom yes) (on_board yes)
-    (property "Reference" "R97" (id 0) (at 97.79 67.31 0)
+  (symbol (lib_id "Device:R") (at 96.52 67.31 0)
+    (in_bom yes) (on_board yes)
+    (property "Reference" "R91" (id 0) (at 97.79 67.31 0)
       (effects (font (size 1.27 1.27)) (justify left))
     )
@@
     (pin "2")
   )
-  (symbol (lib_id "power:GND") (at 118.11 80.01 0) (unit 1)
-    (in_bom yes) (on_board yes)
-    (property "Reference" "#PWR0106" (id 0) (at 118.11 86.36 0)
+  (symbol (lib_id "power:GND") (at 118.11 80.01 0)
+    (in_bom yes) (on_board yes)
+    (property "Reference" "#PWR0100" (id 0) (at 118.11 86.36 0)
       (effects (font (size 1.27 1.27)) hide)
     )
@@
     (pin "1")
   )
-  (symbol (lib_id "Device:R") (at 144.78 59.69 270) (unit 1)
-    (in_bom yes) (on_board yes)
-    (property "Reference" "R101" (id 0) (at 144.78 57.15 90))
+  (symbol (lib_id "Device:R") (at 144.78 59.69 270)
+    (in_bom yes) (on_board yes)
+    (property "Reference" "R95" (id 0) (at 144.78 57.15 90))
     (property "Value" "4m" (id 1) (at 144.78 59.69 90))
     (property "Footprint" "Resistor_SMD:R_1206_3216Metric" (id 2) (at 144.78 57.912 90)
@@
     (pin "2")
   )
-  (symbol (lib_id "Device:R") (at 118.11 74.93 0) (unit 1)
-    (in_bom yes) (on_board yes)
-    (property "Reference" "R100" (id 0) (at 119.38 74.93 0)
+  (symbol (lib_id "Device:R") (at 118.11 74.93 0)
+    (in_bom yes) (on_board yes)
+    (property "Reference" "R94" (id 0) (at 119.38 74.93 0)
       (effects (font (size 1.27 1.27)) (justify left))
     )
@@
     (pin "2")
   )
-  (symbol (lib_id "Amplifier_Current:INA138") (at 158.75 72.39 0) (unit 1)
-    (in_bom yes) (on_board yes)
-    (property "Reference" "U24" (id 0) (at 167.4876 71.2216 0)
+  (symbol (lib_id "Amplifier_Current:INA138") (at 158.75 72.39 0)
+    (in_bom yes) (on_board yes)
+    (property "Reference" "U23" (id 0) (at 167.4876 71.2216 0)
       (effects (font (size 1.27 1.27)) (justify left))
     )
@@
     (pin "5")
   )
-  (symbol (lib_id "power:VCC") (at 156.21 64.77 0) (unit 1)
-    (in_bom yes) (on_board yes)
-    (property "Reference" "#PWR0108" (id 0) (at 156.21 68.58 0)
+  (symbol (lib_id "power:VCC") (at 156.21 64.77 0)
+    (in_bom yes) (on_board yes)
+    (property "Reference" "#PWR0102" (id 0) (at 156.21 68.58 0)
       (effects (font (size 1.27 1.27)) hide)
     )
@@
     (pin "1")
   )
-  (symbol (lib_id "Device:C") (at 160.02 64.77 90) (unit 1)
-    (in_bom yes) (on_board yes)
-    (property "Reference" "C46" (id 0) (at 161.29 60.96 90)
+  (symbol (lib_id "Device:C") (at 160.02 64.77 90)
+    (in_bom yes) (on_board yes)
+    (property "Reference" "C45" (id 0) (at 161.29 60.96 90)
       (effects (font (size 1.27 1.27)) (justify right))
     )
@@
     (pin "2")
   )
-  (symbol (lib_id "power:GND") (at 163.83 64.77 0) (unit 1)
-    (in_bom yes) (on_board yes)
-    (property "Reference" "#PWR0109" (id 0) (at 163.83 71.12 0)
+  (symbol (lib_id "power:GND") (at 163.83 64.77 0)
+    (in_bom yes) (on_board yes)
+    (property "Reference" "#PWR0103" (id 0) (at 163.83 71.12 0)
       (effects (font (size 1.27 1.27)) hide)
     )
@@
     (pin "1")
   )
-  (symbol (lib_id "symbols:SolderJumper_4_Open") (at 118.11 39.37 0) (unit 1)
-    (in_bom yes) (on_board yes)
-    (property "Reference" "JP8" (id 0) (at 120.65 35.56 0)
+  (symbol (lib_id "symbols:SolderJumper_4_Open") (at 118.11 39.37 0)
+    (in_bom yes) (on_board yes)
+    (property "Reference" "JP7" (id 0) (at 120.65 35.56 0)
       (effects (font (size 1.27 1.27)) (justify left))
     )
@@
     (pin "4")
   )
-  (symbol (lib_id "power:+5V") (at 127 39.37 0) (unit 1)
+  (symbol (lib_id "power:+5V") (at 127 39.37 0)
     (in_bom yes) (on_board yes) (fields_autoplaced)
-    (property "Reference" "#PWR0107" (id 0) (at 127 43.18 0)
+    (property "Reference" "#PWR0101" (id 0) (at 127 43.18 0)
       (effects (font (size 1.27 1.27)) hide)
     )
@@
     (pin "1")
   )
-  (symbol (lib_id "power:+3V3") (at 109.22 39.37 0) (unit 1)
+  (symbol (lib_id "power:+3V3") (at 109.22 39.37 0)
     (in_bom yes) (on_board yes) (fields_autoplaced)
-    (property "Reference" "#PWR0104" (id 0) (at 109.22 43.18 0)
-      (effects (font (size 1.27 1.27)) hide)
-    )
+    (property "Reference" "#PWR098" (id 0) (at 109.22 43.18 0)
+      (effects (font (size 1.27 1.27)) hide)
+    )
