File: ECAD/EPS/PDM.kicad_sch (KiCad schematic)
At the start: 12 parts, among them Q24 2N7002, Q25 IRF7458, U18 INA180A3

Commit message: proposed switch layout
Parts:
- C39: renamed from C40; footprint Capacitor_SMD:C_0603_1608Metric -> (none)
Changed lines of the file:
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@@
   (symbol (lib_id "Device:C") (at 160.02 64.77 90) (unit 1)
     (in_bom yes) (on_board yes)
-    (property "Reference" "C40" (id 0) (at 161.29 60.96 90)
+    (property "Reference" "C39" (id 0) (at 161.29 60.96 90)
       (effects (font (size 1.27 1.27)) (justify right))
     )
@@
       (effects (font (size 1.27 1.27)) (justify right))
     )
-    (property "Footprint" "Capacitor_SMD:C_0603_1608Metric" (id 2) (at 163.83 63.8048 0)
+    (property "Footprint" "" (id 2) (at 163.83 63.8048 0)
       (effects (font (size 1.27 1.27)) hide)
     )

Commit message: flip PDM current monitors
Parts:
- C39: footprint (none) -> Capacitor_SMD:C_0805_2012Metric
Changed lines of the file:
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@@
       (effects (font (size 1.27 1.27)) (justify right))
     )
-    (property "Footprint" "" (id 2) (at 163.83 63.8048 0)
+    (property "Footprint" "Capacitor_SMD:C_0805_2012Metric" (id 2) (at 163.83 63.8048 0)
       (effects (font (size 1.27 1.27)) hide)
     )

Commit message: Thick PCM->BCR
Thick PCM->BCR
Parts:
- renumbered C39 to C38, D7 to D6, JP8 to JP7, Q24 to Q22, Q25 to Q23, R74 to R68, R75 to R69, R76 to R70, R77 to R71, R78 to R72, R79 to R73, U18 to U17
Changed lines of the file:
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@@
     (effects (font (size 1.27 1.27)) (justify left))
   )
-  (symbol (lib_id "Device:D") (at 189.23 63.5 270) (unit 1)
-    (in_bom yes) (on_board yes)
-    (property "Reference" "D7" (id 0) (at 191.262 62.3316 90)
+  (symbol (lib_id "Device:D") (at 189.23 63.5 270)
+    (in_bom yes) (on_board yes)
+    (property "Reference" "D6" (id 0) (at 191.262 62.3316 90)
       (effects (font (size 1.27 1.27)) (justify left))
     )
@@
     (pin "2")
   )
-  (symbol (lib_id "Device:R") (at 118.11 64.77 0) (unit 1)
-    (in_bom yes) (on_board yes)
-    (property "Reference" "R77" (id 0) (at 119.38 64.77 0)
+  (symbol (lib_id "Device:R") (at 118.11 64.77 0)
+    (in_bom yes) (on_board yes)
+    (property "Reference" "R71" (id 0) (at 119.38 64.77 0)
       (effects (font (size 1.27 1.27)) (justify left))
     )
@@
     (pin "2")
   )
-  (symbol (lib_id "power:+BATT") (at 118.11 34.29 0) (unit 1)
-    (in_bom yes) (on_board yes)
-    (property "Reference" "#PWR093" (id 0) (at 118.11 38.1 0)
+  (symbol (lib_id "power:+BATT") (at 118.11 34.29 0)
+    (in_bom yes) (on_board yes)
+    (property "Reference" "#PWR0111" (id 0) (at 118.11 38.1 0)
       (effects (font (size 1.27 1.27)) hide)
     )
@@
     (pin "1")
   )
-  (symbol (lib_id "Transistor_FET:IRF7404") (at 115.57 54.61 0) (mirror x) (unit 1)
-    (in_bom yes) (on_board yes)
-    (property "Reference" "Q25" (id 0) (at 120.777 55.7784 0)
+  (symbol (lib_id "Transistor_FET:IRF7404") (at 115.57 54.61 0) (mirror x)
+    (in_bom yes) (on_board yes)
+    (property "Reference" "Q23" (id 0) (at 120.777 55.7784 0)
       (effects (font (size 1.27 1.27)) (justify left))
     )
@@
     (pin "8")
   )
-  (symbol (lib_id "Transistor_FET:2N7002") (at 104.14 63.5 0) (unit 1)
-    (in_bom yes) (on_board yes)
-    (property "Reference" "Q24" (id 0) (at 109.3216 62.3316 0)
+  (symbol (lib_id "Transistor_FET:2N7002") (at 104.14 63.5 0)
+    (in_bom yes) (on_board yes)
+    (property "Reference" "Q22" (id 0) (at 109.3216 62.3316 0)
       (effects (font (size 1.27 1.27)) (justify left))
     )
@@
     (pin "3")
   )
-  (symbol (lib_id "Device:R") (at 106.68 46.99 0) (unit 1)
-    (in_bom yes) (on_board yes)
-    (property "Reference" "R76" (id 0) (at 107.95 46.99 0)
+  (symbol (lib_id "Device:R") (at 106.68 46.99 0)
+    (in_bom yes) (on_board yes)
+    (property "Reference" "R70" (id 0) (at 107.95 46.99 0)
       (effects (font (size 1.27 1.27)) (justify left))
     )
@@
     (pin "2")
   )
-  (symbol (lib_id "Device:R") (at 90.17 63.5 270) (unit 1)
-    (in_bom yes) (on_board yes)
-    (property "Reference" "R74" (id 0) (at 90.17 60.96 90))
+  (symbol (lib_id "Device:R") (at 90.17 63.5 270)
+    (in_bom yes) (on_board yes)
+    (property "Reference" "R68" (id 0) (at 90.17 60.96 90))
     (property "Value" "100R" (id 1) (at 90.17 63.5 90))
     (property "Footprint" "Resistor_SMD:R_0805_2012Metric" (id 2) (at 90.17 61.722 90)
@@
     (pin "2")
   )
-  (symbol (lib_id "Device:R") (at 96.52 67.31 0) (unit 1)
-    (in_bom yes) (on_board yes)
-    (property "Reference" "R75" (id 0) (at 97.79 67.31 0)
+  (symbol (lib_id "Device:R") (at 96.52 67.31 0)
+    (in_bom yes) (on_board yes)
+    (property "Reference" "R69" (id 0) (at 97.79 67.31 0)
       (effects (font (size 1.27 1.27)) (justify left))
     )
@@
     (pin "2")
   )
-  (symbol (lib_id "power:GND") (at 118.11 80.01 0) (unit 1)
-    (in_bom yes) (on_board yes)
-    (property "Reference" "#PWR094" (id 0) (at 118.11 86.36 0)
+  (symbol (lib_id "power:GND") (at 118.11 80.01 0)
+    (in_bom yes) (on_board yes)
+    (property "Reference" "#PWR0112" (id 0) (at 118.11 86.36 0)
       (effects (font (size 1.27 1.27)) hide)
     )
@@
     (pin "1")
   )
-  (symbol (lib_id "Device:R") (at 144.78 59.69 270) (unit 1)
-    (in_bom yes) (on_board yes)
-    (property "Reference" "R79" (id 0) (at 144.78 57.15 90))
+  (symbol (lib_id "Device:R") (at 144.78 59.69 270)
+    (in_bom yes) (on_board yes)
+    (property "Reference" "R73" (id 0) (at 144.78 57.15 90))
     (property "Value" "4m" (id 1) (at 144.78 59.69 90))
     (property "Footprint" "Resistor_SMD:R_1206_3216Metric" (id 2) (at 144.78 57.912 90)
@@
     (pin "2")
   )
-  (symbol (lib_id "Device:R") (at 118.11 74.93 0) (unit 1)
-    (in_bom yes) (on_board yes)
-    (property "Reference" "R78" (id 0) (at 119.38 74.93 0)
+  (symbol (lib_id "Device:R") (at 118.11 74.93 0)
+    (in_bom yes) (on_board yes)
+    (property "Reference" "R72" (id 0) (at 119.38 74.93 0)
       (effects (font (size 1.27 1.27)) (justify left))
     )
@@
     (pin "2")
   )
-  (symbol (lib_id "Amplifier_Current:INA138") (at 158.75 72.39 0) (unit 1)
-    (in_bom yes) (on_board yes)
-    (property "Reference" "U18" (id 0) (at 167.4876 71.2216 0)
+  (symbol (lib_id "Amplifier_Current:INA138") (at 158.75 72.39 0)
+    (in_bom yes) (on_board yes)
+    (property "Reference" "U17" (id 0) (at 167.4876 71.2216 0)
       (effects (font (size 1.27 1.27)) (justify left))
     )
@@
     (pin "5")
   )
-  (symbol (lib_id "power:VCC") (at 156.21 64.77 0) (unit 1)
-    (in_bom yes) (on_board yes)
-    (property "Reference" "#PWR096" (id 0) (at 156.21 68.58 0)
+  (symbol (lib_id "power:VCC") (at 156.21 64.77 0)
+    (in_bom yes) (on_board yes)
+    (property "Reference" "#PWR0114" (id 0) (at 156.21 68.58 0)
       (effects (font (size 1.27 1.27)) hide)
     )
@@
     (pin "1")
   )
-  (symbol (lib_id "Device:C") (at 160.02 64.77 90) (unit 1)
-    (in_bom yes) (on_board yes)
-    (property "Reference" "C39" (id 0) (at 161.29 60.96 90)
+  (symbol (lib_id "Device:C") (at 160.02 64.77 90)
+    (in_bom yes) (on_board yes)
+    (property "Reference" "C38" (id 0) (at 161.29 60.96 90)
       (effects (font (size 1.27 1.27)) (justify right))
     )
@@
     (pin "2")
   )
-  (symbol (lib_id "power:GND") (at 163.83 64.77 0) (unit 1)
-    (in_bom yes) (on_board yes)
-    (property "Reference" "#PWR097" (id 0) (at 163.83 71.12 0)
+  (symbol (lib_id "power:GND") (at 163.83 64.77 0)
+    (in_bom yes) (on_board yes)
+    (property "Reference" "#PWR0115" (id 0) (at 163.83 71.12 0)
       (effects (font (size 1.27 1.27)) hide)
     )
@@
     (pin "1")
   )
-  (symbol (lib_id "symbols:SolderJumper_4_Open") (at 118.11 39.37 0) (unit 1)
-    (in_bom yes) (on_board yes)
-    (property "Reference" "JP8" (id 0) (at 120.65 35.56 0)
+  (symbol (lib_id "symbols:SolderJumper_4_Open") (at 118.11 39.37 0)
+    (in_bom yes) (on_board yes)
+    (property "Reference" "JP7" (id 0) (at 120.65 35.56 0)
       (effects (font (size 1.27 1.27)) (justify left))
     )
@@
     (pin "4")
   )
-  (symbol (lib_id "power:+5V") (at 127 39.37 0) (unit 1)
+  (symbol (lib_id "power:+5V") (at 127 39.37 0)
     (in_bom yes) (on_board yes) (fields_autoplaced)
-    (property "Reference" "#PWR095" (id 0) (at 127 43.18 0)
+    (property "Reference" "#PWR0113" (id 0) (at 127 43.18 0)
       (effects (font (size 1.27 1.27)) hide)
     )
@@
     (pin "1")
   )
-  (symbol (lib_id "power:+3V3") (at 109.22 39.37 0) (unit 1)
+  (symbol (lib_id "power:+3V3") (at 109.22 39.37 0)
     (in_bom yes) (on_board yes) (fields_autoplaced)
-    (property "Reference" "#PWR092" (id 0) (at 109.22 43.18 0)
-      (effects (font (size 1.27 1.27)) hide)
-    )
+    (property "Reference" "#PWR0110" (id 0) (at 109.22 43.18 0)
+      (effects (font (size 1.27 1.27)) hide)
+    )

Commit message: finish battery
Parts:
- Q25: renamed from Q23; value IRF7458 -> DMP3015LSSQ
- renumbered C38 to C39, D6 to D7, JP7 to JP8, Q22 to Q24, R68 to R74, R69 to R75, R70 to R76, R71 to R77, R72 to R78, R73 to R79, U17 to U18
Changed lines of the file:
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@@
     (effects (font (size 1.27 1.27)) (justify left))
   )
-  (symbol (lib_id "Device:D") (at 189.23 63.5 270)
-    (in_bom yes) (on_board yes)
-    (property "Reference" "D6" (id 0) (at 191.262 62.3316 90)
+  (symbol (lib_id "Device:D") (at 189.23 63.5 270) (unit 1)
+    (in_bom yes) (on_board yes)
+    (property "Reference" "D7" (id 0) (at 191.262 62.3316 90)
       (effects (font (size 1.27 1.27)) (justify left))
     )
@@
     (pin "2")
   )
-  (symbol (lib_id "Device:R") (at 118.11 64.77 0)
-    (in_bom yes) (on_board yes)
-    (property "Reference" "R71" (id 0) (at 119.38 64.77 0)
+  (symbol (lib_id "Device:R") (at 118.11 64.77 0) (unit 1)
+    (in_bom yes) (on_board yes)
+    (property "Reference" "R77" (id 0) (at 119.38 64.77 0)
       (effects (font (size 1.27 1.27)) (justify left))
     )
@@
     (pin "2")
   )
-  (symbol (lib_id "power:+BATT") (at 118.11 34.29 0)
-    (in_bom yes) (on_board yes)
-    (property "Reference" "#PWR0111" (id 0) (at 118.11 38.1 0)
+  (symbol (lib_id "power:+BATT") (at 118.11 34.29 0) (unit 1)
+    (in_bom yes) (on_board yes)
+    (property "Reference" "#PWR093" (id 0) (at 118.11 38.1 0)
       (effects (font (size 1.27 1.27)) hide)
     )
@@
     (pin "1")
   )
-  (symbol (lib_id "Transistor_FET:IRF7404") (at 115.57 54.61 0) (mirror x)
-    (in_bom yes) (on_board yes)
-    (property "Reference" "Q23" (id 0) (at 120.777 55.7784 0)
-      (effects (font (size 1.27 1.27)) (justify left))
-    )
-    (property "Value" "IRF7458" (id 1) (at 120.777 53.467 0)
+  (symbol (lib_id "Transistor_FET:IRF7404") (at 115.57 54.61 0) (mirror x) (unit 1)
+    (in_bom yes) (on_board yes)
+    (property "Reference" "Q25" (id 0) (at 120.777 55.7784 0)
+      (effects (font (size 1.27 1.27)) (justify left))
+    )
+    (property "Value" "DMP3015LSSQ" (id 1) (at 120.777 53.467 0)
       (effects (font (size 1.27 1.27)) (justify left))
     )
@@
     (pin "8")
   )
-  (symbol (lib_id "Transistor_FET:2N7002") (at 104.14 63.5 0)
-    (in_bom yes) (on_board yes)
-    (property "Reference" "Q22" (id 0) (at 109.3216 62.3316 0)
+  (symbol (lib_id "Transistor_FET:2N7002") (at 104.14 63.5 0) (unit 1)
+    (in_bom yes) (on_board yes)
+    (property "Reference" "Q24" (id 0) (at 109.3216 62.3316 0)
       (effects (font (size 1.27 1.27)) (justify left))
     )
@@
     (pin "3")
   )
-  (symbol (lib_id "Device:R") (at 106.68 46.99 0)
-    (in_bom yes) (on_board yes)
-    (property "Reference" "R70" (id 0) (at 107.95 46.99 0)
+  (symbol (lib_id "Device:R") (at 106.68 46.99 0) (unit 1)
+    (in_bom yes) (on_board yes)
+    (property "Reference" "R76" (id 0) (at 107.95 46.99 0)
       (effects (font (size 1.27 1.27)) (justify left))
     )
@@
     (pin "2")
   )
-  (symbol (lib_id "Device:R") (at 90.17 63.5 270)
-    (in_bom yes) (on_board yes)
-    (property "Reference" "R68" (id 0) (at 90.17 60.96 90))
+  (symbol (lib_id "Device:R") (at 90.17 63.5 270) (unit 1)
+    (in_bom yes) (on_board yes)
+    (property "Reference" "R74" (id 0) (at 90.17 60.96 90))
     (property "Value" "100R" (id 1) (at 90.17 63.5 90))
     (property "Footprint" "Resistor_SMD:R_0805_2012Metric" (id 2) (at 90.17 61.722 90)
@@
     (pin "2")
   )
-  (symbol (lib_id "Device:R") (at 96.52 67.31 0)
-    (in_bom yes) (on_board yes)
-    (property "Reference" "R69" (id 0) (at 97.79 67.31 0)
+  (symbol (lib_id "Device:R") (at 96.52 67.31 0) (unit 1)
+    (in_bom yes) (on_board yes)
+    (property "Reference" "R75" (id 0) (at 97.79 67.31 0)
       (effects (font (size 1.27 1.27)) (justify left))
     )
@@
     (pin "2")
   )
-  (symbol (lib_id "power:GND") (at 118.11 80.01 0)
-    (in_bom yes) (on_board yes)
-    (property "Reference" "#PWR0112" (id 0) (at 118.11 86.36 0)
+  (symbol (lib_id "power:GND") (at 118.11 80.01 0) (unit 1)
+    (in_bom yes) (on_board yes)
+    (property "Reference" "#PWR094" (id 0) (at 118.11 86.36 0)
       (effects (font (size 1.27 1.27)) hide)
     )
@@
     (pin "1")
   )
-  (symbol (lib_id "Device:R") (at 144.78 59.69 270)
-    (in_bom yes) (on_board yes)
-    (property "Reference" "R73" (id 0) (at 144.78 57.15 90))
+  (symbol (lib_id "Device:R") (at 144.78 59.69 270) (unit 1)
+    (in_bom yes) (on_board yes)
+    (property "Reference" "R79" (id 0) (at 144.78 57.15 90))
     (property "Value" "4m" (id 1) (at 144.78 59.69 90))
     (property "Footprint" "Resistor_SMD:R_1206_3216Metric" (id 2) (at 144.78 57.912 90)
@@
     (pin "2")
   )
-  (symbol (lib_id "Device:R") (at 118.11 74.93 0)
-    (in_bom yes) (on_board yes)
-    (property "Reference" "R72" (id 0) (at 119.38 74.93 0)
+  (symbol (lib_id "Device:R") (at 118.11 74.93 0) (unit 1)
+    (in_bom yes) (on_board yes)
+    (property "Reference" "R78" (id 0) (at 119.38 74.93 0)
       (effects (font (size 1.27 1.27)) (justify left))
     )
@@
     (pin "2")
   )
-  (symbol (lib_id "Amplifier_Current:INA138") (at 158.75 72.39 0)
-    (in_bom yes) (on_board yes)
-    (property "Reference" "U17" (id 0) (at 167.4876 71.2216 0)
+  (symbol (lib_id "Amplifier_Current:INA138") (at 158.75 72.39 0) (unit 1)
+    (in_bom yes) (on_board yes)
+    (property "Reference" "U18" (id 0) (at 167.4876 71.2216 0)
       (effects (font (size 1.27 1.27)) (justify left))
     )
@@
     (pin "5")
   )
-  (symbol (lib_id "power:VCC") (at 156.21 64.77 0)
-    (in_bom yes) (on_board yes)
-    (property "Reference" "#PWR0114" (id 0) (at 156.21 68.58 0)
+  (symbol (lib_id "power:VCC") (at 156.21 64.77 0) (unit 1)
+    (in_bom yes) (on_board yes)
+    (property "Reference" "#PWR096" (id 0) (at 156.21 68.58 0)
       (effects (font (size 1.27 1.27)) hide)
     )
@@
     (pin "1")
   )
-  (symbol (lib_id "Device:C") (at 160.02 64.77 90)
-    (in_bom yes) (on_board yes)
-    (property "Reference" "C38" (id 0) (at 161.29 60.96 90)
+  (symbol (lib_id "Device:C") (at 160.02 64.77 90) (unit 1)
+    (in_bom yes) (on_board yes)
+    (property "Reference" "C39" (id 0) (at 161.29 60.96 90)
       (effects (font (size 1.27 1.27)) (justify right))
     )
@@
     (pin "2")
   )
-  (symbol (lib_id "power:GND") (at 163.83 64.77 0)
-    (in_bom yes) (on_board yes)
-    (property "Reference" "#PWR0115" (id 0) (at 163.83 71.12 0)
+  (symbol (lib_id "power:GND") (at 163.83 64.77 0) (unit 1)
+    (in_bom yes) (on_board yes)
+    (property "Reference" "#PWR097" (id 0) (at 163.83 71.12 0)
       (effects (font (size 1.27 1.27)) hide)
     )
@@
     (pin "1")
   )
-  (symbol (lib_id "symbols:SolderJumper_4_Open") (at 118.11 39.37 0)
-    (in_bom yes) (on_board yes)
-    (property "Reference" "JP7" (id 0) (at 120.65 35.56 0)
+  (symbol (lib_id "symbols:SolderJumper_4_Open") (at 118.11 39.37 0) (unit 1)
+    (in_bom yes) (on_board yes)
+    (property "Reference" "JP8" (id 0) (at 120.65 35.56 0)
       (effects (font (size 1.27 1.27)) (justify left))
     )
@@
     (pin "4")
   )
-  (symbol (lib_id "power:+5V") (at 127 39.37 0)
+  (symbol (lib_id "power:+5V") (at 127 39.37 0) (unit 1)
     (in_bom yes) (on_board yes) (fields_autoplaced)
-    (property "Reference" "#PWR0113" (id 0) (at 127 43.18 0)
+    (property "Reference" "#PWR095" (id 0) (at 127 43.18 0)
       (effects (font (size 1.27 1.27)) hide)
     )
@@
     (pin "1")
   )
-  (symbol (lib_id "power:+3V3") (at 109.22 39.37 0)
+  (symbol (lib_id "power:+3V3") (at 109.22 39.37 0) (unit 1)
     (in_bom yes) (on_board yes) (fields_autoplaced)
-    (property "Reference" "#PWR0110" (id 0) (at 109.22 43.18 0)
-      (effects (font (size 1.27 1.27)) hide)
-    )
+    (property "Reference" "#PWR092" (id 0) (at 109.22 43.18 0)
+      (effects (font (size 1.27 1.27)) hide)
+    )
