File: ECAD/EPS/Pulse+RetryTimer.kicad_sch (KiCad schematic)
At the start: 13 parts, among them Q21 2N7002, Q22 2N7002, U34 AD8603, U35 LTC6993xS6-4

Commit message: respec and consolidate
Parts:
- C59: renamed from C70; footprint Capacitor_SMD:C_0805_2012Metric -> Capacitor_SMD:C_1210_3225Metric
- renumbered C71 to C60, Q21 to Q19, Q22 to Q20, U34 to U33, U35 to U34
Changed lines of the file:
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@@
   (symbol (lib_id "Transistor_FET:2N7002") (at 38.1 43.18 0) (unit 1)
     (in_bom yes) (on_board yes)
-    (property "Reference" "Q21" (id 0) (at 43.2816 42.0116 0)
+    (property "Reference" "Q19" (id 0) (at 43.2816 42.0116 0)
       (effects (font (size 1.27 1.27)) (justify left))
     )
@@
   (symbol (lib_id "Amplifier_Operational:AD8603") (at 77.47 40.64 0) (unit 1)
     (in_bom yes) (on_board yes)
-    (property "Reference" "U34" (id 0) (at 86.2076 39.4716 0)
+    (property "Reference" "U33" (id 0) (at 86.2076 39.4716 0)
       (effects (font (size 1.27 1.27)) (justify left))
     )
@@
   (symbol (lib_id "Transistor_FET:2N7002") (at 99.06 40.64 0) (unit 1)
     (in_bom yes) (on_board yes)
-    (property "Reference" "Q22" (id 0) (at 104.2416 39.4716 0)
+    (property "Reference" "Q20" (id 0) (at 104.2416 39.4716 0)
       (effects (font (size 1.27 1.27)) (justify left))
     )
@@
   (symbol (lib_id "Device:C") (at 53.34 43.18 0) (unit 1)
     (in_bom yes) (on_board yes)
-    (property "Reference" "C70" (id 0) (at 56.261 42.0116 0)
+    (property "Reference" "C59" (id 0) (at 56.261 42.0116 0)
       (effects (font (size 1.27 1.27)) (justify left))
     )
@@
       (effects (font (size 1.27 1.27)) (justify left))
     )
-    (property "Footprint" "Capacitor_SMD:C_0805_2012Metric" (id 2) (at 54.3052 46.99 0)
+    (property "Footprint" "Capacitor_SMD:C_1210_3225Metric" (id 2) (at 54.3052 46.99 0)
       (effects (font (size 1.27 1.27)) hide)
     )
@@
   (symbol (lib_id "Timer:LTC6993xS6-4") (at 161.29 43.18 0) (unit 1)
     (in_bom yes) (on_board yes)
-    (property "Reference" "U35" (id 0) (at 167.64 40.64 0)
+    (property "Reference" "U34" (id 0) (at 167.64 40.64 0)
       (effects (font (size 1.27 1.27)) (justify left))
     )
@@
   (symbol (lib_id "Device:C") (at 132.08 36.83 0) (unit 1)
     (in_bom yes) (on_board yes)
-    (property "Reference" "C71" (id 0) (at 135.001 35.6616 0)
-      (effects (font (size 1.27 1.27)) (justify left))
-    )
+    (property "Reference" "C60" (id 0) (at 135.001 35.6616 0)
+      (effects (font (size 1.27 1.27)) (justify left))
+    )

Commit message: selectable voltages on PDMs
Parts:
- renumbered C59 to C61, C60 to C62, Q19 to Q21, Q20 to Q22, R82 to R89, R83 to R90, R84 to R91, R85 to R92, R86 to R93, R87 to R94, R88 to R95, U33 to U35, U34 to U36
Changed lines of the file:
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@@
   (symbol (lib_id "Transistor_FET:2N7002") (at 38.1 43.18 0) (unit 1)
     (in_bom yes) (on_board yes)
-    (property "Reference" "Q19" (id 0) (at 43.2816 42.0116 0)
+    (property "Reference" "Q21" (id 0) (at 43.2816 42.0116 0)
       (effects (font (size 1.27 1.27)) (justify left))
     )
@@
   (symbol (lib_id "Amplifier_Operational:AD8603") (at 77.47 40.64 0) (unit 1)
     (in_bom yes) (on_board yes)
-    (property "Reference" "U33" (id 0) (at 86.2076 39.4716 0)
+    (property "Reference" "U35" (id 0) (at 86.2076 39.4716 0)
       (effects (font (size 1.27 1.27)) (justify left))
     )
@@
   (symbol (lib_id "Transistor_FET:2N7002") (at 99.06 40.64 0) (unit 1)
     (in_bom yes) (on_board yes)
-    (property "Reference" "Q20" (id 0) (at 104.2416 39.4716 0)
+    (property "Reference" "Q22" (id 0) (at 104.2416 39.4716 0)
       (effects (font (size 1.27 1.27)) (justify left))
     )
@@
   (symbol (lib_id "Device:R") (at 62.23 33.02 0) (unit 1)
     (in_bom yes) (on_board yes)
-    (property "Reference" "R83" (id 0) (at 63.5 33.02 0)
+    (property "Reference" "R90" (id 0) (at 63.5 33.02 0)
       (effects (font (size 1.27 1.27)) (justify left))
     )
@@
   (symbol (lib_id "Device:R") (at 62.23 48.26 0) (unit 1)
     (in_bom yes) (on_board yes)
-    (property "Reference" "R84" (id 0) (at 63.5 48.26 0)
+    (property "Reference" "R91" (id 0) (at 63.5 48.26 0)
       (effects (font (size 1.27 1.27)) (justify left))
     )
@@
   (symbol (lib_id "power:VCC") (at 74.93 29.21 0) (unit 1)
     (in_bom yes) (on_board yes)
-    (property "Reference" "#PWR0100" (id 0) (at 74.93 33.02 0)
+    (property "Reference" "#PWR0104" (id 0) (at 74.93 33.02 0)
       (effects (font (size 1.27 1.27)) hide)
     )
@@
   (symbol (lib_id "Device:R") (at 53.34 33.02 0) (unit 1)
     (in_bom yes) (on_board yes)
-    (property "Reference" "R82" (id 0) (at 54.61 33.02 0)
+    (property "Reference" "R89" (id 0) (at 54.61 33.02 0)
       (effects (font (size 1.27 1.27)) (justify left))
     )
@@
   (symbol (lib_id "Device:C") (at 53.34 43.18 0) (unit 1)
     (in_bom yes) (on_board yes)
-    (property "Reference" "C59" (id 0) (at 56.261 42.0116 0)
+    (property "Reference" "C61" (id 0) (at 56.261 42.0116 0)
       (effects (font (size 1.27 1.27)) (justify left))
     )
@@
   (symbol (lib_id "power:GND") (at 74.93 52.07 0) (unit 1)
     (in_bom yes) (on_board yes)
-    (property "Reference" "#PWR0101" (id 0) (at 74.93 58.42 0)
+    (property "Reference" "#PWR0105" (id 0) (at 74.93 58.42 0)
       (effects (font (size 1.27 1.27)) hide)
     )
@@
   (symbol (lib_id "Timer:LTC6993xS6-4") (at 161.29 43.18 0) (unit 1)
     (in_bom yes) (on_board yes)
-    (property "Reference" "U34" (id 0) (at 167.64 40.64 0)
+    (property "Reference" "U36" (id 0) (at 167.64 40.64 0)
       (effects (font (size 1.27 1.27)) (justify left))
     )
@@
   (symbol (lib_id "power:VCC") (at 161.29 33.02 0) (unit 1)
     (in_bom yes) (on_board yes)
-    (property "Reference" "#PWR0102" (id 0) (at 161.29 36.83 0)
+    (property "Reference" "#PWR0106" (id 0) (at 161.29 36.83 0)
       (effects (font (size 1.27 1.27)) hide)
     )
@@
   (symbol (lib_id "Device:R") (at 143.51 48.26 0) (unit 1)
     (in_bom yes) (on_board yes)
-    (property "Reference" "R86" (id 0) (at 144.78 48.26 0)
+    (property "Reference" "R93" (id 0) (at 144.78 48.26 0)
       (effects (font (size 1.27 1.27)) (justify left))
     )
@@
   (symbol (lib_id "Device:R") (at 143.51 36.83 0) (unit 1)
     (in_bom yes) (on_board yes)
-    (property "Reference" "R85" (id 0) (at 144.78 36.83 0)
+    (property "Reference" "R92" (id 0) (at 144.78 36.83 0)
       (effects (font (size 1.27 1.27)) (justify left))
     )
@@
   (symbol (lib_id "Device:R") (at 151.13 49.53 0) (unit 1)
     (in_bom yes) (on_board yes)
-    (property "Reference" "R88" (id 0) (at 152.4 49.53 0)
+    (property "Reference" "R95" (id 0) (at 152.4 49.53 0)
       (effects (font (size 1.27 1.27)) (justify left))
     )
@@
   (symbol (lib_id "Device:C") (at 132.08 36.83 0) (unit 1)
     (in_bom yes) (on_board yes)
-    (property "Reference" "C60" (id 0) (at 135.001 35.6616 0)
+    (property "Reference" "C62" (id 0) (at 135.001 35.6616 0)
       (effects (font (size 1.27 1.27)) (justify left))
     )
@@
   (symbol (lib_id "Device:R") (at 148.59 38.1 0) (unit 1)
     (in_bom yes) (on_board yes)
-    (property "Reference" "R87" (id 0) (at 149.86 38.1 0)
+    (property "Reference" "R94" (id 0) (at 149.86 38.1 0)
       (effects (font (size 1.27 1.27)) (justify left))
     )
@@
   (symbol (lib_id "power:GND") (at 161.29 53.34 0) (unit 1)
     (in_bom yes) (on_board yes)
-    (property "Reference" "#PWR0103" (id 0) (at 161.29 59.69 0)
-      (effects (font (size 1.27 1.27)) hide)
-    )
+    (property "Reference" "#PWR0107" (id 0) (at 161.29 59.69 0)
+      (effects (font (size 1.27 1.27)) hide)
+    )

Commit message: push rev 2 (no more silly numbering conventions)
Parts:
- renumbered C61 to C59, C62 to C60, Q21 to Q19, Q22 to Q20, R89 to R82, R90 to R83, R91 to R84, R92 to R85, R93 to R86, R94 to R87, R95 to R88, U35 to U33, U36 to U34
Changed lines of the file:
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@@
   (title_block
     (title "TJ Custom EPS")
-    (rev "0.1")
+    (rev "2")
     (company "TJHSST Nanosatellite Club")
     (comment 4 "Engineer: Alan Hsu")
@@
   (symbol (lib_id "Transistor_FET:2N7002") (at 38.1 43.18 0) (unit 1)
     (in_bom yes) (on_board yes)
-    (property "Reference" "Q21" (id 0) (at 43.2816 42.0116 0)
+    (property "Reference" "Q19" (id 0) (at 43.2816 42.0116 0)
       (effects (font (size 1.27 1.27)) (justify left))
     )
@@
   (symbol (lib_id "Amplifier_Operational:AD8603") (at 77.47 40.64 0) (unit 1)
     (in_bom yes) (on_board yes)
-    (property "Reference" "U35" (id 0) (at 86.2076 39.4716 0)
+    (property "Reference" "U33" (id 0) (at 86.2076 39.4716 0)
       (effects (font (size 1.27 1.27)) (justify left))
     )
@@
   (symbol (lib_id "Transistor_FET:2N7002") (at 99.06 40.64 0) (unit 1)
     (in_bom yes) (on_board yes)
-    (property "Reference" "Q22" (id 0) (at 104.2416 39.4716 0)
+    (property "Reference" "Q20" (id 0) (at 104.2416 39.4716 0)
       (effects (font (size 1.27 1.27)) (justify left))
     )
@@
   (symbol (lib_id "Device:R") (at 62.23 33.02 0) (unit 1)
     (in_bom yes) (on_board yes)
-    (property "Reference" "R90" (id 0) (at 63.5 33.02 0)
+    (property "Reference" "R83" (id 0) (at 63.5 33.02 0)
       (effects (font (size 1.27 1.27)) (justify left))
     )
@@
   (symbol (lib_id "Device:R") (at 62.23 48.26 0) (unit 1)
     (in_bom yes) (on_board yes)
-    (property "Reference" "R91" (id 0) (at 63.5 48.26 0)
+    (property "Reference" "R84" (id 0) (at 63.5 48.26 0)
       (effects (font (size 1.27 1.27)) (justify left))
     )
@@
   (symbol (lib_id "power:VCC") (at 74.93 29.21 0) (unit 1)
     (in_bom yes) (on_board yes)
-    (property "Reference" "#PWR0104" (id 0) (at 74.93 33.02 0)
+    (property "Reference" "#PWR0100" (id 0) (at 74.93 33.02 0)
       (effects (font (size 1.27 1.27)) hide)
     )
@@
   (symbol (lib_id "Device:R") (at 53.34 33.02 0) (unit 1)
     (in_bom yes) (on_board yes)
-    (property "Reference" "R89" (id 0) (at 54.61 33.02 0)
+    (property "Reference" "R82" (id 0) (at 54.61 33.02 0)
       (effects (font (size 1.27 1.27)) (justify left))
     )
@@
   (symbol (lib_id "Device:C") (at 53.34 43.18 0) (unit 1)
     (in_bom yes) (on_board yes)
-    (property "Reference" "C61" (id 0) (at 56.261 42.0116 0)
+    (property "Reference" "C59" (id 0) (at 56.261 42.0116 0)
       (effects (font (size 1.27 1.27)) (justify left))
     )
@@
   (symbol (lib_id "power:GND") (at 74.93 52.07 0) (unit 1)
     (in_bom yes) (on_board yes)
-    (property "Reference" "#PWR0105" (id 0) (at 74.93 58.42 0)
+    (property "Reference" "#PWR0101" (id 0) (at 74.93 58.42 0)
       (effects (font (size 1.27 1.27)) hide)
     )
@@
   (symbol (lib_id "Timer:LTC6993xS6-4") (at 161.29 43.18 0) (unit 1)
     (in_bom yes) (on_board yes)
-    (property "Reference" "U36" (id 0) (at 167.64 40.64 0)
+    (property "Reference" "U34" (id 0) (at 167.64 40.64 0)
       (effects (font (size 1.27 1.27)) (justify left))
     )
@@
   (symbol (lib_id "power:VCC") (at 161.29 33.02 0) (unit 1)
     (in_bom yes) (on_board yes)
-    (property "Reference" "#PWR0106" (id 0) (at 161.29 36.83 0)
+    (property "Reference" "#PWR0102" (id 0) (at 161.29 36.83 0)
       (effects (font (size 1.27 1.27)) hide)
     )
@@
   (symbol (lib_id "Device:R") (at 143.51 48.26 0) (unit 1)
     (in_bom yes) (on_board yes)
-    (property "Reference" "R93" (id 0) (at 144.78 48.26 0)
+    (property "Reference" "R86" (id 0) (at 144.78 48.26 0)
       (effects (font (size 1.27 1.27)) (justify left))
     )
@@
   (symbol (lib_id "Device:R") (at 143.51 36.83 0) (unit 1)
     (in_bom yes) (on_board yes)
-    (property "Reference" "R92" (id 0) (at 144.78 36.83 0)
+    (property "Reference" "R85" (id 0) (at 144.78 36.83 0)
       (effects (font (size 1.27 1.27)) (justify left))
     )
@@
   (symbol (lib_id "Device:R") (at 151.13 49.53 0) (unit 1)
     (in_bom yes) (on_board yes)
-    (property "Reference" "R95" (id 0) (at 152.4 49.53 0)
+    (property "Reference" "R88" (id 0) (at 152.4 49.53 0)
       (effects (font (size 1.27 1.27)) (justify left))
     )
@@
   (symbol (lib_id "Device:C") (at 132.08 36.83 0) (unit 1)
     (in_bom yes) (on_board yes)
-    (property "Reference" "C62" (id 0) (at 135.001 35.6616 0)
+    (property "Reference" "C60" (id 0) (at 135.001 35.6616 0)
       (effects (font (size 1.27 1.27)) (justify left))
     )
@@
   (symbol (lib_id "Device:R") (at 148.59 38.1 0) (unit 1)
     (in_bom yes) (on_board yes)
-    (property "Reference" "R94" (id 0) (at 149.86 38.1 0)
+    (property "Reference" "R87" (id 0) (at 149.86 38.1 0)
       (effects (font (size 1.27 1.27)) (justify left))
     )
@@
   (symbol (lib_id "power:GND") (at 161.29 53.34 0) (unit 1)
     (in_bom yes) (on_board yes)
-    (property "Reference" "#PWR0107" (id 0) (at 161.29 59.69 0)
-      (effects (font (size 1.27 1.27)) hide)
-    )
+    (property "Reference" "#PWR0103" (id 0) (at 161.29 59.69 0)
+      (effects (font (size 1.27 1.27)) hide)
+    )

Commit message: layout and footprints
Parts:
- renumbered C59 to C63, C60 to C64, Q19 to Q14, Q20 to Q15, R82 to R74, R83 to R75, R84 to R76, R85 to R77, R86 to R78, R87 to R79, R88 to R80, U33 to U34, U34 to U35
Changed lines of the file:
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@@
   (symbol (lib_id "Transistor_FET:2N7002") (at 38.1 43.18 0) (unit 1)
     (in_bom yes) (on_board yes)
-    (property "Reference" "Q19" (id 0) (at 43.2816 42.0116 0)
+    (property "Reference" "Q14" (id 0) (at 43.2816 42.0116 0)
       (effects (font (size 1.27 1.27)) (justify left))
     )
@@
   (symbol (lib_id "Amplifier_Operational:AD8603") (at 77.47 40.64 0) (unit 1)
     (in_bom yes) (on_board yes)
-    (property "Reference" "U33" (id 0) (at 86.2076 39.4716 0)
+    (property "Reference" "U34" (id 0) (at 86.2076 39.4716 0)
       (effects (font (size 1.27 1.27)) (justify left))
     )
@@
   (symbol (lib_id "Transistor_FET:2N7002") (at 99.06 40.64 0) (unit 1)
     (in_bom yes) (on_board yes)
-    (property "Reference" "Q20" (id 0) (at 104.2416 39.4716 0)
+    (property "Reference" "Q15" (id 0) (at 104.2416 39.4716 0)
       (effects (font (size 1.27 1.27)) (justify left))
     )
@@
   (symbol (lib_id "Device:R") (at 62.23 33.02 0) (unit 1)
     (in_bom yes) (on_board yes)
-    (property "Reference" "R83" (id 0) (at 63.5 33.02 0)
+    (property "Reference" "R75" (id 0) (at 63.5 33.02 0)
       (effects (font (size 1.27 1.27)) (justify left))
     )
@@
   (symbol (lib_id "Device:R") (at 62.23 48.26 0) (unit 1)
     (in_bom yes) (on_board yes)
-    (property "Reference" "R84" (id 0) (at 63.5 48.26 0)
+    (property "Reference" "R76" (id 0) (at 63.5 48.26 0)
       (effects (font (size 1.27 1.27)) (justify left))
     )
@@
   (symbol (lib_id "power:VCC") (at 74.93 29.21 0) (unit 1)
     (in_bom yes) (on_board yes)
-    (property "Reference" "#PWR0100" (id 0) (at 74.93 33.02 0)
+    (property "Reference" "#PWR097" (id 0) (at 74.93 33.02 0)
       (effects (font (size 1.27 1.27)) hide)
     )
@@
   (symbol (lib_id "Device:R") (at 53.34 33.02 0) (unit 1)
     (in_bom yes) (on_board yes)
-    (property "Reference" "R82" (id 0) (at 54.61 33.02 0)
+    (property "Reference" "R74" (id 0) (at 54.61 33.02 0)
       (effects (font (size 1.27 1.27)) (justify left))
     )
@@
   (symbol (lib_id "Device:C") (at 53.34 43.18 0) (unit 1)
     (in_bom yes) (on_board yes)
-    (property "Reference" "C59" (id 0) (at 56.261 42.0116 0)
+    (property "Reference" "C63" (id 0) (at 56.261 42.0116 0)
       (effects (font (size 1.27 1.27)) (justify left))
     )
@@
   (symbol (lib_id "power:GND") (at 74.93 52.07 0) (unit 1)
     (in_bom yes) (on_board yes)
-    (property "Reference" "#PWR0101" (id 0) (at 74.93 58.42 0)
+    (property "Reference" "#PWR098" (id 0) (at 74.93 58.42 0)
       (effects (font (size 1.27 1.27)) hide)
     )
@@
   (symbol (lib_id "Timer:LTC6993xS6-4") (at 161.29 43.18 0) (unit 1)
     (in_bom yes) (on_board yes)
-    (property "Reference" "U34" (id 0) (at 167.64 40.64 0)
+    (property "Reference" "U35" (id 0) (at 167.64 40.64 0)
       (effects (font (size 1.27 1.27)) (justify left))
     )
@@
   (symbol (lib_id "power:VCC") (at 161.29 33.02 0) (unit 1)
     (in_bom yes) (on_board yes)
-    (property "Reference" "#PWR0102" (id 0) (at 161.29 36.83 0)
+    (property "Reference" "#PWR099" (id 0) (at 161.29 36.83 0)
       (effects (font (size 1.27 1.27)) hide)
     )
@@
   (symbol (lib_id "Device:R") (at 143.51 48.26 0) (unit 1)
     (in_bom yes) (on_board yes)
-    (property "Reference" "R86" (id 0) (at 144.78 48.26 0)
+    (property "Reference" "R78" (id 0) (at 144.78 48.26 0)
       (effects (font (size 1.27 1.27)) (justify left))
     )
@@
   (symbol (lib_id "Device:R") (at 143.51 36.83 0) (unit 1)
     (in_bom yes) (on_board yes)
-    (property "Reference" "R85" (id 0) (at 144.78 36.83 0)
+    (property "Reference" "R77" (id 0) (at 144.78 36.83 0)
       (effects (font (size 1.27 1.27)) (justify left))
     )
@@
   (symbol (lib_id "Device:R") (at 151.13 49.53 0) (unit 1)
     (in_bom yes) (on_board yes)
-    (property "Reference" "R88" (id 0) (at 152.4 49.53 0)
+    (property "Reference" "R80" (id 0) (at 152.4 49.53 0)
       (effects (font (size 1.27 1.27)) (justify left))
     )
@@
   (symbol (lib_id "Device:C") (at 132.08 36.83 0) (unit 1)
     (in_bom yes) (on_board yes)
-    (property "Reference" "C60" (id 0) (at 135.001 35.6616 0)
+    (property "Reference" "C64" (id 0) (at 135.001 35.6616 0)
       (effects (font (size 1.27 1.27)) (justify left))
     )
@@
   (symbol (lib_id "Device:R") (at 148.59 38.1 0) (unit 1)
     (in_bom yes) (on_board yes)
-    (property "Reference" "R87" (id 0) (at 149.86 38.1 0)
+    (property "Reference" "R79" (id 0) (at 149.86 38.1 0)
       (effects (font (size 1.27 1.27)) (justify left))
     )
@@
   (symbol (lib_id "power:GND") (at 161.29 53.34 0) (unit 1)
     (in_bom yes) (on_board yes)
-    (property "Reference" "#PWR0103" (id 0) (at 161.29 59.69 0)
-      (effects (font (size 1.27 1.27)) hide)
-    )
+    (property "Reference" "#PWR0100" (id 0) (at 161.29 59.69 0)
+      (effects (font (size 1.27 1.27)) hide)
+    )

Commit message: routing and stuff
Parts:
- removed U34: AD8603, Package_TO_SOT_SMD:TSOT-23-5, symbol Amplifier_Operational:AD8603
- added U36: (no value), symbol Amplifier_Operational:LM321
Connections:
- net GND: now also U36.2 (V-)
- net VCC: now also U36.5 (V+)
- net at C63.1, Q14.3 (D), R74.2: now also U36.1 (+)
- net at Q15.1 (G): now also U36.4
- net at R75.2, R76.1: now also U36.3 (-)
Changed lines of the file:
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@@
     (pin "3")
-  )
-  (symbol (lib_id "Amplifier_Operational:AD8603") (at 77.47 40.64 0) (unit 1)
-    (in_bom yes) (on_board yes)
-    (property "Reference" "U34" (id 0) (at 86.2076 39.4716 0)
-      (effects (font (size 1.27 1.27)) (justify left))
-    )
-    (property "Value" "AD8603" (id 1) (at 86.2076 41.783 0)
-      (effects (font (size 1.27 1.27)) (justify left))
-    )
-    (property "Footprint" "Package_TO_SOT_SMD:TSOT-23-5" (id 2) (at 77.47 40.64 0)
-      (effects (font (size 1.27 1.27)) hide)
-    )
-    (property "Datasheet" "https://www.analog.com/media/en/technical-documentation/data-sheets/AD8603_8607_8609.pdf" (id 3) (at 77.47 35.56 0)
-      (effects (font (size 1.27 1.27)) hide)
-    )
-    (pin "2")
-    (pin "5")
-    (pin "1")
-    (pin "3")
-    (pin "4")
   )
   (symbol (lib_id "Transistor_FET:2N7002") (at 99.06 40.64 0) (unit 1)
@@
     (pin "1")
   )
+  (symbol (lib_id "Amplifier_Operational:LM321") (at 77.47 40.64 0) (unit 1)
+    (in_bom yes) (on_board yes) (fields_autoplaced)
+    (property "Reference" "U36" (id 0) (at 87.63 35.941 0))
+    (property "Value" "" (id 1) (at 87.63 38.481 0))
+    (property "Footprint" "" (id 2) (at 77.47 40.64 0)
+      (effects (font (size 1.27 1.27)) hide)
+    )
+    (property "Datasheet" "http://www.ti.com/lit/ds/symlink/lm321.pdf" (id 3) (at 77.47 40.64 0)
+      (effects (font (size 1.27 1.27)) hide)
+    )
+    (pin "1")
+    (pin "2")
+    (pin "3")
+    (pin "4")
+    (pin "5")
+  )
 )
