File: ECAD/EPS/MPPT.kicad_sch (KiCad schematic)
At the start: 22 parts, among them U17 INA180A3, U18 INA180A3, U19 LM358, U20 LT3652EMSE

Commit message: respec and consolidate
Parts:
- L1: renamed from L2; value 22uH -> 10uH; footprint Inductor_SMD:L_Bourns_SRP7028A_7.3x6.6mm -> Inductor_SMD:L_AVX_LMLP07A7
- renumbered C28 to C23, C29 to C24, C30 to C25, C31 to C26, C32 to C27, D15 to D17, D16 to D18, R27 to R17, R28 to R18, R29 to R19, R30 to R20, R32 to R21, R31 to R22, R33 to R23, R34 to R24, R35 to R25, R36 to R26, U17 to U13, U18 to U14, U19 to U15, U20 to U16

Commit message: note about input
Other:
- note added: "Up to 26V input"
Changed lines of the file:
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@@
+    (effects (font (size 1.27 1.27)) (justify left bottom))
+  )
+  (text "Up to 26V input" (at 15.24 41.91 90)
     (effects (font (size 1.27 1.27)) (justify left bottom))
   )

Commit message: layout and footprints
Parts:
- renumbered C23 to C27, C24 to C28, C25 to C29, C26 to C30, C27 to C31, R17 to R13, R18 to R14, R19 to R15, R20 to R16, R21 to R17, R22 to R18, R23 to R19, R24 to R20, R25 to R21, R26 to R22
Changed lines of the file:
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@@
   (symbol (lib_id "Device:R") (at 80.01 40.64 0) (unit 1)
     (in_bom yes) (on_board yes)
-    (property "Reference" "R19" (id 0) (at 81.28 40.64 0)
+    (property "Reference" "R15" (id 0) (at 81.28 40.64 0)
       (effects (font (size 1.27 1.27)) (justify left))
     )
@@
   (symbol (lib_id "Device:R") (at 80.01 55.88 0) (unit 1)
     (in_bom yes) (on_board yes)
-    (property "Reference" "R20" (id 0) (at 81.28 55.88 0)
+    (property "Reference" "R16" (id 0) (at 81.28 55.88 0)
       (effects (font (size 1.27 1.27)) (justify left))
     )
@@
   (symbol (lib_id "Device:R") (at 128.27 39.37 0) (unit 1)
     (in_bom yes) (on_board yes)
-    (property "Reference" "R21" (id 0) (at 129.54 39.37 0)
+    (property "Reference" "R17" (id 0) (at 129.54 39.37 0)
       (effects (font (size 1.27 1.27)) (justify left))
     )
@@
   (symbol (lib_id "Device:R") (at 128.27 59.69 0) (unit 1)
     (in_bom yes) (on_board yes)
-    (property "Reference" "R22" (id 0) (at 129.54 59.69 0)
+    (property "Reference" "R18" (id 0) (at 129.54 59.69 0)
       (effects (font (size 1.27 1.27)) (justify left))
     )
@@
   (symbol (lib_id "power:GND") (at 128.27 64.77 0) (unit 1)
     (in_bom yes) (on_board yes)
-    (property "Reference" "#PWR057" (id 0) (at 128.27 71.12 0)
+    (property "Reference" "#PWR053" (id 0) (at 128.27 71.12 0)
       (effects (font (size 1.27 1.27)) hide)
     )
@@
   (symbol (lib_id "Device:C") (at 152.4 38.1 0) (unit 1)
     (in_bom yes) (on_board yes)
-    (property "Reference" "C25" (id 0) (at 155.321 36.9316 0)
+    (property "Reference" "C29" (id 0) (at 155.321 36.9316 0)
       (effects (font (size 1.27 1.27)) (justify left))
     )
@@
   (symbol (lib_id "Device:R") (at 193.04 57.15 270) (unit 1)
     (in_bom yes) (on_board yes)
-    (property "Reference" "R23" (id 0) (at 193.04 54.61 90))
+    (property "Reference" "R19" (id 0) (at 193.04 54.61 90))
     (property "Value" "52.8K" (id 1) (at 193.04 57.15 90))
     (property "Footprint" "Resistor_SMD:R_0805_2012Metric" (id 2) (at 193.04 55.372 90)
@@
   (symbol (lib_id "Device:R") (at 198.12 60.96 180) (unit 1)
     (in_bom yes) (on_board yes)
-    (property "Reference" "R25" (id 0) (at 199.39 60.96 0)
+    (property "Reference" "R21" (id 0) (at 199.39 60.96 0)
       (effects (font (size 1.27 1.27)) (justify right))
     )
@@
   (symbol (lib_id "Device:R") (at 198.12 53.34 180) (unit 1)
     (in_bom yes) (on_board yes)
-    (property "Reference" "R24" (id 0) (at 199.39 53.34 0)
+    (property "Reference" "R20" (id 0) (at 199.39 53.34 0)
       (effects (font (size 1.27 1.27)) (justify right))
     )
@@
   (symbol (lib_id "Device:C") (at 191.77 40.64 0) (unit 1)
     (in_bom yes) (on_board yes)
-    (property "Reference" "C26" (id 0) (at 191.77 38.1 0)
+    (property "Reference" "C30" (id 0) (at 191.77 38.1 0)
       (effects (font (size 1.27 1.27)) (justify left))
     )
@@
   (symbol (lib_id "power:GND") (at 199.39 31.75 0) (unit 1)
     (in_bom yes) (on_board yes)
-    (property "Reference" "#PWR058" (id 0) (at 199.39 38.1 0)
+    (property "Reference" "#PWR054" (id 0) (at 199.39 38.1 0)
       (effects (font (size 1.27 1.27)) hide)
     )
@@
   (symbol (lib_id "Device:R") (at 214.63 46.99 270) (unit 1)
     (in_bom yes) (on_board yes)
-    (property "Reference" "R26" (id 0) (at 218.44 44.45 90))
+    (property "Reference" "R22" (id 0) (at 218.44 44.45 90))
     (property "Value" "50m" (id 1) (at 214.63 46.99 90))
     (property "Footprint" "Resistor_SMD:R_2512_6332Metric" (id 2) (at 214.63 45.212 90)
@@
   (symbol (lib_id "Device:C") (at 209.55 53.34 0) (unit 1)
     (in_bom yes) (on_board yes)
-    (property "Reference" "C27" (id 0) (at 212.471 52.1716 0)
+    (property "Reference" "C31" (id 0) (at 212.471 52.1716 0)
       (effects (font (size 1.27 1.27)) (justify left))
     )
@@
   (symbol (lib_id "power:GND") (at 39.37 39.37 0) (unit 1)
     (in_bom yes) (on_board yes)
-    (property "Reference" "#PWR051" (id 0) (at 39.37 45.72 0)
+    (property "Reference" "#PWR047" (id 0) (at 39.37 45.72 0)
       (effects (font (size 1.27 1.27)) hide)
     )
@@
   (symbol (lib_id "Device:R") (at 27.94 19.05 270) (unit 1)
     (in_bom yes) (on_board yes)
-    (property "Reference" "R17" (id 0) (at 27.94 16.51 90))
+    (property "Reference" "R13" (id 0) (at 27.94 16.51 90))
     (property "Value" "4m" (id 1) (at 27.94 19.05 90))
     (property "Footprint" "Resistor_SMD:R_1206_3216Metric" (id 2) (at 27.94 17.272 90)
@@
   (symbol (lib_id "Device:C") (at 43.18 24.13 90) (unit 1)
     (in_bom yes) (on_board yes)
-    (property "Reference" "C23" (id 0) (at 44.45 20.32 90)
+    (property "Reference" "C27" (id 0) (at 44.45 20.32 90)
       (effects (font (size 1.27 1.27)) (justify right))
     )
@@
   (symbol (lib_id "power:GND") (at 46.99 24.13 0) (unit 1)
     (in_bom yes) (on_board yes)
-    (property "Reference" "#PWR054" (id 0) (at 46.99 30.48 0)
+    (property "Reference" "#PWR050" (id 0) (at 46.99 30.48 0)
       (effects (font (size 1.27 1.27)) hide)
     )
@@
   (symbol (lib_id "power:+3.3VA") (at 39.37 24.13 0) (unit 1)
     (in_bom yes) (on_board yes)
-    (property "Reference" "#PWR050" (id 0) (at 39.37 27.94 0)
+    (property "Reference" "#PWR046" (id 0) (at 39.37 27.94 0)
       (effects (font (size 1.27 1.27)) hide)
     )
@@
   (symbol (lib_id "power:GND") (at 39.37 66.04 0) (unit 1)
     (in_bom yes) (on_board yes)
-    (property "Reference" "#PWR053" (id 0) (at 39.37 72.39 0)
+    (property "Reference" "#PWR049" (id 0) (at 39.37 72.39 0)
       (effects (font (size 1.27 1.27)) hide)
     )
@@
   (symbol (lib_id "Device:R") (at 27.94 45.72 270) (unit 1)
     (in_bom yes) (on_board yes)
-    (property "Reference" "R18" (id 0) (at 27.94 43.18 90))
+    (property "Reference" "R14" (id 0) (at 27.94 43.18 90))
     (property "Value" "4m" (id 1) (at 27.94 45.72 90))
     (property "Footprint" "Resistor_SMD:R_1206_3216Metric" (id 2) (at 27.94 43.942 90)
@@
   (symbol (lib_id "Device:C") (at 43.18 50.8 90) (unit 1)
     (in_bom yes) (on_board yes)
-    (property "Reference" "C24" (id 0) (at 44.45 46.99 90)
+    (property "Reference" "C28" (id 0) (at 44.45 46.99 90)
       (effects (font (size 1.27 1.27)) (justify right))
     )
@@
   (symbol (lib_id "power:GND") (at 46.99 50.8 0) (unit 1)
     (in_bom yes) (on_board yes)
-    (property "Reference" "#PWR055" (id 0) (at 46.99 57.15 0)
+    (property "Reference" "#PWR051" (id 0) (at 46.99 57.15 0)
       (effects (font (size 1.27 1.27)) hide)
     )
@@
   (symbol (lib_id "power:+3.3VA") (at 39.37 50.8 0) (unit 1)
     (in_bom yes) (on_board yes)
-    (property "Reference" "#PWR052" (id 0) (at 39.37 54.61 0)
+    (property "Reference" "#PWR048" (id 0) (at 39.37 54.61 0)
       (effects (font (size 1.27 1.27)) hide)
     )
@@
   (symbol (lib_id "power:+3.3VA") (at 118.11 49.53 0) (unit 1)
     (in_bom yes) (on_board yes)
-    (property "Reference" "#PWR056" (id 0) (at 118.11 53.34 0)
-      (effects (font (size 1.27 1.27)) hide)
-    )
+    (property "Reference" "#PWR052" (id 0) (at 118.11 53.34 0)
+      (effects (font (size 1.27 1.27)) hide)
+    )

Commit message: routing and stuff
Parts:
- removed U15: LM358, Package_SO:SO-8_3.9x4.9mm_P1.27mm, symbol Amplifier_Operational:LM358
- added U?: (no value), symbol Amplifier_Operational:LM321
Connections:
- net +3.3VA: now also U?.5 (V+)
- net GND: now also U?.2 (V-)
- net TELEM_VIN: now also R15.2, R16.1
- net Vset: now also U?.3 (-)
- net at U16.2 (VIN_REG): now also U?.4
- net at R17.2, R18.1: now also U?.1 (+)
Other:
- moved on the sheet: C29, C30, C31, D17, D18, L1, R17, R18, R19, R20, R21, R22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

Commit message: move solar to daughterboard... again. Also replace all 0603 resistor with 0805
Parts:
- C10: renamed from C27; value 0.1uF -> (none); footprint Capacitor_SMD:C_0603_1608Metric -> (none)
- C11: renamed from C28; value 0.1uF -> (none); footprint Capacitor_SMD:C_0603_1608Metric -> (none)
- C12: renamed from C29; value 10uF -> (none); footprint Capacitor_SMD:C_0805_2012Metric -> (none)
- C13: renamed from C30; value 1uF -> (none); footprint Capacitor_SMD:C_0805_2012Metric -> (none)
- C14: renamed from C31; value 10uF -> (none); footprint Capacitor_SMD:C_0805_2012Metric -> (none)
- D17: value CMSH3-40MA -> (none); footprint Diode_SMD:D_SMA -> (none)
- D18: value RB051MM-2Y -> (none); footprint Diode_SMD:D_SOD-123F -> (none)
- L1: value 10uH -> (none); footprint Inductor_SMD:L_AVX_LMLP07A7 -> (none)
- R10: renamed from R19; value 52.8K -> (none); footprint Resistor_SMD:R_0805_2012Metric -> (none)
- R11: renamed from R20; value 490K -> (none); footprint Resistor_SMD:R_0805_2012Metric -> (none)
- R12: renamed from R21; value 330K -> (none); footprint Resistor_SMD:R_0805_2012Metric -> (none)
- R13: renamed from R22; value 50m -> (none); footprint Resistor_SMD:R_2512_6332Metric -> (none)
- R4: renamed from R13; value 4m -> (none); footprint Resistor_SMD:R_1206_3216Metric -> (none)
- R5: renamed from R14; value 4m -> (none); footprint Resistor_SMD:R_1206_3216Metric -> (none)
- R6: renamed from R15; value 750K -> (none); footprint Resistor_SMD:R_0805_2012Metric -> (none)
- R7: renamed from R16; value 100K -> (none); footprint Resistor_SMD:R_0805_2012Metric -> (none)
- R8: renamed from R17; value 75K -> (none); footprint Resistor_SMD:R_0805_2012Metric -> (none)
- R9: renamed from R18; value 10K -> (none); footprint Resistor_SMD:R_0805_2012Metric -> (none)
- U10: renamed from U13; value INA180A3 -> (none); footprint Package_TO_SOT_SMD:SOT-23-5 -> (none)
- U11: renamed from U14; value INA180A3 -> (none); footprint Package_TO_SOT_SMD:SOT-23-5 -> (none)
- U13: renamed from U16; value LT3652EMSE -> (none); footprint Package_SO:MSOP-12-1EP_3x4mm_P0.65mm_EP1.65x2.85mm -> (none)
- gave numbers to parts that had none: 1

Commit message: flip PDM current monitors
Parts:
- C10, C11: value (none) -> 0.1uF; footprint (none) -> Capacitor_SMD:C_0603_1608Metric
- C12, C14: value (none) -> 10uF; footprint (none) -> Capacitor_SMD:C_0805_2012Metric
- C13: value (none) -> 1uF; footprint (none) -> Capacitor_SMD:C_0805_2012Metric
- D17: value (none) -> CMSH3-40MA; footprint (none) -> Diode_SMD:D_SMA
- D18: value (none) -> RB051MM-2Y; footprint (none) -> Diode_SMD:D_SOD-123F
- L1: value (none) -> 10uH; footprint (none) -> Inductor_SMD:L_AVX_LMLP07A7
- R10: value (none) -> 52.8K; footprint (none) -> Resistor_SMD:R_0805_2012Metric
- R11: value (none) -> 490K; footprint (none) -> Resistor_SMD:R_0805_2012Metric
- R12: value (none) -> 330K; footprint (none) -> Resistor_SMD:R_0805_2012Metric
- R13: value (none) -> 50m; footprint (none) -> Resistor_SMD:R_2512_6332Metric
- R4, R5: value (none) -> 4m; footprint (none) -> Resistor_SMD:R_1206_3216Metric
- R6: value (none) -> 750K; footprint (none) -> Resistor_SMD:R_0805_2012Metric
- R7: value (none) -> 100K; footprint (none) -> Resistor_SMD:R_0805_2012Metric
- R8: value (none) -> 75K; footprint (none) -> Resistor_SMD:R_0805_2012Metric
- R9: value (none) -> 10K; footprint (none) -> Resistor_SMD:R_0805_2012Metric
- U10, U11: value (none) -> INA180A3; footprint (none) -> Package_TO_SOT_SMD:SOT-23-5
- U12: value (none) -> LM321; footprint (none) -> Package_TO_SOT_SMD:SOT-23-5
- U13: value (none) -> LT3652EMSE; footprint (none) -> Package_SO:MSOP-12-1EP_3x4mm_P0.65mm_EP1.65x2.85mm

Commit message: add parts and work on battery
Parts:
- removed U12: LM321, Package_TO_SOT_SMD:SOT-23-5, symbol Amplifier_Operational:LM321
- added U12: TLV9361IDBVR, symbol Amplifier_Operational:OPA842xDBV
Connections:
- net +3.3VA: now also U12.5 (V+)
- net GND: now also U12.2 (V-)
- net Vset: now also U12.4 (-)
- net at U13.2 (VIN_REG): now also U12.1
- net at R8.2, R9.1: now also U12.3 (+)
Changed lines of the file:
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@@
     (pin "1")
   )
-  (symbol (lib_id "Amplifier_Operational:LM321") (at 107.95 46.99 0) (unit 1)
-    (in_bom yes) (on_board yes) (fields_autoplaced)
-    (property "Reference" "U12" (id 0) (at 118.11 42.291 0))
-    (property "Value" "LM321" (id 1) (at 118.11 44.831 0))
-    (property "Footprint" "Package_TO_SOT_SMD:SOT-23-5" (id 2) (at 107.95 46.99 0)
+  (symbol (lib_id "Amplifier_Operational:OPA842xDBV") (at 107.95 46.99 0) (unit 1)
+    (in_bom yes) (on_board yes)
+    (property "Reference" "U12" (id 0) (at 105.41 53.34 0)
+      (effects (font (size 1.27 1.27)) (justify left))
+    )
+    (property "Value" "TLV9361IDBVR" (id 1) (at 105.41 55.88 0)
+      (effects (font (size 1.27 1.27)) (justify left))
+    )
+    (property "Footprint" "" (id 2) (at 105.41 52.07 0)
+      (effects (font (size 1.27 1.27)) (justify left) hide)
+    )
+    (property "Datasheet" "http://www.ti.com/lit/ds/symlink/opa842.pdf" (id 3) (at 107.95 41.91 0)
       (effects (font (size 1.27 1.27)) hide)
     )
-    (property "Datasheet" "http://www.ti.com/lit/ds/symlink/lm321.pdf" (id 3) (at 107.95 46.99 0)
-      (effects (font (size 1.27 1.27)) hide)
-    )
+    (pin "2")
+    (pin "5")
     (pin "1")
-    (pin "2")
     (pin "3")
     (pin "4")
-    (pin "5")
   )
 )
