File: ECAD/EPS/MPPT.kicad_sch (KiCad schematic)
At the start: 22 parts, among them U10 INA180A3, U11 INA180A3, U12 TLV9361IDBVR, U13 LT3652EMSE

Commit message: finish battery
Parts:
- U12: footprint (none) -> Package_TO_SOT_SMD:SOT-23-5
Changed lines of the file:
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@@
       (effects (font (size 1.27 1.27)) (justify left))
     )
-    (property "Footprint" "" (id 2) (at 105.41 52.07 0)
+    (property "Footprint" "Package_TO_SOT_SMD:SOT-23-5" (id 2) (at 105.41 52.07 0)
       (effects (font (size 1.27 1.27)) (justify left) hide)
     )

Commit message: solar route
Parts:
- removed R6: 750K, Resistor_SMD:R_0805_2012Metric, symbol Device:R
- removed R7: 100K, Resistor_SMD:R_0805_2012Metric, symbol Device:R
- C10, C11: footprint Capacitor_SMD:C_0603_1608Metric -> (none)
- R11: renamed from R13; footprint Resistor_SMD:R_2512_6332Metric -> (none)
- renumbered D17 to D18, D18 to D19, R12 to R10, R8 to R6, R9 to R7, R10 to R8, R11 to R9
Connections:
- net TELEM_VIN: now also R6.2, R7.1, U12.3 (+)
Changed lines of the file:
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@@
   (junction (at 31.75 45.72) (diameter 0) (color 0 0 0 0)
-  )
-  (junction (at 80.01 34.29) (diameter 0) (color 0 0 0 0)
   )
   (junction (at 171.45 49.53) (diameter 0) (color 0 0 0 0)
@@
     (stroke (width 0) (type default) (color 0 0 0 0))
   )
+  (wire (pts (xy 92.71 44.45) (xy 97.79 44.45))
+    (stroke (width 0) (type default) (color 0 0 0 0))
+  )
   (wire (pts (xy 24.13 19.05) (xy 22.86 21.59))
     (stroke (width 0) (type default) (color 0 0 0 0))
   )
-  (wire (pts (xy 80.01 34.29) (xy 97.79 34.29))
+  (wire (pts (xy 74.93 34.29) (xy 97.79 34.29))
     (stroke (width 0) (type default) (color 0 0 0 0))
   )
@@
     (stroke (width 0) (type default) (color 0 0 0 0))
   )
-  (wire (pts (xy 80.01 36.83) (xy 80.01 34.29))
-    (stroke (width 0) (type default) (color 0 0 0 0))
-  )
   (wire (pts (xy 179.07 49.53) (xy 182.88 49.53))
     (stroke (width 0) (type default) (color 0 0 0 0))
   )
-  (wire (pts (xy 80.01 44.45) (xy 80.01 52.07))
-    (stroke (width 0) (type default) (color 0 0 0 0))
-  )
   (wire (pts (xy 182.88 38.1) (xy 182.88 36.83))
     (stroke (width 0) (type default) (color 0 0 0 0))
@@
     (stroke (width 0) (type default) (color 0 0 0 0))
   )
-  (wire (pts (xy 80.01 64.77) (xy 97.79 64.77))
-    (stroke (width 0) (type default) (color 0 0 0 0))
-  )
   (wire (pts (xy 31.75 45.72) (xy 74.93 45.72))
     (stroke (width 0) (type default) (color 0 0 0 0))
@@
     (stroke (width 0) (type default) (color 0 0 0 0))
   )
-  (wire (pts (xy 80.01 59.69) (xy 80.01 64.77))
-    (stroke (width 0) (type default) (color 0 0 0 0))
-  )
   (wire (pts (xy 33.02 60.96) (xy 34.29 60.96))
     (stroke (width 0) (type default) (color 0 0 0 0))
@@
   )
   (wire (pts (xy 191.77 46.99) (xy 200.66 46.99))
-    (stroke (width 0) (type default) (color 0 0 0 0))
-  )
-  (wire (pts (xy 80.01 34.29) (xy 74.93 34.29))
     (stroke (width 0) (type default) (color 0 0 0 0))
   )
@@
     (effects (font (size 1.27 1.27)) (justify right))
   )
-  (hierarchical_label "TELEM_VIN" (shape input) (at 80.01 46.99 0)
-    (effects (font (size 1.27 1.27)) (justify left))
+  (hierarchical_label "TELEM_VIN" (shape input) (at 92.71 44.45 180)
+    (effects (font (size 1.27 1.27)) (justify right))
   )
   (hierarchical_label "TELEM_I_A" (shape input) (at 58.42 31.75 0)
     (effects (font (size 1.27 1.27)) (justify left))
-  )
-  (symbol (lib_id "Device:R") (at 80.01 40.64 0) (unit 1)
-    (in_bom yes) (on_board yes)
-    (property "Reference" "R6" (id 0) (at 81.28 40.64 0)
-      (effects (font (size 1.27 1.27)) (justify left))
-    )
-    (property "Value" "750K" (id 1) (at 80.01 43.18 90)
-      (effects (font (size 1.27 1.27)) (justify left))
-    )
-    (property "Footprint" "Resistor_SMD:R_0805_2012Metric" (id 2) (at 78.232 40.64 90)
-      (effects (font (size 1.27 1.27)) hide)
-    )
-    (property "Datasheet" "~" (id 3) (at 80.01 40.64 0)
-      (effects (font (size 1.27 1.27)) hide)
-    )
-    (pin "1")
-    (pin "2")
-  )
-  (symbol (lib_id "Device:R") (at 80.01 55.88 0) (unit 1)
-    (in_bom yes) (on_board yes)
-    (property "Reference" "R7" (id 0) (at 81.28 55.88 0)
-      (effects (font (size 1.27 1.27)) (justify left))
-    )
-    (property "Value" "100K" (id 1) (at 80.01 58.42 90)
-      (effects (font (size 1.27 1.27)) (justify left))
-    )
-    (property "Footprint" "Resistor_SMD:R_0805_2012Metric" (id 2) (at 78.232 55.88 90)
-      (effects (font (size 1.27 1.27)) hide)
-    )
-    (property "Datasheet" "~" (id 3) (at 80.01 55.88 0)
-      (effects (font (size 1.27 1.27)) hide)
-    )
-    (pin "1")
-    (pin "2")
   )
   (symbol (lib_id "Battery_Management:LT3652EMSE") (at 148.59 46.99 0) (unit 1)
@@
   (symbol (lib_id "Device:R") (at 97.79 39.37 0) (unit 1)
     (in_bom yes) (on_board yes)
-    (property "Reference" "R8" (id 0) (at 99.06 39.37 0)
+    (property "Reference" "R6" (id 0) (at 99.06 39.37 0)
       (effects (font (size 1.27 1.27)) (justify left))
     )
@@
   (symbol (lib_id "Device:R") (at 97.79 59.69 0) (unit 1)
     (in_bom yes) (on_board yes)
-    (property "Reference" "R9" (id 0) (at 99.06 59.69 0)
+    (property "Reference" "R7" (id 0) (at 99.06 59.69 0)
       (effects (font (size 1.27 1.27)) (justify left))
     )
@@
   (symbol (lib_id "power:GND") (at 97.79 64.77 0) (unit 1)
     (in_bom yes) (on_board yes)
-    (property "Reference" "#PWR026" (id 0) (at 97.79 71.12 0)
+    (property "Reference" "#PWR028" (id 0) (at 97.79 71.12 0)
       (effects (font (size 1.27 1.27)) hide)
     )
@@
   (symbol (lib_id "Device:R") (at 166.37 57.15 270) (unit 1)
     (in_bom yes) (on_board yes)
-    (property "Reference" "R10" (id 0) (at 166.37 54.61 90))
+    (property "Reference" "R8" (id 0) (at 166.37 54.61 90))
     (property "Value" "52.8K" (id 1) (at 166.37 57.15 90))
     (property "Footprint" "Resistor_SMD:R_0805_2012Metric" (id 2) (at 166.37 55.372 90)
@@
   (symbol (lib_id "Device:R") (at 171.45 60.96 180) (unit 1)
     (in_bom yes) (on_board yes)
-    (property "Reference" "R12" (id 0) (at 172.72 60.96 0)
+    (property "Reference" "R10" (id 0) (at 172.72 60.96 0)
       (effects (font (size 1.27 1.27)) (justify right))
     )
@@
   (symbol (lib_id "Device:R") (at 171.45 53.34 180) (unit 1)
     (in_bom yes) (on_board yes)
-    (property "Reference" "R11" (id 0) (at 172.72 53.34 0)
+    (property "Reference" "R9" (id 0) (at 172.72 53.34 0)
       (effects (font (size 1.27 1.27)) (justify right))
     )
@@
   (symbol (lib_id "Device:D_Schottky") (at 175.26 44.45 0) (unit 1)
     (in_bom yes) (on_board yes)
-    (property "Reference" "D18" (id 0) (at 175.26 38.9382 0))
+    (property "Reference" "D19" (id 0) (at 175.26 38.9382 0))
     (property "Value" "RB051MM-2Y" (id 1) (at 175.26 41.2496 0))
     (property "Footprint" "Diode_SMD:D_SOD-123F" (id 2) (at 175.26 44.45 0)
@@
   (symbol (lib_id "Device:D_Schottky") (at 168.91 31.75 0) (unit 1)
     (in_bom yes) (on_board yes)
-    (property "Reference" "D17" (id 0) (at 168.91 26.2382 0))
+    (property "Reference" "D18" (id 0) (at 168.91 26.2382 0))
     (property "Value" "CMSH3-40MA" (id 1) (at 168.91 28.5496 0))
     (property "Footprint" "Diode_SMD:D_SMA" (id 2) (at 168.91 31.75 0)
@@
   (symbol (lib_id "power:GND") (at 172.72 31.75 0) (unit 1)
     (in_bom yes) (on_board yes)
-    (property "Reference" "#PWR028" (id 0) (at 172.72 38.1 0)
+    (property "Reference" "#PWR030" (id 0) (at 172.72 38.1 0)
       (effects (font (size 1.27 1.27)) hide)
     )
@@
   (symbol (lib_id "Device:R") (at 187.96 46.99 270) (unit 1)
     (in_bom yes) (on_board yes)
-    (property "Reference" "R13" (id 0) (at 191.77 44.45 90))
+    (property "Reference" "R11" (id 0) (at 191.77 44.45 90))
     (property "Value" "50m" (id 1) (at 187.96 46.99 90))
-    (property "Footprint" "Resistor_SMD:R_2512_6332Metric" (id 2) (at 187.96 45.212 90)
+    (property "Footprint" "" (id 2) (at 187.96 45.212 90)
       (effects (font (size 1.27 1.27)) hide)
     )
@@
   (symbol (lib_id "power:GND") (at 39.37 39.37 0) (unit 1)
     (in_bom yes) (on_board yes)
-    (property "Reference" "#PWR021" (id 0) (at 39.37 45.72 0)
+    (property "Reference" "#PWR023" (id 0) (at 39.37 45.72 0)
       (effects (font (size 1.27 1.27)) hide)
     )
@@
       (effects (font (size 1.27 1.27)) (justify right))
     )
-    (property "Footprint" "Capacitor_SMD:C_0603_1608Metric" (id 2) (at 46.99 23.1648 0)
+    (property "Footprint" "" (id 2) (at 46.99 23.1648 0)
       (effects (font (size 1.27 1.27)) hide)
     )
@@
   (symbol (lib_id "power:GND") (at 46.99 24.13 0) (unit 1)
     (in_bom yes) (on_board yes)
-    (property "Reference" "#PWR024" (id 0) (at 46.99 30.48 0)
+    (property "Reference" "#PWR026" (id 0) (at 46.99 30.48 0)
       (effects (font (size 1.27 1.27)) hide)
     )
@@
   (symbol (lib_id "power:+3.3VA") (at 39.37 24.13 0) (unit 1)
     (in_bom yes) (on_board yes)
-    (property "Reference" "#PWR020" (id 0) (at 39.37 27.94 0)
+    (property "Reference" "#PWR022" (id 0) (at 39.37 27.94 0)
       (effects (font (size 1.27 1.27)) hide)
     )
@@
   (symbol (lib_id "power:GND") (at 39.37 66.04 0) (unit 1)
     (in_bom yes) (on_board yes)
-    (property "Reference" "#PWR023" (id 0) (at 39.37 72.39 0)
+    (property "Reference" "#PWR025" (id 0) (at 39.37 72.39 0)
       (effects (font (size 1.27 1.27)) hide)
     )
@@
       (effects (font (size 1.27 1.27)) (justify right))
     )
-    (property "Footprint" "Capacitor_SMD:C_0603_1608Metric" (id 2) (at 46.99 49.8348 0)
+    (property "Footprint" "" (id 2) (at 46.99 49.8348 0)
       (effects (font (size 1.27 1.27)) hide)
     )
@@
   (symbol (lib_id "power:GND") (at 46.99 50.8 0) (unit 1)
     (in_bom yes) (on_board yes)
-    (property "Reference" "#PWR025" (id 0) (at 46.99 57.15 0)
+    (property "Reference" "#PWR027" (id 0) (at 46.99 57.15 0)
       (effects (font (size 1.27 1.27)) hide)
     )
@@
   (symbol (lib_id "power:+3.3VA") (at 39.37 50.8 0) (unit 1)
     (in_bom yes) (on_board yes)
-    (property "Reference" "#PWR022" (id 0) (at 39.37 54.61 0)
+    (property "Reference" "#PWR024" (id 0) (at 39.37 54.61 0)
       (effects (font (size 1.27 1.27)) hide)
     )
@@
   (symbol (lib_id "power:+3.3VA") (at 105.41 39.37 0) (unit 1)
     (in_bom yes) (on_board yes)
-    (property "Reference" "#PWR027" (id 0) (at 105.41 43.18 0)
-      (effects (font (size 1.27 1.27)) hide)
-    )
+    (property "Reference" "#PWR029" (id 0) (at 105.41 43.18 0)
+      (effects (font (size 1.27 1.27)) hide)
+    )

Commit message: solar footprint work
Parts:
- removed U12: TLV9361IDBVR, Package_TO_SOT_SMD:SOT-23-5, symbol Amplifier_Operational:OPA842xDBV
- added RV1: 100K, footprints:Bourns PVG3A, symbol Device:R_Potentiometer_Trim
- added TP1: VIN, TestPoint:TestPoint_2Pads_Pitch2.54mm_Drill0.8mm, symbol Connector:TestPoint_2Pole
- added TP2: Vmpp, TestPoint:TestPoint_Pad_2.0x2.0mm, symbol Connector:TestPoint
- C6: renamed from C10; footprint (none) -> Capacitor_SMD:C_0805_2012Metric
- C7: renamed from C11; footprint (none) -> Capacitor_SMD:C_0805_2012Metric
- R11: footprint (none) -> Resistor_SMD:R_1206_3216Metric
- renumbered C14 to C10, C12 to C8, C13 to C9, D19 to D10, D18 to D9, U10 to U5, U11 to U6, U13 to U7
Connections:
- net GND: now also RV1.3, TP1.1
- net at C8.1, R4.1, R5.1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: now also RV1.1, TP1.2
- net at U7.2 (VIN_REG): now also RV1.2, TP2.1
- net +3.3VA renamed VDD
Other:
- moved on the sheet: R6, R7

Commit message: descope solar LV input
Parts:
- renumbered U5 to U4, U6 to U5, U7 to U6
Changed lines of the file:
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@@
   (symbol (lib_id "Battery_Management:LT3652EMSE") (at 148.59 46.99 0) (unit 1)
     (in_bom yes) (on_board yes)
-    (property "Reference" "U7" (id 0) (at 148.59 29.6926 0))
+    (property "Reference" "U6" (id 0) (at 148.59 29.6926 0))
     (property "Value" "LT3652EMSE" (id 1) (at 148.59 32.004 0))
     (property "Footprint" "Package_SO:MSOP-12-1EP_3x4mm_P0.65mm_EP1.65x2.85mm" (id 2) (at 148.59 62.23 0)
@@
   (symbol (lib_id "Amplifier_Current:INA138") (at 41.91 31.75 0) (unit 1)
     (in_bom yes) (on_board yes)
-    (property "Reference" "U5" (id 0) (at 50.6476 30.5816 0)
+    (property "Reference" "U4" (id 0) (at 50.6476 30.5816 0)
       (effects (font (size 1.27 1.27)) (justify left))
     )
@@
   (symbol (lib_id "Amplifier_Current:INA138") (at 41.91 58.42 0) (unit 1)
     (in_bom yes) (on_board yes)
-    (property "Reference" "U6" (id 0) (at 50.6476 57.2516 0)
-      (effects (font (size 1.27 1.27)) (justify left))
-    )
+    (property "Reference" "U5" (id 0) (at 50.6476 57.2516 0)
+      (effects (font (size 1.27 1.27)) (justify left))
+    )

Commit message: value editing
Parts:
- R10: value 330K -> (none)
- R8: value 52.8K -> (none)
- R9: value 490K -> (none)
Other:
- note added: "Float voltage selection 8.27V Rbottom/Rtop = 3.3/(Vbat - 3.3) Rmiddle = 250K - Rtop || Rbottom"
- note removed: "Float voltage selection Rbottom/Rtop = 3.3/(Vbat - 3.3) Rmiddle = 250K - Rtop || Rbottom"
Changed lines of the file:
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@@
     (effects (font (size 1.27 1.27)) (justify left bottom))
   )
-  (text "Float voltage selection\nRbottom/Rtop = 3.3/(Vbat - 3.3)\nRmiddle = 250K - Rtop || Rbottom\n"
+  (text "Float voltage selection 8.27V\nRbottom/Rtop = 3.3/(Vbat - 3.3)\nRmiddle = 250K - Rtop || Rbottom\n"
     (at 158.75 71.12 0)
     (effects (font (size 1.27 1.27)) (justify left bottom))
@@
     (in_bom yes) (on_board yes)
     (property "Reference" "R8" (id 0) (at 166.37 54.61 90))
-    (property "Value" "52.8K" (id 1) (at 166.37 57.15 90))
+    (property "Value" "" (id 1) (at 166.37 57.15 90))
     (property "Footprint" "Resistor_SMD:R_0805_2012Metric" (id 2) (at 166.37 55.372 90)
       (effects (font (size 1.27 1.27)) hide)
@@
       (effects (font (size 1.27 1.27)) (justify right))
     )
-    (property "Value" "330K" (id 1) (at 171.45 60.96 90))
+    (property "Value" "" (id 1) (at 171.45 60.96 90))
     (property "Footprint" "Resistor_SMD:R_0805_2012Metric" (id 2) (at 173.228 60.96 90)
       (effects (font (size 1.27 1.27)) hide)
@@
       (effects (font (size 1.27 1.27)) (justify right))
     )
-    (property "Value" "490K" (id 1) (at 171.45 53.34 90))
+    (property "Value" "" (id 1) (at 171.45 53.34 90))
     (property "Footprint" "Resistor_SMD:R_0805_2012Metric" (id 2) (at 173.228 53.34 90)
       (effects (font (size 1.27 1.27)) hide)

Commit message: finish solar routing except telem
Parts:
- R10: value (none) -> 97.6K
- R8: value (none) -> 191K
- R9: value (none) -> 147K
- renumbered C6 to C4, C7 to C5, C8 to C6, C9 to C7, C10 to C8, U4 to U3, U5 to U4, U6 to U5
Changed lines of the file:
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@@
   (symbol (lib_id "Battery_Management:LT3652EMSE") (at 148.59 46.99 0) (unit 1)
     (in_bom yes) (on_board yes)
-    (property "Reference" "U6" (id 0) (at 148.59 29.6926 0))
+    (property "Reference" "U5" (id 0) (at 148.59 29.6926 0))
     (property "Value" "LT3652EMSE" (id 1) (at 148.59 32.004 0))
     (property "Footprint" "Package_SO:MSOP-12-1EP_3x4mm_P0.65mm_EP1.65x2.85mm" (id 2) (at 148.59 62.23 0)
@@
   (symbol (lib_id "power:GND") (at 97.79 64.77 0) (unit 1)
     (in_bom yes) (on_board yes)
-    (property "Reference" "#PWR021" (id 0) (at 97.79 71.12 0)
+    (property "Reference" "#PWR020" (id 0) (at 97.79 71.12 0)
       (effects (font (size 1.27 1.27)) hide)
     )
@@
   (symbol (lib_id "Device:C") (at 125.73 38.1 0) (unit 1)
     (in_bom yes) (on_board yes)
-    (property "Reference" "C8" (id 0) (at 128.651 36.9316 0)
+    (property "Reference" "C6" (id 0) (at 128.651 36.9316 0)
       (effects (font (size 1.27 1.27)) (justify left))
     )
@@
     (in_bom yes) (on_board yes)
     (property "Reference" "R8" (id 0) (at 166.37 54.61 90))
-    (property "Value" "" (id 1) (at 166.37 57.15 90))
+    (property "Value" "191K" (id 1) (at 166.37 57.15 90))
     (property "Footprint" "Resistor_SMD:R_0805_2012Metric" (id 2) (at 166.37 55.372 90)
       (effects (font (size 1.27 1.27)) hide)
@@
       (effects (font (size 1.27 1.27)) (justify right))
     )
-    (property "Value" "" (id 1) (at 171.45 60.96 90))
+    (property "Value" "97.6K" (id 1) (at 171.45 60.96 90))
     (property "Footprint" "Resistor_SMD:R_0805_2012Metric" (id 2) (at 173.228 60.96 90)
       (effects (font (size 1.27 1.27)) hide)
@@
       (effects (font (size 1.27 1.27)) (justify right))
     )
-    (property "Value" "" (id 1) (at 171.45 53.34 90))
+    (property "Value" "147K" (id 1) (at 171.45 53.34 90))
     (property "Footprint" "Resistor_SMD:R_0805_2012Metric" (id 2) (at 173.228 53.34 90)
       (effects (font (size 1.27 1.27)) hide)
@@
   (symbol (lib_id "Device:C") (at 165.1 40.64 0) (unit 1)
     (in_bom yes) (on_board yes)
-    (property "Reference" "C9" (id 0) (at 165.1 38.1 0)
+    (property "Reference" "C7" (id 0) (at 165.1 38.1 0)
       (effects (font (size 1.27 1.27)) (justify left))
     )
@@
   (symbol (lib_id "power:GND") (at 172.72 31.75 0) (unit 1)
     (in_bom yes) (on_board yes)
-    (property "Reference" "#PWR022" (id 0) (at 172.72 38.1 0)
+    (property "Reference" "#PWR021" (id 0) (at 172.72 38.1 0)
       (effects (font (size 1.27 1.27)) hide)
     )
@@
   (symbol (lib_id "Device:C") (at 182.88 53.34 0) (unit 1)
     (in_bom yes) (on_board yes)
-    (property "Reference" "C10" (id 0) (at 185.801 52.1716 0)
+    (property "Reference" "C8" (id 0) (at 185.801 52.1716 0)
       (effects (font (size 1.27 1.27)) (justify left))
     )
@@
   (symbol (lib_id "power:GND") (at 39.37 39.37 0) (unit 1)
     (in_bom yes) (on_board yes)
-    (property "Reference" "#PWR016" (id 0) (at 39.37 45.72 0)
+    (property "Reference" "#PWR015" (id 0) (at 39.37 45.72 0)
       (effects (font (size 1.27 1.27)) hide)
     )
@@
   (symbol (lib_id "Amplifier_Current:INA138") (at 41.91 31.75 0) (unit 1)
     (in_bom yes) (on_board yes)
-    (property "Reference" "U4" (id 0) (at 50.6476 30.5816 0)
+    (property "Reference" "U3" (id 0) (at 50.6476 30.5816 0)
       (effects (font (size 1.27 1.27)) (justify left))
     )
@@
   (symbol (lib_id "Device:C") (at 43.18 24.13 90) (unit 1)
     (in_bom yes) (on_board yes)
-    (property "Reference" "C6" (id 0) (at 44.45 20.32 90)
+    (property "Reference" "C4" (id 0) (at 44.45 20.32 90)
       (effects (font (size 1.27 1.27)) (justify right))
     )
@@
   (symbol (lib_id "power:GND") (at 46.99 24.13 0) (unit 1)
     (in_bom yes) (on_board yes)
-    (property "Reference" "#PWR019" (id 0) (at 46.99 30.48 0)
+    (property "Reference" "#PWR018" (id 0) (at 46.99 30.48 0)
       (effects (font (size 1.27 1.27)) hide)
     )
@@
   (symbol (lib_id "power:GND") (at 39.37 66.04 0) (unit 1)
     (in_bom yes) (on_board yes)
-    (property "Reference" "#PWR018" (id 0) (at 39.37 72.39 0)
+    (property "Reference" "#PWR017" (id 0) (at 39.37 72.39 0)
       (effects (font (size 1.27 1.27)) hide)
     )
@@
   (symbol (lib_id "Amplifier_Current:INA138") (at 41.91 58.42 0) (unit 1)
     (in_bom yes) (on_board yes)
-    (property "Reference" "U5" (id 0) (at 50.6476 57.2516 0)
+    (property "Reference" "U4" (id 0) (at 50.6476 57.2516 0)
       (effects (font (size 1.27 1.27)) (justify left))
     )
@@
   (symbol (lib_id "Device:C") (at 43.18 50.8 90) (unit 1)
     (in_bom yes) (on_board yes)
-    (property "Reference" "C7" (id 0) (at 44.45 46.99 90)
+    (property "Reference" "C5" (id 0) (at 44.45 46.99 90)
       (effects (font (size 1.27 1.27)) (justify right))
     )
@@
   (symbol (lib_id "power:GND") (at 46.99 50.8 0) (unit 1)
     (in_bom yes) (on_board yes)
-    (property "Reference" "#PWR020" (id 0) (at 46.99 57.15 0)
+    (property "Reference" "#PWR019" (id 0) (at 46.99 57.15 0)
       (effects (font (size 1.27 1.27)) hide)
     )
@@
   (symbol (lib_id "power:VDD") (at 39.37 50.8 0) (unit 1)
     (in_bom yes) (on_board yes)
-    (property "Reference" "#PWR017" (id 0) (at 39.37 54.61 0)
+    (property "Reference" "#PWR016" (id 0) (at 39.37 54.61 0)
       (effects (font (size 1.27 1.27)) hide)
     )
@@
   (symbol (lib_id "power:VDD") (at 39.37 24.13 0) (unit 1)
     (in_bom yes) (on_board yes)
-    (property "Reference" "#PWR015" (id 0) (at 39.37 27.94 0)
-      (effects (font (size 1.27 1.27)) hide)
-    )
+    (property "Reference" "#PWR014" (id 0) (at 39.37 27.94 0)
+      (effects (font (size 1.27 1.27)) hide)
+    )
