File: ECAD/EPS/PowerConditioning.kicad_sch (KiCad schematic)
At the start: 63 parts, among them Q10 2N7002, Q11 IRF7458, Q12 2N7002, Q13 2N7002, Q14 2N7002, Q15 IRF7458, Q16 IRF7458, Q17 2N7002, Q18 2N7002, U28 TPS54394RSAR, U29 LM1117-3.3, U30 MAX4373F, U31 MAX4373F, U32 MAX4373F

Commit message: layout and footprints
Parts:
- U31: renamed from U?; value ~ -> 74HC595; footprint (none) -> Package_SO:SOIC-16_3.9x9.9mm_P1.27mm
- gave numbers to parts that had none: 4
- renumbered C50 to C47, C45 to C48, C46 to C49, C47 to C50, C48 to C51, C55 to C52, C56 to C53, C49 to C55, C51 to C56, C52 to C57, C53 to C58, C54 to C59, C57 to C61, C58 to C62, Q15 to Q10, Q16 to Q11, Q17 to Q12, Q18 to Q13, Q10 to Q5, Q11 to Q6, Q14 to Q7, Q12 to Q8, Q13 to Q9, R51 to R45, R52 to R46, R58 to R47, R61 to R48, R64 to R49, R67 to R50, R70 to R51, R71 to R52, R76 to R54, R77 to R55, R59 to R58, R60 to R59, R62 to R60, R63 to R61, R65 to R62, R66 to R63, R68 to R64, R69 to R65, R72 to R66, R73 to R67, R74 to R68, R75 to R69, R78 to R70, R79 to R71, R80 to R72, R81 to R73, U29 to U27, U30 to U29, U31 to U32, U32 to U33

Commit message: move solar to daughterboard... again. Also replace all 0603 resistor with 0805
Parts:
- renumbered C47 to C18, C48 to C19, C49 to C20, C50 to C21, C51 to C22, C52 to C23, C53 to C24, C54 to C25, C55 to C26, C56 to C27, C57 to C28, C58 to C29, C59 to C30, C60 to C31, C61 to C32, C62 to C33, L5 to L1, L6 to L2, Q12 to Q10, Q13 to Q11, Q5 to Q3, Q6 to Q4, Q7 to Q5, Q8 to Q6, Q9 to Q7, Q10 to Q8, Q11 to Q9, R45 to R10, R46 to R11, R47 to R12, R48 to R13, R49 to R14, R50 to R15, R51 to R16, R52 to R17, R53 to R18, R54 to R19, R55 to R20, R56 to R21, R57 to R22, R58 to R23, R59 to R24, R60 to R25, R61 to R26, R62 to R27, R63 to R28, R64 to R29, R65 to R30, R66 to R31, R67 to R32, R68 to R33, R69 to R34, R70 to R35, R71 to R36, R72 to R37, R73 to R38, U32 to U10, U33 to U11, U27 to U5, U28 to U6, U29 to U7, U30 to U8, U31 to U9

Commit message: simplify reset and retry
Parts:
- removed R18: 10K, Resistor_SMD:R_0805_2012Metric, symbol Device:R
Connections:
- net PDMRST is gone; now on net VDD: U8.10 (~{SRCLR})
- net RST3V3PLS is gone; now on net RST3V3: Q7.1 (G)
- net RST5VPLS is gone; now on net RST5V: Q6.1 (G)
- net RSTBATVPLS is gone; now on net RSTBATV: Q3.1 (G)
- net +3.3VA: now reaches C29.1, C30.1, L2.2, Q9.1 (S), Q9.2 (S), Q9.3 (S), R21.1, R24.1
- net GATE3V3: no longer names the net of Q11.1 (G), R26.2, U11.6 (COUT1)
- net GATE5V: no longer names the net of Q10.1 (G), R25.2, U10.6 (COUT1)
- net GATEBATV: no longer names the net of Q5.1 (G), R13.2, U7.6 (COUT1)
Other:
- removed sheet Timer3V3
- removed sheet Timer5V
- removed sheet TimerBATV

Commit message: reannotate and cleanup some more
Parts:
- renumbered R19 to R18, R20 to R19, R21 to R20, R22 to R21, R23 to R22, R24 to R23, R25 to R24, R26 to R25, R27 to R26, R28 to R27, R29 to R28, R30 to R29, R31 to R30, R32 to R31, R33 to R32, R34 to R33, R35 to R34, R36 to R35, R37 to R36, R38 to R37

Commit message: proposed switch layout
Parts:
- renumbered C18 to C17, C19 to C18, C20 to C19, C21 to C20, C22 to C21, C23 to C22, C24 to C23, C25 to C24, C26 to C25, C27 to C26, C28 to C27, C29 to C28, C30 to C29, C31 to C30, C32 to C31, C33 to C32
Changed lines of the file:
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@@
   (symbol (lib_id "Device:C") (at 46.99 93.98 180) (unit 1)
     (in_bom yes) (on_board yes)
-    (property "Reference" "C21" (id 0) (at 44.069 95.1484 0)
+    (property "Reference" "C20" (id 0) (at 44.069 95.1484 0)
       (effects (font (size 1.27 1.27)) (justify left))
     )
@@
   (symbol (lib_id "Device:C") (at 50.8 107.95 0) (mirror y) (unit 1)
     (in_bom yes) (on_board yes)
-    (property "Reference" "C22" (id 0) (at 47.879 106.7816 0)
+    (property "Reference" "C21" (id 0) (at 47.879 106.7816 0)
       (effects (font (size 1.27 1.27)) (justify left))
     )
@@
   (symbol (lib_id "Device:C") (at 73.66 107.95 0) (unit 1)
     (in_bom yes) (on_board yes)
-    (property "Reference" "C26" (id 0) (at 76.581 106.7816 0)
+    (property "Reference" "C25" (id 0) (at 76.581 106.7816 0)
       (effects (font (size 1.27 1.27)) (justify left))
     )
@@
   (symbol (lib_id "Device:C") (at 26.67 163.83 0) (unit 1)
     (in_bom yes) (on_board yes)
-    (property "Reference" "C18" (id 0) (at 29.591 162.6616 0)
+    (property "Reference" "C17" (id 0) (at 29.591 162.6616 0)
       (effects (font (size 1.27 1.27)) (justify left))
     )
@@
   (symbol (lib_id "Device:C") (at 50.8 163.83 0) (unit 1)
     (in_bom yes) (on_board yes)
-    (property "Reference" "C23" (id 0) (at 53.721 162.6616 0)
+    (property "Reference" "C22" (id 0) (at 53.721 162.6616 0)
       (effects (font (size 1.27 1.27)) (justify left))
     )
@@
   (symbol (lib_id "Device:C") (at 52.07 19.05 0) (unit 1)
     (in_bom yes) (on_board yes)
-    (property "Reference" "C24" (id 0) (at 54.991 17.8816 0)
+    (property "Reference" "C23" (id 0) (at 54.991 17.8816 0)
       (effects (font (size 1.27 1.27)) (justify left))
     )
@@
   (symbol (lib_id "Device:C") (at 152.4 66.04 0) (unit 1)
     (in_bom yes) (on_board yes)
-    (property "Reference" "C32" (id 0) (at 155.321 64.8716 0)
+    (property "Reference" "C31" (id 0) (at 155.321 64.8716 0)
       (effects (font (size 1.27 1.27)) (justify left))
     )
@@
   (symbol (lib_id "Device:C") (at 152.4 109.22 0) (unit 1)
     (in_bom yes) (on_board yes)
-    (property "Reference" "C33" (id 0) (at 155.321 108.0516 0)
+    (property "Reference" "C32" (id 0) (at 155.321 108.0516 0)
       (effects (font (size 1.27 1.27)) (justify left))
     )
@@
   (symbol (lib_id "Device:C") (at 35.56 115.57 0) (unit 1)
     (in_bom yes) (on_board yes)
-    (property "Reference" "C20" (id 0) (at 38.481 114.4016 0)
+    (property "Reference" "C19" (id 0) (at 38.481 114.4016 0)
       (effects (font (size 1.27 1.27)) (justify left))
     )
@@
   (symbol (lib_id "Device:C") (at 30.48 115.57 0) (mirror y) (unit 1)
     (in_bom yes) (on_board yes)
-    (property "Reference" "C19" (id 0) (at 27.559 114.4016 0)
+    (property "Reference" "C18" (id 0) (at 27.559 114.4016 0)
       (effects (font (size 1.27 1.27)) (justify left))
     )
@@
   (symbol (lib_id "Device:C") (at 88.9 115.57 0) (mirror y) (unit 1)
     (in_bom yes) (on_board yes)
-    (property "Reference" "C29" (id 0) (at 85.979 114.4016 0)
+    (property "Reference" "C28" (id 0) (at 85.979 114.4016 0)
       (effects (font (size 1.27 1.27)) (justify left))
     )
@@
   (symbol (lib_id "Device:C") (at 64.77 158.75 0) (unit 1)
     (in_bom yes) (on_board yes)
-    (property "Reference" "C25" (id 0) (at 67.31 157.48 0)
+    (property "Reference" "C24" (id 0) (at 67.31 157.48 0)
       (effects (font (size 1.27 1.27)) (justify left))
     )
@@
   (symbol (lib_id "Device:C") (at 81.28 93.98 180) (unit 1)
     (in_bom yes) (on_board yes)
-    (property "Reference" "C28" (id 0) (at 78.359 95.1484 0)
+    (property "Reference" "C27" (id 0) (at 78.359 95.1484 0)
       (effects (font (size 1.27 1.27)) (justify left))
     )
@@
   (symbol (lib_id "Device:C") (at 78.74 134.62 180) (unit 1)
     (in_bom yes) (on_board yes)
-    (property "Reference" "C27" (id 0) (at 75.819 135.7884 0)
+    (property "Reference" "C26" (id 0) (at 75.819 135.7884 0)
       (effects (font (size 1.27 1.27)) (justify left))
     )
@@
   (symbol (lib_id "Device:C") (at 93.98 115.57 0) (unit 1)
     (in_bom yes) (on_board yes)
-    (property "Reference" "C30" (id 0) (at 96.901 114.4016 0)
+    (property "Reference" "C29" (id 0) (at 96.901 114.4016 0)
       (effects (font (size 1.27 1.27)) (justify left))
     )
@@
   (symbol (lib_id "Device:C") (at 114.3 158.75 0) (unit 1)
     (in_bom yes) (on_board yes)
-    (property "Reference" "C31" (id 0) (at 117.221 157.5816 0)
-      (effects (font (size 1.27 1.27)) (justify left))
-    )
+    (property "Reference" "C30" (id 0) (at 117.221 157.5816 0)
+      (effects (font (size 1.27 1.27)) (justify left))
+    )

Commit message: finish battery
Parts:
- Q4, Q8, Q9: value IRF7458 -> DMP3015LSSQ
Changed lines of the file:
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@@
     (in_bom yes) (on_board yes)
     (property "Reference" "Q4" (id 0) (at 35.56 15.4432 90))
-    (property "Value" "IRF7458" (id 1) (at 35.56 17.7546 90))
+    (property "Value" "DMP3015LSSQ" (id 1) (at 35.56 17.7546 90))
     (property "Footprint" "Package_SO:SOIC-8_3.9x4.9mm_P1.27mm" (id 2) (at 33.655 19.05 0)
       (effects (font (size 1.27 1.27) italic) (justify left) hide)
@@
     (in_bom yes) (on_board yes)
     (property "Reference" "Q8" (id 0) (at 135.89 62.4332 90))
-    (property "Value" "IRF7458" (id 1) (at 135.89 64.7446 90))
+    (property "Value" "DMP3015LSSQ" (id 1) (at 135.89 64.7446 90))
     (property "Footprint" "Package_SO:SOIC-8_3.9x4.9mm_P1.27mm" (id 2) (at 133.985 66.04 0)
       (effects (font (size 1.27 1.27) italic) (justify left) hide)
@@
     (in_bom yes) (on_board yes)
     (property "Reference" "Q9" (id 0) (at 135.89 105.6132 90))
-    (property "Value" "IRF7458" (id 1) (at 135.89 107.9246 90))
+    (property "Value" "DMP3015LSSQ" (id 1) (at 135.89 107.9246 90))
     (property "Footprint" "Package_SO:SOIC-8_3.9x4.9mm_P1.27mm" (id 2) (at 133.985 109.22 0)
       (effects (font (size 1.27 1.27) italic) (justify left) hide)

Commit message: value editing
Parts:
- C17, C20, C22, C27: value 10uF -> (none); footprint Capacitor_SMD:C_0805_2012Metric -> (none)
- C18, C19, C28, C29: value 22uF -> (none); footprint Capacitor_SMD:C_1210_3225Metric -> (none)
- C21, C23, C24, C25, C30, C31, C32: value 0.1uF -> (none); footprint Capacitor_SMD:C_0805_2012Metric -> (none)
- C26: value 1uF -> (none); footprint Capacitor_SMD:C_0805_2012Metric -> (none)
- L1: value 4.7uH -> (none); footprint Inductor_SMD:L_Abracon_ASPI-0630LR -> (none)
- L2: value 3.3uH -> (none); footprint Inductor_SMD:L_Abracon_ASPI-0630LR -> (none)
- Q10, Q11, Q3, Q5, Q6, Q7: value 2N7002 -> (none); footprint Package_TO_SOT_SMD:SOT-23 -> (none)
- Q4, Q8, Q9: value DMP3015LSSQ -> (none); footprint Package_SO:SOIC-8_3.9x4.9mm_P1.27mm -> (none)
- R10: value 124K -> (none); footprint Resistor_SMD:R_0805_2012Metric -> (none)
- R11, R21: value 22.1K -> (none); footprint Resistor_SMD:R_0805_2012Metric -> (none)
- R12, R13, R14, R22, R23, R24, R25, R26, R27: value 10K -> (none); footprint Resistor_SMD:R_0805_2012Metric -> (none)
- R15, R28, R29: value 10m -> (none); footprint Resistor_SMD:R_1206_3216Metric -> (none)
- R16: value 9.5K -> (none); footprint Resistor_SMD:R_0805_2012Metric -> (none)
- R17: value 3K -> (none); footprint Resistor_SMD:R_0805_2012Metric -> (none)
- R18: value 200K -> (none); footprint Resistor_SMD:R_0805_2012Metric -> (none)
- R19, R34, R35, R36, R37: value 100K -> (none); footprint Resistor_SMD:R_0805_2012Metric -> (none)
- R20: value 73.2K -> (none); footprint Resistor_SMD:R_0805_2012Metric -> (none)
- R30, R32: value 6K -> (none); footprint Resistor_SMD:R_0805_2012Metric -> (none)
- R31, R33: value 4K -> (none); footprint Resistor_SMD:R_0805_2012Metric -> (none)
- U10, U11, U7: value MAX4373F -> (none); footprint Package_SO:SO-8_3.9x4.9mm_P1.27mm -> (none)
- U5: value LM1117-3.3 -> (none); footprint Package_TO_SOT_SMD:SOT-223-3_TabPin2 -> (none)
- U6: value TPS54394RSAR -> (none); footprint Package_DFN_QFN:Texas_S-PVQFN-N16_EP2.7x2.7mm_ThermalVias -> (none)
- U8, U9: value 74HC595 -> (none); footprint Package_SO:SOIC-16_3.9x9.9mm_P1.27mm -> (none)
