File: ECAD/EPS/SolarConditioning.kicad_pcb (KiCad board)
At the start: 2 copper layers, 83.8 x 59.4 mm, 120 parts, among them J1 S1A, J2 S1B, J3 S2A, J4 S2B, J5 S3A, J6 S3B, J7 S4A, J8 S4B, J9 Solar Daughterboard Connector, U1 INA180A3, U10 INA180A3, U11 INA180A3, U12 LT3652EMSE, U13 INA180A3, U14 INA180A3, U15 LT3652EMSE, U2 CD74HC4067SM, U3 CD74HC4067SM, U4 INA180A3, U5 INA180A3, U6 LT3652EMSE, U7 INA180A3, U8 INA180A3, U9 LT3652EMSE

Commit message: value editing
Parts:
- moved D16 2.27 mm to (148.8, 104.7)
Routing:
- net /MPPT1/VOUT: track 71.6 -> 81.5 mm
Changed lines of the file:
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@@
   )
   (footprint "Diode_SMD:D_SOD-123F" (layer "F.Cu")
-    (at 146.812 105.661 -90)
+    (at 148.844 104.651 -90)
     (descr "D_SOD-123F")
     (tags "D_SOD-123F")
@@
     (property "Sheetname" "MPPT4")
     (attr smd)
-    (fp_text reference "D16" (at -0.127 -1.905 90) (layer "F.SilkS")
+    (fp_text reference "D16" (at 0 1.778 90) (layer "F.SilkS")
       (effects (font (size 1 1) (thickness 0.15)))
     )
@@
   (segment (start 146.431 72.898) (end 146.431 84.963) (width 0.381) (layer "F.Cu") (net 7))
   (segment (start 149.165853 71.179147) (end 146.939 73.406) (width 0.254) (layer "F.Cu") (net 7))
+  (segment (start 148.844 106.938) (end 148.7825 106.9995) (width 0.508) (layer "F.Cu") (net 7))
+  (segment (start 148.844 106.051) (end 148.844 106.938) (width 0.508) (layer "F.Cu") (net 7))
   (segment (start 156.7185 84.9015) (end 156.911 84.709) (width 0.762) (layer "F.Cu") (net 7))
   (segment (start 148.971 84.077) (end 148.971 84.963) (width 0.762) (layer "F.Cu") (net 7))
   (segment (start 153.924 106.9995) (end 156.7225 106.9995) (width 0.762) (layer "F.Cu") (net 7))
+  (segment (start 148.7825 106.9995) (end 144.9725 106.9995) (width 0.762) (layer "F.Cu") (net 7))
   (segment (start 161.095147 71.179147) (end 149.165853 71.179147) (width 0.254) (layer "F.Cu") (net 7))
   (segment (start 154.051 82.87652) (end 154.051 84.9015) (width 0.254) (layer "F.Cu") (net 7))
   (segment (start 153.9895 84.963) (end 148.971 84.963) (width 0.762) (layer "F.Cu") (net 7))
+  (segment (start 153.924 106.9995) (end 148.7825 106.9995) (width 0.762) (layer "F.Cu") (net 7))
   (segment (start 148.844 70.485) (end 146.431 72.898) (width 0.381) (layer "F.Cu") (net 7))
   (segment (start 148.971 84.963) (end 144.653 84.963) (width 0.762) (layer "F.Cu") (net 7))

Commit message: solar progress
Parts:
- R1: value 220K -> 200K
- R10, R18, R26, R34: value 330K -> 97.6K
- R16, R24, R32, R8: value 52.8K -> 191K
- R17, R25, R33, R9: value 490K -> 147K
- moved C5 203.6 mm to (199.1, 131.7), turned to 0 degrees
- moved U3 199.6 mm to (200.9, 137.3)
- moved C1 193.2 mm to (202.6, 131.7), turned to 180 degrees
- moved C3 172.5 mm to (155.9, 135.5)
- moved U2 161.6 mm to (150.1, 137.2), turned to -90 degrees
- moved C2 131.1 mm to (155.9, 139.0), turned to 90 degrees
- moved R3 100.1 mm to (134.9, 103.7), turned to 90 degrees
- moved C4 99.5 mm to (140.7, 103.8), turned to 90 degrees
- moved J1 98.6 mm to (107.4, 107.2), turned to 90 degrees
- moved U1 93.6 mm to (137.9, 103.8), turned to -90 degrees
- moved J4 91.4 mm to (107.4, 75.3), turned to 90 degrees
- moved D1 88.9 mm to (110.7, 106.8), turned to 90 degrees
- moved D2 87.4 mm to (110.7, 97.7), turned to 90 degrees
- moved J2 86.1 mm to (107.4, 97.9), turned to 90 degrees
- moved J3 84.6 mm to (107.4, 84.7), turned to 90 degrees
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Routing:
- net /MPPT1/VOUT: track 81.5 -> 135.0 mm
- net Net-(L4-Pad2): track 2.09 -> 33.2 mm
- net Net-(C24-Pad2): track 2.73 -> 22.2 mm
- net Net-(C13-Pad1): track 0.00 -> 17.5 mm
- net Net-(C8-Pad1): track 0.00 -> 17.1 mm
- net GND: track 27.8 -> 43.7 mm
- net VDD: track 7.69 -> 15.4 mm
- net Net-(C23-Pad1): track 34.5 -> 40.1 mm
- net Net-(D1-Pad2): track 0.00 -> 4.77 mm
- net Net-(D4-Pad2): track 0.00 -> 4.72 mm
- net Net-(D2-Pad2): track 0.00 -> 4.72 mm
- net Net-(D3-Pad2): track 0.00 -> 4.72 mm
- net /MPPT2/B_PWR: track 0.00 -> 4.63 mm
- net /MPPT2/A_PWR: track 0.00 -> 4.59 mm
- net /MPPT1/B_PWR: track 0.00 -> 4.52 mm
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
Commit message: finish placing solar components
Parts:
- moved R2 114.5 mm to (149.2, 125.1)
- moved R1 111.3 mm to (145.9, 125.1)
- moved L1 77.4 mm to (135.4, 98.4), turned to 90 degrees
- moved R10 74.1 mm to (133.1, 106.0), turned to 90 degrees
- moved R19 72.2 mm to (136.4, 70.5), turned to -90 degrees
- moved C9 70.7 mm to (130.0, 102.0), turned to -90 degrees
- moved D9 70.3 mm to (128.0, 98.2), turned to 180 degrees
- moved R9 70.1 mm to (135.9, 105.3)
- moved L2 70.0 mm to (136.4, 76.8), turned to 90 degrees
- moved D10 68.0 mm to (139.7, 92.1), turned to 90 degrees
- moved R11 67.5 mm to (135.4, 92.1), turned to -90 degrees
- moved TP4 64.4 mm to (124.5, 88.0)
- moved R8 64.2 mm to (130.3, 105.3), turned to 180 degrees
- moved C8 62.8 mm to (122.7, 98.9)
- moved U9 61.7 mm to (126.2, 81.9)
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Routing:
- net /MPPT1/VOUT: track 135.0 -> 297.0 mm
- net Net-(L2-Pad2): track 0.00 -> 32.0 mm
- net Net-(L1-Pad2): track 0.00 -> 31.9 mm
- net Net-(C14-Pad2): track 0.00 -> 21.4 mm
- net Net-(C9-Pad2): track 0.00 -> 21.3 mm
- net Net-(C13-Pad1): track 17.5 -> 38.7 mm, vias 0 -> 2
- net Net-(C8-Pad1): track 17.1 -> 38.0 mm, vias 0 -> 2
- net Net-(RV2-Pad2): track 0.00 -> 12.2 mm
- net Net-(C9-Pad1): track 0.00 -> 11.6 mm
- net Net-(C14-Pad1): track 0.00 -> 11.3 mm
- net Net-(RV1-Pad2): track 0.00 -> 10.3 mm
- net Net-(R10-Pad2): track 0.00 -> 3.89 mm
- net Net-(R16-Pad1): track 0.00 -> 3.89 mm
- net Net-(R16-Pad2): track 0.00 -> 2.19 mm
- net Net-(R8-Pad2): track 0.00 -> 2.13 mm
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- added copper zone on B.Cu, net GND
- added copper zone on F.Cu, net GND

Commit message: current monitor
Parts:
- moved C4 25.4 mm to (146.3, 107.3)
- moved R3 25.4 mm to (140.5, 107.3)
- moved U1 25.4 mm to (143.5, 107.3)
- moved D16 1.82 mm to (150.6, 105.0)
- moved L4 1.52 mm to (155.4, 99.2)
- moved R35 1.52 mm to (155.4, 105.5)
- moved C25 1.27 mm to (159.0, 107.1)
- moved C24 0.51 mm to (160.8, 95.6)
- moved R32 0.51 mm to (160.0, 91.8)
- moved R34 0.51 mm to (157.2, 90.8)
- moved TP8 0.51 mm to (171.2, 90.0)
- moved C23 0.51 mm to (168.4, 98.9)
- moved D15 0.51 mm to (162.8, 99.4)
- moved R33 0.51 mm to (154.4, 91.8)
- moved U15 0.51 mm to (165.4, 94.3)
Routing:
- net BCR_OUT: track 0.00 -> 9.71 mm
- net /MPPT1/VOUT: track 297.0 -> 301.9 mm
- net GND: track 43.7 -> 47.8 mm
- net VDD: track 15.4 -> 17.3 mm
- net Net-(C24-Pad2): track 22.2 -> 21.0 mm
- net Net-(C24-Pad1): track 12.1 -> 11.1 mm
- net Net-(RV4-Pad2): track 9.78 -> 9.06 mm
- net Net-(L4-Pad2): track 33.2 -> 32.5 mm

Commit message: finish solar routing except telem
Parts:
- removed the C2 at (155.9, 139.0)
- removed the C5 at (199.1, 131.7)
- removed the U3 at (200.9, 137.3)
- J9: footprint Connector_PinHeader_2.54mm:PinHeader_2x06_P2.54mm_Vertical -> Connector_PinHeader_2.54mm:PinHeader_2x05_P2.54mm_Vertical
- moved C1 32.0 mm to (175.3, 115.2), turned to 90 degrees
- moved C2 30.7 mm to (175.3, 111.7)
- moved U2 30.5 mm to (169.2, 113.4)
- moved R1 17.1 mm to (152.7, 109.3), turned to -90 degrees
- moved R2 15.8 mm to (150.6, 109.3), turned to 90 degrees
- moved RV2 1.27 mm to (119.9, 80.6)
- renumbered C12 to C10, C13 to C11, C14 to C12, C15 to C13, C16 to C14, C17 to C15, C18 to C16, C19 to C17, C20 to C18, C21 to C19, C3 to C2, C22 to C20, C23 to C21, C24 to C22, C25 to C23, C4 to C3, C6 to C4, C7 to C5, C8 to C6, C9 to C7, C10 to C8, C11 to C9, U11 to U10, U12 to U11, U13 to U12, U14 to U13, U15 to U14, U4 to U3, U5 to U4, U6 to U5, U7 to U6, U8 to U7, U9 to U8, U10 to U9
Connections:
- J9 pad 10: VDD -> GND
- J9 pad 6: MUX4OUT -> VDD
- J9 pad 9: VDD -> GND
Routing:
- net VDD: track 17.3 -> 199.3 mm, vias 0 -> 12
- net MUX3OUT: track 0.00 -> 45.4 mm, vias 0 -> 2
- net S1: track 0.00 -> 30.3 mm, vias 0 -> 2
- net S2: track 0.00 -> 28.5 mm
- net S0: track 0.00 -> 26.4 mm, vias 0 -> 2
- net S3: track 0.00 -> 24.2 mm
- net GND: track 47.8 -> 50.8 mm, vias 0 -> 38
- net TELEM_IBCROUT: track 0.00 -> 2.30 mm, vias 0 -> 1
- net Net-(C11-Pad1): track 38.7 -> 37.4 mm
- net /MPPT1/VOUT: track 301.9 -> 302.6 mm
- net BCR_OUT: track 9.71 -> 10.4 mm

Commit message: finish solar
Routing:
- net I_SA2B: track 0.00 -> 137.4 mm, vias 0 -> 2
- net I_SA2A: track 0.00 -> 111.5 mm, vias 0 -> 4
- net I_SA1B: track 0.00 -> 96.0 mm, vias 0 -> 4
- net I_SA1A: track 0.00 -> 85.5 mm, vias 0 -> 4
- net V_SA2: track 2.03 -> 86.7 mm, vias 0 -> 4
- net V_SA1: track 2.03 -> 69.2 mm, vias 0 -> 4
- net V_SA3: track 2.03 -> 68.0 mm, vias 0 -> 2
- net I_SA3A: track 0.00 -> 60.5 mm, vias 0 -> 2
- net I_SA3B: track 0.00 -> 50.2 mm, vias 0 -> 2
- net I_SA4A: track 0.00 -> 43.4 mm, vias 0 -> 4
- net TELEM_IBCROUT: track 2.30 -> 41.4 mm, vias 1 -> 2
- net I_SA4B: track 0.00 -> 30.0 mm, vias 0 -> 2
- net TELEM_VBCROUT: track 0.00 -> 23.3 mm, vias 0 -> 2
- net V_SA4: track 2.03 -> 9.04 mm
- net GND: track 50.8 -> 51.5 mm, vias 38 -> 39
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Other:
- board text added: "Alan H. '23 TJ EPS Solar Daughterboard v1"

Commit message: boost
Parts:
- added MH5: M2, MountingHole:MountingHole_2.2mm_M2, F.Cu at (187.1, 132.5)
Changed lines of the file:
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@@
     )
+  )
+  (footprint "MountingHole:MountingHole_2.2mm_M2" (layer "F.Cu")
+    (at 187.071 132.461)
+    (descr "Mounting Hole 2.2mm, no annular, M2")
+    (tags "mounting hole 2.2mm no annular m2")
+    (property "Sheetfile" "SolarConditioning.kicad_sch")
+    (property "Sheetname" "")
+    (attr exclude_from_pos_files)
+    (fp_text reference "MH5" (at 0 -3.2) (layer "F.SilkS")
+      (effects (font (size 1 1) (thickness 0.15)))
+    )
+    (fp_text value "M2" (at 0 3.2) (layer "F.Fab")
+      (effects (font (size 1 1) (thickness 0.15)))
+    )
+    (fp_text user "${REFERENCE}" (at 0 0) (layer "F.Fab")
+      (effects (font (size 1 1) (thickness 0.15)))
+    )
+    (fp_circle (center 0 0) (end 2.2 0) (layer "Cmts.User") (width 0.15) (fill none))
+    (fp_circle (center 0 0) (end 2.45 0) (layer "F.CrtYd") (width 0.05) (fill none))
+    (pad "" np_thru_hole circle (at 0 0) (size 2.2 2.2) (drill 2.2) (layers *.Cu *.Mask))
   )
   (footprint "Capacitor_SMD:C_0805_2012Metric" (layer "F.Cu")

Commit message: add 5v charge back in
Parts:
- added C24: 22uF, Capacitor_SMD:C_1210_3225Metric, F.Cu at (181.6, 127.9)
- added C25: 22uF, Capacitor_SMD:C_1210_3225Metric, F.Cu at (174.9, 133.3)
- added C26: 22uF, Capacitor_SMD:C_1210_3225Metric, F.Cu at (183.5, 123.3)
- added C27: 22uF, Capacitor_SMD:C_1210_3225Metric, F.Cu at (180.5, 133.3)
- added D17: CMSH3-40MA, Diode_SMD:D_SMA, F.Cu at (176.6, 123.5)
- added J10: USBCHG, Connector_Hirose:Hirose_DF13-02P-1.25DSA_1x02_P1.25mm_Vertical, F.Cu at (175.1, 129.0)
- added L5: 33uH, Inductor_SMD:L_Coilcraft_XAL60xx_6.36x6.56mm, F.Cu at (168.1, 131.7)
- added U15: LT1301, Package_SO:SO-8_3.9x4.9mm_P1.27mm, F.Cu at (168.4, 124.4)
