File: ECAD/EPS/SolarConditioning.kicad_sch (KiCad schematic)
At the start: 53 parts, among them J1 S1A, J2 S1B, J3 S2A, J4 S2B, J5 S3A, J6 S3B, J7 S4A, J8 S4B, J9 Solar Daughterboard Connector, Q1 DMP3015LSSQ, U1 LTC4412xS6, U2 MCP3008, U3 INA180A3, U4 ATtiny84A-SSU, U5 L78L33_SO8, U6 CD74HC4067SM, U7 MCP4812, U8 MCP4812, U9 CD74HC4067SM

Commit message: solar route
Parts:
- C1: footprint Capacitor_SMD:C_0603_1608Metric -> (none)
- J9: renamed from J10; value (none) -> ICSP; footprint (none) -> Connector_PinHeader_2.54mm:PinHeader_2x03_P2.54mm_Vertical
- MH1, MH2, MH3, MH4: value (none) -> M2; footprint (none) -> MountingHole:MountingHole_2.2mm_M2
- renumbered D26 to D17, J9 to J10

Commit message: solar footprint work
Parts:
- removed C2, C6, C7, C8: 0.1uF, Capacitor_SMD:C_0805_2012Metric, symbol Device:C
- removed C4: 0.47uF, Capacitor_SMD:C_0805_2012Metric, symbol Device:C
- removed D10, D11, D12, D13, D14, D15, D16, D9: RR264MM, Diode_SMD:D_SOD-123F, symbol Device:D
- removed D17: RB051MM-2Y, Diode_SMD:D_SOD-123F, symbol Device:D_Schottky
- removed J9: ICSP, Connector_PinHeader_2.54mm:PinHeader_2x03_P2.54mm_Vertical, symbol Connector_Generic:Conn_02x03_Odd_Even
- removed U2: MCP3008, Package_SO:SOIC-16_3.9x9.9mm_P1.27mm, symbol Analog_ADC:MCP3008
- removed U4: ATtiny84A-SSU, Package_SO:SOIC-14_3.9x8.7mm_P1.27mm, symbol MCU_Microchip_ATtiny:ATtiny84A-SS
- removed U5: L78L33_SO8, Package_SO:SOIC-8_3.9x4.9mm_P1.27mm, symbol Regulator_Linear:L78L33_SO8
- removed U7, U8: MCP4812, Package_SO:MSOP-8_3x3mm_P0.65mm, symbol Analog_DAC:MCP4812
- added C5: 0.1uF, Capacitor_SMD:C_0805_2012Metric, symbol Device:C
- C1: footprint (none) -> Capacitor_SMD:C_0805_2012Metric
- D1, D2: value CMSH3-40MA -> (none); footprint Diode_SMD:D_SMA -> (none)
- D3, D4, D5, D6, D7, D8: value CMSH3-40MA -> SS34FA; footprint Diode_SMD:D_SMA -> (none)
- renumbered C5 to C2, C9 to C4, J10 to J9, U3 to U2, U6 to U3, U9 to U4
Connections:
- net GND: now also C5.2
- net MUX3OUT: now also C3.1
- net MUX4OUT: now also C5.1
- net VUSB: no longer J9.10 (Pin_10)
- net +3.3VA renamed VDD
- net VDD: now also J9.10 (Pin_10); no longer C3.1
Other:
- sheet MPPT1 ports: added none; removed Vset
- sheet MPPT2 ports: added none; removed Vset
- sheet MPPT3 ports: added none; removed Vset
- sheet MPPT4 ports: added none; removed Vset
- note removed: "MPPT Setpoint Controller"
- moved on the sheet: C4, U4

Commit message: descope solar LV input
Parts:
- removed Q1: DMP3015LSSQ, Package_SO:SOIC-8_3.9x4.9mm_P1.27mm, symbol Transistor_FET:IRF7404
- removed U1: LTC4412xS6, Package_TO_SOT_SMD:TSOT-23-6, symbol Power_Management:LTC4412xS6
- D1, D2: value (none) -> SS34FA; footprint (none) -> Diode_SMD:D_SOD-123F
- D3, D4, D5, D6, D7, D8: footprint (none) -> Diode_SMD:D_SOD-123F
- renumbered U2 to U1, U3 to U2, U4 to U3
Connections:
- net VUSB is gone; now on net VDD: J9.9 (Pin_9)
- no-connect marks 1 -> 0
Other:
- sheet MPPT4: file Boost-BuckMPPT.kicad_sch -> MPPT.kicad_sch

Commit message: work
Other:
- note added: "Space for more telemetry"
- note removed: "Add panel telemetry here if we implement"
Changed lines of the file:
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@@
     (effects (font (size 1.27 1.27)) (justify left bottom))
   )
-  (text "Add panel telemetry here if we implement" (at 250.19 77.47 90)
+  (text "Space for more telemetry\n" (at 250.19 77.47 90)
     (effects (font (size 1.27 1.27)) (justify left bottom))
   )

Commit message: value editing
Parts:
- R1: value 220K -> (none)
Changed lines of the file:
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@@
       (effects (font (size 1.27 1.27)) (justify left))
     )
-    (property "Value" "220K" (id 1) (at 100.33 43.18 90)
+    (property "Value" "" (id 1) (at 100.33 43.18 90)
       (effects (font (size 1.27 1.27)) (justify left))
     )
@@
     )
     (path "/00000000-0000-0000-0000-000061c37b40"
-      (reference "R1") (unit 1) (value "220K") (footprint "Resistor_SMD:R_0805_2012Metric")
+      (reference "R1") (unit 1) (value "200K") (footprint "Resistor_SMD:R_0805_2012Metric")
     )
     (path "/00000000-0000-0000-0000-000061c37b46"
@@
     )
     (path "/00000000-0000-0000-0000-000061bec848/00000000-0000-0000-0000-000061d5e781"
-      (reference "R8") (unit 1) (value "52.8K") (footprint "Resistor_SMD:R_0805_2012Metric")
+      (reference "R8") (unit 1) (value "191K") (footprint "Resistor_SMD:R_0805_2012Metric")
     )
     (path "/00000000-0000-0000-0000-000061bec848/00000000-0000-0000-0000-000061d73998"
-      (reference "R9") (unit 1) (value "490K") (footprint "Resistor_SMD:R_0805_2012Metric")
+      (reference "R9") (unit 1) (value "147K") (footprint "Resistor_SMD:R_0805_2012Metric")
     )
     (path "/00000000-0000-0000-0000-000061bec848/00000000-0000-0000-0000-000061d6d602"
-      (reference "R10") (unit 1) (value "330K") (footprint "Resistor_SMD:R_0805_2012Metric")
+      (reference "R10") (unit 1) (value "97.6K") (footprint "Resistor_SMD:R_0805_2012Metric")
     )
     (path "/00000000-0000-0000-0000-000061bec848/00000000-0000-0000-0000-000061dc7062"
@@
     )
     (path "/00000000-0000-0000-0000-000061e10014/00000000-0000-0000-0000-000061d5e781"
-      (reference "R16") (unit 1) (value "52.8K") (footprint "Resistor_SMD:R_0805_2012Metric")
+      (reference "R16") (unit 1) (value "191K") (footprint "Resistor_SMD:R_0805_2012Metric")
     )
     (path "/00000000-0000-0000-0000-000061e10014/00000000-0000-0000-0000-000061d73998"
-      (reference "R17") (unit 1) (value "490K") (footprint "Resistor_SMD:R_0805_2012Metric")
+      (reference "R17") (unit 1) (value "147K") (footprint "Resistor_SMD:R_0805_2012Metric")
     )
     (path "/00000000-0000-0000-0000-000061e10014/00000000-0000-0000-0000-000061d6d602"
-      (reference "R18") (unit 1) (value "330K") (footprint "Resistor_SMD:R_0805_2012Metric")
+      (reference "R18") (unit 1) (value "97.6K") (footprint "Resistor_SMD:R_0805_2012Metric")
     )
     (path "/00000000-0000-0000-0000-000061e10014/00000000-0000-0000-0000-000061dc7062"
@@
     )
     (path "/3f3e5af9-b6d1-4725-9068-724c489d3608/00000000-0000-0000-0000-000061d5e781"
-      (reference "R24") (unit 1) (value "52.8K") (footprint "Resistor_SMD:R_0805_2012Metric")
+      (reference "R24") (unit 1) (value "191K") (footprint "Resistor_SMD:R_0805_2012Metric")
     )
     (path "/3f3e5af9-b6d1-4725-9068-724c489d3608/00000000-0000-0000-0000-000061d73998"
-      (reference "R25") (unit 1) (value "490K") (footprint "Resistor_SMD:R_0805_2012Metric")
+      (reference "R25") (unit 1) (value "147K") (footprint "Resistor_SMD:R_0805_2012Metric")
     )
     (path "/3f3e5af9-b6d1-4725-9068-724c489d3608/00000000-0000-0000-0000-000061d6d602"
-      (reference "R26") (unit 1) (value "330K") (footprint "Resistor_SMD:R_0805_2012Metric")
+      (reference "R26") (unit 1) (value "97.6K") (footprint "Resistor_SMD:R_0805_2012Metric")
     )
     (path "/3f3e5af9-b6d1-4725-9068-724c489d3608/00000000-0000-0000-0000-000061dc7062"
@@
     )
     (path "/77ddfb4a-bec3-4f62-8129-0cd32bef34d6/00000000-0000-0000-0000-000061d5e781"
-      (reference "R32") (unit 1) (value "52.8K") (footprint "Resistor_SMD:R_0805_2012Metric")
+      (reference "R32") (unit 1) (value "191K") (footprint "Resistor_SMD:R_0805_2012Metric")
     )
     (path "/77ddfb4a-bec3-4f62-8129-0cd32bef34d6/00000000-0000-0000-0000-000061d73998"
-      (reference "R33") (unit 1) (value "490K") (footprint "Resistor_SMD:R_0805_2012Metric")
+      (reference "R33") (unit 1) (value "147K") (footprint "Resistor_SMD:R_0805_2012Metric")
     )
     (path "/77ddfb4a-bec3-4f62-8129-0cd32bef34d6/00000000-0000-0000-0000-000061d6d602"
-      (reference "R34") (unit 1) (value "330K") (footprint "Resistor_SMD:R_0805_2012Metric")
+      (reference "R34") (unit 1) (value "97.6K") (footprint "Resistor_SMD:R_0805_2012Metric")
     )
     (path "/77ddfb4a-bec3-4f62-8129-0cd32bef34d6/00000000-0000-0000-0000-000061dc7062"

Commit message: finish solar routing except telem
Parts:
- removed C2, C5: 0.1uF, Capacitor_SMD:C_0805_2012Metric, symbol Device:C
- removed J9: Solar Daughterboard Connector, Connector_PinHeader_2.54mm:PinHeader_2x06_P2.54mm_Vertical, symbol Connector_Generic:Conn_02x06_Odd_Even
- removed U3: CD74HC4067SM, Package_SO:SSOP-24_5.3x8.2mm_P0.65mm, symbol 74xx:CD74HC4067SM
- added J9: (no value), symbol Connector_Generic:Conn_02x05_Odd_Even
- R1: value (none) -> 200K
- renumbered C3 to C2, C4 to C3
Connections:
- net BCR_OUT: now also J9.7 (Pin_7), J9.8 (Pin_8)
- net GND: now also J9.10 (Pin_10), J9.9 (Pin_9)
- net MUX3OUT: now also J9.5 (Pin_5)
- net S0: now also J9.2 (Pin_2)
- net S1: now also J9.4 (Pin_4)
- net S2: now also J9.3 (Pin_3)
- net S3: now also J9.1 (Pin_1)
- net VDD: now also J9.6 (Pin_6)
Other:
- note removed: "Space for more telemetry"

Commit message: boost
Parts:
- added MH5: M2, MountingHole:MountingHole_2.2mm_M2, symbol Mechanical:MountingHole
- added U?: (no value), symbol Regulator_Switching:LT1301
- J9: value (none) -> Solar Daughterboard Connector; footprint (none) -> Connector_PinHeader_2.54mm:PinHeader_2x05_P2.54mm_Vertical
Changed lines of the file:
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@@
     (pin "1")
+  )
+  (symbol (lib_id "Mechanical:MountingHole") (at 115.57 92.71 0) (unit 1)
+    (in_bom yes) (on_board yes) (fields_autoplaced)
+    (property "Reference" "MH5" (id 0) (at 118.11 91.4399 0)
+      (effects (font (size 1.27 1.27)) (justify left))
+    )
+    (property "Value" "M2" (id 1) (at 118.11 93.9799 0)
+      (effects (font (size 1.27 1.27)) (justify left))
+    )
+    (property "Footprint" "MountingHole:MountingHole_2.2mm_M2" (id 2) (at 115.57 92.71 0)
+      (effects (font (size 1.27 1.27)) hide)
+    )
+    (property "Datasheet" "~" (id 3) (at 115.57 92.71 0)
+      (effects (font (size 1.27 1.27)) hide)
+    )
   )
   (symbol (lib_id "power:VDD") (at 242.57 30.48 0) (unit 1)
@@
     )
     (pin "1")
+  )
+  (symbol (lib_id "Regulator_Switching:LT1301") (at 226.06 127 0) (unit 1)
+    (in_bom yes) (on_board yes) (fields_autoplaced)
+    (property "Reference" "U?" (id 0) (at 228.0794 111.76 0)
+      (effects (font (size 1.27 1.27)) (justify left))
+    )
+    (property "Value" "" (id 1) (at 228.0794 114.3 0)
+      (effects (font (size 1.27 1.27)) (justify left))
+    )
+    (property "Footprint" "" (id 2) (at 226.06 127 0)
+      (effects (font (size 1.27 1.27)) hide)
+    )
+    (property "Datasheet" "https://www.analog.com/media/en/technical-documentation/data-sheets/lt1301.pdf" (id 3) (at 226.06 127 0)
+      (effects (font (size 1.27 1.27)) hide)
+    )
+    (pin "1")
+    (pin "2")
+    (pin "3")
+    (pin "4")
+    (pin "5")
+    (pin "6")
+    (pin "7")
+    (pin "8")
   )
   (symbol (lib_id "power:VDD") (at 163.83 74.93 0) (unit 1)
@@
     (in_bom yes) (on_board yes) (fields_autoplaced)
     (property "Reference" "J9" (id 0) (at 149.86 63.5 0))
-    (property "Value" "" (id 1) (at 149.86 66.04 0))
-    (property "Footprint" "" (id 2) (at 148.59 74.93 0)
+    (property "Value" "Solar Daughterboard Connector" (id 1) (at 149.86 66.04 0))
+    (property "Footprint" "Connector_PinHeader_2.54mm:PinHeader_2x05_P2.54mm_Vertical" (id 2) (at 148.59 74.93 0)
       (effects (font (size 1.27 1.27)) hide)
     )
@@
       (reference "MH4") (unit 1) (value "M2") (footprint "MountingHole:MountingHole_2.2mm_M2")
     )
+    (path "/2f389684-fc2a-46a1-b11d-5ff1e4efe356"
+      (reference "MH5") (unit 1) (value "M2") (footprint "MountingHole:MountingHole_2.2mm_M2")
+    )
     (path "/00000000-0000-0000-0000-000061c37b40"
       (reference "R1") (unit 1) (value "200K") (footprint "Resistor_SMD:R_0805_2012Metric")
@@
       (reference "U14") (unit 1) (value "LT3652EMSE") (footprint "Package_SO:MSOP-12-1EP_3x4mm_P0.65mm_EP1.65x2.85mm")
     )
-  )
+    (path "/45e3a90b-d22e-4e72-a1c6-03596189a34c"
+      (reference "U?") (unit 1) (value "LT1301") (footprint "")
+    )
+  )

Commit message: add 5v charge back in
Parts:
- removed U?: (no value), symbol Regulator_Switching:LT1301
- added C24, C25, C26, C27: 22uF, Capacitor_SMD:C_1210_3225Metric, symbol Device:C
- added D17: CMSH3-40MA, Diode_SMD:D_SMA, symbol Device:D_Schottky
- added J10: (no value), symbol Connector:Conn_01x02_Female
- added L5: 33uH, symbol Device:L
- added U15: LT1301, symbol Regulator_Switching:LT1301
Connections:
- net GND: now also C24.2, C25.2, C26.2, C27.2, J10.1 (Pin_1), U15.1 (GND), U15.3 (SHDN), U15.8 (PGND)
- net MPPT4/B_PWR: now also C26.1, C27.1, D17.1 (K), U15.4 (SENSE)
- new net: D17.2 (A), L5.2, U15.7 (SW)
- new net 5VIN: C24.1, C25.1, J10.2 (Pin_2), L5.1, U15.2 (SEL), U15.6 (VIN)
- no-connect marks 0 -> 1
Other:
- note added: "12V boost converter"
- moved on the sheet: C1, C2, C3, D1, D2, D3, D4, D5, D6, D7, D8, J1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
