File: ECAD/Battery/Heaters/Cell.kicad_sch (KiCad schematic)
At the start: 12 parts, among them Q23 2N7002, Q24 BSS83P, Q25 BSN20

Commit message: move heater circuitry
Parts:
- removed C24: 0.1uF, Capacitor_SMD:C_0805_2012Metric, symbol Device:C
- removed Q23: 2N7002, Package_TO_SOT_SMD:SOT-23, symbol Transistor_FET:2N7002
- removed Q24: BSS83P, Package_TO_SOT_SMD:SOT-23, symbol Transistor_FET:BSS83P
- removed Q25: BSN20, Package_TO_SOT_SMD:SOT-23, symbol Transistor_FET:BSN20
- removed R51, R54: 100R, Resistor_SMD:R_0805_2012Metric, symbol Device:R
- removed R52, R53, R55: 10K, Resistor_SMD:R_0805_2012Metric, symbol Device:R
- removed R56: Heater (125R), Connector_PinHeader_2.54mm:PinHeader_1x02_P2.54mm_Vertical, symbol Device:Heater
- removed R57: 270K, Resistor_SMD:R_0805_2012Metric, symbol Device:R
- removed TH4: 100K NTC, Connector_Hirose:Hirose_DF13-02P-1.25DSA_1x02_P1.25mm_Vertical, symbol Device:Thermistor_NTC
- added C?: 0.1uF, Capacitor_SMD:C_0805_2012Metric, symbol Device:C
- added Q?: 2N7002, Package_TO_SOT_SMD:SOT-23, symbol Transistor_FET:2N7002
- added Q?: BSN20, Package_TO_SOT_SMD:SOT-23, symbol Transistor_FET:BSN20
- added Q?: BSS83P, Package_TO_SOT_SMD:SOT-23, symbol Transistor_FET:BSS83P
- added R? (x3): 10K, Resistor_SMD:R_0805_2012Metric, symbol Device:R
- added R?: 270K, Resistor_SMD:R_0805_2012Metric, symbol Device:R
- added R? (x2): 100R, Resistor_SMD:R_0805_2012Metric, symbol Device:R
- added R?: Heater (125R), Connector_PinHeader_2.54mm:PinHeader_1x02_P2.54mm_Vertical, symbol Device:Heater
- added TH?: 100K NTC, Connector_Hirose:Hirose_DF13-02P-1.25DSA_1x02_P1.25mm_Vertical, symbol Device:Thermistor_NTC
Connections:
- net +5V: now also Q?.2 (S), R?.1
- net GND: now also C?.2, Q?.2 (S), Q?.2 (S), R?.2, R?.2, TH?.2
- net TELEM_TBAT: now also C?.1, R?.2, TH?.1
- net VDD: now also R?.1
- new net: Q?.1 (G), Q?.3 (D), R?.2
- new net: Q?.1 (G), R?.1, R?.1 (x2)
- new net: Q?.3 (D), R?.2
- new net: Q?.3 (D), R?.1
- new net GATE: R?.2, R?.2
Other:
- company: TJHSST Nanosatellite Club -> (none)
- title: TJ Custom EPS -> (none)
